Commit message: Removed a TON of comments. Down to about 2600 lines from 5300.

File: valkyrie_description/common_xacro/xacro/generic_models.xacro (robot description, xacro)
@@ -265,10 +265,4 @@
     </link>
   </xacro:macro>
-  <!-- Its seems that zero mass links are not kosher. I can't find any solid data, only suggestions from people
-  as to what small but not too small should be for mass numbers.
-  Until better evidence/experience says otherwise, we will use a mass that is ~0.1% * total_mass, and
-  the inertia properties of a cylinder. Justification: Most of these virtual links are the rotor attached
-  to gearing and any attachment structure.
-   -->
   <xacro:property name="virtual_link_mass" value="0.1"/>
   <xacro:property name="virtual_link_radius" value="0.05"/>

File: valkyrie_description/robots/valkyrie_A/xacro/V1.xacro (robot description, xacro)
@@ -5,5 +5,5 @@
     <xacro:property name="mesh_root" value="package://V1/meshes/reduced_polygon_meshes"/>
     <!-- <xacro:include filename="$(find common_xacro)/xacro/mode_setup_hw.xacro" /> -->
-    <xacro:include filename="$(find valkyrie_description)/robots/valkyrie_A/xacro/common/hw_actuator_types.xacro"/>
+    <!-- <xacro:include filename="$(find valkyrie_description)/robots/valkyrie_A/xacro/common/hw_actuator_types.xacro"/> -->
     <xacro:include filename="$(find valkyrie_description)/robots/valkyrie_A/xacro/V1_sim_base.xacro"/>
 </robot>

File: valkyrie_description/robots/valkyrie_A/xacro/V1_sim_base.xacro (robot description, xacro)
@@ -1,6 +1,3 @@
 <robot xmlns:xacro="http://ros.org/wiki/xacro" name="valkyrie">
-    <!-- ======================================================= -->
-    <!-- DO NOT MODIFY URDF BY HAND! YOU ARE A FOOL IF YOU DO! -->
-    <!-- ======================================================= -->
     <xacro:include filename="$(find common_xacro)/xacro/generic_models.xacro" />
     <xacro:include filename="$(find valkyrie_description)/robots/valkyrie_A/xacro/plugins/gazebo_plugins.xacro"/>
@@ -132,5 +129,3 @@
                                        actuator5="${leftleg_name5}"
                                        actuator6="${leftleg_name6}" /> -->
-    <!-- <xacro:v1_leg_sensors prefix="Left" reflect="-1" /> -->
-    <!-- <xacro:v1_hw_sensors prefix="Left" hermes_node="${leftleg_hermes}" atidaq_node="${leftleg_ati}" mpu6000_node="${leftleg_mpu2000}" cop_node="${leftleg_cop}"/> -->
 </robot>

File: valkyrie_description/robots/valkyrie_A/xacro/arm/actuator_names.xacro (robot description, xacro)
@@ -1,8 +1,4 @@
 <?xml version="1.0" ?>
 <robot xmlns:xacro="http://www.ros.org/wiki/xacro" name="v1/arm/joint_names">
-  <!--
-    Reference for kinematic and dynamic parameters comes from:
-      http://bender.jsc.nasa.gov/confluence/pages/viewpage.action?pageId=16417593
-  -->
   <xacro:property name="AJ1_Actuator_Name" value="/Trunk/${prefix}ArmActuator" />
   <xacro:property name="AJ2_Actuator_Name" value="/${prefix}Arm/Actuator2" />

File: valkyrie_description/robots/valkyrie_A/xacro/arm/arm.xacro (robot description, xacro)
@@ -1,8 +1,4 @@
 <?xml version="1.0" ?>
 <robot xmlns:xacro="http://www.ros.org/wiki/xacro" name="v1/arm">
-  <!--
-        Reference for kinematic and dynamic parameters comes from:
-            http://bender.jsc.nasa.gov/confluence/pages/viewpage.action?pageId=16417593
-  -->
   <xacro:include filename="$(find valkyrie_description)/robots/valkyrie_A/xacro/arm/joint_names.xacro"/>
   <xacro:include filename="$(find valkyrie_description)/robots/valkyrie_A/xacro/arm/link_names.xacro"/>

File: valkyrie_description/robots/valkyrie_A/xacro/arm/dh_parameters.xacro (robot description, xacro)
@@ -1,21 +1,8 @@
 <?xml version="1.0" ?>
 <robot xmlns:xacro="http://www.ros.org/wiki/xacro" name="v1/arm/dh_parameters">
-  <!--
-    Reference for kinematic and dynamic parameters comes from:
-      http://bender.jsc.nasa.gov/confluence/pages/viewpage.action?pageId=16417593
-  -->
-  <!--
-    Joint_Offset (d): offset along previous z to the common normal
-    Joint_Angle (theta): angle about previous z, from old x to new x
-    Joint_Radius (a): length of the common normal. Assuming a revolute joint, this is the radius about previous z.
-    Joint_Twist (alpha): angle about common normal, from old z axis to new z axis
-  -->
-  <!-- AJ1 -->
-  <!-- DH Parameters -->
   <xacro:property name="AJ1_Joint_Offset" value="-0.03157" />
   <xacro:property name="AJ1_Joint_Angle" value="0" />
   <xacro:property name="AJ1_Joint_Radius" value="0.29842" />
   <xacro:property name="AJ1_Joint_Twist" value="${pi_2}" />
-  <!-- Derived -->
   <xacro:property name="AJ1_Origin_X" value="0.29842"/>
   <xacro:property name="AJ1_Origin_Y" value="0"/>
@@ -24,11 +11,8 @@
   <xacro:property name="AJ1_Orientation_Pitch" value="0"/>
   <xacro:property name="AJ1_Orientation_Yaw" value="0"/>
-  <!-- AJ2 -->
-  <!-- DH Parameters -->
   <xacro:property name="AJ2_Joint_Offset" value="${reflect * -0.246}" />
   <xacro:property name="AJ2_Joint_Angle" value="${pi}" />
   <xacro:property name="AJ2_Joint_Radius" value="0" />
   <xacro:property name="AJ2_Joint_Twist" value="${reflect * (pi_2)}" />
-  <!-- Derived -->
   <xacro:property name="AJ2_Origin_X" value="0"/>
   <xacro:property name="AJ2_Origin_Y" value="0"/>
@@ -37,11 +21,8 @@
   <xacro:property name="AJ2_Orientation_Pitch" value="0"/>
   <xacro:property name="AJ2_Orientation_Yaw" value="${pi}"/>
-  <!-- AJ3 -->
-  <!-- DH Parameters -->
   <xacro:property name="AJ3_Joint_Offset" value="0" />
   <xacro:property name="AJ3_Joint_Angle" value="${reflect * pi_2}" />
   <xacro:property name="AJ3_Joint_Radius" value="0" />
   <xacro:property name="AJ3_Joint_Twist" value="${-1 * pi_2}" />
-  <!-- Derived -->
   <xacro:property name="AJ3_Origin_X" value="0"/>
   <xacro:property name="AJ3_Origin_Y" value="0"/>
@@ -50,11 +31,8 @@
   <xacro:property name="AJ3_Orientation_Pitch" value="0"/>
   <xacro:property name="AJ3_Orientation_Yaw" value="${reflect * pi_2}"/>
-  <!-- AJ4 -->
-  <!-- DH Parameters -->
   <xacro:property name="AJ4_Joint_Offset" value="${reflect * -0.330}" />
   <xacro:property name="AJ4_Joint_Angle" value="${reflect * pi_2}" />
   <xacro:property name="AJ4_Joint_Radius" value="-0.0254" />
   <xacro:property name="AJ4_Joint_Twist" value="${reflect * pi_2}" />
-  <!-- Derived -->
   <xacro:property name="AJ4_Origin_X" value="0"/>
   <xacro:property name="AJ4_Origin_Y" value="${reflect * -0.0254}"/>
@@ -63,11 +41,8 @@
   <xacro:property name="AJ4_Orientation_Pitch" value="0"/>
   <xacro:property name="AJ4_Orientation_Yaw" value="${reflect * pi_2}"/>
-  <!-- AJ5 -->
-  <!-- DH Parameters -->
   <xacro:property name="AJ5_Joint_Offset" value="0" />
   <xacro:property name="AJ5_Joint_Angle" value="${pi}" />
   <xacro:property name="AJ5_Joint_Radius" value="-0.0254" />
   <xacro:property name="AJ5_Joint_Twist" value="${reflect * pi_2}" />
-  <!-- Derived -->
   <xacro:property name="AJ5_Origin_X" value="0.0254"/>
   <xacro:property name="AJ5_Origin_Y" value="0"/>
@@ -76,11 +51,8 @@
   <xacro:property name="AJ5_Orientation_Pitch" value="0"/>
   <xacro:property name="AJ5_Orientation_Yaw" value="${pi}"/>
-  <!-- AJ6 -->
-  <!-- DH Parameters -->
   <xacro:property name="AJ6_Joint_Offset" value="${reflect * -0.287}" />
   <xacro:property name="AJ6_Joint_Angle" value="${reflect * pi_2}" />
   <xacro:property name="AJ6_Joint_Radius" value="0" />
   <xacro:property name="AJ6_Joint_Twist" value="${reflect * -1 * pi_2}" />
-  <!-- Derived -->
   <xacro:property name="AJ6_Origin_X" value="0"/>
   <xacro:property name="AJ6_Origin_Y" value="0"/>
@@ -89,11 +61,8 @@
   <xacro:property name="AJ6_Orientation_Pitch" value="0"/>
   <xacro:property name="AJ6_Orientation_Yaw" value="${reflect * pi_2}"/>
-  <!-- AJ7 -->
-  <!-- DH Parameters -->
   <xacro:property name="AJ7_Joint_Offset" value="0" />
   <xacro:property name="AJ7_Joint_Angle" value="${reflect * pi_2}" />
   <xacro:property name="AJ7_Joint_Radius" value="0" />
   <xacro:property name="AJ7_Joint_Twist" value="${reflect * pi_2}" />
-  <!-- Derived -->
   <xacro:property name="AJ7_Origin_X" value="0"/>
   <xacro:property name="AJ7_Origin_Y" value="0"/>

File: valkyrie_description/robots/valkyrie_A/xacro/arm/joint_limits.xacro (robot description, xacro)
@@ -1,9 +1,4 @@
 <?xml version="1.0" ?>
 <robot xmlns:xacro="http://www.ros.org/wiki/xacro" name="v1/arm/joint_limits">
-  <!--
-    Reference for kinematic and dynamic parameters comes from:
-      http://bender.jsc.nasa.gov/confluence/pages/viewpage.action?pageId=16417593
-      Note: Some joint limits are set ~5 degrees smaller than the corresponding coeff
-  -->
   <xacro:property name="AJ1_Torque_Limit" value="190" />
   <xacro:property name="AJ2_Torque_Limit" value="190" />

File: valkyrie_description/robots/valkyrie_A/xacro/arm/joint_names.xacro (robot description, xacro)
@@ -1,8 +1,4 @@
 <?xml version="1.0" ?>
 <robot xmlns:xacro="http://www.ros.org/wiki/xacro" name="v1/arm/joint_names">
-  <!--
-    Reference for kinematic and dynamic parameters comes from:
-      http://bender.jsc.nasa.gov/confluence/pages/viewpage.action?pageId=16417593
-  -->
   <xacro:property name="AJ1_Joint_Name" value="${prefix}ShoulderExtensor" />
   <xacro:property name="AJ2_Joint_Name" value="${prefix}ShoulderAdductor" />

File: valkyrie_description/robots/valkyrie_A/xacro/arm/link_names.xacro (robot description, xacro)
@@ -1,8 +1,4 @@
 <?xml version="1.0" ?>
 <robot xmlns:xacro="http://www.ros.org/wiki/xacro" name="v1/arm/link_names">
-  <!--
-    Reference for kinematic and dynamic parameters comes from:
-      http://bender.jsc.nasa.gov/confluence/pages/viewpage.action?pageId=16417593
-  -->
   <xacro:property name="AJ1_Proximal_Link" value="${arm_root_link}" />
   <xacro:property name="AJ1_Distal_Link" value="/v1/${prefix}ShoulderExtensor" />

File: valkyrie_description/robots/valkyrie_A/xacro/arm/mass_parameters.xacro (robot description, xacro)
@@ -1,36 +1,4 @@
 <?xml version="1.0" ?>
 <robot xmlns:xacro="http://www.ros.org/wiki/xacro" name="v1/arm/mass_parameters">
-  <!--
-    Reference for kinematic and dynamic parameters comes from:
-      http://bender.jsc.nasa.gov/confluence/pages/viewpage.action?pageId=16417593
-  -->
-  <!-- AJ1 -->
-<!--   <xacro:property name="AJ1_Link_Mass" value="2.65" />
-  <xacro:property name="AJ2_Link_Mass" value="3.5" />
-  <xacro:property name="AJ3_Link_Mass" value="2.3" /> -->
-<!-- cdr -->
-<!--
-  <xacro:property name="AJ4_Link_Mass" value="1.05" />
-  <xacro:property name="AJ5_Link_Mass" value="0.95" />
-  <xacro:property name="AJ6_Link_Mass" value="0.58" />
-  <xacro:property name="AJ7_Link_Mass" value="0.06" />
- -->
-<!--    default xacro
- -->  <!--
-  <xacro:property name="AJ4_Link_Mass" value="2.3" />
-  <xacro:property name="AJ5_Link_Mass" value="2.95" />
-  <xacro:property name="AJ6_Link_Mass" value="0.73" />
-  <xacro:property name="AJ7_Link_Mass" value="0.06" /> -->
-<!-- wiki -->
-<!--  <xacro:property name="AJ4_Link_Mass" value="2.52" />
-  <xacro:property name="AJ5_Link_Mass" value="2.95" />
-  <xacro:property name="AJ6_Link_Mass" value="0.06" />
-  <xacro:property name="AJ7_Link_Mass" value="0.73" />
- --><!--
- <xacro:property name="AJ4_Link_Mass" value="1.05" />
-  <xacro:property name="AJ5_Link_Mass" value="2.95" />
-  <xacro:property name="AJ6_Link_Mass" value="0.06" />
-  <xacro:property name="AJ7_Link_Mass" value="0.73" /> -->
-  <!-- The following were taken from Christopher McQuin's DRC Master Spreadsheet sept.xlsx, 10/7/13-->
   <xacro:property name="AJ1_Link_Mass" value="2.65" />
   <xacro:property name="AJ2_Link_Mass" value="2.87" />

File: valkyrie_description/robots/valkyrie_A/xacro/common/common_bodies.xacro (robot description, xacro)
@@ -1,6 +1,3 @@
 <robot xmlns:xacro="http://ros.orgt/wiki/xacro" name="v1/common_bodies">
-    <!-- ======================================================= -->
-    <!-- DO NOT MODIFY URDF BY HAND! YOU ARE A FOOL IF YOU DO! -->
-    <!-- ======================================================= -->
     <xacro:include filename="$(find valkyrie_description)/robots/valkyrie_A/xacro/pelvis/pelvis.xacro" />
     <xacro:include filename="$(find valkyrie_description)/robots/valkyrie_A/xacro/waist/waist.xacro" />

File: valkyrie_description/robots/valkyrie_A/xacro/common/hw_actuator_types.xacro (robot description, xacro)
@@ -1,6 +1,3 @@
 <robot xmlns:xacro="http://ros.org/wiki/xacro" name="hw_actuator_types">
-    <!-- ======================================================= -->
-    <!-- DO NOT MODIFY URDF BY HAND! YOU ARE A FOOL IF YOU DO! -->
-    <!-- ======================================================= -->
     <xacro:property name="arm_type1" value="turbodriver_api/TurbodriverAPI_DRCv4"/>
     <xacro:property name="arm_type2" value="turbodriver_api/TurbodriverAPI_DRCv4"/>

File: valkyrie_description/robots/valkyrie_A/xacro/common/sim_actuator_types.xacro (robot description, xacro)
@@ -1,6 +1,3 @@
 <robot xmlns:xacro="http://ros.org/wiki/xacro" name="sim_actuator_types">
-    <!-- ======================================================= -->
-    <!-- DO NOT MODIFY URDF BY HAND! YOU ARE A FOOL IF YOU DO! -->
-    <!-- ======================================================= -->
     <xacro:property name="arm_type1" value="turbodriver_api/TurbodriverSimAPI_DRCv4"/>
     <xacro:property name="arm_type2" value="turbodriver_api/TurbodriverSimAPI_DRCv4"/>

File: valkyrie_description/robots/valkyrie_A/xacro/head/dh_parameters.xacro (robot description, xacro)
@@ -1,21 +1,8 @@
 <?xml version="1.0" ?>
 <robot xmlns:xacro="http://www.ros.org/wiki/xacro" name="v1/head/dh_parameters">
-  <!--
-    Reference for kinematic and dynamic parameters comes from:
-      http://bender.jsc.nasa.gov/confluence/pages/viewpage.action?pageId=16417593
-  -->
-  <!--
-    Joint_Offset (d): offset along previous z to the common normal
-    Joint_Angle (theta): angle about previous z, from old x to new x
-    Joint_Radius (a): length of the common normal. Assuming a revolute joint, this is the radius about previous z.
-    Joint_Twist (alpha): angle about common normal, from old z axis to new z axis
-  -->
-  <!-- NJ1 -->
-  <!-- DH Parameters -->
   <xacro:property name="NJ1_Joint_Offset" value="0.0519" />
   <xacro:property name="NJ1_Joint_Angle" value="0" />
   <xacro:property name="NJ1_Joint_Radius" value="0.33845" />
   <xacro:property name="NJ1_Joint_Twist" value="${-1 * pi_2}" />
-  <!-- Derived -->
   <xacro:property name="NJ1_Origin_X" value="0.3383"/>
   <xacro:property name="NJ1_Origin_Y" value="0"/>
@@ -24,11 +11,8 @@
   <xacro:property name="NJ1_Orientation_Pitch" value="0"/>
   <xacro:property name="NJ1_Orientation_Yaw" value="0"/>
-  <!-- NJ2 -->
-  <!-- DH Parameters -->
   <xacro:property name="NJ2_Joint_Offset" value="0" />
   <xacro:property name="NJ2_Joint_Angle" value="${pi_2}" />
   <xacro:property name="NJ2_Joint_Radius" value="0.0519" />
   <xacro:property name="NJ2_Joint_Twist" value="${pi_2}" />
-  <!-- Derived -->
   <xacro:property name="NJ2_Origin_X" value="0"/>
   <xacro:property name="NJ2_Origin_Y" value="0.0519"/>
@@ -37,11 +21,8 @@
   <xacro:property name="NJ2_Orientation_Pitch" value="0"/>
   <xacro:property name="NJ2_Orientation_Yaw" value="${pi_2}"/>
-  <!-- NJ3 -->
-  <!-- DH Parameters -->
   <xacro:property name="NJ3_Joint_Offset" value="0.196" />
   <xacro:property name="NJ3_Joint_Angle" value="0" />
   <xacro:property name="NJ3_Joint_Radius" value="0.06" />
   <xacro:property name="NJ3_Joint_Twist" value="${-1 * pi_2}" />
-  <!-- Derived -->
   <xacro:property name="NJ3_Origin_X" value="0.06"/>
   <xacro:property name="NJ3_Origin_Y" value="0"/>

File: valkyrie_description/robots/valkyrie_A/xacro/head/head.xacro (robot description, xacro)
@@ -1,7 +1,3 @@
 <robot xmlns:xacro="http://www.ros.org/wiki/xacro" name="v1/head">
-  <!--
-      Reference for kinematic and dynamic parameters comes from:
-          http://bender.jsc.nasa.gov/confluence/pages/viewpage.action?pageId=16417593
-  -->
   <!-- Properties -->
   <xacro:include filename="$(find valkyrie_description)/robots/valkyrie_A/xacro/head/joint_names.xacro"/>

File: valkyrie_description/robots/valkyrie_A/xacro/head/joint_limits.xacro (robot description, xacro)
@@ -1,8 +1,4 @@
 <?xml version="1.0" ?>
 <robot xmlns:xacro="http://www.ros.org/wiki/xacro" name="v1/head/joint_limits">
-  <!--
-    Reference for kinematic and dynamic parameters comes from:
-      http://bender.jsc.nasa.gov/confluence/pages/viewpage.action?pageId=16417593
-  -->
   <xacro:property name="NJ1_Torque_Limit" value="26" />
   <xacro:property name="NJ2_Torque_Limit" value="26" />

File: valkyrie_description/robots/valkyrie_A/xacro/head/joint_names.xacro (robot description, xacro)
@@ -1,8 +1,4 @@
 <?xml version="1.0" ?>
 <robot xmlns:xacro="http://www.ros.org/wiki/xacro" name="v1/head/joint_names">
-  <!--
-    Reference for kinematic and dynamic parameters comes from:
-      http://bender.jsc.nasa.gov/confluence/pages/viewpage.action?pageId=16417593
-  -->
   <xacro:property name="NJ1_Joint_Name" value="LowerNeckExtensor" />
   <xacro:property name="NJ2_Joint_Name" value="NeckRotator" />

File: valkyrie_description/robots/valkyrie_A/xacro/head/link_names.xacro (robot description, xacro)
@@ -1,8 +1,4 @@
 <?xml version="1.0" ?>
 <robot xmlns:xacro="http://www.ros.org/wiki/xacro" name="v1/head/link_names">
-  <!--
-    Reference for kinematic and dynamic parameters comes from:
-      http://bender.jsc.nasa.gov/confluence/pages/viewpage.action?pageId=16417593
-  -->
   <xacro:property name="NJ1_Proximal_Link" value="${head_root_link}" />
   <xacro:property name="NJ1_Distal_Link" value="/v1/LowerNeckExtensor" />

File: valkyrie_description/robots/valkyrie_A/xacro/head/mass_parameters.xacro (robot description, xacro)
@@ -1,13 +1,4 @@
 <?xml version="1.0" ?>
 <robot xmlns:xacro="http://www.ros.org/wiki/xacro" name="v1/head/mass_parameters">
-  <!--
-    Reference for kinematic and dynamic parameters comes from:
-      http://bender.jsc.nasa.gov/confluence/pages/viewpage.action?pageId=16417593
-  -->
-<!--   <xacro:property name="NJ1_Link_Mass" value="1.08" />
-  <xacro:property name="NJ2_Link_Mass" value="1.08" />
-  <xacro:property name="NJ3_Link_Mass" value="4.34" /> -->
-<!--  <xacro:property name="NJ3_Link_Mass" value="3.58" /> -->
-  <!-- The following were taken from Christopher McQuin's DRC Master Spreadsheet sept.xlsx, 10/7/13-->
   <xacro:property name="NJ1_Link_Mass" value="0.471" />
   <xacro:property name="NJ2_Link_Mass" value="1.4" />

File: valkyrie_description/robots/valkyrie_A/xacro/leg/dh_parameters.xacro (robot description, xacro)
@@ -1,21 +1,8 @@
 <?xml version="1.0" ?>
 <robot xmlns:xacro="http://www.ros.org/wiki/xacro" name="v1/leg/dh_parameters">
-  <!--
-    Reference for kinematic and dynamic parameters comes from:
-      http://bender.jsc.nasa.gov/confluence/pages/viewpage.action?pageId=16417593
-  -->
-  <!--
-    Joint_Offset (d): offset along previous z to the common normal
-    Joint_Angle (theta): angle about previous z, from old x to new x
-    Joint_Radius (a): length of the common normal. Assuming a revolute joint, this is the radius about previous z.
-    Joint_Twist (alpha): angle about common normal, from old z axis to new z axis
-  -->
-  <!-- LJ1 -->
-  <!-- DH Parameters -->
   <xacro:property name="LJ1_Joint_Offset" value="-0.183" />
   <xacro:property name="LJ1_Joint_Angle" value="${reflect * -1 * pi_2}" />
   <xacro:property name="LJ1_Joint_Radius" value="0.1016" />
   <xacro:property name="LJ1_Joint_Twist" value="${pi * ((1 - reflect)/2)}" />
-  <!-- Derived -->
   <xacro:property name="LJ1_Origin_X" value="0"/>
   <xacro:property name="LJ1_Origin_Y" value="${reflect * -0.1016}"/>
@@ -24,11 +11,8 @@
   <xacro:property name="LJ1_Orientation_Pitch" value="0"/>
   <xacro:property name="LJ1_Orientation_Yaw" value="${reflect * -1 * pi_2}"/>
-  <!-- LJ2 -->
-  <!-- DH Parameters -->
   <xacro:property name="LJ2_Joint_Offset" value="0" />
   <xacro:property name="LJ2_Joint_Angle" value="0" />
   <xacro:property name="LJ2_Joint_Radius" value="0" />
   <xacro:property name="LJ2_Joint_Twist" value="${reflect * -1 * pi_2}" />
-  <!-- Derived -->
   <xacro:property name="LJ2_Origin_X" value="0"/>
   <xacro:property name="LJ2_Origin_Y" value="0"/>
@@ -37,11 +21,8 @@
   <xacro:property name="LJ2_Orientation_Pitch" value="0"/>
   <xacro:property name="LJ2_Orientation_Yaw" value="0"/>
-  <!-- LJ3 -->
-  <!-- DH Parameters -->
   <xacro:property name="LJ3_Joint_Offset" value="0" />
   <xacro:property name="LJ3_Joint_Angle" value="${pi_2}" />
   <xacro:property name="LJ3_Joint_Radius" value="0.061" />
   <xacro:property name="LJ3_Joint_Twist" value="${reflect * -1 * pi_2}" />
-  <!-- Derived -->
   <xacro:property name="LJ3_Origin_X" value="0"/>
   <xacro:property name="LJ3_Origin_Y" value="0.061"/>
@@ -50,11 +31,8 @@
   <xacro:property name="LJ3_Orientation_Pitch" value="0"/>
   <xacro:property name="LJ3_Orientation_Yaw" value="${pi_2}"/>
-  <!-- LJ4 -->
-  <!-- DH Parameters -->
   <xacro:property name="LJ4_Joint_Offset" value="${reflect * -1 * 0.0374}" />
   <xacro:property name="LJ4_Joint_Angle" value="0" />
   <xacro:property name="LJ4_Joint_Radius" value="0.431" />
   <xacro:property name="LJ4_Joint_Twist" value="${pi}" />
-  <!-- Derived -->
   <xacro:property name="LJ4_Origin_X" value="0.431"/>
   <xacro:property name="LJ4_Origin_Y" value="0"/>
@@ -63,11 +41,8 @@
   <xacro:property name="LJ4_Orientation_Pitch" value="0"/>
   <xacro:property name="LJ4_Orientation_Yaw" value="0"/>
-  <!-- LJ5 -->
-  <!-- DH Parameters -->
   <xacro:property name="LJ5_Joint_Offset" value="0" />
   <xacro:property name="LJ5_Joint_Angle" value="0" />
   <xacro:property name="LJ5_Joint_Radius" value="0.406" />
   <xacro:property name="LJ5_Joint_Twist" value="${pi}" />
-  <!-- Derived -->
   <xacro:property name="LJ5_Origin_X" value="0.406"/>
   <xacro:property name="LJ5_Origin_Y" value="0"/>
@@ -76,11 +51,8 @@
   <xacro:property name="LJ5_Orientation_Pitch" value="0"/>
   <xacro:property name="LJ5_Orientation_Yaw" value="0"/>
-  <!-- LJ6 -->
-  <!-- DH Parameters -->
   <xacro:property name="LJ6_Joint_Offset" value="0" />
   <xacro:property name="LJ6_Joint_Angle" value="0" />
   <xacro:property name="LJ6_Joint_Radius" value="0.0127" />
   <xacro:property name="LJ6_Joint_Twist" value="${reflect * pi_2}" />
-  <!-- Derived -->
   <xacro:property name="LJ6_Origin_X" value="0.0127"/>
   <xacro:property name="LJ6_Origin_Y" value="0"/>
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