Commit message: Removing some comments.

File: valkyrie_description/common_xacro/xacro/generic_models.xacro (robot description, xacro)
@@ -63,8 +63,6 @@
         <geometry>
           <mesh filename="${visual_mesh}"/>
-          <!-- <box size="${width} ${height} ${depth}"/> -->
-        </geometry>
-        <origin rpy="0 0 0" xyz="0 0 0"/>
-        <!-- <origin rpy="${origin_rpy}" xyz="${origin_xyz}"/> -->
+        </geometry>
+        <origin rpy="0 0 0" xyz="0 0 0"/>
         <material name="${material}"/>
       </visual>
@@ -92,8 +90,6 @@
         <geometry>
           <mesh filename="${visual_mesh}"/>
-          <!-- <box size="${width} ${height} ${depth}"/> -->
         </geometry>
         <origin rpy="${origin_offset_rpy}" xyz="${origin_offset_xyz}"/>
-        <!-- <origin rpy="${origin_rpy}" xyz="${origin_xyz}"/> -->
         <material name="${material}"/>
       </visual>
@@ -131,8 +127,6 @@
         <geometry>
           <mesh filename="${visual_mesh}" scale="${visual_mesh_scale}"/>
-          <!-- <box size="${width} ${height} ${depth}"/> -->
-        </geometry>
-        <origin rpy="0 0 0" xyz="0 0 0"/>
-        <!-- <origin rpy="${origin_rpy}" xyz="${origin_xyz}"/> -->
+        </geometry>
+        <origin rpy="0 0 0" xyz="0 0 0"/>
         <material name="${material}"/>
       </visual>
@@ -208,5 +202,4 @@
         <geometry>
           <mesh filename="${visual_mesh}"/>
-          <!-- <box size="${width} ${height} ${depth}"/> -->
         </geometry>
         <origin rpy="0 0 0" xyz="0 0 0"/>
@@ -229,8 +222,6 @@
       <visual>
         <origin rpy="0 0 0" xyz="0 0 0"/>
-        <!-- <origin rpy="${origin_rpy}" xyz="${origin_xyz}"/> -->
         <geometry>
           <mesh filename="${visual_mesh}"/>
-          <!-- <sphere radius="${radius}"/> -->
         </geometry>
         <material name="${material}"/>

File: valkyrie_description/robots/valkyrie_A/valkyrie_A.urdf (robot description, URDF)
Before this commit: robot valkyrie, 63 links, 62 joints
Links:
- link /v1/Head: geometry collision mesh filename=package://valkyrie_description/meshes/reduced_polygon_meshe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; visual mesh filename=package://valkyrie_description/meshes/reduced_polygon_meshe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
- link /v1/LeftElbowExtensor: geometry collision mesh filename=package://valkyrie_description/meshes/reduced_polygon_meshe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; visual mesh filename=package://valkyrie_description/meshes/reduced_polygon_meshe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
- link /v1/LeftForearm: geometry collision mesh filename=package://valkyrie_description/meshes/reduced_polygon_meshe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; visual mesh filename=package://valkyrie_description/meshes/reduced_polygon_meshe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
- link /v1/LeftHipAdductor: geometry collision mesh filename=package://valkyrie_description/meshes/reduced_polygon_meshe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; visual mesh filename=package://valkyrie_description/meshes/reduced_polygon_meshe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
- link /v1/LeftHipRotator: geometry collision mesh filename=package://valkyrie_description/meshes/reduced_polygon_meshe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; visual mesh filename=package://valkyrie_description/meshes/reduced_polygon_meshe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
- link /v1/LeftLeg: geometry collision mesh filename=package://valkyrie_description/meshes/reduced_polygon_meshe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; visual mesh filename=package://valkyrie_description/meshes/reduced_polygon_meshe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
- link /v1/LeftLittleDistalPhalanx: geometry collision mesh filename=package://valkyrie_description/meshes/reduced_polygon_meshe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; visual mesh filename=package://valkyrie_description/meshes/reduced_polygon_meshe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
- link /v1/LeftLittleMedialPhalanx: geometry collision mesh filename=package://valkyrie_description/meshes/reduced_polygon_meshe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; visual mesh filename=package://valkyrie_description/meshes/reduced_polygon_meshe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
- link /v1/LeftLittleProximalPhalanx: geometry collision mesh filename=package://valkyrie_description/meshes/reduced_polygon_meshe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; visual mesh filename=package://valkyrie_description/meshes/reduced_polygon_meshe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
- link /v1/LeftMedialMetacarpal: geometry collision mesh filename=package://valkyrie_description/meshes/reduced_polygon_meshe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; visual mesh filename=package://valkyrie_description/meshes/reduced_polygon_meshe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
- link /v1/LeftMiddleDistalPhalanx: geometry collision mesh filename=package://valkyrie_description/meshes/reduced_polygon_meshe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; visual mesh filename=package://valkyrie_description/meshes/reduced_polygon_meshe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
- link /v1/LeftMiddleMedialPhalanx: geometry collision mesh filename=package://valkyrie_description/meshes/reduced_polygon_meshe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; visual mesh filename=package://valkyrie_description/meshes/reduced_polygon_meshe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
- link /v1/LeftMiddleProximalPhalanx: geometry collision mesh filename=package://valkyrie_description/meshes/reduced_polygon_meshe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; visual mesh filename=package://valkyrie_description/meshes/reduced_polygon_meshe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
- link /v1/LeftPalm: geometry collision mesh filename=package://valkyrie_description/meshes/reduced_polygon_meshe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; visual mesh filename=package://valkyrie_description/meshes/reduced_polygon_meshe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
- link /v1/LeftPrimaryDistalPhalanx: geometry collision mesh filename=package://valkyrie_description/meshes/reduced_polygon_meshe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; visual mesh filename=package://valkyrie_description/meshes/reduced_polygon_meshe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
- link /v1/LeftPrimaryMedialPhalanx: geometry collision mesh filename=package://valkyrie_description/meshes/reduced_polygon_meshe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; visual mesh filename=package://valkyrie_description/meshes/reduced_polygon_meshe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
- link /v1/LeftPrimaryMetacarpal: geometry collision mesh filename=package://valkyrie_description/meshes/reduced_polygon_meshe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; visual mesh filename=package://valkyrie_description/meshes/reduced_polygon_meshe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
- link /v1/LeftPrimaryProximalPhalanx: geometry collision mesh filename=package://valkyrie_description/meshes/reduced_polygon_meshe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; visual mesh filename=package://valkyrie_description/meshes/reduced_polygon_meshe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
- link /v1/LeftShankStructure: geometry collision mesh filename=package://valkyrie_description/meshes/reduced_polygon_meshe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; visual mesh filename=package://valkyrie_description/meshes/reduced_polygon_meshe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
- link /v1/LeftShoulderAdductor: geometry collision mesh filename=package://valkyrie_description/meshes/reduced_polygon_meshe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; visual mesh filename=package://valkyrie_description/meshes/reduced_polygon_meshe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
- link /v1/LeftShoulderExtensor: geometry collision mesh filename=package://valkyrie_description/meshes/reduced_polygon_meshe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; visual mesh filename=package://valkyrie_description/meshes/reduced_polygon_meshe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
- link /v1/LeftShoulderRotator: geometry collision mesh filename=package://valkyrie_description/meshes/reduced_polygon_meshe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; visual mesh filename=package://valkyrie_description/meshes/reduced_polygon_meshe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
- link /v1/LeftThumbDistalPhalanx: geometry collision mesh filename=package://valkyrie_description/meshes/reduced_polygon_meshe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; visual mesh filename=package://valkyrie_description/meshes/reduced_polygon_meshe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
- link /v1/LeftThumbMedialPhalanx: geometry collision mesh filename=package://valkyrie_description/meshes/reduced_polygon_meshe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; visual mesh filename=package://valkyrie_description/meshes/reduced_polygon_meshe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
- link /v1/LeftThumbMetacarpal: geometry collision mesh filename=package://valkyrie_description/meshes/reduced_polygon_meshe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; visual mesh filename=package://valkyrie_description/meshes/reduced_polygon_meshe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
- link /v1/LeftThumbProximalPhalanx: geometry collision mesh filename=package://valkyrie_description/meshes/reduced_polygon_meshe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; visual mesh filename=package://valkyrie_description/meshes/reduced_polygon_meshe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
- link /v1/LeftUpperFoot: geometry collision box size=0.082 0.128 0.3; visual mesh filename=package://valkyrie_description/meshes/reduced_polygon_meshe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
- link /v1/LowerNeckExtensor: geometry collision mesh filename=package://valkyrie_description/meshes/reduced_polygon_meshe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; visual mesh filename=package://valkyrie_description/meshes/reduced_polygon_meshe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
- link /v1/NeckRotator: geometry collision mesh filename=package://valkyrie_description/meshes/reduced_polygon_meshe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; visual mesh filename=package://valkyrie_description/meshes/reduced_polygon_meshe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
- link /v1/Pelvis: geometry collision mesh filename=package://valkyrie_description/meshes/reduced_polygon_meshe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; visual mesh filename=package://valkyrie_description/meshes/reduced_polygon_meshe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
- link /v1/RightElbowExtensor: geometry collision mesh filename=package://valkyrie_description/meshes/reduced_polygon_meshe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; visual mesh filename=package://valkyrie_description/meshes/reduced_polygon_meshe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
- link /v1/RightForearm: geometry collision mesh filename=package://valkyrie_description/meshes/reduced_polygon_meshe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; visual mesh filename=package://valkyrie_description/meshes/reduced_polygon_meshe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
- link /v1/RightHipAdductor: geometry collision mesh filename=package://valkyrie_description/meshes/reduced_polygon_meshe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; visual mesh filename=package://valkyrie_description/meshes/reduced_polygon_meshe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
- link /v1/RightHipRotator: geometry collision mesh filename=package://valkyrie_description/meshes/reduced_polygon_meshe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; visual mesh filename=package://valkyrie_description/meshes/reduced_polygon_meshe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
- link /v1/RightLeg: geometry collision mesh filename=package://valkyrie_description/meshes/reduced_polygon_meshe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; visual mesh filename=package://valkyrie_description/meshes/reduced_polygon_meshe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
- link /v1/RightLittleDistalPhalanx: geometry collision mesh filename=package://valkyrie_description/meshes/reduced_polygon_meshe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; visual mesh filename=package://valkyrie_description/meshes/reduced_polygon_meshe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
- link /v1/RightLittleMedialPhalanx: geometry collision mesh filename=package://valkyrie_description/meshes/reduced_polygon_meshe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; visual mesh filename=package://valkyrie_description/meshes/reduced_polygon_meshe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
- link /v1/RightLittleProximalPhalanx: geometry collision mesh filename=package://valkyrie_description/meshes/reduced_polygon_meshe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; visual mesh filename=package://valkyrie_description/meshes/reduced_polygon_meshe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
- link /v1/RightMedialMetacarpal: geometry collision mesh filename=package://valkyrie_description/meshes/reduced_polygon_meshe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; visual mesh filename=package://valkyrie_description/meshes/reduced_polygon_meshe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
- link /v1/RightMiddleDistalPhalanx: geometry collision mesh filename=package://valkyrie_description/meshes/reduced_polygon_meshe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; visual mesh filename=package://valkyrie_description/meshes/reduced_polygon_meshe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
- link /v1/RightMiddleMedialPhalanx: geometry collision mesh filename=package://valkyrie_description/meshes/reduced_polygon_meshe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; visual mesh filename=package://valkyrie_description/meshes/reduced_polygon_meshe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
- link /v1/RightMiddleProximalPhalanx: geometry collision mesh filename=package://valkyrie_description/meshes/reduced_polygon_meshe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; visual mesh filename=package://valkyrie_description/meshes/reduced_polygon_meshe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
- link /v1/RightPalm: geometry collision mesh filename=package://valkyrie_description/meshes/reduced_polygon_meshe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; visual mesh filename=package://valkyrie_description/meshes/reduced_polygon_meshe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
- link /v1/RightPrimaryDistalPhalanx: geometry collision mesh filename=package://valkyrie_description/meshes/reduced_polygon_meshe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; visual mesh filename=package://valkyrie_description/meshes/reduced_polygon_meshe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
- link /v1/RightPrimaryMedialPhalanx: geometry collision mesh filename=package://valkyrie_description/meshes/reduced_polygon_meshe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; visual mesh filename=package://valkyrie_description/meshes/reduced_polygon_meshe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
- link /v1/RightPrimaryMetacarpal: geometry collision mesh filename=package://valkyrie_description/meshes/reduced_polygon_meshe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; visual mesh filename=package://valkyrie_description/meshes/reduced_polygon_meshe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
- link /v1/RightPrimaryProximalPhalanx: geometry collision mesh filename=package://valkyrie_description/meshes/reduced_polygon_meshe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; visual mesh filename=package://valkyrie_description/meshes/reduced_polygon_meshe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
- link /v1/RightShankStructure: geometry collision mesh filename=package://valkyrie_description/meshes/reduced_polygon_meshe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; visual mesh filename=package://valkyrie_description/meshes/reduced_polygon_meshe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
- link /v1/RightShoulderAdductor: geometry collision mesh filename=package://valkyrie_description/meshes/reduced_polygon_meshe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; visual mesh filename=package://valkyrie_description/meshes/reduced_polygon_meshe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
- link /v1/RightShoulderExtensor: geometry collision mesh filename=package://valkyrie_description/meshes/reduced_polygon_meshe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; visual mesh filename=package://valkyrie_description/meshes/reduced_polygon_meshe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
- link /v1/RightShoulderRotator: geometry collision mesh filename=package://valkyrie_description/meshes/reduced_polygon_meshe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; visual mesh filename=package://valkyrie_description/meshes/reduced_polygon_meshe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
- link /v1/RightThumbDistalPhalanx: geometry collision mesh filename=package://valkyrie_description/meshes/reduced_polygon_meshe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; visual mesh filename=package://valkyrie_description/meshes/reduced_polygon_meshe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
- link /v1/RightThumbMedialPhalanx: geometry collision mesh filename=package://valkyrie_description/meshes/reduced_polygon_meshe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; visual mesh filename=package://valkyrie_description/meshes/reduced_polygon_meshe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
- link /v1/RightThumbMetacarpal: geometry collision mesh filename=package://valkyrie_description/meshes/reduced_polygon_meshe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; visual mesh filename=package://valkyrie_description/meshes/reduced_polygon_meshe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
- link /v1/RightThumbProximalPhalanx: geometry collision mesh filename=package://valkyrie_description/meshes/reduced_polygon_meshe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; visual mesh filename=package://valkyrie_description/meshes/reduced_polygon_meshe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
- link /v1/RightUpperFoot: geometry collision box size=0.082 0.128 0.3; visual mesh filename=package://valkyrie_description/meshes/reduced_polygon_meshe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
- link /v1/Trunk: geometry collision mesh filename=package://valkyrie_description/meshes/reduced_polygon_meshe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; visual mesh filename=package://valkyrie_description/meshes/reduced_polygon_meshe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

File: valkyrie_description/robots/valkyrie_A/xacro/V1.xacro (robot description, xacro)
@@ -3,5 +3,5 @@
     <!-- DO NOT MODIFY URDF BY HAND! YOU ARE A FOOL IF YOU DO! -->
     <!-- ======================================================= -->
-    <xacro:property name="mesh_root" value="package://V1/meshes/reduced_polygon_meshes"/>
+    <xacro:property name="mesh_root" value="package://valkyrie_description/meshes/reduced_polygon_meshes"/>
     <!-- <xacro:include filename="$(find common_xacro)/xacro/mode_setup_hw.xacro" /> -->
     <!-- <xacro:include filename="$(find valkyrie_description)/robots/valkyrie_A/xacro/common/hw_actuator_types.xacro"/> -->

File: valkyrie_description/robots/valkyrie_A/xacro/arm/arm.xacro (robot description, xacro)
@@ -7,5 +7,4 @@
   <xacro:include filename="$(find valkyrie_description)/robots/valkyrie_A/xacro/arm/mass_parameters.xacro"/>
   <xacro:include filename="$(find valkyrie_description)/robots/valkyrie_A/xacro/sensors/camboard.xacro"/>
-  <!-- Link properties. -->
   <xacro:property name="AJ1_Link_Width" value="0.162"/>
   <xacro:property name="AJ1_Link_Height" value="0.202"/>
@@ -241,5 +240,4 @@
                                 actuator1="${actuator2}"   actuator2="${actuator3}"
                                 reflect="1"/>
-                                <!-- because of the hardware configuration, wrist and waist transmissions should always have reflection=1 -->
   </xacro:macro>
   <xacro:macro name="v1_lower_arm_transmissions_simple" params="prefix actuator1 actuator2 actuator3">

File: valkyrie_description/robots/valkyrie_A/xacro/leg/leg.xacro (robot description, xacro)
@@ -97,28 +97,4 @@
       <minDepth>0.00</minDepth>
     </gazebo>
-    <!-- <xacro:box_link_no_mesh name="v1/${prefix}_Foot_Segment1"
-                    width="${Foot_Segment_Width}" height="${Foot_Segment_Height}" depth="${Foot_Segment_Depth}" mass="${Foot_Segment_Mass}"
-                    origin_rpy="0 0 0"
-                    origin_xyz="${Foot_Segment1_Origin_X} ${reflect * Foot_Segment1_Origin_Y} ${reflect * Foot_Segment1_Origin_Z}"/>
-    <xacro:box_link_no_mesh name="v1/${prefix}_Foot_Segment2"
-                    width="${Foot_Segment_Width}" height="${Foot_Segment_Height}" depth="${Foot_Segment_Depth}" mass="${Foot_Segment_Mass}"
-                    origin_rpy="0 0 0"
-                    origin_xyz="${Foot_Segment2_Origin_X} ${reflect * Foot_Segment2_Origin_Y} ${reflect * Foot_Segment2_Origin_Z}"/>
-    <xacro:box_link_no_mesh name="v1/${prefix}_Foot_Segment3"
-                    width="${Foot_Segment_Width}" height="${Foot_Segment_Height}" depth="${Foot_Segment_Depth}" mass="${Foot_Segment_Mass}"
-                    origin_rpy="0 0 0"
-                    origin_xyz="${Foot_Segment3_Origin_X} ${reflect * Foot_Segment3_Origin_Y} ${reflect * Foot_Segment3_Origin_Z}"/> -->
-<!--     <xacro:box_link_no_mesh name="v1/${prefix}_Foot_Segment4"
-                    width="${Foot_Segment_Width}" height="${Foot_Segment_Height}" depth="${Foot_Segment_Depth}" mass="${Foot_Segment_Mass}"
-                    origin_rpy="0 0 0"
-                    origin_xyz="${Foot_Segment4_Origin_X} ${reflect * Foot_Segment4_Origin_Y} ${reflect * Foot_Segment4_Origin_Z}"/> -->
-    <!-- <xacro:box_link_no_mesh name="v1/${prefix}_Foot_Segment5"
-                    width="${Foot_Segment_Width}" height="${Foot_Segment_Height}" depth="${Foot_Segment_Depth}" mass="${Foot_Segment_Mass}"
-                    origin_rpy="0 0 0"
-                    origin_xyz="${Foot_Segment5_Origin_X} ${reflect * Foot_Segment5_Origin_Y} ${reflect * Foot_Segment5_Origin_Z}"/>
-    <xacro:box_link_no_mesh name="v1/${prefix}_Foot_Segment6"
-                    width="${Foot_Segment_Width}" height="${Foot_Segment_Height}" depth="${Foot_Segment_Depth}" mass="${Foot_Segment_Mass}"
-                    origin_rpy="0 0 0"
-                    origin_xyz="${Foot_Segment6_Origin_X} ${reflect * Foot_Segment6_Origin_Y} ${reflect * Foot_Segment6_Origin_Z}"/> -->
   </xacro:macro>
   <xacro:macro name="make_leg_joints" params="prefix reflect leg_root_link">
@@ -231,32 +207,4 @@
                           origin_rpy="${LJ6_Orientation_Roll} ${LJ6_Orientation_Pitch} ${LJ6_Orientation_Yaw}">
     </xacro:fixed_joint>
-  </xacro:macro>
-  <xacro:macro name="make_foot_joints" params="prefix reflect leg_root_link">
-    <!-- JOINTS -->
-    <!-- <xacro:fixed_joint jointName="${prefix}FootSegment1Offset"
-                       parent="${LJ6_Distal_Link}" child="v1/${prefix}_Foot_Segment1"
-                       origin_rpy="0 0 0"
-                       origin_xyz="0 0 0"/>
-    <xacro:fixed_joint jointName="${prefix}FootSegment2Offset"
-                       parent="${LJ6_Distal_Link}" child="v1/${prefix}_Foot_Segment2"
-                       origin_rpy="0 0 0"
-                       origin_xyz="0 0 0"/>
-    <xacro:fixed_joint jointName="${prefix}FootSegment3Offset"
-                       parent="${LJ6_Distal_Link}" child="v1/${prefix}_Foot_Segment3"
-                       origin_rpy="0 0 0"
-                       origin_xyz="0 0 0"/> -->
-<!--
-    <xacro:fixed_joint jointName="${prefix}FootSegment4Offset"
-                       parent="${LJ6_Distal_Link}" child="v1/${prefix}_Foot_Segment4"
-                       origin_rpy="0 0 0"
-                       origin_xyz="0 0 0"/> -->
-    <!-- <xacro:fixed_joint jointName="${prefix}FootSegment5Offset"
-                       parent="${LJ6_Distal_Link}" child="v1/${prefix}_Foot_Segment5"
-                       origin_rpy="0 0 0"
-                       origin_xyz="0 0 0"/>
-    <xacro:fixed_joint jointName="${prefix}FootSegmen65Offset"
-                       parent="${LJ6_Distal_Link}" child="v1/${prefix}_Foot_Segment6"
-                       origin_rpy="0 0 0"
-                       origin_xyz="0 0 0"/> -->
   </xacro:macro>
   <xacro:macro name="make_leg" params="prefix reflect leg_root_link">
