Commit message: Commented out all sensors from xacros to simpify the urdf for now.

File: valkyrie_description/robots/valkyrie_A/valkyrie_A.urdf (robot description, URDF)
Before this commit: robot V1, 85 links, 84 joints
Links:
- removed link /v1/LeftCOP_Frame
- removed link /v1/LeftCamBoardIR_Frame
- removed link /v1/LeftCamBoard_Frame
- removed link /v1/LeftHazardCamera_Frame
- removed link /v1/LeftIMU_Frame
- removed link /v1/LeftLeg6Axis_Frame
- removed link /v1/LeftLegCamBoardIR_Frame
- removed link /v1/LeftLegCamBoard_Frame
- removed link /v1/LeftLegHermes_Frame
- removed link /v1/LeftMPU6000_Frame
- removed link /v1/LeftPelvisIMU_Frame
- removed link /v1/RightCOP_Frame
- removed link /v1/RightCamBoardIR_Frame
- removed link /v1/RightCamBoard_Frame
- removed link /v1/RightHazardCamera_Frame
- removed link /v1/RightIMU_Frame
- removed link /v1/RightLeg6Axis_Frame
- removed link /v1/RightLegCamBoardIR_Frame
- removed link /v1/RightLegCamBoard_Frame
- removed link /v1/RightLegHermes_Frame
- removed link /v1/RightMPU6000_Frame
- removed link /v1/RightPelvisIMU_Frame
Joints:
- removed joint /v1/LeftCOP_Offset
- removed joint /v1/LeftCamBoardIR_Offset
- removed joint /v1/LeftCamBoard_Offset
- removed joint /v1/LeftHazardCamera_Offset
- removed joint /v1/LeftIMU_Offset
- removed joint /v1/LeftLeg6Axis_Offset
- removed joint /v1/LeftLegCamBoardIR_Offset
- removed joint /v1/LeftLegCamBoard_Offset
- removed joint /v1/LeftLegHermes_Offset
- removed joint /v1/LeftMPU6000_Offset
- removed joint /v1/LeftPelvisIMU_Offset
- removed joint /v1/RightCOP_Offset
- removed joint /v1/RightCamBoardIR_Offset
- removed joint /v1/RightCamBoard_Offset
- removed joint /v1/RightHazardCamera_Offset
- removed joint /v1/RightIMU_Offset
- removed joint /v1/RightLeg6Axis_Offset
- removed joint /v1/RightLegCamBoardIR_Offset
- removed joint /v1/RightLegCamBoard_Offset
- removed joint /v1/RightLegHermes_Offset
- removed joint /v1/RightMPU6000_Offset
- removed joint /v1/RightPelvisIMU_Offset

File: valkyrie_description/robots/valkyrie_A/xacro/V1.xacro (robot description, xacro)
@@ -1,3 +1,3 @@
-<robot xmlns:xacro="http://ros.org/wiki/xacro" name="V1">
+<robot xmlns:xacro="http://ros.org/wiki/xacro" name="valkyrie">
     <!-- ======================================================= -->
     <!-- DO NOT MODIFY URDF BY HAND! YOU ARE A FOOL IF YOU DO! -->

File: valkyrie_description/robots/valkyrie_A/xacro/V1_sim_base.xacro (robot description, xacro)
@@ -1,3 +1,3 @@
-<robot xmlns:xacro="http://ros.org/wiki/xacro" name="V1">
+<robot xmlns:xacro="http://ros.org/wiki/xacro" name="valkyrie">
     <!-- ======================================================= -->
     <!-- DO NOT MODIFY URDF BY HAND! YOU ARE A FOOL IF YOU DO! -->
@@ -26,11 +26,11 @@
     <!-- ===== PELVIS ===== -->
     <xacro:make_pelvis />
-    <xacro:v1_pelvis_sensors/>
+    <!-- <xacro:v1_pelvis_sensors/> -->
    <!-- ===== TRUNK ===== -->
     <xacro:make_waist waist_root_link="${Pelvis_Link_Name}" />
     <xacro:v1_waist_actuators name1="${waist_name1}" type1="${waist_type1}" name2="${waist_name2}" type2="${waist_type2}" name3="${waist_name3}" type3="${waist_type3}"/>
-    <xacro:v1_waist_transmissions actuator1="${waist_name1}" actuator2="${waist_name2}" actuator3="${waist_name3}" />
+    <!-- <xacro:v1_waist_transmissions actuator1="${waist_name1}" actuator2="${waist_name2}" actuator3="${waist_name3}" /> -->
     <xacro:v1_waist_modes actuator1="${waist_name1}" actuator2="${waist_name2}" actuator3="${waist_name3}" />
-    <xacro:v1_trunk_sensors/>
+    <!-- <xacro:v1_trunk_sensors/> -->
     <!-- ===== HEAD ===== -->
     <xacro:make_head head_root_link="${WJ3_Distal_Link}" />
@@ -47,9 +47,9 @@
                             name6="${rightarm_name6}" type6="${arm_type6}"
                             name7="${rightarm_name7}" type7="${arm_type7}"/>
-    <xacro:v1_upper_arm_transmissions prefix="Right" actuator1="${rightarm_name1}" actuator2="${rightarm_name2}" actuator3="${rightarm_name3}" actuator4="${rightarm_name4}"/>
-    <xacro:v1_lower_arm_transmissions prefix="Right" actuator1="${rightarm_name5}" actuator2="${rightarm_name6}" actuator3="${rightarm_name7}"/>
+    <!-- <xacro:v1_upper_arm_transmissions prefix="Right" actuator1="${rightarm_name1}" actuator2="${rightarm_name2}" actuator3="${rightarm_name3}" actuator4="${rightarm_name4}"/> -->
+    <!-- <xacro:v1_lower_arm_transmissions prefix="Right" actuator1="${rightarm_name5}" actuator2="${rightarm_name6}" actuator3="${rightarm_name7}"/> -->
     <xacro:v1_arm_modes prefix="Right" actuator1="${rightarm_name1}" actuator2="${rightarm_name2}" actuator3="${rightarm_name3}" actuator4="${rightarm_name4}" actuator5="${rightarm_name5}" actuator6="${rightarm_name6}" actuator7="${rightarm_name7}"/>
     <!-- Why is this not symmetric?? -->
-    <xacro:v1_arm_sensors />
+    <!-- <xacro:v1_arm_sensors /> -->
     <!-- ===== RIGHT THUMB ===== -->
     <xacro:make_thumb_fixed prefix="Right" reflect="1" thumb_root_link="/v1/RightPalm"/>
@@ -73,6 +73,6 @@
                             name6="${leftarm_name6}" type6="${arm_type6}"
                             name7="${leftarm_name7}" type7="${arm_type7}"/>
-    <xacro:v1_upper_arm_transmissions prefix="Left" actuator1="${leftarm_name1}" actuator2="${leftarm_name2}" actuator3="${leftarm_name3}" actuator4="${leftarm_name4}"/>
-    <xacro:v1_lower_arm_transmissions prefix="Left" actuator1="${leftarm_name5}" actuator2="${leftarm_name6}" actuator3="${leftarm_name7}"/>
+    <!-- <xacro:v1_upper_arm_transmissions prefix="Left" actuator1="${leftarm_name1}" actuator2="${leftarm_name2}" actuator3="${leftarm_name3}" actuator4="${leftarm_name4}"/> -->
+    <!-- <xacro:v1_lower_arm_transmissions prefix="Left" actuator1="${leftarm_name5}" actuator2="${leftarm_name6}" actuator3="${leftarm_name7}"/> -->
     <xacro:v1_arm_modes prefix="Left" actuator1="${leftarm_name1}" actuator2="${leftarm_name2}" actuator3="${leftarm_name3}" actuator4="${leftarm_name4}" actuator5="${leftarm_name5}" actuator6="${leftarm_name6}" actuator7="${leftarm_name7}"/>
     <!-- ===== LEFT THUMB ===== -->
@@ -96,5 +96,5 @@
                             name5="${rightleg_name5}" type5="${leg_type5}"
                             name6="${rightleg_name6}" type6="${leg_type6}"/>
-    <xacro:v1_leg_transmissions prefix="Right" reflect="1"
+    <!-- <xacro:v1_leg_transmissions prefix="Right" reflect="1"
                                                actuator1="${rightleg_name1}"
                                                actuator2="${rightleg_name2}"
@@ -102,5 +102,5 @@
                                                actuator4="${rightleg_name4}"
                                                actuator5="${rightleg_name5}"
-                                               actuator6="${rightleg_name6}" />
+                                               actuator6="${rightleg_name6}" /> -->
     <xacro:v1_leg_modes prefix="Right" actuator1="${rightleg_name1}"
                                        actuator2="${rightleg_name2}"
@@ -109,6 +109,6 @@
                                        actuator5="${rightleg_name5}"
                                        actuator6="${rightleg_name6}" />
-    <xacro:v1_leg_sensors prefix="Right" reflect="1" />
-    <xacro:v1_hw_sensors prefix="Right" hermes_node="${rightleg_hermes}" atidaq_node="${rightleg_ati}" mpu6000_node="${rightleg_mpu2000}" cop_node="${rightleg_cop}"/>
+    <!-- <xacro:v1_leg_sensors prefix="Right" reflect="1" /> -->
+    <!-- <xacro:v1_hw_sensors prefix="Right" hermes_node="${rightleg_hermes}" atidaq_node="${rightleg_ati}" mpu6000_node="${rightleg_mpu2000}" cop_node="${rightleg_cop}"/> -->
     <!-- ===== LEFT LEG ===== -->
     <xacro:make_leg prefix="Left" reflect="-1" leg_root_link="${Pelvis_Link_Name}" />
@@ -119,5 +119,5 @@
                             name5="${leftleg_name5}" type5="${leg_type5}"
                             name6="${leftleg_name6}" type6="${leg_type6}"/>
-    <xacro:v1_leg_transmissions prefix="Left" reflect="-1"
+    <!-- <xacro:v1_leg_transmissions prefix="Left" reflect="-1"
                                                actuator1="${leftleg_name1}"
                                                actuator2="${leftleg_name2}"
@@ -125,5 +125,5 @@
                                                actuator4="${leftleg_name4}"
                                                actuator5="${leftleg_name5}"
-                                               actuator6="${leftleg_name6}" />
+                                               actuator6="${leftleg_name6}" /> -->
     <xacro:v1_leg_modes prefix="Left" actuator1="${leftleg_name1}"
                                        actuator2="${leftleg_name2}"
@@ -132,5 +132,5 @@
                                        actuator5="${leftleg_name5}"
                                        actuator6="${leftleg_name6}" />
-    <xacro:v1_leg_sensors prefix="Left" reflect="-1" />
-    <xacro:v1_hw_sensors prefix="Left" hermes_node="${leftleg_hermes}" atidaq_node="${leftleg_ati}" mpu6000_node="${leftleg_mpu2000}" cop_node="${leftleg_cop}"/>
+    <!-- <xacro:v1_leg_sensors prefix="Left" reflect="-1" /> -->
+    <!-- <xacro:v1_hw_sensors prefix="Left" hermes_node="${leftleg_hermes}" atidaq_node="${leftleg_ati}" mpu6000_node="${leftleg_mpu2000}" cop_node="${leftleg_cop}"/> -->
 </robot>
