Commit message: Changed link/joint names of everything but a few of the fingers. Also removed 4th pinky joint/link because they don't actually exist.

File: valkyrie_description/robots/valkyrie_A/valkyrie_A.urdf (robot description, URDF)
Before this commit: robot valkyrie, 63 links, 62 joints
Links:
- removed link /v1/Head
- removed link /v1/LeftAnkleYoke
- removed link /v1/LeftElbowExtensor
- removed link /v1/LeftForearm
- removed link /v1/LeftHipAdductor
- removed link /v1/LeftHipRotator
- removed link /v1/LeftLeg
- removed link /v1/LeftLittleDistalPhalanx
- removed link /v1/LeftLittleMedialPhalanx
- removed link /v1/LeftLittleProximalPhalanx
- removed link /v1/LeftMedialMetacarpal
- removed link /v1/LeftPalm
- removed link /v1/LeftShankStructure
- removed link /v1/LeftShoulderAdductor
- removed link /v1/LeftShoulderExtensor
- removed link /v1/LeftShoulderRotator
- removed link /v1/LeftUpperFoot
- removed link /v1/LeftWristYoke
- removed link /v1/LowerNeckExtensor
- removed link /v1/NeckRotator
- removed link /v1/Pelvis
- removed link /v1/RightAnkleYoke
- removed link /v1/RightElbowExtensor
- removed link /v1/RightForearm
- removed link /v1/RightHipAdductor
- removed link /v1/RightHipRotator
- removed link /v1/RightLeg
- removed link /v1/RightLittleDistalPhalanx
- removed link /v1/RightLittleMedialPhalanx
- removed link /v1/RightLittleProximalPhalanx
- removed link /v1/RightMedialMetacarpal
- removed link /v1/RightPalm
- removed link /v1/RightShankStructure
- removed link /v1/RightShoulderAdductor
- removed link /v1/RightShoulderExtensor
- removed link /v1/RightShoulderRotator
- removed link /v1/RightUpperFoot
- removed link /v1/RightWristYoke
- removed link /v1/Trunk
- removed link /v1/WaistExtensor
- removed link /v1/WaistRotator
- added link /v1/LeftPinkyPitch1, mass 0.047; collision mesh filename=package://valkyrie_description/meshes/reduced_polygon_meshe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; visual mesh filename=package://valkyrie_description/meshes/reduced_polygon_meshe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
- added link /v1/LeftPinkyPitch2, mass 0.02; collision mesh filename=package://valkyrie_description/meshes/reduced_polygon_meshe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; visual mesh filename=package://valkyrie_description/meshes/reduced_polygon_meshe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
- added link /v1/LeftPinkyPitch3, mass 0.011; collision mesh filename=package://valkyrie_description/meshes/reduced_polygon_meshe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; visual mesh filename=package://valkyrie_description/meshes/reduced_polygon_meshe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
- added link /v1/RightPinkyPitch1, mass 0.047; collision mesh filename=package://valkyrie_description/meshes/reduced_polygon_meshe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; visual mesh filename=package://valkyrie_description/meshes/reduced_polygon_meshe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
- added link /v1/RightPinkyPitch2, mass 0.02; collision mesh filename=package://valkyrie_description/meshes/reduced_polygon_meshe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; visual mesh filename=package://valkyrie_description/meshes/reduced_polygon_meshe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
- added link /v1/RightPinkyPitch3, mass 0.011; collision mesh filename=package://valkyrie_description/meshes/reduced_polygon_meshe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; visual mesh filename=package://valkyrie_description/meshes/reduced_polygon_meshe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
- added link Head, mass 4.06; collision mesh filename=package://valkyrie_description/meshes/reduced_polygon_meshe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; visual mesh filename=package://valkyrie_description/meshes/reduced_polygon_meshe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
- added link LeftAnkleRoll, mass 0.395; collision box size=0.033 0.076 0.025; visual box size=0.033 0.076 0.025
- added link LeftElbowPitch, mass 2.367; collision mesh filename=package://valkyrie_description/meshes/reduced_polygon_meshe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; visual mesh filename=package://valkyrie_description/meshes/reduced_polygon_meshe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
- added link LeftFoot, mass 1.888; collision box size=0.082 0.128 0.3; visual mesh filename=package://valkyrie_description/meshes/reduced_polygon_meshe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
- added link LeftForearm, mass 2.903; collision mesh filename=package://valkyrie_description/meshes/reduced_polygon_meshe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; visual mesh filename=package://valkyrie_description/meshes/reduced_polygon_meshe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
- added link LeftHipPitch, mass 10.3; collision mesh filename=package://valkyrie_description/meshes/reduced_polygon_meshe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; visual mesh filename=package://valkyrie_description/meshes/reduced_polygon_meshe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
- added link LeftHipRoll, mass 5.95; collision mesh filename=package://valkyrie_description/meshes/reduced_polygon_meshe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; visual mesh filename=package://valkyrie_description/meshes/reduced_polygon_meshe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
- added link LeftHipYaw, mass 2.39; collision mesh filename=package://valkyrie_description/meshes/reduced_polygon_meshe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; visual mesh filename=package://valkyrie_description/meshes/reduced_polygon_meshe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
- added link LeftKneePitch, mass 7.4; collision mesh filename=package://valkyrie_description/meshes/reduced_polygon_meshe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; visual mesh filename=package://valkyrie_description/meshes/reduced_polygon_meshe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
- added link LeftPalm, mass 0.712; collision mesh filename=package://valkyrie_description/meshes/reduced_polygon_meshe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; visual mesh filename=package://valkyrie_description/meshes/reduced_polygon_meshe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
- added link LeftShoulderPitch, mass 2.65; collision mesh filename=package://valkyrie_description/meshes/reduced_polygon_meshe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; visual mesh filename=package://valkyrie_description/meshes/reduced_polygon_meshe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
- added link LeftShoulderRoll, mass 2.87; collision mesh filename=package://valkyrie_description/meshes/reduced_polygon_meshe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; visual mesh filename=package://valkyrie_description/meshes/reduced_polygon_meshe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
- added link LeftShoulderYaw, mass 2.575; collision mesh filename=package://valkyrie_description/meshes/reduced_polygon_meshe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; visual mesh filename=package://valkyrie_description/meshes/reduced_polygon_meshe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
- added link LeftWristPitch, mass 0.1; collision box size=0.03 0.01 0.051; visual box size=0.03 0.01 0.051
- added link LowerNeckPitch, mass 0.1; collision mesh filename=package://valkyrie_description/meshes/reduced_polygon_meshe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; visual mesh filename=package://valkyrie_description/meshes/reduced_polygon_meshe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
- added link NeckYaw, mass 0.1; collision mesh filename=package://valkyrie_description/meshes/reduced_polygon_meshe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; visual mesh filename=package://valkyrie_description/meshes/reduced_polygon_meshe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
- added link Pelvis, mass 6.986; collision mesh filename=package://valkyrie_description/meshes/reduced_polygon_meshe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; visual mesh filename=package://valkyrie_description/meshes/reduced_polygon_meshe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
- added link RightAnkleRoll, mass 0.395; collision box size=0.033 0.076 0.025; visual box size=0.033 0.076 0.025
- added link RightElbowPitch, mass 2.367; collision mesh filename=package://valkyrie_description/meshes/reduced_polygon_meshe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; visual mesh filename=package://valkyrie_description/meshes/reduced_polygon_meshe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
- added link RightFoot, mass 1.888; collision box size=0.082 0.128 0.3; visual mesh filename=package://valkyrie_description/meshes/reduced_polygon_meshe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
- added link RightForearm, mass 2.903; collision mesh filename=package://valkyrie_description/meshes/reduced_polygon_meshe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; visual mesh filename=package://valkyrie_description/meshes/reduced_polygon_meshe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
- added link RightHipPitch, mass 10.3; collision mesh filename=package://valkyrie_description/meshes/reduced_polygon_meshe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; visual mesh filename=package://valkyrie_description/meshes/reduced_polygon_meshe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
- added link RightHipRoll, mass 5.95; collision mesh filename=package://valkyrie_description/meshes/reduced_polygon_meshe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; visual mesh filename=package://valkyrie_description/meshes/reduced_polygon_meshe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
- added link RightHipYaw, mass 2.39; collision mesh filename=package://valkyrie_description/meshes/reduced_polygon_meshe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; visual mesh filename=package://valkyrie_description/meshes/reduced_polygon_meshe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
- added link RightKneePitch, mass 7.4; collision mesh filename=package://valkyrie_description/meshes/reduced_polygon_meshe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; visual mesh filename=package://valkyrie_description/meshes/reduced_polygon_meshe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
- added link RightPalm, mass 0.712; collision mesh filename=package://valkyrie_description/meshes/reduced_polygon_meshe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; visual mesh filename=package://valkyrie_description/meshes/reduced_polygon_meshe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
- added link RightShoulderPitch, mass 2.65; collision mesh filename=package://valkyrie_description/meshes/reduced_polygon_meshe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; visual mesh filename=package://valkyrie_description/meshes/reduced_polygon_meshe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
- added link RightShoulderRoll, mass 2.87; collision mesh filename=package://valkyrie_description/meshes/reduced_polygon_meshe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; visual mesh filename=package://valkyrie_description/meshes/reduced_polygon_meshe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
- added link RightShoulderYaw, mass 2.575; collision mesh filename=package://valkyrie_description/meshes/reduced_polygon_meshe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; visual mesh filename=package://valkyrie_description/meshes/reduced_polygon_meshe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
- added link RightWristPitch, mass 0.1; collision box size=0.03 0.01 0.051; visual box size=0.03 0.01 0.051
- added link TorsoPitch, mass 0.1
- added link TorsoRoll, mass 42.6; collision mesh filename=package://valkyrie_description/meshes/reduced_polygon_meshe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; visual mesh filename=package://valkyrie_description/meshes/reduced_polygon_meshe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
- added link TorsoYaw, mass 0.1
Joints:
- removed joint LeftAnkle
- removed joint LeftAnkleExtensor
- removed joint LeftElbowExtensor
- removed joint LeftForearmSupinator
- removed joint LeftHipAdductor
- removed joint LeftHipExtensor
- removed joint LeftHipRotator
- removed joint LeftKneeExtensor
- removed joint LeftLittleDIPExtensor
- removed joint LeftLittleMPExtensor
- removed joint LeftLittleMPYaw
- removed joint LeftLittlePIPExtensor
- removed joint LeftShoulderAdductor
- removed joint LeftShoulderExtensor
- removed joint LeftShoulderSupinator
- removed joint LeftWrist
- removed joint LeftWristExtensor
- removed joint LowerNeckExtensor
- removed joint NeckRotator
- removed joint RightAnkle
- removed joint RightAnkleExtensor
- removed joint RightElbowExtensor
- removed joint RightForearmSupinator
- removed joint RightHipAdductor
- removed joint RightHipExtensor
- removed joint RightHipRotator
- removed joint RightKneeExtensor
- removed joint RightLittleDIPExtensor
- removed joint RightLittleMPExtensor
- removed joint RightLittleMPYaw
- removed joint RightLittlePIPExtensor
- removed joint RightShoulderAdductor
- removed joint RightShoulderExtensor
- removed joint RightShoulderSupinator
- removed joint RightWrist
- removed joint RightWristExtensor
- removed joint UpperNeckExtensor
- removed joint WaistExtensor
- removed joint WaistLateralExtensor
- removed joint WaistRotator
- added joint LeftAnklePitch: type revolute, parent LeftKneePitch, child LeftAnkleRoll, origin xyz=0.406 0 0 rpy=3.14159265359 0 0, axis 0 0 1, limit lower=-0.8726646255 upper=0.8726646255 effort=205 velocity=11
- added joint LeftAnkleRoll: type revolute, parent LeftAnkleRoll, child LeftFoot, origin xyz=0.0127 0 0 rpy=-1.57079632679 0 -0.13, axis 0 0 1, limit lower=-0.3490658502 upper=0.3490658502 effort=205 velocity=11
- added joint LeftElbowPitch: type revolute, parent LeftShoulderYaw, child LeftElbowPitch, origin xyz=0 0.0254 0.33 rpy=-1.57079632679 0 -1.57079632679, axis 0 0 1, limit lower=-1.9198621761 upper=-0.08726646255 effort=65 velocity=11.5
- added joint LeftForearmYaw: type revolute, parent LeftElbowPitch, child LeftForearm, origin xyz=0.0254 0 0 rpy=-1.57079632679 0 3.14159265359, axis 0 0 1, limit lower=-2.35619448885 upper=2.35619448885 effort=26 velocity=5
- added joint LeftHipPitch: type revolute, parent LeftHipRoll, child LeftHipPitch, origin xyz=0 0.061 0 rpy=1.57079632679 0 1.57079632679, axis 0 0 1, limit lower=-2.35619448885 upper=1.71042266598 effort=350 velocity=6.11
- added joint LeftHipRoll: type revolute, parent LeftHipYaw, child LeftHipRoll, origin xyz=0 0 0 rpy=1.57079632679 0 0, axis 0 0 1, limit lower=-0.5235987753 upper=0.26179938765 effort=350 velocity=7
- added joint LeftHipYaw: type revolute, parent Pelvis, child LeftHipYaw, origin xyz=0 0.1016 -0.183 rpy=3.14159265359 0 1.57079632679, axis 0 0 1, limit lower=-0.5235987753 upper=0.169296937347 effort=190 velocity=5.89
- added joint LeftKneePitch: type revolute, parent LeftHipPitch, child LeftKneePitch, origin xyz=0.431 0 0.0374 rpy=3.14159265359 0 0, axis 0 0 1, limit lower=-1.90240888359 upper=0.218166156375 effort=350 velocity=6.11
- added joint LeftPinkyPitch1: type fixed, parent LeftPalm, child /v1/LeftPinkyPitch1, origin xyz=0.0427072303336 0.0352928446888 0.007747 rpy=1.57079632679 0 0.690626785, axis 0 0 1
- added joint LeftPinkyPitch2: type fixed, parent /v1/LeftPinkyPitch1, child /v1/LeftPinkyPitch2, origin xyz=0 -0.010287 0.071327 rpy=-0.690626785 0 1.57079632679, axis 0 0 1
- added joint LeftPinkyPitch3: type fixed, parent /v1/LeftPinkyPitch2, child /v1/LeftPinkyPitch3, origin xyz=0 -0.0381 -0.050169 rpy=0 0 -1.57079632679, axis 0 0 1
- added joint LeftShoulderPitch: type revolute, parent TorsoRoll, child LeftShoulderPitch, origin xyz=0.29842 0 -0.03157 rpy=1.57079632679 0 0, axis 0 0 1, limit lower=-3.1415926518 upper=3.1415926518 effort=190 velocity=5.89
- added joint LeftShoulderRoll: type revolute, parent LeftShoulderPitch, child LeftShoulderRoll, origin xyz=0 0 0.246 rpy=-1.57079632679 0 3.14159265359, axis 0 0 1, limit lower=-3.05432618925 upper=-0.155 effort=190 velocity=5.89
- added joint LeftShoulderYaw: type revolute, parent LeftShoulderRoll, child LeftShoulderYaw, origin xyz=0 0 0 rpy=-1.57079632679 0 -1.57079632679, axis 0 0 1, limit lower=-1.5707963259 upper=1.7 effort=65 velocity=11.5
- added joint LeftWristPitch: type revolute, parent LeftForearm, child LeftWristPitch, origin xyz=0 0 0.287 rpy=-1.57079632679 0 -1.57079632679, axis 0 0 1, limit lower=-0.8726646255 upper=0.6981317004 effort=14 velocity=1
- added joint LeftWristRoll: type revolute, parent LeftWristPitch, child LeftPalm, origin xyz=0 0 0 rpy=-1.57079632679 0 -1.57079632679, axis 0 0 1, limit lower=-0.5235987753 upper=0.43633231275 effort=14 velocity=1
- added joint LowerNeckPitch: type revolute, parent TorsoRoll, child LowerNeckPitch, origin xyz=0.3383 0 0.0519 rpy=-1.57079632679 0 0, axis 0 0 1, limit lower=-1.5707963259 upper=0 effort=26 velocity=5
- added joint NeckYaw: type revolute, parent LowerNeckPitch, child NeckYaw, origin xyz=0 0.0519 0 rpy=1.57079632679 0 1.57079632679, axis 0 0 1, limit lower=-1.5707963259 upper=1.5707963259 effort=26 velocity=5
- added joint RightAnklePitch: type revolute, parent RightKneePitch, child RightAnkleRoll, origin xyz=0.406 0 0 rpy=3.14159265359 0 0, axis 0 0 1, limit lower=-0.8726646255 upper=0.8726646255 effort=205 velocity=11
- added joint RightAnkleRoll: type revolute, parent RightAnkleRoll, child RightFoot, origin xyz=0.0127 0 0 rpy=1.57079632679 0 -0.13, axis 0 0 1, limit lower=-0.3490658502 upper=0.3490658502 effort=205 velocity=11
- added joint RightElbowPitch: type revolute, parent RightShoulderYaw, child RightElbowPitch, origin xyz=0 -0.0254 -0.33 rpy=1.57079632679 0 1.57079632679, axis 0 0 1, limit lower=-1.9198621761 upper=-0.08726646255 effort=65 velocity=11.5
- added joint RightForearmYaw: type revolute, parent RightElbowPitch, child RightForearm, origin xyz=0.0254 0 0 rpy=1.57079632679 0 3.14159265359, axis 0 0 1, limit lower=-2.35619448885 upper=2.35619448885 effort=26 velocity=5
- added joint RightHipPitch: type revolute, parent RightHipRoll, child RightHipPitch, origin xyz=0 0.061 0 rpy=-1.57079632679 0 1.57079632679, axis 0 0 1, limit lower=-2.35619448885 upper=1.71042266598 effort=350 velocity=6.11
- added joint RightHipRoll: type revolute, parent RightHipYaw, child RightHipRoll, origin xyz=0 0 0 rpy=-1.57079632679 0 0, axis 0 0 1, limit lower=-0.5235987753 upper=0.26179938765 effort=350 velocity=7
- added joint RightHipYaw: type revolute, parent Pelvis, child RightHipYaw, origin xyz=0 -0.1016 -0.183 rpy=0.0 0 -1.57079632679, axis 0 0 1, limit lower=-0.5235987753 upper=0.169296937347 effort=190 velocity=5.89
- added joint RightKneePitch: type revolute, parent RightHipPitch, child RightKneePitch, origin xyz=0.431 0 -0.0374 rpy=3.14159265359 0 0, axis 0 0 1, limit lower=-1.90240888359 upper=0.218166156375 effort=350 velocity=6.11
- added joint RightPinkyPitch1: type fixed, parent RightPalm, child /v1/RightPinkyPitch1, origin xyz=0.0427072303336 0.0352928446888 -0.007747 rpy=-1.57079632679 0 0.690626785, axis 0 0 1
- added joint RightPinkyPitch2: type fixed, parent /v1/RightPinkyPitch1, child /v1/RightPinkyPitch2, origin xyz=0 -0.010287 -0.071327 rpy=-0.690626785 0 -1.57079632679, axis 0 0 1
- added joint RightPinkyPitch3: type fixed, parent /v1/RightPinkyPitch2, child /v1/RightPinkyPitch3, origin xyz=0 0.0381 0.050169 rpy=0 0 1.57079632679, axis 0 0 1
- added joint RightShoulderPitch: type revolute, parent TorsoRoll, child RightShoulderPitch, origin xyz=0.29842 0 -0.03157 rpy=1.57079632679 0 0, axis 0 0 1, limit lower=-3.1415926518 upper=3.1415926518 effort=190 velocity=5.89
- added joint RightShoulderRoll: type revolute, parent RightShoulderPitch, child RightShoulderRoll, origin xyz=0 0 -0.246 rpy=1.57079632679 0 3.14159265359, axis 0 0 1, limit lower=-3.05432618925 upper=-0.155 effort=190 velocity=5.89
- added joint RightShoulderYaw: type revolute, parent RightShoulderRoll, child RightShoulderYaw, origin xyz=0 0 0 rpy=-1.57079632679 0 1.57079632679, axis 0 0 1, limit lower=-1.5707963259 upper=1.7 effort=65 velocity=11.5
- added joint RightWristPitch: type revolute, parent RightForearm, child RightWristPitch, origin xyz=0 0 -0.287 rpy=-1.57079632679 0 1.57079632679, axis 0 0 1, limit lower=-0.8726646255 upper=0.6981317004 effort=14 velocity=1
- added joint RightWristRoll: type revolute, parent RightWristPitch, child RightPalm, origin xyz=0 0 0 rpy=1.57079632679 0 1.57079632679, axis 0 0 1, limit lower=-0.5235987753 upper=0.43633231275 effort=14 velocity=1
- added joint TorsoPitch: type revolute, parent TorsoYaw, child TorsoPitch, origin xyz=0.04191 0 0 rpy=1.57079632679 0 0, axis 0 0 1, limit lower=-0.6981317004 upper=0.08726646255 effort=150 velocity=9
- added joint TorsoRoll: type revolute, parent TorsoPitch, child TorsoRoll, origin xyz=0 0.020352 0 rpy=1.57079632679 0 1.57079632679, axis 0 0 1, limit lower=-0.26179938765 upper=0.26179938765 effort=150 velocity=9
- added joint TorsoYaw: type revolute, parent Pelvis, child TorsoYaw, origin xyz=0 0 0 rpy=0 0 0, axis 0 0 1, limit lower=-0.6981317004 upper=0.6981317004 effort=190 velocity=5.89
- added joint UpperNeckPitch: type revolute, parent NeckYaw, child Head, origin xyz=0.06 0 0.196 rpy=-1.57079632679 0 0, axis 0 0 1, limit lower=-0.08726646255 upper=0.78539816295 effort=26 velocity=5
- joint LeftMiddleMPExtensor: parent /v1/LeftPalm -> LeftPalm
- joint LeftPrimaryMPYaw: parent /v1/LeftPalm -> LeftPalm
- joint LeftThumbMPYaw: parent /v1/LeftPalm -> LeftPalm
- joint RightMiddleMPExtensor: parent /v1/RightPalm -> RightPalm
- joint RightPrimaryMPYaw: parent /v1/RightPalm -> RightPalm
- joint RightThumbMPYaw: parent /v1/RightPalm -> RightPalm

File: valkyrie_description/robots/valkyrie_A/xacro/V1_sim_base.xacro (robot description, xacro)
@@ -50,14 +50,14 @@
     <!-- <xacro:v1_arm_sensors /> -->
     <!-- ===== RIGHT THUMB ===== -->
-    <xacro:make_thumb_fixed prefix="Right" reflect="1" thumb_root_link="/v1/RightPalm"/>
+    <xacro:make_thumb_fixed prefix="Right" reflect="1" thumb_root_link="RightPalm"/>
     <!-- <xacro:make_right_thumb_interface api="${finger_api}"/> -->
     <!-- ===== RIGHT PRIMARY FINGER ===== -->
-    <xacro:make_primary_finger_fixed prefix="Right" reflect="1" primary_finger_root_link="/v1/RightPalm"/>
+    <xacro:make_primary_finger_fixed prefix="Right" reflect="1" primary_finger_root_link="RightPalm"/>
     <!-- <xacro:make_right_primary_finger_interface api="${finger_api}"/> -->
     <!-- ===== RIGHT MIDDLE FINGER ===== -->
-    <xacro:make_middle_finger_fixed prefix="Right" reflect="1" middle_finger_root_link="/v1/RightPalm"/>
+    <xacro:make_middle_finger_fixed prefix="Right" reflect="1" middle_finger_root_link="RightPalm"/>
     <!-- <xacro:make_right_middle_finger_interface api="${finger_api}"/> -->
     <!-- ===== RIGHT LITTLE FINGER ===== -->
-    <xacro:make_little_finger_fixed prefix="Right" reflect="1" little_finger_root_link="/v1/RightPalm"/>
+    <xacro:make_little_finger_fixed prefix="Right" reflect="1" little_finger_root_link="RightPalm"/>
     <!-- <xacro:make_right_little_finger_interface api="${finger_api}"/> -->
     <!-- ===== LEFT ARM ===== -->
@@ -74,14 +74,14 @@
     <!-- <xacro:v1_arm_modes prefix="Left" actuator1="${leftarm_name1}" actuator2="${leftarm_name2}" actuator3="${leftarm_name3}" actuator4="${leftarm_name4}" actuator5="${leftarm_name5}" actuator6="${leftarm_name6}" actuator7="${leftarm_name7}"/> -->
     <!-- ===== LEFT THUMB ===== -->
-    <xacro:make_thumb_fixed prefix="Left" reflect="-1" thumb_root_link="/v1/LeftPalm"/>
+    <xacro:make_thumb_fixed prefix="Left" reflect="-1" thumb_root_link="LeftPalm"/>
     <!-- <xacro:make_left_thumb_interface api="${finger_api}"/> -->
     <!-- ===== LEFT PRIMARY FINGER ===== -->
-    <xacro:make_primary_finger_fixed prefix="Left" reflect="-1" primary_finger_root_link="/v1/LeftPalm"/>
+    <xacro:make_primary_finger_fixed prefix="Left" reflect="-1" primary_finger_root_link="LeftPalm"/>
     <!-- <xacro:make_left_primary_finger_interface api="${finger_api}"/> -->
     <!-- ===== LEFT MIDDLE FINGER ===== -->
-    <xacro:make_middle_finger_fixed prefix="Left" reflect="-1" middle_finger_root_link="/v1/LeftPalm"/>
+    <xacro:make_middle_finger_fixed prefix="Left" reflect="-1" middle_finger_root_link="LeftPalm"/>
     <!-- <xacro:make_left_middle_finger_interface api="${finger_api}"/> -->
     <!-- ===== LEFT LITTLE FINGER ===== -->
-    <xacro:make_little_finger_fixed prefix="Left" reflect="-1" little_finger_root_link="/v1/LeftPalm"/>
+    <xacro:make_little_finger_fixed prefix="Left" reflect="-1" little_finger_root_link="LeftPalm"/>
     <!-- <xacro:make_left_little_finger_interface api="${finger_api}"/> -->
     <!-- ===== RIGHT LEG ===== -->

File: valkyrie_description/robots/valkyrie_A/xacro/arm/joint_names.xacro (robot description, xacro)
@@ -1,10 +1,10 @@
 <?xml version="1.0" ?>
 <robot xmlns:xacro="http://www.ros.org/wiki/xacro" name="v1/arm/joint_names">
-  <xacro:property name="AJ1_Joint_Name" value="${prefix}ShoulderExtensor" />
-  <xacro:property name="AJ2_Joint_Name" value="${prefix}ShoulderAdductor" />
-  <xacro:property name="AJ3_Joint_Name" value="${prefix}ShoulderSupinator" />
-  <xacro:property name="AJ4_Joint_Name" value="${prefix}ElbowExtensor" />
-  <xacro:property name="AJ5_Joint_Name" value="${prefix}ForearmSupinator" />
-  <xacro:property name="AJ6_Joint_Name" value="${prefix}WristExtensor" />
-  <xacro:property name="AJ7_Joint_Name" value="${prefix}Wrist" />
+  <xacro:property name="AJ1_Joint_Name" value="${prefix}ShoulderPitch" />
+  <xacro:property name="AJ2_Joint_Name" value="${prefix}ShoulderRoll" />
+  <xacro:property name="AJ3_Joint_Name" value="${prefix}ShoulderYaw" />
+  <xacro:property name="AJ4_Joint_Name" value="${prefix}ElbowPitch" />
+  <xacro:property name="AJ5_Joint_Name" value="${prefix}ForearmYaw" />
+  <xacro:property name="AJ6_Joint_Name" value="${prefix}WristPitch" />
+  <xacro:property name="AJ7_Joint_Name" value="${prefix}WristRoll" />
 </robot>
