Commit message: Changed link/joint names of everything but a few of the fingers. Also removed 4th pinky joint/link because they don't actually exist.

File: valkyrie_description/robots/valkyrie_A/xacro/arm/link_names.xacro (robot description, xacro)
@@ -2,16 +2,16 @@
 <robot xmlns:xacro="http://www.ros.org/wiki/xacro" name="v1/arm/link_names">
   <xacro:property name="AJ1_Proximal_Link" value="${arm_root_link}" />
-  <xacro:property name="AJ1_Distal_Link" value="/v1/${prefix}ShoulderExtensor" />
-  <xacro:property name="AJ2_Proximal_Link" value="/v1/${prefix}ShoulderExtensor" />
-  <xacro:property name="AJ2_Distal_Link" value="/v1/${prefix}ShoulderAdductor" />
-  <xacro:property name="AJ3_Proximal_Link" value="/v1/${prefix}ShoulderAdductor" />
-  <xacro:property name="AJ3_Distal_Link" value="/v1/${prefix}ShoulderRotator" />
-  <xacro:property name="AJ4_Proximal_Link" value="/v1/${prefix}ShoulderRotator" />
-  <xacro:property name="AJ4_Distal_Link" value="/v1/${prefix}ElbowExtensor" />
-  <xacro:property name="AJ5_Proximal_Link" value="/v1/${prefix}ElbowExtensor" />
-  <xacro:property name="AJ5_Distal_Link" value="/v1/${prefix}Forearm" />
-  <xacro:property name="AJ6_Proximal_Link" value="/v1/${prefix}Forearm" />
-  <xacro:property name="AJ6_Distal_Link" value="/v1/${prefix}WristYoke" />
-  <xacro:property name="AJ7_Proximal_Link" value="/v1/${prefix}WristYoke" />
-  <xacro:property name="AJ7_Distal_Link" value="/v1/${prefix}Palm" />
+  <xacro:property name="AJ1_Distal_Link" value="${prefix}ShoulderPitch" />
+  <xacro:property name="AJ2_Proximal_Link" value="${prefix}ShoulderPitch" />
+  <xacro:property name="AJ2_Distal_Link" value="${prefix}ShoulderRoll" />
+  <xacro:property name="AJ3_Proximal_Link" value="${prefix}ShoulderRoll" />
+  <xacro:property name="AJ3_Distal_Link" value="${prefix}ShoulderYaw" />
+  <xacro:property name="AJ4_Proximal_Link" value="${prefix}ShoulderYaw" />
+  <xacro:property name="AJ4_Distal_Link" value="${prefix}ElbowPitch" />
+  <xacro:property name="AJ5_Proximal_Link" value="${prefix}ElbowPitch" />
+  <xacro:property name="AJ5_Distal_Link" value="${prefix}Forearm" />
+  <xacro:property name="AJ6_Proximal_Link" value="${prefix}Forearm" />
+  <xacro:property name="AJ6_Distal_Link" value="${prefix}WristPitch" />
+  <xacro:property name="AJ7_Proximal_Link" value="${prefix}WristPitch" />
+  <xacro:property name="AJ7_Distal_Link" value="${prefix}Palm" />
 </robot>

File: valkyrie_description/robots/valkyrie_A/xacro/head/joint_names.xacro (robot description, xacro)
@@ -1,6 +1,6 @@
 <?xml version="1.0" ?>
 <robot xmlns:xacro="http://www.ros.org/wiki/xacro" name="v1/head/joint_names">
-  <xacro:property name="NJ1_Joint_Name" value="LowerNeckExtensor" />
-  <xacro:property name="NJ2_Joint_Name" value="NeckRotator" />
-  <xacro:property name="NJ3_Joint_Name" value="UpperNeckExtensor" />
+  <xacro:property name="NJ1_Joint_Name" value="LowerNeckPitch" />
+  <xacro:property name="NJ2_Joint_Name" value="NeckYaw" />
+  <xacro:property name="NJ3_Joint_Name" value="UpperNeckPitch" />
 </robot>

File: valkyrie_description/robots/valkyrie_A/xacro/head/link_names.xacro (robot description, xacro)
@@ -2,8 +2,8 @@
 <robot xmlns:xacro="http://www.ros.org/wiki/xacro" name="v1/head/link_names">
   <xacro:property name="NJ1_Proximal_Link" value="${head_root_link}" />
-  <xacro:property name="NJ1_Distal_Link" value="/v1/LowerNeckExtensor" />
-  <xacro:property name="NJ2_Proximal_Link" value="/v1/LowerNeckExtensor" />
-  <xacro:property name="NJ2_Distal_Link" value="/v1/NeckRotator" />
-  <xacro:property name="NJ3_Proximal_Link" value="/v1/NeckRotator" />
-  <xacro:property name="NJ3_Distal_Link" value="/v1/Head" />
+  <xacro:property name="NJ1_Distal_Link" value="LowerNeckPitch" />
+  <xacro:property name="NJ2_Proximal_Link" value="LowerNeckPitch" />
+  <xacro:property name="NJ2_Distal_Link" value="NeckYaw" />
+  <xacro:property name="NJ3_Proximal_Link" value="NeckYaw" />
+  <xacro:property name="NJ3_Distal_Link" value="Head" />
 </robot>

File: valkyrie_description/robots/valkyrie_A/xacro/leg/joint_names.xacro (robot description, xacro)
@@ -1,9 +1,9 @@
 <?xml version="1.0" ?>
 <robot xmlns:xacro="http://www.ros.org/wiki/xacro" name="v1/leg/joint_names">
-  <xacro:property name="LJ1_Joint_Name" value="${prefix}HipRotator" />
-  <xacro:property name="LJ2_Joint_Name" value="${prefix}HipAdductor" />
-  <xacro:property name="LJ3_Joint_Name" value="${prefix}HipExtensor" />
-  <xacro:property name="LJ4_Joint_Name" value="${prefix}KneeExtensor" />
-  <xacro:property name="LJ5_Joint_Name" value="${prefix}AnkleExtensor" />
-  <xacro:property name="LJ6_Joint_Name" value="${prefix}Ankle" />
+  <xacro:property name="LJ1_Joint_Name" value="${prefix}HipYaw" />
+  <xacro:property name="LJ2_Joint_Name" value="${prefix}HipRoll" />
+  <xacro:property name="LJ3_Joint_Name" value="${prefix}HipPitch" />
+  <xacro:property name="LJ4_Joint_Name" value="${prefix}KneePitch" />
+  <xacro:property name="LJ5_Joint_Name" value="${prefix}AnklePitch" />
+  <xacro:property name="LJ6_Joint_Name" value="${prefix}AnkleRoll" />
 </robot>

File: valkyrie_description/robots/valkyrie_A/xacro/leg/link_names.xacro (robot description, xacro)
@@ -2,16 +2,16 @@
 <robot xmlns:xacro="http://www.ros.org/wiki/xacro" name="v1/leg/link_names">
   <xacro:property name="LJ1_Proximal_Link" value="${leg_root_link}" />
-  <xacro:property name="LJ1_Distal_Link" value="/v1/${prefix}HipRotator" />
-  <xacro:property name="LJ2_Proximal_Link" value="/v1/${prefix}HipRotator" />
-  <xacro:property name="LJ2_Distal_Link" value="/v1/${prefix}HipAdductor" />
-  <xacro:property name="LJ3_Proximal_Link" value="/v1/${prefix}HipAdductor" />
-  <xacro:property name="LJ3_Distal_Link" value="/v1/${prefix}Leg" />
-  <xacro:property name="LJ4_Proximal_Link" value="/v1/${prefix}Leg" />
-  <xacro:property name="LJ4_Distal_Link_Box" value="/v1/${prefix}ShankStructure" />
-  <xacro:property name="LJ4_Distal_Link_Cylinder1" value="/v1/${prefix}MedialAnkleActuator" />
-  <xacro:property name="LJ4_Distal_Link_Cylinder2" value="/v1/${prefix}LateralAnkleActuator" />
-  <xacro:property name="LJ5_Proximal_Link" value="/v1/${prefix}ShankStructure" />
-  <xacro:property name="LJ5_Distal_Link" value="/v1/${prefix}AnkleYoke" />
-  <xacro:property name="LJ6_Proximal_Link" value="/v1/${prefix}AnkleYoke" />
-  <xacro:property name="LJ6_Distal_Link" value="/v1/${prefix}UpperFoot" />
+  <xacro:property name="LJ1_Distal_Link" value="${prefix}HipYaw" />
+  <xacro:property name="LJ2_Proximal_Link" value="${prefix}HipYaw" />
+  <xacro:property name="LJ2_Distal_Link" value="${prefix}HipRoll" />
+  <xacro:property name="LJ3_Proximal_Link" value="${prefix}HipRoll" />
+  <xacro:property name="LJ3_Distal_Link" value="${prefix}HipPitch" />
+  <xacro:property name="LJ4_Proximal_Link" value="${prefix}HipPitch" />
+  <xacro:property name="LJ4_Distal_Link_Box" value="${prefix}KneePitch" />
+  <xacro:property name="LJ4_Distal_Link_Cylinder1" value="${prefix}MedialAnkleActuator" />
+  <xacro:property name="LJ4_Distal_Link_Cylinder2" value="${prefix}LateralAnkleActuator" />
+  <xacro:property name="LJ5_Proximal_Link" value="${prefix}KneePitch" />
+  <xacro:property name="LJ5_Distal_Link" value="${prefix}AnkleRoll" />
+  <xacro:property name="LJ6_Proximal_Link" value="${prefix}AnkleRoll" />
+  <xacro:property name="LJ6_Distal_Link" value="${prefix}Foot" />
 </robot>

File: valkyrie_description/robots/valkyrie_A/xacro/little_finger/joint_names.xacro (robot description, xacro)
@@ -1,7 +1,7 @@
 <?xml version="1.0" ?>
 <robot xmlns:xacro="http://www.ros.org/wiki/xacro" name="v1/little_finger/mass_parameters">
-  <xacro:property name="LFJ1_Joint_Name" value="${prefix}LittleMPYaw" />
-  <xacro:property name="LFJ2_Joint_Name" value="${prefix}LittleMPExtensor" />
-  <xacro:property name="LFJ3_Joint_Name" value="${prefix}LittlePIPExtensor" />
-  <xacro:property name="LFJ4_Joint_Name" value="${prefix}LittleDIPExtensor" />
+  <xacro:property name="LFJ1_Joint_Name" value="${prefix}PinkyPitch1" />
+  <xacro:property name="LFJ2_Joint_Name" value="${prefix}PinkyPitch2" />
+  <xacro:property name="LFJ3_Joint_Name" value="${prefix}PinkyPitch3" />
+  <xacro:property name="LFJ4_Joint_Name" value="${prefix}PinkyPitch4" />
 </robot>

File: valkyrie_description/robots/valkyrie_A/xacro/little_finger/link_names.xacro (robot description, xacro)
@@ -2,10 +2,10 @@
 <robot xmlns:xacro="http://www.ros.org/wiki/xacro" name="v1/little_finger/dh_parameters">
   <xacro:property name="LFJ1_Proximal_Link" value="${little_finger_root_link}" />
-  <xacro:property name="LFJ1_Distal_Link" value="/v1/${prefix}MedialMetacarpal" />
-  <xacro:property name="LFJ2_Proximal_Link" value="/v1/${prefix}MedialMetacarpal" />
-  <xacro:property name="LFJ2_Distal_Link" value="/v1/${prefix}LittleProximalPhalanx" />
-  <xacro:property name="LFJ3_Proximal_Link" value="/v1/${prefix}LittleProximalPhalanx" />
-  <xacro:property name="LFJ3_Distal_Link" value="/v1/${prefix}LittleMedialPhalanx" />
-  <xacro:property name="LFJ4_Proximal_Link" value="/v1/${prefix}LittleMedialPhalanx" />
-  <xacro:property name="LFJ4_Distal_Link" value="/v1/${prefix}LittleDistalPhalanx" />
+  <xacro:property name="LFJ1_Distal_Link" value="/v1/${prefix}PinkyPitch1" />
+  <xacro:property name="LFJ2_Proximal_Link" value="/v1/${prefix}PinkyPitch1" />
+  <xacro:property name="LFJ2_Distal_Link" value="/v1/${prefix}PinkyPitch2" />
+  <xacro:property name="LFJ3_Proximal_Link" value="/v1/${prefix}PinkyPitch2" />
+  <xacro:property name="LFJ3_Distal_Link" value="/v1/${prefix}PinkyPitch3" />
+  <xacro:property name="LFJ4_Proximal_Link" value="/v1/${prefix}PinkyPitch4" />
+  <xacro:property name="LFJ4_Distal_Link" value="/v1/${prefix}PinkyPitch5" />
 </robot>

File: valkyrie_description/robots/valkyrie_A/xacro/little_finger/little_finger.xacro (robot description, xacro)
@@ -26,10 +26,4 @@
   <xacro:property name="LFJ3_Link_Origin_Y" value="0"/>
   <xacro:property name="LFJ3_Link_Origin_Z" value="0"/>
-  <xacro:property name="LFJ4_Link_Width" value="0.027"/>
-  <xacro:property name="LFJ4_Link_Height" value="0.012"/>
-  <xacro:property name="LFJ4_Link_Length" value="0.019"/>
-  <xacro:property name="LFJ4_Link_Origin_X" value="0.0086"/>
-  <xacro:property name="LFJ4_Link_Origin_Y" value="0"/>
-  <xacro:property name="LFJ4_Link_Origin_Z" value="0"/>
   <xacro:macro name="make_little_finger" params="prefix reflect little_finger_root_link">
     <!-- LINKS -->
@@ -83,11 +77,4 @@
         <limit effort="${LFJ3_Torque_Limit}" lower="${LFJ3_Lower_Limit}" upper="${LFJ3_Upper_Limit}" velocity="${LFJ3_Speed_Limit}"/>
     </xacro:revolute_joint>
-    <!-- LFJ4 -->
-    <xacro:revolute_joint jointName="${LFJ4_Joint_Name}"
-                          parent="${LFJ4_Proximal_Link}" child="${LFJ4_Distal_Link}"
-                          origin_xyz="${LFJ4_Origin_X} ${LFJ4_Origin_Y} ${LFJ4_Origin_Z}"
-                          origin_rpy="${LFJ4_Orientation_Roll} ${LFJ4_Orientation_Pitch} ${LFJ4_Orientation_Yaw}">
-        <limit effort="${LFJ4_Torque_Limit}" lower="${LFJ4_Lower_Limit}" upper="${LFJ4_Upper_Limit}" velocity="${LFJ4_Speed_Limit}"/>
-    </xacro:revolute_joint>
   </xacro:macro>
   <xacro:macro name="make_little_finger_fixed" params="prefix reflect little_finger_root_link">
@@ -114,11 +101,4 @@
                     material="Gold"
                     collision_mesh="${mesh_root}/sf2_ssf3.stl"/>
-    <xacro:box_link name="${LFJ4_Distal_Link}"
-                    width="${LFJ4_Link_Width}" height="${LFJ4_Link_Height}" depth="${LFJ4_Link_Length}" mass="${LFJ4_Link_Mass}"
-                    origin_rpy="0 0 0"
-                    origin_xyz="${LFJ4_Link_Origin_X} ${LFJ4_Link_Origin_Y} ${LFJ4_Link_Origin_Z}"
-                    visual_mesh="${mesh_root}/sf3_ssf4.stl"
-                    material="Gold"
-                    collision_mesh="${mesh_root}/sf3_ssf4.stl"/>
     <!-- LFJ1 -->
     <xacro:fixed_joint jointName="${LFJ1_Joint_Name}"
@@ -136,9 +116,4 @@
                           origin_xyz="${LFJ3_Origin_X} ${LFJ3_Origin_Y} ${LFJ3_Origin_Z}"
                           origin_rpy="${LFJ3_Orientation_Roll} ${LFJ3_Orientation_Pitch} ${LFJ3_Orientation_Yaw}"/>
-    <!-- LFJ4 -->
-    <xacro:fixed_joint jointName="${LFJ4_Joint_Name}"
-                          parent="${LFJ4_Proximal_Link}" child="${LFJ4_Distal_Link}"
-                          origin_xyz="${LFJ4_Origin_X} ${LFJ4_Origin_Y} ${LFJ4_Origin_Z}"
-                          origin_rpy="${LFJ4_Orientation_Roll} ${LFJ4_Orientation_Pitch} ${LFJ4_Orientation_Yaw}"/>
   </xacro:macro>
   <!-- Actuators -->
@@ -155,5 +130,4 @@
                                 joint2="${LFJ2_Joint_Name}"
                                 joint3="${LFJ3_Joint_Name}"
-                                joint4="${LFJ4_Joint_Name}"
                                 actuator="${RLFA_Actuator_Name}" />
   </xacro:macro>
@@ -163,5 +137,4 @@
                                 joint2="${LFJ2_Joint_Name}"
                                 joint3="${LFJ3_Joint_Name}"
-                                joint4="${LFJ4_Joint_Name}"
                                 actuator="${LLFA_Actuator_Name}" />
   </xacro:macro>

File: valkyrie_description/robots/valkyrie_A/xacro/pelvis/pelvis.xacro (robot description, xacro)
@@ -1,4 +1,4 @@
-<robot xmlns:xacro="http://ros.org/wiki/xacro" name="v1/Pelvis">
-    <xacro:property name="Pelvis_Link_Name" value="/v1/Pelvis" />
+<robot xmlns:xacro="http://ros.org/wiki/xacro" name="Pelvis">
+    <xacro:property name="Pelvis_Link_Name" value="Pelvis" />
     <xacro:macro name="make_pelvis">
         <xacro:box_link name="${Pelvis_Link_Name}"

File: valkyrie_description/robots/valkyrie_A/xacro/waist/joint_names.xacro (robot description, xacro)
@@ -1,6 +1,6 @@
 <?xml version="1.0" ?>
 <robot xmlns:xacro="http://www.ros.org/wiki/xacro" name="v1/waist/mass_parameters">
-  <xacro:property name="WJ1_Joint_Name" value="WaistRotator" />
-  <xacro:property name="WJ2_Joint_Name" value="WaistExtensor" />
-  <xacro:property name="WJ3_Joint_Name" value="WaistLateralExtensor" />
+  <xacro:property name="WJ1_Joint_Name" value="TorsoYaw" />
+  <xacro:property name="WJ2_Joint_Name" value="TorsoPitch" />
+  <xacro:property name="WJ3_Joint_Name" value="TorsoRoll" />
 </robot>

File: valkyrie_description/robots/valkyrie_A/xacro/waist/link_names.xacro (robot description, xacro)
@@ -2,8 +2,8 @@
 <robot xmlns:xacro="http://www.ros.org/wiki/xacro" name="v1/waist/dh_parameters">
   <xacro:property name="WJ1_Proximal_Link" value="${waist_root_link}" />
-  <xacro:property name="WJ1_Distal_Link" value="/v1/WaistRotator" />
-  <xacro:property name="WJ2_Proximal_Link" value="/v1/WaistRotator" />
-  <xacro:property name="WJ2_Distal_Link" value="/v1/WaistExtensor" />
-  <xacro:property name="WJ3_Proximal_Link" value="/v1/WaistExtensor" />
-  <xacro:property name="WJ3_Distal_Link" value="/v1/Trunk" />
+  <xacro:property name="WJ1_Distal_Link" value="TorsoYaw" />
+  <xacro:property name="WJ2_Proximal_Link" value="TorsoYaw" />
+  <xacro:property name="WJ2_Distal_Link" value="TorsoPitch" />
+  <xacro:property name="WJ3_Proximal_Link" value="TorsoPitch" />
+  <xacro:property name="WJ3_Distal_Link" value="TorsoRoll" />
 </robot>
