Commit message: Removed head sensors from urdf.

File: valkyrie_description/robots/valkyrie_A/V1.urdf (robot description, URDF)
Before this commit: robot V1, 94 links, 93 joints
Links:
- removed link /v1/EnsensoIR_Frame
- removed link /v1/Ensenso_Frame
- removed link /v1/HeadCamBoardIR_Frame
- removed link /v1/HeadCamBoard_Frame
- removed link /v1/HeadIMU_Frame
- removed link /v1/HeadWebcam_Frame
- removed link /v1/Ibeo_Frame
Joints:
- removed joint /v1/EnsensoIR_Offset
- removed joint /v1/Ensenso_Offset
- removed joint /v1/HeadCamBoardIR_Offset
- removed joint /v1/HeadCamBoard_Offset
- removed joint /v1/HeadIMU_Offset
- removed joint /v1/HeadWebcam_Offset
- removed joint /v1/Ibeo_Offset

File: valkyrie_description/robots/valkyrie_A/xacro/utility/utility.xacro (robot description, xacro)
@@ -10,5 +10,5 @@
     <xacro:v1_head_transmissions actuator1="${name1}" actuator2="${name2}" actuator3="${name3}" />
     <xacro:v1_head_modes actuator1="${name1}" actuator2="${name2}" actuator3="${name3}" />
-    <xacro:v1_head_sensors/>
+    <!-- <xacro:v1_head_sensors/> @TODO: Updated head sensors and add this back in. Head sensors are in head.xacro. -->
   </xacro:macro>
   <xacro:macro name="make_arm_interface" params="prefix name1 type1 name2 type2 name3 type3 name4 type4 name5 type5 name6 type6 name7 type7">

Commit message: Removed leg hokoyuo from xacro's and urdf since they are not in the robot anymore.

File: valkyrie_description/robots/valkyrie_A/V1.urdf (robot description, URDF)
Before this commit: robot V1, 87 links, 86 joints
Links:
- removed link /v1/LeftLegHokuyo_Frame
- removed link /v1/RightLegHokuyo_Frame
Joints:
- removed joint /v1/LeftLegHokuyo_Offset
- removed joint /v1/RightLegHokuyo_Offset

File: valkyrie_description/robots/valkyrie_A/xacro/leg/leg.xacro (robot description, xacro)
@@ -319,8 +319,9 @@
   <!-- Sensors -->
   <xacro:macro name="v1_leg_sensors" params="prefix reflect">
-    <xacro:hokuyo_sensor sensorName="/v1/${prefix}LegHokuyo"
+    <!-- HOKUYO IS NOT IN THE ROBOT ANYMORE -->
+    <!-- <xacro:hokuyo_sensor sensorName="/v1/${prefix}LegHokuyo"
                          parentLink="${LJ3_Distal_Link}"
                          origin_xyz="0.350849 -0.098349 ${reflect * -0.036021}"
-                         origin_rpy="${pi_2} 0 -0.38394"/>
+                         origin_rpy="${pi_2} 0 -0.38394"/> -->
     <xacro:camboard_sensor sensorName="/v1/${prefix}LegCamBoard"
                        parentLink="${LJ4_Distal_Link_Box}"

Commit message: More neck renaming. I think everything with the neck is now rename.

File: valkyrie_description/robots/valkyrie_A/V1.urdf (robot description, URDF)
Before this commit: robot valkyrie, 61 links, 60 joints
Joints:
- joint LowerNeckPitch: limit lower=-1.5707963259 upper=0 effort=26 velocity=5 -> lower=-1.57 upper=0 effort=26 velocity=5
- joint NeckYaw: limit lower=-1.5707963259 upper=1.5707963259 effort=26 velocity=5 -> lower=-1.57 upper=1.57 effort=26 velocity=5
- joint UpperNeckPitch: limit lower=-0.08726646255 upper=0.78539816295 effort=26 velocity=5 -> lower=-0.087 upper=0.785 effort=26 velocity=5

File: valkyrie_description/robots/valkyrie_A/xacro/head/head.xacro (robot description, xacro)
@@ -39,5 +39,5 @@
                           origin_rpy="${LowerNeckPitchFrameOrientation_Roll} ${LowerNeckPitchFrameOrientation_Roll} ${LowerNeckPitchFrameOrientation_Yaw}"
                           damping="1.0" friction="0.0">
-      <limit effort="${NJ1_Torque_Limit}" lower="${NJ1_Lower_Limit}" upper="${NJ1_Upper_Limit}" velocity="${NJ1_Speed_Limit}"/>
+      <limit effort="${LowerNeckPitchTorqueLimit}" lower="${LowerNeckPitchPositionLimit_Lower}" upper="${LowerNeckPitchPositionLimit_Upper}" velocity="${LowerNeckPitchVelocityLimit}"/>
       <controller_gains Kp="20000" Kd="0"/>
     </xacro:revolute_joint_ex>
@@ -48,5 +48,5 @@
                           origin_rpy="${NeckYawFrameOrientation_Roll} ${NeckYawFrameOrientation_Pitch} ${NeckYawFrameOrientation_Yaw}"
                           damping="1.0" friction="0.0">
-      <limit effort="${NJ2_Torque_Limit}" lower="${NJ2_Lower_Limit}" upper="${NJ2_Upper_Limit}" velocity="${NJ2_Speed_Limit}"/>
+      <limit effort="${NeckYawTorqueLimit}" lower="${NeckYawPositionLimit_Lower}" upper="${NeckYawPositionLimit_Upper}" velocity="${NeckYawVelocityLimit}"/>
       <controller_gains Kp="20000" Kd="0"/>
     </xacro:revolute_joint_ex>
@@ -57,5 +57,5 @@
                           origin_rpy="${UpperNeckPitchFrameOrientation_Roll} ${UpperNeckPitchFrameOrientation_Pitch} ${UpperNeckPitchFrameOrientation_Yaw}"
                           damping="1.0" friction="0.0">
-      <limit effort="${NJ3_Torque_Limit}" lower="${NJ3_Lower_Limit}" upper="${NJ3_Upper_Limit}" velocity="${NJ3_Speed_Limit}"/>
+      <limit effort="${UpperNeckPitchTorqueLimit}" lower="${UpperNeckPitchPositionLimit_Lower}" upper="${UpperNeckPitchPositionLimit_Upper}" velocity="${UpperNeckPitchVelocityLimit}"/>
       <controller_gains Kp="20000" Kd="0"/>
     </xacro:revolute_joint_ex>
@@ -82,5 +82,5 @@
                           origin_xyz="${LowerNeckPitchFrameOrigin_X} ${LowerNeckPitchFrameOrigin_Y} ${LowerNeckPitchFrameOrigin_Z}"
                           origin_rpy="${LowerNeckPitchFrameOrientation_Roll} ${LowerNeckPitchFrameOrientation_Roll} ${LowerNeckPitchFrameOrientation_Yaw}">
-      <limit effort="${NJ1_Torque_Limit}" lower="${NJ1_Lower_Limit}" upper="${NJ1_Upper_Limit}" velocity="${NJ1_Speed_Limit}"/>
+      <limit effort="${LowerNeckPitchTorqueLimit}" lower="${LowerNeckPitchPositionLimit_Lower}" upper="${LowerNeckPitchPositionLimit_Upper}" velocity="${LowerNeckPitchVelocityLimit}"/>
     </xacro:fixed_joint>
     <!-- NJ2 -->
@@ -89,5 +89,5 @@
                           origin_xyz="${NeckYawFrameOrigin_X} ${NeckYawFrameOrigin_Y} ${NeckYawFrameOrigin_Z}"
                           origin_rpy="${NeckYawFrameOrientation_Roll} ${NeckYawFrameOrientation_Pitch} ${NeckYawFrameOrientation_Yaw}">
-      <limit effort="${NJ2_Torque_Limit}" lower="${NJ2_Lower_Limit}" upper="${NJ2_Upper_Limit}" velocity="${NJ2_Speed_Limit}"/>
+      <limit effort="${NeckYawTorqueLimit}" lower="${NeckYawPositionLimit_Lower}" upper="${NeckYawPositionLimit_Upper}" velocity="${NeckYawVelocityLimit}"/>
     </xacro:fixed_joint>
     <!-- NJ3 -->
@@ -96,5 +96,5 @@
                           origin_xyz="${UpperNeckPitchFrameOrigin_X} ${UpperNeckPitchFrameOrigin_Y} ${UpperNeckPitchFrameOrigin_Z}"
                           origin_rpy="${UpperNeckPitchFrameOrientation_Roll} ${UpperNeckPitchFrameOrientation_Pitch} ${UpperNeckPitchFrameOrientation_Yaw}">
-      <limit effort="${NJ3_Torque_Limit}" lower="${NJ3_Lower_Limit}" upper="${NJ3_Upper_Limit}" velocity="${NJ3_Speed_Limit}"/>
+      <limit effort="${UpperNeckPitchTorqueLimit}" lower="${UpperNeckPitchPositionLimit_Lower}" upper="${UpperNeckPitchPositionLimit_Upper}" velocity="${UpperNeckPitchVelocityLimit}"/>
     </xacro:fixed_joint>
   </xacro:macro>

File: valkyrie_description/robots/valkyrie_A/xacro/head/joint_limits.xacro (robot description, xacro)
@@ -1,15 +1,15 @@
 <?xml version="1.0" ?>
 <robot xmlns:xacro="http://www.ros.org/wiki/xacro" name="v1/head/joint_limits">
-  <xacro:property name="NJ1_Torque_Limit" value="26" />
-  <xacro:property name="NJ2_Torque_Limit" value="26" />
-  <xacro:property name="NJ3_Torque_Limit" value="26" />
-  <xacro:property name="NJ1_Lower_Limit" value="${-90 * DEG2RAD}" />
-  <xacro:property name="NJ2_Lower_Limit" value="${-90 * DEG2RAD}" />
-  <xacro:property name="NJ3_Lower_Limit" value="${-5 * DEG2RAD}" />
-  <xacro:property name="NJ1_Upper_Limit" value="0" />
-  <xacro:property name="NJ2_Upper_Limit" value="${90 * DEG2RAD}" />
-  <xacro:property name="NJ3_Upper_Limit" value="${45 * DEG2RAD}" />
-  <xacro:property name="NJ1_Speed_Limit" value="5" />
-  <xacro:property name="NJ2_Speed_Limit" value="5" />
-  <xacro:property name="NJ3_Speed_Limit" value="5" />
+  <xacro:property name="LowerNeckPitchTorqueLimit" value="26" />
+  <xacro:property name="NeckYawTorqueLimit" value="26" />
+  <xacro:property name="UpperNeckPitchTorqueLimit" value="26" />
+  <xacro:property name="LowerNeckPitchPositionLimit_Lower" value="-1.57" />
+  <xacro:property name="NeckYawPositionLimit_Lower" value="-1.57" />
+  <xacro:property name="UpperNeckPitchPositionLimit_Lower" value="-0.087" />
+  <xacro:property name="LowerNeckPitchPositionLimit_Upper" value="0" />
+  <xacro:property name="NeckYawPositionLimit_Upper" value="1.57" />
+  <xacro:property name="UpperNeckPitchPositionLimit_Upper" value="0.785" />
+  <xacro:property name="LowerNeckPitchVelocityLimit" value="5" />
+  <xacro:property name="NeckYawVelocityLimit" value="5" />
+  <xacro:property name="UpperNeckPitchVelocityLimit" value="5" />
 </robot>
