Commit message: Renamed position and orientation parameters for neck frames.

File: valkyrie_description/robots/valkyrie_A/xacro/arm/actuator_names.xacro (robot description, xacro)
@@ -1,9 +1,9 @@
 <?xml version="1.0" ?>
 <robot xmlns:xacro="http://www.ros.org/wiki/xacro" name="v1/arm/joint_names">
-  <xacro:property name="AJ1_Actuator_Name" value="/Trunk/${prefix}ArmActuator" />
-  <xacro:property name="AJ2_Actuator_Name" value="/${prefix}Arm/Actuator2" />
-  <xacro:property name="AJ3_Actuator_Name" value="/${prefix}Arm/Actuator3" />
-  <xacro:property name="AJ4_Actuator_Name" value="/${prefix}Arm/Actuator4" />
-  <xacro:property name="AJ5_Actuator_Name" value="/${prefix}Arm/Actuator5" />
+  <xacro:property name="ShoulderPitchActuatorName" value="/Trunk/${prefix}ArmActuator" />
+  <xacro:property name="ShoulderRollActuatorName" value="/${prefix}Arm/Actuator2" />
+  <xacro:property name="ShoulderYawActuatorName" value="/${prefix}Arm/Actuator3" />
+  <xacro:property name="ElbowPitchActuatorName" value="/${prefix}Arm/Actuator4" />
+  <xacro:property name="ForearmYawActuatorName" value="/${prefix}Arm/Actuator5" />
   <xacro:property name="RAJ6_Actuator_Name" value="/RightArm/ForearmDriver1/RightWristActuator" />
   <xacro:property name="RAJ7_Actuator_Name" value="/RightArm/ForearmDriver1/LeftWristActuator" />

File: valkyrie_description/robots/valkyrie_A/xacro/arm/arm.xacro (robot description, xacro)
@@ -58,5 +58,5 @@
     <xacro:revolute_joint_ex jointName="${AJ1_Joint_Name}"
                           parent="${upper_arm_root_link}" child="${AJ1_Distal_Link}"
-                          origin_xyz="${AJ1_Origin_X} ${AJ1_Origin_Y} ${AJ1_Origin_Z}"
+                          origin_xyz="${ArmPitchFrameOrigin_X} ${AJ1_Origin_Y} ${AJ1_Origin_Z}"
                           origin_rpy="${AJ1_Orientation_Roll} ${AJ1_Orientation_Pitch} ${AJ1_Orientation_Yaw}"
                           damping="1.0" friction="0.0">

File: valkyrie_description/robots/valkyrie_A/xacro/arm/dh_parameters.xacro (robot description, xacro)
@@ -1,9 +1,5 @@
 <?xml version="1.0" ?>
 <robot xmlns:xacro="http://www.ros.org/wiki/xacro" name="v1/arm/dh_parameters">
-  <xacro:property name="AJ1_Joint_Offset" value="-0.03157" />
-  <xacro:property name="AJ1_Joint_Angle" value="0" />
-  <xacro:property name="AJ1_Joint_Radius" value="0.29842" />
-  <xacro:property name="AJ1_Joint_Twist" value="${pi_2}" />
-  <xacro:property name="AJ1_Origin_X" value="0.29842"/>
+  <xacro:property name="ArmPitchFrameOrigin_X" value="0.29842"/>
   <xacro:property name="AJ1_Origin_Y" value="0"/>
   <xacro:property name="AJ1_Origin_Z" value="-0.03157"/>
@@ -11,8 +7,4 @@
   <xacro:property name="AJ1_Orientation_Pitch" value="0"/>
   <xacro:property name="AJ1_Orientation_Yaw" value="0"/>
-  <xacro:property name="AJ2_Joint_Offset" value="${reflect * -0.246}" />
-  <xacro:property name="AJ2_Joint_Angle" value="${pi}" />
-  <xacro:property name="AJ2_Joint_Radius" value="0" />
-  <xacro:property name="AJ2_Joint_Twist" value="${reflect * (pi_2)}" />
   <xacro:property name="AJ2_Origin_X" value="0"/>
   <xacro:property name="AJ2_Origin_Y" value="0"/>
@@ -21,8 +13,4 @@
   <xacro:property name="AJ2_Orientation_Pitch" value="0"/>
   <xacro:property name="AJ2_Orientation_Yaw" value="${pi}"/>
-  <xacro:property name="AJ3_Joint_Offset" value="0" />
-  <xacro:property name="AJ3_Joint_Angle" value="${reflect * pi_2}" />
-  <xacro:property name="AJ3_Joint_Radius" value="0" />
-  <xacro:property name="AJ3_Joint_Twist" value="${-1 * pi_2}" />
   <xacro:property name="AJ3_Origin_X" value="0"/>
   <xacro:property name="AJ3_Origin_Y" value="0"/>
@@ -31,8 +19,4 @@
   <xacro:property name="AJ3_Orientation_Pitch" value="0"/>
   <xacro:property name="AJ3_Orientation_Yaw" value="${reflect * pi_2}"/>
-  <xacro:property name="AJ4_Joint_Offset" value="${reflect * -0.330}" />
-  <xacro:property name="AJ4_Joint_Angle" value="${reflect * pi_2}" />
-  <xacro:property name="AJ4_Joint_Radius" value="-0.0254" />
-  <xacro:property name="AJ4_Joint_Twist" value="${reflect * pi_2}" />
   <xacro:property name="AJ4_Origin_X" value="0"/>
   <xacro:property name="AJ4_Origin_Y" value="${reflect * -0.0254}"/>
@@ -41,8 +25,4 @@
   <xacro:property name="AJ4_Orientation_Pitch" value="0"/>
   <xacro:property name="AJ4_Orientation_Yaw" value="${reflect * pi_2}"/>
-  <xacro:property name="AJ5_Joint_Offset" value="0" />
-  <xacro:property name="AJ5_Joint_Angle" value="${pi}" />
-  <xacro:property name="AJ5_Joint_Radius" value="-0.0254" />
-  <xacro:property name="AJ5_Joint_Twist" value="${reflect * pi_2}" />
   <xacro:property name="AJ5_Origin_X" value="0.0254"/>
   <xacro:property name="AJ5_Origin_Y" value="0"/>
@@ -51,8 +31,4 @@
   <xacro:property name="AJ5_Orientation_Pitch" value="0"/>
   <xacro:property name="AJ5_Orientation_Yaw" value="${pi}"/>
-  <xacro:property name="AJ6_Joint_Offset" value="${reflect * -0.287}" />
-  <xacro:property name="AJ6_Joint_Angle" value="${reflect * pi_2}" />
-  <xacro:property name="AJ6_Joint_Radius" value="0" />
-  <xacro:property name="AJ6_Joint_Twist" value="${reflect * -1 * pi_2}" />
   <xacro:property name="AJ6_Origin_X" value="0"/>
   <xacro:property name="AJ6_Origin_Y" value="0"/>
@@ -61,8 +37,4 @@
   <xacro:property name="AJ6_Orientation_Pitch" value="0"/>
   <xacro:property name="AJ6_Orientation_Yaw" value="${reflect * pi_2}"/>
-  <xacro:property name="AJ7_Joint_Offset" value="0" />
-  <xacro:property name="AJ7_Joint_Angle" value="${reflect * pi_2}" />
-  <xacro:property name="AJ7_Joint_Radius" value="0" />
-  <xacro:property name="AJ7_Joint_Twist" value="${reflect * pi_2}" />
   <xacro:property name="AJ7_Origin_X" value="0"/>
   <xacro:property name="AJ7_Origin_Y" value="0"/>

File: valkyrie_description/robots/valkyrie_A/xacro/head/dh_parameters.xacro (robot description, xacro)
@@ -1,21 +1,21 @@
 <?xml version="1.0" ?>
 <robot xmlns:xacro="http://www.ros.org/wiki/xacro" name="v1/head/dh_parameters">
-  <xacro:property name="LowerNeckPitchOrigin_X" value="0.3383"/>
-  <xacro:property name="LowerNeckPitchOrigin_Y" value="0"/>
-  <xacro:property name="LowerNeckPitchOrigin_Z" value="0.0519"/>
-  <xacro:property name="LowerNeckPitchFrame_Roll" value="0.0"/>
-  <xacro:property name="LowerNeckPitchFrame_Pitch" value="0.0"/>
-  <xacro:property name="LowerNeckPitchFrame_Yaw" value="0.0"/>
-  <xacro:property name="NeckYawOrigin_X" value="0"/>
-  <xacro:property name="NJ2_Origin_Y" value="0.0519"/>
-  <xacro:property name="NJ2_Origin_Z" value="0"/>
-  <xacro:property name="NJ2_Orientation_Roll" value="0.0"/>
-  <xacro:property name="NJ2_Orientation_Pitch" value="0.0"/>
-  <xacro:property name="NJ2_Orientation_Yaw" value="0.0"/>
-  <xacro:property name="NJ3_Origin_X" value="0.06"/>
-  <xacro:property name="NJ3_Origin_Y" value="0"/>
-  <xacro:property name="NJ3_Origin_Z" value="0.196"/>
-  <xacro:property name="NJ3_Orientation_Roll" value="0.0"/>
-  <xacro:property name="NJ3_Orientation_Pitch" value="0.0"/>
-  <xacro:property name="NJ3_Orientation_Yaw" value="0.0"/>
+  <xacro:property name="LowerNeckPitchFrameOrigin_X" value="0.3383"/>
+  <xacro:property name="LowerNeckPitchFrameOrigin_Y" value="0"/>
+  <xacro:property name="LowerNeckPitchFrameOrigin_Z" value="0.0519"/>
+  <xacro:property name="LowerNeckPitchFrameOrientation_Roll" value="0.0"/>
+  <xacro:property name="LowerNeckPitchFrameOrientation_Pitch" value="0.0"/>
+  <xacro:property name="LowerNeckPitchFrameOrientation_Yaw" value="0.0"/>
+  <xacro:property name="NeckYawFrameOrigin_X" value="0"/>
+  <xacro:property name="NeckYawFrameOrigin_Y" value="0.0519"/>
+  <xacro:property name="NeckYawFrameOrigin_Z" value="0"/>
+  <xacro:property name="NeckYawFrameOrientation_Roll" value="0.0"/>
+  <xacro:property name="NeckYawFrameOrientation_Pitch" value="0.0"/>
+  <xacro:property name="NeckYawFrameOrientation_Yaw" value="0.0"/>
+  <xacro:property name="UpperNeckPitchFrameOrigin_X" value="0.06"/>
+  <xacro:property name="UpperNeckPitchFrameOrigin_Y" value="0"/>
+  <xacro:property name="UpperNeckPitchFrameOrigin_Z" value="0.196"/>
+  <xacro:property name="UpperNeckPitchFrameOrientation_Roll" value="0.0"/>
+  <xacro:property name="UpperNeckPitchFrameOrientation_Pitch" value="0.0"/>
+  <xacro:property name="UpperNeckPitchFrameOrientation_Yaw" value="0.0"/>
 </robot>

File: valkyrie_description/robots/valkyrie_A/xacro/head/head.xacro (robot description, xacro)
@@ -36,6 +36,6 @@
     <xacro:revolute_joint_ex jointName="${LowerNeckPitchJointName}"
                           parent="${LowerNeckPitchParentLink}" child="${LowerNeckPitchLinkName}"
-                          origin_xyz="${LowerNeckPitchOrigin_X} ${LowerNeckPitchOrigin_Y} ${LowerNeckPitchOrigin_Z}"
-                          origin_rpy="${LowerNeckPitchFrame_Roll} ${LowerNeckPitchFrame_Roll} ${LowerNeckPitchFrame_Yaw}"
+                          origin_xyz="${LowerNeckPitchFrameOrigin_X} ${LowerNeckPitchFrameOrigin_Y} ${LowerNeckPitchFrameOrigin_Z}"
+                          origin_rpy="${LowerNeckPitchFrameOrientation_Roll} ${LowerNeckPitchFrameOrientation_Roll} ${LowerNeckPitchFrameOrientation_Yaw}"
                           damping="1.0" friction="0.0">
       <limit effort="${NJ1_Torque_Limit}" lower="${NJ1_Lower_Limit}" upper="${NJ1_Upper_Limit}" velocity="${NJ1_Speed_Limit}"/>
@@ -45,6 +45,6 @@
     <xacro:revolute_joint_ex jointName="${NeckYawJointName}"
                           parent="${LowerNeckPitchLinkName}" child="${NeckYawLinkName}"
-                          origin_xyz="${NeckYawOrigin_X} ${NJ2_Origin_Y} ${NJ2_Origin_Z}"
-                          origin_rpy="${NJ2_Orientation_Roll} ${NJ2_Orientation_Pitch} ${NJ2_Orientation_Yaw}"
+                          origin_xyz="${NeckYawFrameOrigin_X} ${NeckYawFrameOrigin_Y} ${NeckYawFrameOrigin_Z}"
+                          origin_rpy="${NeckYawFrameOrientation_Roll} ${NeckYawFrameOrientation_Pitch} ${NeckYawFrameOrientation_Yaw}"
                           damping="1.0" friction="0.0">
       <limit effort="${NJ2_Torque_Limit}" lower="${NJ2_Lower_Limit}" upper="${NJ2_Upper_Limit}" velocity="${NJ2_Speed_Limit}"/>
@@ -54,6 +54,6 @@
     <xacro:revolute_joint_ex jointName="${UpperNeckPitchJointName}"
                           parent="${NeckYawLinkName}" child="${UpperNeckPitchLinkName}"
-                          origin_xyz="${NJ3_Origin_X} ${NJ3_Origin_Y} ${NJ3_Origin_Z}"
-                          origin_rpy="${NJ3_Orientation_Roll} ${NJ3_Orientation_Pitch} ${NJ3_Orientation_Yaw}"
+                          origin_xyz="${UpperNeckPitchFrameOrigin_X} ${UpperNeckPitchFrameOrigin_Y} ${UpperNeckPitchFrameOrigin_Z}"
+                          origin_rpy="${UpperNeckPitchFrameOrientation_Roll} ${UpperNeckPitchFrameOrientation_Pitch} ${UpperNeckPitchFrameOrientation_Yaw}"
                           damping="1.0" friction="0.0">
       <limit effort="${NJ3_Torque_Limit}" lower="${NJ3_Lower_Limit}" upper="${NJ3_Upper_Limit}" velocity="${NJ3_Speed_Limit}"/>
@@ -80,6 +80,6 @@
     <xacro:fixed_joint jointName="${LowerNeckPitchJointName}"
                           parent="${LowerNeckPitchParentLink}" child="${LowerNeckPitchLinkName}"
-                          origin_xyz="${LowerNeckPitchOrigin_X} ${LowerNeckPitchOrigin_Y} ${LowerNeckPitchOrigin_Z}"
-                          origin_rpy="${LowerNeckPitchFrame_Roll} ${LowerNeckPitchFrame_Roll} ${LowerNeckPitchFrame_Yaw}">
+                          origin_xyz="${LowerNeckPitchFrameOrigin_X} ${LowerNeckPitchFrameOrigin_Y} ${LowerNeckPitchFrameOrigin_Z}"
+                          origin_rpy="${LowerNeckPitchFrameOrientation_Roll} ${LowerNeckPitchFrameOrientation_Roll} ${LowerNeckPitchFrameOrientation_Yaw}">
       <limit effort="${NJ1_Torque_Limit}" lower="${NJ1_Lower_Limit}" upper="${NJ1_Upper_Limit}" velocity="${NJ1_Speed_Limit}"/>
     </xacro:fixed_joint>
@@ -87,6 +87,6 @@
     <xacro:fixed_joint jointName="${NeckYawJointName}"
                           parent="${LowerNeckPitchLinkName}" child="${NeckYawLinkName}"
-                          origin_xyz="${NeckYawOrigin_X} ${NJ2_Origin_Y} ${NJ2_Origin_Z}"
-                          origin_rpy="${NJ2_Orientation_Roll} ${NJ2_Orientation_Pitch} ${NJ2_Orientation_Yaw}">
+                          origin_xyz="${NeckYawFrameOrigin_X} ${NeckYawFrameOrigin_Y} ${NeckYawFrameOrigin_Z}"
+                          origin_rpy="${NeckYawFrameOrientation_Roll} ${NeckYawFrameOrientation_Pitch} ${NeckYawFrameOrientation_Yaw}">
       <limit effort="${NJ2_Torque_Limit}" lower="${NJ2_Lower_Limit}" upper="${NJ2_Upper_Limit}" velocity="${NJ2_Speed_Limit}"/>
     </xacro:fixed_joint>
@@ -94,6 +94,6 @@
     <xacro:fixed_joint jointName="${UpperNeckPitchJointName}"
                           parent="${NeckYawLinkName}" child="${UpperNeckPitchLinkName}"
-                          origin_xyz="${NJ3_Origin_X} ${NJ3_Origin_Y} ${NJ3_Origin_Z}"
-                          origin_rpy="${NJ3_Orientation_Roll} ${NJ3_Orientation_Pitch} ${NJ3_Orientation_Yaw}">
+                          origin_xyz="${UpperNeckPitchFrameOrigin_X} ${UpperNeckPitchFrameOrigin_Y} ${UpperNeckPitchFrameOrigin_Z}"
+                          origin_rpy="${UpperNeckPitchFrameOrientation_Roll} ${UpperNeckPitchFrameOrientation_Pitch} ${UpperNeckPitchFrameOrientation_Yaw}">
       <limit effort="${NJ3_Torque_Limit}" lower="${NJ3_Lower_Limit}" upper="${NJ3_Upper_Limit}" velocity="${NJ3_Speed_Limit}"/>
     </xacro:fixed_joint>

Commit message: Removed some more extra crap. More to come. Rename dh_parameters.xacro for head and arms to frames_parameters.xacro.

File: valkyrie_description/robots/valkyrie_A/xacro/arm/actuator_names.xacro (robot description, xacro)
@@ -6,7 +6,3 @@
   <xacro:property name="ElbowPitchActuatorName" value="/${prefix}Arm/Actuator4" />
   <xacro:property name="ForearmYawActuatorName" value="/${prefix}Arm/Actuator5" />
-  <xacro:property name="RAJ6_Actuator_Name" value="/RightArm/ForearmDriver1/RightWristActuator" />
-  <xacro:property name="RAJ7_Actuator_Name" value="/RightArm/ForearmDriver1/LeftWristActuator" />
-  <xacro:property name="LAJ6_Actuator_Name" value="/LeftArm/ForearmDriver1/LeftWristActuator" />
-  <xacro:property name="LAJ7_Actuator_Name" value="/LeftArm/ForearmDriver1/RightWristActuator" />
 </robot>

File: valkyrie_description/robots/valkyrie_A/xacro/arm/arm.xacro (robot description, xacro)
@@ -4,5 +4,5 @@
   <xacro:include filename="$(find valkyrie_description)/robots/valkyrie_A/xacro/arm/link_names.xacro"/>
   <xacro:include filename="$(find valkyrie_description)/robots/valkyrie_A/xacro/arm/joint_limits.xacro"/>
-  <xacro:include filename="$(find valkyrie_description)/robots/valkyrie_A/xacro/arm/dh_parameters.xacro"/>
+  <xacro:include filename="$(find valkyrie_description)/robots/valkyrie_A/xacro/arm/frame_parameters.xacro"/>
   <xacro:include filename="$(find valkyrie_description)/robots/valkyrie_A/xacro/arm/mass_parameters.xacro"/>
   <xacro:include filename="$(find valkyrie_description)/robots/valkyrie_A/xacro/sensors/camboard.xacro"/>

File: valkyrie_description/robots/valkyrie_A/xacro/head/head.xacro (robot description, xacro)
@@ -4,5 +4,5 @@
   <xacro:include filename="$(find valkyrie_description)/robots/valkyrie_A/xacro/head/link_names.xacro"/>
   <xacro:include filename="$(find valkyrie_description)/robots/valkyrie_A/xacro/head/joint_limits.xacro"/>
-  <xacro:include filename="$(find valkyrie_description)/robots/valkyrie_A/xacro/head/dh_parameters.xacro"/>
+  <xacro:include filename="$(find valkyrie_description)/robots/valkyrie_A/xacro/head/frame_parameters.xacro"/>
   <xacro:include filename="$(find valkyrie_description)/robots/valkyrie_A/xacro/head/mass_parameters.xacro"/>
   <xacro:include filename="$(find valkyrie_description)/robots/valkyrie_A/xacro/sensors/camboard.xacro"/>
