Commit message: Fixed naming bug.

File: valkyrie_description/robots/valkyrie_A/xacro/arm/link_names.xacro (robot description, xacro)
@@ -9,4 +9,4 @@
   <xacro:property name="ForearmLinkName" value="${prefix}ForearmLink" />
   <xacro:property name="WristRollLinkName" value="${prefix}WristRollLink" />
-  <xacro:property name="WristPitchLinkName" value="${prefix}PalmLink" />
+  <xacro:property name="WristPitchLinkName" value="${prefix}Palm" />
 </robot>

File: valkyrie_description/robots/valkyrie_A/xacro/head/link_names.xacro (robot description, xacro)
@@ -4,4 +4,4 @@
   <xacro:property name="LowerNeckPitchLinkName" value="LowerNeckPitchLink" />
   <xacro:property name="NeckYawLinkName" value="NeckYawLink" />
-  <xacro:property name="UpperNeckPitchLinkName" value="HeadLink" />
+  <xacro:property name="UpperNeckPitchLinkName" value="Head" />
 </robot>
