Commit message: Rename arm frame orientations and frame origin locations. Will need to rename entire file eventually.

File: valkyrie_description/robots/valkyrie_A/xacro/arm/arm.xacro (robot description, xacro)
@@ -58,6 +58,6 @@
     <xacro:revolute_joint_ex jointName="${AJ1_Joint_Name}"
                           parent="${upper_arm_root_link}" child="${AJ1_Distal_Link}"
-                          origin_xyz="${ArmPitchFrameOrigin_X} ${AJ1_Origin_Y} ${AJ1_Origin_Z}"
-                          origin_rpy="${AJ1_Orientation_Roll} ${AJ1_Orientation_Pitch} ${AJ1_Orientation_Yaw}"
+                          origin_xyz="${ShoulderPitchFrameOrigin_X} ${ShoulderPitchFrameOrigin_Y} ${ShoulderPitchFrameOrigin_Z}"
+                          origin_rpy="${ShoulderPitchFrameOrientation_Roll} ${ShoulderPitchFrameOrientation_Pitch} ${ShoulderPitchFrameOrientation_Yaw}"
                           damping="1.0" friction="0.0">
         <limit effort="${AJ1_Torque_Limit}" lower="${AJ1_Lower_Limit}" upper="${AJ1_Upper_Limit}" velocity="${AJ1_Speed_Limit}"/>
@@ -67,6 +67,6 @@
     <xacro:revolute_joint_ex jointName="${AJ2_Joint_Name}"
                           parent="${AJ2_Proximal_Link}" child="${AJ2_Distal_Link}"
-                          origin_xyz="${AJ2_Origin_X} ${AJ2_Origin_Y} ${AJ2_Origin_Z}"
-                          origin_rpy="${AJ2_Orientation_Roll} ${AJ2_Orientation_Pitch} ${AJ2_Orientation_Yaw}"
+                          origin_xyz="${ShoulderRollFrameOrigin_X} ${ShoulderRollFrameOrigin_Y} ${ShoulderRollFrameOrigin_Z}"
+                          origin_rpy="${ShoulderRollFrameOrientation_Roll} ${ShoulderRollFrameOrientation_Pitch} ${ShoulderRollFrameOrientation_Yaw}"
                           damping="1.0" friction="0.0">
         <limit effort="${AJ2_Torque_Limit}" lower="${AJ2_Lower_Limit}" upper="${AJ2_Upper_Limit}" velocity="${AJ2_Speed_Limit}"/>
@@ -76,6 +76,6 @@
     <xacro:revolute_joint_ex jointName="${AJ3_Joint_Name}"
                           parent="${AJ3_Proximal_Link}" child="${AJ3_Distal_Link}"
-                          origin_xyz="${AJ3_Origin_X} ${AJ3_Origin_Y} ${AJ3_Origin_Z}"
-                          origin_rpy="${AJ3_Orientation_Roll} ${AJ3_Orientation_Pitch} ${AJ3_Orientation_Yaw}"
+                          origin_xyz="${ShoulderYawFrameOrigin_X} ${ShoulderYawFrameOrigin_Y} ${ShoulderYawFrameOrigin_Z}"
+                          origin_rpy="${ShoulderYawFrameOrientation_Roll} ${ShoulderYawFrameOrientation_Pitch} ${ShoulderYawFrameOrientation_Yaw}"
                           damping="1.0" friction="0.0">
         <limit effort="${AJ3_Torque_Limit}" lower="${AJ3_Lower_Limit}" upper="${AJ3_Upper_Limit}" velocity="${AJ3_Speed_Limit}"/>
@@ -85,6 +85,6 @@
     <xacro:revolute_joint_ex jointName="${AJ4_Joint_Name}"
                           parent="${AJ4_Proximal_Link}" child="${AJ4_Distal_Link}"
-                          origin_xyz="${AJ4_Origin_X} ${AJ4_Origin_Y} ${AJ4_Origin_Z}"
-                          origin_rpy="${AJ4_Orientation_Roll} ${AJ4_Orientation_Pitch} ${AJ4_Orientation_Yaw}"
+                          origin_xyz="${ElbowPitchFrameOrigin_X} ${ElbowPitchFrameOrigin_Y} ${ElbowPitchFrameOrigin_Z}"
+                          origin_rpy="${ElbowPitchFrameOrientation_Roll} ${ElbowPitchFrameOrientation_Pitch} ${ElbowPitchFrameOrientation_Yaw}"
                           damping="1.0" friction="0.0">
         <limit effort="${AJ4_Torque_Limit}" lower="${AJ4_Lower_Limit}" upper="${AJ4_Upper_Limit}" velocity="${AJ4_Speed_Limit}"/>
@@ -115,6 +115,6 @@
     <xacro:revolute_joint_ex jointName="${AJ5_Joint_Name}"
                           parent="${lower_arm_root_link}" child="${AJ5_Distal_Link}"
-                          origin_xyz="${AJ5_Origin_X} ${AJ5_Origin_Y} ${AJ5_Origin_Z}"
-                          origin_rpy="${AJ5_Orientation_Roll} ${AJ5_Orientation_Pitch} ${AJ5_Orientation_Yaw}"
+                          origin_xyz="${ForearmYawFrameOrigin_X} ${ForearmYawFrameOrigin_Y} ${ForearmYawFrameOrigin_Z}"
+                          origin_rpy="${ForearmYawFrameOrientation_Roll} ${ForearmYawFrameOrientation_Pitch} ${ForearmYawFrameOrientation_Yaw}"
                           damping="1.0" friction="0.0">
         <limit effort="${AJ5_Torque_Limit}" lower="${AJ5_Lower_Limit}" upper="${AJ5_Upper_Limit}" velocity="${AJ5_Speed_Limit}"/>
@@ -124,6 +124,6 @@
     <xacro:revolute_joint_ex jointName="${AJ6_Joint_Name}"
                           parent="${AJ6_Proximal_Link}" child="${AJ6_Distal_Link}"
-                          origin_xyz="${AJ6_Origin_X} ${AJ6_Origin_Y} ${AJ6_Origin_Z}"
-                          origin_rpy="${AJ6_Orientation_Roll} ${AJ6_Orientation_Pitch} ${AJ6_Orientation_Yaw}"
+                          origin_xyz="${WristRollFrameOrigin_X} ${WristRollFrameOrigin_Y} ${WristRollFrameOrigin_Z}"
+                          origin_rpy="${WristRollFrameOrientation_Roll} ${WristRollFrameOrientation_Pitch} ${WristRollFrameOrientation_Yaw}"
                           damping="1.0" friction="0.0">
         <limit effort="${AJ6_Torque_Limit}" lower="${AJ6_Lower_Limit}" upper="${AJ6_Upper_Limit}" velocity="${AJ6_Speed_Limit}"/>
@@ -133,6 +133,6 @@
     <xacro:revolute_joint_ex jointName="${AJ7_Joint_Name}"
                           parent="${AJ7_Proximal_Link}" child="${AJ7_Distal_Link}"
-                          origin_xyz="${AJ7_Origin_X} ${AJ7_Origin_Y} ${AJ7_Origin_Z}"
-                          origin_rpy="${AJ7_Orientation_Roll} ${AJ7_Orientation_Pitch} ${AJ7_Orientation_Yaw}"
+                          origin_xyz="${WristPitchFrameOrigin_X} ${WristPitchFrameOrigin_Y} ${WristPitchFrameOrigin_Z}"
+                          origin_rpy="${WristPitchFrameOrientation_Roll} ${WristPitchFrameOrientation_Pitch} ${WristPitchFrameOrientation_Yaw}"
                           damping="1.0" friction="0.0">
         <limit effort="${AJ7_Torque_Limit}" lower="${AJ7_Lower_Limit}" upper="${AJ7_Upper_Limit}" velocity="${AJ7_Speed_Limit}"/>
@@ -170,6 +170,6 @@
     <xacro:fixed_joint jointName="${AJ5_Joint_Name}"
                           parent="${lower_arm_root_link}" child="${AJ5_Distal_Link}"
-                          origin_xyz="${AJ5_Origin_X} ${AJ5_Origin_Y} ${AJ5_Origin_Z}"
-                          origin_rpy="${AJ5_Orientation_Roll} ${AJ5_Orientation_Pitch} ${AJ5_Orientation_Yaw}">
+                          origin_xyz="${ForearmYawFrameOrigin_X} ${ForearmYawFrameOrigin_Y} ${ForearmYawFrameOrigin_Z}"
+                          origin_rpy="${ForearmYawFrameOrientation_Roll} ${ForearmYawFrameOrientation_Pitch} ${ForearmYawFrameOrientation_Yaw}">
         <limit effort="${AJ5_Torque_Limit}" lower="${AJ5_Lower_Limit}" upper="${AJ5_Upper_Limit}" velocity="${AJ5_Speed_Limit}"/>
     </xacro:fixed_joint>
@@ -177,6 +177,6 @@
     <xacro:fixed_joint jointName="${AJ6_Joint_Name}"
                           parent="${AJ6_Proximal_Link}" child="${AJ6_Distal_Link}"
-                          origin_xyz="${AJ6_Origin_X} ${AJ6_Origin_Y} ${AJ6_Origin_Z}"
-                          origin_rpy="${AJ6_Orientation_Roll} ${AJ6_Orientation_Pitch} ${AJ6_Orientation_Yaw}">
+                          origin_xyz="${WristRollFrameOrigin_X} ${WristRollFrameOrigin_Y} ${WristRollFrameOrigin_Z}"
+                          origin_rpy="${WristRollFrameOrientation_Roll} ${WristRollFrameOrientation_Pitch} ${WristRollFrameOrientation_Yaw}">
         <limit effort="${AJ6_Torque_Limit}" lower="${AJ6_Lower_Limit}" upper="${AJ6_Upper_Limit}" velocity="${AJ6_Speed_Limit}"/>
     </xacro:fixed_joint>
@@ -184,6 +184,6 @@
     <xacro:fixed_joint jointName="${AJ7_Joint_Name}"
                           parent="${AJ7_Proximal_Link}" child="${AJ7_Distal_Link}"
-                          origin_xyz="${AJ7_Origin_X} ${AJ7_Origin_Y} ${AJ7_Origin_Z}"
-                          origin_rpy="${AJ7_Orientation_Roll} ${AJ7_Orientation_Pitch} ${AJ7_Orientation_Yaw}">
+                          origin_xyz="${WristPitchFrameOrigin_X} ${WristPitchFrameOrigin_Y} ${WristPitchFrameOrigin_Z}"
+                          origin_rpy="${WristPitchFrameOrientation_Roll} ${WristPitchFrameOrientation_Pitch} ${WristPitchFrameOrientation_Yaw}">
         <limit effort="${AJ7_Torque_Limit}" lower="${AJ7_Lower_Limit}" upper="${AJ7_Upper_Limit}" velocity="${AJ7_Speed_Limit}"/>
     </xacro:fixed_joint>

File: valkyrie_description/robots/valkyrie_A/xacro/arm/dh_parameters.xacro (robot description, xacro)
@@ -1,45 +1,45 @@
 <?xml version="1.0" ?>
 <robot xmlns:xacro="http://www.ros.org/wiki/xacro" name="v1/arm/dh_parameters">
-  <xacro:property name="ArmPitchFrameOrigin_X" value="0.29842"/>
-  <xacro:property name="AJ1_Origin_Y" value="0"/>
-  <xacro:property name="AJ1_Origin_Z" value="-0.03157"/>
-  <xacro:property name="AJ1_Orientation_Roll" value="${pi_2}"/>
-  <xacro:property name="AJ1_Orientation_Pitch" value="0"/>
-  <xacro:property name="AJ1_Orientation_Yaw" value="0"/>
-  <xacro:property name="AJ2_Origin_X" value="0"/>
-  <xacro:property name="AJ2_Origin_Y" value="0"/>
-  <xacro:property name="AJ2_Origin_Z" value="${reflect * -0.246}"/>
-  <xacro:property name="AJ2_Orientation_Roll" value="${reflect * (pi_2)}"/>
-  <xacro:property name="AJ2_Orientation_Pitch" value="0"/>
-  <xacro:property name="AJ2_Orientation_Yaw" value="${pi}"/>
-  <xacro:property name="AJ3_Origin_X" value="0"/>
-  <xacro:property name="AJ3_Origin_Y" value="0"/>
-  <xacro:property name="AJ3_Origin_Z" value="0"/>
-  <xacro:property name="AJ3_Orientation_Roll" value="${-1 * pi_2}"/>
-  <xacro:property name="AJ3_Orientation_Pitch" value="0"/>
-  <xacro:property name="AJ3_Orientation_Yaw" value="${reflect * pi_2}"/>
-  <xacro:property name="AJ4_Origin_X" value="0"/>
-  <xacro:property name="AJ4_Origin_Y" value="${reflect * -0.0254}"/>
-  <xacro:property name="AJ4_Origin_Z" value="${reflect * -0.330}"/>
-  <xacro:property name="AJ4_Orientation_Roll" value="${reflect * pi_2}"/>
-  <xacro:property name="AJ4_Orientation_Pitch" value="0"/>
-  <xacro:property name="AJ4_Orientation_Yaw" value="${reflect * pi_2}"/>
-  <xacro:property name="AJ5_Origin_X" value="0.0254"/>
-  <xacro:property name="AJ5_Origin_Y" value="0"/>
-  <xacro:property name="AJ5_Origin_Z" value="0"/>
-  <xacro:property name="AJ5_Orientation_Roll" value="${reflect * pi_2}"/>
-  <xacro:property name="AJ5_Orientation_Pitch" value="0"/>
-  <xacro:property name="AJ5_Orientation_Yaw" value="${pi}"/>
-  <xacro:property name="AJ6_Origin_X" value="0"/>
-  <xacro:property name="AJ6_Origin_Y" value="0"/>
-  <xacro:property name="AJ6_Origin_Z" value="${reflect * -0.287}"/>
-  <xacro:property name="AJ6_Orientation_Roll" value="${-1 * pi_2}"/>
-  <xacro:property name="AJ6_Orientation_Pitch" value="0"/>
-  <xacro:property name="AJ6_Orientation_Yaw" value="${reflect * pi_2}"/>
-  <xacro:property name="AJ7_Origin_X" value="0"/>
-  <xacro:property name="AJ7_Origin_Y" value="0"/>
-  <xacro:property name="AJ7_Origin_Z" value="0"/>
-  <xacro:property name="AJ7_Orientation_Roll" value="${reflect * pi_2}"/>
-  <xacro:property name="AJ7_Orientation_Pitch" value="0"/>
-  <xacro:property name="AJ7_Orientation_Yaw" value="${reflect * pi_2}"/>
+  <xacro:property name="ShoulderPitchFrameOrigin_X" value="0.29842"/>
+  <xacro:property name="ShoulderPitchFrameOrigin_Y" value="0"/>
+  <xacro:property name="ShoulderPitchFrameOrigin_Z" value="-0.03157"/>
+  <xacro:property name="ShoulderPitchFrameOrientation_Roll" value="${pi_2}"/>
+  <xacro:property name="ShoulderPitchFrameOrientation_Pitch" value="0"/>
+  <xacro:property name="ShoulderPitchFrameOrientation_Yaw" value="0"/>
+  <xacro:property name="ShoulderRollFrameOrigin_X" value="0"/>
+  <xacro:property name="ShoulderRollFrameOrigin_Y" value="0"/>
+  <xacro:property name="ShoulderRollFrameOrigin_Z" value="${reflect * -0.246}"/>
+  <xacro:property name="ShoulderRollFrameOrientation_Roll" value="${reflect * (pi_2)}"/>
+  <xacro:property name="ShoulderRollFrameOrientation_Pitch" value="0"/>
+  <xacro:property name="ShoulderRollFrameOrientation_Yaw" value="${pi}"/>
+  <xacro:property name="ShoulderYawFrameOrigin_X" value="0"/>
+  <xacro:property name="ShoulderYawFrameOrigin_Y" value="0"/>
+  <xacro:property name="ShoulderYawFrameOrigin_Z" value="0"/>
+  <xacro:property name="ShoulderYawFrameOrientation_Roll" value="${-1 * pi_2}"/>
+  <xacro:property name="ShoulderYawFrameOrientation_Pitch" value="0"/>
+  <xacro:property name="ShoulderYawFrameOrientation_Yaw" value="${reflect * pi_2}"/>
+  <xacro:property name="ElbowPitchFrameOrigin_X" value="0"/>
+  <xacro:property name="ElbowPitchFrameOrigin_Y" value="${reflect * -0.0254}"/>
+  <xacro:property name="ElbowPitchFrameOrigin_Z" value="${reflect * -0.330}"/>
+  <xacro:property name="ElbowPitchFrameOrientation_Roll" value="${reflect * pi_2}"/>
+  <xacro:property name="ElbowPitchFrameOrientation_Pitch" value="0"/>
+  <xacro:property name="ElbowPitchFrameOrientation_Yaw" value="${reflect * pi_2}"/>
+  <xacro:property name="ForearmYawFrameOrigin_X" value="0.0254"/>
+  <xacro:property name="ForearmYawFrameOrigin_Y" value="0"/>
+  <xacro:property name="ForearmYawFrameOrigin_Z" value="0"/>
+  <xacro:property name="ForearmYawFrameOrientation_Roll" value="${reflect * pi_2}"/>
+  <xacro:property name="ForearmYawFrameOrientation_Pitch" value="0"/>
+  <xacro:property name="ForearmYawFrameOrientation_Yaw" value="${pi}"/>
+  <xacro:property name="WristRollFrameOrigin_X" value="0"/>
+  <xacro:property name="WristRollFrameOrigin_Y" value="0"/>
+  <xacro:property name="WristRollFrameOrigin_Z" value="${reflect * -0.287}"/>
+  <xacro:property name="WristRollFrameOrientation_Roll" value="${-1 * pi_2}"/>
+  <xacro:property name="WristRollFrameOrientation_Pitch" value="0"/>
+  <xacro:property name="WristRollFrameOrientation_Yaw" value="${reflect * pi_2}"/>
+  <xacro:property name="WristPitchFrameOrigin_X" value="0"/>
+  <xacro:property name="WristPitchFrameOrigin_Y" value="0"/>
+  <xacro:property name="WristPitchFrameOrigin_Z" value="0"/>
+  <xacro:property name="WristPitchFrameOrientation_Roll" value="${reflect * pi_2}"/>
+  <xacro:property name="WristPitchFrameOrientation_Pitch" value="0"/>
+  <xacro:property name="WristPitchFrameOrientation_Yaw" value="${reflect * pi_2}"/>
 </robot>

File: valkyrie_description/robots/valkyrie_A/xacro/head/dh_parameters.xacro (robot description, xacro)
@@ -7,7 +7,7 @@
   <xacro:property name="LowerNeckPitchFrameOrientation_Pitch" value="0.0"/>
   <xacro:property name="LowerNeckPitchFrameOrientation_Yaw" value="0.0"/>
-  <xacro:property name="NeckYawFrameOrigin_X" value="0"/>
-  <xacro:property name="NeckYawFrameOrigin_Y" value="0.0519"/>
-  <xacro:property name="NeckYawFrameOrigin_Z" value="0"/>
+  <xacro:property name="NeckShoulderYawFrameOrigin_X" value="0"/>
+  <xacro:property name="NeckShoulderYawFrameOrigin_Y" value="0.0519"/>
+  <xacro:property name="NeckShoulderYawFrameOrigin_Z" value="0"/>
   <xacro:property name="NeckYawFrameOrientation_Roll" value="0.0"/>
   <xacro:property name="NeckYawFrameOrientation_Pitch" value="0.0"/>

File: valkyrie_description/robots/valkyrie_A/xacro/head/head.xacro (robot description, xacro)
@@ -45,5 +45,5 @@
     <xacro:revolute_joint_ex jointName="${NeckYawJointName}"
                           parent="${LowerNeckPitchLinkName}" child="${NeckYawLinkName}"
-                          origin_xyz="${NeckYawFrameOrigin_X} ${NeckYawFrameOrigin_Y} ${NeckYawFrameOrigin_Z}"
+                          origin_xyz="${NeckShoulderYawFrameOrigin_X} ${NeckShoulderYawFrameOrigin_Y} ${NeckShoulderYawFrameOrigin_Z}"
                           origin_rpy="${NeckYawFrameOrientation_Roll} ${NeckYawFrameOrientation_Pitch} ${NeckYawFrameOrientation_Yaw}"
                           damping="1.0" friction="0.0">
@@ -87,5 +87,5 @@
     <xacro:fixed_joint jointName="${NeckYawJointName}"
                           parent="${LowerNeckPitchLinkName}" child="${NeckYawLinkName}"
-                          origin_xyz="${NeckYawFrameOrigin_X} ${NeckYawFrameOrigin_Y} ${NeckYawFrameOrigin_Z}"
+                          origin_xyz="${NeckShoulderYawFrameOrigin_X} ${NeckShoulderYawFrameOrigin_Y} ${NeckShoulderYawFrameOrigin_Z}"
                           origin_rpy="${NeckYawFrameOrientation_Roll} ${NeckYawFrameOrientation_Pitch} ${NeckYawFrameOrientation_Yaw}">
       <limit effort="${NeckYawTorqueLimit}" lower="${NeckYawPositionLimit_Lower}" upper="${NeckYawPositionLimit_Upper}" velocity="${NeckYawVelocityLimit}"/>
