Commit message: Renamed xacro properties for arm joint torque limits.

File: valkyrie_description/robots/valkyrie_A/xacro/arm/arm.xacro (robot description, xacro)
@@ -61,5 +61,5 @@
                           origin_rpy="${ShoulderPitchFrameOrientation_Roll} ${ShoulderPitchFrameOrientation_Pitch} ${ShoulderPitchFrameOrientation_Yaw}"
                           damping="1.0" friction="0.0">
-        <limit effort="${AJ1_Torque_Limit}" lower="${AJ1_Lower_Limit}" upper="${AJ1_Upper_Limit}" velocity="${AJ1_Speed_Limit}"/>
+        <limit effort="${ShoulderPitchTorqueLimit}" lower="${AJ1_Lower_Limit}" upper="${AJ1_Upper_Limit}" velocity="${AJ1_Speed_Limit}"/>
         <controller_gains Kp="20000" Kd="400"/>
     </xacro:revolute_joint_ex>
@@ -70,5 +70,5 @@
                           origin_rpy="${ShoulderRollFrameOrientation_Roll} ${ShoulderRollFrameOrientation_Pitch} ${ShoulderRollFrameOrientation_Yaw}"
                           damping="1.0" friction="0.0">
-        <limit effort="${AJ2_Torque_Limit}" lower="${AJ2_Lower_Limit}" upper="${AJ2_Upper_Limit}" velocity="${AJ2_Speed_Limit}"/>
+        <limit effort="${ShoulderRollTorqueLimit}" lower="${AJ2_Lower_Limit}" upper="${AJ2_Upper_Limit}" velocity="${AJ2_Speed_Limit}"/>
         <controller_gains Kp="20000" Kd="400"/>
     </xacro:revolute_joint_ex>
@@ -79,5 +79,5 @@
                           origin_rpy="${ShoulderYawFrameOrientation_Roll} ${ShoulderYawFrameOrientation_Pitch} ${ShoulderYawFrameOrientation_Yaw}"
                           damping="1.0" friction="0.0">
-        <limit effort="${AJ3_Torque_Limit}" lower="${AJ3_Lower_Limit}" upper="${AJ3_Upper_Limit}" velocity="${AJ3_Speed_Limit}"/>
+        <limit effort="${ShoulderYawTorqueLimit}" lower="${AJ3_Lower_Limit}" upper="${AJ3_Upper_Limit}" velocity="${AJ3_Speed_Limit}"/>
         <controller_gains Kp="20000" Kd="400"/>
     </xacro:revolute_joint_ex>
@@ -88,5 +88,5 @@
                           origin_rpy="${ElbowPitchFrameOrientation_Roll} ${ElbowPitchFrameOrientation_Pitch} ${ElbowPitchFrameOrientation_Yaw}"
                           damping="1.0" friction="0.0">
-        <limit effort="${AJ4_Torque_Limit}" lower="${AJ4_Lower_Limit}" upper="${AJ4_Upper_Limit}" velocity="${AJ4_Speed_Limit}"/>
+        <limit effort="${ElbowPitchTorqueLimit}" lower="${AJ4_Lower_Limit}" upper="${AJ4_Upper_Limit}" velocity="${AJ4_Speed_Limit}"/>
         <controller_gains Kp="20000" Kd="400"/>
     </xacro:revolute_joint_ex>
@@ -118,5 +118,5 @@
                           origin_rpy="${ForearmYawFrameOrientation_Roll} ${ForearmYawFrameOrientation_Pitch} ${ForearmYawFrameOrientation_Yaw}"
                           damping="1.0" friction="0.0">
-        <limit effort="${AJ5_Torque_Limit}" lower="${AJ5_Lower_Limit}" upper="${AJ5_Upper_Limit}" velocity="${AJ5_Speed_Limit}"/>
+        <limit effort="${ForearmYawTorqueLimit}" lower="${AJ5_Lower_Limit}" upper="${AJ5_Upper_Limit}" velocity="${AJ5_Speed_Limit}"/>
         <controller_gains Kp="20000" Kd="0"/>
     </xacro:revolute_joint_ex>
@@ -127,5 +127,5 @@
                           origin_rpy="${WristRollFrameOrientation_Roll} ${WristRollFrameOrientation_Pitch} ${WristRollFrameOrientation_Yaw}"
                           damping="1.0" friction="0.0">
-        <limit effort="${AJ6_Torque_Limit}" lower="${AJ6_Lower_Limit}" upper="${AJ6_Upper_Limit}" velocity="${AJ6_Speed_Limit}"/>
+        <limit effort="${WristRollTorqueLimit}" lower="${AJ6_Lower_Limit}" upper="${AJ6_Upper_Limit}" velocity="${AJ6_Speed_Limit}"/>
         <controller_gains Kp="20000" Kd="400"/>
     </xacro:revolute_joint_ex>
@@ -136,5 +136,5 @@
                           origin_rpy="${WristPitchFrameOrientation_Roll} ${WristPitchFrameOrientation_Pitch} ${WristPitchFrameOrientation_Yaw}"
                           damping="1.0" friction="0.0">
-        <limit effort="${AJ7_Torque_Limit}" lower="${AJ7_Lower_Limit}" upper="${AJ7_Upper_Limit}" velocity="${AJ7_Speed_Limit}"/>
+        <limit effort="${WristPitchTorqueLimit}" lower="${AJ7_Lower_Limit}" upper="${AJ7_Upper_Limit}" velocity="${AJ7_Speed_Limit}"/>
         <controller_gains Kp="20000" Kd="400"/>
     </xacro:revolute_joint_ex>
@@ -172,5 +172,5 @@
                           origin_xyz="${ForearmYawFrameOrigin_X} ${ForearmYawFrameOrigin_Y} ${ForearmYawFrameOrigin_Z}"
                           origin_rpy="${ForearmYawFrameOrientation_Roll} ${ForearmYawFrameOrientation_Pitch} ${ForearmYawFrameOrientation_Yaw}">
-        <limit effort="${AJ5_Torque_Limit}" lower="${AJ5_Lower_Limit}" upper="${AJ5_Upper_Limit}" velocity="${AJ5_Speed_Limit}"/>
+        <limit effort="${ForearmYawTorqueLimit}" lower="${AJ5_Lower_Limit}" upper="${AJ5_Upper_Limit}" velocity="${AJ5_Speed_Limit}"/>
     </xacro:fixed_joint>
     <!-- AJ6 -->
@@ -179,5 +179,5 @@
                           origin_xyz="${WristRollFrameOrigin_X} ${WristRollFrameOrigin_Y} ${WristRollFrameOrigin_Z}"
                           origin_rpy="${WristRollFrameOrientation_Roll} ${WristRollFrameOrientation_Pitch} ${WristRollFrameOrientation_Yaw}">
-        <limit effort="${AJ6_Torque_Limit}" lower="${AJ6_Lower_Limit}" upper="${AJ6_Upper_Limit}" velocity="${AJ6_Speed_Limit}"/>
+        <limit effort="${WristRollTorqueLimit}" lower="${AJ6_Lower_Limit}" upper="${AJ6_Upper_Limit}" velocity="${AJ6_Speed_Limit}"/>
     </xacro:fixed_joint>
     <!-- AJ7 -->
@@ -186,5 +186,5 @@
                           origin_xyz="${WristPitchFrameOrigin_X} ${WristPitchFrameOrigin_Y} ${WristPitchFrameOrigin_Z}"
                           origin_rpy="${WristPitchFrameOrientation_Roll} ${WristPitchFrameOrientation_Pitch} ${WristPitchFrameOrientation_Yaw}">
-        <limit effort="${AJ7_Torque_Limit}" lower="${AJ7_Lower_Limit}" upper="${AJ7_Upper_Limit}" velocity="${AJ7_Speed_Limit}"/>
+        <limit effort="${WristPitchTorqueLimit}" lower="${AJ7_Lower_Limit}" upper="${AJ7_Upper_Limit}" velocity="${AJ7_Speed_Limit}"/>
     </xacro:fixed_joint>
   </xacro:macro>

File: valkyrie_description/robots/valkyrie_A/xacro/arm/joint_limits.xacro (robot description, xacro)
@@ -1,11 +1,11 @@
 <?xml version="1.0" ?>
 <robot xmlns:xacro="http://www.ros.org/wiki/xacro" name="v1/arm/joint_limits">
-  <xacro:property name="AJ1_Torque_Limit" value="190" />
-  <xacro:property name="AJ2_Torque_Limit" value="190" />
-  <xacro:property name="AJ3_Torque_Limit" value="65" />
-  <xacro:property name="AJ4_Torque_Limit" value="65" />
-  <xacro:property name="AJ5_Torque_Limit" value="26" />
-  <xacro:property name="AJ6_Torque_Limit" value="14" />
-  <xacro:property name="AJ7_Torque_Limit" value="14" />
+  <xacro:property name="ShoulderPitchTorqueLimit" value="190" />
+  <xacro:property name="ShoulderRollTorqueLimit" value="190" />
+  <xacro:property name="ShoulderYawTorqueLimit" value="65" />
+  <xacro:property name="ElbowPitchTorqueLimit" value="65" />
+  <xacro:property name="ForearmYawTorqueLimit" value="26" />
+  <xacro:property name="WristRollTorqueLimit" value="14" />
+  <xacro:property name="WristPitchTorqueLimit" value="14" />
   <xacro:property name="AJ1_Lower_Limit" value="${-180 * DEG2RAD}" />
   <xacro:property name="AJ2_Lower_Limit" value="${-175 * DEG2RAD}" />

Commit message: Renamed lower limits of arm joints and got rid of degree to rad conversion via xacro property.

File: valkyrie_description/robots/valkyrie_A/xacro/arm/arm.xacro (robot description, xacro)
@@ -61,5 +61,5 @@
                           origin_rpy="${ShoulderPitchFrameOrientation_Roll} ${ShoulderPitchFrameOrientation_Pitch} ${ShoulderPitchFrameOrientation_Yaw}"
                           damping="1.0" friction="0.0">
-        <limit effort="${ShoulderPitchTorqueLimit}" lower="${AJ1_Lower_Limit}" upper="${AJ1_Upper_Limit}" velocity="${AJ1_Speed_Limit}"/>
+        <limit effort="${ShoulderPitchTorqueLimit}" lower="${ShoulderPitchPositionLimit_Lower}" upper="${AJ1_Upper_Limit}" velocity="${AJ1_Speed_Limit}"/>
         <controller_gains Kp="20000" Kd="400"/>
     </xacro:revolute_joint_ex>
@@ -70,5 +70,5 @@
                           origin_rpy="${ShoulderRollFrameOrientation_Roll} ${ShoulderRollFrameOrientation_Pitch} ${ShoulderRollFrameOrientation_Yaw}"
                           damping="1.0" friction="0.0">
-        <limit effort="${ShoulderRollTorqueLimit}" lower="${AJ2_Lower_Limit}" upper="${AJ2_Upper_Limit}" velocity="${AJ2_Speed_Limit}"/>
+        <limit effort="${ShoulderRollTorqueLimit}" lower="${ShoulderRollPositionLimit_Lower}" upper="${AJ2_Upper_Limit}" velocity="${AJ2_Speed_Limit}"/>
         <controller_gains Kp="20000" Kd="400"/>
     </xacro:revolute_joint_ex>
@@ -79,5 +79,5 @@
                           origin_rpy="${ShoulderYawFrameOrientation_Roll} ${ShoulderYawFrameOrientation_Pitch} ${ShoulderYawFrameOrientation_Yaw}"
                           damping="1.0" friction="0.0">
-        <limit effort="${ShoulderYawTorqueLimit}" lower="${AJ3_Lower_Limit}" upper="${AJ3_Upper_Limit}" velocity="${AJ3_Speed_Limit}"/>
+        <limit effort="${ShoulderYawTorqueLimit}" lower="${ShoulderYawPositionLimit_Lower}" upper="${AJ3_Upper_Limit}" velocity="${AJ3_Speed_Limit}"/>
         <controller_gains Kp="20000" Kd="400"/>
     </xacro:revolute_joint_ex>
@@ -88,5 +88,5 @@
                           origin_rpy="${ElbowPitchFrameOrientation_Roll} ${ElbowPitchFrameOrientation_Pitch} ${ElbowPitchFrameOrientation_Yaw}"
                           damping="1.0" friction="0.0">
-        <limit effort="${ElbowPitchTorqueLimit}" lower="${AJ4_Lower_Limit}" upper="${AJ4_Upper_Limit}" velocity="${AJ4_Speed_Limit}"/>
+        <limit effort="${ElbowPitchTorqueLimit}" lower="${ElbowPitchPositionLimit_Lower}" upper="${AJ4_Upper_Limit}" velocity="${AJ4_Speed_Limit}"/>
         <controller_gains Kp="20000" Kd="400"/>
     </xacro:revolute_joint_ex>
@@ -118,5 +118,5 @@
                           origin_rpy="${ForearmYawFrameOrientation_Roll} ${ForearmYawFrameOrientation_Pitch} ${ForearmYawFrameOrientation_Yaw}"
                           damping="1.0" friction="0.0">
-        <limit effort="${ForearmYawTorqueLimit}" lower="${AJ5_Lower_Limit}" upper="${AJ5_Upper_Limit}" velocity="${AJ5_Speed_Limit}"/>
+        <limit effort="${ForearmYawTorqueLimit}" lower="${ForearmYawPositionLimit_Lower}" upper="${AJ5_Upper_Limit}" velocity="${AJ5_Speed_Limit}"/>
         <controller_gains Kp="20000" Kd="0"/>
     </xacro:revolute_joint_ex>
@@ -127,5 +127,5 @@
                           origin_rpy="${WristRollFrameOrientation_Roll} ${WristRollFrameOrientation_Pitch} ${WristRollFrameOrientation_Yaw}"
                           damping="1.0" friction="0.0">
-        <limit effort="${WristRollTorqueLimit}" lower="${AJ6_Lower_Limit}" upper="${AJ6_Upper_Limit}" velocity="${AJ6_Speed_Limit}"/>
+        <limit effort="${WristRollTorqueLimit}" lower="${WristRollPositionLimit_Lower}" upper="${AJ6_Upper_Limit}" velocity="${AJ6_Speed_Limit}"/>
         <controller_gains Kp="20000" Kd="400"/>
     </xacro:revolute_joint_ex>
@@ -136,5 +136,5 @@
                           origin_rpy="${WristPitchFrameOrientation_Roll} ${WristPitchFrameOrientation_Pitch} ${WristPitchFrameOrientation_Yaw}"
                           damping="1.0" friction="0.0">
-        <limit effort="${WristPitchTorqueLimit}" lower="${AJ7_Lower_Limit}" upper="${AJ7_Upper_Limit}" velocity="${AJ7_Speed_Limit}"/>
+        <limit effort="${WristPitchTorqueLimit}" lower="${WristPitchPositionLimit_Lower}" upper="${AJ7_Upper_Limit}" velocity="${AJ7_Speed_Limit}"/>
         <controller_gains Kp="20000" Kd="400"/>
     </xacro:revolute_joint_ex>
@@ -172,5 +172,5 @@
                           origin_xyz="${ForearmYawFrameOrigin_X} ${ForearmYawFrameOrigin_Y} ${ForearmYawFrameOrigin_Z}"
                           origin_rpy="${ForearmYawFrameOrientation_Roll} ${ForearmYawFrameOrientation_Pitch} ${ForearmYawFrameOrientation_Yaw}">
-        <limit effort="${ForearmYawTorqueLimit}" lower="${AJ5_Lower_Limit}" upper="${AJ5_Upper_Limit}" velocity="${AJ5_Speed_Limit}"/>
+        <limit effort="${ForearmYawTorqueLimit}" lower="${ForearmYawPositionLimit_Lower}" upper="${AJ5_Upper_Limit}" velocity="${AJ5_Speed_Limit}"/>
     </xacro:fixed_joint>
     <!-- AJ6 -->
@@ -179,5 +179,5 @@
                           origin_xyz="${WristRollFrameOrigin_X} ${WristRollFrameOrigin_Y} ${WristRollFrameOrigin_Z}"
                           origin_rpy="${WristRollFrameOrientation_Roll} ${WristRollFrameOrientation_Pitch} ${WristRollFrameOrientation_Yaw}">
-        <limit effort="${WristRollTorqueLimit}" lower="${AJ6_Lower_Limit}" upper="${AJ6_Upper_Limit}" velocity="${AJ6_Speed_Limit}"/>
+        <limit effort="${WristRollTorqueLimit}" lower="${WristRollPositionLimit_Lower}" upper="${AJ6_Upper_Limit}" velocity="${AJ6_Speed_Limit}"/>
     </xacro:fixed_joint>
     <!-- AJ7 -->
@@ -186,5 +186,5 @@
                           origin_xyz="${WristPitchFrameOrigin_X} ${WristPitchFrameOrigin_Y} ${WristPitchFrameOrigin_Z}"
                           origin_rpy="${WristPitchFrameOrientation_Roll} ${WristPitchFrameOrientation_Pitch} ${WristPitchFrameOrientation_Yaw}">
-        <limit effort="${WristPitchTorqueLimit}" lower="${AJ7_Lower_Limit}" upper="${AJ7_Upper_Limit}" velocity="${AJ7_Speed_Limit}"/>
+        <limit effort="${WristPitchTorqueLimit}" lower="${WristPitchPositionLimit_Lower}" upper="${AJ7_Upper_Limit}" velocity="${AJ7_Speed_Limit}"/>
     </xacro:fixed_joint>
   </xacro:macro>

File: valkyrie_description/robots/valkyrie_A/xacro/arm/joint_limits.xacro (robot description, xacro)
@@ -8,11 +8,11 @@
   <xacro:property name="WristRollTorqueLimit" value="14" />
   <xacro:property name="WristPitchTorqueLimit" value="14" />
-  <xacro:property name="AJ1_Lower_Limit" value="${-180 * DEG2RAD}" />
-  <xacro:property name="AJ2_Lower_Limit" value="${-175 * DEG2RAD}" />
-  <xacro:property name="AJ3_Lower_Limit" value="${-90 * DEG2RAD}" />
-  <xacro:property name="AJ4_Lower_Limit" value="${-110 * DEG2RAD}" />
-  <xacro:property name="AJ5_Lower_Limit" value="${-135 * DEG2RAD}" />
-  <xacro:property name="AJ6_Lower_Limit" value="${-50 * DEG2RAD}" />
-  <xacro:property name="AJ7_Lower_Limit" value="${-30 * DEG2RAD}" />
+  <xacro:property name="ShoulderPitchPositionLimit_Lower" value="-3.14" />
+  <xacro:property name="ShoulderRollPositionLimit_Lower" value="-3.05" />
+  <xacro:property name="ShoulderYawPositionLimit_Lower" value="-1.57" />
+  <xacro:property name="ElbowPitchPositionLimit_Lower" value="-1.92" />
+  <xacro:property name="ForearmYawPositionLimit_Lower" value="-2.36" />
+  <xacro:property name="WristRollPositionLimit_Lower" value="-0.873" />
+  <xacro:property name="WristPitchPositionLimit_Lower" value="-0.524" />
   <xacro:property name="AJ1_Upper_Limit" value="${180 * DEG2RAD}" />
   <xacro:property name="AJ2_Upper_Limit" value="-0.155" />

Commit message: Renamed variables for position limits of arm joints.

File: valkyrie_description/robots/valkyrie_A/xacro/arm/arm.xacro (robot description, xacro)
@@ -61,5 +61,5 @@
                           origin_rpy="${ShoulderPitchFrameOrientation_Roll} ${ShoulderPitchFrameOrientation_Pitch} ${ShoulderPitchFrameOrientation_Yaw}"
                           damping="1.0" friction="0.0">
-        <limit effort="${ShoulderPitchTorqueLimit}" lower="${ShoulderPitchPositionLimit_Lower}" upper="${AJ1_Upper_Limit}" velocity="${AJ1_Speed_Limit}"/>
+        <limit effort="${ShoulderPitchTorqueLimit}" lower="${ShoulderPitchPositionLimit_Lower}" upper="${ShoulderPitchPositionLimit_Upper}" velocity="${AJ1_Speed_Limit}"/>
         <controller_gains Kp="20000" Kd="400"/>
     </xacro:revolute_joint_ex>
@@ -70,5 +70,5 @@
                           origin_rpy="${ShoulderRollFrameOrientation_Roll} ${ShoulderRollFrameOrientation_Pitch} ${ShoulderRollFrameOrientation_Yaw}"
                           damping="1.0" friction="0.0">
-        <limit effort="${ShoulderRollTorqueLimit}" lower="${ShoulderRollPositionLimit_Lower}" upper="${AJ2_Upper_Limit}" velocity="${AJ2_Speed_Limit}"/>
+        <limit effort="${ShoulderRollTorqueLimit}" lower="${ShoulderRollPositionLimit_Lower}" upper="${ShoulderRollPositionLimit_Upper}" velocity="${AJ2_Speed_Limit}"/>
         <controller_gains Kp="20000" Kd="400"/>
     </xacro:revolute_joint_ex>
@@ -79,5 +79,5 @@
                           origin_rpy="${ShoulderYawFrameOrientation_Roll} ${ShoulderYawFrameOrientation_Pitch} ${ShoulderYawFrameOrientation_Yaw}"
                           damping="1.0" friction="0.0">
-        <limit effort="${ShoulderYawTorqueLimit}" lower="${ShoulderYawPositionLimit_Lower}" upper="${AJ3_Upper_Limit}" velocity="${AJ3_Speed_Limit}"/>
+        <limit effort="${ShoulderYawTorqueLimit}" lower="${ShoulderYawPositionLimit_Lower}" upper="${ShoulderYawPositionLimit_Upper}" velocity="${AJ3_Speed_Limit}"/>
         <controller_gains Kp="20000" Kd="400"/>
     </xacro:revolute_joint_ex>
@@ -88,5 +88,5 @@
                           origin_rpy="${ElbowPitchFrameOrientation_Roll} ${ElbowPitchFrameOrientation_Pitch} ${ElbowPitchFrameOrientation_Yaw}"
                           damping="1.0" friction="0.0">
-        <limit effort="${ElbowPitchTorqueLimit}" lower="${ElbowPitchPositionLimit_Lower}" upper="${AJ4_Upper_Limit}" velocity="${AJ4_Speed_Limit}"/>
+        <limit effort="${ElbowPitchTorqueLimit}" lower="${ElbowPitchPositionLimit_Lower}" upper="${ElbowPitchPositionLimit_Upper}" velocity="${AJ4_Speed_Limit}"/>
         <controller_gains Kp="20000" Kd="400"/>
     </xacro:revolute_joint_ex>
@@ -118,5 +118,5 @@
                           origin_rpy="${ForearmYawFrameOrientation_Roll} ${ForearmYawFrameOrientation_Pitch} ${ForearmYawFrameOrientation_Yaw}"
                           damping="1.0" friction="0.0">
-        <limit effort="${ForearmYawTorqueLimit}" lower="${ForearmYawPositionLimit_Lower}" upper="${AJ5_Upper_Limit}" velocity="${AJ5_Speed_Limit}"/>
+        <limit effort="${ForearmYawTorqueLimit}" lower="${ForearmYawPositionLimit_Lower}" upper="${ForearmYawPositionLimit_Upper}" velocity="${AJ5_Speed_Limit}"/>
         <controller_gains Kp="20000" Kd="0"/>
     </xacro:revolute_joint_ex>
@@ -127,5 +127,5 @@
                           origin_rpy="${WristRollFrameOrientation_Roll} ${WristRollFrameOrientation_Pitch} ${WristRollFrameOrientation_Yaw}"
                           damping="1.0" friction="0.0">
-        <limit effort="${WristRollTorqueLimit}" lower="${WristRollPositionLimit_Lower}" upper="${AJ6_Upper_Limit}" velocity="${AJ6_Speed_Limit}"/>
+        <limit effort="${WristRollTorqueLimit}" lower="${WristRollPositionLimit_Lower}" upper="${WristRollPositionLimit_Upper}" velocity="${AJ6_Speed_Limit}"/>
         <controller_gains Kp="20000" Kd="400"/>
     </xacro:revolute_joint_ex>
@@ -136,5 +136,5 @@
                           origin_rpy="${WristPitchFrameOrientation_Roll} ${WristPitchFrameOrientation_Pitch} ${WristPitchFrameOrientation_Yaw}"
                           damping="1.0" friction="0.0">
-        <limit effort="${WristPitchTorqueLimit}" lower="${WristPitchPositionLimit_Lower}" upper="${AJ7_Upper_Limit}" velocity="${AJ7_Speed_Limit}"/>
+        <limit effort="${WristPitchTorqueLimit}" lower="${WristPitchPositionLimit_Lower}" upper="${WristPitchPositionLimit_Upper}" velocity="${AJ7_Speed_Limit}"/>
         <controller_gains Kp="20000" Kd="400"/>
     </xacro:revolute_joint_ex>
@@ -172,5 +172,5 @@
                           origin_xyz="${ForearmYawFrameOrigin_X} ${ForearmYawFrameOrigin_Y} ${ForearmYawFrameOrigin_Z}"
                           origin_rpy="${ForearmYawFrameOrientation_Roll} ${ForearmYawFrameOrientation_Pitch} ${ForearmYawFrameOrientation_Yaw}">
-        <limit effort="${ForearmYawTorqueLimit}" lower="${ForearmYawPositionLimit_Lower}" upper="${AJ5_Upper_Limit}" velocity="${AJ5_Speed_Limit}"/>
+        <limit effort="${ForearmYawTorqueLimit}" lower="${ForearmYawPositionLimit_Lower}" upper="${ForearmYawPositionLimit_Upper}" velocity="${AJ5_Speed_Limit}"/>
     </xacro:fixed_joint>
     <!-- AJ6 -->
@@ -179,5 +179,5 @@
                           origin_xyz="${WristRollFrameOrigin_X} ${WristRollFrameOrigin_Y} ${WristRollFrameOrigin_Z}"
                           origin_rpy="${WristRollFrameOrientation_Roll} ${WristRollFrameOrientation_Pitch} ${WristRollFrameOrientation_Yaw}">
-        <limit effort="${WristRollTorqueLimit}" lower="${WristRollPositionLimit_Lower}" upper="${AJ6_Upper_Limit}" velocity="${AJ6_Speed_Limit}"/>
+        <limit effort="${WristRollTorqueLimit}" lower="${WristRollPositionLimit_Lower}" upper="${WristRollPositionLimit_Upper}" velocity="${AJ6_Speed_Limit}"/>
     </xacro:fixed_joint>
     <!-- AJ7 -->
@@ -186,5 +186,5 @@
                           origin_xyz="${WristPitchFrameOrigin_X} ${WristPitchFrameOrigin_Y} ${WristPitchFrameOrigin_Z}"
                           origin_rpy="${WristPitchFrameOrientation_Roll} ${WristPitchFrameOrientation_Pitch} ${WristPitchFrameOrientation_Yaw}">
-        <limit effort="${WristPitchTorqueLimit}" lower="${WristPitchPositionLimit_Lower}" upper="${AJ7_Upper_Limit}" velocity="${AJ7_Speed_Limit}"/>
+        <limit effort="${WristPitchTorqueLimit}" lower="${WristPitchPositionLimit_Lower}" upper="${WristPitchPositionLimit_Upper}" velocity="${AJ7_Speed_Limit}"/>
     </xacro:fixed_joint>
   </xacro:macro>

File: valkyrie_description/robots/valkyrie_A/xacro/arm/joint_limits.xacro (robot description, xacro)
@@ -15,11 +15,11 @@
   <xacro:property name="WristRollPositionLimit_Lower" value="-0.873" />
   <xacro:property name="WristPitchPositionLimit_Lower" value="-0.524" />
-  <xacro:property name="AJ1_Upper_Limit" value="${180 * DEG2RAD}" />
-  <xacro:property name="AJ2_Upper_Limit" value="-0.155" />
-  <xacro:property name="AJ3_Upper_Limit" value="1.7" />
-  <xacro:property name="AJ4_Upper_Limit" value="${-5 * DEG2RAD}" />
-  <xacro:property name="AJ5_Upper_Limit" value="${135 * DEG2RAD}" />
-  <xacro:property name="AJ6_Upper_Limit" value="${40 * DEG2RAD}" />
-  <xacro:property name="AJ7_Upper_Limit" value="${25 * DEG2RAD}" />
+  <xacro:property name="ShoulderPitchPositionLimit_Upper" value="3.14" />
+  <xacro:property name="ShoulderRollPositionLimit_Upper" value="-0.155" />
+  <xacro:property name="ShoulderYawPositionLimit_Upper" value="1.7" />
+  <xacro:property name="ElbowPitchPositionLimit_Upper" value="0.087" />
+  <xacro:property name="ForearmYawPositionLimit_Upper" value="2.356" />
+  <xacro:property name="WristRollPositionLimit_Upper" value="0.698" />
+  <xacro:property name="WristPitchPositionLimit_Upper" value="0.436" />
   <xacro:property name="AJ1_Speed_Limit" value="5.89" />
   <xacro:property name="AJ2_Speed_Limit" value="5.89" />
