Commit message: Rename velocity limit properties for arm joints.

File: valkyrie_description/robots/valkyrie_A/xacro/arm/arm.xacro (robot description, xacro)
@@ -61,5 +61,5 @@
                           origin_rpy="${ShoulderPitchFrameOrientation_Roll} ${ShoulderPitchFrameOrientation_Pitch} ${ShoulderPitchFrameOrientation_Yaw}"
                           damping="1.0" friction="0.0">
-        <limit effort="${ShoulderPitchTorqueLimit}" lower="${ShoulderPitchPositionLimit_Lower}" upper="${ShoulderPitchPositionLimit_Upper}" velocity="${AJ1_Speed_Limit}"/>
+        <limit effort="${ShoulderPitchTorqueLimit}" lower="${ShoulderPitchPositionLimit_Lower}" upper="${ShoulderPitchPositionLimit_Upper}" velocity="${ShoulderPitchVelocityLimit}"/>
         <controller_gains Kp="20000" Kd="400"/>
     </xacro:revolute_joint_ex>
@@ -70,5 +70,5 @@
                           origin_rpy="${ShoulderRollFrameOrientation_Roll} ${ShoulderRollFrameOrientation_Pitch} ${ShoulderRollFrameOrientation_Yaw}"
                           damping="1.0" friction="0.0">
-        <limit effort="${ShoulderRollTorqueLimit}" lower="${ShoulderRollPositionLimit_Lower}" upper="${ShoulderRollPositionLimit_Upper}" velocity="${AJ2_Speed_Limit}"/>
+        <limit effort="${ShoulderRollTorqueLimit}" lower="${ShoulderRollPositionLimit_Lower}" upper="${ShoulderRollPositionLimit_Upper}" velocity="${ShoulderRollVelocityLimit}"/>
         <controller_gains Kp="20000" Kd="400"/>
     </xacro:revolute_joint_ex>
@@ -79,5 +79,5 @@
                           origin_rpy="${ShoulderYawFrameOrientation_Roll} ${ShoulderYawFrameOrientation_Pitch} ${ShoulderYawFrameOrientation_Yaw}"
                           damping="1.0" friction="0.0">
-        <limit effort="${ShoulderYawTorqueLimit}" lower="${ShoulderYawPositionLimit_Lower}" upper="${ShoulderYawPositionLimit_Upper}" velocity="${AJ3_Speed_Limit}"/>
+        <limit effort="${ShoulderYawTorqueLimit}" lower="${ShoulderYawPositionLimit_Lower}" upper="${ShoulderYawPositionLimit_Upper}" velocity="${ShoulderYawVelocityLimit}"/>
         <controller_gains Kp="20000" Kd="400"/>
     </xacro:revolute_joint_ex>
@@ -88,5 +88,5 @@
                           origin_rpy="${ElbowPitchFrameOrientation_Roll} ${ElbowPitchFrameOrientation_Pitch} ${ElbowPitchFrameOrientation_Yaw}"
                           damping="1.0" friction="0.0">
-        <limit effort="${ElbowPitchTorqueLimit}" lower="${ElbowPitchPositionLimit_Lower}" upper="${ElbowPitchPositionLimit_Upper}" velocity="${AJ4_Speed_Limit}"/>
+        <limit effort="${ElbowPitchTorqueLimit}" lower="${ElbowPitchPositionLimit_Lower}" upper="${ElbowPitchPositionLimit_Upper}" velocity="${ElbowPitchVelocityLimit}"/>
         <controller_gains Kp="20000" Kd="400"/>
     </xacro:revolute_joint_ex>
@@ -118,5 +118,5 @@
                           origin_rpy="${ForearmYawFrameOrientation_Roll} ${ForearmYawFrameOrientation_Pitch} ${ForearmYawFrameOrientation_Yaw}"
                           damping="1.0" friction="0.0">
-        <limit effort="${ForearmYawTorqueLimit}" lower="${ForearmYawPositionLimit_Lower}" upper="${ForearmYawPositionLimit_Upper}" velocity="${AJ5_Speed_Limit}"/>
+        <limit effort="${ForearmYawTorqueLimit}" lower="${ForearmYawPositionLimit_Lower}" upper="${ForearmYawPositionLimit_Upper}" velocity="${ForearmYawVelocityLimit}"/>
         <controller_gains Kp="20000" Kd="0"/>
     </xacro:revolute_joint_ex>
@@ -127,5 +127,5 @@
                           origin_rpy="${WristRollFrameOrientation_Roll} ${WristRollFrameOrientation_Pitch} ${WristRollFrameOrientation_Yaw}"
                           damping="1.0" friction="0.0">
-        <limit effort="${WristRollTorqueLimit}" lower="${WristRollPositionLimit_Lower}" upper="${WristRollPositionLimit_Upper}" velocity="${AJ6_Speed_Limit}"/>
+        <limit effort="${WristRollTorqueLimit}" lower="${WristRollPositionLimit_Lower}" upper="${WristRollPositionLimit_Upper}" velocity="${WristRollVelocityLimit}"/>
         <controller_gains Kp="20000" Kd="400"/>
     </xacro:revolute_joint_ex>
@@ -136,5 +136,5 @@
                           origin_rpy="${WristPitchFrameOrientation_Roll} ${WristPitchFrameOrientation_Pitch} ${WristPitchFrameOrientation_Yaw}"
                           damping="1.0" friction="0.0">
-        <limit effort="${WristPitchTorqueLimit}" lower="${WristPitchPositionLimit_Lower}" upper="${WristPitchPositionLimit_Upper}" velocity="${AJ7_Speed_Limit}"/>
+        <limit effort="${WristPitchTorqueLimit}" lower="${WristPitchPositionLimit_Lower}" upper="${WristPitchPositionLimit_Upper}" velocity="${WristPitchVelocityLimit}"/>
         <controller_gains Kp="20000" Kd="400"/>
     </xacro:revolute_joint_ex>
@@ -172,5 +172,5 @@
                           origin_xyz="${ForearmYawFrameOrigin_X} ${ForearmYawFrameOrigin_Y} ${ForearmYawFrameOrigin_Z}"
                           origin_rpy="${ForearmYawFrameOrientation_Roll} ${ForearmYawFrameOrientation_Pitch} ${ForearmYawFrameOrientation_Yaw}">
-        <limit effort="${ForearmYawTorqueLimit}" lower="${ForearmYawPositionLimit_Lower}" upper="${ForearmYawPositionLimit_Upper}" velocity="${AJ5_Speed_Limit}"/>
+        <limit effort="${ForearmYawTorqueLimit}" lower="${ForearmYawPositionLimit_Lower}" upper="${ForearmYawPositionLimit_Upper}" velocity="${ForearmYawVelocityLimit}"/>
     </xacro:fixed_joint>
     <!-- AJ6 -->
@@ -179,5 +179,5 @@
                           origin_xyz="${WristRollFrameOrigin_X} ${WristRollFrameOrigin_Y} ${WristRollFrameOrigin_Z}"
                           origin_rpy="${WristRollFrameOrientation_Roll} ${WristRollFrameOrientation_Pitch} ${WristRollFrameOrientation_Yaw}">
-        <limit effort="${WristRollTorqueLimit}" lower="${WristRollPositionLimit_Lower}" upper="${WristRollPositionLimit_Upper}" velocity="${AJ6_Speed_Limit}"/>
+        <limit effort="${WristRollTorqueLimit}" lower="${WristRollPositionLimit_Lower}" upper="${WristRollPositionLimit_Upper}" velocity="${WristRollVelocityLimit}"/>
     </xacro:fixed_joint>
     <!-- AJ7 -->
@@ -186,5 +186,5 @@
                           origin_xyz="${WristPitchFrameOrigin_X} ${WristPitchFrameOrigin_Y} ${WristPitchFrameOrigin_Z}"
                           origin_rpy="${WristPitchFrameOrientation_Roll} ${WristPitchFrameOrientation_Pitch} ${WristPitchFrameOrientation_Yaw}">
-        <limit effort="${WristPitchTorqueLimit}" lower="${WristPitchPositionLimit_Lower}" upper="${WristPitchPositionLimit_Upper}" velocity="${AJ7_Speed_Limit}"/>
+        <limit effort="${WristPitchTorqueLimit}" lower="${WristPitchPositionLimit_Lower}" upper="${WristPitchPositionLimit_Upper}" velocity="${WristPitchVelocityLimit}"/>
     </xacro:fixed_joint>
   </xacro:macro>

File: valkyrie_description/robots/valkyrie_A/xacro/arm/joint_limits.xacro (robot description, xacro)
@@ -22,10 +22,10 @@
   <xacro:property name="WristRollPositionLimit_Upper" value="0.698" />
   <xacro:property name="WristPitchPositionLimit_Upper" value="0.436" />
-  <xacro:property name="AJ1_Speed_Limit" value="5.89" />
-  <xacro:property name="AJ2_Speed_Limit" value="5.89" />
-  <xacro:property name="AJ3_Speed_Limit" value="11.5" />
-  <xacro:property name="AJ4_Speed_Limit" value="11.5" />
-  <xacro:property name="AJ5_Speed_Limit" value="5" />
-  <xacro:property name="AJ6_Speed_Limit" value="1" />
-  <xacro:property name="AJ7_Speed_Limit" value="1" />
+  <xacro:property name="ShoulderPitchVelocityLimit" value="5.89" />
+  <xacro:property name="ShoulderRollVelocityLimit" value="5.89" />
+  <xacro:property name="ShoulderYawVelocityLimit" value="11.5" />
+  <xacro:property name="ElbowPitchVelocityLimit" value="11.5" />
+  <xacro:property name="ForearmYawVelocityLimit" value="5" />
+  <xacro:property name="WristRollVelocityLimit" value="1" />
+  <xacro:property name="WristPitchVelocityLimit" value="1" />
 </robot>

Commit message: Renamed xacro property names pertaining to arm joint names.

File: valkyrie_description/robots/valkyrie_A/xacro/arm/arm.xacro (robot description, xacro)
@@ -56,5 +56,5 @@
                     collision_mesh="${mesh_root}/aj4.stl" />
     <!-- AJ1 -->
-    <xacro:revolute_joint_ex jointName="${AJ1_Joint_Name}"
+    <xacro:revolute_joint_ex jointName="${ShoulderPitchJointName}"
                           parent="${upper_arm_root_link}" child="${AJ1_Distal_Link}"
                           origin_xyz="${ShoulderPitchFrameOrigin_X} ${ShoulderPitchFrameOrigin_Y} ${ShoulderPitchFrameOrigin_Z}"
@@ -65,5 +65,5 @@
     </xacro:revolute_joint_ex>
     <!-- AJ2 -->
-    <xacro:revolute_joint_ex jointName="${AJ2_Joint_Name}"
+    <xacro:revolute_joint_ex jointName="${ShoulderRollJointName}"
                           parent="${AJ2_Proximal_Link}" child="${AJ2_Distal_Link}"
                           origin_xyz="${ShoulderRollFrameOrigin_X} ${ShoulderRollFrameOrigin_Y} ${ShoulderRollFrameOrigin_Z}"
@@ -74,5 +74,5 @@
     </xacro:revolute_joint_ex>
     <!-- AJ3 -->
-    <xacro:revolute_joint_ex jointName="${AJ3_Joint_Name}"
+    <xacro:revolute_joint_ex jointName="${ShoulderYawJointName}"
                           parent="${AJ3_Proximal_Link}" child="${AJ3_Distal_Link}"
                           origin_xyz="${ShoulderYawFrameOrigin_X} ${ShoulderYawFrameOrigin_Y} ${ShoulderYawFrameOrigin_Z}"
@@ -83,5 +83,5 @@
     </xacro:revolute_joint_ex>
     <!-- AJ4 -->
-    <xacro:revolute_joint_ex jointName="${AJ4_Joint_Name}"
+    <xacro:revolute_joint_ex jointName="${ElbowPitchJointName}"
                           parent="${AJ4_Proximal_Link}" child="${AJ4_Distal_Link}"
                           origin_xyz="${ElbowPitchFrameOrigin_X} ${ElbowPitchFrameOrigin_Y} ${ElbowPitchFrameOrigin_Z}"
@@ -113,5 +113,5 @@
                     collision_mesh="${mesh_root}/palm_${prefix}.stl"/>
     <!-- AJ5 -->
-    <xacro:revolute_joint_ex jointName="${AJ5_Joint_Name}"
+    <xacro:revolute_joint_ex jointName="${ForearmYawJointName}"
                           parent="${lower_arm_root_link}" child="${AJ5_Distal_Link}"
                           origin_xyz="${ForearmYawFrameOrigin_X} ${ForearmYawFrameOrigin_Y} ${ForearmYawFrameOrigin_Z}"
@@ -122,5 +122,5 @@
     </xacro:revolute_joint_ex>
     <!-- AJ6 -->
-    <xacro:revolute_joint_ex jointName="${AJ6_Joint_Name}"
+    <xacro:revolute_joint_ex jointName="${WristRollJointName}"
                           parent="${AJ6_Proximal_Link}" child="${AJ6_Distal_Link}"
                           origin_xyz="${WristRollFrameOrigin_X} ${WristRollFrameOrigin_Y} ${WristRollFrameOrigin_Z}"
@@ -131,5 +131,5 @@
     </xacro:revolute_joint_ex>
     <!-- AJ7 -->
-    <xacro:revolute_joint_ex jointName="${AJ7_Joint_Name}"
+    <xacro:revolute_joint_ex jointName="${WristPitchJointName}"
                           parent="${AJ7_Proximal_Link}" child="${AJ7_Distal_Link}"
                           origin_xyz="${WristPitchFrameOrigin_X} ${WristPitchFrameOrigin_Y} ${WristPitchFrameOrigin_Z}"
@@ -168,5 +168,5 @@
                     collision_mesh="${mesh_root}/palm_${prefix}.stl"/>
     <!-- AJ5 -->
-    <xacro:fixed_joint jointName="${AJ5_Joint_Name}"
+    <xacro:fixed_joint jointName="${ForearmYawJointName}"
                           parent="${lower_arm_root_link}" child="${AJ5_Distal_Link}"
                           origin_xyz="${ForearmYawFrameOrigin_X} ${ForearmYawFrameOrigin_Y} ${ForearmYawFrameOrigin_Z}"
@@ -175,5 +175,5 @@
     </xacro:fixed_joint>
     <!-- AJ6 -->
-    <xacro:fixed_joint jointName="${AJ6_Joint_Name}"
+    <xacro:fixed_joint jointName="${WristRollJointName}"
                           parent="${AJ6_Proximal_Link}" child="${AJ6_Distal_Link}"
                           origin_xyz="${WristRollFrameOrigin_X} ${WristRollFrameOrigin_Y} ${WristRollFrameOrigin_Z}"
@@ -182,5 +182,5 @@
     </xacro:fixed_joint>
     <!-- AJ7 -->
-    <xacro:fixed_joint jointName="${AJ7_Joint_Name}"
+    <xacro:fixed_joint jointName="${WristPitchJointName}"
                           parent="${AJ7_Proximal_Link}" child="${AJ7_Distal_Link}"
                           origin_xyz="${WristPitchFrameOrigin_X} ${WristPitchFrameOrigin_Y} ${WristPitchFrameOrigin_Z}"

File: valkyrie_description/robots/valkyrie_A/xacro/arm/joint_names.xacro (robot description, xacro)
@@ -1,10 +1,10 @@
 <?xml version="1.0" ?>
 <robot xmlns:xacro="http://www.ros.org/wiki/xacro" name="v1/arm/joint_names">
-  <xacro:property name="AJ1_Joint_Name" value="${prefix}ShoulderPitch" />
-  <xacro:property name="AJ2_Joint_Name" value="${prefix}ShoulderRoll" />
-  <xacro:property name="AJ3_Joint_Name" value="${prefix}ShoulderYaw" />
-  <xacro:property name="AJ4_Joint_Name" value="${prefix}ElbowPitch" />
-  <xacro:property name="AJ5_Joint_Name" value="${prefix}ForearmYaw" />
-  <xacro:property name="AJ6_Joint_Name" value="${prefix}WristPitch" />
-  <xacro:property name="AJ7_Joint_Name" value="${prefix}WristRoll" />
+  <xacro:property name="ShoulderPitchJointName" value="${prefix}ShoulderPitch" />
+  <xacro:property name="ShoulderRollJointName" value="${prefix}ShoulderRoll" />
+  <xacro:property name="ShoulderYawJointName" value="${prefix}ShoulderYaw" />
+  <xacro:property name="ElbowPitchJointName" value="${prefix}ElbowPitch" />
+  <xacro:property name="ForearmYawJointName" value="${prefix}ForearmYaw" />
+  <xacro:property name="WristRollJointName" value="${prefix}WristPitch" />
+  <xacro:property name="WristPitchJointName" value="${prefix}WristRoll" />
 </robot>
