Commit message: Renamed the link name properties for the arm links.

File: valkyrie_description/robots/valkyrie_A/xacro/arm/arm.xacro (robot description, xacro)
@@ -30,5 +30,5 @@
   <xacro:macro name="make_upper_arm" params="prefix reflect upper_arm_root_link">
     <!-- LINKS -->
-    <xacro:box_link name="${AJ1_Distal_Link}"
+    <xacro:box_link name="${ShoulderPitchLink}"
                     width="${AJ1_Link_Width}" height="${AJ1_Link_Height}" depth="${AJ1_Link_Length}" mass="${AJ1_Link_Mass}"
                     origin_xyz="0 -0.01204 ${reflect * -0.251}" origin_rpy="0 0 0"
@@ -36,5 +36,5 @@
                     material="Gold"
                     collision_mesh="${mesh_root}/aj1_${prefix}.stl" />
-    <xacro:box_link name="${AJ2_Distal_Link}"
+    <xacro:box_link name="${ShoulderRollLink}"
                     width="${AJ2_Link_Width}" height="${AJ2_Link_Height}" depth="${AJ2_Link_Length}" mass="${AJ2_Link_Mass}"
                     origin_xyz="0.04 0.005 ${reflect * -0.02}" origin_rpy="0 0 0"
@@ -42,5 +42,5 @@
                     material="White"
                     collision_mesh="${mesh_root}/aj2.stl" />
-    <xacro:box_link name="${AJ3_Distal_Link}"
+    <xacro:box_link name="${ShoulderYawLink}"
                     width="${AJ3_Link_Width}" height="${AJ3_Link_Height}" depth="${AJ3_Link_Length}" mass="${AJ3_Link_Mass}"
                     origin_xyz="${reflect * 0.02} ${reflect * -0.004} ${reflect * -0.273}" origin_rpy="0 0 0"
@@ -48,5 +48,5 @@
                     material="White"
                     collision_mesh="${mesh_root}/aj3_${prefix}.stl" />
-    <xacro:box_link name="${AJ4_Distal_Link}"
+    <xacro:box_link name="${ElbowPitchLink}"
                     width="${AJ4_Link_Width}" height="${AJ4_Link_Height}" depth="${AJ4_Link_Length}" mass="${AJ4_Link_Mass}"
                     origin_rpy="0 0 0"
@@ -57,5 +57,5 @@
     <!-- AJ1 -->
     <xacro:revolute_joint_ex jointName="${ShoulderPitchJointName}"
-                          parent="${upper_arm_root_link}" child="${AJ1_Distal_Link}"
+                          parent="${upper_arm_root_link}" child="${ShoulderPitchLink}"
                           origin_xyz="${ShoulderPitchFrameOrigin_X} ${ShoulderPitchFrameOrigin_Y} ${ShoulderPitchFrameOrigin_Z}"
                           origin_rpy="${ShoulderPitchFrameOrientation_Roll} ${ShoulderPitchFrameOrientation_Pitch} ${ShoulderPitchFrameOrientation_Yaw}"
@@ -66,5 +66,5 @@
     <!-- AJ2 -->
     <xacro:revolute_joint_ex jointName="${ShoulderRollJointName}"
-                          parent="${AJ2_Proximal_Link}" child="${AJ2_Distal_Link}"
+                          parent="${ShoulderPitchLink}" child="${ShoulderRollLink}"
                           origin_xyz="${ShoulderRollFrameOrigin_X} ${ShoulderRollFrameOrigin_Y} ${ShoulderRollFrameOrigin_Z}"
                           origin_rpy="${ShoulderRollFrameOrientation_Roll} ${ShoulderRollFrameOrientation_Pitch} ${ShoulderRollFrameOrientation_Yaw}"
@@ -75,5 +75,5 @@
     <!-- AJ3 -->
     <xacro:revolute_joint_ex jointName="${ShoulderYawJointName}"
-                          parent="${AJ3_Proximal_Link}" child="${AJ3_Distal_Link}"
+                          parent="${ShoulderRollLink}" child="${ShoulderYawLink}"
                           origin_xyz="${ShoulderYawFrameOrigin_X} ${ShoulderYawFrameOrigin_Y} ${ShoulderYawFrameOrigin_Z}"
                           origin_rpy="${ShoulderYawFrameOrientation_Roll} ${ShoulderYawFrameOrientation_Pitch} ${ShoulderYawFrameOrientation_Yaw}"
@@ -84,5 +84,5 @@
     <!-- AJ4 -->
     <xacro:revolute_joint_ex jointName="${ElbowPitchJointName}"
-                          parent="${AJ4_Proximal_Link}" child="${AJ4_Distal_Link}"
+                          parent="${ShoulderYawLink}" child="${ElbowPitchLink}"
                           origin_xyz="${ElbowPitchFrameOrigin_X} ${ElbowPitchFrameOrigin_Y} ${ElbowPitchFrameOrigin_Z}"
                           origin_rpy="${ElbowPitchFrameOrientation_Roll} ${ElbowPitchFrameOrientation_Pitch} ${ElbowPitchFrameOrientation_Yaw}"
@@ -94,5 +94,5 @@
   <xacro:macro name="make_lower_arm" params="prefix reflect lower_arm_root_link">
     <!-- LINKS -->
-    <xacro:box_link name="${AJ5_Distal_Link}"
+    <xacro:box_link name="${ForearmLinkName}"
                     width="${AJ5_Link_Width}" height="${AJ5_Link_Height}" depth="${AJ5_Link_Length}" mass="${AJ5_Link_Mass}"
                     origin_rpy="0 0 0"
@@ -101,9 +101,9 @@
                     material="White"
                     collision_mesh="${mesh_root}/aj5_${prefix}.stl" />
-    <xacro:box_link_no_mesh name="${AJ6_Distal_Link}"
+    <xacro:box_link_no_mesh name="${WristRollLinkName}"
                     width="${AJ6_Link_Width}" height="${AJ6_Link_Height}" depth="${AJ6_Link_Length}" mass="${AJ6_Link_Mass}"
                     origin_rpy="0 0 0"
                     origin_xyz="0 0 0"/>
-    <xacro:box_link name="${AJ7_Distal_Link}"
+    <xacro:box_link name="${WristPitchLinkName}"
                     width="${AJ7_Link_Width}" height="${AJ7_Link_Height}" depth="${AJ7_Link_Length}" mass="${AJ7_Link_Mass}"
                     origin_rpy="0 0 0"
@@ -114,5 +114,5 @@
     <!-- AJ5 -->
     <xacro:revolute_joint_ex jointName="${ForearmYawJointName}"
-                          parent="${lower_arm_root_link}" child="${AJ5_Distal_Link}"
+                          parent="${lower_arm_root_link}" child="${ForearmLinkName}"
                           origin_xyz="${ForearmYawFrameOrigin_X} ${ForearmYawFrameOrigin_Y} ${ForearmYawFrameOrigin_Z}"
                           origin_rpy="${ForearmYawFrameOrientation_Roll} ${ForearmYawFrameOrientation_Pitch} ${ForearmYawFrameOrientation_Yaw}"
@@ -123,5 +123,5 @@
     <!-- AJ6 -->
     <xacro:revolute_joint_ex jointName="${WristRollJointName}"
-                          parent="${AJ6_Proximal_Link}" child="${AJ6_Distal_Link}"
+                          parent="${ForearmLinkName}" child="${WristRollLinkName}"
                           origin_xyz="${WristRollFrameOrigin_X} ${WristRollFrameOrigin_Y} ${WristRollFrameOrigin_Z}"
                           origin_rpy="${WristRollFrameOrientation_Roll} ${WristRollFrameOrientation_Pitch} ${WristRollFrameOrientation_Yaw}"
@@ -132,5 +132,5 @@
     <!-- AJ7 -->
     <xacro:revolute_joint_ex jointName="${WristPitchJointName}"
-                          parent="${AJ7_Proximal_Link}" child="${AJ7_Distal_Link}"
+                          parent="${WristRollLinkName}" child="${WristPitchLinkName}"
                           origin_xyz="${WristPitchFrameOrigin_X} ${WristPitchFrameOrigin_Y} ${WristPitchFrameOrigin_Z}"
                           origin_rpy="${WristPitchFrameOrientation_Roll} ${WristPitchFrameOrientation_Pitch} ${WristPitchFrameOrientation_Yaw}"
@@ -142,5 +142,5 @@
   <xacro:macro name="make_lower_arm_fixed" params="prefix reflect lower_arm_root_link">
     <!-- LINKS -->
-    <xacro:box_link name="${AJ5_Distal_Link}"
+    <xacro:box_link name="${ForearmLinkName}"
                     width="${AJ5_Link_Width}" height="${AJ5_Link_Height}" depth="${AJ5_Link_Length}" mass="${AJ5_Link_Mass}"
                     origin_rpy="0 0 0"
@@ -149,5 +149,5 @@
                     material="White"
                     collision_mesh="${mesh_root}/aj5_${prefix}.stl" />
-<!--     <xacro:box_link name="${AJ5_Distal_Link}"
+<!--     <xacro:box_link name="${ForearmLinkName}"
                     width="${AJ5_Link_Width}" height="${AJ5_Link_Height}" depth="${AJ5_Link_Length}" mass="${AJ5_Link_Mass}"
                     origin_rpy="0 0 0"
@@ -156,9 +156,9 @@
                     material="White"
                     collision_mesh="${mesh_root}/aj5_${prefix}.stl" />
- -->    <xacro:box_link_no_mesh name="${AJ6_Distal_Link}"
+ -->    <xacro:box_link_no_mesh name="${WristRollLinkName}"
                     width="${AJ6_Link_Width}" height="${AJ6_Link_Height}" depth="${AJ6_Link_Length}" mass="${AJ6_Link_Mass}"
                     origin_rpy="0 0 0"
                     origin_xyz="0 0 0"/>
-    <xacro:box_link name="${AJ7_Distal_Link}"
+    <xacro:box_link name="${WristPitchLinkName}"
                     width="${AJ7_Link_Width}" height="${AJ7_Link_Height}" depth="${AJ7_Link_Length}" mass="${AJ7_Link_Mass}"
                     origin_rpy="0 0 0"
@@ -169,5 +169,5 @@
     <!-- AJ5 -->
     <xacro:fixed_joint jointName="${ForearmYawJointName}"
-                          parent="${lower_arm_root_link}" child="${AJ5_Distal_Link}"
+                          parent="${lower_arm_root_link}" child="${ForearmLinkName}"
                           origin_xyz="${ForearmYawFrameOrigin_X} ${ForearmYawFrameOrigin_Y} ${ForearmYawFrameOrigin_Z}"
                           origin_rpy="${ForearmYawFrameOrientation_Roll} ${ForearmYawFrameOrientation_Pitch} ${ForearmYawFrameOrientation_Yaw}">
@@ -176,5 +176,5 @@
     <!-- AJ6 -->
     <xacro:fixed_joint jointName="${WristRollJointName}"
-                          parent="${AJ6_Proximal_Link}" child="${AJ6_Distal_Link}"
+                          parent="${ForearmLinkName}" child="${WristRollLinkName}"
                           origin_xyz="${WristRollFrameOrigin_X} ${WristRollFrameOrigin_Y} ${WristRollFrameOrigin_Z}"
                           origin_rpy="${WristRollFrameOrientation_Roll} ${WristRollFrameOrientation_Pitch} ${WristRollFrameOrientation_Yaw}">
@@ -183,5 +183,5 @@
     <!-- AJ7 -->
     <xacro:fixed_joint jointName="${WristPitchJointName}"
-                          parent="${AJ7_Proximal_Link}" child="${AJ7_Distal_Link}"
+                          parent="${WristRollLinkName}" child="${WristPitchLinkName}"
                           origin_xyz="${WristPitchFrameOrigin_X} ${WristPitchFrameOrigin_Y} ${WristPitchFrameOrigin_Z}"
                           origin_rpy="${WristPitchFrameOrientation_Roll} ${WristPitchFrameOrientation_Pitch} ${WristPitchFrameOrientation_Yaw}">
@@ -191,5 +191,5 @@
   <xacro:macro name="make_arm" params="prefix reflect arm_root_link">
     <xacro:make_upper_arm prefix="${prefix}" reflect="${reflect}" upper_arm_root_link="${arm_root_link}" />
-    <xacro:make_lower_arm prefix="${prefix}" reflect="${reflect}" lower_arm_root_link="${AJ5_Proximal_Link}" />
+    <xacro:make_lower_arm prefix="${prefix}" reflect="${reflect}" lower_arm_root_link="${ElbowPitchLink}" />
   </xacro:macro>
   <!-- Sensors -->

File: valkyrie_description/robots/valkyrie_A/xacro/arm/link_names.xacro (robot description, xacro)
@@ -1,17 +1,12 @@
 <?xml version="1.0" ?>
 <robot xmlns:xacro="http://www.ros.org/wiki/xacro" name="v1/arm/link_names">
-  <xacro:property name="AJ1_Proximal_Link" value="${arm_root_link}" />
-  <xacro:property name="AJ1_Distal_Link" value="${prefix}ShoulderPitch" />
-  <xacro:property name="AJ2_Proximal_Link" value="${prefix}ShoulderPitch" />
-  <xacro:property name="AJ2_Distal_Link" value="${prefix}ShoulderRoll" />
-  <xacro:property name="AJ3_Proximal_Link" value="${prefix}ShoulderRoll" />
-  <xacro:property name="AJ3_Distal_Link" value="${prefix}ShoulderYaw" />
-  <xacro:property name="AJ4_Proximal_Link" value="${prefix}ShoulderYaw" />
-  <xacro:property name="AJ4_Distal_Link" value="${prefix}ElbowPitch" />
-  <xacro:property name="AJ5_Proximal_Link" value="${prefix}ElbowPitch" />
-  <xacro:property name="AJ5_Distal_Link" value="${prefix}Forearm" />
-  <xacro:property name="AJ6_Proximal_Link" value="${prefix}Forearm" />
-  <xacro:property name="AJ6_Distal_Link" value="${prefix}WristPitch" />
-  <xacro:property name="AJ7_Proximal_Link" value="${prefix}WristPitch" />
-  <xacro:property name="AJ7_Distal_Link" value="${prefix}Palm" />
+  <xacro:property name="ShoulderPitchParentLink" value="${arm_root_link}" />
+  <xacro:property name="ShoulderPitchLink" value="${prefix}ShoulderPitchLink" />
+  <xacro:property name="ShoulderRollLink" value="${prefix}ShoulderRollLink" />
+  <xacro:property name="ShoulderYawLink" value="${prefix}ShoulderYawLink" />
+  <xacro:property name="ElbowPitchLink" value="${prefix}ElbowPitchLink" />
+  <xacro:property name="ElbowPitchLink" value="${prefix}ElbowPitchLink" />
+  <xacro:property name="ForearmLinkName" value="${prefix}ForearmLink" />
+  <xacro:property name="WristRollLinkName" value="${prefix}WristRollLink" />
+  <xacro:property name="WristPitchLinkName" value="${prefix}PalmLink" />
 </robot>

File: valkyrie_description/robots/valkyrie_A/xacro/head/link_names.xacro (robot description, xacro)
@@ -4,4 +4,4 @@
   <xacro:property name="LowerNeckPitchLinkName" value="LowerNeckPitchLink" />
   <xacro:property name="NeckYawLinkName" value="NeckYawLink" />
-  <xacro:property name="UpperNeckPitchLinkName" value="Head" />
+  <xacro:property name="UpperNeckPitchLinkName" value="HeadLink" />
 </robot>
