Commit message: Think I finished renaming arm stuff. At least for a first pass.

File: valkyrie_description/robots/valkyrie_A/xacro/arm/arm.xacro (robot description, xacro)
@@ -31,5 +31,5 @@
     <!-- LINKS -->
     <xacro:box_link name="${ShoulderPitchLink}"
-                    width="${AJ1_Link_Width}" height="${AJ1_Link_Height}" depth="${AJ1_Link_Length}" mass="${AJ1_Link_Mass}"
+                    width="${AJ1_Link_Width}" height="${AJ1_Link_Height}" depth="${AJ1_Link_Length}" mass="${ShoulderPitchLinkMass}"
                     origin_xyz="0 -0.01204 ${reflect * -0.251}" origin_rpy="0 0 0"
                     visual_mesh="${mesh_root}/aj1_${prefix}.stl"
@@ -37,5 +37,5 @@
                     collision_mesh="${mesh_root}/aj1_${prefix}.stl" />
     <xacro:box_link name="${ShoulderRollLink}"
-                    width="${AJ2_Link_Width}" height="${AJ2_Link_Height}" depth="${AJ2_Link_Length}" mass="${AJ2_Link_Mass}"
+                    width="${AJ2_Link_Width}" height="${AJ2_Link_Height}" depth="${AJ2_Link_Length}" mass="${ShoulderRollLinkMass}"
                     origin_xyz="0.04 0.005 ${reflect * -0.02}" origin_rpy="0 0 0"
                     visual_mesh="${mesh_root}/aj2.stl"
@@ -43,5 +43,5 @@
                     collision_mesh="${mesh_root}/aj2.stl" />
     <xacro:box_link name="${ShoulderYawLink}"
-                    width="${AJ3_Link_Width}" height="${AJ3_Link_Height}" depth="${AJ3_Link_Length}" mass="${AJ3_Link_Mass}"
+                    width="${AJ3_Link_Width}" height="${AJ3_Link_Height}" depth="${AJ3_Link_Length}" mass="${ShoulderYawLinkMass}"
                     origin_xyz="${reflect * 0.02} ${reflect * -0.004} ${reflect * -0.273}" origin_rpy="0 0 0"
                     visual_mesh="${mesh_root}/aj3_${prefix}.stl"
@@ -49,5 +49,5 @@
                     collision_mesh="${mesh_root}/aj3_${prefix}.stl" />
     <xacro:box_link name="${ElbowPitchLink}"
-                    width="${AJ4_Link_Width}" height="${AJ4_Link_Height}" depth="${AJ4_Link_Length}" mass="${AJ4_Link_Mass}"
+                    width="${AJ4_Link_Width}" height="${AJ4_Link_Height}" depth="${AJ4_Link_Length}" mass="${ElbowPitchLinkMass}"
                     origin_rpy="0 0 0"
                     origin_xyz="0.0270 -0.0802 0"
@@ -95,5 +95,5 @@
     <!-- LINKS -->
     <xacro:box_link name="${ForearmLinkName}"
-                    width="${AJ5_Link_Width}" height="${AJ5_Link_Height}" depth="${AJ5_Link_Length}" mass="${AJ5_Link_Mass}"
+                    width="${AJ5_Link_Width}" height="${AJ5_Link_Height}" depth="${AJ5_Link_Length}" mass="${ForearmYawLinkMass}"
                     origin_rpy="0 0 0"
                     origin_xyz="0.015 ${reflect * 0.02} ${reflect * -0.11}"
@@ -102,9 +102,9 @@
                     collision_mesh="${mesh_root}/aj5_${prefix}.stl" />
     <xacro:box_link_no_mesh name="${WristRollLinkName}"
-                    width="${AJ6_Link_Width}" height="${AJ6_Link_Height}" depth="${AJ6_Link_Length}" mass="${AJ6_Link_Mass}"
+                    width="${AJ6_Link_Width}" height="${AJ6_Link_Height}" depth="${AJ6_Link_Length}" mass="${WristRollLinkMass}"
                     origin_rpy="0 0 0"
                     origin_xyz="0 0 0"/>
     <xacro:box_link name="${WristPitchLinkName}"
-                    width="${AJ7_Link_Width}" height="${AJ7_Link_Height}" depth="${AJ7_Link_Length}" mass="${AJ7_Link_Mass}"
+                    width="${AJ7_Link_Width}" height="${AJ7_Link_Height}" depth="${AJ7_Link_Length}" mass="${PalmMass}"
                     origin_rpy="0 0 0"
                     origin_xyz="${AJ7_Link_Width/2} 0 0"
@@ -143,5 +143,5 @@
     <!-- LINKS -->
     <xacro:box_link name="${ForearmLinkName}"
-                    width="${AJ5_Link_Width}" height="${AJ5_Link_Height}" depth="${AJ5_Link_Length}" mass="${AJ5_Link_Mass}"
+                    width="${AJ5_Link_Width}" height="${AJ5_Link_Height}" depth="${AJ5_Link_Length}" mass="${ForearmYawLinkMass}"
                     origin_rpy="0 0 0"
                     origin_xyz="0 ${reflect * 0.0006} ${reflect * -0.14}"
@@ -150,5 +150,5 @@
                     collision_mesh="${mesh_root}/aj5_${prefix}.stl" />
 <!--     <xacro:box_link name="${ForearmLinkName}"
-                    width="${AJ5_Link_Width}" height="${AJ5_Link_Height}" depth="${AJ5_Link_Length}" mass="${AJ5_Link_Mass}"
+                    width="${AJ5_Link_Width}" height="${AJ5_Link_Height}" depth="${AJ5_Link_Length}" mass="${ForearmYawLinkMass}"
                     origin_rpy="0 0 0"
                     origin_xyz="0 ${reflect * 0.0006} ${reflect * -0.176}"
@@ -157,9 +157,9 @@
                     collision_mesh="${mesh_root}/aj5_${prefix}.stl" />
  -->    <xacro:box_link_no_mesh name="${WristRollLinkName}"
-                    width="${AJ6_Link_Width}" height="${AJ6_Link_Height}" depth="${AJ6_Link_Length}" mass="${AJ6_Link_Mass}"
+                    width="${AJ6_Link_Width}" height="${AJ6_Link_Height}" depth="${AJ6_Link_Length}" mass="${WristRollLinkMass}"
                     origin_rpy="0 0 0"
                     origin_xyz="0 0 0"/>
     <xacro:box_link name="${WristPitchLinkName}"
-                    width="${AJ7_Link_Width}" height="${AJ7_Link_Height}" depth="${AJ7_Link_Length}" mass="${AJ7_Link_Mass}"
+                    width="${AJ7_Link_Width}" height="${AJ7_Link_Height}" depth="${AJ7_Link_Length}" mass="${PalmMass}"
                     origin_rpy="0 0 0"
                     origin_xyz="${AJ7_Link_Width/2} 0 0"

File: valkyrie_description/robots/valkyrie_A/xacro/arm/frame_parameters.xacro (robot description, xacro)
@@ -4,42 +4,42 @@
   <xacro:property name="ShoulderPitchFrameOrigin_Y" value="0"/>
   <xacro:property name="ShoulderPitchFrameOrigin_Z" value="-0.03157"/>
-  <xacro:property name="ShoulderPitchFrameOrientation_Roll" value="${pi_2}"/>
-  <xacro:property name="ShoulderPitchFrameOrientation_Pitch" value="0"/>
-  <xacro:property name="ShoulderPitchFrameOrientation_Yaw" value="0"/>
+  <xacro:property name="ShoulderPitchFrameOrientation_Roll" value="0.0"/>
+  <xacro:property name="ShoulderPitchFrameOrientation_Pitch" value="0.0"/>
+  <xacro:property name="ShoulderPitchFrameOrientation_Yaw" value="0.0"/>
   <xacro:property name="ShoulderRollFrameOrigin_X" value="0"/>
   <xacro:property name="ShoulderRollFrameOrigin_Y" value="0"/>
   <xacro:property name="ShoulderRollFrameOrigin_Z" value="${reflect * -0.246}"/>
-  <xacro:property name="ShoulderRollFrameOrientation_Roll" value="${reflect * (pi_2)}"/>
-  <xacro:property name="ShoulderRollFrameOrientation_Pitch" value="0"/>
-  <xacro:property name="ShoulderRollFrameOrientation_Yaw" value="${pi}"/>
-  <xacro:property name="ShoulderYawFrameOrigin_X" value="0"/>
-  <xacro:property name="ShoulderYawFrameOrigin_Y" value="0"/>
-  <xacro:property name="ShoulderYawFrameOrigin_Z" value="0"/>
-  <xacro:property name="ShoulderYawFrameOrientation_Roll" value="${-1 * pi_2}"/>
-  <xacro:property name="ShoulderYawFrameOrientation_Pitch" value="0"/>
-  <xacro:property name="ShoulderYawFrameOrientation_Yaw" value="${reflect * pi_2}"/>
+  <xacro:property name="ShoulderRollFrameOrientation_Roll" value="0.0"/>
+  <xacro:property name="ShoulderRollFrameOrientation_Pitch" value="0.0"/>
+  <xacro:property name="ShoulderRollFrameOrientation_Yaw" value="0.0"/>
+  <xacro:property name="ShoulderYawFrameOrigin_X" value="0.0"/>
+  <xacro:property name="ShoulderYawFrameOrigin_Y" value="0.0"/>
+  <xacro:property name="ShoulderYawFrameOrigin_Z" value="0.0"/>
+  <xacro:property name="ShoulderYawFrameOrientation_Roll" value="0.0"/>
+  <xacro:property name="ShoulderYawFrameOrientation_Pitch" value="0.0"/>
+  <xacro:property name="ShoulderYawFrameOrientation_Yaw" value="0.0"/>
   <xacro:property name="ElbowPitchFrameOrigin_X" value="0"/>
   <xacro:property name="ElbowPitchFrameOrigin_Y" value="${reflect * -0.0254}"/>
   <xacro:property name="ElbowPitchFrameOrigin_Z" value="${reflect * -0.330}"/>
-  <xacro:property name="ElbowPitchFrameOrientation_Roll" value="${reflect * pi_2}"/>
-  <xacro:property name="ElbowPitchFrameOrientation_Pitch" value="0"/>
-  <xacro:property name="ElbowPitchFrameOrientation_Yaw" value="${reflect * pi_2}"/>
+  <xacro:property name="ElbowPitchFrameOrientation_Roll" value="0.0"/>
+  <xacro:property name="ElbowPitchFrameOrientation_Pitch" value="0.0"/>
+  <xacro:property name="ElbowPitchFrameOrientation_Yaw" value="0.0"/>
   <xacro:property name="ForearmYawFrameOrigin_X" value="0.0254"/>
   <xacro:property name="ForearmYawFrameOrigin_Y" value="0"/>
   <xacro:property name="ForearmYawFrameOrigin_Z" value="0"/>
-  <xacro:property name="ForearmYawFrameOrientation_Roll" value="${reflect * pi_2}"/>
-  <xacro:property name="ForearmYawFrameOrientation_Pitch" value="0"/>
-  <xacro:property name="ForearmYawFrameOrientation_Yaw" value="${pi}"/>
+  <xacro:property name="ForearmYawFrameOrientation_Roll" value="0.0"/>
+  <xacro:property name="ForearmYawFrameOrientation_Pitch" value="0.0"/>
+  <xacro:property name="ForearmYawFrameOrientation_Yaw" value="0.0"/>
   <xacro:property name="WristRollFrameOrigin_X" value="0"/>
   <xacro:property name="WristRollFrameOrigin_Y" value="0"/>
   <xacro:property name="WristRollFrameOrigin_Z" value="${reflect * -0.287}"/>
-  <xacro:property name="WristRollFrameOrientation_Roll" value="${-1 * pi_2}"/>
-  <xacro:property name="WristRollFrameOrientation_Pitch" value="0"/>
-  <xacro:property name="WristRollFrameOrientation_Yaw" value="${reflect * pi_2}"/>
-  <xacro:property name="WristPitchFrameOrigin_X" value="0"/>
-  <xacro:property name="WristPitchFrameOrigin_Y" value="0"/>
-  <xacro:property name="WristPitchFrameOrigin_Z" value="0"/>
-  <xacro:property name="WristPitchFrameOrientation_Roll" value="${reflect * pi_2}"/>
-  <xacro:property name="WristPitchFrameOrientation_Pitch" value="0"/>
-  <xacro:property name="WristPitchFrameOrientation_Yaw" value="${reflect * pi_2}"/>
+  <xacro:property name="WristRollFrameOrientation_Roll" value="0.0"/>
+  <xacro:property name="WristRollFrameOrientation_Pitch" value="0.0"/>
+  <xacro:property name="WristRollFrameOrientation_Yaw" value="0.0"/>
+  <xacro:property name="WristPitchFrameOrigin_X" value="0.0"/>
+  <xacro:property name="WristPitchFrameOrigin_Y" value="0.0"/>
+  <xacro:property name="WristPitchFrameOrigin_Z" value="0.0"/>
+  <xacro:property name="WristPitchFrameOrientation_Roll" value="0.0"/>
+  <xacro:property name="WristPitchFrameOrientation_Pitch" value="0.0"/>
+  <xacro:property name="WristPitchFrameOrientation_Yaw" value="0.0"/>
 </robot>

File: valkyrie_description/robots/valkyrie_A/xacro/arm/mass_parameters.xacro (robot description, xacro)
@@ -1,10 +1,10 @@
 <?xml version="1.0" ?>
 <robot xmlns:xacro="http://www.ros.org/wiki/xacro" name="v1/arm/mass_parameters">
-  <xacro:property name="AJ1_Link_Mass" value="2.65" />
-  <xacro:property name="AJ2_Link_Mass" value="2.87" />
-  <xacro:property name="AJ3_Link_Mass" value="2.575" />
-  <xacro:property name="AJ4_Link_Mass" value="2.367" />
-  <xacro:property name="AJ5_Link_Mass" value="2.903" />
-  <xacro:property name="AJ6_Link_Mass" value="0.1" />
-  <xacro:property name="AJ7_Link_Mass" value="0.712" />
+  <xacro:property name="ShoulderPitchLinkMass" value="2.65" />
+  <xacro:property name="ShoulderRollLinkMass" value="2.87" />
+  <xacro:property name="ShoulderYawLinkMass" value="2.575" />
+  <xacro:property name="ElbowPitchLinkMass" value="2.367" />
+  <xacro:property name="ForearmYawLinkMass" value="2.903" />
+  <xacro:property name="WristRollLinkMass" value="0.1" />
+  <xacro:property name="PalmMass" value="0.712" />
 </robot>
