Commit message: Renamed a bunch of middle finger xacro properties and fixed an arm naming typo I had.

File: valkyrie_description/robots/valkyrie_A/xacro/arm/arm.xacro (robot description, xacro)
@@ -30,5 +30,5 @@
   <xacro:macro name="make_upper_arm" params="prefix reflect upper_arm_root_link">
     <!-- LINKS -->
-    <xacro:box_link name="${ShoulderPitchLink}"
+    <xacro:box_link name="${ShoulderPitchLinkName}"
                     width="${AJ1_Link_Width}" height="${AJ1_Link_Height}" depth="${AJ1_Link_Length}" mass="${ShoulderPitchLinkMass}"
                     origin_xyz="0 -0.01204 ${reflect * -0.251}" origin_rpy="0 0 0"
@@ -36,5 +36,5 @@
                     material="Gold"
                     collision_mesh="${mesh_root}/aj1_${prefix}.stl" />
-    <xacro:box_link name="${ShoulderRollLink}"
+    <xacro:box_link name="${ShoulderRollLinkName}"
                     width="${AJ2_Link_Width}" height="${AJ2_Link_Height}" depth="${AJ2_Link_Length}" mass="${ShoulderRollLinkMass}"
                     origin_xyz="0.04 0.005 ${reflect * -0.02}" origin_rpy="0 0 0"
@@ -42,5 +42,5 @@
                     material="White"
                     collision_mesh="${mesh_root}/aj2.stl" />
-    <xacro:box_link name="${ShoulderYawLink}"
+    <xacro:box_link name="${ShoulderYawLinkName}"
                     width="${AJ3_Link_Width}" height="${AJ3_Link_Height}" depth="${AJ3_Link_Length}" mass="${ShoulderYawLinkMass}"
                     origin_xyz="${reflect * 0.02} ${reflect * -0.004} ${reflect * -0.273}" origin_rpy="0 0 0"
@@ -48,5 +48,5 @@
                     material="White"
                     collision_mesh="${mesh_root}/aj3_${prefix}.stl" />
-    <xacro:box_link name="${ElbowPitchLink}"
+    <xacro:box_link name="${ElbowPitchLinkName}"
                     width="${AJ4_Link_Width}" height="${AJ4_Link_Height}" depth="${AJ4_Link_Length}" mass="${ElbowPitchLinkMass}"
                     origin_rpy="0 0 0"
@@ -57,5 +57,5 @@
     <!-- AJ1 -->
     <xacro:revolute_joint_ex jointName="${ShoulderPitchJointName}"
-                          parent="${upper_arm_root_link}" child="${ShoulderPitchLink}"
+                          parent="${upper_arm_root_link}" child="${ShoulderPitchLinkName}"
                           origin_xyz="${ShoulderPitchFrameOrigin_X} ${ShoulderPitchFrameOrigin_Y} ${ShoulderPitchFrameOrigin_Z}"
                           origin_rpy="${ShoulderPitchFrameOrientation_Roll} ${ShoulderPitchFrameOrientation_Pitch} ${ShoulderPitchFrameOrientation_Yaw}"
@@ -66,5 +66,5 @@
     <!-- AJ2 -->
     <xacro:revolute_joint_ex jointName="${ShoulderRollJointName}"
-                          parent="${ShoulderPitchLink}" child="${ShoulderRollLink}"
+                          parent="${ShoulderPitchLinkName}" child="${ShoulderRollLinkName}"
                           origin_xyz="${ShoulderRollFrameOrigin_X} ${ShoulderRollFrameOrigin_Y} ${ShoulderRollFrameOrigin_Z}"
                           origin_rpy="${ShoulderRollFrameOrientation_Roll} ${ShoulderRollFrameOrientation_Pitch} ${ShoulderRollFrameOrientation_Yaw}"
@@ -75,5 +75,5 @@
     <!-- AJ3 -->
     <xacro:revolute_joint_ex jointName="${ShoulderYawJointName}"
-                          parent="${ShoulderRollLink}" child="${ShoulderYawLink}"
+                          parent="${ShoulderRollLinkName}" child="${ShoulderYawLinkName}"
                           origin_xyz="${ShoulderYawFrameOrigin_X} ${ShoulderYawFrameOrigin_Y} ${ShoulderYawFrameOrigin_Z}"
                           origin_rpy="${ShoulderYawFrameOrientation_Roll} ${ShoulderYawFrameOrientation_Pitch} ${ShoulderYawFrameOrientation_Yaw}"
@@ -84,5 +84,5 @@
     <!-- AJ4 -->
     <xacro:revolute_joint_ex jointName="${ElbowPitchJointName}"
-                          parent="${ShoulderYawLink}" child="${ElbowPitchLink}"
+                          parent="${ShoulderYawLinkName}" child="${ElbowPitchLinkName}"
                           origin_xyz="${ElbowPitchFrameOrigin_X} ${ElbowPitchFrameOrigin_Y} ${ElbowPitchFrameOrigin_Z}"
                           origin_rpy="${ElbowPitchFrameOrientation_Roll} ${ElbowPitchFrameOrientation_Pitch} ${ElbowPitchFrameOrientation_Yaw}"
@@ -191,5 +191,5 @@
   <xacro:macro name="make_arm" params="prefix reflect arm_root_link">
     <xacro:make_upper_arm prefix="${prefix}" reflect="${reflect}" upper_arm_root_link="${arm_root_link}" />
-    <xacro:make_lower_arm prefix="${prefix}" reflect="${reflect}" lower_arm_root_link="${ElbowPitchLink}" />
+    <xacro:make_lower_arm prefix="${prefix}" reflect="${reflect}" lower_arm_root_link="${ElbowPitchLinkName}" />
   </xacro:macro>
   <!-- Sensors -->

File: valkyrie_description/robots/valkyrie_A/xacro/arm/link_names.xacro (robot description, xacro)
@@ -1,10 +1,9 @@
 <?xml version="1.0" ?>
 <robot xmlns:xacro="http://www.ros.org/wiki/xacro" name="v1/arm/link_names">
-  <xacro:property name="ShoulderPitchParentLink" value="${arm_root_link}" />
-  <xacro:property name="ShoulderPitchLink" value="${prefix}ShoulderPitchLink" />
-  <xacro:property name="ShoulderRollLink" value="${prefix}ShoulderRollLink" />
-  <xacro:property name="ShoulderYawLink" value="${prefix}ShoulderYawLink" />
-  <xacro:property name="ElbowPitchLink" value="${prefix}ElbowPitchLink" />
-  <xacro:property name="ElbowPitchLink" value="${prefix}ElbowPitchLink" />
+  <xacro:property name="ShoulderPitchParentLinkName" value="${arm_root_link}" />
+  <xacro:property name="ShoulderPitchLinkName" value="${prefix}ShoulderPitchLink" />
+  <xacro:property name="ShoulderRollLinkName" value="${prefix}ShoulderRollLink" />
+  <xacro:property name="ShoulderYawLinkName" value="${prefix}ShoulderYawLink" />
+  <xacro:property name="ElbowPitchLinkName" value="${prefix}ElbowPitchLink" />
   <xacro:property name="ForearmLinkName" value="${prefix}ForearmLink" />
   <xacro:property name="WristRollLinkName" value="${prefix}WristRollLink" />

File: valkyrie_description/robots/valkyrie_A/xacro/little_finger/link_names.xacro (robot description, xacro)
@@ -2,7 +2,7 @@
 <robot xmlns:xacro="http://www.ros.org/wiki/xacro" name="v1/little_finger/dh_parameters">
   <xacro:property name="PinkyPitch1ParentLinkName" value="${little_finger_root_link}" />
-  <xacro:property name="PinkyPitch1LinkName" value="${prefix}PinkyPitch1" />
-  <xacro:property name="PinkyPitch2LinkName" value="${prefix}PinkyPitch2" />
-  <xacro:property name="PinkyPitch3LinkName" value="${prefix}PinkyPitch3" />
-  <xacro:property name="PinkyPitch4LinkName" value="${prefix}PinkyPitch4" />
+  <xacro:property name="PinkyPitch1LinkName" value="${prefix}PinkyPitch1Link" />
+  <xacro:property name="PinkyPitch2LinkName" value="${prefix}PinkyPitch2Link" />
+  <xacro:property name="PinkyPitch3LinkName" value="${prefix}PinkyPitch3Link" />
+  <xacro:property name="PinkyPitch4LinkName" value="${prefix}PinkyPitch4Link" />
 </robot>

File: valkyrie_description/robots/valkyrie_A/xacro/middle_finger/dh_parameters.xacro (robot description, xacro)
@@ -1,21 +1,21 @@
 <?xml version="1.0" ?>
 <robot xmlns:xacro="http://www.ros.org/wiki/xacro" name="v1/middle_finger/dh_parameters">
-  <xacro:property name="MFJ1_Origin_X" value="0.09767"/>
-  <xacro:property name="MFJ1_Origin_Y" value="0"/>
-  <xacro:property name="MFJ1_Origin_Z" value="${reflect * 0.00254}"/>
-  <xacro:property name="MFJ1_Orientation_Roll" value="${reflect * -1 * 1.57}"/>
-  <xacro:property name="MFJ1_Orientation_Pitch" value="0"/>
-  <xacro:property name="MFJ1_Orientation_Yaw" value="0"/>
-  <xacro:property name="MFJ2_Origin_X" value="0.0381"/>
-  <xacro:property name="MFJ2_Origin_Y" value="0"/>
-  <xacro:property name="MFJ2_Origin_Z" value="0"/>
-  <xacro:property name="MFJ2_Orientation_Roll" value="0"/>
-  <xacro:property name="MFJ2_Orientation_Pitch" value="0"/>
-  <xacro:property name="MFJ2_Orientation_Yaw" value="0"/>
-  <xacro:property name="MFJ3_Origin_X" value="0.02286"/>
-  <xacro:property name="MFJ3_Origin_Y" value="0"/>
-  <xacro:property name="MFJ3_Origin_Z" value="0"/>
-  <xacro:property name="MFJ3_Orientation_Roll" value="0"/>
-  <xacro:property name="MFJ3_Orientation_Pitch" value="0"/>
-  <xacro:property name="MFJ3_Orientation_Yaw" value="0"/>
+  <xacro:property name="MiddleFingerPitch1FrameOrigin_X" value="0.09767"/>
+  <xacro:property name="MiddleFingerPitch1FrameOrigin_Y" value="0"/>
+  <xacro:property name="MiddleFingerPitch1FrameOrigin_Z" value="${reflect * 0.00254}"/>
+  <xacro:property name="MiddleFingerPitch1FrameOrientation_Roll" value="0.0"/>
+  <xacro:property name="MiddleFingerPitch1FrameOrientation_Pitch" value="0.0"/>
+  <xacro:property name="MiddleFingerPitch1FrameOrientation_Yaw" value="0.0"/>
+  <xacro:property name="MiddleFingerPitch2FrameOrigin_X" value="0.0381"/>
+  <xacro:property name="MiddleFingerPitch2FrameOrigin_Y" value="0"/>
+  <xacro:property name="MiddleFingerPitch2FrameOrigin_Z" value="0"/>
+  <xacro:property name="MiddleFingerPitch2FrameOrientation_Roll" value="0.0"/>
+  <xacro:property name="MiddleFingerPitch2FrameOrientation_Pitch" value="0.0"/>
+  <xacro:property name="MiddleFingerPitch2FrameOrientation_Yaw" value="0.0"/>
+  <xacro:property name="MiddleFingerPitch3FrameOrigin_X" value="0.02286"/>
+  <xacro:property name="MiddleFingerPitch3FrameOrigin_Y" value="0"/>
+  <xacro:property name="MiddleFingerPitch3FrameOrigin_Z" value="0"/>
+  <xacro:property name="MiddleFingerPitch3FrameOrientation_Roll" value="0.0"/>
+  <xacro:property name="MiddleFingerPitch3FrameOrientation_Pitch" value="0.0"/>
+  <xacro:property name="MiddleFingerPitch3FrameOrientation_Yaw" value="0.0"/>
 </robot>

File: valkyrie_description/robots/valkyrie_A/xacro/middle_finger/joint_limits.xacro (robot description, xacro)
@@ -1,15 +1,15 @@
 <?xml version="1.0" ?>
 <robot xmlns:xacro="http://www.ros.org/wiki/xacro" name="v1/middle_finger/joint_limits">
-  <xacro:property name="MFJ1_Torque_Limit" value="10" />
-  <xacro:property name="MFJ2_Torque_Limit" value="10" />
-  <xacro:property name="MFJ3_Torque_Limit" value="10" />
-  <xacro:property name="MFJ1_Lower_Limit" value="-1.658" />
-  <xacro:property name="MFJ2_Lower_Limit" value="-1.920" />
-  <xacro:property name="MFJ3_Lower_Limit" value="-1.57" />
-  <xacro:property name="MFJ1_Upper_Limit" value="0.175" />
-  <xacro:property name="MFJ2_Upper_Limit" value="0" />
-  <xacro:property name="MFJ3_Upper_Limit" value="0.175" />
-  <xacro:property name="MFJ1_Speed_Limit" value="1" />
-  <xacro:property name="MFJ2_Speed_Limit" value="1" />
-  <xacro:property name="MFJ3_Speed_Limit" value="1" />
+  <xacro:property name="MiddleFingerPitch1TorqueLimit" value="10" />
+  <xacro:property name="MiddleFingerPitch2TorqueLimit" value="10" />
+  <xacro:property name="MiddleFingerPitch3TorqueLimit" value="10" />
+  <xacro:property name="MiddleFingerPitch1PositionLimit_Lower" value="-1.658" />
+  <xacro:property name="MiddleFingerPitch2PositionLimit_Lower" value="-1.920" />
+  <xacro:property name="MiddleFingerPitch3PositionLimit_Lower" value="-1.57" />
+  <xacro:property name="MiddleFingerPitch1PositionLimit_Upper" value="0.175" />
+  <xacro:property name="MiddleFingerPitch2PositionLimit_Upper" value="0" />
+  <xacro:property name="MiddleFingerPitch3PositionLimit_Upper" value="0.175" />
+  <xacro:property name="MiddleFingerPitch1VelocityLimit" value="1" />
+  <xacro:property name="MiddleFingerPitch2VelocityLimit" value="1" />
+  <xacro:property name="MiddleFingerPitch3VelocityLimit" value="1" />
 </robot>

File: valkyrie_description/robots/valkyrie_A/xacro/middle_finger/joint_names.xacro (robot description, xacro)
@@ -1,6 +1,6 @@
 <?xml version="1.0" ?>
 <robot xmlns:xacro="http://www.ros.org/wiki/xacro" name="v1/middle_finger/mass_parameters">
-  <xacro:property name="MFJ1_Joint_Name" value="${prefix}MiddleFingerPitch1" />
-  <xacro:property name="MFJ2_Joint_Name" value="${prefix}MiddleFingerPitch2" />
-  <xacro:property name="MFJ3_Joint_Name" value="${prefix}MiddleFingerPitch3" />
+  <xacro:property name="MiddleFingerPitch1JointName" value="${prefix}MiddleFingerPitch1" />
+  <xacro:property name="MiddleFingerPitch2JointName" value="${prefix}MiddleFingerPitch2" />
+  <xacro:property name="MiddleFingerPitch3JointName" value="${prefix}MiddleFingerPitch3" />
 </robot>

File: valkyrie_description/robots/valkyrie_A/xacro/middle_finger/link_names.xacro (robot description, xacro)
@@ -1,9 +1,7 @@
 <?xml version="1.0" ?>
 <robot xmlns:xacro="http://www.ros.org/wiki/xacro" name="v1/middle_finger/dh_parameters">
-  <xacro:property name="MFJ1_Proximal_Link" value="${middle_finger_root_link}" />
-  <xacro:property name="MFJ1_Distal_Link" value="${prefix}MiddleFingerPitch1" />
-  <xacro:property name="MFJ2_Proximal_Link" value="${prefix}MiddleFingerPitch1" />
-  <xacro:property name="MFJ2_Distal_Link" value="${prefix}MiddleFingerPitch2" />
-  <xacro:property name="MFJ3_Proximal_Link" value="${prefix}MiddleFingerPitch2" />
-  <xacro:property name="MFJ3_Distal_Link" value="${prefix}MiddleFingerPitch3" />
+  <xacro:property name="MiddleFingerPitch1ParentLinkName" value="${middle_finger_root_link}" />
+  <xacro:property name="MiddleFingerPitch1LinkName" value="${prefix}MiddleFingerPitch1" />
+  <xacro:property name="MiddleFingerPitch2LinkName" value="${prefix}MiddleFingerPitch2" />
+  <xacro:property name="MiddleFingerPitch3LinkName" value="${prefix}MiddleFingerPitch3" />
 </robot>
