Commit message: Renamed a bunch of middle finger xacro properties and fixed an arm naming typo I had.

File: valkyrie_description/robots/valkyrie_A/xacro/middle_finger/middle_finger.xacro (robot description, xacro)
@@ -28,5 +28,5 @@
   <xacro:macro name="make_middle_finger" params="prefix reflect middle_finger_root_link">
     <!-- LINKS -->
-    <xacro:box_link name="${MFJ1_Distal_Link}"
+    <xacro:box_link name="${MiddleFingerPitch1LinkName}"
                     width="${MFJ1_Link_Width}" height="${MFJ1_Link_Height}" depth="${MFJ1_Link_Length}" mass="${MFJ1_Link_Mass}"
                     origin_rpy="0 0 0"
@@ -35,5 +35,5 @@
                     material="Gold"
                     collision_mesh="${mesh_root}/sf1.stl"/>
-    <xacro:box_link name="${MFJ2_Distal_Link}"
+    <xacro:box_link name="${MiddleFingerPitch2LinkName}"
                     width="${MFJ2_Link_Width}" height="${MFJ2_Link_Height}" depth="${MFJ2_Link_Length}" mass="${MFJ2_Link_Mass}"
                     origin_rpy="0 0 0"
@@ -42,5 +42,5 @@
                     material="Gold"
                     collision_mesh="${mesh_root}/sf2_ssf3.stl"/>
-    <xacro:box_link name="${MFJ3_Distal_Link}"
+    <xacro:box_link name="${MiddleFingerPitch3LinkName}"
                     width="${MFJ3_Link_Width}" height="${MFJ3_Link_Height}" depth="${MFJ3_Link_Length}" mass="${MFJ3_Link_Mass}"
                     origin_rpy="0 0 0"
@@ -50,28 +50,28 @@
                     collision_mesh="${mesh_root}/sf3_ssf4.stl"/>
     <!-- MFJ1 -->
-    <xacro:revolute_joint jointName="${MFJ1_Joint_Name}"
-                          parent="${MFJ1_Proximal_Link}" child="${MFJ1_Distal_Link}"
-                          origin_xyz="${MFJ1_Origin_X} ${MFJ1_Origin_Y} ${MFJ1_Origin_Z}"
-                          origin_rpy="${MFJ1_Orientation_Roll} ${MFJ1_Orientation_Pitch} ${MFJ1_Orientation_Yaw}">
-        <limit effort="${MFJ1_Torque_Limit}" lower="${MFJ1_Lower_Limit}" upper="${MFJ1_Upper_Limit}" velocity="${MFJ1_Speed_Limit}"/>
+    <xacro:revolute_joint jointName="${MiddleFingerPitch1JointName}"
+                          parent="${MiddleFingerPitch1ParentLinkName}" child="${MiddleFingerPitch1LinkName}"
+                          origin_xyz="${MiddleFingerPitch1FrameOrigin_X} ${MiddleFingerPitch1FrameOrigin_Y} ${MiddleFingerPitch1FrameOrigin_Z}"
+                          origin_rpy="${MiddleFingerPitch1FrameOrientation_Roll} ${MiddleFingerPitch1FrameOrientation_Pitch} ${MiddleFingerPitch1FrameOrientation_Yaw}">
+        <limit effort="${MiddleFingerPitch1TorqueLimit}" lower="${MiddleFingerPitch1PositionLimit_Lower}" upper="${MiddleFingerPitch1PositionLimit_Upper}" velocity="${MiddleFingerPitch1VelocityLimit}"/>
     </xacro:revolute_joint>
     <!-- MFJ2 -->
-    <xacro:revolute_joint jointName="${MFJ2_Joint_Name}"
-                          parent="${MFJ2_Proximal_Link}" child="${MFJ2_Distal_Link}"
-                          origin_xyz="${MFJ2_Origin_X} ${MFJ2_Origin_Y} ${MFJ2_Origin_Z}"
-                          origin_rpy="${MFJ2_Orientation_Roll} ${MFJ2_Orientation_Pitch} ${MFJ2_Orientation_Yaw}">
-        <limit effort="${MFJ2_Torque_Limit}" lower="${MFJ2_Lower_Limit}" upper="${MFJ2_Upper_Limit}" velocity="${MFJ2_Speed_Limit}"/>
+    <xacro:revolute_joint jointName="${MiddleFingerPitch2JointName}"
+                          parent="${MiddleFingerPitch1LinkName}" child="${MiddleFingerPitch2LinkName}"
+                          origin_xyz="${MiddleFingerPitch2FrameOrigin_X} ${MiddleFingerPitch2FrameOrigin_Y} ${MiddleFingerPitch2FrameOrigin_Z}"
+                          origin_rpy="${MiddleFingerPitch2FrameOrientation_Roll} ${MiddleFingerPitch2FrameOrientation_Pitch} ${MiddleFingerPitch2FrameOrientation_Yaw}">
+        <limit effort="${MiddleFingerPitch2TorqueLimit}" lower="${MiddleFingerPitch2PositionLimit_Lower}" upper="${MiddleFingerPitch2PositionLimit_Upper}" velocity="${MiddleFingerPitch2VelocityLimit}"/>
     </xacro:revolute_joint>
     <!-- MFJ3 -->
-    <xacro:revolute_joint jointName="${MFJ3_Joint_Name}"
-                          parent="${MFJ3_Proximal_Link}" child="${MFJ3_Distal_Link}"
-                          origin_xyz="${MFJ3_Origin_X} ${MFJ3_Origin_Y} ${MFJ3_Origin_Z}"
-                          origin_rpy="${MFJ3_Orientation_Roll} ${MFJ3_Orientation_Pitch} ${MFJ3_Orientation_Yaw}">
-        <limit effort="${MFJ3_Torque_Limit}" lower="${MFJ3_Lower_Limit}" upper="${MFJ3_Upper_Limit}" velocity="${MFJ3_Speed_Limit}"/>
+    <xacro:revolute_joint jointName="${MiddleFingerPitch3JointName}"
+                          parent="${MiddleFingerPitch2LinkName}" child="${MiddleFingerPitch3LinkName}"
+                          origin_xyz="${MiddleFingerPitch3FrameOrigin_X} ${MiddleFingerPitch3FrameOrigin_Y} ${MiddleFingerPitch3FrameOrigin_Z}"
+                          origin_rpy="${MiddleFingerPitch3FrameOrientation_Roll} ${MiddleFingerPitch3FrameOrientation_Pitch} ${MiddleFingerPitch3FrameOrientation_Yaw}">
+        <limit effort="${MiddleFingerPitch3TorqueLimit}" lower="${MiddleFingerPitch3PositionLimit_Lower}" upper="${MiddleFingerPitch3PositionLimit_Upper}" velocity="${MiddleFingerPitch3VelocityLimit}"/>
     </xacro:revolute_joint>
   </xacro:macro>
   <xacro:macro name="make_middle_finger_fixed" params="prefix reflect middle_finger_root_link">
     <!-- LINKS -->
-    <xacro:box_link name="${MFJ1_Distal_Link}"
+    <xacro:box_link name="${MiddleFingerPitch1LinkName}"
                     width="${MFJ1_Link_Width}" height="${MFJ1_Link_Height}" depth="${MFJ1_Link_Length}" mass="${MFJ1_Link_Mass}"
                     origin_rpy="0 0 0"
@@ -80,5 +80,5 @@
                     material="Gold"
                     collision_mesh="${mesh_root}/sf1.stl"/>
-    <xacro:box_link name="${MFJ2_Distal_Link}"
+    <xacro:box_link name="${MiddleFingerPitch2LinkName}"
                     width="${MFJ2_Link_Width}" height="${MFJ2_Link_Height}" depth="${MFJ2_Link_Length}" mass="${MFJ2_Link_Mass}"
                     origin_rpy="0 0 0"
@@ -87,5 +87,5 @@
                     material="Gold"
                     collision_mesh="${mesh_root}/sf2_ssf3.stl"/>
-    <xacro:box_link name="${MFJ3_Distal_Link}"
+    <xacro:box_link name="${MiddleFingerPitch3LinkName}"
                     width="${MFJ3_Link_Width}" height="${MFJ3_Link_Height}" depth="${MFJ3_Link_Length}" mass="${MFJ3_Link_Mass}"
                     origin_rpy="0 0 0"
@@ -95,18 +95,18 @@
                     collision_mesh="${mesh_root}/sf3_ssf4.stl"/>
     <!-- MFJ1 -->
-    <xacro:fixed_joint jointName="${MFJ1_Joint_Name}"
-                          parent="${MFJ1_Proximal_Link}" child="${MFJ1_Distal_Link}"
-                          origin_xyz="${MFJ1_Origin_X} ${MFJ1_Origin_Y} ${MFJ1_Origin_Z}"
-                          origin_rpy="${MFJ1_Orientation_Roll} ${MFJ1_Orientation_Pitch} ${MFJ1_Orientation_Yaw}"/>
+    <xacro:fixed_joint jointName="${MiddleFingerPitch1JointName}"
+                          parent="${MiddleFingerPitch1ParentLinkName}" child="${MiddleFingerPitch1LinkName}"
+                          origin_xyz="${MiddleFingerPitch1FrameOrigin_X} ${MiddleFingerPitch1FrameOrigin_Y} ${MiddleFingerPitch1FrameOrigin_Z}"
+                          origin_rpy="${MiddleFingerPitch1FrameOrientation_Roll} ${MiddleFingerPitch1FrameOrientation_Pitch} ${MiddleFingerPitch1FrameOrientation_Yaw}"/>
     <!-- MFJ2 -->
-    <xacro:fixed_joint jointName="${MFJ2_Joint_Name}"
-                          parent="${MFJ2_Proximal_Link}" child="${MFJ2_Distal_Link}"
-                          origin_xyz="${MFJ2_Origin_X} ${MFJ2_Origin_Y} ${MFJ2_Origin_Z}"
-                          origin_rpy="${MFJ2_Orientation_Roll} ${MFJ2_Orientation_Pitch} ${MFJ2_Orientation_Yaw}"/>
+    <xacro:fixed_joint jointName="${MiddleFingerPitch2JointName}"
+                          parent="${MiddleFingerPitch1LinkName}" child="${MiddleFingerPitch2LinkName}"
+                          origin_xyz="${MiddleFingerPitch2FrameOrigin_X} ${MiddleFingerPitch2FrameOrigin_Y} ${MiddleFingerPitch2FrameOrigin_Z}"
+                          origin_rpy="${MiddleFingerPitch2FrameOrientation_Roll} ${MiddleFingerPitch2FrameOrientation_Pitch} ${MiddleFingerPitch2FrameOrientation_Yaw}"/>
     <!-- MFJ3 -->
-    <xacro:fixed_joint jointName="${MFJ3_Joint_Name}"
-                          parent="${MFJ3_Proximal_Link}" child="${MFJ3_Distal_Link}"
-                          origin_xyz="${MFJ3_Origin_X} ${MFJ3_Origin_Y} ${MFJ3_Origin_Z}"
-                          origin_rpy="${MFJ3_Orientation_Roll} ${MFJ3_Orientation_Pitch} ${MFJ3_Orientation_Yaw}"/>
+    <xacro:fixed_joint jointName="${MiddleFingerPitch3JointName}"
+                          parent="${MiddleFingerPitch2LinkName}" child="${MiddleFingerPitch3LinkName}"
+                          origin_xyz="${MiddleFingerPitch3FrameOrigin_X} ${MiddleFingerPitch3FrameOrigin_Y} ${MiddleFingerPitch3FrameOrigin_Z}"
+                          origin_rpy="${MiddleFingerPitch3FrameOrientation_Roll} ${MiddleFingerPitch3FrameOrientation_Pitch} ${MiddleFingerPitch3FrameOrientation_Yaw}"/>
   </xacro:macro>
   <!-- Actuators -->
@@ -120,32 +120,32 @@
   <xacro:macro name="v1_right_middle_finger_transmissions" params="prefix">
     <xacro:finger3_transmission tranName="${prefix}MiddleFingerTransmission"
-                                joint1="${MFJ1_Joint_Name}"
-                                joint2="${MFJ2_Joint_Name}"
-                                joint3="${MFJ3_Joint_Name}"
+                                joint1="${MiddleFingerPitch1JointName}"
+                                joint2="${MiddleFingerPitch2JointName}"
+                                joint3="${MiddleFingerPitch3JointName}"
                                 actuator="${RMFA_Actuator_Name}" />
   </xacro:macro>
   <xacro:macro name="v1_left_middle_finger_transmissions" params="prefix">
     <xacro:finger3_transmission tranName="${prefix}MiddleFingerTransmission"
-                                joint1="${MFJ1_Joint_Name}"
-                                joint2="${MFJ2_Joint_Name}"
-                                joint3="${MFJ3_Joint_Name}"
+                                joint1="${MiddleFingerPitch1JointName}"
+                                joint2="${MiddleFingerPitch2JointName}"
+                                joint3="${MiddleFingerPitch3JointName}"
                                 actuator="${LMFA_Actuator_Name}" />
   </xacro:macro>
   <xacro:macro name="v1_right_middle_finger_transmissions_simple" params="prefix">
-    <xacro:simple_transmission jointName="${MFJ1_Joint_Name}" actuatorName="${RMFA_Actuator_Name}" reduction="1" offset="0"/>
+    <xacro:simple_transmission jointName="${MiddleFingerPitch1JointName}" actuatorName="${RMFA_Actuator_Name}" reduction="1" offset="0"/>
   </xacro:macro>
   <xacro:macro name="v1_left_middle_finger_transmissions_simple" params="prefix">
-    <xacro:simple_transmission jointName="${MFJ1_Joint_Name}" actuatorName="${LMFA_Actuator_Name}" reduction="1" offset="0"/>
+    <xacro:simple_transmission jointName="${MiddleFingerPitch1JointName}" actuatorName="${LMFA_Actuator_Name}" reduction="1" offset="0"/>
   </xacro:macro>
   <!-- Modes -->
   <xacro:macro name="v1_right_middle_finger_modes" params="prefix">
-    <xacro:v1_modes jointName="${MFJ1_Joint_Name}" actuatorName="${RMFA_Actuator_Name}" />
-    <xacro:v1_modes jointName="${MFJ2_Joint_Name}" actuatorName="${RMFA_Actuator_Name}" />
-    <xacro:v1_modes jointName="${MFJ3_Joint_Name}" actuatorName="${RMFA_Actuator_Name}" />
+    <xacro:v1_modes jointName="${MiddleFingerPitch1JointName}" actuatorName="${RMFA_Actuator_Name}" />
+    <xacro:v1_modes jointName="${MiddleFingerPitch2JointName}" actuatorName="${RMFA_Actuator_Name}" />
+    <xacro:v1_modes jointName="${MiddleFingerPitch3JointName}" actuatorName="${RMFA_Actuator_Name}" />
   </xacro:macro>
   <xacro:macro name="v1_left_middle_finger_modes" params="prefix">
-    <xacro:v1_modes jointName="${MFJ1_Joint_Name}" actuatorName="${LMFA_Actuator_Name}" />
-    <xacro:v1_modes jointName="${MFJ2_Joint_Name}" actuatorName="${LMFA_Actuator_Name}" />
-    <xacro:v1_modes jointName="${MFJ3_Joint_Name}" actuatorName="${LMFA_Actuator_Name}" />
+    <xacro:v1_modes jointName="${MiddleFingerPitch1JointName}" actuatorName="${LMFA_Actuator_Name}" />
+    <xacro:v1_modes jointName="${MiddleFingerPitch2JointName}" actuatorName="${LMFA_Actuator_Name}" />
+    <xacro:v1_modes jointName="${MiddleFingerPitch3JointName}" actuatorName="${LMFA_Actuator_Name}" />
   </xacro:macro>
   <!-- Complete interface -->

Commit message: Updated COM values for arms.

File: valkyrie_description/robots/valkyrie_A/xacro/arm/arm.xacro (robot description, xacro)
@@ -33,5 +33,5 @@
     <xacro:box_link name="${ShoulderPitchLinkName}"
                     width="${AJ1_Link_Width}" height="${AJ1_Link_Height}" depth="${AJ1_Link_Length}" mass="${ShoulderPitchLinkMass}"
-                    origin_xyz="0 -0.01204 ${reflect * -0.251}" origin_rpy="0 0 0"
+                    origin_xyz="${ShoulderPitchLinkComPosition}" origin_rpy="0 0 0"
                     visual_mesh="${mesh_root}/aj1_${prefix}.stl"
                     material="Gold"
@@ -39,5 +39,5 @@
     <xacro:box_link name="${ShoulderRollLinkName}"
                     width="${AJ2_Link_Width}" height="${AJ2_Link_Height}" depth="${AJ2_Link_Length}" mass="${ShoulderRollLinkMass}"
-                    origin_xyz="0.04 0.005 ${reflect * -0.02}" origin_rpy="0 0 0"
+                    origin_xyz="${ShoulderRollLinkComPosition}" origin_rpy="0 0 0"
                     visual_mesh="${mesh_root}/aj2_${prefix}.stl"
                     material="White"
@@ -45,5 +45,5 @@
     <xacro:box_link name="${ShoulderYawLinkName}"
                     width="${AJ3_Link_Width}" height="${AJ3_Link_Height}" depth="${AJ3_Link_Length}" mass="${ShoulderYawLinkMass}"
-                    origin_xyz="${reflect * 0.02} ${reflect * -0.004} ${reflect * -0.273}" origin_rpy="0 0 0"
+                    origin_xyz="${ShoulderYawLinkComPosition}" origin_rpy="0 0 0"
                     visual_mesh="${mesh_root}/aj3_${prefix}.stl"
                     material="White"
@@ -51,6 +51,6 @@
     <xacro:box_link name="${ElbowPitchLinkName}"
                     width="${AJ4_Link_Width}" height="${AJ4_Link_Height}" depth="${AJ4_Link_Length}" mass="${ElbowPitchLinkMass}"
+                    origin_xyz="${ElbowPitchLinkComPosition}"
                     origin_rpy="0 0 0"
-                    origin_xyz="0.0270 -0.0802 0"
                     visual_mesh="${mesh_root}/aj4_${prefix}.stl"
                     material="Gold"
@@ -101,6 +101,6 @@
     <xacro:box_link name="${ForearmLinkName}"
                     width="${AJ5_Link_Width}" height="${AJ5_Link_Height}" depth="${AJ5_Link_Length}" mass="${ForearmYawLinkMass}"
+                    origin_xyz="${ForearmYawLinkComPosition}"
                     origin_rpy="0 0 0"
-                    origin_xyz="0.015 ${reflect * 0.02} ${reflect * -0.11}"
                     visual_mesh="${mesh_root}/aj5_${prefix}.stl"
                     material="White"
@@ -108,6 +108,6 @@
     <xacro:box_link name="${WristRollLinkName}"
                     width="${AJ6_Link_Width}" height="${AJ6_Link_Height}" depth="${AJ6_Link_Length}" mass="${WristRollLinkMass}"
+                    origin_xyz="${WristRollLinkComPosition}"
                     origin_rpy="0 0 0"
-                    origin_xyz="0 0 0"
                     visual_mesh="${mesh_root}/aj6_${prefix}.stl"
                     material="White"
@@ -115,6 +115,6 @@
     <xacro:box_link name="${WristPitchLinkName}"
                     width="${AJ7_Link_Width}" height="${AJ7_Link_Height}" depth="${AJ7_Link_Length}" mass="${PalmMass}"
+                    origin_xyz="${PalmComPosition}"
                     origin_rpy="0 0 0"
-                    origin_xyz="${AJ7_Link_Width/2} 0 0"
                     visual_mesh="${mesh_root}/palm_${prefix}.stl"
                     material="Gold"

File: valkyrie_description/robots/valkyrie_A/xacro/arm/mass_parameters.xacro (robot description, xacro)
@@ -2,9 +2,16 @@
 <robot xmlns:xacro="http://www.ros.org/wiki/xacro" name="v1/arm/mass_parameters">
   <xacro:property name="ShoulderPitchLinkMass" value="2.65" />
+  <xacro:property name="ShoulderPitchLinkComPosition" value="-0.012000 ${reflect}*0.251000 0.000000" />
   <xacro:property name="ShoulderRollLinkMass" value="2.87" />
+  <xacro:property name="ShoulderRollLinkComPosition" value="-0.020086 ${reflect}*0.040000 -0.004999" />
   <xacro:property name="ShoulderYawLinkMass" value="2.575" />
+  <xacro:property name="ShoulderYawLinkComPosition" value="0.004000	${reflect}*0.273000	-0.019953" />
   <xacro:property name="ElbowPitchLinkMass" value="2.367" />
+  <xacro:property name="ElbowPitchLinkComPosition" value="-0.027000	${reflect}*0.080200 0.000000" />
   <xacro:property name="ForearmYawLinkMass" value="2.903" />
+  <xacro:property name="ForearmYawLinkComPosition" value="0.015000	${reflect}*0.110000 0.019564" />
   <xacro:property name="WristRollLinkMass" value="0.1" />
+  <xacro:property name="WristRollLinkComPosition" value="0 0 0" />
   <xacro:property name="PalmMass" value="0.712" />
+  <xacro:property name="PalmComPosition" value="0.002954 ${reflect}*0.052034 -0.000236" />
 </robot>
