Commit message: Fixed COM values of fingers.

File: valkyrie_description/robots/valkyrie_A/xacro/arm/mass_parameters.xacro (robot description, xacro)
@@ -2,16 +2,16 @@
 <robot xmlns:xacro="http://www.ros.org/wiki/xacro" name="v1/arm/mass_parameters">
   <xacro:property name="ShoulderPitchLinkMass" value="2.65" />
-  <xacro:property name="ShoulderPitchLinkComPosition" value="-0.012000 ${reflect}*0.251000 0.000000" />
+  <xacro:property name="ShoulderPitchLinkComPosition" value="-0.012000 ${reflect*0.251000} 0.000000" />
   <xacro:property name="ShoulderRollLinkMass" value="2.87" />
-  <xacro:property name="ShoulderRollLinkComPosition" value="-0.020086 ${reflect}*0.040000 -0.004999" />
+  <xacro:property name="ShoulderRollLinkComPosition" value="-0.020086 ${reflect*0.040000} -0.004999" />
   <xacro:property name="ShoulderYawLinkMass" value="2.575" />
-  <xacro:property name="ShoulderYawLinkComPosition" value="0.004000	${reflect}*0.273000	-0.019953" />
+  <xacro:property name="ShoulderYawLinkComPosition" value="0.004000	${reflect*0.273000}	-0.019953" />
   <xacro:property name="ElbowPitchLinkMass" value="2.367" />
-  <xacro:property name="ElbowPitchLinkComPosition" value="-0.027000	${reflect}*0.080200 0.000000" />
+  <xacro:property name="ElbowPitchLinkComPosition" value="-0.027000	${reflect*0.080200} 0.000000" />
   <xacro:property name="ForearmYawLinkMass" value="2.903" />
-  <xacro:property name="ForearmYawLinkComPosition" value="0.015000	${reflect}*0.110000 0.019564" />
+  <xacro:property name="ForearmYawLinkComPosition" value="0.015000	${reflect*0.110000} 0.019564" />
   <xacro:property name="WristRollLinkMass" value="0.1" />
-  <xacro:property name="WristRollLinkComPosition" value="0 0 0" />
+  <xacro:property name="WristRollLinkComPosition" value="0 ${reflect*0} 0" />
   <xacro:property name="PalmMass" value="0.712" />
-  <xacro:property name="PalmComPosition" value="0.002954 ${reflect}*0.052034 -0.000236" />
+  <xacro:property name="PalmComPosition" value="0.002954 ${reflect*0.052034} -0.000236" />
 </robot>

File: valkyrie_description/robots/valkyrie_A/xacro/head/head.xacro (robot description, xacro)
@@ -1,4 +1,3 @@
 <robot xmlns:xacro="http://www.ros.org/wiki/xacro" name="v1/head">
-  <!-- Properties -->
   <xacro:include filename="$(find valkyrie_description)/robots/valkyrie_A/xacro/head/joint_names.xacro"/>
   <xacro:include filename="$(find valkyrie_description)/robots/valkyrie_A/xacro/head/joint_axes.xacro"/>
@@ -9,11 +8,8 @@
   <xacro:include filename="$(find valkyrie_description)/robots/valkyrie_A/xacro/sensors/ensenso.xacro"/>
   <xacro:include filename="$(find valkyrie_description)/robots/valkyrie_A/xacro/sensors/webcam.xacro"/>
-  <!-- Link properties. -->
   <xacro:property name="NJ3_Link_Radius" value="0.139"/>
   <xacro:macro name="include_head" params="lower_neck_pitch_root_link">
-    <!-- <xacro:standard_link name="${LowerNeckPitchLinkName}" "${LowerNeckPitchLinkMass" > -->
   </xacro:macro>
   <xacro:macro name="make_head" params="head_root_link">
-    <!-- LINKS -->
     <xacro:virtual_link_with_visual name="${LowerNeckPitchLinkName}"
                                     origin_xyz="${LowerNeckPitchLinkComPosition}"
@@ -30,5 +26,4 @@
                        material="White"
                        collision_mesh="${mesh_root}/head.stl"/>
-    <!-- NJ1 -->
     <xacro:revolute_joint_ex jointName="${LowerNeckPitchJointName}"
                           parent="${LowerNeckPitchParentLinkName}" child="${LowerNeckPitchLinkName}"
@@ -40,5 +35,4 @@
       <controller_gains Kp="20000" Kd="0"/>
     </xacro:revolute_joint_ex>
-    <!-- NJ2 -->
     <xacro:revolute_joint_ex jointName="${NeckYawJointName}"
                           parent="${LowerNeckPitchLinkName}" child="${NeckYawLinkName}"
@@ -50,5 +44,4 @@
       <controller_gains Kp="20000" Kd="0"/>
     </xacro:revolute_joint_ex>
-    <!-- NJ3 -->
     <xacro:revolute_joint_ex jointName="${UpperNeckPitchJointName}"
                           parent="${NeckYawLinkName}" child="${UpperNeckPitchLinkName}"
@@ -61,5 +54,4 @@
     </xacro:revolute_joint_ex>
   </xacro:macro>
-  <!-- Sensors -->
   <xacro:macro name="v1_head_sensors">
     <xacro:ensenso_sensor sensorName="Ensenso"
@@ -78,5 +70,4 @@
                         frameRate="60"/>
   </xacro:macro>
-  <!-- Actuators -->
   <xacro:macro name="v1_head_actuators" params="name1 type1 name2 type2 name3 type3">
     <actuator name="${name1}" type="${type1}"/>

File: valkyrie_description/robots/valkyrie_A/xacro/index_finger/index_finger.xacro (robot description, xacro)
@@ -11,24 +11,15 @@
   <xacro:property name="PFJ1_Link_Height" value="0.019"/>
   <xacro:property name="PFJ1_Link_Length" value="0.022"/>
-  <xacro:property name="PFJ1_Link_Origin_X" value="-0.0048"/>
-  <xacro:property name="PFJ1_Link_Origin_Y" value="0"/>
-  <xacro:property name="PFJ1_Link_Origin_Z" value="0"/>
   <xacro:property name="PFJ2_Link_Width" value="0.054"/>
   <xacro:property name="PFJ2_Link_Height" value="0.019"/>
   <xacro:property name="PFJ2_Link_Length" value="0.021"/>
-  <xacro:property name="PFJ2_Link_Origin_X" value="0.0175"/>
-  <xacro:property name="PFJ2_Link_Origin_Y" value="0"/>
-  <xacro:property name="PFJ2_Link_Origin_Z" value="0"/>
   <xacro:property name="PFJ3_Link_Width" value="0.034"/>
   <xacro:property name="PFJ3_Link_Height" value="0.013"/>
   <xacro:property name="PFJ3_Link_Length" value="0.017"/>
-  <xacro:property name="PFJ3_Link_Origin_X" value="0.0108"/>
-  <xacro:property name="PFJ3_Link_Origin_Y" value="-0.0003"/>
-  <xacro:property name="PFJ3_Link_Origin_Z" value="0"/>
   <xacro:macro name="make_index_finger" params="prefix reflect index_finger_root_link">
     <xacro:box_link name="${IndexFingerPitch1LinkName}"
                     width="${PFJ1_Link_Width}" height="${PFJ1_Link_Height}" depth="${PFJ1_Link_Length}" mass="${IndexFingerPitch1LinkMass}"
+                    origin_xyz="${IndexFingerPitch1ComPosition}"
                     origin_rpy="0 0 0"
-                    origin_xyz="${PFJ1_Link_Origin_X} ${PFJ1_Link_Origin_Y} ${PFJ1_Link_Origin_Z}"
                     visual_mesh="${mesh_root}/indexj1_${prefix}.stl"
                     material="Gold"
@@ -36,6 +27,6 @@
     <xacro:box_link name="${IndexFingerPitch2LinkName}"
                     width="${PFJ2_Link_Width}" height="${PFJ2_Link_Height}" depth="${PFJ2_Link_Length}" mass="${IndexFingerPitch2LinkMass}"
+                    origin_xyz="${IndexFingerPitch2ComPosition}"
                     origin_rpy="0 0 0"
-                    origin_xyz="${PFJ2_Link_Origin_X} ${PFJ2_Link_Origin_Y} ${PFJ2_Link_Origin_Z}"
                     visual_mesh="${mesh_root}/indexj2_${prefix}.stl"
                     material="Gold"
@@ -43,6 +34,6 @@
     <xacro:box_link name="${IndexFingerPitch3LinkName}"
                     width="${PFJ3_Link_Width}" height="${PFJ3_Link_Height}" depth="${PFJ3_Link_Length}" mass="${IndexFingerPitch3LinkMass}"
+                    origin_xyz="${IndexFingerPitch3ComPosition}"
                     origin_rpy="0 0 0"
-                    origin_xyz="${PFJ3_Link_Origin_X} ${PFJ3_Link_Origin_Y} ${PFJ3_Link_Origin_Z}"
                     visual_mesh="${mesh_root}/indexj3_${prefix}.stl"
                     material="Gold"

File: valkyrie_description/robots/valkyrie_A/xacro/index_finger/mass_parameters.xacro (robot description, xacro)
@@ -2,6 +2,8 @@
 <robot xmlns:xacro="http://www.ros.org/wiki/xacro" name="v1/index_finger/mass_parameters">
   <xacro:property name="IndexFingerPitch1LinkMass" value="0.006" />
+  <xacro:property name="IndexFingerPitch1ComPosition" value="0 ${reflect*0.02} 0" />
   <xacro:property name="IndexFingerPitch2LinkMass" value="0.018" />
+  <xacro:property name="IndexFingerPitch2ComPosition" value="0 ${reflect*0.013} 0" />
   <xacro:property name="IndexFingerPitch3LinkMass" value="0.01" />
-  <xacro:property name="IndexFingerPitch4LinkMass" value="0.005" />
+  <xacro:property name="IndexFingerPitch3ComPosition" value="0 ${reflect*0.01} 0" />
 </robot>

File: valkyrie_description/robots/valkyrie_A/xacro/leg/mass_parameters.xacro (robot description, xacro)
@@ -2,14 +2,14 @@
 <robot xmlns:xacro="http://www.ros.org/wiki/xacro" name="v1/leg/mass_parameters">
   <xacro:property name="HipYawLinkMass" value="2.39" />
-  <xacro:property name="HipYawLinkComPosition" value="0.02176 ${reflect}*-0.00131 0.03867" />
+  <xacro:property name="HipYawLinkComPosition" value="0.02176 ${reflect*-0.00131} 0.03867" />
   <xacro:property name="HipRollLinkMass" value="5.95" />
-  <xacro:property name="HipRollLinkComPosition" value="-0.00185 ${reflect}*0.02426 -0.019260" />
+  <xacro:property name="HipRollLinkComPosition" value="-0.00185 ${reflect*0.02426} -0.019260" />
   <xacro:property name="HipPitchLinkMass" value="10.3" />
-  <xacro:property name="HipPitchLinkComPosition" value="0.000057 ${reflect}*0.050000 -0.220000" />
+  <xacro:property name="HipPitchLinkComPosition" value="0.000057 ${reflect*0.050000} -0.220000" />
   <xacro:property name="KneePitchLinkMass" value="7.4" />
-  <xacro:property name="KneePitchLinkComPosition" value="-0.004670 ${reflect}*0.045000 -0.184940" />
+  <xacro:property name="KneePitchLinkComPosition" value="-0.004670 ${reflect*0.045000} -0.184940" />
   <xacro:property name="AnklePitchLinkMass" value="0.395" />
-  <xacro:property name="AnklePitchLinkComPosition" value="-0.001270 ${reflect}*0.000000 -0.006010" />
+  <xacro:property name="AnklePitchLinkComPosition" value="-0.001270 ${reflect*0.000000} -0.006010" />
   <xacro:property name="FootMass" value="1.888" />
-  <xacro:property name="FootComPosition" value="0.068860 ${reflect}*-0.000285 -0.051830" />
+  <xacro:property name="FootComPosition" value="0.068860 ${reflect*-0.000285} -0.051830" />
 </robot>

File: valkyrie_description/robots/valkyrie_A/xacro/middle_finger/mass_parameters.xacro (robot description, xacro)
@@ -2,5 +2,8 @@
 <robot xmlns:xacro="http://www.ros.org/wiki/xacro" name="v1/middle_finger/mass_parameters">
   <xacro:property name="MiddleFingerPitch1LinkMass" value="0.02" />
+  <xacro:property name="MiddleFingerPitch1ComPosition" value="0 ${reflect*0.02} 0" />
   <xacro:property name="MiddleFingerPitch2LinkMass" value="0.011" />
+  <xacro:property name="MiddleFingerPitch2ComPosition" value="0 ${reflect*0.013} 0" />
   <xacro:property name="MiddleFingerPitch3LinkMass" value="0.006" />
+  <xacro:property name="MiddleFingerPitch3ComPosition" value="0 ${reflect*0.01} 0" />
 </robot>

File: valkyrie_description/robots/valkyrie_A/xacro/middle_finger/middle_finger.xacro (robot description, xacro)
@@ -11,24 +11,15 @@
   <xacro:property name="MFJ1_Link_Height" value="0.019"/>
   <xacro:property name="MFJ1_Link_Length" value="0.026"/>
-  <xacro:property name="MFJ1_Link_Origin_X" value="0.017"/>
-  <xacro:property name="MFJ1_Link_Origin_Y" value="0"/>
-  <xacro:property name="MFJ1_Link_Origin_Z" value="0"/>
   <xacro:property name="MFJ2_Link_Width" value="0.034"/>
   <xacro:property name="MFJ2_Link_Height" value="0.013"/>
   <xacro:property name="MFJ2_Link_Length" value="0.022"/>
-  <xacro:property name="MFJ2_Link_Origin_X" value="0.011"/>
-  <xacro:property name="MFJ2_Link_Origin_Y" value="0"/>
-  <xacro:property name="MFJ2_Link_Origin_Z" value="0"/>
   <xacro:property name="MFJ3_Link_Width" value="0.027"/>
   <xacro:property name="MFJ3_Link_Height" value="0.012"/>
   <xacro:property name="MFJ3_Link_Length" value="0.019"/>
-  <xacro:property name="MFJ3_Link_Origin_X" value="0.0086"/>
-  <xacro:property name="MFJ3_Link_Origin_Y" value="0"/>
-  <xacro:property name="MFJ3_Link_Origin_Z" value="0"/>
   <xacro:macro name="make_middle_finger" params="prefix reflect middle_finger_root_link">
     <xacro:box_link name="${MiddleFingerPitch1LinkName}"
                     width="${MFJ1_Link_Width}" height="${MFJ1_Link_Height}" depth="${MFJ1_Link_Length}" mass="${MiddleFingerPitch1LinkMass}"
+                    origin_xyz="${MiddleFingerPitch1ComPosition}"
                     origin_rpy="0 0 0"
-                    origin_xyz="${MFJ1_Link_Origin_X} ${MFJ1_Link_Origin_Y} ${MFJ1_Link_Origin_Z}"
                     visual_mesh="${mesh_root}/middlej1_${prefix}.stl"
                     material="Gold"
@@ -36,6 +27,6 @@
     <xacro:box_link name="${MiddleFingerPitch2LinkName}"
                     width="${MFJ2_Link_Width}" height="${MFJ2_Link_Height}" depth="${MFJ2_Link_Length}" mass="${MiddleFingerPitch2LinkMass}"
+                    origin_xyz="${MiddleFingerPitch2ComPosition}"
                     origin_rpy="0 0 0"
-                    origin_xyz="${MFJ2_Link_Origin_X} ${MFJ2_Link_Origin_Y} ${MFJ2_Link_Origin_Z}"
                     visual_mesh="${mesh_root}/middlej2_${prefix}.stl"
                     material="Gold"
@@ -43,6 +34,6 @@
     <xacro:box_link name="${MiddleFingerPitch3LinkName}"
                     width="${MFJ3_Link_Width}" height="${MFJ3_Link_Height}" depth="${MFJ3_Link_Length}" mass="${MiddleFingerPitch3LinkMass}"
+                    origin_xyz="${MiddleFingerPitch3ComPosition}"
                     origin_rpy="0 0 0"
-                    origin_xyz="${MFJ3_Link_Origin_X} ${MFJ3_Link_Origin_Y} ${MFJ3_Link_Origin_Z}"
                     visual_mesh="${mesh_root}/middlej3_${prefix}.stl"
                     material="Gold"

File: valkyrie_description/robots/valkyrie_A/xacro/pinky_finger/mass_parameters.xacro (robot description, xacro)
@@ -2,6 +2,8 @@
 <robot xmlns:xacro="http://www.ros.org/wiki/xacro" name="v1/pinky_finger/mass_parameters">
   <xacro:property name="PinkyPitch1LinkMass" value="0.047" />
+  <xacro:property name="PinkyFingerPitch1ComPosition" value="0 ${reflect*0.02} 0" />
   <xacro:property name="PinkyPitch2LinkMass" value="0.02" />
+  <xacro:property name="PinkyFingerPitch2ComPosition" value="0 ${reflect*0.013} 0" />
   <xacro:property name="PinkyPitch3LinkMass" value="0.011" />
-  <xacro:property name="PinkyPitch4LinkMass" value="0.006" />
+  <xacro:property name="PinkyFingerPitch3ComPosition" value="0 ${reflect*0.01} 0" />
 </robot>

File: valkyrie_description/robots/valkyrie_A/xacro/pinky_finger/pinky_finger.xacro (robot description, xacro)
@@ -11,24 +11,15 @@
   <xacro:property name="LFJ1_Link_Height" value="0.010"/>
   <xacro:property name="LFJ1_Link_Length" value="0.010"/>
-  <xacro:property name="LFJ1_Link_Origin_X" value="0"/>
-  <xacro:property name="LFJ1_Link_Origin_Y" value="0"/>
-  <xacro:property name="LFJ1_Link_Origin_Z" value="0"/>
   <xacro:property name="LFJ2_Link_Width" value="0.019"/>
   <xacro:property name="LFJ2_Link_Height" value="0.054"/>
   <xacro:property name="LFJ2_Link_Length" value="0.026"/>
-  <xacro:property name="LFJ2_Link_Origin_X" value="0"/>
-  <xacro:property name="LFJ2_Link_Origin_Y" value="${reflect * 0.017}"/>
-  <xacro:property name="LFJ2_Link_Origin_Z" value="${reflect * 0.050169}"/>
   <xacro:property name="LFJ3_Link_Width" value="0.034"/>
   <xacro:property name="LFJ3_Link_Height" value="0.013"/>
   <xacro:property name="LFJ3_Link_Length" value="0.022"/>
-  <xacro:property name="LFJ3_Link_Origin_X" value="0.011"/>
-  <xacro:property name="LFJ3_Link_Origin_Y" value="0"/>
-  <xacro:property name="LFJ3_Link_Origin_Z" value="0"/>
   <xacro:macro name="make_pinky_finger" params="prefix reflect pinky_finger_root_link">
     <xacro:box_link name="${PinkyPitch1LinkName}"
                     width="${LFJ1_Link_Width}" height="${LFJ1_Link_Height}" depth="${LFJ1_Link_Length}" mass="${PinkyPitch1LinkMass}"
+                    origin_xyz="${PinkyFingerPitch1ComPosition}"
                     origin_rpy="0 0 0"
-                    origin_xyz="${LFJ1_Link_Origin_X} ${LFJ1_Link_Origin_Y} ${LFJ1_Link_Origin_Z}"
                     visual_mesh="${mesh_root}/pinkyj1_${prefix}.stl"
                     material="Gold"
@@ -36,6 +27,6 @@
     <xacro:box_link name="${PinkyPitch2LinkName}"
                     width="${LFJ2_Link_Width}" height="${LFJ2_Link_Height}" depth="${LFJ2_Link_Length}" mass="${PinkyPitch2LinkMass}"
+                    origin_xyz="${PinkyFingerPitch2ComPosition}"
                     origin_rpy="0 0 0"
-                    origin_xyz="${LFJ2_Link_Origin_X} ${LFJ2_Link_Origin_Y} ${LFJ2_Link_Origin_Z}"
                     visual_mesh="${mesh_root}/pinkyj2_${prefix}.stl"
                     material="Gold"
@@ -43,6 +34,6 @@
     <xacro:box_link name="${PinkyPitch3LinkName}"
                     width="${LFJ3_Link_Width}" height="${LFJ3_Link_Height}" depth="${LFJ3_Link_Length}" mass="${PinkyPitch3LinkMass}"
+                    origin_xyz="${PinkyFingerPitch3ComPosition}"
                     origin_rpy="0 0 0"
-                    origin_xyz="${LFJ3_Link_Origin_X} ${LFJ3_Link_Origin_Y} ${LFJ3_Link_Origin_Z}"
                     visual_mesh="${mesh_root}/pinkyj3_${prefix}.stl"
                     material="Gold"
@@ -70,5 +61,4 @@
     </xacro:revolute_joint>
   </xacro:macro>
-  <!-- Actuators -->
   <xacro:macro name="v1_right_pinky_finger_actuators" params="prefix api">
     <xacro:v1_actuator name="${RLFA_Actuator_Name}" api="${api}" />

File: valkyrie_description/robots/valkyrie_A/xacro/thumb/mass_parameters.xacro (robot description, xacro)
@@ -2,6 +2,10 @@
 <robot xmlns:xacro="http://www.ros.org/wiki/xacro" name="v1/thumb/mass_parameters">
   <xacro:property name="ThumbRollLinkMass" value="0.017" />
+  <xacro:property name="ThumbRollLinkComPosition" value="0 ${reflect*0} 0.015" />
   <xacro:property name="ThumbPitch1LinkMass" value="0.02" />
+  <xacro:property name="ThumbPitch1LinkComPosition" value="0.0 ${reflect*0.002} 0.02" />
   <xacro:property name="ThumbPitch2LinkMass" value="0.013" />
+  <xacro:property name="ThumbPitch2LinkComPosition" value="0 ${reflect*0.002} 0.015" />
   <xacro:property name="ThumbPitch3LinkMass" value="0.006" />
+  <xacro:property name="ThumbPitch3LinkComPosition" value="0 ${reflect*0} 0.01" />
 </robot>

File: valkyrie_description/robots/valkyrie_A/xacro/thumb/thumb.xacro (robot description, xacro)
@@ -11,30 +11,18 @@
   <xacro:property name="TJ1_Link_Height" value="0.010"/>
   <xacro:property name="TJ1_Link_Length" value="0.010"/>
-  <xacro:property name="TJ1_Link_Origin_X" value="0"/>
-  <xacro:property name="TJ1_Link_Origin_Y" value="0"/>
-  <xacro:property name="TJ1_Link_Origin_Z" value="0"/>
   <xacro:property name="TJ2_Link_Width" value="0.054"/>
   <xacro:property name="TJ2_Link_Height" value="0.019"/>
   <xacro:property name="TJ2_Link_Length" value="0.026"/>
-  <xacro:property name="TJ2_Link_Origin_X" value="0.017"/>
-  <xacro:property name="TJ2_Link_Origin_Y" value="0"/>
-  <xacro:property name="TJ2_Link_Origin_Z" value="0"/>
   <xacro:property name="TJ3_Link_Width" value="0.034"/>
   <xacro:property name="TJ3_Link_Height" value="0.013"/>
   <xacro:property name="TJ3_Link_Length" value="0.022"/>
-  <xacro:property name="TJ3_Link_Origin_X" value="0.011"/>
-  <xacro:property name="TJ3_Link_Origin_Y" value="0"/>
-  <xacro:property name="TJ3_Link_Origin_Z" value="0"/>
   <xacro:property name="TJ4_Link_Width" value="0.027"/>
   <xacro:property name="TJ4_Link_Height" value="0.012"/>
   <xacro:property name="TJ4_Link_Length" value="0.019"/>
-  <xacro:property name="TJ4_Link_Origin_X" value="0.0086"/>
-  <xacro:property name="TJ4_Link_Origin_Y" value="0"/>
-  <xacro:property name="TJ4_Link_Origin_Z" value="0"/>
   <xacro:macro name="make_thumb" params="prefix reflect thumb_root_link">
     <xacro:box_link name="${ThumbRollLinkName}"
                     width="${TJ1_Link_Width}" height="${TJ1_Link_Height}" depth="${TJ1_Link_Length}" mass="${ThumbRollLinkMass}"
+                    origin_xyz="${ThumbRollLinkComPosition}"
                     origin_rpy="0 0 0"
-                    origin_xyz="${TJ1_Link_Origin_X} ${TJ1_Link_Origin_Y} ${TJ1_Link_Origin_Z}"
                     visual_mesh="${mesh_root}/thumbj1_${prefix}.stl"
                     material="Gold"
@@ -42,6 +30,6 @@
     <xacro:box_link name="${ThumbPitch1LinkName}"
                     width="${TJ2_Link_Width}" height="${TJ2_Link_Height}" depth="${TJ2_Link_Length}" mass="${ThumbPitch1LinkMass}"
+                    origin_xyz="${ThumbPitch1LinkComPosition}"
                     origin_rpy="0 0 0"
-                    origin_xyz="${TJ2_Link_Origin_X} ${TJ2_Link_Origin_Y} ${TJ2_Link_Origin_Z}"
                     visual_mesh="${mesh_root}/thumbj2_${prefix}.stl"
                     material="Gold"
@@ -49,6 +37,6 @@
     <xacro:box_link name="${ThumbPitch2LinkName}"
                     width="${TJ3_Link_Width}" height="${TJ3_Link_Height}" depth="${TJ3_Link_Length}" mass="${ThumbPitch2LinkMass}"
+                    origin_xyz="${ThumbPitch2LinkComPosition}"
                     origin_rpy="0 0 0"
-                    origin_xyz="${TJ3_Link_Origin_X} ${TJ3_Link_Origin_Y} ${TJ3_Link_Origin_Z}"
                     visual_mesh="${mesh_root}/thumbj3_${prefix}.stl"
                     material="Gold"
@@ -56,6 +44,6 @@
     <xacro:box_link name="${ThumbPitch3LinkName}"
                     width="${TJ4_Link_Width}" height="${TJ4_Link_Height}" depth="${TJ4_Link_Length}" mass="${ThumbPitch3LinkMass}"
+                    origin_xyz="${ThumbPitch3LinkComPosition}"
                     origin_rpy="0 0 0"
-                    origin_xyz="${TJ4_Link_Origin_X} ${TJ4_Link_Origin_Y} ${TJ4_Link_Origin_Z}"
                     visual_mesh="${mesh_root}/thumbj4_${prefix}.stl"
                     material="Gold"
