Commit message: Fixed error in names of wrist joints.

File: valkyrie_description/robots/valkyrie_A/xacro/arm/joint_names.xacro (robot description, xacro)
@@ -6,5 +6,5 @@
   <xacro:property name="ElbowPitchJointName" value="${prefix}ElbowPitch" />
   <xacro:property name="ForearmYawJointName" value="${prefix}ForearmYaw" />
-  <xacro:property name="WristRollJointName" value="${prefix}WristPitch" />
-  <xacro:property name="WristPitchJointName" value="${prefix}WristRoll" />
+  <xacro:property name="WristRollJointName" value="${prefix}WristRoll" />
+  <xacro:property name="WristPitchJointName" value="${prefix}WristPitch" />
 </robot>
