Commit message: Removed trash from dh_parameters for the legs.

File: valkyrie_description/robots/valkyrie_A/xacro/leg/dh_parameters.xacro (robot description, xacro)
@@ -1,8 +1,4 @@
 <?xml version="1.0" ?>
 <robot xmlns:xacro="http://www.ros.org/wiki/xacro" name="v1/leg/dh_parameters">
-  <xacro:property name="LJ1_Joint_Offset" value="-0.183" />
-  <xacro:property name="LJ1_Joint_Angle" value="${reflect * -1 * pi_2}" />
-  <xacro:property name="LJ1_Joint_Radius" value="0.1016" />
-  <xacro:property name="LJ1_Joint_Twist" value="${pi * ((1 - reflect)/2)}" />
   <xacro:property name="LJ1_Origin_X" value="0"/>
   <xacro:property name="LJ1_Origin_Y" value="${reflect * -0.1016}"/>
@@ -11,8 +7,4 @@
   <xacro:property name="LJ1_Orientation_Pitch" value="0"/>
   <xacro:property name="LJ1_Orientation_Yaw" value="${reflect * -1 * pi_2}"/>
-  <xacro:property name="LJ2_Joint_Offset" value="0" />
-  <xacro:property name="LJ2_Joint_Angle" value="0" />
-  <xacro:property name="LJ2_Joint_Radius" value="0" />
-  <xacro:property name="LJ2_Joint_Twist" value="${reflect * -1 * pi_2}" />
   <xacro:property name="LJ2_Origin_X" value="0"/>
   <xacro:property name="LJ2_Origin_Y" value="0"/>
@@ -21,8 +13,4 @@
   <xacro:property name="LJ2_Orientation_Pitch" value="0"/>
   <xacro:property name="LJ2_Orientation_Yaw" value="0"/>
-  <xacro:property name="LJ3_Joint_Offset" value="0" />
-  <xacro:property name="LJ3_Joint_Angle" value="${pi_2}" />
-  <xacro:property name="LJ3_Joint_Radius" value="0.061" />
-  <xacro:property name="LJ3_Joint_Twist" value="${reflect * -1 * pi_2}" />
   <xacro:property name="LJ3_Origin_X" value="0"/>
   <xacro:property name="LJ3_Origin_Y" value="0.061"/>
@@ -31,8 +19,4 @@
   <xacro:property name="LJ3_Orientation_Pitch" value="0"/>
   <xacro:property name="LJ3_Orientation_Yaw" value="${pi_2}"/>
-  <xacro:property name="LJ4_Joint_Offset" value="${reflect * -1 * 0.0374}" />
-  <xacro:property name="LJ4_Joint_Angle" value="0" />
-  <xacro:property name="LJ4_Joint_Radius" value="0.431" />
-  <xacro:property name="LJ4_Joint_Twist" value="${pi}" />
   <xacro:property name="LJ4_Origin_X" value="0.431"/>
   <xacro:property name="LJ4_Origin_Y" value="0"/>
@@ -41,8 +25,4 @@
   <xacro:property name="LJ4_Orientation_Pitch" value="0"/>
   <xacro:property name="LJ4_Orientation_Yaw" value="0"/>
-  <xacro:property name="LJ5_Joint_Offset" value="0" />
-  <xacro:property name="LJ5_Joint_Angle" value="0" />
-  <xacro:property name="LJ5_Joint_Radius" value="0.406" />
-  <xacro:property name="LJ5_Joint_Twist" value="${pi}" />
   <xacro:property name="LJ5_Origin_X" value="0.406"/>
   <xacro:property name="LJ5_Origin_Y" value="0"/>
@@ -51,8 +31,4 @@
   <xacro:property name="LJ5_Orientation_Pitch" value="0"/>
   <xacro:property name="LJ5_Orientation_Yaw" value="0"/>
-  <xacro:property name="LJ6_Joint_Offset" value="0" />
-  <xacro:property name="LJ6_Joint_Angle" value="0" />
-  <xacro:property name="LJ6_Joint_Radius" value="0.0127" />
-  <xacro:property name="LJ6_Joint_Twist" value="${reflect * pi_2}" />
   <xacro:property name="LJ6_Origin_X" value="0.0127"/>
   <xacro:property name="LJ6_Origin_Y" value="0"/>
