Commit message: Renamed a bunch of the leg joint stuff. Not quite finished with it yet.

File: valkyrie_description/robots/valkyrie_A/xacro/leg/joint_limits.xacro (robot description, xacro)
@@ -1,27 +1,27 @@
 <?xml version="1.0" ?>
 <robot xmlns:xacro="http://www.ros.org/wiki/xacro" name="v1/leg/joint_limits">
-  <xacro:property name="LJ1_Torque_Limit" value="190" />
-  <xacro:property name="LJ2_Torque_Limit" value="350" />
-  <xacro:property name="LJ3_Torque_Limit" value="350" />
-  <xacro:property name="LJ4_Torque_Limit" value="350" />
-  <xacro:property name="LJ5_Torque_Limit" value="205" />
-  <xacro:property name="LJ6_Torque_Limit" value="205" />
-  <xacro:property name="LJ1_Lower_Limit" value="-0.524" />
-  <xacro:property name="LJ2_Lower_Limit" value="-0.524" />
-  <xacro:property name="LJ3_Lower_Limit" value="-2.356" />
-  <xacro:property name="LJ4_Lower_Limit" value="-1.902" />
-  <xacro:property name="LJ5_Lower_Limit" value="-0.873" />
-  <xacro:property name="LJ6_Lower_Limit" value="-0.349" />
-  <xacro:property name="LJ1_Upper_Limit" value="0.169" />
-  <xacro:property name="LJ2_Upper_Limit" value="0.262" />
-  <xacro:property name="LJ3_Upper_Limit" value="1.710" />
-  <xacro:property name="LJ4_Upper_Limit" value="0.218" />
-  <xacro:property name="LJ5_Upper_Limit" value="0.873" />
-  <xacro:property name="LJ6_Upper_Limit" value="0.349" />
-  <xacro:property name="LJ1_Speed_Limit" value="5.89" />
-  <xacro:property name="LJ2_Speed_Limit" value="7" />
-  <xacro:property name="LJ3_Speed_Limit" value="6.11" />
-  <xacro:property name="LJ4_Speed_Limit" value="6.11" />
-  <xacro:property name="LJ5_Speed_Limit" value="11" />
-  <xacro:property name="LJ6_Speed_Limit" value="11" />
+  <xacro:property name="HipYawTorqueLimit" value="190" />
+  <xacro:property name="HipRollTorqueLimit" value="350" />
+  <xacro:property name="HipPitchTorqueLimit" value="350" />
+  <xacro:property name="KneePitchTorqueLimit" value="350" />
+  <xacro:property name="AnklePitchTorqueLimit" value="205" />
+  <xacro:property name="AnkleRollTorqueLimit" value="205" />
+  <xacro:property name="HipYawPositionLimit_Lower" value="-0.524" />
+  <xacro:property name="HipRollPositionLimit_Lower" value="-0.524" />
+  <xacro:property name="HipPitchPositionLimit_Lower" value="-2.356" />
+  <xacro:property name="KneePitchPositionLimit_Lower" value="-1.902" />
+  <xacro:property name="AnklePitchPositionLimit_Lower" value="-0.873" />
+  <xacro:property name="AnkleRollPositionLimit_Lower" value="-0.349" />
+  <xacro:property name="HipYawPositionLimit_Upper" value="0.169" />
+  <xacro:property name="HipRollPositionLimit_Upper" value="0.262" />
+  <xacro:property name="HipPitchPositionLimit_Upper" value="1.710" />
+  <xacro:property name="KneePitchPositionLimit_Upper" value="0.218" />
+  <xacro:property name="AnklePitchPositionLimit_Upper" value="0.873" />
+  <xacro:property name="AnkleRollPositionLimit_Upper" value="0.349" />
+  <xacro:property name="HipYawVelocityLimit" value="5.89" />
+  <xacro:property name="HipRollVelocityLimit" value="7" />
+  <xacro:property name="HipPitchVelocityLimit" value="6.11" />
+  <xacro:property name="KneePitchVelocityLimit" value="6.11" />
+  <xacro:property name="AnklePitchVelocityLimit" value="11" />
+  <xacro:property name="AnkleRollVelocityLimit" value="11" />
 </robot>

File: valkyrie_description/robots/valkyrie_A/xacro/leg/joint_names.xacro (robot description, xacro)
@@ -1,9 +1,9 @@
 <?xml version="1.0" ?>
 <robot xmlns:xacro="http://www.ros.org/wiki/xacro" name="v1/leg/joint_names">
-  <xacro:property name="LJ1_Joint_Name" value="${prefix}HipYaw" />
-  <xacro:property name="LJ2_Joint_Name" value="${prefix}HipRoll" />
-  <xacro:property name="LJ3_Joint_Name" value="${prefix}HipPitch" />
-  <xacro:property name="LJ4_Joint_Name" value="${prefix}KneePitch" />
-  <xacro:property name="LJ5_Joint_Name" value="${prefix}AnklePitch" />
-  <xacro:property name="LJ6_Joint_Name" value="${prefix}AnkleRoll" />
+  <xacro:property name="HipYawJointName" value="${prefix}HipYaw" />
+  <xacro:property name="HipRollJointName" value="${prefix}HipRoll" />
+  <xacro:property name="HipPitchJointName" value="${prefix}HipPitch" />
+  <xacro:property name="KneePitchJointName" value="${prefix}KneePitch" />
+  <xacro:property name="AnklePitchJointName" value="${prefix}AnklePitch" />
+  <xacro:property name="AnkleRollJointName" value="${prefix}AnkleRoll" />
 </robot>

File: valkyrie_description/robots/valkyrie_A/xacro/leg/leg.xacro (robot description, xacro)
@@ -4,5 +4,5 @@
   <xacro:include filename="$(find valkyrie_description)/robots/valkyrie_A/xacro/leg/link_names.xacro"/>
   <xacro:include filename="$(find valkyrie_description)/robots/valkyrie_A/xacro/leg/joint_limits.xacro"/>
-  <xacro:include filename="$(find valkyrie_description)/robots/valkyrie_A/xacro/leg/dh_parameters.xacro"/>
+  <xacro:include filename="$(find valkyrie_description)/robots/valkyrie_A/xacro/leg/frame_parameters.xacro"/>
   <xacro:include filename="$(find valkyrie_description)/robots/valkyrie_A/xacro/leg/mass_parameters.xacro"/>
   <xacro:include filename="$(find valkyrie_description)/robots/valkyrie_A/xacro/sensors/camboard.xacro"/>
@@ -46,5 +46,5 @@
   <xacro:property name="LJ6_Link_Box_Origin_Z" value="7.7849126e-02"/>
   <xacro:macro name="make_leg_links" params="prefix reflect leg_root_link">
-    <xacro:box_link name="${LJ1_Distal_Link}"
+    <xacro:box_link name="${HipYawLinkName}"
                     width="${LJ1_Link_Width}" height="${LJ1_Link_Height}" depth="${LJ1_Link_Length}" mass="${LJ1_Link_Mass}"
                     origin_xyz="${LJ1_Link_Origin_X} ${LJ1_Link_Origin_Y} ${reflect * LJ1_Link_Origin_Z}" origin_rpy="0 0 0"
@@ -52,5 +52,5 @@
                     material="Gold"
                     collision_mesh="${mesh_root}/lj1_${prefix}.stl"/>
-    <xacro:box_link name="${LJ2_Distal_Link}"
+    <xacro:box_link name="${HipRollLinkName}"
                     width="${LJ2_Link_Width}" height="${LJ2_Link_Height}" depth="${LJ2_Link_Length}" mass="${LJ2_Link_Mass}"
                     origin_rpy="0 0 0"
@@ -59,5 +59,5 @@
                     material="White"
                     collision_mesh="${mesh_root}/lj2.stl"/>
-    <xacro:box_link name="${LJ3_Distal_Link}"
+    <xacro:box_link name="${HipPitchLinkName}"
                     width="${LJ3_Link_Width}" height="${LJ3_Link_Height}" depth="${LJ3_Link_Length}" mass="${LJ3_Link_Mass}"
                     origin_rpy="0 0 0"
@@ -66,5 +66,5 @@
                     material="White"
                     collision_mesh="${mesh_root}/lj3_${prefix}.stl"/>
-    <xacro:box_link name="${LJ4_Distal_Link_Box}"
+    <xacro:box_link name="${KneePitchLinkName}"
                     width="${LJ4_Link_Box_Width}" height="${LJ4_Link_Box_Height}" depth="${LJ4_Link_Box_Length}" mass="${LJ4_Link_Box_Mass}"
                     origin_rpy="0 0 0"
@@ -73,9 +73,9 @@
                     material="White"
                     collision_mesh="${mesh_root}/lj4_${prefix}.stl"/>
-    <xacro:box_link_no_mesh name="${LJ5_Distal_Link}"
+    <xacro:box_link_no_mesh name="${AnklePitchLinkName}"
                     width="${LJ5_Link_Width}" height="${LJ5_Link_Height}" depth="${LJ5_Link_Length}" mass="${LJ5_Link_Mass}"
                     origin_rpy="0 0 0"
                     origin_xyz="${LJ5_Link_Box_Origin_X} ${LJ5_Link_Box_Origin_Y} ${LJ5_Link_Box_Origin_Z}"/>
-    <xacro:box_link_primitive_collision_origin_offset name="${LJ6_Distal_Link}"
+    <xacro:box_link_primitive_collision_origin_offset name="${AnkleRollLinkName}"
                     width="${LJ6_Link_Width}" height="${LJ6_Link_Height}" depth="${LJ6_Link_Length}" mass="${LJ6_Link_Mass}"
                     origin_rpy="0 ${reflect * 0.13} 0"
@@ -85,5 +85,5 @@
                     origin_offset_xyz="0 0 0"
                     origin_offset_rpy="0 ${reflect * 0.13} 0"/>
-    <gazebo reference="${LJ6_Distal_Link}">
+    <gazebo reference="${AnkleRollLinkName}">
       <kp>100000.0</kp>
       <kd>1000.0</kd>
@@ -97,86 +97,86 @@
   <xacro:macro name="make_leg_joints" params="prefix reflect leg_root_link">
     <!-- LJ1 -->
-    <xacro:revolute_joint_ex jointName="${LJ1_Joint_Name}"
-                          parent="${LJ1_Proximal_Link}" child="${LJ1_Distal_Link}"
+    <xacro:revolute_joint_ex jointName="${HipYawJointName}"
+                          parent="${HipYawParentLinkName}" child="${HipYawLinkName}"
                           origin_xyz="${HipYawFrameOrigin_X} ${HipYawFrameOrigin_Y} ${HipYawFrameOrigin_Z}"
                           origin_rpy="${HipYawFrameOrientation_Roll} ${HipYawFrameOrientation_Pitch} ${HipYawFrameOrientation_Yaw}"
                           damping="1.0" friction="0.0">
-        <limit effort="${LJ1_Torque_Limit}" lower="${LJ1_Lower_Limit}" upper="${LJ1_Upper_Limit}" velocity="${LJ1_Speed_Limit}"/>
-        <controller_gains Kp="15000" Kd="500"/>
-    </xacro:revolute_joint_ex>
-    <xacro:revolute_joint_ex jointName="${LJ2_Joint_Name}"
-                          parent="${LJ2_Proximal_Link}" child="${LJ2_Distal_Link}"
+        <limit effort="${HipYawTorqueLimit}" lower="${HipYawPositionLimit_Lower}" upper="${HipYawPositionLimit_Upper}" velocity="${HipYawVelocityLimit}"/>
+        <controller_gains Kp="15000" Kd="500"/>
+    </xacro:revolute_joint_ex>
+    <xacro:revolute_joint_ex jointName="${HipRollJointName}"
+                          parent="${HipYawLinkName}" child="${HipRollLinkName}"
                           origin_xyz="${HipRollFrameOrigin_X} ${HipRollFrameOrigin_Y} ${HipRollFrameOrigin_Z}"
                           origin_rpy="${HipRollFrameOrientation_Roll} ${HipRollFrameOrientation_Pitch} ${HipRollFrameOrientation_Yaw}"
                           damping="1.0" friction="0.0">
-        <limit effort="${LJ2_Torque_Limit}" lower="${LJ2_Lower_Limit}" upper="${LJ2_Upper_Limit}" velocity="${LJ2_Speed_Limit}"/>
-        <controller_gains Kp="15000" Kd="500"/>
-    </xacro:revolute_joint_ex>
-    <xacro:revolute_joint_ex jointName="${LJ3_Joint_Name}"
-                          parent="${LJ3_Proximal_Link}" child="${LJ3_Distal_Link}"
+        <limit effort="${HipRollTorqueLimit}" lower="${HipRollPositionLimit_Lower}" upper="${HipRollPositionLimit_Upper}" velocity="${HipRollVelocityLimit}"/>
+        <controller_gains Kp="15000" Kd="500"/>
+    </xacro:revolute_joint_ex>
+    <xacro:revolute_joint_ex jointName="${HipPitchJointName}"
+                          parent="${HipRollLinkName}" child="${HipPitchLinkName}"
                           origin_xyz="${HipPitchFrameOrigin_X} ${HipPitchFrameOrigin_Y} ${HipPitchFrameOrigin_Z}"
                           origin_rpy="${HipPitchFrameOrientation_Roll} ${HipPitchFrameOrientation_Pitch} ${HipPitchFrameOrientation_Yaw}"
                           damping="1.0" friction="0.0">
-        <limit effort="${LJ3_Torque_Limit}" lower="${LJ3_Lower_Limit}" upper="${LJ3_Upper_Limit}" velocity="${LJ3_Speed_Limit}"/>
-        <controller_gains Kp="15000" Kd="500"/>
-    </xacro:revolute_joint_ex>
-    <xacro:revolute_joint_ex jointName="${LJ4_Joint_Name}"
-                          parent="${LJ4_Proximal_Link}" child="${LJ4_Distal_Link_Box}"
+        <limit effort="${HipPitchTorqueLimit}" lower="${HipPitchPositionLimit_Lower}" upper="${HipPitchPositionLimit_Upper}" velocity="${HipPitchVelocityLimit}"/>
+        <controller_gains Kp="15000" Kd="500"/>
+    </xacro:revolute_joint_ex>
+    <xacro:revolute_joint_ex jointName="${KneePitchJointName}"
+                          parent="${HipPitchLinkName}" child="${KneePitchLinkName}"
                           origin_xyz="${KneePitchFrameOrigin_X} ${KneePitchFrameOrigin_Y} ${KneePitchFrameOrigin_Z}"
                           origin_rpy="${KneePitchFrameOrientation_Roll} ${KneePitchFrameOrientation_Pitch} ${KneePitchFrameOrientation_Yaw}"
                           damping="1.0" friction="0.0">
-        <limit effort="${LJ4_Torque_Limit}" lower="${LJ4_Lower_Limit}" upper="${LJ4_Upper_Limit}" velocity="${LJ4_Speed_Limit}"/>
+        <limit effort="${KneePitchTorqueLimit}" lower="${KneePitchPositionLimit_Lower}" upper="${KneePitchPositionLimit_Upper}" velocity="${KneePitchVelocityLimit}"/>
         <controller_gains Kp="15000" Kd="500"/>
     </xacro:revolute_joint_ex>
   </xacro:macro>
   <xacro:macro name="make_leg_joints_fixed" params="prefix reflect leg_root_link">
-    <xacro:fixed_joint jointName="${LJ1_Joint_Name}"
-                          parent="${LJ1_Proximal_Link}" child="${LJ1_Distal_Link}"
+    <xacro:fixed_joint jointName="${HipYawJointName}"
+                          parent="${HipYawParentLinkName}" child="${HipYawLinkName}"
                           origin_xyz="${HipYawFrameOrigin_X} ${HipYawFrameOrigin_Y} ${HipYawFrameOrigin_Z}"
                           origin_rpy="${HipYawFrameOrientation_Roll} ${HipYawFrameOrientation_Pitch} ${HipYawFrameOrientation_Yaw}">
-        <limit effort="${LJ1_Torque_Limit}" lower="${LJ1_Lower_Limit}" upper="${LJ1_Upper_Limit}" velocity="${LJ1_Speed_Limit}"/>
-    </xacro:fixed_joint>
-    <xacro:fixed_joint jointName="${LJ2_Joint_Name}"
-                          parent="${LJ2_Proximal_Link}" child="${LJ2_Distal_Link}"
+        <limit effort="${HipYawTorqueLimit}" lower="${HipYawPositionLimit_Lower}" upper="${HipYawPositionLimit_Upper}" velocity="${HipYawVelocityLimit}"/>
+    </xacro:fixed_joint>
+    <xacro:fixed_joint jointName="${HipRollJointName}"
+                          parent="${HipYawLinkName}" child="${HipRollLinkName}"
                           origin_xyz="${HipRollFrameOrigin_X} ${HipRollFrameOrigin_Y} ${HipRollFrameOrigin_Z}"
                           origin_rpy="${HipRollFrameOrientation_Roll} ${HipRollFrameOrientation_Pitch} ${HipRollFrameOrientation_Yaw}">
-        <limit effort="${LJ2_Torque_Limit}" lower="${LJ2_Lower_Limit}" upper="${LJ2_Upper_Limit}" velocity="${LJ2_Speed_Limit}"/>
-    </xacro:fixed_joint>
-    <xacro:fixed_joint jointName="${LJ3_Joint_Name}"
-                          parent="${LJ3_Proximal_Link}" child="${LJ3_Distal_Link}"
+        <limit effort="${HipRollTorqueLimit}" lower="${HipRollPositionLimit_Lower}" upper="${HipRollPositionLimit_Upper}" velocity="${HipRollVelocityLimit}"/>
+    </xacro:fixed_joint>
+    <xacro:fixed_joint jointName="${HipPitchJointName}"
+                          parent="${HipRollLinkName}" child="${HipPitchLinkName}"
                           origin_xyz="${HipPitchFrameOrigin_X} ${HipPitchFrameOrigin_Y} ${HipPitchFrameOrigin_Z}"
                           origin_rpy="${HipPitchFrameOrientation_Roll} ${HipPitchFrameOrientation_Pitch} ${HipPitchFrameOrientation_Yaw}">
-        <limit effort="${LJ3_Torque_Limit}" lower="${LJ3_Lower_Limit}" upper="${LJ3_Upper_Limit}" velocity="${LJ3_Speed_Limit}"/>
-    </xacro:fixed_joint>
-    <xacro:fixed_joint jointName="${LJ4_Joint_Name}"
-                          parent="${LJ4_Proximal_Link}" child="${LJ4_Distal_Link_Box}"
+        <limit effort="${HipPitchTorqueLimit}" lower="${HipPitchPositionLimit_Lower}" upper="${HipPitchPositionLimit_Upper}" velocity="${HipPitchVelocityLimit}"/>
+    </xacro:fixed_joint>
+    <xacro:fixed_joint jointName="${KneePitchJointName}"
+                          parent="${HipPitchLinkName}" child="${KneePitchLinkName}"
                           origin_xyz="${KneePitchFrameOrigin_X} ${KneePitchFrameOrigin_Y} ${KneePitchFrameOrigin_Z}"
                           origin_rpy="${KneePitchFrameOrientation_Roll} ${KneePitchFrameOrientation_Pitch} ${KneePitchFrameOrientation_Yaw}">
-        <limit effort="${LJ4_Torque_Limit}" lower="${LJ4_Lower_Limit}" upper="${LJ4_Upper_Limit}" velocity="${LJ4_Speed_Limit}"/>
+        <limit effort="${KneePitchTorqueLimit}" lower="${KneePitchPositionLimit_Lower}" upper="${KneePitchPositionLimit_Upper}" velocity="${KneePitchVelocityLimit}"/>
     </xacro:fixed_joint>
   </xacro:macro>
   <xacro:macro name="make_ankle_joints" params="prefix reflect leg_root_link">
     <!--     <xacro:fixed_joint jointName="${prefix}MedialAnkleActuatorOffset"
-                       parent="${LJ4_Distal_Link_Box}" child="${LJ4_Distal_Link_Cylinder1}"
+                       parent="${KneePitchLinkName}" child="${LJ4_Distal_Link_Cylinder1}"
                        origin_xyz="0 0 0"
                        origin_rpy="0 0 0"/><controller_gains Kp="15000" Kd="2<controller_gains Kp="15000" Kd="500"/>
     <xacro:fixed_joint jointName="${prefix}LateralAnkleActuatorOffset"
-                       parent="${LJ4_Distal_Link_Box}" child="${LJ4_Distal_Link_Cylinder2}"
+                       parent="${KneePitchLinkName}" child="${LJ4_Distal_Link_Cylinder2}"
                        origin_xyz="0 0 0"
                        origin_rpy="0 0 0"/> -->
-    <xacro:revolute_joint_ex jointName="${LJ5_Joint_Name}"
-                          parent="${LJ5_Proximal_Link}" child="${LJ5_Distal_Link}"
+    <xacro:revolute_joint_ex jointName="${AnklePitchJointName}"
+                          parent="${KneePitchLinkName}" child="${AnklePitchLinkName}"
                           origin_xyz="${AnklePitchFrameOrigin_X} ${AnklePitchFrameOrigin_Y} ${AnklePitchFrameOrigin_Z}"
                           origin_rpy="${AnklePitchFrameOrientation_Roll} ${AnklePitchFrameOrientation_Pitch} ${AnklePitchFrameOrientation_Yaw}"
                           damping="1.0" friction="0.0">
-        <limit effort="${LJ5_Torque_Limit}" lower="${LJ5_Lower_Limit}" upper="${LJ5_Upper_Limit}" velocity="${LJ5_Speed_Limit}"/>
+        <limit effort="${AnklePitchTorqueLimit}" lower="${AnklePitchPositionLimit_Lower}" upper="${AnklePitchPositionLimit_Upper}" velocity="${AnklePitchVelocityLimit}"/>
         <controller_gains Kp="15000" Kd="400"/>
     </xacro:revolute_joint_ex>
-    <xacro:revolute_joint_ex jointName="${LJ6_Joint_Name}"
-                          parent="${LJ6_Proximal_Link}" child="${LJ6_Distal_Link}"
+    <xacro:revolute_joint_ex jointName="${AnkleRollJointName}"
+                          parent="${AnklePitchLinkName}" child="${AnkleRollLinkName}"
                           origin_xyz="${AnkleRollFrameOrigin_X} ${AnkleRollFrameOrigin_Y} ${AnkleRollFrameOrigin_Z}"
                           origin_rpy="${AnkleRollFrameOrientation_Roll} ${AnkleRollFrameOrientation_Pitch} ${AnkleRollFrameOrientation_Yaw}"
                           damping="0.3" friction="0.0">
-        <limit effort="${LJ6_Torque_Limit}" lower="${LJ6_Lower_Limit}" upper="${LJ6_Upper_Limit}" velocity="${LJ6_Speed_Limit}"/>
+        <limit effort="${AnkleRollTorqueLimit}" lower="${AnkleRollPositionLimit_Lower}" upper="${AnkleRollPositionLimit_Upper}" velocity="${AnkleRollVelocityLimit}"/>
         <controller_gains Kp="15000" Kd="400"/>
     </xacro:revolute_joint_ex>
@@ -184,12 +184,12 @@
   <xacro:macro name="make_ankle_joints_fixed" params="prefix reflect leg_root_link">
     <!-- LJ5 -->
-    <xacro:fixed_joint jointName="${LJ5_Joint_Name}"
-                       parent="${LJ5_Proximal_Link}" child="${LJ5_Distal_Link}"
+    <xacro:fixed_joint jointName="${AnklePitchJointName}"
+                       parent="${KneePitchLinkName}" child="${AnklePitchLinkName}"
                        origin_xyz="${AnklePitchFrameOrigin_X} ${AnklePitchFrameOrigin_Y} ${AnklePitchFrameOrigin_Z}"
                        origin_rpy="${AnklePitchFrameOrientation_Roll} ${AnklePitchFrameOrientation_Pitch} ${AnklePitchFrameOrientation_Yaw}">
     </xacro:fixed_joint>
     <!-- LJ6 -->
-    <xacro:fixed_joint jointName="${LJ6_Joint_Name}"
-                          parent="${LJ6_Proximal_Link}" child="${LJ6_Distal_Link}"
+    <xacro:fixed_joint jointName="${AnkleRollJointName}"
+                          parent="${AnklePitchLinkName}" child="${AnkleRollLinkName}"
                           origin_xyz="${AnkleRollFrameOrigin_X} ${AnkleRollFrameOrigin_Y} ${AnkleRollFrameOrigin_Z}"
                           origin_rpy="${AnkleRollFrameOrientation_Roll} ${AnkleRollFrameOrientation_Pitch} ${AnkleRollFrameOrientation_Yaw}">
@@ -217,21 +217,21 @@
   <xacro:macro name="v1_leg_sensors" params="prefix reflect">
     <xacro:camboard_sensor sensorName="/v1/${prefix}LegCamBoard"
-                       parentLink="${LJ4_Distal_Link_Box}"
+                       parentLink="${KneePitchLinkName}"
                        origin_xyz="0.344887 0.069118 ${reflect * -0.008500}"
                        origin_rpy="-1.57 0 1.3"/>
     <xacro:virtual_fixed_frame_offset name="/v1/${prefix}COP"
-                       parentLink="${LJ6_Distal_Link}"
+                       parentLink="${AnkleRollLinkName}"
                        origin_xyz="0.0845 0 0"
                        origin_rpy="${1.57 + reflect * -1.57} ${reflect * -1.57} 0"/>
     <xacro:virtual_fixed_frame_offset name="/v1/${prefix}Leg6Axis"
-                       parentLink="${LJ6_Distal_Link}"
+                       parentLink="${AnkleRollLinkName}"
                        origin_xyz="0.058547 0 ${reflect * 0.0215}"
                        origin_rpy="0 0 0"/>
     <xacro:virtual_fixed_frame_offset name="/v1/${prefix}LegHermes"
-                       parentLink="${LJ6_Distal_Link}"
+                       parentLink="${AnkleRollLinkName}"
                        origin_xyz="0.0845 0 0"
                        origin_rpy="${1.57 + reflect * -1.57} ${reflect * -1.57} 0"/>
     <xacro:virtual_fixed_frame_offset name="/v1/${prefix}MPU6000"
-                       parentLink="${LJ6_Distal_Link}"
+                       parentLink="${AnkleRollLinkName}"
                        origin_xyz="0.0471 ${reflect * 0.00722} ${reflect * 0.0843}"
                        origin_rpy="0 ${reflect * 1.57 - 0.13} ${1.57 + reflect * 1.57}"/>
