Commit message: Updated frame parameters for waist and legs.

File: valkyrie_description/robots/valkyrie_A/xacro/leg/frame_parameters.xacro (robot description, xacro)
@@ -2,6 +2,6 @@
 <robot xmlns:xacro="http://www.ros.org/wiki/xacro" name="v1/leg/dh_parameters">
   <xacro:property name="HipYawFrameOrigin_X" value="0.0"/>
-  <xacro:property name="HipYawFrameOrigin_Y" value="${reflect * -0.1016}"/>
-  <xacro:property name="HipYawFrameOrigin_Z" value="-0.183"/>
+  <xacro:property name="HipYawFrameOrigin_Y" value="${reflect * 0.1016}"/>
+  <xacro:property name="HipYawFrameOrigin_Z" value="-0.1853"/>
   <xacro:property name="HipYawFrameOrientation_Roll" value="0.0"/>
   <xacro:property name="HipYawFrameOrientation_Pitch" value="0.0"/>
@@ -13,27 +13,27 @@
   <xacro:property name="HipRollFrameOrientation_Pitch" value="0.0"/>
   <xacro:property name="HipRollFrameOrientation_Yaw" value="0.0"/>
-  <xacro:property name="HipPitchFrameOrigin_X" value="0"/>
-  <xacro:property name="HipPitchFrameOrigin_Y" value="0.061"/>
-  <xacro:property name="HipPitchFrameOrigin_Z" value="0"/>
+  <xacro:property name="HipPitchFrameOrigin_X" value="0.0"/>
+  <xacro:property name="HipPitchFrameOrigin_Y" value="0.0"/>
+  <xacro:property name="HipPitchFrameOrigin_Z" value="-0.0609"/>
   <xacro:property name="HipPitchFrameOrientation_Roll" value="0.0"/>
   <xacro:property name="HipPitchFrameOrientation_Pitch" value="0.0"/>
   <xacro:property name="HipPitchFrameOrientation_Yaw" value="0.0"/>
-  <xacro:property name="KneePitchFrameOrigin_X" value="0.431"/>
-  <xacro:property name="KneePitchFrameOrigin_Y" value="0.0"/>
-  <xacro:property name="KneePitchFrameOrigin_Z" value="${reflect * -1 * 0.0374}"/>
+  <xacro:property name="KneePitchFrameOrigin_X" value="0.0001"/>
+  <xacro:property name="KneePitchFrameOrigin_Y" value="${reflect * 0.0361}"/>
+  <xacro:property name="KneePitchFrameOrigin_Z" value="-0.4306"/>
   <xacro:property name="KneePitchFrameOrientation_Roll" value="0.0"/>
   <xacro:property name="KneePitchFrameOrientation_Pitch" value="0.0"/>
   <xacro:property name="KneePitchFrameOrientation_Yaw" value="0.0"/>
-  <xacro:property name="AnklePitchFrameOrigin_X" value="0.406"/>
+  <xacro:property name="AnklePitchFrameOrigin_X" value="-0.0103"/>
   <xacro:property name="AnklePitchFrameOrigin_Y" value="0.0"/>
-  <xacro:property name="AnklePitchFrameOrigin_Z" value="0.0"/>
+  <xacro:property name="AnklePitchFrameOrigin_Z" value="-0.4064"/>
   <xacro:property name="AnklePitchFrameOrientation_Roll" value="0.0"/>
   <xacro:property name="AnklePitchFrameOrientation_Pitch" value="0.0"/>
   <xacro:property name="AnklePitchFrameOrientation_Yaw" value="0.0"/>
-  <xacro:property name="AnkleRollFrameOrigin_X" value="0.0127"/>
+  <xacro:property name="AnkleRollFrameOrigin_X" value="0.0017"/>
   <xacro:property name="AnkleRollFrameOrigin_Y" value="0.0"/>
-  <xacro:property name="AnkleRollFrameOrigin_Z" value="0.0"/>
+  <xacro:property name="AnkleRollFrameOrigin_Z" value="-0.0126"/>
   <xacro:property name="AnkleRollFrameOrientation_Roll" value="0.0"/>
-  <xacro:property name="AnkleRollFrameOrientation_Pitch" value="0.0"/>
-  <xacro:property name="AnkleRollFrameOrientation_Yaw" value="-0.13"/>
+  <xacro:property name="AnkleRollFrameOrientation_Pitch" value="-0.1309"/>
+  <xacro:property name="AnkleRollFrameOrientation_Yaw" value="0.0"/>
 </robot>

File: valkyrie_description/robots/valkyrie_A/xacro/waist/frame_parameters.xacro (robot description, xacro)
@@ -1,19 +1,19 @@
 <?xml version="1.0" ?>
 <robot xmlns:xacro="http://www.ros.org/wiki/xacro" name="v1/waist/dh_parameters">
-  <xacro:property name="TorsoYawFrameOrigin_X" value="0"/>
-  <xacro:property name="TorsoYawFrameOrigin_Y" value="0"/>
-  <xacro:property name="TorsoYawFrameOrigin_Z" value="0"/>
+  <xacro:property name="TorsoYawFrameOrigin_X" value="0.0"/>
+  <xacro:property name="TorsoYawFrameOrigin_Y" value="0.0"/>
+  <xacro:property name="TorsoYawFrameOrigin_Z" value="0.0"/>
   <xacro:property name="TorsoYawFrameOrientation_Roll" value="0.0"/>
   <xacro:property name="TorsoYawFrameOrientation_Pitch" value="0.0"/>
   <xacro:property name="TorsoYawFrameOrientation_Yaw" value="0.0"/>
   <xacro:property name="TorsoPitchFrameOrigin_X" value="0.04191"/>
-  <xacro:property name="TorsoPitchFrameOrigin_Y" value="0"/>
-  <xacro:property name="TorsoPitchFrameOrigin_Z" value="0"/>
+  <xacro:property name="TorsoPitchFrameOrigin_Y" value="0.0"/>
+  <xacro:property name="TorsoPitchFrameOrigin_Z" value="0.0"/>
   <xacro:property name="TorsoPitchFrameOrientation_Roll" value="0.0"/>
   <xacro:property name="TorsoPitchFrameOrientation_Pitch" value="0.0"/>
   <xacro:property name="TorsoPitchFrameOrientation_Yaw" value="0.0"/>
-  <xacro:property name="TorsoRollFrameOrigin_X" value="0"/>
-  <xacro:property name="TorsoRollFrameOrigin_Y" value="0.020352"/>
-  <xacro:property name="TorsoRollFrameOrigin_Z" value="0"/>
+  <xacro:property name="TorsoRollFrameOrigin_X" value="0.0"/>
+  <xacro:property name="TorsoRollFrameOrigin_Y" value="0.0"/>
+  <xacro:property name="TorsoRollFrameOrigin_Z" value="0.0203"/>
   <xacro:property name="TorsoRollFrameOrientation_Roll" value="0.0"/>
   <xacro:property name="TorsoRollFrameOrientation_Pitch" value="0.0"/>
