Commit message: First pass of renaming stuff for the leg xacros is done.

File: valkyrie_description/robots/valkyrie_A/xacro/leg/leg.xacro (robot description, xacro)
@@ -47,5 +47,5 @@
   <xacro:macro name="make_leg_links" params="prefix reflect leg_root_link">
     <xacro:box_link name="${HipYawLinkName}"
-                    width="${LJ1_Link_Width}" height="${LJ1_Link_Height}" depth="${LJ1_Link_Length}" mass="${LJ1_Link_Mass}"
+                    width="${LJ1_Link_Width}" height="${LJ1_Link_Height}" depth="${LJ1_Link_Length}" mass="${HipYawLinkMass}"
                     origin_xyz="${LJ1_Link_Origin_X} ${LJ1_Link_Origin_Y} ${reflect * LJ1_Link_Origin_Z}" origin_rpy="0 0 0"
                     visual_mesh="${mesh_root}/lj1_${prefix}.stl"
@@ -53,5 +53,5 @@
                     collision_mesh="${mesh_root}/lj1_${prefix}.stl"/>
     <xacro:box_link name="${HipRollLinkName}"
-                    width="${LJ2_Link_Width}" height="${LJ2_Link_Height}" depth="${LJ2_Link_Length}" mass="${LJ2_Link_Mass}"
+                    width="${LJ2_Link_Width}" height="${LJ2_Link_Height}" depth="${LJ2_Link_Length}" mass="${HipRollLinkMass}"
                     origin_rpy="0 0 0"
                     origin_xyz="${LJ2_Link_Origin_X} ${LJ2_Link_Origin_Y} ${LJ2_Link_Origin_Z}"
@@ -60,5 +60,5 @@
                     collision_mesh="${mesh_root}/lj2.stl"/>
     <xacro:box_link name="${HipPitchLinkName}"
-                    width="${LJ3_Link_Width}" height="${LJ3_Link_Height}" depth="${LJ3_Link_Length}" mass="${LJ3_Link_Mass}"
+                    width="${LJ3_Link_Width}" height="${LJ3_Link_Height}" depth="${LJ3_Link_Length}" mass="${HipPitchLinkMass}"
                     origin_rpy="0 0 0"
                     origin_xyz="${LJ3_Link_Origin_X} ${LJ3_Link_Origin_Y} ${reflect * LJ3_Link_Origin_Z}"
@@ -67,5 +67,5 @@
                     collision_mesh="${mesh_root}/lj3_${prefix}.stl"/>
     <xacro:box_link name="${KneePitchLinkName}"
-                    width="${LJ4_Link_Box_Width}" height="${LJ4_Link_Box_Height}" depth="${LJ4_Link_Box_Length}" mass="${LJ4_Link_Box_Mass}"
+                    width="${LJ4_Link_Box_Width}" height="${LJ4_Link_Box_Height}" depth="${LJ4_Link_Box_Length}" mass="${KneePitchLinkMass}"
                     origin_rpy="0 0 0"
                     origin_xyz="${LJ4_Link_Box_Origin_X} ${LJ4_Link_Box_Origin_Y} ${reflect * LJ4_Link_Box_Origin_Z}"
@@ -74,9 +74,9 @@
                     collision_mesh="${mesh_root}/lj4_${prefix}.stl"/>
     <xacro:box_link_no_mesh name="${AnklePitchLinkName}"
-                    width="${LJ5_Link_Width}" height="${LJ5_Link_Height}" depth="${LJ5_Link_Length}" mass="${LJ5_Link_Mass}"
+                    width="${LJ5_Link_Width}" height="${LJ5_Link_Height}" depth="${LJ5_Link_Length}" mass="${AnklePitchLinkMass}"
                     origin_rpy="0 0 0"
                     origin_xyz="${LJ5_Link_Box_Origin_X} ${LJ5_Link_Box_Origin_Y} ${LJ5_Link_Box_Origin_Z}"/>
     <xacro:box_link_primitive_collision_origin_offset name="${AnkleRollLinkName}"
-                    width="${LJ6_Link_Width}" height="${LJ6_Link_Height}" depth="${LJ6_Link_Length}" mass="${LJ6_Link_Mass}"
+                    width="${LJ6_Link_Width}" height="${LJ6_Link_Height}" depth="${LJ6_Link_Length}" mass="${FootMass}"
                     origin_rpy="0 ${reflect * 0.13} 0"
                     origin_xyz="${LJ6_Link_Box_Origin_X} ${LJ6_Link_Box_Origin_Y} ${reflect * LJ6_Link_Box_Origin_Z}"

File: valkyrie_description/robots/valkyrie_A/xacro/leg/mass_parameters.xacro (robot description, xacro)
@@ -1,9 +1,9 @@
 <?xml version="1.0" ?>
 <robot xmlns:xacro="http://www.ros.org/wiki/xacro" name="v1/leg/mass_parameters">
-  <xacro:property name="LJ1_Link_Mass" value="2.39" />
-  <xacro:property name="LJ2_Link_Mass" value="5.95" />
-  <xacro:property name="LJ3_Link_Mass" value="10.3" />
-  <xacro:property name="LJ4_Link_Box_Mass" value="7.4" />
-  <xacro:property name="LJ5_Link_Mass" value="0.395" />
-  <xacro:property name="LJ6_Link_Mass" value="1.888" />
+  <xacro:property name="HipYawLinkMass" value="2.39" />
+  <xacro:property name="HipRollLinkMass" value="5.95" />
+  <xacro:property name="HipPitchLinkMass" value="10.3" />
+  <xacro:property name="KneePitchLinkMass" value="7.4" />
+  <xacro:property name="AnklePitchLinkMass" value="0.395" />
+  <xacro:property name="FootMass" value="1.888" />
 </robot>

Commit message: Updated COM locations of legs for new frame orientations. Also extracted out the xacro properties for leg COM positions to mass_parameters.xacro. Will continue on with all the other links.

File: valkyrie_description/robots/valkyrie_A/xacro/leg/leg.xacro (robot description, xacro)
@@ -11,41 +11,29 @@
   <xacro:property name="LJ1_Link_Height" value="0.185"/>
   <xacro:property name="LJ1_Link_Length" value="0.229"/>
-  <xacro:property name="LJ1_Link_Origin_X" value="1.3078570e-03"/>
+  <xacro:property name="LJ1_Link_Origin_X" value="0.02176"/>
+  <xacro:property name="LJ1_Link_Origin_Y" value="0.0013"/>
+  <xacro:property name="LJ1_Link_Origin_Z" value="0.03867"/>
+  <!-- <xacro:property name="LJ1_Link_Origin_X" value="1.3078570e-03"/>
   <xacro:property name="LJ1_Link_Origin_Y" value="2.1764163e-02"/>
-  <xacro:property name="LJ1_Link_Origin_Z" value="3.8670367e-02"/>
+  <xacro:property name="LJ1_Link_Origin_Z" value="3.8670367e-02"/> -->
   <xacro:property name="LJ2_Link_Width" value="0.131"/>
   <xacro:property name="LJ2_Link_Height" value="0.185"/>
   <xacro:property name="LJ2_Link_Length" value="0.123"/>
-  <xacro:property name="LJ2_Link_Origin_X" value="2.4260044e-02"/>
-  <xacro:property name="LJ2_Link_Origin_Y" value="1.9261751e-02"/>
-  <xacro:property name="LJ2_Link_Origin_Z" value="-1.8458616e-03"/>
   <xacro:property name="LJ3_Link_Width" value="0.55419965909040602714"/>
   <xacro:property name="LJ3_Link_Height" value="0.24253719562602335524"/>
   <xacro:property name="LJ3_Link_Length" value="0.18520578950459243295"/>
-  <xacro:property name="LJ3_Link_Origin_X" value="0.220"/>
-  <xacro:property name="LJ3_Link_Origin_Y" value="0"/>
-  <xacro:property name="LJ3_Link_Origin_Z" value="-0.05"/>
   <xacro:property name="LJ4_Link_Box_Width" value="0.44528684954574881960"/>
   <xacro:property name="LJ4_Link_Box_Height" value="0.20288766696230062236"/>
   <xacro:property name="LJ4_Link_Box_Length" value="0.20551228016178813007"/>
-  <xacro:property name="LJ4_Link_Box_Origin_X" value="0.185"/>
-  <xacro:property name="LJ4_Link_Box_Origin_Y" value="0.0"/>
-  <xacro:property name="LJ4_Link_Box_Origin_Z" value="0.045"/>
   <xacro:property name="LJ5_Link_Width" value="0.033"/>
   <xacro:property name="LJ5_Link_Height" value="0.076"/>
   <xacro:property name="LJ5_Link_Length" value="0.025"/>
-  <xacro:property name="LJ5_Link_Box_Origin_X" value="5.7963439e-03"/>
-  <xacro:property name="LJ5_Link_Box_Origin_Y" value="2.0433211e-03"/>
-  <xacro:property name="LJ5_Link_Box_Origin_Z" value="9.0424431e-05"/>
   <xacro:property name="LJ6_Link_Width" value="0.082"/>
   <xacro:property name="LJ6_Link_Height" value="0.128"/>
   <xacro:property name="LJ6_Link_Length" value="0.300"/>
-  <xacro:property name="LJ6_Link_Box_Origin_X" value="4.8263578e-02"/>
-  <xacro:property name="LJ6_Link_Box_Origin_Y" value="-3.1591183e-05"/>
-  <xacro:property name="LJ6_Link_Box_Origin_Z" value="7.7849126e-02"/>
   <xacro:macro name="make_leg_links" params="prefix reflect leg_root_link">
     <xacro:box_link name="${HipYawLinkName}"
                     width="${LJ1_Link_Width}" height="${LJ1_Link_Height}" depth="${LJ1_Link_Length}" mass="${HipYawLinkMass}"
-                    origin_xyz="${LJ1_Link_Origin_X} ${LJ1_Link_Origin_Y} ${reflect * LJ1_Link_Origin_Z}" origin_rpy="0 0 0"
+                    origin_xyz="${HipYawLinkComPosition}" origin_rpy="0 0 0"
                     visual_mesh="${mesh_root}/lj1_${prefix}.stl"
                     material="Gold"
@@ -53,6 +41,6 @@
     <xacro:box_link name="${HipRollLinkName}"
                     width="${LJ2_Link_Width}" height="${LJ2_Link_Height}" depth="${LJ2_Link_Length}" mass="${HipRollLinkMass}"
+                    origin_xyz="${HipRollLinkComPosition}"
                     origin_rpy="0 0 0"
-                    origin_xyz="${LJ2_Link_Origin_X} ${LJ2_Link_Origin_Y} ${LJ2_Link_Origin_Z}"
                     visual_mesh="${mesh_root}/lj2_${prefix}.stl"
                     material="White"
@@ -60,6 +48,6 @@
     <xacro:box_link name="${HipPitchLinkName}"
                     width="${LJ3_Link_Width}" height="${LJ3_Link_Height}" depth="${LJ3_Link_Length}" mass="${HipPitchLinkMass}"
+                    origin_xyz="${HipPitchLinkComPosition}"
                     origin_rpy="0 0 0"
-                    origin_xyz="${LJ3_Link_Origin_X} ${LJ3_Link_Origin_Y} ${reflect * LJ3_Link_Origin_Z}"
                     visual_mesh="${mesh_root}/lj3_${prefix}.stl"
                     material="White"
@@ -67,6 +55,6 @@
     <xacro:box_link name="${KneePitchLinkName}"
                     width="${LJ4_Link_Box_Width}" height="${LJ4_Link_Box_Height}" depth="${LJ4_Link_Box_Length}" mass="${KneePitchLinkMass}"
+                    origin_xyz="${KneePitchLinkComPosition}"
                     origin_rpy="0 0 0"
-                    origin_xyz="${LJ4_Link_Box_Origin_X} ${LJ4_Link_Box_Origin_Y} ${reflect * LJ4_Link_Box_Origin_Z}"
                     visual_mesh="${mesh_root}/lj4_${prefix}.stl"
                     material="White"
@@ -74,6 +62,6 @@
     <xacro:box_link name="${AnklePitchLinkName}"
                     width="${LJ5_Link_Width}" height="${LJ5_Link_Height}" depth="${LJ5_Link_Length}" mass="${AnklePitchLinkMass}"
+                    origin_xyz="${AnklePitchLinkComPosition}"
                     origin_rpy="0 0 0"
-                    origin_xyz="${LJ5_Link_Box_Origin_X} ${LJ5_Link_Box_Origin_Y} ${LJ5_Link_Box_Origin_Z}"
                     visual_mesh="${mesh_root}/lj5.stl"
                     material="White"
@@ -81,6 +69,6 @@
     <xacro:box_link name="${AnkleRollLinkName}"
                     width="${LJ6_Link_Width}" height="${LJ6_Link_Height}" depth="${LJ6_Link_Length}" mass="${FootMass}"
+                    origin_xyz="${FootComPosition}"
                     origin_rpy="0 0 0"
-                    origin_xyz="${LJ6_Link_Box_Origin_X} ${LJ6_Link_Box_Origin_Y} ${reflect * LJ6_Link_Box_Origin_Z}"
                     visual_mesh="${mesh_root}/foot_${prefix}.stl"
                     material="White"

File: valkyrie_description/robots/valkyrie_A/xacro/leg/mass_parameters.xacro (robot description, xacro)
@@ -2,8 +2,14 @@
 <robot xmlns:xacro="http://www.ros.org/wiki/xacro" name="v1/leg/mass_parameters">
   <xacro:property name="HipYawLinkMass" value="2.39" />
+  <xacro:property name="HipYawLinkComPosition" value="0.02176 ${reflect}*-0.00131 0.03867" />
   <xacro:property name="HipRollLinkMass" value="5.95" />
+  <xacro:property name="HipRollLinkComPosition" value="-0.00185 ${reflect}*0.02426 -0.019260" />
   <xacro:property name="HipPitchLinkMass" value="10.3" />
+  <xacro:property name="HipPitchLinkComPosition" value="0.000057 ${reflect}*0.050000 -0.220000" />
   <xacro:property name="KneePitchLinkMass" value="7.4" />
+  <xacro:property name="KneePitchLinkComPosition" value="-0.004670 ${reflect}*0.045000 -0.184940" />
   <xacro:property name="AnklePitchLinkMass" value="0.395" />
+  <xacro:property name="AnklePitchLinkComPosition" value="-0.001270 ${reflect}*0.000000 -0.006010" />
   <xacro:property name="FootMass" value="1.888" />
+  <xacro:property name="FootComPosition" value="0.068860 ${reflect}*-0.000285 -0.051830" />
 </robot>
