Commit message: Zero'd out a few of the orientation parameters for the pinky finger.

File: valkyrie_description/robots/valkyrie_A/xacro/little_finger/dh_parameters.xacro (robot description, xacro)
@@ -1,43 +1,27 @@
 <?xml version="1.0" ?>
 <robot xmlns:xacro="http://www.ros.org/wiki/xacro" name="v1/little_finger/dh_parameters">
-  <xacro:property name="LFJ1_Joint_Offset" value="$​{reflect * -0.007747}" />
-  <xacro:property name="LFJ1_Joint_Angle" value="0.690626785" />
-  <xacro:property name="LFJ1_Joint_Radius" value="0.055403" />
-  <xacro:property name="LFJ1_Joint_Twist" value="${reflect * -1 * 1.57}" />
  <xacro:property name="LFJ1_Origin_X" value="0.0427072303336"/>
   <xacro:property name="LFJ1_Origin_Y" value="0.0352928446888"/>
   <xacro:property name="LFJ1_Origin_Z" value="${reflect * -0.007747}"/>
-  <xacro:property name="LFJ1_Orientation_Roll" value="${reflect * -1 * 1.57}"/>
-  <xacro:property name="LFJ1_Orientation_Pitch" value="0"/>
-  <xacro:property name="LFJ1_Orientation_Yaw" value="0.690626785"/>
-  <xacro:property name="LFJ2_Joint_Offset" value="${reflect * -0.071327}" />
-  <xacro:property name="LFJ2_Joint_Angle" value="${reflect * -1 * 1.57}" />
-  <xacro:property name="LFJ2_Joint_Radius" value="{reflect * 0.010287}" />
-  <xacro:property name="LFJ2_Joint_Twist" value="-0.690626785" />
+  <xacro:property name="LFJ1_Orientation_Roll" value="0.0"/>
+  <xacro:property name="LFJ1_Orientation_Pitch" value="0.0"/>
+  <xacro:property name="LFJ1_Orientation_Yaw" value="0.0"/>
   <xacro:property name="LFJ2_Origin_X" value="0"/>
   <xacro:property name="LFJ2_Origin_Y" value="-0.010287"/>
   <xacro:property name="LFJ2_Origin_Z" value="${reflect * -0.071327}"/>
-  <xacro:property name="LFJ2_Orientation_Roll" value="-0.690626785"/>
-  <xacro:property name="LFJ2_Orientation_Pitch" value="0"/>
-  <xacro:property name="LFJ2_Orientation_Yaw" value="${reflect * -1 * 1.57}"/>
-  <xacro:property name="LFJ3_Joint_Offset" value="${reflect * 0.050169}" />
-  <xacro:property name="LFJ3_Joint_Angle" value="${reflect * 1.57}" />
-  <xacro:property name="LFJ3_Joint_Radius" value="0.0381" />
-  <xacro:property name="LFJ3_Joint_Twist" value="0" />
-  <xacro:property name="LFJ3_Origin_X" value="0"/>
-  <xacro:property name="LFJ3_Origin_Y" value="${reflect * 0.0381}"/>
-  <xacro:property name="LFJ3_Origin_Z" value="${reflect * 0.050169}"/>
-  <xacro:property name="LFJ3_Orientation_Roll" value="0"/>
-  <xacro:property name="LFJ3_Orientation_Pitch" value="0"/>
-  <xacro:property name="LFJ3_Orientation_Yaw" value="${reflect * 1.57}"/>
-  <xacro:property name="LFJ4_Joint_Offset" value="0" />
-  <xacro:property name="LFJ4_Joint_Angle" value="0" />
-  <xacro:property name="LFJ4_Joint_Radius" value="0.02286" />
-  <xacro:property name="LFJ4_Joint_Twist" value="0" />
+  <xacro:property name="LFJ2_Orientation_Roll" value="0.0"/>
+  <xacro:property name="LFJ2_Orientation_Pitch" value="0.0"/>
+  <xacro:property name="LFJ2_Orientation_Yaw" value="0.0"/>
+  <xacro:property name="LFJ3_Origin_X" value="0.0"/>
+  <xacro:property name="LFJ3_Origin_Y" value="0.0"/>
+  <xacro:property name="LFJ3_Origin_Z" value="0.0"/>
+  <xacro:property name="LFJ3_Orientation_Roll" value="0.0"/>
+  <xacro:property name="LFJ3_Orientation_Pitch" value="0.0"/>
+  <xacro:property name="LFJ3_Orientation_Yaw" value="0.0"/>
   <xacro:property name="LFJ4_Origin_X" value="0.02286"/>
   <xacro:property name="LFJ4_Origin_Y" value="0"/>
   <xacro:property name="LFJ4_Origin_Z" value="0"/>
-  <xacro:property name="LFJ4_Orientation_Roll" value="0"/>
-  <xacro:property name="LFJ4_Orientation_Pitch" value="0"/>
-  <xacro:property name="LFJ4_Orientation_Yaw" value="0"/>
+  <xacro:property name="LFJ4_Orientation_Roll" value="0.0"/>
+  <xacro:property name="LFJ4_Orientation_Pitch" value="0.0"/>
+  <xacro:property name="LFJ4_Orientation_Yaw" value="0.0"/>
 </robot>

Commit message: Changed xacro property names for pinky finger frame parameters.

File: valkyrie_description/robots/valkyrie_A/xacro/little_finger/dh_parameters.xacro (robot description, xacro)
@@ -1,27 +1,27 @@
 <?xml version="1.0" ?>
 <robot xmlns:xacro="http://www.ros.org/wiki/xacro" name="v1/little_finger/dh_parameters">
- <xacro:property name="LFJ1_Origin_X" value="0.0427072303336"/>
-  <xacro:property name="LFJ1_Origin_Y" value="0.0352928446888"/>
-  <xacro:property name="LFJ1_Origin_Z" value="${reflect * -0.007747}"/>
-  <xacro:property name="LFJ1_Orientation_Roll" value="0.0"/>
-  <xacro:property name="LFJ1_Orientation_Pitch" value="0.0"/>
-  <xacro:property name="LFJ1_Orientation_Yaw" value="0.0"/>
-  <xacro:property name="LFJ2_Origin_X" value="0"/>
-  <xacro:property name="LFJ2_Origin_Y" value="-0.010287"/>
-  <xacro:property name="LFJ2_Origin_Z" value="${reflect * -0.071327}"/>
-  <xacro:property name="LFJ2_Orientation_Roll" value="0.0"/>
-  <xacro:property name="LFJ2_Orientation_Pitch" value="0.0"/>
-  <xacro:property name="LFJ2_Orientation_Yaw" value="0.0"/>
-  <xacro:property name="LFJ3_Origin_X" value="0.0"/>
-  <xacro:property name="LFJ3_Origin_Y" value="0.0"/>
-  <xacro:property name="LFJ3_Origin_Z" value="0.0"/>
-  <xacro:property name="LFJ3_Orientation_Roll" value="0.0"/>
-  <xacro:property name="LFJ3_Orientation_Pitch" value="0.0"/>
-  <xacro:property name="LFJ3_Orientation_Yaw" value="0.0"/>
-  <xacro:property name="LFJ4_Origin_X" value="0.02286"/>
-  <xacro:property name="LFJ4_Origin_Y" value="0"/>
-  <xacro:property name="LFJ4_Origin_Z" value="0"/>
-  <xacro:property name="LFJ4_Orientation_Roll" value="0.0"/>
-  <xacro:property name="LFJ4_Orientation_Pitch" value="0.0"/>
-  <xacro:property name="LFJ4_Orientation_Yaw" value="0.0"/>
+ <xacro:property name="PinkyPitch1FrameOrigin_X" value="0.0427072303336"/>
+  <xacro:property name="PinkyPitch1FrameOrigin_Y" value="0.0352928446888"/>
+  <xacro:property name="PinkyPitch1FrameOrigin_Z" value="${reflect * -0.007747}"/>
+  <xacro:property name="PinkyPitch1FrameOrientation_Roll" value="0.0"/>
+  <xacro:property name="PinkyPitch1FrameOrientation_Pitch" value="0.0"/>
+  <xacro:property name="PinkyPitch1FrameOrientation_Yaw" value="0.0"/>
+  <xacro:property name="PinkyPitch2FrameOrigin_X" value="0"/>
+  <xacro:property name="PinkyPitch2FrameOrigin_Y" value="-0.010287"/>
+  <xacro:property name="PinkyPitch2FrameOrigin_Z" value="${reflect * -0.071327}"/>
+  <xacro:property name="PinkyPitch2FrameOrientation_Roll" value="0.0"/>
+  <xacro:property name="PinkyPitch2FrameOrientation_Pitch" value="0.0"/>
+  <xacro:property name="PinkyPitch2FrameOrientation_Yaw" value="0.0"/>
+  <xacro:property name="PinkyPitch3FrameOrigin_X" value="0.0"/>
+  <xacro:property name="PinkyPitch3FrameOrigin_Y" value="0.0"/>
+  <xacro:property name="PinkyPitch3FrameOrigin_Z" value="0.0"/>
+  <xacro:property name="PinkyPitch3FrameOrientation_Roll" value="0.0"/>
+  <xacro:property name="PinkyPitch3FrameOrientation_Pitch" value="0.0"/>
+  <xacro:property name="PinkyPitch3FrameOrientation_Yaw" value="0.0"/>
+  <xacro:property name="PinkyPitch4FrameOrigin_X" value="0.02286"/>
+  <xacro:property name="PinkyPitch4FrameOrigin_Y" value="0"/>
+  <xacro:property name="PinkyPitch4FrameOrigin_Z" value="0"/>
+  <xacro:property name="PinkyPitch4FrameOrientation_Roll" value="0.0"/>
+  <xacro:property name="PinkyPitch4FrameOrientation_Pitch" value="0.0"/>
+  <xacro:property name="PinkyPitch4FrameOrientation_Yaw" value="0.0"/>
 </robot>

File: valkyrie_description/robots/valkyrie_A/xacro/little_finger/little_finger.xacro (robot description, xacro)
@@ -58,6 +58,6 @@
     <xacro:revolute_joint jointName="${LFJ1_Joint_Name}"
                           parent="${LFJ1_Proximal_Link}" child="${LFJ1_Distal_Link}"
-                          origin_xyz="${LFJ1_Origin_X} ${LFJ1_Origin_Y} ${LFJ1_Origin_Z}"
-                          origin_rpy="${LFJ1_Orientation_Roll} ${LFJ1_Orientation_Pitch} ${LFJ1_Orientation_Yaw}">
+                          origin_xyz="${PinkyPitch1FrameOrigin_X} ${PinkyPitch1FrameOrigin_Y} ${PinkyPitch1FrameOrigin_Z}"
+                          origin_rpy="${PinkyPitch1FrameOrientation_Roll} ${PinkyPitch1FrameOrientation_Pitch} ${PinkyPitch1FrameOrientation_Yaw}">
         <limit effort="${LFJ1_Torque_Limit}" lower="${LFJ1_Lower_Limit}" upper="${LFJ1_Upper_Limit}" velocity="${LFJ1_Speed_Limit}"/>
     </xacro:revolute_joint>
@@ -65,6 +65,6 @@
     <xacro:revolute_joint jointName="${LFJ2_Joint_Name}"
                           parent="${LFJ2_Proximal_Link}" child="${LFJ2_Distal_Link}"
-                          origin_xyz="${LFJ2_Origin_X} ${LFJ2_Origin_Y} ${LFJ2_Origin_Z}"
-                          origin_rpy="${LFJ2_Orientation_Roll} ${LFJ2_Orientation_Pitch} ${LFJ2_Orientation_Yaw}">
+                          origin_xyz="${PinkyPitch2FrameOrigin_X} ${PinkyPitch2FrameOrigin_Y} ${PinkyPitch2FrameOrigin_Z}"
+                          origin_rpy="${PinkyPitch2FrameOrientation_Roll} ${PinkyPitch2FrameOrientation_Pitch} ${PinkyPitch2FrameOrientation_Yaw}">
         <limit effort="${LFJ2_Torque_Limit}" lower="${LFJ2_Lower_Limit}" upper="${LFJ2_Upper_Limit}" velocity="${LFJ2_Speed_Limit}"/>
     </xacro:revolute_joint>
@@ -72,6 +72,6 @@
     <xacro:revolute_joint jointName="${LFJ3_Joint_Name}"
                           parent="${LFJ3_Proximal_Link}" child="${LFJ3_Distal_Link}"
-                          origin_xyz="${LFJ3_Origin_X} ${LFJ3_Origin_Y} ${LFJ3_Origin_Z}"
-                          origin_rpy="${LFJ3_Orientation_Roll} ${LFJ3_Orientation_Pitch} ${LFJ3_Orientation_Yaw}">
+                          origin_xyz="${PinkyPitch3FrameOrigin_X} ${PinkyPitch3FrameOrigin_Y} ${PinkyPitch3FrameOrigin_Z}"
+                          origin_rpy="${PinkyPitch3FrameOrientation_Roll} ${PinkyPitch3FrameOrientation_Pitch} ${PinkyPitch3FrameOrientation_Yaw}">
         <limit effort="${LFJ3_Torque_Limit}" lower="${LFJ3_Lower_Limit}" upper="${LFJ3_Upper_Limit}" velocity="${LFJ3_Speed_Limit}"/>
     </xacro:revolute_joint>
@@ -103,16 +103,16 @@
     <xacro:fixed_joint jointName="${LFJ1_Joint_Name}"
                        parent="${LFJ1_Proximal_Link}" child="${LFJ1_Distal_Link}"
-                       origin_xyz="${LFJ1_Origin_X} ${LFJ1_Origin_Y} ${LFJ1_Origin_Z}"
-                       origin_rpy="${LFJ1_Orientation_Roll} ${LFJ1_Orientation_Pitch} ${LFJ1_Orientation_Yaw}"/>
+                       origin_xyz="${PinkyPitch1FrameOrigin_X} ${PinkyPitch1FrameOrigin_Y} ${PinkyPitch1FrameOrigin_Z}"
+                       origin_rpy="${PinkyPitch1FrameOrientation_Roll} ${PinkyPitch1FrameOrientation_Pitch} ${PinkyPitch1FrameOrientation_Yaw}"/>
     <!-- LFJ2 -->
     <xacro:fixed_joint jointName="${LFJ2_Joint_Name}"
                           parent="${LFJ2_Proximal_Link}" child="${LFJ2_Distal_Link}"
-                          origin_xyz="${LFJ2_Origin_X} ${LFJ2_Origin_Y} ${LFJ2_Origin_Z}"
-                          origin_rpy="${LFJ2_Orientation_Roll} ${LFJ2_Orientation_Pitch} ${LFJ2_Orientation_Yaw}"/>
+                          origin_xyz="${PinkyPitch2FrameOrigin_X} ${PinkyPitch2FrameOrigin_Y} ${PinkyPitch2FrameOrigin_Z}"
+                          origin_rpy="${PinkyPitch2FrameOrientation_Roll} ${PinkyPitch2FrameOrientation_Pitch} ${PinkyPitch2FrameOrientation_Yaw}"/>
     <!-- LFJ3 -->
     <xacro:fixed_joint jointName="${LFJ3_Joint_Name}"
                           parent="${LFJ3_Proximal_Link}" child="${LFJ3_Distal_Link}"
-                          origin_xyz="${LFJ3_Origin_X} ${LFJ3_Origin_Y} ${LFJ3_Origin_Z}"
-                          origin_rpy="${LFJ3_Orientation_Roll} ${LFJ3_Orientation_Pitch} ${LFJ3_Orientation_Yaw}"/>
+                          origin_xyz="${PinkyPitch3FrameOrigin_X} ${PinkyPitch3FrameOrigin_Y} ${PinkyPitch3FrameOrigin_Z}"
+                          origin_rpy="${PinkyPitch3FrameOrientation_Roll} ${PinkyPitch3FrameOrientation_Pitch} ${PinkyPitch3FrameOrientation_Yaw}"/>
   </xacro:macro>
   <!-- Actuators -->
