Commit message: Updated frame parameters  for pinky finger.

File: valkyrie_description/robots/valkyrie_A/xacro/little_finger/frame_parameters.xacro (robot description, xacro)
@@ -1,27 +1,21 @@
 <?xml version="1.0" ?>
 <robot xmlns:xacro="http://www.ros.org/wiki/xacro" name="v1/little_finger/dh_parameters">
- <xacro:property name="PinkyPitch1FrameOrigin_X" value="0.0427072303336"/>
-  <xacro:property name="PinkyPitch1FrameOrigin_Y" value="0.0352928446888"/>
-  <xacro:property name="PinkyPitch1FrameOrigin_Z" value="${reflect * -0.007747}"/>
-  <xacro:property name="PinkyPitch1FrameOrientation_Roll" value="0.0"/>
+ <xacro:property name="PinkyPitch1FrameOrigin_X" value="0.0022"/>
+  <xacro:property name="PinkyPitch1FrameOrigin_Y" value="${reflect * 0.0838}"/>
+  <xacro:property name="PinkyPitch1FrameOrigin_Z" value="-0.041"/>
+  <xacro:property name="PinkyPitch1FrameOrientation_Roll" value="${reflect * -0.1222}"/>
   <xacro:property name="PinkyPitch1FrameOrientation_Pitch" value="0.0"/>
   <xacro:property name="PinkyPitch1FrameOrientation_Yaw" value="0.0"/>
-  <xacro:property name="PinkyPitch2FrameOrigin_X" value="0"/>
-  <xacro:property name="PinkyPitch2FrameOrigin_Y" value="-0.010287"/>
-  <xacro:property name="PinkyPitch2FrameOrigin_Z" value="${reflect * -0.071327}"/>
+  <xacro:property name="PinkyPitch2FrameOrigin_X" value="0.0"/>
+  <xacro:property name="PinkyPitch2FrameOrigin_Y" value="${reflect * 0.0381}"/>
+  <xacro:property name="PinkyPitch2FrameOrigin_Z" value="0.0"/>
   <xacro:property name="PinkyPitch2FrameOrientation_Roll" value="0.0"/>
   <xacro:property name="PinkyPitch2FrameOrientation_Pitch" value="0.0"/>
   <xacro:property name="PinkyPitch2FrameOrientation_Yaw" value="0.0"/>
   <xacro:property name="PinkyPitch3FrameOrigin_X" value="0.0"/>
-  <xacro:property name="PinkyPitch3FrameOrigin_Y" value="0.0"/>
+  <xacro:property name="PinkyPitch3FrameOrigin_Y" value="${reflect * 0.0229}"/>
   <xacro:property name="PinkyPitch3FrameOrigin_Z" value="0.0"/>
   <xacro:property name="PinkyPitch3FrameOrientation_Roll" value="0.0"/>
   <xacro:property name="PinkyPitch3FrameOrientation_Pitch" value="0.0"/>
   <xacro:property name="PinkyPitch3FrameOrientation_Yaw" value="0.0"/>
-  <xacro:property name="PinkyPitch4FrameOrigin_X" value="0.02286"/>
-  <xacro:property name="PinkyPitch4FrameOrigin_Y" value="0"/>
-  <xacro:property name="PinkyPitch4FrameOrigin_Z" value="0"/>
-  <xacro:property name="PinkyPitch4FrameOrientation_Roll" value="0.0"/>
-  <xacro:property name="PinkyPitch4FrameOrientation_Pitch" value="0.0"/>
-  <xacro:property name="PinkyPitch4FrameOrientation_Yaw" value="0.0"/>
 </robot>

File: valkyrie_description/robots/valkyrie_A/xacro/little_finger/little_finger.xacro (robot description, xacro)
@@ -26,5 +26,4 @@
   <xacro:property name="LFJ3_Link_Origin_Z" value="0"/>
   <xacro:macro name="make_little_finger" params="prefix reflect little_finger_root_link">
-    <!-- LINKS -->
     <xacro:box_link name="${PinkyPitch1LinkName}"
                     width="${LFJ1_Link_Width}" height="${LFJ1_Link_Height}" depth="${LFJ1_Link_Length}" mass="${PinkyPitch1LinkMass}"
@@ -48,12 +47,4 @@
                     material="Gold"
                     collision_mesh="${mesh_root}/sf2_ssf3.stl"/>
-    <xacro:box_link name="${PinkyPitch4LinkName}"
-                    width="${LFJ4_Link_Width}" height="${LFJ4_Link_Height}" depth="${LFJ4_Link_Length}" mass="${PinkyPitch4LinkMass}"
-                    origin_rpy="0 0 0"
-                    origin_xyz="${LFJ4_Link_Origin_X} ${LFJ4_Link_Origin_Y} ${LFJ4_Link_Origin_Z}"
-                    visual_mesh="${mesh_root}/sf3_ssf4.stl"
-                    material="Gold"
-                    collision_mesh="${mesh_root}/sf3_ssf4.stl"/>
-    <!-- LFJ1 -->
     <xacro:revolute_joint jointName="${PinkyPitch1JointName}"
                           parent="${PinkyPitch1ParentLinkName}" child="${PinkyPitch1LinkName}"
@@ -62,5 +53,4 @@
         <limit effort="${PinkyPitch1TorqueLimit}" lower="${PinkyPitch1PositionLimit_Lower}" upper="${PinkyPitch1PositionLimit_Upper}" velocity="${PinkyPitch1VelocityLimit}"/>
     </xacro:revolute_joint>
-    <!-- LFJ2 -->
     <xacro:revolute_joint jointName="${PinkyPitch2JointName}"
                           parent="${PinkyPitch1LinkName}" child="${PinkyPitch2LinkName}"
@@ -69,5 +59,4 @@
         <limit effort="${PinkyPitch2TorqueLimit}" lower="${PinkyPitch2PositionLimit_Lower}" upper="${PinkyPitch2PositionLimit_Upper}" velocity="${PinkyPitch2VelocityLimit}"/>
     </xacro:revolute_joint>
-    <!-- LFJ3 -->
     <xacro:revolute_joint jointName="${PinkyPitch3JointName}"
                           parent="${PinkyPitch2LinkName}" child="${PinkyPitch3LinkName}"
@@ -78,5 +67,4 @@
   </xacro:macro>
   <xacro:macro name="make_little_finger_fixed" params="prefix reflect little_finger_root_link">
-    <!-- LINKS -->
     <xacro:box_link name="${PinkyPitch1LinkName}"
                     width="${LFJ1_Link_Width}" height="${LFJ1_Link_Height}" depth="${LFJ1_Link_Length}" mass="${PinkyPitch1LinkMass}"
@@ -100,15 +88,12 @@
                     material="Gold"
                     collision_mesh="${mesh_root}/sf2_ssf3.stl"/>
-    <!-- LFJ1 -->
     <xacro:fixed_joint jointName="${PinkyPitch1JointName}"
                        parent="${PinkyPitch1ParentLinkName}" child="${PinkyPitch1LinkName}"
                        origin_xyz="${PinkyPitch1FrameOrigin_X} ${PinkyPitch1FrameOrigin_Y} ${PinkyPitch1FrameOrigin_Z}"
                        origin_rpy="${PinkyPitch1FrameOrientation_Roll} ${PinkyPitch1FrameOrientation_Pitch} ${PinkyPitch1FrameOrientation_Yaw}"/>
-    <!-- LFJ2 -->
     <xacro:fixed_joint jointName="${PinkyPitch2JointName}"
                           parent="${PinkyPitch1LinkName}" child="${PinkyPitch2LinkName}"
                           origin_xyz="${PinkyPitch2FrameOrigin_X} ${PinkyPitch2FrameOrigin_Y} ${PinkyPitch2FrameOrigin_Z}"
                           origin_rpy="${PinkyPitch2FrameOrientation_Roll} ${PinkyPitch2FrameOrientation_Pitch} ${PinkyPitch2FrameOrientation_Yaw}"/>
-    <!-- LFJ3 -->
     <xacro:fixed_joint jointName="${PinkyPitch3JointName}"
                           parent="${PinkyPitch2LinkName}" child="${PinkyPitch3LinkName}"
