Commit message: Renamed mass params of middle finger.

File: valkyrie_description/robots/valkyrie_A/xacro/middle_finger/mass_parameters.xacro (robot description, xacro)
@@ -1,6 +1,6 @@
 <?xml version="1.0" ?>
 <robot xmlns:xacro="http://www.ros.org/wiki/xacro" name="v1/middle_finger/mass_parameters">
-  <xacro:property name="MFJ1_Link_Mass" value="0.02" />
-  <xacro:property name="MFJ2_Link_Mass" value="0.011" />
-  <xacro:property name="MFJ3_Link_Mass" value="0.006" />
+  <xacro:property name="MiddleFingerPitch1LinkMass" value="0.02" />
+  <xacro:property name="MiddleFingerPitch2LinkMass" value="0.011" />
+  <xacro:property name="MiddleFingerPitch3LinkMass" value="0.006" />
 </robot>

File: valkyrie_description/robots/valkyrie_A/xacro/middle_finger/middle_finger.xacro (robot description, xacro)
@@ -29,5 +29,5 @@
     <!-- LINKS -->
     <xacro:box_link name="${MiddleFingerPitch1LinkName}"
-                    width="${MFJ1_Link_Width}" height="${MFJ1_Link_Height}" depth="${MFJ1_Link_Length}" mass="${MFJ1_Link_Mass}"
+                    width="${MFJ1_Link_Width}" height="${MFJ1_Link_Height}" depth="${MFJ1_Link_Length}" mass="${MiddleFingerPitch1LinkMass}"
                     origin_rpy="0 0 0"
                     origin_xyz="${MFJ1_Link_Origin_X} ${MFJ1_Link_Origin_Y} ${MFJ1_Link_Origin_Z}"
@@ -36,5 +36,5 @@
                     collision_mesh="${mesh_root}/sf1.stl"/>
     <xacro:box_link name="${MiddleFingerPitch2LinkName}"
-                    width="${MFJ2_Link_Width}" height="${MFJ2_Link_Height}" depth="${MFJ2_Link_Length}" mass="${MFJ2_Link_Mass}"
+                    width="${MFJ2_Link_Width}" height="${MFJ2_Link_Height}" depth="${MFJ2_Link_Length}" mass="${MiddleFingerPitch2LinkMass}"
                     origin_rpy="0 0 0"
                     origin_xyz="${MFJ2_Link_Origin_X} ${MFJ2_Link_Origin_Y} ${MFJ2_Link_Origin_Z}"
@@ -43,5 +43,5 @@
                     collision_mesh="${mesh_root}/sf2_ssf3.stl"/>
     <xacro:box_link name="${MiddleFingerPitch3LinkName}"
-                    width="${MFJ3_Link_Width}" height="${MFJ3_Link_Height}" depth="${MFJ3_Link_Length}" mass="${MFJ3_Link_Mass}"
+                    width="${MFJ3_Link_Width}" height="${MFJ3_Link_Height}" depth="${MFJ3_Link_Length}" mass="${MiddleFingerPitch3LinkMass}"
                     origin_rpy="0 0 0"
                     origin_xyz="${MFJ3_Link_Origin_X} ${MFJ3_Link_Origin_Y} ${MFJ3_Link_Origin_Z}"
@@ -74,5 +74,5 @@
     <!-- LINKS -->
     <xacro:box_link name="${MiddleFingerPitch1LinkName}"
-                    width="${MFJ1_Link_Width}" height="${MFJ1_Link_Height}" depth="${MFJ1_Link_Length}" mass="${MFJ1_Link_Mass}"
+                    width="${MFJ1_Link_Width}" height="${MFJ1_Link_Height}" depth="${MFJ1_Link_Length}" mass="${MiddleFingerPitch1LinkMass}"
                     origin_rpy="0 0 0"
                     origin_xyz="${MFJ1_Link_Origin_X} ${MFJ1_Link_Origin_Y} ${MFJ1_Link_Origin_Z}"
@@ -81,5 +81,5 @@
                     collision_mesh="${mesh_root}/sf1.stl"/>
     <xacro:box_link name="${MiddleFingerPitch2LinkName}"
-                    width="${MFJ2_Link_Width}" height="${MFJ2_Link_Height}" depth="${MFJ2_Link_Length}" mass="${MFJ2_Link_Mass}"
+                    width="${MFJ2_Link_Width}" height="${MFJ2_Link_Height}" depth="${MFJ2_Link_Length}" mass="${MiddleFingerPitch2LinkMass}"
                     origin_rpy="0 0 0"
                     origin_xyz="${MFJ2_Link_Origin_X} ${MFJ2_Link_Origin_Y} ${MFJ2_Link_Origin_Z}"
@@ -88,5 +88,5 @@
                     collision_mesh="${mesh_root}/sf2_ssf3.stl"/>
     <xacro:box_link name="${MiddleFingerPitch3LinkName}"
-                    width="${MFJ3_Link_Width}" height="${MFJ3_Link_Height}" depth="${MFJ3_Link_Length}" mass="${MFJ3_Link_Mass}"
+                    width="${MFJ3_Link_Width}" height="${MFJ3_Link_Height}" depth="${MFJ3_Link_Length}" mass="${MiddleFingerPitch3LinkMass}"
                     origin_rpy="0 0 0"
                     origin_xyz="${MFJ3_Link_Origin_X} ${MFJ3_Link_Origin_Y} ${MFJ3_Link_Origin_Z}"
