Commit message: Updated thumb index and middle finger frame parameters.

File: valkyrie_description/robots/valkyrie_A/xacro/index_finger/frame_parameters.xacro (robot description, xacro)
@@ -1,27 +1,21 @@
 <?xml version="1.0" ?>
 <robot xmlns:xacro="http://www.ros.org/wiki/xacro" name="v1/index_finger/dh_parameters">
-  <xacro:property name="IndexFingerPitch1FrameOrigin_X" value="0.0776738914821"/>
-  <xacro:property name="IndexFingerPitch1FrameOrigin_Y" value="-0.0298162134085"/>
-  <xacro:property name="IndexFingerPitch1FrameOrigin_Z" value="${reflect * 0.00254}"/>
-  <xacro:property name="IndexFingerPitch1FrameOrientation_Roll" value="0.0"/>
+  <xacro:property name="IndexFingerPitch1FrameOrigin_X" value="0.0022"/>
+  <xacro:property name="IndexFingerPitch1FrameOrigin_Y" value="${reflect * 0.0976}"/>
+  <xacro:property name="IndexFingerPitch1FrameOrigin_Z" value="0.0235"/>
+  <xacro:property name="IndexFingerPitch1FrameOrientation_Roll" value="${reflect * 0.1745}"/>
   <xacro:property name="IndexFingerPitch1FrameOrientation_Pitch" value="0.0"/>
   <xacro:property name="IndexFingerPitch1FrameOrientation_Yaw" value="0.0"/>
-  <xacro:property name="IndexFingerPitch2FrameOrigin_X" value="0.0169724899301"/>
-  <xacro:property name="IndexFingerPitch2FrameOrigin_Y" value="0.000966739661347"/>
-  <xacro:property name="IndexFingerPitch2FrameOrigin_Z" value="0"/>
+  <xacro:property name="IndexFingerPitch2FrameOrigin_X" value="0.0"/>
+  <xacro:property name="IndexFingerPitch2FrameOrigin_Y" value="${reflect * 0.0381}"/>
+  <xacro:property name="IndexFingerPitch2FrameOrigin_Z" value="0.0"/>
   <xacro:property name="IndexFingerPitch2FrameOrientation_Roll" value="0.0"/>
   <xacro:property name="IndexFingerPitch2FrameOrientation_Pitch" value="0.0"/>
   <xacro:property name="IndexFingerPitch2FrameOrientation_Yaw" value="0.0"/>
-  <xacro:property name="IndexFingerPitch3FrameOrigin_X" value="0.0381"/>
-  <xacro:property name="IndexFingerPitch3FrameOrigin_Y" value="0"/>
+  <xacro:property name="IndexFingerPitch3FrameOrigin_X" value="0.0"/>
+  <xacro:property name="IndexFingerPitch3FrameOrigin_Y" value="${reflect * 0.0229}"/>
   <xacro:property name="IndexFingerPitch3FrameOrigin_Z" value="0"/>
   <xacro:property name="IndexFingerPitch3FrameOrientation_Roll" value="0.0"/>
   <xacro:property name="IndexFingerPitch3FrameOrientation_Pitch" value="0.0"/>
   <xacro:property name="IndexFingerPitch3FrameOrientation_Yaw" value="0.0"/>
-  <xacro:property name="IndexFingerPitch4FrameOrigin_X" value="0.02286"/>
-  <xacro:property name="IndexFingerPitch4FrameOrigin_Y" value="0"/>
-  <xacro:property name="IndexFingerPitch4FrameOrigin_Z" value="0"/>
-  <xacro:property name="IndexFingerPitch4FrameOrientation_Roll" value="0.0"/>
-  <xacro:property name="IndexFingerPitch4FrameOrientation_Pitch" value="0.0"/>
-  <xacro:property name="IndexFingerPitch4FrameOrientation_Yaw" value="0.0"/>
 </robot>

File: valkyrie_description/robots/valkyrie_A/xacro/index_finger/index_finger.xacro (robot description, xacro)
@@ -25,10 +25,4 @@
   <xacro:property name="PFJ3_Link_Origin_Y" value="-0.0003"/>
   <xacro:property name="PFJ3_Link_Origin_Z" value="0"/>
-  <xacro:property name="PFJ4_Link_Width" value="0.027"/>
-  <xacro:property name="PFJ4_Link_Height" value="0.012"/>
-  <xacro:property name="PFJ4_Link_Length" value="0.015"/>
-  <xacro:property name="PFJ4_Link_Origin_X" value="0.00857"/>
-  <xacro:property name="PFJ4_Link_Origin_Y" value="-0.000696"/>
-  <xacro:property name="PFJ4_Link_Origin_Z" value="0"/>
   <xacro:macro name="make_index_finger" params="prefix reflect index_finger_root_link">
     <xacro:box_link name="${IndexFingerPitch1LinkName}"
@@ -53,11 +47,4 @@
                     material="Gold"
                     collision_mesh="${mesh_root}/pf3.stl"/>
-    <xacro:box_link name="${IndexFingerPitch4LinkName}"
-                    width="${PFJ4_Link_Width}" height="${PFJ4_Link_Height}" depth="${PFJ4_Link_Length}" mass="${IndexFingerPitch4LinkMass}"
-                    origin_rpy="0 0 0"
-                    origin_xyz="${PFJ4_Link_Origin_X} ${PFJ4_Link_Origin_Y} ${PFJ4_Link_Origin_Z}"
-                    visual_mesh="${mesh_root}/pf4.stl"
-                    material="Gold"
-                    collision_mesh="${mesh_root}/pf4.stl"/>
     <xacro:revolute_joint jointName="${IndexFingerPitch1JointName}"
                           parent="${IndexFingerPitch1ParentLinkName}" child="${IndexFingerPitch1LinkName}"
@@ -77,10 +64,4 @@
                           origin_rpy="${IndexFingerPitch3FrameOrientation_Roll} ${IndexFingerPitch3FrameOrientation_Pitch} ${IndexFingerPitch3FrameOrientation_Yaw}">
         <limit effort="${IndexFingerPitch3TorqueLimit}" lower="${IndexFingerPitch3PositionLimit_Lower}" upper="${IndexFingerPitch3PositionLimit_Upper}" velocity="${IndexFingerPitch3VelocityLimit}"/>
-    </xacro:revolute_joint>
-    <xacro:revolute_joint jointName="${IndexFingerPitch4JointName}"
-                          parent="${IndexFingerPitch3LinkName}" child="${IndexFingerPitch4LinkName}"
-                          origin_xyz="${IndexFingerPitch4FrameOrigin_X} ${IndexFingerPitch4FrameOrigin_Y} ${IndexFingerPitch4FrameOrigin_Z}"
-                          origin_rpy="${IndexFingerPitch4FrameOrientation_Roll} ${IndexFingerPitch4FrameOrientation_Pitch} ${IndexFingerPitch4FrameOrientation_Yaw}">
-        <limit effort="${IndexFingerPitch4TorqueLimit}" lower="${IndexFingerPitch4PositionLimit_Lower}" upper="${IndexFingerPitch4PositionLimit_Upper}" velocity="${IndexFingerPitch4VelocityLimit}"/>
     </xacro:revolute_joint>
   </xacro:macro>
@@ -107,11 +88,4 @@
                     material="Gold"
                     collision_mesh="${mesh_root}/pf3.stl"/>
-    <xacro:box_link name="${IndexFingerPitch4LinkName}"
-                    width="${PFJ4_Link_Width}" height="${PFJ4_Link_Height}" depth="${PFJ4_Link_Length}" mass="${IndexFingerPitch4LinkMass}"
-                    origin_rpy="0 0 0"
-                    origin_xyz="${PFJ4_Link_Origin_X} ${PFJ4_Link_Origin_Y} ${PFJ4_Link_Origin_Z}"
-                    visual_mesh="${mesh_root}/pf4.stl"
-                    material="Gold"
-                    collision_mesh="${mesh_root}/pf4.stl"/>
     <xacro:fixed_joint jointName="${IndexFingerPitch1JointName}"
                           parent="${IndexFingerPitch1ParentLinkName}" child="${IndexFingerPitch1LinkName}"
@@ -126,8 +100,4 @@
                           origin_xyz="${IndexFingerPitch3FrameOrigin_X} ${IndexFingerPitch3FrameOrigin_Y} ${IndexFingerPitch3FrameOrigin_Z}"
                           origin_rpy="${IndexFingerPitch3FrameOrientation_Roll} ${IndexFingerPitch3FrameOrientation_Pitch} ${IndexFingerPitch3FrameOrientation_Yaw}"/>
-    <xacro:fixed_joint jointName="${IndexFingerPitch4JointName}"
-                          parent="${IndexFingerPitch3LinkName}" child="${IndexFingerPitch4LinkName}"
-                          origin_xyz="${IndexFingerPitch4FrameOrigin_X} ${IndexFingerPitch4FrameOrigin_Y} ${IndexFingerPitch4FrameOrigin_Z}"
-                          origin_rpy="${IndexFingerPitch4FrameOrientation_Roll} ${IndexFingerPitch4FrameOrientation_Pitch} ${IndexFingerPitch4FrameOrientation_Yaw}"/>
   </xacro:macro>
   <xacro:macro name="v1_right_index_finger_actuators" params="prefix api">

File: valkyrie_description/robots/valkyrie_A/xacro/middle_finger/frame_parameters.xacro (robot description, xacro)
@@ -1,19 +1,19 @@
 <?xml version="1.0" ?>
 <robot xmlns:xacro="http://www.ros.org/wiki/xacro" name="v1/middle_finger/dh_parameters">
-  <xacro:property name="MiddleFingerPitch1FrameOrigin_X" value="0.09767"/>
-  <xacro:property name="MiddleFingerPitch1FrameOrigin_Y" value="0"/>
-  <xacro:property name="MiddleFingerPitch1FrameOrigin_Z" value="${reflect * 0.00254}"/>
-  <xacro:property name="MiddleFingerPitch1FrameOrientation_Roll" value="0.0"/>
+  <xacro:property name="MiddleFingerPitch1FrameOrigin_X" value="0.0022"/>
+  <xacro:property name="MiddleFingerPitch1FrameOrigin_Y" value="${reflect * 0.097}"/>
+  <xacro:property name="MiddleFingerPitch1FrameOrigin_Z" value="-0.0119"/>
+  <xacro:property name="MiddleFingerPitch1FrameOrientation_Roll" value="${reflect * -0.1222}"/>
   <xacro:property name="MiddleFingerPitch1FrameOrientation_Pitch" value="0.0"/>
   <xacro:property name="MiddleFingerPitch1FrameOrientation_Yaw" value="0.0"/>
-  <xacro:property name="MiddleFingerPitch2FrameOrigin_X" value="0.0381"/>
-  <xacro:property name="MiddleFingerPitch2FrameOrigin_Y" value="0"/>
-  <xacro:property name="MiddleFingerPitch2FrameOrigin_Z" value="0"/>
+  <xacro:property name="MiddleFingerPitch2FrameOrigin_X" value="0.0"/>
+  <xacro:property name="MiddleFingerPitch2FrameOrigin_Y" value="${reflect * 0.0381}"/>
+  <xacro:property name="MiddleFingerPitch2FrameOrigin_Z" value="0.0"/>
   <xacro:property name="MiddleFingerPitch2FrameOrientation_Roll" value="0.0"/>
   <xacro:property name="MiddleFingerPitch2FrameOrientation_Pitch" value="0.0"/>
   <xacro:property name="MiddleFingerPitch2FrameOrientation_Yaw" value="0.0"/>
-  <xacro:property name="MiddleFingerPitch3FrameOrigin_X" value="0.02286"/>
-  <xacro:property name="MiddleFingerPitch3FrameOrigin_Y" value="0"/>
-  <xacro:property name="MiddleFingerPitch3FrameOrigin_Z" value="0"/>
+  <xacro:property name="MiddleFingerPitch3FrameOrigin_X" value="0.0"/>
+  <xacro:property name="MiddleFingerPitch3FrameOrigin_Y" value="${reflect * 0.0229}"/>
+  <xacro:property name="MiddleFingerPitch3FrameOrigin_Z" value="0.0"/>
   <xacro:property name="MiddleFingerPitch3FrameOrientation_Roll" value="0.0"/>
   <xacro:property name="MiddleFingerPitch3FrameOrientation_Pitch" value="0.0"/>
