Commit message: Fixed orientation of right pelvis IMU frame.

File: valkyrie_description/robots/valkyrie_A/xacro/index_finger/index_finger.xacro (robot description, xacro)
@@ -69,5 +69,5 @@
         <limit effort="${IndexFingerPitch3TorqueLimit}" lower="${IndexFingerPitch3PositionLimit_Lower}" upper="${IndexFingerPitch3PositionLimit_Upper}" velocity="${IndexFingerPitch3VelocityLimit}"/>
     </xacro:revolute_joint>
-  </xacro:macro>]
+  </xacro:macro>
   <xacro:macro name="v1_right_index_finger_actuators" params="prefix api">
     <xacro:v1_actuator name="${RPFA_Actuator_Name}" api="${api}" />

File: valkyrie_description/robots/valkyrie_A/xacro/pelvis/pelvis.xacro (robot description, xacro)
@@ -13,5 +13,5 @@
                                   parentLink="${Pelvis_Link_Name}"
                                   origin_xyz="0.0515 -0.115 -0.042"
-                                  origin_rpy="-1.57 -1.274 0.0" />
+                                  origin_rpy="-1.57 0.0 1.274" />
         <xacro:microstrain_sensor sensorName="LeftPelvisIMU"
                                   parentLink="${Pelvis_Link_Name}"
