Commit message: Fixed joint names of some fingers. Removed comment.

File: valkyrie_description/robots/valkyrie_A/xacro/index_finger/joint_names.xacro (robot description, xacro)
@@ -1,7 +1,6 @@
 <?xml version="1.0" ?>
 <robot xmlns:xacro="http://www.ros.org/wiki/xacro" name="v1/index_finger/mass_parameters">
-  <xacro:property name="IndexFingerPitch1JointName" value="${prefix}PrimaryMPYaw" />
-  <xacro:property name="IndexFingerPitch2JointName" value="${prefix}PrimaryMPExtensor" />
-  <xacro:property name="IndexFingerPitch3JointName" value="${prefix}PrimaryPIPExtensor" />
-  <xacro:property name="IndexFingerPitch4JointName" value="${prefix}PrimaryDIPExtensor" />
+  <xacro:property name="IndexFingerPitch1JointName" value="${prefix}IndexFingerPitch1" />
+  <xacro:property name="IndexFingerPitch2JointName" value="${prefix}IndexFingerPitch2" />
+  <xacro:property name="IndexFingerPitch3JointName" value="${prefix}IndexFingerPitch3" />
 </robot>

File: valkyrie_description/robots/valkyrie_A/xacro/valkyrie_A_sim_base.xacro (robot description, xacro)
@@ -10,5 +10,4 @@
     <!-- <xacro:v1_waist_actuators name1="${waist_name1}" type1="${waist_type1}" name2="${waist_name2}" type2="${waist_type2}" name3="${waist_name3}" type3="${waist_type3}"/> -->
     <xacro:v1_trunk_sensors/>
-    <!-- ===== HEAD ===== -->
     <xacro:make_head head_root_link="${TorsoRollLinkName}" />
     <xacro:v1_head_sensors />
