Commit message: Added a bunch of stl meshes. Looks like the frames are done for the robots joints. I viewed them in rviz and everything looks good.

File: valkyrie_description/robots/valkyrie_A/xacro/V1.xacro (robot description, xacro)
@@ -1,4 +1,4 @@
 <robot xmlns:xacro="http://ros.org/wiki/xacro" name="valkyrie">
-    <xacro:property name="mesh_root" value="package://valkyrie_description/meshes/reduced_polygon_meshes"/>
+    <xacro:property name="mesh_root" value="package://valkyrie_description/meshes"/>
     <!-- <xacro:include filename="$(find valkyrie_description)/robots/valkyrie_A/xacro/common/hw_actuator_types.xacro"/> -->
     <xacro:include filename="$(find valkyrie_description)/robots/valkyrie_A/xacro/V1_sim_base.xacro"/>

File: valkyrie_description/robots/valkyrie_A/xacro/arm/joint_limits.xacro (robot description, xacro)
@@ -16,5 +16,5 @@
   <xacro:property name="WristPitchPositionLimit_Lower" value="-0.524" />
   <xacro:property name="ShoulderPitchPositionLimit_Upper" value="3.14" />
-  <xacro:property name="ShoulderRollPositionLimit_Upper" value="-0.155" />
+  <xacro:property name="ShoulderRollPositionLimit_Upper" value="0.155" />
   <xacro:property name="ShoulderYawPositionLimit_Upper" value="1.7" />
   <xacro:property name="ElbowPitchPositionLimit_Upper" value="0.087" />
