Commit message: I seem to have renamed all joints/links.

File: valkyrie_description/robots/valkyrie_A/xacro/V1_sim_base.xacro (robot description, xacro)
@@ -28,10 +28,10 @@
     <!-- <xacro:v1_trunk_sensors/> -->
     <!-- ===== HEAD ===== -->
-    <xacro:make_head head_root_link="${WJ3_Distal_Link}" />
+    <xacro:make_head head_root_link="${TorsoRollLinkName}" />
     <!-- <xacro:make_head_interface name1="/neck/j1" type1="${neck_type1}"
                                name2="/neck/j2" type2="${neck_type2}"
                                name3="/neck/j3" type3="${neck_type3}"/> -->
     <!-- ===== RIGHT ARM ===== -->
-    <xacro:make_arm prefix="Right" reflect="1" arm_root_link="${WJ3_Distal_Link}" />
+    <xacro:make_arm prefix="Right" reflect="1" arm_root_link="${TorsoRollLinkName}" />
     <!-- <xacro:v1_arm_actuators name1="${rightarm_name1}" type1="${arm_type1}"
                             name2="${rightarm_name2}" type2="${arm_type2}"
@@ -51,5 +51,5 @@
     <xacro:make_little_finger_fixed prefix="Right" reflect="1" little_finger_root_link="RightPalm"/>
     <!-- ===== LEFT ARM ===== -->
-    <xacro:make_arm prefix="Left" reflect="-1" arm_root_link="${WJ3_Distal_Link}" />
+    <xacro:make_arm prefix="Left" reflect="-1" arm_root_link="${TorsoRollLinkName}" />
     <!-- <xacro:v1_arm_actuators name1="${leftarm_name1}" type1="${arm_type1}"
                             name2="${leftarm_name2}" type2="${arm_type2}"

File: valkyrie_description/robots/valkyrie_A/xacro/middle_finger/link_names.xacro (robot description, xacro)
@@ -2,6 +2,6 @@
 <robot xmlns:xacro="http://www.ros.org/wiki/xacro" name="v1/middle_finger/dh_parameters">
   <xacro:property name="MiddleFingerPitch1ParentLinkName" value="${middle_finger_root_link}" />
-  <xacro:property name="MiddleFingerPitch1LinkName" value="${prefix}MiddleFingerPitch1" />
-  <xacro:property name="MiddleFingerPitch2LinkName" value="${prefix}MiddleFingerPitch2" />
-  <xacro:property name="MiddleFingerPitch3LinkName" value="${prefix}MiddleFingerPitch3" />
+  <xacro:property name="MiddleFingerPitch1LinkName" value="${prefix}MiddleFingerPitch1Link" />
+  <xacro:property name="MiddleFingerPitch2LinkName" value="${prefix}MiddleFingerPitch2Link" />
+  <xacro:property name="MiddleFingerPitch3LinkName" value="${prefix}MiddleFingerPitch3Link" />
 </robot>

File: valkyrie_description/robots/valkyrie_A/xacro/middle_finger/middle_finger.xacro (robot description, xacro)
@@ -5,5 +5,5 @@
   <xacro:include filename="$(find valkyrie_description)/robots/valkyrie_A/xacro/middle_finger/link_names.xacro"/>
   <xacro:include filename="$(find valkyrie_description)/robots/valkyrie_A/xacro/middle_finger/joint_limits.xacro"/>
-  <xacro:include filename="$(find valkyrie_description)/robots/valkyrie_A/xacro/middle_finger/dh_parameters.xacro"/>
+  <xacro:include filename="$(find valkyrie_description)/robots/valkyrie_A/xacro/middle_finger/frame_parameters.xacro"/>
   <xacro:include filename="$(find valkyrie_description)/robots/valkyrie_A/xacro/middle_finger/mass_parameters.xacro"/>
   <!-- Link properties. -->

File: valkyrie_description/robots/valkyrie_A/xacro/primary_finger/primary_finger.xacro (robot description, xacro)
@@ -5,5 +5,5 @@
   <xacro:include filename="$(find valkyrie_description)/robots/valkyrie_A/xacro/primary_finger/link_names.xacro"/>
   <xacro:include filename="$(find valkyrie_description)/robots/valkyrie_A/xacro/primary_finger/joint_limits.xacro"/>
-  <xacro:include filename="$(find valkyrie_description)/robots/valkyrie_A/xacro/primary_finger/dh_parameters.xacro"/>
+  <xacro:include filename="$(find valkyrie_description)/robots/valkyrie_A/xacro/primary_finger/frame_parameters.xacro"/>
   <xacro:include filename="$(find valkyrie_description)/robots/valkyrie_A/xacro/primary_finger/mass_parameters.xacro"/>
   <!-- Link properties. -->

File: valkyrie_description/robots/valkyrie_A/xacro/waist/joint_limits.xacro (robot description, xacro)
@@ -1,15 +1,15 @@
 <?xml version="1.0" ?>
 <robot xmlns:xacro="http://www.ros.org/wiki/xacro" name="v1/waist/joint_limits">
-  <xacro:property name="WJ1_Torque_Limit" value="190" />
-  <xacro:property name="WJ2_Torque_Limit" value="150" />
-  <xacro:property name="WJ3_Torque_Limit" value="150" />
-  <xacro:property name="WJ1_Lower_Limit" value="-0.698" />
-  <xacro:property name="WJ2_Lower_Limit" value="-0.698" />
-  <xacro:property name="WJ3_Lower_Limit" value="-0.262" />
-  <xacro:property name="WJ1_Upper_Limit" value="0.698" />
-  <xacro:property name="WJ2_Upper_Limit" value="0.087" />
-  <xacro:property name="WJ3_Upper_Limit" value="0.262" />
-  <xacro:property name="WJ1_Speed_Limit" value="5.89" />
-  <xacro:property name="WJ2_Speed_Limit" value="9" />
-  <xacro:property name="WJ3_Speed_Limit" value="9" />
+  <xacro:property name="TorsoYawTorqueLimit" value="190" />
+  <xacro:property name="TorsoPitchTorqueLimit" value="150" />
+  <xacro:property name="TorsoRollTorqueLimit" value="150" />
+  <xacro:property name="TorsoYawPositionLimit_Lower" value="-0.698" />
+  <xacro:property name="TorsoPitchPositionLimit_Lower" value="-0.698" />
+  <xacro:property name="TorsoRollPositionLimit_Lower" value="-0.262" />
+  <xacro:property name="TorsoYawPositionLimit_Upper" value="0.698" />
+  <xacro:property name="TorsoPitchPositionLimit_Upper" value="0.087" />
+  <xacro:property name="TorsoRollPositionLimit_Upper" value="0.262" />
+  <xacro:property name="TorsoYawVelocityLimit" value="5.89" />
+  <xacro:property name="TorsoPitchVelocityLimit" value="9" />
+  <xacro:property name="TorsoRollVelocityLimit" value="9" />
 </robot>

File: valkyrie_description/robots/valkyrie_A/xacro/waist/joint_names.xacro (robot description, xacro)
@@ -1,6 +1,6 @@
 <?xml version="1.0" ?>
 <robot xmlns:xacro="http://www.ros.org/wiki/xacro" name="v1/waist/mass_parameters">
-  <xacro:property name="WJ1_Joint_Name" value="TorsoYaw" />
-  <xacro:property name="WJ2_Joint_Name" value="TorsoPitch" />
-  <xacro:property name="WJ3_Joint_Name" value="TorsoRoll" />
+  <xacro:property name="TorsoYawJointName" value="TorsoYaw" />
+  <xacro:property name="TorsoPitchJointName" value="TorsoPitch" />
+  <xacro:property name="TorsoRollJointName" value="TorsoRoll" />
 </robot>

File: valkyrie_description/robots/valkyrie_A/xacro/waist/link_names.xacro (robot description, xacro)
@@ -1,9 +1,7 @@
 <?xml version="1.0" ?>
 <robot xmlns:xacro="http://www.ros.org/wiki/xacro" name="v1/waist/dh_parameters">
-  <xacro:property name="WJ1_Proximal_Link" value="${waist_root_link}" />
-  <xacro:property name="WJ1_Distal_Link" value="TorsoYaw" />
-  <xacro:property name="WJ2_Proximal_Link" value="TorsoYaw" />
-  <xacro:property name="WJ2_Distal_Link" value="TorsoPitch" />
-  <xacro:property name="WJ3_Proximal_Link" value="TorsoPitch" />
-  <xacro:property name="WJ3_Distal_Link" value="TorsoRoll" />
+  <xacro:property name="TorsoYawParentLinkName" value="${waist_root_link}" />
+  <xacro:property name="TorsoYawLinkName" value="TorsoYawLink" />
+  <xacro:property name="TorsoPitchLinkName" value="TorsoPitchLink" />
+  <xacro:property name="TorsoRollLinkName" value="Torso" />
 </robot>

File: valkyrie_description/robots/valkyrie_A/xacro/waist/mass_parameters.xacro (robot description, xacro)
@@ -1,7 +1,6 @@
 <?xml version="1.0" ?>
 <robot xmlns:xacro="http://www.ros.org/wiki/xacro" name="v1/waist/mass_parameters">
-  <xacro:property name="WJ3_Link_Mass_No_Battery_No_Neck" value="23.9" />
-  <xacro:property name="Battery_Mass" value="14.4" />
-  <xacro:property name="WJ3_Link_Mass" value="42.6" />
-  <xacro:property name="WJ3_Link_Mass_No_Battery" value="24.371" />
+	<xacro:property name="TorsoYawLinkMass" value="2.858" />
+	<xacro:property name="TorsoPitchLinkMass" value="0.001"/>
+  <xacro:property name="TorsoRollLinkMass" value="42.6" />
 </robot>
