Commit message: I seem to have renamed all joints/links.

File: valkyrie_description/robots/valkyrie_A/xacro/waist/waist.xacro (robot description, xacro)
@@ -4,5 +4,5 @@
   <xacro:include filename="$(find valkyrie_description)/robots/valkyrie_A/xacro/waist/link_names.xacro"/>
   <xacro:include filename="$(find valkyrie_description)/robots/valkyrie_A/xacro/waist/joint_limits.xacro"/>
-  <xacro:include filename="$(find valkyrie_description)/robots/valkyrie_A/xacro/waist/dh_parameters.xacro"/>
+  <xacro:include filename="$(find valkyrie_description)/robots/valkyrie_A/xacro/waist/frame_parameters.xacro"/>
   <xacro:include filename="$(find valkyrie_description)/robots/valkyrie_A/xacro/waist/mass_parameters.xacro"/>
   <xacro:include filename="$(find valkyrie_description)/robots/valkyrie_A/xacro/sensors/microstrain.xacro"/>
@@ -14,37 +14,37 @@
   <xacro:macro name="make_waist_common" params="waist_root_link">
     <!-- Links -->
-    <xacro:virtual_link name="${WJ1_Distal_Link}" origin_xyz="0 0 0" origin_rpy="0 0 0"/>
-    <xacro:virtual_link name="${WJ2_Distal_Link}" origin_xyz="0 0 0" origin_rpy="0 0 0"/>
+    <xacro:virtual_link name="${TorsoYawLinkName}" origin_xyz="0 0 0" origin_rpy="0 0 0"/>
+    <xacro:virtual_link name="${TorsoPitchLinkName}" origin_xyz="0 0 0" origin_rpy="0 0 0"/>
     <!-- WJ1 -->
-    <xacro:revolute_joint_ex jointName="${WJ1_Joint_Name}"
-                          parent="${WJ1_Proximal_Link}" child="${WJ1_Distal_Link}"
-                          origin_xyz="${WJ1_Origin_X} ${WJ1_Origin_Y} ${WJ1_Origin_Z}"
-                          origin_rpy="${WJ1_Orientation_Roll} ${WJ1_Orientation_Pitch} ${WJ1_Orientation_Yaw}"
+    <xacro:revolute_joint_ex jointName="${TorsoYawJointName}"
+                          parent="${TorsoYawParentLinkName}" child="${TorsoYawLinkName}"
+                          origin_xyz="${TorsoYawFrameOrigin_X} ${TorsoYawFrameOrigin_Y} ${TorsoYawFrameOrigin_Z}"
+                          origin_rpy="${TorsoYawFrameOrientation_Roll} ${TorsoYawFrameOrientation_Pitch} ${TorsoYawFrameOrientation_Yaw}"
                           damping="1.0" friction="0.0">
-        <limit effort="${WJ1_Torque_Limit}" lower="${WJ1_Lower_Limit}" upper="${WJ1_Upper_Limit}" velocity="${WJ1_Speed_Limit}"/>
+        <limit effort="${TorsoYawTorqueLimit}" lower="${TorsoYawPositionLimit_Lower}" upper="${TorsoYawPositionLimit_Upper}" velocity="${TorsoYawVelocityLimit}"/>
         <controller_gains Kp="20000" Kd="400"/>
     </xacro:revolute_joint_ex>
     <!-- WJ2 -->
-    <xacro:revolute_joint_ex jointName="${WJ2_Joint_Name}"
-                          parent="${WJ2_Proximal_Link}" child="${WJ2_Distal_Link}"
-                          origin_xyz="${WJ2_Origin_X} ${WJ2_Origin_Y} ${WJ2_Origin_Z}"
-                          origin_rpy="${WJ2_Orientation_Roll} ${WJ2_Orientation_Pitch} ${WJ2_Orientation_Yaw}"
+    <xacro:revolute_joint_ex jointName="${TorsoPitchJointName}"
+                          parent="${TorsoYawLinkName}" child="${TorsoPitchLinkName}"
+                          origin_xyz="${TorsoPitchFrameOrigin_X} ${TorsoPitchFrameOrigin_Y} ${TorsoPitchFrameOrigin_Z}"
+                          origin_rpy="${TorsoPitchFrameOrientation_Roll} ${TorsoPitchFrameOrientation_Pitch} ${TorsoPitchFrameOrientation_Yaw}"
                           damping="1.0" friction="0.0">
-        <limit effort="${WJ2_Torque_Limit}" lower="${WJ2_Lower_Limit}" upper="${WJ2_Upper_Limit}" velocity="${WJ2_Speed_Limit}"/>
+        <limit effort="${TorsoPitchTorqueLimit}" lower="${TorsoPitchPositionLimit_Lower}" upper="${TorsoPitchPositionLimit_Upper}" velocity="${TorsoPitchVelocityLimit}"/>
         <controller_gains Kp="20000" Kd="400"/>
     </xacro:revolute_joint_ex>
     <!-- WJ3 -->
-    <xacro:revolute_joint_ex jointName="${WJ3_Joint_Name}"
-                          parent="${WJ3_Proximal_Link}" child="${WJ3_Distal_Link}"
-                          origin_xyz="${WJ3_Origin_X} ${WJ3_Origin_Y} ${WJ3_Origin_Z}"
-                          origin_rpy="${WJ3_Orientation_Roll} ${WJ3_Orientation_Pitch} ${WJ3_Orientation_Yaw}"
+    <xacro:revolute_joint_ex jointName="${TorsoRollJointName}"
+                          parent="${TorsoPitchLinkName}" child="${TorsoRollLinkName}"
+                          origin_xyz="${TorsoRollFrameOrigin_X} ${TorsoRollFrameOrigin_Y} ${TorsoRollFrameOrigin_Z}"
+                          origin_rpy="${TorsoRollFrameOrientation_Roll} ${TorsoRollFrameOrientation_Pitch} ${TorsoRollFrameOrientation_Yaw}"
                           damping="1.0" friction="0.0">
-        <limit effort="${WJ3_Torque_Limit}" lower="${WJ3_Lower_Limit}" upper="${WJ3_Upper_Limit}" velocity="${WJ3_Speed_Limit}"/>
+        <limit effort="${TorsoRollTorqueLimit}" lower="${TorsoRollPositionLimit_Lower}" upper="${TorsoRollPositionLimit_Upper}" velocity="${TorsoRollVelocityLimit}"/>
         <controller_gains Kp="20000" Kd="400"/>
     </xacro:revolute_joint_ex>
   </xacro:macro>
   <xacro:macro name="make_waist" params="waist_root_link">
-    <xacro:box_link name="${WJ3_Distal_Link}"
-                    width="${Trunk_Width}" height="${Trunk_Height}" depth="${Trunk_Length}" mass="${WJ3_Link_Mass}"
+    <xacro:box_link name="${TorsoRollLinkName}"
+                    width="${Trunk_Width}" height="${Trunk_Height}" depth="${Trunk_Length}" mass="${TorsoRollLinkMass}"
                     origin_rpy="0 0 0"
                     origin_xyz="0.219 0.03 -0.104"
@@ -54,30 +54,10 @@
     <xacro:make_waist_common waist_root_link="${waist_root_link}"/>
   </xacro:macro>
-  <xacro:macro name="make_waist_no_battery_no_nj1" params="waist_root_link">
-    <xacro:box_link name="${WJ3_Distal_Link}"
-                    width="${Trunk_Width}" height="${Trunk_Height}" depth="${Trunk_Length}" mass="${WJ3_Link_Mass_No_Battery_No_Neck}"
-                    origin_rpy="0 0 0"
-                    origin_xyz="0.239 0 -0.060"
-                    visual_mesh="${mesh_root}/wj3.stl"
-                    material="White"
-                    collision_mesh="${mesh_root}/wj3.stl" />
-    <xacro:make_waist_common waist_root_link="${waist_root_link}"/>
-  </xacro:macro>
-  <xacro:macro name="make_waist_no_battery" params="waist_root_link">
-    <xacro:box_link name="${WJ3_Distal_Link}"
-                    width="${Trunk_Width}" height="${Trunk_Height}" depth="${Trunk_Length}" mass="${WJ3_Link_Mass_No_Battery_No_Neck + NJ1_Link_Mass}"
-                    origin_rpy="0 0 0"
-                    origin_xyz="0.239 0 -0.060"
-                    visual_mesh="${mesh_root}/wj3.stl"
-                    material="White"
-                    collision_mesh="${mesh_root}/wj3.stl" />
-    <xacro:make_waist_common waist_root_link="${waist_root_link}"/>
-  </xacro:macro>
   <xacro:macro name="make_fixed_waist" params="waist_root_link">
     <!-- Links -->
-    <xacro:virtual_link name="${WJ1_Distal_Link}" origin_xyz="0 0 0" origin_rpy="0 0 0"/>
-    <xacro:virtual_link name="${WJ2_Distal_Link}" origin_xyz="0 0 0" origin_rpy="0 0 0"/>
-    <xacro:box_link name="${WJ3_Distal_Link}"
-                    width="${Trunk_Width}" height="${Trunk_Height}" depth="${Trunk_Length}" mass="${WJ3_Link_Mass}"
+    <xacro:virtual_link name="${TorsoYawLinkName}" origin_xyz="0 0 0" origin_rpy="0 0 0"/>
+    <xacro:virtual_link name="${TorsoPitchLinkName}" origin_xyz="0 0 0" origin_rpy="0 0 0"/>
+    <xacro:box_link name="${TorsoRollLinkName}"
+                    width="${Trunk_Width}" height="${Trunk_Height}" depth="${Trunk_Length}" mass="${TorsoRollLinkMass}"
                     origin_rpy="0 0 0"
                     origin_xyz="0.226 0 -0.078"
@@ -86,29 +66,29 @@
                     collision_mesh="${mesh_root}/wj3.stl" />
     <!-- WJ1 -->
-    <xacro:fixed_joint jointName="${WJ1_Joint_Name}"
-                          parent="${WJ1_Proximal_Link}" child="${WJ1_Distal_Link}"
-                          origin_xyz="${WJ1_Origin_X} ${WJ1_Origin_Y} ${WJ1_Origin_Z}"
-                          origin_rpy="${WJ1_Orientation_Roll} ${WJ1_Orientation_Pitch} ${WJ1_Orientation_Yaw}">
-        <limit effort="${WJ1_Torque_Limit}" lower="${WJ1_Lower_Limit}" upper="${WJ1_Upper_Limit}" velocity="${WJ1_Speed_Limit}"/>
+    <xacro:fixed_joint jointName="${TorsoYawJointName}"
+                          parent="${TorsoYawParentLinkName}" child="${TorsoYawLinkName}"
+                          origin_xyz="${TorsoYawFrameOrigin_X} ${TorsoYawFrameOrigin_Y} ${TorsoYawFrameOrigin_Z}"
+                          origin_rpy="${TorsoYawFrameOrientation_Roll} ${TorsoYawFrameOrientation_Pitch} ${TorsoYawFrameOrientation_Yaw}">
+        <limit effort="${TorsoYawTorqueLimit}" lower="${TorsoYawPositionLimit_Lower}" upper="${TorsoYawPositionLimit_Upper}" velocity="${TorsoYawVelocityLimit}"/>
     </xacro:fixed_joint>
     <!-- WJ2 -->
-    <xacro:fixed_joint jointName="${WJ2_Joint_Name}"
-                          parent="${WJ2_Proximal_Link}" child="${WJ2_Distal_Link}"
-                          origin_xyz="${WJ2_Origin_X} ${WJ2_Origin_Y} ${WJ2_Origin_Z}"
-                          origin_rpy="${WJ2_Orientation_Roll} ${WJ2_Orientation_Pitch} ${WJ2_Orientation_Yaw}">
-        <limit effort="${WJ2_Torque_Limit}" lower="${WJ2_Lower_Limit}" upper="${WJ2_Upper_Limit}" velocity="${WJ2_Speed_Limit}"/>
+    <xacro:fixed_joint jointName="${TorsoPitchJointName}"
+                          parent="${TorsoYawLinkName}" child="${TorsoPitchLinkName}"
+                          origin_xyz="${TorsoPitchFrameOrigin_X} ${TorsoPitchFrameOrigin_Y} ${TorsoPitchFrameOrigin_Z}"
+                          origin_rpy="${TorsoPitchFrameOrientation_Roll} ${TorsoPitchFrameOrientation_Pitch} ${TorsoPitchFrameOrientation_Yaw}">
+        <limit effort="${TorsoPitchTorqueLimit}" lower="${TorsoPitchPositionLimit_Lower}" upper="${TorsoPitchPositionLimit_Upper}" velocity="${TorsoPitchVelocityLimit}"/>
     </xacro:fixed_joint>
     <!-- WJ3 -->
-    <xacro:fixed_joint jointName="${WJ3_Joint_Name}"
-                          parent="${WJ3_Proximal_Link}" child="${WJ3_Distal_Link}"
-                          origin_xyz="${WJ3_Origin_X} ${WJ3_Origin_Y} ${WJ3_Origin_Z}"
-                          origin_rpy="${WJ3_Orientation_Roll} ${WJ3_Orientation_Pitch} ${WJ3_Orientation_Yaw}">
-        <limit effort="${WJ3_Torque_Limit}" lower="${WJ3_Lower_Limit}" upper="${WJ3_Upper_Limit}" velocity="${WJ3_Speed_Limit}"/>
+    <xacro:fixed_joint jointName="${TorsoRollJointName}"
+                          parent="${TorsoPitchLinkName}" child="${TorsoRollLinkName}"
+                          origin_xyz="${TorsoRollFrameOrigin_X} ${TorsoRollFrameOrigin_Y} ${TorsoRollFrameOrigin_Z}"
+                          origin_rpy="${TorsoRollFrameOrientation_Roll} ${TorsoRollFrameOrientation_Pitch} ${TorsoRollFrameOrientation_Yaw}">
+        <limit effort="${TorsoRollTorqueLimit}" lower="${TorsoRollPositionLimit_Lower}" upper="${TorsoRollPositionLimit_Upper}" velocity="${TorsoRollVelocityLimit}"/>
     </xacro:fixed_joint>
   </xacro:macro>
   <xacro:macro name="make_no_waist">
     <!-- Links -->
-    <xacro:box_link name="${WJ3_Distal_Link}"
-                    width="${Trunk_Width}" height="${Trunk_Height}" depth="${Trunk_Length}" mass="${WJ3_Link_Mass}"
+    <xacro:box_link name="${TorsoRollLinkName}"
+                    width="${Trunk_Width}" height="${Trunk_Height}" depth="${Trunk_Length}" mass="${TorsoRollLinkMass}"
                     origin_rpy="0 0 0"
                     origin_xyz="0 0 0"
@@ -119,10 +99,10 @@
   <xacro:macro name="make_waist_fixed_wj2_wj3" params="waist_root_link">
     <!-- Links -->
-    <!-- <xacro:virtual_link name="${WJ1_Distal_Link}" origin_xyz="0 0 0" origin_rpy="0 0 0"/> -->
+    <!-- <xacro:virtual_link name="${TorsoYawLinkName}" origin_xyz="0 0 0" origin_rpy="0 0 0"/> -->
     <!--NOTE : This is for lower body testbed setup-->
     <xacro:link_no_mesh
-      name="${WJ1_Distal_Link}"
+      name="${TorsoYawLinkName}"
       width="0.01" height="0.01" depth="0.01"
-      mass="2.858"
+      mass="${TorsoYawLinkMass}"
       origin_xyz="0.0008 0.0002 0.0221"
       origin_rpy="0 0 0"
@@ -130,28 +110,28 @@
       iyy="1.12e-2" iyz="1.07e-5"
       izz="1.181e-2"/>
-    <xacro:virtual_link name="${WJ2_Distal_Link}" origin_xyz="0 0 0" origin_rpy="0 0 0"/>
-    <xacro:virtual_link name="${WJ3_Distal_Link}" origin_rpy="0 0 0" origin_xyz="0.226 0 -0.078" />
+    <xacro:virtual_link name="${TorsoPitchLinkName}" origin_xyz="0 0 0" origin_rpy="0 0 0"/>
+    <xacro:virtual_link name="${TorsoRollLinkName}" origin_rpy="0 0 0" origin_xyz="0.226 0 -0.078" />
     <!-- WJ1 -->
-    <xacro:revolute_joint_ex jointName="${WJ1_Joint_Name}"
-                          parent="${WJ1_Proximal_Link}" child="${WJ1_Distal_Link}"
-                          origin_xyz="${WJ1_Origin_X} ${WJ1_Origin_Y} ${WJ1_Origin_Z}"
-                          origin_rpy="${WJ1_Orientation_Roll} ${WJ1_Orientation_Pitch} ${WJ1_Orientation_Yaw}"
+    <xacro:revolute_joint_ex jointName="${TorsoYawJointName}"
+                          parent="${TorsoYawParentLinkName}" child="${TorsoYawLinkName}"
+                          origin_xyz="${TorsoYawFrameOrigin_X} ${TorsoYawFrameOrigin_Y} ${TorsoYawFrameOrigin_Z}"
+                          origin_rpy="${TorsoYawFrameOrientation_Roll} ${TorsoYawFrameOrientation_Pitch} ${TorsoYawFrameOrientation_Yaw}"
                           damping="1.0" friction="0.0">
-        <limit effort="${WJ1_Torque_Limit}" lower="${WJ1_Lower_Limit}" upper="${WJ1_Upper_Limit}" velocity="${WJ1_Speed_Limit}"/>
+        <limit effort="${TorsoYawTorqueLimit}" lower="${TorsoYawPositionLimit_Lower}" upper="${TorsoYawPositionLimit_Upper}" velocity="${TorsoYawVelocityLimit}"/>
         <controller_gains Kp="20000" Kd="400"/>
     </xacro:revolute_joint_ex>
     <!-- WJ2 -->
-    <xacro:fixed_joint jointName="${WJ2_Joint_Name}"
-                          parent="${WJ2_Proximal_Link}" child="${WJ2_Distal_Link}"
-                          origin_xyz="${WJ2_Origin_X} ${WJ2_Origin_Y} ${WJ2_Origin_Z}"
-                          origin_rpy="${WJ2_Orientation_Roll} ${WJ2_Orientation_Pitch} ${WJ2_Orientation_Yaw}">
-        <limit effort="${WJ2_Torque_Limit}" lower="${WJ2_Lower_Limit}" upper="${WJ2_Upper_Limit}" velocity="${WJ2_Speed_Limit}"/>
+    <xacro:fixed_joint jointName="${TorsoPitchJointName}"
+                          parent="${TorsoYawLinkName}" child="${TorsoPitchLinkName}"
+                          origin_xyz="${TorsoPitchFrameOrigin_X} ${TorsoPitchFrameOrigin_Y} ${TorsoPitchFrameOrigin_Z}"
+                          origin_rpy="${TorsoPitchFrameOrientation_Roll} ${TorsoPitchFrameOrientation_Pitch} ${TorsoPitchFrameOrientation_Yaw}">
+        <limit effort="${TorsoPitchTorqueLimit}" lower="${TorsoPitchPositionLimit_Lower}" upper="${TorsoPitchPositionLimit_Upper}" velocity="${TorsoPitchVelocityLimit}"/>
     </xacro:fixed_joint>
     <!-- WJ3 -->
-    <xacro:fixed_joint jointName="${WJ3_Joint_Name}"
-                          parent="${WJ3_Proximal_Link}" child="${WJ3_Distal_Link}"
-                          origin_xyz="${WJ3_Origin_X} ${WJ3_Origin_Y} ${WJ3_Origin_Z}"
-                          origin_rpy="${WJ3_Orientation_Roll} ${WJ3_Orientation_Pitch} ${WJ3_Orientation_Yaw}">
-        <limit effort="${WJ3_Torque_Limit}" lower="${WJ3_Lower_Limit}" upper="${WJ3_Upper_Limit}" velocity="${WJ3_Speed_Limit}"/>
+    <xacro:fixed_joint jointName="${TorsoRollJointName}"
+                          parent="${TorsoPitchLinkName}" child="${TorsoRollLinkName}"
+                          origin_xyz="${TorsoRollFrameOrigin_X} ${TorsoRollFrameOrigin_Y} ${TorsoRollFrameOrigin_Z}"
+                          origin_rpy="${TorsoRollFrameOrientation_Roll} ${TorsoRollFrameOrientation_Pitch} ${TorsoRollFrameOrientation_Yaw}">
+        <limit effort="${TorsoRollTorqueLimit}" lower="${TorsoRollPositionLimit_Lower}" upper="${TorsoRollPositionLimit_Upper}" velocity="${TorsoRollVelocityLimit}"/>
     </xacro:fixed_joint>
   </xacro:macro>
@@ -171,13 +151,13 @@
      -->
     <xacro:microstrain_sensor sensorName="/v1/RightIMU"
-                              parentLink="${WJ3_Distal_Link}"
+                              parentLink="${TorsoRollLinkName}"
                               origin_xyz="0.363038 0.134239 -0.0468630"
                               origin_rpy="-1.57 1.57 0" />
     <xacro:microstrain_sensor sensorName="/v1/LeftIMU"
-                              parentLink="${WJ3_Distal_Link}"
+                              parentLink="${TorsoRollLinkName}"
                               origin_xyz="0.363038 -0.134239  -0.0468630"
                               origin_rpy="1.57 1.57 0" />
     <xacro:flea3_camera sensorName="/v1/RightHazardCamera"
-                        parentLink="${WJ3_Distal_Link}"
+                        parentLink="${TorsoRollLinkName}"
                         origin_xyz="0.0446987 0.0406146 0.0182674"
                         origin_rpy="0 0 0"
@@ -185,5 +165,5 @@
                         frameRate="60"/>
     <xacro:flea3_camera sensorName="/v1/LeftHazardCamera"
-                        parentLink="${WJ3_Distal_Link}"
+                        parentLink="${TorsoRollLinkName}"
                         origin_xyz="0.0446987 -0.0406146 0.0182674"
                         origin_rpy="0 0 0"
@@ -191,5 +171,5 @@
                         frameRate="60"/>
     <xacro:massless_virtual_sensor sensorName="/v1/StereoHazardCamera"
-                          parentLink="${WJ3_Distal_Link}"
+                          parentLink="${TorsoRollLinkName}"
                           origin_xyz=".1723 -0.04535 0.0344"
                           origin_rpy="0 0 1.57" />
@@ -197,7 +177,7 @@
   <!-- Transmissions -->
   <xacro:macro name="v1_waist_transmissions" params="actuator1 actuator2 actuator3">
-    <xacro:simple_transmission jointName="${WJ1_Joint_Name}" actuatorName="${actuator1}" reduction="1" offset="0"/>
+    <xacro:simple_transmission jointName="${TorsoYawJointName}" actuatorName="${actuator1}" reduction="1" offset="0"/>
     <xacro:pushrod_transmission tranName="Waist" namespace="v1_waist"
-                                joint1="${WJ2_Joint_Name}" joint2="${WJ3_Joint_Name}"
+                                joint1="${TorsoPitchJointName}" joint2="${TorsoRollJointName}"
                                 actuator1="${actuator2}"   actuator2="${actuator3}"
                                 reflect="1"/>
@@ -205,24 +185,13 @@
   </xacro:macro>
   <xacro:macro name="v1_waist_transmissions_simple" params="actuator1 actuator2 actuator3">
-    <xacro:simple_transmission jointName="${WJ1_Joint_Name}" actuatorName="${actuator1}" reduction="1" offset="0"/>
-    <xacro:simple_transmission jointName="${WJ2_Joint_Name}" actuatorName="${actuator2}" reduction="1" offset="0"/>
-    <xacro:simple_transmission jointName="${WJ3_Joint_Name}" actuatorName="${actuator3}" reduction="1" offset="0"/>
+    <xacro:simple_transmission jointName="${TorsoYawJointName}" actuatorName="${actuator1}" reduction="1" offset="0"/>
+    <xacro:simple_transmission jointName="${TorsoPitchJointName}" actuatorName="${actuator2}" reduction="1" offset="0"/>
+    <xacro:simple_transmission jointName="${TorsoRollJointName}" actuatorName="${actuator3}" reduction="1" offset="0"/>
   </xacro:macro>
   <!-- Modes -->
   <xacro:macro name="v1_waist_modes" params="actuator1 actuator2 actuator3">
-    <xacro:v1_modes jointName="${WJ1_Joint_Name}" actuatorName="${actuator1}" />
-    <xacro:v1_modes jointName="${WJ2_Joint_Name}" actuatorName="${actuator2}" />
-    <xacro:v1_modes jointName="${WJ3_Joint_Name}" actuatorName="${actuator3}" />
+    <xacro:v1_modes jointName="${TorsoYawJointName}" actuatorName="${actuator1}" />
+    <xacro:v1_modes jointName="${TorsoPitchJointName}" actuatorName="${actuator2}" />
+    <xacro:v1_modes jointName="${TorsoRollJointName}" actuatorName="${actuator3}" />
   </xacro:macro>
-  <!-- Battery -->
-  <!-- TODO: Get better numbers for battery center from mech team -->
-  <!-- <xacro:fixed_joint jointName="battery_offset"
-                     parent="/v1/trunk" child="/v1/battery"
-                     origin_xyz=".3 0 -0.2"
-                     origin_rpy="0 0 0" /> -->
-  <!-- TODO: Get better approximation for battery -->
-  <!-- <xacro:link_box name="/v1/battery"
-                  width=".2" height="0.2" depth="0.2" mass="15.0"
-                  origin_rpy="0 0 0"
-                  origin_xyz="0 0 0" /> -->
 </robot>
