Commit message: Rename primary to index because I really don't like primary.

File: valkyrie_description/robots/valkyrie_A/xacro/V1_sim_base.xacro (robot description, xacro)
@@ -45,5 +45,5 @@
     <xacro:make_thumb_fixed prefix="Right" reflect="1" thumb_root_link="RightPalm"/>
     <!-- ===== RIGHT PRIMARY FINGER ===== -->
-    <xacro:make_primary_finger_fixed prefix="Right" reflect="1" primary_finger_root_link="RightPalm"/>
+    <xacro:make_index_finger_fixed prefix="Right" reflect="1" index_finger_root_link="RightPalm"/>
     <!-- ===== RIGHT MIDDLE FINGER ===== -->
     <xacro:make_middle_finger_fixed prefix="Right" reflect="1" middle_finger_root_link="RightPalm"/>
@@ -62,5 +62,5 @@
     <xacro:make_thumb_fixed prefix="Left" reflect="-1" thumb_root_link="LeftPalm"/>
     <!-- ===== LEFT PRIMARY FINGER ===== -->
-    <xacro:make_primary_finger_fixed prefix="Left" reflect="-1" primary_finger_root_link="LeftPalm"/>
+    <xacro:make_index_finger_fixed prefix="Left" reflect="-1" index_finger_root_link="LeftPalm"/>
     <!-- ===== LEFT MIDDLE FINGER ===== -->
     <xacro:make_middle_finger_fixed prefix="Left" reflect="-1" middle_finger_root_link="LeftPalm"/>

File: valkyrie_description/robots/valkyrie_A/xacro/arm/frame_parameters.xacro (robot description, xacro)
@@ -1,13 +1,13 @@
 <?xml version="1.0" ?>
 <robot xmlns:xacro="http://www.ros.org/wiki/xacro" name="v1/arm/dh_parameters">
-  <xacro:property name="ShoulderPitchFrameOrigin_X" value="0.29842"/>
-  <xacro:property name="ShoulderPitchFrameOrigin_Y" value="0"/>
-  <xacro:property name="ShoulderPitchFrameOrigin_Z" value="-0.03157"/>
+  <xacro:property name="ShoulderPitchFrameOrigin_X" value="-0.0316"/>
+  <xacro:property name="ShoulderPitchFrameOrigin_Y" value="0.0"/>
+  <xacro:property name="ShoulderPitchFrameOrigin_Z" value="0.2984"/>
   <xacro:property name="ShoulderPitchFrameOrientation_Roll" value="0.0"/>
   <xacro:property name="ShoulderPitchFrameOrientation_Pitch" value="0.0"/>
   <xacro:property name="ShoulderPitchFrameOrientation_Yaw" value="0.0"/>
-  <xacro:property name="ShoulderRollFrameOrigin_X" value="0"/>
-  <xacro:property name="ShoulderRollFrameOrigin_Y" value="0"/>
-  <xacro:property name="ShoulderRollFrameOrigin_Z" value="${reflect * -0.246}"/>
+  <xacro:property name="ShoulderRollFrameOrigin_X" value="0.0"/>
+  <xacro:property name="ShoulderRollFrameOrigin_Y" value="${reflect * 0.2499}"/>
+  <xacro:property name="ShoulderRollFrameOrigin_Z" value="0.0"/>
   <xacro:property name="ShoulderRollFrameOrientation_Roll" value="0.0"/>
   <xacro:property name="ShoulderRollFrameOrientation_Pitch" value="0.0"/>
@@ -19,11 +19,11 @@
   <xacro:property name="ShoulderYawFrameOrientation_Pitch" value="0.0"/>
   <xacro:property name="ShoulderYawFrameOrientation_Yaw" value="0.0"/>
-  <xacro:property name="ElbowPitchFrameOrigin_X" value="0"/>
-  <xacro:property name="ElbowPitchFrameOrigin_Y" value="${reflect * -0.0254}"/>
-  <xacro:property name="ElbowPitchFrameOrigin_Z" value="${reflect * -0.330}"/>
+  <xacro:property name="ElbowPitchFrameOrigin_X" value="0.0254"/>
+  <xacro:property name="ElbowPitchFrameOrigin_Y" value="${reflect * 0.33}"/>
+  <xacro:property name="ElbowPitchFrameOrigin_Z" value="0.0"/>
   <xacro:property name="ElbowPitchFrameOrientation_Roll" value="0.0"/>
   <xacro:property name="ElbowPitchFrameOrientation_Pitch" value="0.0"/>
   <xacro:property name="ElbowPitchFrameOrientation_Yaw" value="0.0"/>
-  <xacro:property name="ForearmYawFrameOrigin_X" value="0.0254"/>
+  <xacro:property name="ForearmYawFrameOrigin_X" value="-0.0254"/>
   <xacro:property name="ForearmYawFrameOrigin_Y" value="0"/>
   <xacro:property name="ForearmYawFrameOrigin_Z" value="0"/>
@@ -31,7 +31,7 @@
   <xacro:property name="ForearmYawFrameOrientation_Pitch" value="0.0"/>
   <xacro:property name="ForearmYawFrameOrientation_Yaw" value="0.0"/>
-  <xacro:property name="WristRollFrameOrigin_X" value="0"/>
-  <xacro:property name="WristRollFrameOrigin_Y" value="0"/>
-  <xacro:property name="WristRollFrameOrigin_Z" value="${reflect * -0.287}"/>
+  <xacro:property name="WristRollFrameOrigin_X" value="0.0"/>
+  <xacro:property name="WristRollFrameOrigin_Y" value="${reflect * 0.2871}"/>
+  <xacro:property name="WristRollFrameOrigin_Z" value="0.0"/>
   <xacro:property name="WristRollFrameOrientation_Roll" value="0.0"/>
   <xacro:property name="WristRollFrameOrientation_Pitch" value="0.0"/>

File: valkyrie_description/robots/valkyrie_A/xacro/common/common_bodies.xacro (robot description, xacro)
@@ -6,5 +6,5 @@
     <xacro:include filename="$(find valkyrie_description)/robots/valkyrie_A/xacro/leg/leg.xacro" />
     <xacro:include filename="$(find valkyrie_description)/robots/valkyrie_A/xacro/thumb/thumb.xacro" />
-    <xacro:include filename="$(find valkyrie_description)/robots/valkyrie_A/xacro/primary_finger/primary_finger.xacro" />
+    <xacro:include filename="$(find valkyrie_description)/robots/valkyrie_A/xacro/index_finger/index_finger.xacro" />
     <xacro:include filename="$(find valkyrie_description)/robots/valkyrie_A/xacro/middle_finger/middle_finger.xacro" />
     <xacro:include filename="$(find valkyrie_description)/robots/valkyrie_A/xacro/little_finger/little_finger.xacro" />

File: valkyrie_description/robots/valkyrie_A/xacro/head/frame_parameters.xacro (robot description, xacro)
@@ -1,17 +1,17 @@
 <?xml version="1.0" ?>
 <robot xmlns:xacro="http://www.ros.org/wiki/xacro" name="v1/head/dh_parameters">
-  <xacro:property name="LowerNeckPitchFrameOrigin_X" value="0.3383"/>
-  <xacro:property name="LowerNeckPitchFrameOrigin_Y" value="0"/>
-  <xacro:property name="LowerNeckPitchFrameOrigin_Z" value="0.0519"/>
+  <xacro:property name="LowerNeckPitchFrameOrigin_X" value="0.0204"/>
+  <xacro:property name="LowerNeckPitchFrameOrigin_Y" value="0.0"/>
+  <xacro:property name="LowerNeckPitchFrameOrigin_Z" value="0.3385"/>
   <xacro:property name="LowerNeckPitchFrameOrientation_Roll" value="0.0"/>
   <xacro:property name="LowerNeckPitchFrameOrientation_Pitch" value="0.0"/>
   <xacro:property name="LowerNeckPitchFrameOrientation_Yaw" value="0.0"/>
-  <xacro:property name="NeckShoulderYawFrameOrigin_X" value="0"/>
-  <xacro:property name="NeckShoulderYawFrameOrigin_Y" value="0.0519"/>
-  <xacro:property name="NeckShoulderYawFrameOrigin_Z" value="0"/>
+  <xacro:property name="NeckYawFrameOrigin_X" value="-0.0519"/>
+  <xacro:property name="NeckYawFrameOrigin_Y" value="0.0"/>
+  <xacro:property name="NeckYawFrameOrigin_Z" value="0.0"/>
   <xacro:property name="NeckYawFrameOrientation_Roll" value="0.0"/>
   <xacro:property name="NeckYawFrameOrientation_Pitch" value="0.0"/>
   <xacro:property name="NeckYawFrameOrientation_Yaw" value="0.0"/>
-  <xacro:property name="UpperNeckPitchFrameOrigin_X" value="0.06"/>
+  <xacro:property name="UpperNeckPitchFrameOrigin_X" value="-0.06"/>
   <xacro:property name="UpperNeckPitchFrameOrigin_Y" value="0"/>
   <xacro:property name="UpperNeckPitchFrameOrigin_Z" value="0.196"/>

File: valkyrie_description/robots/valkyrie_A/xacro/head/head.xacro (robot description, xacro)
@@ -45,5 +45,5 @@
     <xacro:revolute_joint_ex jointName="${NeckYawJointName}"
                           parent="${LowerNeckPitchLinkName}" child="${NeckYawLinkName}"
-                          origin_xyz="${NeckShoulderYawFrameOrigin_X} ${NeckShoulderYawFrameOrigin_Y} ${NeckShoulderYawFrameOrigin_Z}"
+                          origin_xyz="${NeckYawFrameOrigin_X} ${NeckYawFrameOrigin_Y} ${NeckYawFrameOrigin_Z}"
                           origin_rpy="${NeckYawFrameOrientation_Roll} ${NeckYawFrameOrientation_Pitch} ${NeckYawFrameOrientation_Yaw}"
                           damping="1.0" friction="0.0">
@@ -87,5 +87,5 @@
     <xacro:fixed_joint jointName="${NeckYawJointName}"
                           parent="${LowerNeckPitchLinkName}" child="${NeckYawLinkName}"
-                          origin_xyz="${NeckShoulderYawFrameOrigin_X} ${NeckShoulderYawFrameOrigin_Y} ${NeckShoulderYawFrameOrigin_Z}"
+                          origin_xyz="${NeckYawFrameOrigin_X} ${NeckYawFrameOrigin_Y} ${NeckYawFrameOrigin_Z}"
                           origin_rpy="${NeckYawFrameOrientation_Roll} ${NeckYawFrameOrientation_Pitch} ${NeckYawFrameOrientation_Yaw}">
       <limit effort="${NeckYawTorqueLimit}" lower="${NeckYawPositionLimit_Lower}" upper="${NeckYawPositionLimit_Upper}" velocity="${NeckYawVelocityLimit}"/>

File: valkyrie_description/robots/valkyrie_A/xacro/index_finger/actuator_names.xacro (robot description, xacro)
@@ -1,4 +1,4 @@
 <?xml version="1.0" ?>
-<robot xmlns:xacro="http://www.ros.org/wiki/xacro" name="v1/arm/primary_finger/actuator_names">
+<robot xmlns:xacro="http://www.ros.org/wiki/xacro" name="v1/arm/index_finger/actuator_names">
   <xacro:property name="RPFA_Actuator_Name" value="/right_arm/forearm_driver2/index" />
   <xacro:property name="LPFA_Actuator_Name" value="/left_arm/forearm_driver2/index" />

File: valkyrie_description/robots/valkyrie_A/xacro/index_finger/frame_parameters.xacro (robot description, xacro)
@@ -1,4 +1,4 @@
 <?xml version="1.0" ?>
-<robot xmlns:xacro="http://www.ros.org/wiki/xacro" name="v1/primary_finger/dh_parameters">
+<robot xmlns:xacro="http://www.ros.org/wiki/xacro" name="v1/index_finger/dh_parameters">
   <xacro:property name="IndexFingerPitch1FrameOrigin_X" value="0.0776738914821"/>
   <xacro:property name="IndexFingerPitch1FrameOrigin_Y" value="-0.0298162134085"/>

File: valkyrie_description/robots/valkyrie_A/xacro/index_finger/index_finger.xacro (robot description, xacro)
@@ -1,10 +1,10 @@
 <?xml version="1.0" ?>
-<robot xmlns:xacro="http://www.ros.org/wiki/xacro" name="v1/primary_finger">
-  <xacro:include filename="$(find valkyrie_description)/robots/valkyrie_A/xacro/primary_finger/joint_names.xacro"/>
-  <xacro:include filename="$(find valkyrie_description)/robots/valkyrie_A/xacro/primary_finger/actuator_names.xacro"/>
-  <xacro:include filename="$(find valkyrie_description)/robots/valkyrie_A/xacro/primary_finger/link_names.xacro"/>
-  <xacro:include filename="$(find valkyrie_description)/robots/valkyrie_A/xacro/primary_finger/joint_limits.xacro"/>
-  <xacro:include filename="$(find valkyrie_description)/robots/valkyrie_A/xacro/primary_finger/frame_parameters.xacro"/>
-  <xacro:include filename="$(find valkyrie_description)/robots/valkyrie_A/xacro/primary_finger/mass_parameters.xacro"/>
+<robot xmlns:xacro="http://www.ros.org/wiki/xacro" name="v1/index_finger">
+  <xacro:include filename="$(find valkyrie_description)/robots/valkyrie_A/xacro/index_finger/joint_names.xacro"/>
+  <xacro:include filename="$(find valkyrie_description)/robots/valkyrie_A/xacro/index_finger/actuator_names.xacro"/>
+  <xacro:include filename="$(find valkyrie_description)/robots/valkyrie_A/xacro/index_finger/link_names.xacro"/>
+  <xacro:include filename="$(find valkyrie_description)/robots/valkyrie_A/xacro/index_finger/joint_limits.xacro"/>
+  <xacro:include filename="$(find valkyrie_description)/robots/valkyrie_A/xacro/index_finger/frame_parameters.xacro"/>
+  <xacro:include filename="$(find valkyrie_description)/robots/valkyrie_A/xacro/index_finger/mass_parameters.xacro"/>
   <xacro:property name="PFJ1_Link_Width" value="0.029"/>
   <xacro:property name="PFJ1_Link_Height" value="0.019"/>
@@ -31,5 +31,5 @@
   <xacro:property name="PFJ4_Link_Origin_Y" value="-0.000696"/>
   <xacro:property name="PFJ4_Link_Origin_Z" value="0"/>
-  <xacro:macro name="make_primary_finger" params="prefix reflect primary_finger_root_link">
+  <xacro:macro name="make_index_finger" params="prefix reflect index_finger_root_link">
     <xacro:box_link name="${IndexFingerPitch1LinkName}"
                     width="${PFJ1_Link_Width}" height="${PFJ1_Link_Height}" depth="${PFJ1_Link_Length}" mass="${IndexFingerPitch1LinkMass}"
@@ -85,5 +85,5 @@
     </xacro:revolute_joint>
   </xacro:macro>
-  <xacro:macro name="make_primary_finger_fixed" params="prefix reflect primary_finger_root_link">
+  <xacro:macro name="make_index_finger_fixed" params="prefix reflect index_finger_root_link">
     <xacro:box_link name="${IndexFingerPitch1LinkName}"
                     width="${PFJ1_Link_Width}" height="${PFJ1_Link_Height}" depth="${PFJ1_Link_Length}" mass="${IndexFingerPitch1LinkMass}"
@@ -131,12 +131,12 @@
                           origin_rpy="${IndexFingerPitch4FrameOrientation_Roll} ${IndexFingerPitch4FrameOrientation_Pitch} ${IndexFingerPitch4FrameOrientation_Yaw}"/>
   </xacro:macro>
-  <xacro:macro name="v1_right_primary_finger_actuators" params="prefix api">
+  <xacro:macro name="v1_right_index_finger_actuators" params="prefix api">
     <xacro:v1_actuator name="${RPFA_Actuator_Name}" api="${api}" />
   </xacro:macro>
-  <xacro:macro name="v1_left_primary_finger_actuators" params="prefix api">
+  <xacro:macro name="v1_left_index_finger_actuators" params="prefix api">
     <xacro:v1_actuator name="${LPFA_Actuator_Name}" api="${api}" />
   </xacro:macro>
-  <xacro:macro name="v1_right_primary_finger_transmissions" params="prefix">
-    <xacro:finger3_transmission tranName="${prefix}PrimaryFingerTransmission"
+  <xacro:macro name="v1_right_index_finger_transmissions" params="prefix">
+    <xacro:finger3_transmission tranName="${prefix}indexFingerTransmission"
                                 joint1="${IndexFingerPitch1JointName}"
                                 joint2="${IndexFingerPitch2JointName}"
@@ -144,6 +144,6 @@
                                 actuator="${RPFA_Actuator_Name}" />
   </xacro:macro>
-  <xacro:macro name="v1_left_primary_finger_transmissions" params="prefix">
-    <xacro:finger3_transmission tranName="${prefix}PrimaryFingerTransmission"
+  <xacro:macro name="v1_left_index_finger_transmissions" params="prefix">
+    <xacro:finger3_transmission tranName="${prefix}indexFingerTransmission"
                                 joint1="${IndexFingerPitch1JointName}"
                                 joint2="${IndexFingerPitch2JointName}"
@@ -151,40 +151,40 @@
                                 actuator="${LPFA_Actuator_Name}" />
   </xacro:macro>
-  <xacro:macro name="v1_right_primary_finger_transmissions_simple" params="prefix">
+  <xacro:macro name="v1_right_index_finger_transmissions_simple" params="prefix">
     <xacro:simple_transmission jointName="${IndexFingerPitch2JointName}" actuatorName="${RPFA_Actuator_Name}" reduction="1" offset="0"/>
   </xacro:macro>
-  <xacro:macro name="v1_left_primary_finger_transmissions_simple" params="prefix">
+  <xacro:macro name="v1_left_index_finger_transmissions_simple" params="prefix">
     <xacro:simple_transmission jointName="${IndexFingerPitch2JointName}" actuatorName="${LPFA_Actuator_Name}" reduction="1" offset="0"/>
   </xacro:macro>
-  <xacro:macro name="v1_right_primary_finger_modes" params="prefix">
+  <xacro:macro name="v1_right_index_finger_modes" params="prefix">
     <xacro:v1_modes jointName="${IndexFingerPitch1JointName}" actuatorName="${RPFA_Actuator_Name}" />
     <xacro:v1_modes jointName="${IndexFingerPitch2JointName}" actuatorName="${RPFA_Actuator_Name}" />
     <xacro:v1_modes jointName="${IndexFingerPitch3JointName}" actuatorName="${RPFA_Actuator_Name}" />
   </xacro:macro>
-  <xacro:macro name="v1_left_primary_finger_modes" params="prefix">
+  <xacro:macro name="v1_left_index_finger_modes" params="prefix">
     <xacro:v1_modes jointName="${IndexFingerPitch1JointName}" actuatorName="${LPFA_Actuator_Name}" />
     <xacro:v1_modes jointName="${IndexFingerPitch2JointName}" actuatorName="${LPFA_Actuator_Name}" />
     <xacro:v1_modes jointName="${IndexFingerPitch3JointName}" actuatorName="${LPFA_Actuator_Name}" />
   </xacro:macro>
-  <xacro:macro name="make_right_primary_finger_interface" params="api">
-    <xacro:v1_right_primary_finger_actuators prefix="Right" api="${api}" />
-    <xacro:v1_right_primary_finger_transmissions prefix="Right" />
-    <xacro:v1_right_primary_finger_modes prefix="Right" />
+  <xacro:macro name="make_right_index_finger_interface" params="api">
+    <xacro:v1_right_index_finger_actuators prefix="Right" api="${api}" />
+    <xacro:v1_right_index_finger_transmissions prefix="Right" />
+    <xacro:v1_right_index_finger_modes prefix="Right" />
   </xacro:macro>
-  <xacro:macro name="make_left_primary_finger_interface" params="api">
-    <xacro:v1_left_primary_finger_actuators prefix="Left" api="${api}" />
-    <xacro:v1_left_primary_finger_transmissions prefix="Left" />
-    <xacro:v1_left_primary_finger_modes prefix="Left" />
+  <xacro:macro name="make_left_index_finger_interface" params="api">
+    <xacro:v1_left_index_finger_actuators prefix="Left" api="${api}" />
+    <xacro:v1_left_index_finger_transmissions prefix="Left" />
+    <xacro:v1_left_index_finger_modes prefix="Left" />
   </xacro:macro>
   <!-- Simple interface -->
-  <xacro:macro name="make_right_primary_finger_interface_simple" params="api">
-    <xacro:v1_right_primary_finger_actuators prefix="Right" api="${api}" />
-    <xacro:v1_right_primary_finger_transmissions_simple prefix="Right" />
-    <xacro:v1_right_primary_finger_modes prefix="Right" />
+  <xacro:macro name="make_right_index_finger_interface_simple" params="api">
+    <xacro:v1_right_index_finger_actuators prefix="Right" api="${api}" />
+    <xacro:v1_right_index_finger_transmissions_simple prefix="Right" />
+    <xacro:v1_right_index_finger_modes prefix="Right" />
   </xacro:macro>
-  <xacro:macro name="make_left_primary_finger_interface_simple" params="api">
-    <xacro:v1_left_primary_finger_actuators prefix="Left" api="${api}" />
-    <xacro:v1_left_primary_finger_transmissions_simple prefix="Left" />
-    <xacro:v1_left_primary_finger_modes prefix="Left" />
+  <xacro:macro name="make_left_index_finger_interface_simple" params="api">
+    <xacro:v1_left_index_finger_actuators prefix="Left" api="${api}" />
+    <xacro:v1_left_index_finger_transmissions_simple prefix="Left" />
+    <xacro:v1_left_index_finger_modes prefix="Left" />
   </xacro:macro>
 </robot>

File: valkyrie_description/robots/valkyrie_A/xacro/index_finger/joint_limits.xacro (robot description, xacro)
@@ -1,4 +1,4 @@
 <?xml version="1.0" ?>
-<robot xmlns:xacro="http://www.ros.org/wiki/xacro" name="v1/primary_finger/joint_limits">
+<robot xmlns:xacro="http://www.ros.org/wiki/xacro" name="v1/index_finger/joint_limits">
   <xacro:property name="IndexFingerPitch1TorqueLimit" value="10" />
   <xacro:property name="IndexFingerPitch2TorqueLimit" value="10" />

File: valkyrie_description/robots/valkyrie_A/xacro/index_finger/joint_names.xacro (robot description, xacro)
@@ -1,4 +1,4 @@
 <?xml version="1.0" ?>
-<robot xmlns:xacro="http://www.ros.org/wiki/xacro" name="v1/primary_finger/mass_parameters">
+<robot xmlns:xacro="http://www.ros.org/wiki/xacro" name="v1/index_finger/mass_parameters">
   <xacro:property name="IndexFingerPitch1JointName" value="${prefix}PrimaryMPYaw" />
   <xacro:property name="IndexFingerPitch2JointName" value="${prefix}PrimaryMPExtensor" />

File: valkyrie_description/robots/valkyrie_A/xacro/index_finger/link_names.xacro (robot description, xacro)
@@ -1,5 +1,5 @@
 <?xml version="1.0" ?>
-<robot xmlns:xacro="http://www.ros.org/wiki/xacro" name="v1/primary_finger/dh_parameters">
-  <xacro:property name="IndexFingerPitch1ParentLinkName" value="${primary_finger_root_link}" />
+<robot xmlns:xacro="http://www.ros.org/wiki/xacro" name="v1/index_finger/dh_parameters">
+  <xacro:property name="IndexFingerPitch1ParentLinkName" value="${index_finger_root_link}" />
   <xacro:property name="IndexFingerPitch1LinkName" value="${prefix}IndexFingerPitch1Link" />
   <xacro:property name="IndexFingerPitch2LinkName" value="${prefix}IndexFingerPitch2Link" />

File: valkyrie_description/robots/valkyrie_A/xacro/index_finger/mass_parameters.xacro (robot description, xacro)
@@ -1,4 +1,4 @@
 <?xml version="1.0" ?>
-<robot xmlns:xacro="http://www.ros.org/wiki/xacro" name="v1/primary_finger/mass_parameters">
+<robot xmlns:xacro="http://www.ros.org/wiki/xacro" name="v1/index_finger/mass_parameters">
   <xacro:property name="IndexFingerPitch1LinkMass" value="0.006" />
   <xacro:property name="IndexFingerPitch2LinkMass" value="0.018" />

File: valkyrie_description/robots/valkyrie_A/xacro/thumb/frame_parameters.xacro (robot description, xacro)
@@ -1,25 +1,25 @@
 <?xml version="1.0" ?>
 <robot xmlns:xacro="http://www.ros.org/wiki/xacro" name="v1/thumb/dh_parameters">
-  <xacro:property name="ThumbRollFrameOrigin_X" value="0.00748367180673"/>
-  <xacro:property name="ThumbRollFrameOrigin_Y" value="-0.0324153432851"/>
-  <xacro:property name="ThumbRollFrameOrigin_Z" value="${reflect * 0.005182}"/>
-  <xacro:property name="ThumbRollFrameOrientation_Roll" value="0.0"/>
+  <xacro:property name="ThumbRollFrameOrigin_X" value="0.0049"/>
+  <xacro:property name="ThumbRollFrameOrigin_Y" value="${reflect * 0.0351}"/>
+  <xacro:property name="ThumbRollFrameOrigin_Z" value="0.0228"/>
+  <xacro:property name="ThumbRollFrameOrientation_Roll" value="${reflect * -0.3491}"/>
   <xacro:property name="ThumbRollFrameOrientation_Pitch" value="0.0"/>
   <xacro:property name="ThumbRollFrameOrientation_Yaw" value="0.0"/>
-  <xacro:property name="ThumbPitch1FrameOrigin_X" value="0.02286"/>
-  <xacro:property name="ThumbPitch1FrameOrigin_Y" value="0"/>
-  <xacro:property name="ThumbPitch1FrameOrigin_Z" value="${reflect * -0.025091}"/>
-  <xacro:property name="ThumbPitch1FrameOrientation_Roll" value="0.0"/>
+  <xacro:property name="ThumbPitch1FrameOrigin_X" value="0.0"/>
+  <xacro:property name="ThumbPitch1FrameOrigin_Y" value="0.0"/>
+  <xacro:property name="ThumbPitch1FrameOrigin_Z" value="0.0229"/>
+  <xacro:property name="ThumbPitch1FrameOrientation_Roll" value="${reflect * 0.3491}"/>
   <xacro:property name="ThumbPitch1FrameOrientation_Pitch" value="0.0"/>
   <xacro:property name="ThumbPitch1FrameOrientation_Yaw" value="0.0"/>
-  <xacro:property name="ThumbPitch2FrameOrigin_X" value="0.0381"/>
-  <xacro:property name="ThumbPitch2FrameOrigin_Y" value="0"/>
-  <xacro:property name="ThumbPitch2FrameOrigin_Z" value="0"/>
+  <xacro:property name="ThumbPitch2FrameOrigin_X" value="0.0"/>
+  <xacro:property name="ThumbPitch2FrameOrigin_Y" value="${reflect * 0.0066}"/>
+  <xacro:property name="ThumbPitch2FrameOrigin_Z" value="0.0375"/>
   <xacro:property name="ThumbPitch2FrameOrientation_Roll" value="0.0"/>
   <xacro:property name="ThumbPitch2FrameOrientation_Pitch" value="0.0"/>
   <xacro:property name="ThumbPitch2FrameOrientation_Yaw" value="0.0"/>
-  <xacro:property name="ThumbPitch3FrameOrigin_X" value="0.02794"/>
-  <xacro:property name="ThumbPitch3FrameOrigin_Y" value="0"/>
-  <xacro:property name="ThumbPitch3FrameOrigin_Z" value="0"/>
+  <xacro:property name="ThumbPitch3FrameOrigin_X" value="0.0"/>
+  <xacro:property name="ThumbPitch3FrameOrigin_Y" value="${reflect * 0.0049}"/>
+  <xacro:property name="ThumbPitch3FrameOrigin_Z" value="0.0275"/>
   <xacro:property name="ThumbPitch3FrameOrientation_Roll" value="0.0"/>
   <xacro:property name="ThumbPitch3FrameOrientation_Pitch" value="0.0"/>
