Commit message: Rename primary to index because I really don't like primary.

File: valkyrie_description/robots/valkyrie_A/xacro/utility/utility.xacro (robot description, xacro)
@@ -29,8 +29,8 @@
        </xacro:macro>
   -->
-  <!-- 	<xacro:macro name="make_primary_finger_interface" params="prefix channel">
-       <xacro:v1_primary_finger_actuators channel="${channel}" />
-       <xacro:v1_primary_finger_transmissions prefix="${prefix}" channel="${channel}" />
-       <xacro:v1_primary_finger_modes prefix="${prefix}" channel="${channel}" />
+  <!-- 	<xacro:macro name="make_index_finger_interface" params="prefix channel">
+       <xacro:v1_index_finger_actuators channel="${channel}" />
+       <xacro:v1_index_finger_transmissions prefix="${prefix}" channel="${channel}" />
+       <xacro:v1_index_finger_modes prefix="${prefix}" channel="${channel}" />
        </xacro:macro> -->
   <!-- 	<xacro:macro name="make_middle_finger_interface" params="prefix channel">

Commit message: Added in COP sensor and ATI sensor in the feet. Frames look good in rviz.

File: valkyrie_description/robots/valkyrie_A/xacro/V1_sim_base.xacro (robot description, xacro)
@@ -63,7 +63,8 @@
                             name5="${rightleg_name5}" type5="${leg_type5}"
                             name6="${rightleg_name6}" type6="${leg_type6}"/> -->
-    <!-- <xacro:v1_leg_sensors prefix="Right" reflect="1" /> -->
+    <xacro:v1_leg_sensors prefix="Right" reflect="-1" />
     <!-- <xacro:v1_hw_sensors prefix="Right" hermes_node="${rightleg_hermes}" atidaq_node="${rightleg_ati}" mpu6000_node="${rightleg_mpu2000}" cop_node="${rightleg_cop}"/> -->
     <xacro:make_leg prefix="Left" reflect="1" leg_root_link="${Pelvis_Link_Name}" />
+    <xacro:v1_leg_sensors prefix="Left" reflect="1" />
     <!-- <xacro:v1_leg_actuators name1="${leftleg_name1}" type1="${leg_type1}"
                             name2="${leftleg_name2}" type2="${leg_type2}"

File: valkyrie_description/robots/valkyrie_A/xacro/leg/leg.xacro (robot description, xacro)
@@ -9,4 +9,5 @@
   <xacro:include filename="$(find valkyrie_description)/robots/valkyrie_A/xacro/sensors/hokuyo.xacro"/>
   <xacro:include filename="$(find valkyrie_description)/robots/valkyrie_A/xacro/sensors/hw_sensors.xacro"/>
+  <xacro:include filename="$(find valkyrie_description)/robots/valkyrie_A/xacro/sensors/ati_force_torque.xacro"/>
   <xacro:property name="LJ1_Link_Width" value="0.149"/>
   <xacro:property name="LJ1_Link_Height" value="0.185"/>
@@ -208,30 +209,16 @@
   <!-- Sensors -->
   <xacro:macro name="v1_leg_sensors" params="prefix reflect">
-    <xacro:camboard_sensor sensorName="/v1/${prefix}LegCamBoard"
-                       parentLink="${KneePitchLinkName}"
-                       origin_xyz="0.344887 0.069118 ${reflect * -0.008500}"
-                       origin_rpy="-1.57 0 1.3"/>
-    <xacro:virtual_fixed_frame_offset name="/v1/${prefix}COP"
+    <xacro:virtual_fixed_frame_offset name="${prefix}COP"
                        parentLink="${AnkleRollLinkName}"
-                       origin_xyz="0.0845 0 0"
-                       origin_rpy="${1.57 + reflect * -1.57} ${reflect * -1.57} 0"/>
-    <xacro:virtual_fixed_frame_offset name="/v1/${prefix}Leg6Axis"
-                       parentLink="${AnkleRollLinkName}"
-                       origin_xyz="0.058547 0 ${reflect * 0.0215}"
-                       origin_rpy="0 0 0"/>
-    <xacro:virtual_fixed_frame_offset name="/v1/${prefix}LegHermes"
-                       parentLink="${AnkleRollLinkName}"
-                       origin_xyz="0.0845 0 0"
-                       origin_rpy="${1.57 + reflect * -1.57} ${reflect * -1.57} 0"/>
-    <xacro:virtual_fixed_frame_offset name="/v1/${prefix}MPU6000"
-                       parentLink="${AnkleRollLinkName}"
-                       origin_xyz="0.0471 ${reflect * 0.00722} ${reflect * 0.0843}"
-                       origin_rpy="0 ${reflect * 1.57 - 0.13} ${1.57 + reflect * 1.57}"/>
-  </xacro:macro>
-  <xacro:macro name="v1_hw_sensors" params="prefix cop_node hermes_node atidaq_node mpu6000_node">
-    <xacro:cop_sensor sensorName="/v1/${prefix}ValkyrieCOP" nodePath="${cop_node}" type="ValkyrieCOPSensor"/>
-<!--     <xacro:cop_sensor sensorName="/v1/${prefix}LegHermes" nodePath="${hermes_node}" type="COPSensorHermes"/>
+                       origin_xyz="0.0189 0.0 -0.0783"
+                       origin_rpy="0.0 0.13 0.0"/>
+    <xacro:ati_force_torque_sensor sensorName="${prefix}Leg6Axis"
+                        parentLink="${AnkleRollLinkName}"
+                        origin_xyz="0.022 0.0 -0.059"
+                        origin_rpy="3.14 0.0 -1.047"/>
+  </xacro:macro>
+  <xacro:macro name="v1_hw_sensors" params="prefix cop_node hermes_node atidaq_node">
+    <xacro:cop_sensor sensorName="${prefix}ValkyrieCOP" nodePath="${cop_node}" type="ValkyrieCOPSensor"/>
     <xacro:cop_sensor sensorName="/v1/${prefix}Leg6Axis" nodePath="${atidaq_node}" type="COPSensorAti"/> -->
-    <xacro:imu_sensor sensorName="/v1/${prefix}MPU6000" nodePath="${mpu6000_node}" type="IMUSensorMPU6000"/>
   </xacro:macro>
   <xacro:macro name="v1_leg_actuators" params="name1 type1 name2 type2 name3 type3 name4 type4 name5 type5 name6 type6">

File: valkyrie_description/robots/valkyrie_A/xacro/sensors/ati_force_torque.xacro (robot description, xacro)
@@ -1,5 +1,5 @@
 <?xml version="1.0" ?>
-<robot xmlns:xacro="http://www.ros.org/wiki/xacro" name="v1/asus">
-  <xacro:macro name="ensenso_sensor" params="sensorName parentLink origin_xyz origin_rpy">
+<robot xmlns:xacro="http://www.ros.org/wiki/xacro" name="ati_force_torque_sensor">
+  <xacro:macro name="ati_force_torque_sensor" params="sensorName parentLink origin_xyz origin_rpy">
     <xacro:massless_virtual_link name="${sensorName}_Frame"
                     origin_rpy="0 0 0"

Commit message: Deleted a bunch of unused stuff. Removed the utility directory and utility.xacro. The info in there doesn't belong in the urdf.

File: valkyrie_description/robots/valkyrie_A/xacro/V1_sim_base.xacro (robot description, xacro)
@@ -4,5 +4,4 @@
     <xacro:include filename="$(find common_xacro)/xacro/materials.xacro" />
     <xacro:include filename="$(find valkyrie_description)/robots/valkyrie_A/xacro/common/common_bodies.xacro" />
-    <xacro:include filename="$(find valkyrie_description)/robots/valkyrie_A/xacro/utility/utility.xacro" />
     <xacro:include filename="$(find valkyrie_description)/robots/valkyrie_A/xacro/common/actuator_names.xacro" />
     <!-- ===== GAZEBO PLUGINS ===== -->

File: valkyrie_description/robots/valkyrie_A/xacro/head/head.xacro (robot description, xacro)
@@ -6,7 +6,4 @@
   <xacro:include filename="$(find valkyrie_description)/robots/valkyrie_A/xacro/head/frame_parameters.xacro"/>
   <xacro:include filename="$(find valkyrie_description)/robots/valkyrie_A/xacro/head/mass_parameters.xacro"/>
-  <xacro:include filename="$(find valkyrie_description)/robots/valkyrie_A/xacro/sensors/camboard.xacro"/>
-  <xacro:include filename="$(find valkyrie_description)/robots/valkyrie_A/xacro/sensors/flea.xacro"/>
-  <xacro:include filename="$(find valkyrie_description)/robots/valkyrie_A/xacro/sensors/ibeo.xacro"/>
   <xacro:include filename="$(find valkyrie_description)/robots/valkyrie_A/xacro/sensors/ensenso.xacro"/>
   <xacro:include filename="$(find valkyrie_description)/robots/valkyrie_A/xacro/sensors/webcam.xacro"/>

File: valkyrie_description/robots/valkyrie_A/xacro/leg/leg.xacro (robot description, xacro)
@@ -6,7 +6,4 @@
   <xacro:include filename="$(find valkyrie_description)/robots/valkyrie_A/xacro/leg/frame_parameters.xacro"/>
   <xacro:include filename="$(find valkyrie_description)/robots/valkyrie_A/xacro/leg/mass_parameters.xacro"/>
-  <xacro:include filename="$(find valkyrie_description)/robots/valkyrie_A/xacro/sensors/camboard.xacro"/>
-  <xacro:include filename="$(find valkyrie_description)/robots/valkyrie_A/xacro/sensors/hokuyo.xacro"/>
-  <xacro:include filename="$(find valkyrie_description)/robots/valkyrie_A/xacro/sensors/hw_sensors.xacro"/>
   <xacro:include filename="$(find valkyrie_description)/robots/valkyrie_A/xacro/sensors/ati_force_torque.xacro"/>
   <xacro:property name="LJ1_Link_Width" value="0.149"/>
@@ -213,12 +210,8 @@
                        origin_xyz="0.0189 0.0 -0.0783"
                        origin_rpy="0.0 0.13 0.0"/>
-    <xacro:ati_force_torque_sensor sensorName="${prefix}Leg6Axis"
+    <xacro:ati_force_torque_sensor sensorName="${prefix}LegSixAxis"
                         parentLink="${AnkleRollLinkName}"
                         origin_xyz="0.022 0.0 -0.059"
                         origin_rpy="3.14 0.0 -1.047"/>
-  </xacro:macro>
-  <xacro:macro name="v1_hw_sensors" params="prefix cop_node hermes_node atidaq_node">
-    <xacro:cop_sensor sensorName="${prefix}ValkyrieCOP" nodePath="${cop_node}" type="ValkyrieCOPSensor"/>
-    <xacro:cop_sensor sensorName="/v1/${prefix}Leg6Axis" nodePath="${atidaq_node}" type="COPSensorAti"/> -->
   </xacro:macro>
   <xacro:macro name="v1_leg_actuators" params="name1 type1 name2 type2 name3 type3 name4 type4 name5 type5 name6 type6">

File: valkyrie_description/robots/valkyrie_A/xacro/leg/link_names.xacro (robot description, xacro)
@@ -6,6 +6,4 @@
   <xacro:property name="HipPitchLinkName" value="${prefix}HipPitchLink" />
   <xacro:property name="KneePitchLinkName" value="${prefix}KneePitchLink" />
-  <xacro:property name="LJ4_Distal_Link_Cylinder1" value="${prefix}MedialAnkleActuator" />
-  <xacro:property name="LJ4_Distal_Link_Cylinder2" value="${prefix}LateralAnkleActuator" />
   <xacro:property name="AnklePitchLinkName" value="${prefix}AnklePitchLink" />
   <xacro:property name="AnkleRollLinkName" value="${prefix}Foot" />
