Commit message: Removed some unused files.

File: valkyrie_description/robots/valkyrie_A/xacro/common/actuator_names.xacro (robot description, xacro)
@@ -26,8 +26,6 @@
     <xacro:property name="rightleg_name5" value="/right_leg/j5"/>
     <xacro:property name="rightleg_name6" value="/right_leg/j6"/>
-    <xacro:property name="rightleg_hermes" value="/right_leg/hermes"/>
     <xacro:property name="rightleg_ati" value="/right_leg/j6"/>
     <xacro:property name="rightleg_cop" value="/right_leg/cop"/>
-    <xacro:property name="rightleg_mpu2000" value="/right_leg/hermes"/>
     <xacro:property name="leftleg_name1" value="/pelvis/lj1"/>
     <xacro:property name="leftleg_name2" value="/left_leg/j2"/>
@@ -36,7 +34,5 @@
     <xacro:property name="leftleg_name5" value="/left_leg/j5"/>
     <xacro:property name="leftleg_name6" value="/left_leg/j6"/>
-    <xacro:property name="leftleg_hermes" value="/left_leg/hermes"/>
     <xacro:property name="leftleg_ati" value="/left_leg/j6"/>
     <xacro:property name="leftleg_cop" value="/left_leg/cop"/>
-    <xacro:property name="leftleg_mpu2000" value="/left_leg/hermes"/>
 </robot>

File: valkyrie_description/robots/valkyrie_A/xacro/waist/waist.xacro (robot description, xacro)
@@ -7,5 +7,4 @@
   <xacro:include filename="$(find valkyrie_description)/robots/valkyrie_A/xacro/waist/mass_parameters.xacro"/>
   <xacro:include filename="$(find valkyrie_description)/robots/valkyrie_A/xacro/sensors/microstrain.xacro"/>
-  <xacro:include filename="$(find valkyrie_description)/robots/valkyrie_A/xacro/sensors/virtual_sensor.xacro"/>
   <xacro:include filename="$(find valkyrie_description)/robots/valkyrie_A/xacro/sensors/flea.xacro"/>
   <xacro:property name="Trunk_Width" value="0.47605775481079287692"/>
