Commit message: Changed name of neck link name property.

File: valkyrie_description/robots/valkyrie_A/xacro/head/head.xacro (robot description, xacro)
@@ -35,5 +35,5 @@
     <!-- NJ1 -->
     <xacro:revolute_joint_ex jointName="${LowerNeckPitchJointName}"
-                          parent="${LowerNeckPitchParentLink}" child="${LowerNeckPitchLinkName}"
+                          parent="${LowerNeckPitchParentLinkName}" child="${LowerNeckPitchLinkName}"
                           origin_xyz="${LowerNeckPitchFrameOrigin_X} ${LowerNeckPitchFrameOrigin_Y} ${LowerNeckPitchFrameOrigin_Z}"
                           origin_rpy="${LowerNeckPitchFrameOrientation_Roll} ${LowerNeckPitchFrameOrientation_Roll} ${LowerNeckPitchFrameOrientation_Yaw}"
@@ -79,5 +79,5 @@
     <!-- NJ1 -->
     <xacro:fixed_joint jointName="${LowerNeckPitchJointName}"
-                          parent="${LowerNeckPitchParentLink}" child="${LowerNeckPitchLinkName}"
+                          parent="${LowerNeckPitchParentLinkName}" child="${LowerNeckPitchLinkName}"
                           origin_xyz="${LowerNeckPitchFrameOrigin_X} ${LowerNeckPitchFrameOrigin_Y} ${LowerNeckPitchFrameOrigin_Z}"
                           origin_rpy="${LowerNeckPitchFrameOrientation_Roll} ${LowerNeckPitchFrameOrientation_Roll} ${LowerNeckPitchFrameOrientation_Yaw}">

File: valkyrie_description/robots/valkyrie_A/xacro/head/link_names.xacro (robot description, xacro)
@@ -1,5 +1,5 @@
 <?xml version="1.0" ?>
 <robot xmlns:xacro="http://www.ros.org/wiki/xacro" name="v1/head/link_names">
-  <xacro:property name="LowerNeckPitchParentLink" value="${head_root_link}" />
+  <xacro:property name="LowerNeckPitchParentLinkName" value="${head_root_link}" />
   <xacro:property name="LowerNeckPitchLinkName" value="LowerNeckPitchLink" />
   <xacro:property name="NeckYawLinkName" value="NeckYawLink" />

Commit message: Updated COM values for head.

File: valkyrie_description/robots/valkyrie_A/xacro/head/head.xacro (robot description, xacro)
@@ -17,14 +17,14 @@
     <!-- LINKS -->
     <xacro:virtual_link_with_visual name="${LowerNeckPitchLinkName}"
-                                    origin_xyz="0 0 0"
+                                    origin_xyz="${LowerNeckPitchLinkComPosition}"
                                     origin_rpy="0 0 0"
                                     mesh_filename="${mesh_root}/neckj1.stl"/>
     <xacro:virtual_link_with_visual name="${NeckYawLinkName}"
-                                    origin_xyz="0 0 0"
+                                    origin_xyz="${NeckYawLinkComPosition}"
                                     origin_rpy="0 0 0"
                                     mesh_filename="${mesh_root}/neckj2.stl"/>
     <xacro:sphere_link name="${UpperNeckPitchLinkName}"
                        radius="${NJ3_Link_Radius}" mass="${UpperNeckPitchLinkMass}"
-                       origin_xyz="-0.08380066 0.01114801 -0.00038569" origin_rpy="0 0 0"
+                       origin_xyz="${UpperNeckPitchLinkComPosition}" origin_rpy="0 0 0"
                        visual_mesh="${mesh_root}/head.stl"
                        material="White"

File: valkyrie_description/robots/valkyrie_A/xacro/head/mass_parameters.xacro (robot description, xacro)
@@ -2,5 +2,8 @@
 <robot xmlns:xacro="http://www.ros.org/wiki/xacro" name="v1/head/mass_parameters">
   <xacro:property name="LowerNeckPitchLinkMass" value="0.471" />
+  <xacro:property name="LowerNeckPitchLinkComPosition" value="0 0 0" />
   <xacro:property name="NeckYawLinkMass" value="1.4" />
+  <xacro:property name="NeckYawLinkComPosition" value="0 0 0" />
   <xacro:property name="UpperNeckPitchLinkMass" value="4.06" />
+  <xacro:property name="UpperNeckPitchLinkComPosition" value="0.091874 0.001012 -0.005277" />
 </robot>
