Commit message: Have hokuyo in meshes now. Fixed offset bug in head mesh.

File: common_xacro/xacro/generic_models.xacro (robot description, xacro)
@@ -356,4 +356,12 @@
     </gazebo>
   </xacro:macro>
+  <xacro:macro name="continuous_joint" params="jointName parent child origin_xyz origin_rpy axis">
+    <joint name="${jointName}" type="continuous">
+      <origin rpy="${origin_rpy}" xyz="${origin_xyz}"/>
+      <axis xyz="${axis}"/>
+      <parent link="${parent}"/>
+      <child link="${child}"/>
+    </joint>
+  </xacro:macro>
   <xacro:macro name="revolute_joint_damped" params="jointName parent child origin_xyz origin_rpy axis damping friction *limits">
     <joint name="${jointName}" type="revolute">

File: robots/valkyrie_A/xacro/head/frame_parameters.xacro (robot description, xacro)
@@ -19,3 +19,9 @@
   <xacro:property name="UpperNeckPitchFrameOrientation_Pitch" value="0.0"/>
   <xacro:property name="UpperNeckPitchFrameOrientation_Yaw" value="0.0"/>
+  <xacro:property name="HokuyoFrameOrigin_X" value="0.001654"/>
+  <xacro:property name="HokuyoFrameOrigin_Y" value="0.0"/>
+  <xacro:property name="HokuyoFrameOrigin_Z" value="0.012564"/>
+  <xacro:property name="HokuyoFrameOrientation_Roll" value="0.0"/>
+  <xacro:property name="HokuyoFrameOrientation_Pitch" value="0.1309"/>
+  <xacro:property name="HokuyoFrameOrientation_Yaw" value="0.0"/>
 </robot>

File: robots/valkyrie_A/xacro/head/head.xacro (robot description, xacro)
@@ -6,6 +6,5 @@
   <xacro:include filename="$(find val_description)/robots/valkyrie_A/xacro/head/frame_parameters.xacro"/>
   <xacro:include filename="$(find val_description)/robots/valkyrie_A/xacro/head/mass_parameters.xacro"/>
-  <xacro:include filename="$(find val_description)/robots/valkyrie_A/xacro/sensors/ensenso.xacro"/>
-  <xacro:include filename="$(find val_description)/robots/valkyrie_A/xacro/sensors/webcam.xacro"/>
+  <xacro:include filename="$(find val_description)/robots/valkyrie_A/xacro/sensors/multisense_sl.xacro"/>
   <xacro:property name="NJ3_Link_Radius" value="0.139"/>
   <xacro:macro name="include_head" params="lower_neck_pitch_root_link">
@@ -23,5 +22,5 @@
                        radius="${NJ3_Link_Radius}" mass="${UpperNeckPitchLinkMass}"
                        origin_xyz="${UpperNeckPitchLinkComPosition}" origin_rpy="0 0 0"
-                       visual_mesh="${mesh_root}/head.stl"
+                       visual_mesh="${mesh_root}/head_multisense_no_visor.stl"
                        material="White"
                        collision_mesh="${mesh_root}/head.stl"/>
@@ -55,18 +54,19 @@
   </xacro:macro>
   <xacro:macro name="v1_head_sensors">
-    <xacro:ensenso_sensor sensorName="Ensenso"
-                        parentLink="${UpperNeckPitchLinkName}"
-                        origin_xyz="0.1781 0.0 0.062"
-                        origin_rpy="1.57 -2.88 0"/>
-    <xacro:microstrain_sensor sensorName="HeadIMU"
+<!-- <xacro:microstrain_sensor sensorName="HeadIMU"
                               parentLink="${UpperNeckPitchLinkName}"
                               origin_xyz="0.098 0.0 0.052"
                               origin_rpy="-1.57 1.57 0.0" />
-    <xacro:webcam_camera sensorName="HeadWebcam"
-                        parentLink="${UpperNeckPitchLinkName}"
-                        origin_xyz="0.1801 0.0 0.102"
-                        origin_rpy="1.57 -2.88 0.0"
-                        imageFormat="R8G8B8"
-                        frameRate="60"/>
+-->
+    <xacro:multisense_sl parentLink="${UpperNeckPitchLinkName}"
+                  joint_axis="1 0 0"
+                  joint_origin_xyz="${HokuyoFrameOrigin_X} ${HokuyoFrameOrigin_Y} ${HokuyoFrameOrigin_Z}"
+                  joint_origin_rpy="${HokuyoFrameOrientation_Roll} ${HokuyoFrameOrientation_Pitch} ${HokuyoFrameOrientation_Yaw}"
+                  com_origin_xyz="${HokuyoLinkComPosition}"
+                  com_origin_rpy="0 0 0"
+                  mass="${HokuyoLinkMass}"
+                  visual_mesh="${mesh_root}/multisense_hokuyo.stl"
+                  material="White"
+                  collision_mesh="${mesh_root}/multisense_hokuyo.stl" />
   </xacro:macro>
   <xacro:macro name="v1_head_actuators" params="name1 type1 name2 type2 name3 type3">

File: robots/valkyrie_A/xacro/head/mass_parameters.xacro (robot description, xacro)
@@ -7,3 +7,5 @@
   <xacro:property name="UpperNeckPitchLinkMass" value="4.06" />
   <xacro:property name="UpperNeckPitchLinkComPosition" value="0.091874 0.001012 -0.005277" />
+  <xacro:property name="HokuyoLinkMass" value="0.057664"/>
+  <xacro:property name="HokuyoLinkComPosition" value="0.14793 0.0 0.01"/>
 </robot>
