Commit message: fix new neck for now

File: robots/valkyrie_A/xacro/head/joint_limits.xacro (robot description, xacro)
@@ -4,8 +4,8 @@
   <xacro:property name="NeckYawTorqueLimit" value="26" />
   <xacro:property name="UpperNeckPitchTorqueLimit" value="26" />
-  <xacro:property name="LowerNeckPitchPositionLimit_Lower" value="-1.57" />
+  <xacro:property name="LowerNeckPitchPositionLimit_Lower" value="0" />
   <xacro:property name="NeckYawPositionLimit_Lower" value="-1.57" />
   <xacro:property name="UpperNeckPitchPositionLimit_Lower" value="-0.087" />
-  <xacro:property name="LowerNeckPitchPositionLimit_Upper" value="0" />
+  <xacro:property name="LowerNeckPitchPositionLimit_Upper" value="1.57" />
   <xacro:property name="NeckYawPositionLimit_Upper" value="1.57" />
   <xacro:property name="UpperNeckPitchPositionLimit_Upper" value="0.785" />
