Commit message: Added gazebo tags to microstrain sensor and to multisense hokuyo.

File: robots/valkyrie_A/xacro/head/head.xacro (robot description, xacro)
@@ -54,9 +54,4 @@
   </xacro:macro>
   <xacro:macro name="v1_head_sensors">
-<!-- <xacro:microstrain_sensor sensorName="HeadIMU"
-                              parentLink="${UpperNeckPitchLinkName}"
-                              origin_xyz="0.098 0.0 0.052"
-                              origin_rpy="-1.57 1.57 0.0" />
--->
     <xacro:multisense_sl parentLink="${UpperNeckPitchLinkName}"
                   joint_axis="1 0 0"

File: robots/valkyrie_A/xacro/sensors/ati_force_torque.xacro (robot description, xacro)
@@ -9,8 +9,10 @@
                        origin_rpy="${origin_rpy}"
                        origin_xyz="${origin_xyz}"/>
-    <sensor name="${sensorName}" type="force_torque">
-      <parent link="${parentLink}"/>
-      <origin rpy="${origin_rpy}" xyz="${origin_xyz}"/>
-  	</sensor>
+    <gazebo reference="${sensorName}_Frame">
+      <sensor name="${sensorName}" type="force_torque">
+        <parent link="${parentLink}"/>
+        <pose>${origin_xyz} ${origin_rpy} </pose>
+    	</sensor>
+    </gazebo>
   </xacro:macro>
 </robot>

File: robots/valkyrie_A/xacro/sensors/microstrain.xacro (robot description, xacro)
@@ -13,25 +13,27 @@
                        origin_rpy="${origin_rpy}"
                        origin_xyz="${origin_xyz}"/>
-    <sensor name="${sensorName}" type="imu">
-      <parent link="${parentLink}"/>
-      <origin rpy="${origin_rpy}" xyz="${origin_xyz}"/>
-      <imu>
-         <noise>
-             <type>gaussian</type>
-             <rate>
-                 <mean>0</mean>
-                 <stddev>0.0002</stddev>
-                 <bias_mean>7.5e-06</bias_mean>
-                 <bias_stddev>8e-07</bias_stddev>
-             </rate>
-             <accel>
-                 <mean>0</mean>
-                 <stddev>0.017</stddev>
-                 <bias_mean>0.1</bias_mean>
-                 <bias_stddev>0.001</bias_stddev>
-             </accel>
-         </noise>
-      </imu>
-      </sensor>
+    <gazebo reference="${sensorName}_Frame">
+      <sensor name="${sensorName}" type="imu">
+        <parent link="${parentLink}"/>
+        <pose>${origin_xyz} ${origin_rpy} </pose>
+        <imu>
+           <noise>
+               <type>gaussian</type>
+               <rate>
+                   <mean>0</mean>
+                   <stddev>0.0002</stddev>
+                   <bias_mean>7.5e-06</bias_mean>
+                   <bias_stddev>8e-07</bias_stddev>
+               </rate>
+               <accel>
+                   <mean>0</mean>
+                   <stddev>0.017</stddev>
+                   <bias_mean>0.1</bias_mean>
+                   <bias_stddev>0.001</bias_stddev>
+               </accel>
+           </noise>
+        </imu>
+        </sensor>
+    </gazebo>
   </xacro:macro>
 </robot>

File: robots/valkyrie_A/xacro/sensors/multisense_sl.xacro (robot description, xacro)
@@ -8,5 +8,5 @@
                           origin_rpy="${joint_origin_rpy}"
                           axis="${joint_axis}"/>
-		<xacro:standard_link name="hokuyo_link"
+		  <xacro:standard_link name="hokuyo_link"
 		    	  mass="${mass}" origin_xyz="${com_origin_xyz}" origin_rpy="${com_origin_rpy}" ixx="3.7174E-05" ixy="4.9927E-08" ixz="1.1015E-05" iyy=".2412E-05" iyz="-9.8165E-09" izz="4.167E-05"
 		    	  visual_mesh="${visual_mesh}"
@@ -14,19 +14,47 @@
 		    	  collision_mesh="${collision_mesh}"
 		    	  />
+      <gazebo reference="hokuyo_link">
+        <sensor type="ray" name="head_hokuyo_sensor">
+          <parent>hokuyo_link</parent>
+          <pose>0 0 0 0 0 0</pose>
+          <visualize>false</visualize>
+          <update_rate>40</update_rate>
+          <ray>
+            <scan>
+              <horizontal>
+                <samples>720</samples>
+                <resolution>1</resolution>
+                <min_angle>-1.570796</min_angle>
+                <max_angle>1.570796</max_angle>
+              </horizontal>
+            </scan>
+            <range>
+              <min>0.10</min>
+              <max>30.0</max>
+              <resolution>0.01</resolution>
+            </range>
+            <noise>
+              <type>gaussian</type>
+              <mean>0.0</mean>
+              <stddev>0.01</stddev>
+            </noise>
+          </ray>
+        </sensor>
+      </gazebo>
 	    <xacro:massless_virtual_link name="head_hokuyo_frame_offset"
                     origin_rpy="0 0 0"
                     origin_xyz="0 0 0"/>
-		<xacro:fixed_joint jointName="head_hokuyo_frame_joint"
+		  <xacro:fixed_joint jointName="head_hokuyo_frame_joint"
 	           parent="hokuyo_link" child="head_hokuyo_frame_offset"
 	           origin_rpy="3.14 0.0 0.0"
 	           origin_xyz="0.16018 0.0 -0.015"/>
-        <xacro:massless_virtual_link name="left_camera_frame_offset"
+      <xacro:massless_virtual_link name="left_camera_frame_offset"
                     origin_rpy="0 0 0"
                     origin_xyz="0 0 0"/>
-        <xacro:fixed_joint jointName="left_camera_frame_joint"
+      <xacro:fixed_joint jointName="left_camera_frame_joint"
          parent="${parentLink}" child="left_camera_frame_offset"
          origin_rpy="-3.14 0.1309 0.0"
        	 origin_xyz="0.18335 0.035 0.0774"/>
-       	<xacro:massless_virtual_link name="right_camera_frame_offset"
+     	<xacro:massless_virtual_link name="right_camera_frame_offset"
                     origin_rpy="0 0 0"
                     origin_xyz="0 0 0"/>

Commit message: Fixed head inertia.

File: robots/valkyrie_A/xacro/head/head.xacro (robot description, xacro)
@@ -19,7 +19,10 @@
                                     origin_rpy="0 0 0"
                                     mesh_filename="${mesh_root}/head/neckj2.stl"/>
-    <xacro:sphere_link name="${UpperNeckPitchLinkName}"
-                       radius="${NJ3_Link_Radius}" mass="${UpperNeckPitchLinkMass}"
-                       origin_xyz="${UpperNeckPitchLinkComPosition}" origin_rpy="0 0 0"
+    <xacro:standard_link name="${UpperNeckPitchLinkName}"
+                       mass="${UpperNeckPitchLinkMass}"
+                       origin_xyz="${UpperNeckPitchLinkComPosition}"
+                       ixx="${UpperNeckPitchLinkInertia_IXX}" ixy="${UpperNeckPitchLinkInertia_IXY}" ixz="${UpperNeckPitchLinkInertia_IXZ}"
+                       iyy="${UpperNeckPitchLinkInertia_IYY}" iyz="${UpperNeckPitchLinkInertia_IYZ}" izz="${UpperNeckPitchLinkInertia_IZZ}"
+                       origin_rpy="0 0 0"
                        visual_mesh="${mesh_root}/head/head_multisense_no_visor.stl"
                        material="White"
@@ -54,9 +57,4 @@
   </xacro:macro>
   <xacro:macro name="v1_head_sensors">
-<!-- <xacro:microstrain_sensor sensorName="HeadIMU"
-                              parentLink="${UpperNeckPitchLinkName}"
-                              origin_xyz="0.098 0.0 0.052"
-                              origin_rpy="-1.57 1.57 0.0" />
--->
     <xacro:multisense_sl parentLink="${UpperNeckPitchLinkName}"
                   joint_axis="1 0 0"

File: robots/valkyrie_A/xacro/head/mass_parameters.xacro (robot description, xacro)
@@ -7,4 +7,10 @@
   <xacro:property name="UpperNeckPitchLinkMass" value="4.59" />
   <xacro:property name="UpperNeckPitchLinkComPosition" value="0.091874 0.001012 -0.005277" />
+  <xacro:property name="UpperNeckPitchLinkInertia_IXX" value="0.041442523" />
+  <xacro:property name="UpperNeckPitchLinkInertia_IXY" value="-0.000055137" />
+  <xacro:property name="UpperNeckPitchLinkInertia_IXZ" value="0.000287605" />
+  <xacro:property name="UpperNeckPitchLinkInertia_IYY" value="0.044208496" />
+  <xacro:property name="UpperNeckPitchLinkInertia_IYZ" value="0.000245121" />
+  <xacro:property name="UpperNeckPitchLinkInertia_IZZ" value="0.041961853" />
   <xacro:property name="HokuyoLinkMass" value="0.057664"/>
   <xacro:property name="HokuyoLinkComPosition" value="0.14793 0.0 0.01"/>

Commit message: Added in xacro file for generating shared memory actuator names. IHMC needs this until the hardware API is ready.

File: robots/valkyrie_A/xacro/head/head.xacro (robot description, xacro)
@@ -65,5 +65,5 @@
                   collision_mesh="${mesh_root}/head/multisense_hokuyo.dae" />
   </xacro:macro>
-  <xacro:macro name="v1_head_actuators" params="name1 type1 name2 type2 name3 type3">
+  <xacro:macro name="neck_actuators" params="name1 type1 name2 type2 name3 type3">
     <actuator name="${name1}" type="${type1}"/>
     <actuator name="${name2}" type="${type2}"/>

File: robots/valkyrie_A/xacro/thumb/thumb.xacro (robot description, xacro)
@@ -139,10 +139,10 @@
                           origin_rpy="${ThumbPitch3FrameOrientation_Roll} ${ThumbPitch3FrameOrientation_Pitch} ${ThumbPitch3FrameOrientation_Yaw}"/>
   </xacro:macro>
-  <xacro:macro name="v1_right_thumb_actuators" params="prefix api">
+  <xacro:macro name="right_thumb_actuators" params="prefix api">
     <xacro:v1_actuator name="${RTA1_Actuator_Name}" api="${api}" />
     <xacro:v1_actuator name="${RTA2_Actuator_Name}" api="${api}" />
     <xacro:v1_actuator name="${RTA3_Actuator_Name}" api="${api}" />
   </xacro:macro>
-  <xacro:macro name="v1_left_thumb_actuators" params="prefix api">
+  <xacro:macro name="left_thumb_actuators" params="prefix api">
     <xacro:v1_actuator name="${LTA1_Actuator_Name}" api="${api}" />
     <xacro:v1_actuator name="${LTA2_Actuator_Name}" api="${api}" />
