Commit message: Updated head mass.

File: robots/valkyrie_A/xacro/head/mass_parameters.xacro (robot description, xacro)
@@ -5,5 +5,5 @@
   <xacro:property name="NeckYawLinkMass" value="1.4" />
   <xacro:property name="NeckYawLinkComPosition" value="0 0 0" />
-  <xacro:property name="UpperNeckPitchLinkMass" value="4.06" />
+  <xacro:property name="UpperNeckPitchLinkMass" value="4.59" />
   <xacro:property name="UpperNeckPitchLinkComPosition" value="0.091874 0.001012 -0.005277" />
   <xacro:property name="HokuyoLinkMass" value="0.057664"/>

Commit message: Renamed a xml tag and updated lower neck pitch link mass.

File: robots/valkyrie_A/xacro/head/mass_parameters.xacro (robot description, xacro)
@@ -1,5 +1,5 @@
 <?xml version="1.0" ?>
 <robot xmlns:xacro="http://www.ros.org/wiki/xacro" name="v1/head/mass_parameters">
-  <xacro:property name="LowerNeckPitchLinkMass" value="0.471" />
+  <xacro:property name="LowerNeckPitchLinkMass" value="1.05" />
   <xacro:property name="LowerNeckPitchLinkComPosition" value="0 0 0" />
   <xacro:property name="NeckYawLinkMass" value="1.4" />

File: robots/valkyrie_A/xacro/leg/mass_parameters.xacro (robot description, xacro)
@@ -1,4 +1,4 @@
 <?xml version="1.0" ?>
-<robot xmlns:xacro="http://www.ros.org/wiki/xacro" name="v1/leg/mass_parameters">
+<robot xmlns:xacro="http://www.ros.org/wiki/xacro" name="leg_mass_parameters">
   <xacro:property name="HipYawLinkMass" value="2.39" />
   <xacro:property name="HipYawLinkComPosition" value="0.02176 ${reflect*-0.00131} 0.03867" />

Commit message: Updated head mass, com location and inertia.

File: robots/valkyrie_A/xacro/head/mass_parameters.xacro (robot description, xacro)
@@ -18,11 +18,11 @@
   <xacro:property name="NeckYawLinkInertia_IZZ" value="0.001766459" />
   <xacro:property name="UpperNeckPitchLinkMass" value="4.59" />
-  <xacro:property name="UpperNeckPitchLinkComPosition" value="0.091874 0.001012 -0.005277" />
-  <xacro:property name="UpperNeckPitchLinkInertia_IXX" value="0.041442523" />
-  <xacro:property name="UpperNeckPitchLinkInertia_IXY" value="-0.000055137" />
-  <xacro:property name="UpperNeckPitchLinkInertia_IXZ" value="0.000287605" />
-  <xacro:property name="UpperNeckPitchLinkInertia_IYY" value="0.044208496" />
-  <xacro:property name="UpperNeckPitchLinkInertia_IYZ" value="0.000245121" />
-  <xacro:property name="UpperNeckPitchLinkInertia_IZZ" value="0.041961853" />
+  <xacro:property name="UpperNeckPitchLinkComPosition" value="0.100912 0.005783 0.034787" />
+  <xacro:property name="UpperNeckPitchLinkInertia_IXX" value="0.039847525" />
+  <xacro:property name="UpperNeckPitchLinkInertia_IXY" value="-0.000470418" />
+  <xacro:property name="UpperNeckPitchLinkInertia_IXZ" value="-0.002829842" />
+  <xacro:property name="UpperNeckPitchLinkInertia_IYY" value="0.041418564" />
+  <xacro:property name="UpperNeckPitchLinkInertia_IYZ" value="-0.000782564" />
+  <xacro:property name="UpperNeckPitchLinkInertia_IZZ" value="0.036841236" />
   <xacro:property name="HokuyoLinkMass" value="0.057664"/>
   <xacro:property name="HokuyoLinkComPosition" value="0.14793 0.0 0.01"/>

Commit message: Updated neck masses based on neckj3 mass and mass of entire head+neck assembly.

File: robots/valkyrie_A/xacro/head/mass_parameters.xacro (robot description, xacro)
@@ -3,18 +3,18 @@
   <xacro:property name="LowerNeckPitchLinkMass" value="1.05" />
   <xacro:property name="LowerNeckPitchLinkComPosition" value="-0.020000 0.000000  0.040000" />
-  <xacro:property name="LowerNeckPitchLinkInertia_IXX" value="0.001161092" />
-  <xacro:property name="LowerNeckPitchLinkInertia_IXY" value="-0.000099490" />
-  <xacro:property name="LowerNeckPitchLinkInertia_IXZ" value="0.000499358" />
-  <xacro:property name="LowerNeckPitchLinkInertia_IYY" value="0.001462041" />
-  <xacro:property name="LowerNeckPitchLinkInertia_IYZ" value="0.000191851" />
-  <xacro:property name="LowerNeckPitchLinkInertia_IZZ" value="0.000656934" />
+  <xacro:property name="LowerNeckPitchLinkInertia_IXX" value="0.001470716" />
+  <xacro:property name="LowerNeckPitchLinkInertia_IXY" value="-0.000126021" />
+  <xacro:property name="LowerNeckPitchLinkInertia_IXZ" value="0.000632521" />
+  <xacro:property name="LowerNeckPitchLinkInertia_IYY" value="0.001851919" />
+  <xacro:property name="LowerNeckPitchLinkInertia_IYZ" value="0.000243012" />
+  <xacro:property name="LowerNeckPitchLinkInertia_IZZ" value="0.000832117" />
   <xacro:property name="NeckYawLinkMass" value="1.4" />
   <xacro:property name="NeckYawLinkComPosition" value="-0.030000  -0.010000 0.150000" />
-  <xacro:property name="NeckYawLinkInertia_IXX" value="0.001664748" />
-  <xacro:property name="NeckYawLinkInertia_IXY" value="-0.000150052" />
-  <xacro:property name="NeckYawLinkInertia_IXZ" value="0.000603064" />
-  <xacro:property name="NeckYawLinkInertia_IYY" value="0.002332736" />
-  <xacro:property name="NeckYawLinkInertia_IYZ" value="0.000205389" />
-  <xacro:property name="NeckYawLinkInertia_IZZ" value="0.001766459" />
+  <xacro:property name="NeckYawLinkInertia_IXX" value="0.001997698" />
+  <xacro:property name="NeckYawLinkInertia_IXY" value="-0.000180062" />
+  <xacro:property name="NeckYawLinkInertia_IXZ" value="0.000723677" />
+  <xacro:property name="NeckYawLinkInertia_IYY" value="0.002919928" />
+  <xacro:property name="NeckYawLinkInertia_IYZ" value="0.000246467" />
+  <xacro:property name="NeckYawLinkInertia_IZZ" value="0.002119751" />
   <xacro:property name="UpperNeckPitchLinkMass" value="4.59" />
   <xacro:property name="UpperNeckPitchLinkComPosition" value="0.100912 0.005783 0.034787" />
