Commit message: flip the order of the legs

File: robots/valkyrie_A/xacro/leg/joint_limits.xacro (robot description, xacro)
@@ -10,5 +10,5 @@
   <xacro:property name="HipRollPositionLimit_Lower" value="-0.524" />
   <xacro:property name="HipPitchPositionLimit_Lower" value="-2.356" />
-  <xacro:property name="KneePitchPositionLimit_Lower" value="-1.902" />
+  <xacro:property name="KneePitchPositionLimit_Lower" value="-0.218" />
   <xacro:property name="AnklePitchPositionLimit_Lower" value="-0.873" />
   <xacro:property name="AnkleRollPositionLimit_Lower" value="-0.349" />
@@ -16,5 +16,5 @@
   <xacro:property name="HipRollPositionLimit_Upper" value="0.262" />
   <xacro:property name="HipPitchPositionLimit_Upper" value="1.710" />
-  <xacro:property name="KneePitchPositionLimit_Upper" value="0.218" />
+  <xacro:property name="KneePitchPositionLimit_Upper" value="1.902" />
   <xacro:property name="AnklePitchPositionLimit_Upper" value="0.873" />
   <xacro:property name="AnkleRollPositionLimit_Upper" value="0.349" />
