Commit message: reflect the hip roll and yaw angles

File: robots/valkyrie_A/xacro/leg/leg.xacro (robot description, xacro)
@@ -92,5 +92,10 @@
                           axis="${HipYawRotationAxis}"
                           damping="0.1" friction="0.0">
+        <xacro:if value="${(reflect+1)/2}">
+        <limit effort="${HipYawTorqueLimit}" lower="${-reflect * HipYawPositionLimit_Upper}" upper="${-reflect * HipYawPositionLimit_Lower}" velocity="${HipYawVelocityLimit}"/>
+        </xacro:if>
+        <xacro:if value="${(-reflect+1)/2}">
         <limit effort="${HipYawTorqueLimit}" lower="${HipYawPositionLimit_Lower}" upper="${HipYawPositionLimit_Upper}" velocity="${HipYawVelocityLimit}"/>
+        </xacro:if>
         <controller_gains Kp="15000" Kd="500"/>
     </xacro:revolute_joint_ex>
@@ -101,5 +106,10 @@
                           axis="${HipRollRotationAxis}"
                           damping="0.1" friction="0.0">
+        <xacro:if value="${(reflect+1)/2}">
+        <limit effort="${HipRollTorqueLimit}" lower="${-reflect * HipRollPositionLimit_Upper}" upper="${-reflect * HipRollPositionLimit_Lower}" velocity="${HipRollVelocityLimit}"/>
+        </xacro:if>
+        <xacro:if value="${(-reflect+1)/2}">
         <limit effort="${HipRollTorqueLimit}" lower="${HipRollPositionLimit_Lower}" upper="${HipRollPositionLimit_Upper}" velocity="${HipRollVelocityLimit}"/>
+        </xacro:if>
         <controller_gains Kp="15000" Kd="500"/>
     </xacro:revolute_joint_ex>

Commit message: Updated foot inertia/mass/com based on sys-id experiments.

File: robots/valkyrie_A/xacro/leg/leg.xacro (robot description, xacro)
@@ -67,7 +67,9 @@
                     material="White"
                     collision_mesh="${mesh_root}/legs/lj5.stl"/>
-    <xacro:box_link name="${AnkleRollLinkName}"
-                    width="${LJ6_Link_Width}" height="${LJ6_Link_Height}" depth="${LJ6_Link_Length}" mass="${FootMass}"
+    <xacro:standard_link name="${AnkleRollLinkName}"
+                    mass="${FootMass}"
                     origin_xyz="${FootComPosition}"
+                    ixx="${FootInertia_IXX}" ixy="${FootInertia_IXY}" ixz="${FootInertia_IXZ}"
+                    iyy="${FootInertia_IYY}" iyz="${FootInertia_IYZ}" izz="${FootInertia_IZZ}"
                     origin_rpy="0 0 0"
                     visual_mesh="${mesh_root}/legs/foot_${prefix}.stl"

File: robots/valkyrie_A/xacro/leg/mass_parameters.xacro (robot description, xacro)
@@ -11,5 +11,11 @@
   <xacro:property name="AnklePitchLinkMass" value="0.395" />
   <xacro:property name="AnklePitchLinkComPosition" value="-0.001270 ${reflect*0.000000} -0.006010" />
-  <xacro:property name="FootMass" value="1.888" />
-  <xacro:property name="FootComPosition" value="0.068860 ${reflect*-0.000285} -0.051830" />
+  <xacro:property name="FootMass" value="3.2549999" />
+  <xacro:property name="FootComPosition" value="0.040004 ${reflect*-0.00381} -0.049558" />
+  <xacro:property name="FootInertia_IXX" value="0.008966273" />
+  <xacro:property name="FootInertia_IXY" value="-0.000086029" />
+  <xacro:property name="FootInertia_IXZ" value="0.003944774" />
+  <xacro:property name="FootInertia_IYY" value="0.023943858" />
+  <xacro:property name="FootInertia_IYZ" value="0.000105218" />
+  <xacro:property name="FootInertia_IZZ" value="0.028128777" />
 </robot>

Commit message: Hotfix: Undefined xml macro was making into urdf rather than throwing error.

File: robots/valkyrie_A/xacro/leg/leg.xacro (robot description, xacro)
@@ -159,17 +159,4 @@
     <xacro:make_leg_joints prefix="${prefix}" reflect="${reflect}" leg_root_link="${leg_root_link}" />
     <xacro:make_ankle_joints prefix="${prefix}" reflect="${reflect}" leg_root_link="${leg_root_link}" />
-    <xacro:make_foot_joints prefix="${prefix}" reflect="${reflect}" leg_root_link="${leg_root_link}" />
-  </xacro:macro>
-  <xacro:macro name="make_leg_fixed_ankle" params="prefix reflect leg_root_link">
-    <xacro:make_leg_links prefix="${prefix}" reflect="${reflect}" leg_root_link="${leg_root_link}" />
-    <xacro:make_leg_joints prefix="${prefix}" reflect="${reflect}" leg_root_link="${leg_root_link}" />
-    <xacro:make_ankle_joints_fixed prefix="${prefix}" reflect="${reflect}" leg_root_link="${leg_root_link}" />
-    <xacro:make_foot_joints prefix="${prefix}" reflect="${reflect}" leg_root_link="${leg_root_link}" />
-  </xacro:macro>
-  <xacro:macro name="make_leg_fixed_upper_leg" params="prefix reflect leg_root_link">
-    <xacro:make_leg_links prefix="${prefix}" reflect="${reflect}" leg_root_link="${leg_root_link}" />
-    <xacro:make_leg_joints_fixed prefix="${prefix}" reflect="${reflect}" leg_root_link="${leg_root_link}" />
-    <xacro:make_ankle_joints prefix="${prefix}" reflect="${reflect}" leg_root_link="${leg_root_link}" />
-    <xacro:make_foot_joints prefix="${prefix}" reflect="${reflect}" leg_root_link="${leg_root_link}" />
   </xacro:macro>
   <!-- Sensors -->

Commit message: Hotfix: Undefined macro was making its way into the URDF somehow rather than throwing an error.

File: robots/valkyrie_A/xacro/leg/leg.xacro (robot description, xacro)
@@ -157,17 +157,4 @@
     <xacro:make_leg_joints prefix="${prefix}" reflect="${reflect}" leg_root_link="${leg_root_link}" />
     <xacro:make_ankle_joints prefix="${prefix}" reflect="${reflect}" leg_root_link="${leg_root_link}" />
-    <xacro:make_foot_joints prefix="${prefix}" reflect="${reflect}" leg_root_link="${leg_root_link}" />
-  </xacro:macro>
-  <xacro:macro name="make_leg_fixed_ankle" params="prefix reflect leg_root_link">
-    <xacro:make_leg_links prefix="${prefix}" reflect="${reflect}" leg_root_link="${leg_root_link}" />
-    <xacro:make_leg_joints prefix="${prefix}" reflect="${reflect}" leg_root_link="${leg_root_link}" />
-    <xacro:make_ankle_joints_fixed prefix="${prefix}" reflect="${reflect}" leg_root_link="${leg_root_link}" />
-    <xacro:make_foot_joints prefix="${prefix}" reflect="${reflect}" leg_root_link="${leg_root_link}" />
-  </xacro:macro>
-  <xacro:macro name="make_leg_fixed_upper_leg" params="prefix reflect leg_root_link">
-    <xacro:make_leg_links prefix="${prefix}" reflect="${reflect}" leg_root_link="${leg_root_link}" />
-    <xacro:make_leg_joints_fixed prefix="${prefix}" reflect="${reflect}" leg_root_link="${leg_root_link}" />
-    <xacro:make_ankle_joints prefix="${prefix}" reflect="${reflect}" leg_root_link="${leg_root_link}" />
-    <xacro:make_foot_joints prefix="${prefix}" reflect="${reflect}" leg_root_link="${leg_root_link}" />
   </xacro:macro>
   <!-- Sensors -->

Commit message: Changing some sensors from fixed_joint to sensor tags.

File: robots/valkyrie_A/xacro/leg/leg.xacro (robot description, xacro)
@@ -164,7 +164,7 @@
                        origin_xyz="0.0189 0.0 -0.0783"
                        origin_rpy="0.0 0.13 0.0"/>
-    <xacro:ati_force_torque_sensor sensorName="${prefix}LegSixAxis"
+    <xacro:ati_force_torque_sensor sensorName="${prefix}FootSixAxis"
                         parentLink="${AnkleRollLinkName}"
-                        origin_xyz="0.022 0.0 -0.059"
+                        origin_xyz="0.0215594 0.0 -0.0585488"
                         origin_rpy="3.14 0.0 -1.047"/>
   </xacro:macro>

File: robots/valkyrie_A/xacro/sensors/ati_force_torque.xacro (robot description, xacro)
@@ -2,11 +2,8 @@
 <robot xmlns:xacro="http://www.ros.org/wiki/xacro" name="ati_force_torque_sensor">
   <xacro:macro name="ati_force_torque_sensor" params="sensorName parentLink origin_xyz origin_rpy">
-    <xacro:massless_virtual_link name="${sensorName}_Frame"
-                    origin_rpy="0 0 0"
-                    origin_xyz="0 0 0"/>
-    <xacro:fixed_joint jointName="${sensorName}_Offset"
-                       parent="${parentLink}" child="${sensorName}_Frame"
-                       origin_rpy="${origin_rpy}"
-                       origin_xyz="${origin_xyz}"/>
+    <sensor name="${sensorName}" type="force_torque">
+      <parent link="${parentLink}"/>
+      <origin rpy="${origin_rpy}" xyz="${origin_xyz}"/>
+  	</sensor>
   </xacro:macro>
 </robot>

File: robots/valkyrie_A/xacro/sensors/microstrain.xacro (robot description, xacro)
@@ -6,11 +6,25 @@
   <xacro:property name="MicrostrainMass" value="0.0000001"/>
   <xacro:macro name="microstrain_sensor" params="sensorName parentLink origin_xyz origin_rpy">
-    <xacro:massless_virtual_link name="${sensorName}_Frame"
-                    origin_rpy="0 0 0"
-                    origin_xyz="0 0 0"/>
-    <xacro:fixed_joint jointName="${sensorName}_Offset"
-                       parent="${parentLink}" child="${sensorName}_Frame"
-                       origin_rpy="${origin_rpy}"
-                       origin_xyz="${origin_xyz}"/>
+    <sensor name="${sensorName}" type="imu">
+      <parent link="${parentLink}"/>
+      <origin rpy="${origin_rpy}" xyz="${origin_xyz}"/>
+      <imu>
+         <noise>
+             <type>gaussian</type>
+             <rate>
+                 <mean>0</mean>
+                 <stddev>0.0002</stddev>
+                 <bias_mean>7.5e-06</bias_mean>
+                 <bias_stddev>8e-07</bias_stddev>
+             </rate>
+             <accel>
+                 <mean>0</mean>
+                 <stddev>0.017</stddev>
+                 <bias_mean>0.1</bias_mean>
+                 <bias_stddev>0.001</bias_stddev>
+             </accel>
+         </noise>
+      </imu>
+      </sensor>
   </xacro:macro>
 </robot>

Commit message: Updated inertias of leg links(minus legj1) based on primitive link shapes created in CAD.

File: robots/valkyrie_A/xacro/leg/leg.xacro (robot description, xacro)
@@ -39,28 +39,36 @@
                     material="Gold"
                     collision_mesh="${mesh_root}/legs/lj1_${prefix}.stl"/>
-    <xacro:box_link name="${HipRollLinkName}"
+    <xacro:standard_link name="${HipRollLinkName}"
                     width="${LJ2_Link_Width}" height="${LJ2_Link_Height}" depth="${LJ2_Link_Length}" mass="${HipRollLinkMass}"
                     origin_xyz="${HipRollLinkComPosition}"
+                    ixx="${HipRollLinkInertia_IXX}" ixy="${HipRollLinkInertia_IXY}" ixz="${HipRollLinkInertia_IXZ}"
+                    iyy="${HipRollLinkInertia_IYY}" iyz="${HipRollLinkInertia_IYZ}" izz="${HipRollLinkInertia_IZZ}"
                     origin_rpy="0 0 0"
                     visual_mesh="${mesh_root}/legs/lj2_${prefix}.stl"
                     material="White"
                     collision_mesh="${mesh_root}/legs/lj2_${prefix}.stl"/>
-    <xacro:box_link name="${HipPitchLinkName}"
+    <xacro:standard_link name="${HipPitchLinkName}"
                     width="${LJ3_Link_Width}" height="${LJ3_Link_Height}" depth="${LJ3_Link_Length}" mass="${HipPitchLinkMass}"
                     origin_xyz="${HipPitchLinkComPosition}"
+                    ixx="${HipPitchLinkInertia_IXX}" ixy="${HipPitchLinkInertia_IXY}" ixz="${HipPitchLinkInertia_IXZ}"
+                    iyy="${HipPitchLinkInertia_IYY}" iyz="${HipPitchLinkInertia_IYZ}" izz="${HipPitchLinkInertia_IZZ}"
                     origin_rpy="0 0 0"
                     visual_mesh="${mesh_root}/legs/lj3_${prefix}.stl"
                     material="White"
                     collision_mesh="${mesh_root}/legs/lj3_${prefix}.stl"/>
-    <xacro:box_link name="${KneePitchLinkName}"
+    <xacro:standard_link name="${KneePitchLinkName}"
                     width="${LJ4_Link_Box_Width}" height="${LJ4_Link_Box_Height}" depth="${LJ4_Link_Box_Length}" mass="${KneePitchLinkMass}"
                     origin_xyz="${KneePitchLinkComPosition}"
+                    ixx="${KneePitchLinkInertia_IXX}" ixy="${KneePitchLinkInertia_IXY}" ixz="${KneePitchLinkInertia_IXZ}"
+                    iyy="${KneePitchLinkInertia_IYY}" iyz="${KneePitchLinkInertia_IYZ}" izz="${KneePitchLinkInertia_IZZ}"
                     origin_rpy="0 0 0"
                     visual_mesh="${mesh_root}/legs/lj4_${prefix}.stl"
                     material="White"
                     collision_mesh="${mesh_root}/legs/lj4_${prefix}.stl"/>
-    <xacro:box_link name="${AnklePitchLinkName}"
+    <xacro:standard_link name="${AnklePitchLinkName}"
                     width="${LJ5_Link_Width}" height="${LJ5_Link_Height}" depth="${LJ5_Link_Length}" mass="${AnklePitchLinkMass}"
                     origin_xyz="${AnklePitchLinkComPosition}"
+                    ixx="${AnklePitchLinkInertia_IXX}" ixy="${AnklePitchLinkInertia_IXY}" ixz="${AnklePitchLinkInertia_IXZ}"
+                    iyy="${AnklePitchLinkInertia_IYY}" iyz="${AnklePitchLinkInertia_IYZ}" izz="${AnklePitchLinkInertia_IZZ}"
                     origin_rpy="0 0 0"
                     visual_mesh="${mesh_root}/legs/lj5.stl"

File: robots/valkyrie_A/xacro/leg/mass_parameters.xacro (robot description, xacro)
@@ -5,10 +5,34 @@
   <xacro:property name="HipRollLinkMass" value="3.665000" />
   <xacro:property name="HipRollLinkComPosition" value="0.012959 ${reflect*-0.007550} -0.015950" />
+  <xacro:property name="HipRollLinkInertia_IXX" value="0.005978962" />
+  <xacro:property name="HipRollLinkInertia_IXY" value="${reflect*0.000234823}" />
+  <xacro:property name="HipRollLinkInertia_IXZ" value="0.000553962" />
+  <xacro:property name="HipRollLinkInertia_IYY" value="0.009372646" />
+  <xacro:property name="HipRollLinkInertia_IYZ" value="${reflect*-0.000778956}" />
+  <xacro:property name="HipRollLinkInertia_IZZ" value="0.008193117" />
   <xacro:property name="HipPitchLinkMass" value="10.20" />
   <xacro:property name="HipPitchLinkComPosition" value="0.016691 ${reflect*-0.091397} -0.207875" />
+  <xacro:property name="HipPitchLinkInertia_IXX" value="0.240834130" />
+  <xacro:property name="HipPitchLinkInertia_IXY" value="${reflect*-0.000035915}" />
+  <xacro:property name="HipPitchLinkInertia_IXZ" value="0.003699383" />
+  <xacro:property name="HipPitchLinkInertia_IYY" value="0.256897050" />
+  <xacro:property name="HipPitchLinkInertia_IYZ" value="${reflect*0.001333005}" />
+  <xacro:property name="HipPitchLinkInertia_IZZ" value="0.023276352" />
   <xacro:property name="KneePitchLinkMass" value="6.600000" />
   <xacro:property name="KneePitchLinkComPosition" value="0.002425 ${reflect*-0.001543} -0.189511" />
+  <xacro:property name="KneePitchLinkInertia_IXX" value="0.096117529" />
+  <xacro:property name="KneePitchLinkInertia_IXY" value="0.000107885" />
+  <xacro:property name="KneePitchLinkInertia_IXZ" value="0.006319047" />
+  <xacro:property name="KneePitchLinkInertia_IYY" value="0.097118447" />
+  <xacro:property name="KneePitchLinkInertia_IYZ" value="-0.000494739" />
+  <xacro:property name="KneePitchLinkInertia_IZZ" value="0.013722874" />
   <xacro:property name="AnklePitchLinkMass" value="0.06" />
   <xacro:property name="AnklePitchLinkComPosition" value="-0.001269 ${reflect*0.00009} -0.006013" />
+  <xacro:property name="AnklePitchLinkInertia_IXX" value="0.000011226" />
+  <xacro:property name="AnklePitchLinkInertia_IXY" value="0.000000000" />
+  <xacro:property name="AnklePitchLinkInertia_IXZ" value="0.000002735" />
+  <xacro:property name="AnklePitchLinkInertia_IYY" value="0.000026700" />
+  <xacro:property name="AnklePitchLinkInertia_IYZ" value="0.0" />
+  <xacro:property name="AnklePitchLinkInertia_IZZ" value="0.000018792" />
   <xacro:property name="FootMass" value="3.2550" />
   <xacro:property name="FootComPosition" value="0.040004 ${reflect*-0.00381} -0.049558" />
