Commit message: Updated mass and COM locations of leg links found from the COM measurement experiments.

File: robots/valkyrie_A/xacro/leg/mass_parameters.xacro (robot description, xacro)
@@ -3,13 +3,13 @@
   <xacro:property name="HipYawLinkMass" value="2.39" />
   <xacro:property name="HipYawLinkComPosition" value="0.02176 ${reflect*-0.00131} 0.03867" />
-  <xacro:property name="HipRollLinkMass" value="5.95" />
-  <xacro:property name="HipRollLinkComPosition" value="-0.00185 ${reflect*0.02426} -0.019260" />
-  <xacro:property name="HipPitchLinkMass" value="10.3" />
-  <xacro:property name="HipPitchLinkComPosition" value="0.000057 ${reflect*0.050000} -0.220000" />
-  <xacro:property name="KneePitchLinkMass" value="7.4" />
-  <xacro:property name="KneePitchLinkComPosition" value="-0.004670 ${reflect*0.045000} -0.184940" />
-  <xacro:property name="AnklePitchLinkMass" value="0.395" />
-  <xacro:property name="AnklePitchLinkComPosition" value="-0.001270 ${reflect*0.000000} -0.006010" />
-  <xacro:property name="FootMass" value="3.2549999" />
+  <xacro:property name="HipRollLinkMass" value="3.665000" />
+  <xacro:property name="HipRollLinkComPosition" value="0.012959 ${reflect*-0.007550} -0.015950" />
+  <xacro:property name="HipPitchLinkMass" value="10.20" />
+  <xacro:property name="HipPitchLinkComPosition" value="0.016691 ${reflect*-0.091397} -0.207875" />
+  <xacro:property name="KneePitchLinkMass" value="6.600000" />
+  <xacro:property name="KneePitchLinkComPosition" value="0.002425 ${reflect*-0.001543} -0.189511" />
+  <xacro:property name="AnklePitchLinkMass" value="0.06" />
+  <xacro:property name="AnklePitchLinkComPosition" value="-0.001269 ${reflect*0.00009} -0.006013" />
+  <xacro:property name="FootMass" value="3.2550" />
   <xacro:property name="FootComPosition" value="0.040004 ${reflect*-0.00381} -0.049558" />
   <xacro:property name="FootInertia_IXX" value="0.008966273" />

Commit message: Fixed reflect bug with leg inertias.

File: robots/valkyrie_A/xacro/leg/mass_parameters.xacro (robot description, xacro)
@@ -6,16 +6,16 @@
   <xacro:property name="HipRollLinkComPosition" value="0.012959 ${reflect*0.007550} -0.015950" />
   <xacro:property name="HipRollLinkInertia_IXX" value="0.005978962" />
-  <xacro:property name="HipRollLinkInertia_IXY" value="${reflect*0.000234823}" />
+  <xacro:property name="HipRollLinkInertia_IXY" value="${reflect*-0.000234823}" />
   <xacro:property name="HipRollLinkInertia_IXZ" value="0.000553962" />
   <xacro:property name="HipRollLinkInertia_IYY" value="0.009372646" />
-  <xacro:property name="HipRollLinkInertia_IYZ" value="${reflect*-0.000778956}" />
+  <xacro:property name="HipRollLinkInertia_IYZ" value="${reflect*0.000778956}" />
   <xacro:property name="HipRollLinkInertia_IZZ" value="0.008193117" />
   <xacro:property name="HipPitchLinkMass" value="10.20" />
   <xacro:property name="HipPitchLinkComPosition" value="0.016691 ${reflect*0.091397} -0.207875" />
   <xacro:property name="HipPitchLinkInertia_IXX" value="0.240834130" />
-  <xacro:property name="HipPitchLinkInertia_IXY" value="${reflect*-0.000035915}" />
+  <xacro:property name="HipPitchLinkInertia_IXY" value="${reflect*0.000035915}" />
   <xacro:property name="HipPitchLinkInertia_IXZ" value="0.003699383" />
   <xacro:property name="HipPitchLinkInertia_IYY" value="0.256897050" />
-  <xacro:property name="HipPitchLinkInertia_IYZ" value="${reflect*0.001333005}" />
+  <xacro:property name="HipPitchLinkInertia_IYZ" value="${reflect*-0.001333005}" />
   <xacro:property name="HipPitchLinkInertia_IZZ" value="0.023276352" />
   <xacro:property name="KneePitchLinkMass" value="6.600000" />

Commit message: Removed stray brace.

File: robots/valkyrie_A/xacro/leg/mass_parameters.xacro (robot description, xacro)
@@ -28,5 +28,5 @@
   <xacro:property name="KneePitchLinkInertia_IZZ" value="0.013722874" />
   <xacro:property name="AnklePitchLinkMass" value="0.06" />
-  <xacro:property name="AnklePitchLinkComPosition" value="-0.001269 0.00009} -0.006013" />
+  <xacro:property name="AnklePitchLinkComPosition" value="-0.001269 0.00009 -0.006013" />
   <xacro:property name="AnklePitchLinkInertia_IXX" value="0.000011226" />
   <xacro:property name="AnklePitchLinkInertia_IXY" value="0.000000000" />
