Commit message: More reorg. Fixed the elbow limit for now. Will update with true values soon.

File: robots/valkyrie_A/xacro/arm/joint_limits.xacro (robot description, xacro)
@@ -18,5 +18,5 @@
   <xacro:property name="ShoulderRollPositionLimit_Upper" value="1.4835" />
   <xacro:property name="ShoulderYawPositionLimit_Upper" value="1.5707" />
-  <xacro:property name="ElbowPitchPositionLimit_Upper" value="-0.087" />
+  <xacro:property name="ElbowPitchPositionLimit_Upper" value="0.0" />
   <xacro:property name="ForearmYawPositionLimit_Upper" value="3.9269" />
   <xacro:property name="WristRollPositionLimit_Upper" value="0.524" />
