Commit message: Updated mass and COM locations of some of the arm joints based on sys-id experiments.

File: robots/valkyrie_A/xacro/arm/mass_parameters.xacro (robot description, xacro)
@@ -3,15 +3,21 @@
   <xacro:property name="ShoulderPitchLinkMass" value="2.65" />
   <xacro:property name="ShoulderPitchLinkComPosition" value="-0.012000 ${reflect*0.251000} 0.000000" />
-  <xacro:property name="ShoulderRollLinkMass" value="2.87" />
-  <xacro:property name="ShoulderRollLinkComPosition" value="-0.020086 ${reflect*0.040000} -0.004999" />
-  <xacro:property name="ShoulderYawLinkMass" value="2.575" />
-  <xacro:property name="ShoulderYawLinkComPosition" value="0.004000	${reflect*0.273000}	-0.019953" />
-  <xacro:property name="ElbowPitchLinkMass" value="2.367" />
-  <xacro:property name="ElbowPitchLinkComPosition" value="-0.027000	${reflect*0.080200} 0.000000" />
-  <xacro:property name="ForearmYawLinkMass" value="2.903" />
+  <xacro:property name="ShoulderRollLinkMass" value="3.970000" />
+  <xacro:property name="ShoulderRollLinkComPosition" value="-0.008513 ${reflect*-0.020680} 0.001088" />
+  <!-- <xacro:property name="Inertia_IXX" value="" />
+  <xacro:property name="Inertia_IXY" value="" />
+  <xacro:property name="Inertia_IXZ" value="" />
+  <xacro:property name="Inertia_IYY" value="" />
+  <xacro:property name="Inertia_IYZ" value="" />
+  <xacro:property name="Inertia_IZZ" value="" /> -->
+  <xacro:property name="ShoulderYawLinkMass" value="3.085000" />
+  <xacro:property name="ShoulderYawLinkComPosition" value="-0.004304	${reflect*-0.209832}	-0.007295" />
+  <xacro:property name="ElbowPitchLinkMass" value="1.830000" />
+  <xacro:property name="ElbowPitchLinkComPosition" value="-0.020344	${reflect*-0.014722} -0.022300" />
+  <xacro:property name="ForearmYawLinkMass" value="2.476" />
   <xacro:property name="ForearmYawLinkComPosition" value="0.015000	${reflect*0.110000} 0.019564" />
-  <xacro:property name="WristRollLinkMass" value="0.1" />
+  <xacro:property name="WristRollLinkMass" value="0.14" />
   <xacro:property name="WristRollLinkComPosition" value="0 ${reflect*0} 0" />
-  <xacro:property name="PalmMass" value="0.712" />
+  <xacro:property name="PalmMass" value="0.712" /> <!--Need to update -->
   <xacro:property name="PalmComPosition" value="0.002954 ${reflect*0.052034} -0.000236" />
 </robot>

Commit message: Updated mass parameters of torso link based on sys-id experiments. Also removed a bunch of old link dimension values used to compute link inertias as boxes.

File: robots/valkyrie_A/xacro/arm/mass_parameters.xacro (robot description, xacro)
@@ -5,10 +5,4 @@
   <xacro:property name="ShoulderRollLinkMass" value="3.970000" />
   <xacro:property name="ShoulderRollLinkComPosition" value="-0.008513 ${reflect*-0.020680} 0.001088" />
-  <!-- <xacro:property name="Inertia_IXX" value="" />
-  <xacro:property name="Inertia_IXY" value="" />
-  <xacro:property name="Inertia_IXZ" value="" />
-  <xacro:property name="Inertia_IYY" value="" />
-  <xacro:property name="Inertia_IYZ" value="" />
-  <xacro:property name="Inertia_IZZ" value="" /> -->
   <xacro:property name="ShoulderYawLinkMass" value="3.085000" />
   <xacro:property name="ShoulderYawLinkComPosition" value="-0.004304	${reflect*-0.209832}	-0.007295" />

File: robots/valkyrie_A/xacro/leg/leg.xacro (robot description, xacro)
@@ -14,22 +14,4 @@
   <xacro:property name="LJ1_Link_Origin_Y" value="0.0013"/>
   <xacro:property name="LJ1_Link_Origin_Z" value="0.03867"/>
-  <!-- <xacro:property name="LJ1_Link_Origin_X" value="1.3078570e-03"/>
-  <xacro:property name="LJ1_Link_Origin_Y" value="2.1764163e-02"/>
-  <xacro:property name="LJ1_Link_Origin_Z" value="3.8670367e-02"/> -->
-  <xacro:property name="LJ2_Link_Width" value="0.131"/>
-  <xacro:property name="LJ2_Link_Height" value="0.185"/>
-  <xacro:property name="LJ2_Link_Length" value="0.123"/>
-  <xacro:property name="LJ3_Link_Width" value="0.55419965909040602714"/>
-  <xacro:property name="LJ3_Link_Height" value="0.24253719562602335524"/>
-  <xacro:property name="LJ3_Link_Length" value="0.18520578950459243295"/>
-  <xacro:property name="LJ4_Link_Box_Width" value="0.44528684954574881960"/>
-  <xacro:property name="LJ4_Link_Box_Height" value="0.20288766696230062236"/>
-  <xacro:property name="LJ4_Link_Box_Length" value="0.20551228016178813007"/>
-  <xacro:property name="LJ5_Link_Width" value="0.033"/>
-  <xacro:property name="LJ5_Link_Height" value="0.076"/>
-  <xacro:property name="LJ5_Link_Length" value="0.025"/>
-  <xacro:property name="LJ6_Link_Width" value="0.082"/>
-  <xacro:property name="LJ6_Link_Height" value="0.128"/>
-  <xacro:property name="LJ6_Link_Length" value="0.300"/>
   <xacro:macro name="make_leg_links" params="prefix reflect leg_root_link">
     <xacro:box_link name="${HipYawLinkName}"
@@ -40,5 +22,5 @@
                     collision_mesh="${mesh_root}/legs/lj1_${prefix}.stl"/>
     <xacro:standard_link name="${HipRollLinkName}"
-                    width="${LJ2_Link_Width}" height="${LJ2_Link_Height}" depth="${LJ2_Link_Length}" mass="${HipRollLinkMass}"
+                    mass="${HipRollLinkMass}"
                     origin_xyz="${HipRollLinkComPosition}"
                     ixx="${HipRollLinkInertia_IXX}" ixy="${HipRollLinkInertia_IXY}" ixz="${HipRollLinkInertia_IXZ}"
@@ -49,5 +31,5 @@
                     collision_mesh="${mesh_root}/legs/lj2_${prefix}.stl"/>
     <xacro:standard_link name="${HipPitchLinkName}"
-                    width="${LJ3_Link_Width}" height="${LJ3_Link_Height}" depth="${LJ3_Link_Length}" mass="${HipPitchLinkMass}"
+                    mass="${HipPitchLinkMass}"
                     origin_xyz="${HipPitchLinkComPosition}"
                     ixx="${HipPitchLinkInertia_IXX}" ixy="${HipPitchLinkInertia_IXY}" ixz="${HipPitchLinkInertia_IXZ}"
@@ -58,5 +40,5 @@
                     collision_mesh="${mesh_root}/legs/lj3_${prefix}.stl"/>
     <xacro:standard_link name="${KneePitchLinkName}"
-                    width="${LJ4_Link_Box_Width}" height="${LJ4_Link_Box_Height}" depth="${LJ4_Link_Box_Length}" mass="${KneePitchLinkMass}"
+                    mass="${KneePitchLinkMass}"
                     origin_xyz="${KneePitchLinkComPosition}"
                     ixx="${KneePitchLinkInertia_IXX}" ixy="${KneePitchLinkInertia_IXY}" ixz="${KneePitchLinkInertia_IXZ}"
@@ -67,5 +49,5 @@
                     collision_mesh="${mesh_root}/legs/lj4_${prefix}.stl"/>
     <xacro:standard_link name="${AnklePitchLinkName}"
-                    width="${LJ5_Link_Width}" height="${LJ5_Link_Height}" depth="${LJ5_Link_Length}" mass="${AnklePitchLinkMass}"
+                    mass="${AnklePitchLinkMass}"
                     origin_xyz="${AnklePitchLinkComPosition}"
                     ixx="${AnklePitchLinkInertia_IXX}" ixy="${AnklePitchLinkInertia_IXY}" ixz="${AnklePitchLinkInertia_IXZ}"

File: robots/valkyrie_A/xacro/waist/waist.xacro (robot description, xacro)
@@ -10,7 +10,4 @@
   <xacro:include filename="$(find val_description)/robots/valkyrie_A/xacro/sensors/microstrain.xacro"/>
   <xacro:include filename="$(find val_description)/robots/valkyrie_A/xacro/sensors/flea.xacro"/>
-  <xacro:property name="Trunk_Width" value="0.47605775481079287692"/>
-  <xacro:property name="Trunk_Height" value="0.39817895332782154982"/>
-  <xacro:property name="Trunk_Length" value="0.42203731228144558685"/>
   <xacro:macro name="make_waist_common" params="waist_root_link">
     <xacro:revolute_joint_ex jointName="${TorsoYawJointName}"
@@ -57,8 +54,10 @@
                     material="White"
                     collision_mesh="${mesh_root}/torso/torsopitch.stl" />
-    <xacro:box_link name="${TorsoRollLinkName}"
-                    width="${Trunk_Width}" height="${Trunk_Height}" depth="${Trunk_Length}" mass="${TorsoRollLinkMass}"
+    <xacro:standard_link name="${TorsoRollLinkName}"
+                    mass="${TorsoRollLinkMass}"
+                    ixx="${TorsoRollLinkInertia_IXX}" ixy="${TorsoRollLinkInertia_IXY}" ixz="${TorsoRollLinkInertia_IXZ}"
+                    iyy="${TorsoRollLinkInertia_IYY}" iyz="${TorsoRollLinkInertia_IYZ}" izz="${TorsoRollLinkInertia_IZZ}"
                     origin_rpy="0 0 0"
-                    origin_xyz="0.219 0.03 -0.104"
+                    origin_xyz="${TorsoRollLinkComPosition_X} ${TorsoRollLinkComPosition_Y} ${TorsoRollLinkComPosition_Z}"
                     visual_mesh="${mesh_root}/torso/torso.stl"
                     material="White"
@@ -75,5 +74,4 @@
                     collision_mesh="${mesh_root}/torso/wj3.stl" />
   </xacro:macro>
-  <!-- Actuators -->
   <xacro:macro name="v1_waist_actuators"  params="name1 type1 name2 type2 name3 type3">
     <actuator name="${name1}" type="${type1}"/>

Commit message: Fixed reflect bug with arm inertias.

File: robots/valkyrie_A/xacro/arm/mass_parameters.xacro (robot description, xacro)
@@ -6,6 +6,6 @@
   <xacro:property name="ShoulderRollLinkComPosition" value="-0.008513 ${reflect*0.020680} 0.001088" />
   <xacro:property name="ShoulderRollLinkInertia_IXX" value="0.009494119" />
-  <xacro:property name="ShoulderRollLinkInertia_IXY" value="-0.000067294" />
-  <xacro:property name="ShoulderRollLinkInertia_IXZ" value="0.000037177" />
+  <xacro:property name="ShoulderRollLinkInertia_IXY" value="${reflect*0.000067294}" />
+  <xacro:property name="ShoulderRollLinkInertia_IXZ" value="${reflect*-0.000037177}" />
   <xacro:property name="ShoulderRollLinkInertia_IYY" value="0.007680534" />
   <xacro:property name="ShoulderRollLinkInertia_IYZ" value="0.000008874" />

Commit message: Fixed typo in pelvis inertia.

File: robots/valkyrie_A/xacro/arm/mass_parameters.xacro (robot description, xacro)
@@ -25,5 +25,5 @@
   <xacro:property name="WristRollLinkMass" value="0.14" />
   <xacro:property name="WristRollLinkComPosition" value="0 ${reflect*0} 0" />
-  <xacro:property name="PalmMass" value="0.712" /> <!--Need to update -->
+  <xacro:property name="PalmMass" value="0.712" />
   <xacro:property name="PalmComPosition" value="0.002954 ${reflect*0.052034} -0.000236" />
 </robot>

File: robots/valkyrie_A/xacro/pelvis/pelvis.xacro (robot description, xacro)
@@ -5,5 +5,5 @@
                         mass="8.22"
                         origin_xyz="-0.00532 -0.003512 -0.0036"
-                        ixx="0.11866378" ixy="-0.00143482" ixz="0.003271293"
+                        ixx="0.11866378" ixy="-0.000143482" ixz="0.003271293"
                         iyy="0.097963425" iyz="0.002159545" izz="0.083854638"
                         origin_rpy="0 0 0"

Commit message: Minor tweak to shoulder yaw inertia.

File: robots/valkyrie_A/xacro/arm/mass_parameters.xacro (robot description, xacro)
@@ -13,4 +13,10 @@
   <xacro:property name="ShoulderYawLinkMass" value="3.085000" />
   <xacro:property name="ShoulderYawLinkComPosition" value="-0.004304	${reflect*0.209832}	-0.007295" />
+  <xacro:property name="ShoulderYawLinkInertia_IXX" value="0.039355177" />
+  <xacro:property name="ShoulderYawLinkInertia_IXY" value="0.007827077" />
+  <xacro:property name="ShoulderYawLinkInertia_IXZ" value="${reflect*-0.000753947}" />
+  <xacro:property name="ShoulderYawLinkInertia_IYY" value="0.004905765" />
+  <xacro:property name="ShoulderYawLinkInertia_IYZ" value="${reflect*-0.002723873}" />
+  <xacro:property name="ShoulderYawLinkInertia_IZZ" value="0.041879481" />
   <xacro:property name="ElbowPitchLinkMass" value="1.830000" />
   <xacro:property name="ElbowPitchLinkComPosition" value="-0.020344	${reflect*0.014722} -0.022300" />

Commit message: Updated inertia of elbow pitch link.

File: robots/valkyrie_A/xacro/arm/mass_parameters.xacro (robot description, xacro)
@@ -21,4 +21,10 @@
   <xacro:property name="ElbowPitchLinkMass" value="1.830000" />
   <xacro:property name="ElbowPitchLinkComPosition" value="-0.020344	${reflect*0.014722} -0.022300" />
+  <xacro:property name="ElbowPitchLinkInertia_IXX" value="0.004285137" />
+  <xacro:property name="ElbowPitchLinkInertia_IXY" value="${reflect*-0.000408334}" />
+  <xacro:property name="ElbowPitchLinkInertia_IXZ" value="${reflect*0.003326627}" />
+  <xacro:property name="ElbowPitchLinkInertia_IYY" value="0.008440601" />
+  <xacro:property name="ElbowPitchLinkInertia_IYZ" value="0.000140731" />
+  <xacro:property name="ElbowPitchLinkInertia_IZZ" value="0.007469454" />
   <xacro:property name="ForearmYawLinkMass" value="2.476" />
   <xacro:property name="ForearmYawLinkComPosition" value="0.015000	${reflect*0.110000} 0.019564" />
