Commit message: Changed all occurences of valkyrie_description to val_description. Updated .gitignore to ignore .bak files.

File: robots/valkyrie_A/xacro/arm/arm.xacro (robot description, xacro)
@@ -1,11 +1,11 @@
 <?xml version="1.0" ?>
 <robot xmlns:xacro="http://www.ros.org/wiki/xacro" name="v1/arm">
-  <xacro:include filename="$(find valkyrie_description)/robots/valkyrie_A/xacro/arm/joint_names.xacro"/>
-  <xacro:include filename="$(find valkyrie_description)/robots/valkyrie_A/xacro/arm/joint_axes.xacro"/>
-  <xacro:include filename="$(find valkyrie_description)/robots/valkyrie_A/xacro/arm/link_names.xacro"/>
-  <xacro:include filename="$(find valkyrie_description)/robots/valkyrie_A/xacro/arm/joint_limits.xacro"/>
-  <xacro:include filename="$(find valkyrie_description)/robots/valkyrie_A/xacro/arm/frame_parameters.xacro"/>
-  <xacro:include filename="$(find valkyrie_description)/robots/valkyrie_A/xacro/arm/mass_parameters.xacro"/>
-  <xacro:include filename="$(find valkyrie_description)/robots/valkyrie_A/xacro/sensors/camboard.xacro"/>
+  <xacro:include filename="$(find val_description)/robots/valkyrie_A/xacro/arm/joint_names.xacro"/>
+  <xacro:include filename="$(find val_description)/robots/valkyrie_A/xacro/arm/joint_axes.xacro"/>
+  <xacro:include filename="$(find val_description)/robots/valkyrie_A/xacro/arm/link_names.xacro"/>
+  <xacro:include filename="$(find val_description)/robots/valkyrie_A/xacro/arm/joint_limits.xacro"/>
+  <xacro:include filename="$(find val_description)/robots/valkyrie_A/xacro/arm/frame_parameters.xacro"/>
+  <xacro:include filename="$(find val_description)/robots/valkyrie_A/xacro/arm/mass_parameters.xacro"/>
+  <xacro:include filename="$(find val_description)/robots/valkyrie_A/xacro/sensors/camboard.xacro"/>
   <xacro:property name="AJ1_Link_Width" value="0.162"/>
   <xacro:property name="AJ1_Link_Height" value="0.202"/>

File: robots/valkyrie_A/xacro/common/common_bodies.xacro (robot description, xacro)
@@ -1,11 +1,11 @@
 <robot xmlns:xacro="http://ros.orgt/wiki/xacro" name="v1/common_bodies">
-    <xacro:include filename="$(find valkyrie_description)/robots/valkyrie_A/xacro/pelvis/pelvis.xacro" />
-    <xacro:include filename="$(find valkyrie_description)/robots/valkyrie_A/xacro/waist/waist.xacro" />
-    <xacro:include filename="$(find valkyrie_description)/robots/valkyrie_A/xacro/head/head.xacro" />
-    <xacro:include filename="$(find valkyrie_description)/robots/valkyrie_A/xacro/arm/arm.xacro" />
-    <xacro:include filename="$(find valkyrie_description)/robots/valkyrie_A/xacro/leg/leg.xacro" />
-    <xacro:include filename="$(find valkyrie_description)/robots/valkyrie_A/xacro/thumb/thumb.xacro" />
-    <xacro:include filename="$(find valkyrie_description)/robots/valkyrie_A/xacro/index_finger/index_finger.xacro" />
-    <xacro:include filename="$(find valkyrie_description)/robots/valkyrie_A/xacro/middle_finger/middle_finger.xacro" />
-    <xacro:include filename="$(find valkyrie_description)/robots/valkyrie_A/xacro/pinky_finger/pinky_finger.xacro" />
+    <xacro:include filename="$(find val_description)/robots/valkyrie_A/xacro/pelvis/pelvis.xacro" />
+    <xacro:include filename="$(find val_description)/robots/valkyrie_A/xacro/waist/waist.xacro" />
+    <xacro:include filename="$(find val_description)/robots/valkyrie_A/xacro/head/head.xacro" />
+    <xacro:include filename="$(find val_description)/robots/valkyrie_A/xacro/arm/arm.xacro" />
+    <xacro:include filename="$(find val_description)/robots/valkyrie_A/xacro/leg/leg.xacro" />
+    <xacro:include filename="$(find val_description)/robots/valkyrie_A/xacro/thumb/thumb.xacro" />
+    <xacro:include filename="$(find val_description)/robots/valkyrie_A/xacro/index_finger/index_finger.xacro" />
+    <xacro:include filename="$(find val_description)/robots/valkyrie_A/xacro/middle_finger/middle_finger.xacro" />
+    <xacro:include filename="$(find val_description)/robots/valkyrie_A/xacro/pinky_finger/pinky_finger.xacro" />
 </robot>

File: robots/valkyrie_A/xacro/head/head.xacro (robot description, xacro)
@@ -1,11 +1,11 @@
 <robot xmlns:xacro="http://www.ros.org/wiki/xacro" name="v1/head">
-  <xacro:include filename="$(find valkyrie_description)/robots/valkyrie_A/xacro/head/joint_names.xacro"/>
-  <xacro:include filename="$(find valkyrie_description)/robots/valkyrie_A/xacro/head/joint_axes.xacro"/>
-  <xacro:include filename="$(find valkyrie_description)/robots/valkyrie_A/xacro/head/link_names.xacro"/>
-  <xacro:include filename="$(find valkyrie_description)/robots/valkyrie_A/xacro/head/joint_limits.xacro"/>
-  <xacro:include filename="$(find valkyrie_description)/robots/valkyrie_A/xacro/head/frame_parameters.xacro"/>
-  <xacro:include filename="$(find valkyrie_description)/robots/valkyrie_A/xacro/head/mass_parameters.xacro"/>
-  <xacro:include filename="$(find valkyrie_description)/robots/valkyrie_A/xacro/sensors/ensenso.xacro"/>
-  <xacro:include filename="$(find valkyrie_description)/robots/valkyrie_A/xacro/sensors/webcam.xacro"/>
+  <xacro:include filename="$(find val_description)/robots/valkyrie_A/xacro/head/joint_names.xacro"/>
+  <xacro:include filename="$(find val_description)/robots/valkyrie_A/xacro/head/joint_axes.xacro"/>
+  <xacro:include filename="$(find val_description)/robots/valkyrie_A/xacro/head/link_names.xacro"/>
+  <xacro:include filename="$(find val_description)/robots/valkyrie_A/xacro/head/joint_limits.xacro"/>
+  <xacro:include filename="$(find val_description)/robots/valkyrie_A/xacro/head/frame_parameters.xacro"/>
+  <xacro:include filename="$(find val_description)/robots/valkyrie_A/xacro/head/mass_parameters.xacro"/>
+  <xacro:include filename="$(find val_description)/robots/valkyrie_A/xacro/sensors/ensenso.xacro"/>
+  <xacro:include filename="$(find val_description)/robots/valkyrie_A/xacro/sensors/webcam.xacro"/>
   <xacro:property name="NJ3_Link_Radius" value="0.139"/>
   <xacro:macro name="include_head" params="lower_neck_pitch_root_link">

File: robots/valkyrie_A/xacro/index_finger/index_finger.xacro (robot description, xacro)
@@ -1,11 +1,11 @@
 <?xml version="1.0" ?>
 <robot xmlns:xacro="http://www.ros.org/wiki/xacro" name="v1/index_finger">
-  <xacro:include filename="$(find valkyrie_description)/robots/valkyrie_A/xacro/index_finger/joint_names.xacro"/>
-  <xacro:include filename="$(find valkyrie_description)/robots/valkyrie_A/xacro/index_finger/joint_axes.xacro"/>
-  <xacro:include filename="$(find valkyrie_description)/robots/valkyrie_A/xacro/index_finger/actuator_names.xacro"/>
-  <xacro:include filename="$(find valkyrie_description)/robots/valkyrie_A/xacro/index_finger/link_names.xacro"/>
-  <xacro:include filename="$(find valkyrie_description)/robots/valkyrie_A/xacro/index_finger/joint_limits.xacro"/>
-  <xacro:include filename="$(find valkyrie_description)/robots/valkyrie_A/xacro/index_finger/frame_parameters.xacro"/>
-  <xacro:include filename="$(find valkyrie_description)/robots/valkyrie_A/xacro/index_finger/mass_parameters.xacro"/>
+  <xacro:include filename="$(find val_description)/robots/valkyrie_A/xacro/index_finger/joint_names.xacro"/>
+  <xacro:include filename="$(find val_description)/robots/valkyrie_A/xacro/index_finger/joint_axes.xacro"/>
+  <xacro:include filename="$(find val_description)/robots/valkyrie_A/xacro/index_finger/actuator_names.xacro"/>
+  <xacro:include filename="$(find val_description)/robots/valkyrie_A/xacro/index_finger/link_names.xacro"/>
+  <xacro:include filename="$(find val_description)/robots/valkyrie_A/xacro/index_finger/joint_limits.xacro"/>
+  <xacro:include filename="$(find val_description)/robots/valkyrie_A/xacro/index_finger/frame_parameters.xacro"/>
+  <xacro:include filename="$(find val_description)/robots/valkyrie_A/xacro/index_finger/mass_parameters.xacro"/>
   <xacro:property name="PFJ1_Link_Width" value="0.029"/>
   <xacro:property name="PFJ1_Link_Height" value="0.019"/>

File: robots/valkyrie_A/xacro/leg/leg.xacro (robot description, xacro)
@@ -1,11 +1,11 @@
 <?xml version="1.0" ?>
 <robot xmlns:xacro="http://www.ros.org/wiki/xacro" name="v1/leg">
-  <xacro:include filename="$(find valkyrie_description)/robots/valkyrie_A/xacro/leg/joint_names.xacro"/>
-  <xacro:include filename="$(find valkyrie_description)/robots/valkyrie_A/xacro/leg/joint_axes.xacro"/>
-  <xacro:include filename="$(find valkyrie_description)/robots/valkyrie_A/xacro/leg/link_names.xacro"/>
-  <xacro:include filename="$(find valkyrie_description)/robots/valkyrie_A/xacro/leg/joint_limits.xacro"/>
-  <xacro:include filename="$(find valkyrie_description)/robots/valkyrie_A/xacro/leg/frame_parameters.xacro"/>
-  <xacro:include filename="$(find valkyrie_description)/robots/valkyrie_A/xacro/leg/mass_parameters.xacro"/>
-  <xacro:include filename="$(find valkyrie_description)/robots/valkyrie_A/xacro/sensors/ati_force_torque.xacro"/>
+  <xacro:include filename="$(find val_description)/robots/valkyrie_A/xacro/leg/joint_names.xacro"/>
+  <xacro:include filename="$(find val_description)/robots/valkyrie_A/xacro/leg/joint_axes.xacro"/>
+  <xacro:include filename="$(find val_description)/robots/valkyrie_A/xacro/leg/link_names.xacro"/>
+  <xacro:include filename="$(find val_description)/robots/valkyrie_A/xacro/leg/joint_limits.xacro"/>
+  <xacro:include filename="$(find val_description)/robots/valkyrie_A/xacro/leg/frame_parameters.xacro"/>
+  <xacro:include filename="$(find val_description)/robots/valkyrie_A/xacro/leg/mass_parameters.xacro"/>
+  <xacro:include filename="$(find val_description)/robots/valkyrie_A/xacro/sensors/ati_force_torque.xacro"/>
   <xacro:property name="LJ1_Link_Width" value="0.149"/>
   <xacro:property name="LJ1_Link_Height" value="0.185"/>

File: robots/valkyrie_A/xacro/middle_finger/middle_finger.xacro (robot description, xacro)
@@ -1,11 +1,11 @@
 <?xml version="1.0" ?>
 <robot xmlns:xacro="http://www.ros.org/wiki/xacro" name="v1/middle_finger">
-  <xacro:include filename="$(find valkyrie_description)/robots/valkyrie_A/xacro/middle_finger/joint_names.xacro"/>
-  <xacro:include filename="$(find valkyrie_description)/robots/valkyrie_A/xacro/middle_finger/joint_axes.xacro"/>
-  <xacro:include filename="$(find valkyrie_description)/robots/valkyrie_A/xacro/middle_finger/actuator_names.xacro"/>
-  <xacro:include filename="$(find valkyrie_description)/robots/valkyrie_A/xacro/middle_finger/link_names.xacro"/>
-  <xacro:include filename="$(find valkyrie_description)/robots/valkyrie_A/xacro/middle_finger/joint_limits.xacro"/>
-  <xacro:include filename="$(find valkyrie_description)/robots/valkyrie_A/xacro/middle_finger/frame_parameters.xacro"/>
-  <xacro:include filename="$(find valkyrie_description)/robots/valkyrie_A/xacro/middle_finger/mass_parameters.xacro"/>
+  <xacro:include filename="$(find val_description)/robots/valkyrie_A/xacro/middle_finger/joint_names.xacro"/>
+  <xacro:include filename="$(find val_description)/robots/valkyrie_A/xacro/middle_finger/joint_axes.xacro"/>
+  <xacro:include filename="$(find val_description)/robots/valkyrie_A/xacro/middle_finger/actuator_names.xacro"/>
+  <xacro:include filename="$(find val_description)/robots/valkyrie_A/xacro/middle_finger/link_names.xacro"/>
+  <xacro:include filename="$(find val_description)/robots/valkyrie_A/xacro/middle_finger/joint_limits.xacro"/>
+  <xacro:include filename="$(find val_description)/robots/valkyrie_A/xacro/middle_finger/frame_parameters.xacro"/>
+  <xacro:include filename="$(find val_description)/robots/valkyrie_A/xacro/middle_finger/mass_parameters.xacro"/>
   <xacro:property name="MFJ1_Link_Width" value="0.054"/>
   <xacro:property name="MFJ1_Link_Height" value="0.019"/>

File: robots/valkyrie_A/xacro/pinky_finger/pinky_finger.xacro (robot description, xacro)
@@ -1,11 +1,11 @@
 <?xml version="1.0" ?>
 <robot xmlns:xacro="http://www.ros.org/wiki/xacro" name="v1/pinky_finger">
-  <xacro:include filename="$(find valkyrie_description)/robots/valkyrie_A/xacro/pinky_finger/joint_names.xacro"/>
-  <xacro:include filename="$(find valkyrie_description)/robots/valkyrie_A/xacro/pinky_finger/joint_axes.xacro"/>
-  <xacro:include filename="$(find valkyrie_description)/robots/valkyrie_A/xacro/pinky_finger/actuator_names.xacro"/>
-  <xacro:include filename="$(find valkyrie_description)/robots/valkyrie_A/xacro/pinky_finger/link_names.xacro"/>
-  <xacro:include filename="$(find valkyrie_description)/robots/valkyrie_A/xacro/pinky_finger/joint_limits.xacro"/>
-  <xacro:include filename="$(find valkyrie_description)/robots/valkyrie_A/xacro/pinky_finger/frame_parameters.xacro"/>
-  <xacro:include filename="$(find valkyrie_description)/robots/valkyrie_A/xacro/pinky_finger/mass_parameters.xacro"/>
+  <xacro:include filename="$(find val_description)/robots/valkyrie_A/xacro/pinky_finger/joint_names.xacro"/>
+  <xacro:include filename="$(find val_description)/robots/valkyrie_A/xacro/pinky_finger/joint_axes.xacro"/>
+  <xacro:include filename="$(find val_description)/robots/valkyrie_A/xacro/pinky_finger/actuator_names.xacro"/>
+  <xacro:include filename="$(find val_description)/robots/valkyrie_A/xacro/pinky_finger/link_names.xacro"/>
+  <xacro:include filename="$(find val_description)/robots/valkyrie_A/xacro/pinky_finger/joint_limits.xacro"/>
+  <xacro:include filename="$(find val_description)/robots/valkyrie_A/xacro/pinky_finger/frame_parameters.xacro"/>
+  <xacro:include filename="$(find val_description)/robots/valkyrie_A/xacro/pinky_finger/mass_parameters.xacro"/>
   <xacro:property name="LFJ1_Link_Width" value="0.010"/>
   <xacro:property name="LFJ1_Link_Height" value="0.010"/>

File: robots/valkyrie_A/xacro/thumb/thumb.xacro (robot description, xacro)
@@ -1,11 +1,11 @@
 <?xml version="1.0" ?>
 <robot xmlns:xacro="http://www.ros.org/wiki/xacro" name="v1/thumb">
-  <xacro:include filename="$(find valkyrie_description)/robots/valkyrie_A/xacro/thumb/joint_names.xacro"/>
-  <xacro:include filename="$(find valkyrie_description)/robots/valkyrie_A/xacro/thumb/joint_axes.xacro"/>
-  <xacro:include filename="$(find valkyrie_description)/robots/valkyrie_A/xacro/thumb/actuator_names.xacro"/>
-  <xacro:include filename="$(find valkyrie_description)/robots/valkyrie_A/xacro/thumb/link_names.xacro"/>
-  <xacro:include filename="$(find valkyrie_description)/robots/valkyrie_A/xacro/thumb/joint_limits.xacro"/>
-  <xacro:include filename="$(find valkyrie_description)/robots/valkyrie_A/xacro/thumb/frame_parameters.xacro"/>
-  <xacro:include filename="$(find valkyrie_description)/robots/valkyrie_A/xacro/thumb/mass_parameters.xacro"/>
+  <xacro:include filename="$(find val_description)/robots/valkyrie_A/xacro/thumb/joint_names.xacro"/>
+  <xacro:include filename="$(find val_description)/robots/valkyrie_A/xacro/thumb/joint_axes.xacro"/>
+  <xacro:include filename="$(find val_description)/robots/valkyrie_A/xacro/thumb/actuator_names.xacro"/>
+  <xacro:include filename="$(find val_description)/robots/valkyrie_A/xacro/thumb/link_names.xacro"/>
+  <xacro:include filename="$(find val_description)/robots/valkyrie_A/xacro/thumb/joint_limits.xacro"/>
+  <xacro:include filename="$(find val_description)/robots/valkyrie_A/xacro/thumb/frame_parameters.xacro"/>
+  <xacro:include filename="$(find val_description)/robots/valkyrie_A/xacro/thumb/mass_parameters.xacro"/>
   <xacro:property name="TJ1_Link_Width" value="0.010"/>
   <xacro:property name="TJ1_Link_Height" value="0.010"/>

File: robots/valkyrie_A/xacro/valkyrie_A.xacro (robot description, xacro)
@@ -1,5 +1,5 @@
 <robot xmlns:xacro="http://ros.org/wiki/xacro" name="valkyrie">
-    <xacro:property name="mesh_root" value="package://valkyrie_description/meshes"/>
-    <!-- <xacro:include filename="$(find valkyrie_description)/robots/valkyrie_A/xacro/common/hw_actuator_types.xacro"/> -->
-    <xacro:include filename="$(find valkyrie_description)/robots/valkyrie_A/xacro/valkyrie_A_sim_base.xacro"/>
+    <xacro:property name="mesh_root" value="package://val_description/meshes"/>
+    <!-- <xacro:include filename="$(find val_description)/robots/valkyrie_A/xacro/common/hw_actuator_types.xacro"/> -->
+    <xacro:include filename="$(find val_description)/robots/valkyrie_A/xacro/valkyrie_A_sim_base.xacro"/>
 </robot>

File: robots/valkyrie_A/xacro/valkyrie_A_sim_base.xacro (robot description, xacro)
@@ -1,8 +1,8 @@
 <robot xmlns:xacro="http://ros.org/wiki/xacro" name="valkyrie">
     <xacro:include filename="$(find common_xacro)/xacro/generic_models.xacro" />
-    <xacro:include filename="$(find valkyrie_description)/robots/valkyrie_A/xacro/plugins/gazebo_plugins.xacro"/>
+    <xacro:include filename="$(find val_description)/robots/valkyrie_A/xacro/plugins/gazebo_plugins.xacro"/>
     <xacro:include filename="$(find common_xacro)/xacro/materials.xacro" />
-    <xacro:include filename="$(find valkyrie_description)/robots/valkyrie_A/xacro/common/common_bodies.xacro" />
-    <xacro:include filename="$(find valkyrie_description)/robots/valkyrie_A/xacro/common/actuator_names.xacro" />
+    <xacro:include filename="$(find val_description)/robots/valkyrie_A/xacro/common/common_bodies.xacro" />
+    <xacro:include filename="$(find val_description)/robots/valkyrie_A/xacro/common/actuator_names.xacro" />
     <xacro:make_pelvis />
     <xacro:v1_pelvis_sensors/>

File: robots/valkyrie_A/xacro/waist/waist.xacro (robot description, xacro)
@@ -1,13 +1,13 @@
 <robot xmlns:xacro="http://www.ros.org/wiki/xacro" name="v1/waist">
   <!-- Properties -->
-  <xacro:include filename="$(find valkyrie_description)/robots/valkyrie_A/xacro/waist/joint_names.xacro"/>
-  <xacro:include filename="$(find valkyrie_description)/robots/valkyrie_A/xacro/waist/joint_axes.xacro"/>
-  <xacro:include filename="$(find valkyrie_description)/robots/valkyrie_A/xacro/waist/joint_axes.xacro"/>
-  <xacro:include filename="$(find valkyrie_description)/robots/valkyrie_A/xacro/waist/link_names.xacro"/>
-  <xacro:include filename="$(find valkyrie_description)/robots/valkyrie_A/xacro/waist/joint_limits.xacro"/>
-  <xacro:include filename="$(find valkyrie_description)/robots/valkyrie_A/xacro/waist/frame_parameters.xacro"/>
-  <xacro:include filename="$(find valkyrie_description)/robots/valkyrie_A/xacro/waist/mass_parameters.xacro"/>
-  <xacro:include filename="$(find valkyrie_description)/robots/valkyrie_A/xacro/sensors/microstrain.xacro"/>
-  <xacro:include filename="$(find valkyrie_description)/robots/valkyrie_A/xacro/sensors/flea.xacro"/>
+  <xacro:include filename="$(find val_description)/robots/valkyrie_A/xacro/waist/joint_names.xacro"/>
+  <xacro:include filename="$(find val_description)/robots/valkyrie_A/xacro/waist/joint_axes.xacro"/>
+  <xacro:include filename="$(find val_description)/robots/valkyrie_A/xacro/waist/joint_axes.xacro"/>
+  <xacro:include filename="$(find val_description)/robots/valkyrie_A/xacro/waist/link_names.xacro"/>
+  <xacro:include filename="$(find val_description)/robots/valkyrie_A/xacro/waist/joint_limits.xacro"/>
+  <xacro:include filename="$(find val_description)/robots/valkyrie_A/xacro/waist/frame_parameters.xacro"/>
+  <xacro:include filename="$(find val_description)/robots/valkyrie_A/xacro/waist/mass_parameters.xacro"/>
+  <xacro:include filename="$(find val_description)/robots/valkyrie_A/xacro/sensors/microstrain.xacro"/>
+  <xacro:include filename="$(find val_description)/robots/valkyrie_A/xacro/sensors/flea.xacro"/>
   <xacro:property name="Trunk_Width" value="0.47605775481079287692"/>
   <xacro:property name="Trunk_Height" value="0.39817895332782154982"/>
