Commit message: supporting new joint limits and mirroring of joint limit upper and lowers
note that 'reflect' is used selectively to flip the joint upper and lower

File: robots/valkyrie_A/xacro/arm/arm.xacro (robot description, xacro)
@@ -73,5 +73,10 @@
                           axis="${ShoulderRollRotationAxis}"
                           damping="0.1" friction="0.0">
+        <xacro:if value="${(reflect+1)/2}">
         <limit effort="${ShoulderRollTorqueLimit}" lower="${ShoulderRollPositionLimit_Lower}" upper="${ShoulderRollPositionLimit_Upper}" velocity="${ShoulderRollVelocityLimit}"/>
+        </xacro:if>
+        <xacro:if value="${(-reflect+1)/2}">
+        <limit effort="${ShoulderRollTorqueLimit}" lower="${reflect * ShoulderRollPositionLimit_Upper}" upper="${reflect * ShoulderRollPositionLimit_Lower}" velocity="${ShoulderRollVelocityLimit}"/>
+        </xacro:if>
         <controller_gains Kp="20000" Kd="400"/>
     </xacro:revolute_joint_ex>
@@ -93,5 +98,10 @@
                           axis="${ElbowPitchRotationAxis}"
                           damping="0.1" friction="0.0">
+        <xacro:if value="${(reflect+1)/2}">
         <limit effort="${ElbowPitchTorqueLimit}" lower="${ElbowPitchPositionLimit_Lower}" upper="${ElbowPitchPositionLimit_Upper}" velocity="${ElbowPitchVelocityLimit}"/>
+        </xacro:if>
+        <xacro:if value="${(-reflect+1)/2}">
+        <limit effort="${ElbowPitchTorqueLimit}" lower="${reflect * ElbowPitchPositionLimit_Upper}" upper="${reflect * ElbowPitchPositionLimit_Lower}" velocity="${ElbowPitchVelocityLimit}"/>
+        </xacro:if>
         <controller_gains Kp="20000" Kd="400"/>
     </xacro:revolute_joint_ex>
@@ -137,5 +147,10 @@
                           axis="${WristRollRotationAxis}"
                           damping="0.1" friction="0.0">
+        <xacro:if value="${(reflect+1)/2}">
         <limit effort="${WristRollTorqueLimit}" lower="${WristRollPositionLimit_Lower}" upper="${WristRollPositionLimit_Upper}" velocity="${WristRollVelocityLimit}"/>
+        </xacro:if>
+        <xacro:if value="${(-reflect+1)/2}">
+        <limit effort="${WristRollTorqueLimit}" lower="${reflect * WristRollPositionLimit_Upper}" upper="${reflect * WristRollPositionLimit_Lower}" velocity="${WristRollVelocityLimit}"/>
+        </xacro:if>
         <controller_gains Kp="20000" Kd="400"/>
     </xacro:revolute_joint_ex>
@@ -147,5 +162,10 @@
                           axis="${WristPitchRotationAxis}"
                           damping="0.1" friction="0.0">
+        <xacro:if value="${(reflect+1)/2}">
         <limit effort="${WristPitchTorqueLimit}" lower="${WristPitchPositionLimit_Lower}" upper="${WristPitchPositionLimit_Upper}" velocity="${WristPitchVelocityLimit}"/>
+        </xacro:if>
+        <xacro:if value="${(-reflect+1)/2}">
+        <limit effort="${WristRollTorqueLimit}" lower="${reflect * WristPitchPositionLimit_Upper}" upper="${reflect * WristPitchPositionLimit_Lower}" velocity="${WristRollVelocityLimit}"/>
+        </xacro:if>
         <controller_gains Kp="20000" Kd="400"/>
     </xacro:revolute_joint_ex>

File: robots/valkyrie_A/xacro/arm/joint_limits.xacro (robot description, xacro)
@@ -9,17 +9,17 @@
   <xacro:property name="WristPitchTorqueLimit" value="14" />
   <xacro:property name="ShoulderPitchPositionLimit_Lower" value="-3.14" />
-  <xacro:property name="ShoulderRollPositionLimit_Lower" value="-3.05" />
+  <xacro:property name="ShoulderRollPositionLimit_Lower" value="-1.3962" />
   <xacro:property name="ShoulderYawPositionLimit_Lower" value="-1.57" />
   <xacro:property name="ElbowPitchPositionLimit_Lower" value="-1.92" />
-  <xacro:property name="ForearmYawPositionLimit_Lower" value="-2.36" />
-  <xacro:property name="WristRollPositionLimit_Lower" value="-0.873" />
-  <xacro:property name="WristPitchPositionLimit_Lower" value="-0.524" />
+  <xacro:property name="ForearmYawPositionLimit_Lower" value="-0.7853" />
+  <xacro:property name="WristRollPositionLimit_Lower" value="-0.436" />
+  <xacro:property name="WristPitchPositionLimit_Lower" value="-0.873" />
   <xacro:property name="ShoulderPitchPositionLimit_Upper" value="3.14" />
-  <xacro:property name="ShoulderRollPositionLimit_Upper" value="0.155" />
-  <xacro:property name="ShoulderYawPositionLimit_Upper" value="1.7" />
-  <xacro:property name="ElbowPitchPositionLimit_Upper" value="0.087" />
-  <xacro:property name="ForearmYawPositionLimit_Upper" value="2.356" />
-  <xacro:property name="WristRollPositionLimit_Upper" value="0.698" />
-  <xacro:property name="WristPitchPositionLimit_Upper" value="0.436" />
+  <xacro:property name="ShoulderRollPositionLimit_Upper" value="1.4835" />
+  <xacro:property name="ShoulderYawPositionLimit_Upper" value="1.5707" />
+  <xacro:property name="ElbowPitchPositionLimit_Upper" value="-0.087" />
+  <xacro:property name="ForearmYawPositionLimit_Upper" value="3.9269" />
+  <xacro:property name="WristRollPositionLimit_Upper" value="0.524" />
+  <xacro:property name="WristPitchPositionLimit_Upper" value="0.698" />
   <xacro:property name="ShoulderPitchVelocityLimit" value="5.89" />
   <xacro:property name="ShoulderRollVelocityLimit" value="5.89" />

Commit message: corrected parameters

File: robots/valkyrie_A/xacro/arm/arm.xacro (robot description, xacro)
@@ -8,19 +8,19 @@
   <xacro:include filename="$(find val_description)/robots/valkyrie_A/xacro/arm/mass_parameters.xacro"/>
   <xacro:include filename="$(find val_description)/robots/valkyrie_A/xacro/sensors/camboard.xacro"/>
-  <xacro:property name="AJ1_Link_Width" value="0.162"/>
-  <xacro:property name="AJ1_Link_Height" value="0.202"/>
+  <xacro:property name="AJ1_Link_Width" value="0.202"/>
+  <xacro:property name="AJ1_Link_Height" value="0.162"/>
   <xacro:property name="AJ1_Link_Length" value="0.146"/>
   <xacro:property name="AJ2_Link_Width" value="0.22179303376297454520"/>
   <xacro:property name="AJ2_Link_Height" value="0.16373203016010165478"/>
   <xacro:property name="AJ2_Link_Length" value="0.15560348965569942292"/>
-  <xacro:property name="AJ3_Link_Width" value="0.136"/>
-  <xacro:property name="AJ3_Link_Height" value="0.158"/>
-  <xacro:property name="AJ3_Link_Length" value="0.285"/>
+  <xacro:property name="AJ3_Link_Width" value="0.158"/>
+  <xacro:property name="AJ3_Link_Height" value="0.285"/>
+  <xacro:property name="AJ3_Link_Length" value="0.136"/>
   <xacro:property name="AJ4_Link_Width" value="0.11323257841518076516"/>
   <xacro:property name="AJ4_Link_Height" value="0.11855222975004402197"/>
   <xacro:property name="AJ4_Link_Length" value="0.10487312631734664603"/>
   <xacro:property name="AJ5_Link_Width" value="0.13557189311158912570"/>
-  <xacro:property name="AJ5_Link_Height" value="0.11439484172804967321"/>
-  <xacro:property name="AJ5_Link_Length" value="0.25365181285234167374"/>
+  <xacro:property name="AJ5_Link_Height" value="0.25365181285234167374"/>
+  <xacro:property name="AJ5_Link_Length" value="0.11439484172804967321"/>
   <xacro:property name="AJ6_Link_Width" value="0.03"/>
   <xacro:property name="AJ6_Link_Height" value="0.01"/>

File: robots/valkyrie_A/xacro/leg/leg.xacro (robot description, xacro)
@@ -17,19 +17,19 @@
   <xacro:property name="LJ1_Link_Origin_Y" value="2.1764163e-02"/>
   <xacro:property name="LJ1_Link_Origin_Z" value="3.8670367e-02"/> -->
-  <xacro:property name="LJ2_Link_Width" value="0.131"/>
-  <xacro:property name="LJ2_Link_Height" value="0.185"/>
-  <xacro:property name="LJ2_Link_Length" value="0.123"/>
-  <xacro:property name="LJ3_Link_Width" value="0.55419965909040602714"/>
-  <xacro:property name="LJ3_Link_Height" value="0.24253719562602335524"/>
-  <xacro:property name="LJ3_Link_Length" value="0.18520578950459243295"/>
-  <xacro:property name="LJ4_Link_Box_Width" value="0.44528684954574881960"/>
-  <xacro:property name="LJ4_Link_Box_Height" value="0.20288766696230062236"/>
-  <xacro:property name="LJ4_Link_Box_Length" value="0.20551228016178813007"/>
+  <xacro:property name="LJ2_Link_Width" value="0.123"/>
+  <xacro:property name="LJ2_Link_Height" value="0.131"/>
+  <xacro:property name="LJ2_Link_Length" value="0.185"/>
+  <xacro:property name="LJ3_Link_Width" value="0.24253719562602335524"/>
+  <xacro:property name="LJ3_Link_Height" value="0.18520578950459243295"/>
+  <xacro:property name="LJ3_Link_Length" value="0.55419965909040602714"/>
+  <xacro:property name="LJ4_Link_Box_Width" value="0.20288766696230062236"/>
+  <xacro:property name="LJ4_Link_Box_Height" value="0.20551228016178813007"/>
+  <xacro:property name="LJ4_Link_Box_Length" value="0.44528684954574881960"/>
   <xacro:property name="LJ5_Link_Width" value="0.033"/>
   <xacro:property name="LJ5_Link_Height" value="0.076"/>
   <xacro:property name="LJ5_Link_Length" value="0.025"/>
-  <xacro:property name="LJ6_Link_Width" value="0.082"/>
+  <xacro:property name="LJ6_Link_Width" value="0.300"/>
   <xacro:property name="LJ6_Link_Height" value="0.128"/>
-  <xacro:property name="LJ6_Link_Length" value="0.300"/>
+  <xacro:property name="LJ6_Link_Length" value="0.082"/>
   <xacro:macro name="make_leg_links" params="prefix reflect leg_root_link">
     <xacro:box_link name="${HipYawLinkName}"

File: robots/valkyrie_A/xacro/waist/waist.xacro (robot description, xacro)
@@ -10,7 +10,7 @@
   <xacro:include filename="$(find val_description)/robots/valkyrie_A/xacro/sensors/microstrain.xacro"/>
   <xacro:include filename="$(find val_description)/robots/valkyrie_A/xacro/sensors/flea.xacro"/>
-  <xacro:property name="Trunk_Width" value="0.47605775481079287692"/>
+  <xacro:property name="Trunk_Width" value="0.42203731228144558685"/>
   <xacro:property name="Trunk_Height" value="0.39817895332782154982"/>
-  <xacro:property name="Trunk_Length" value="0.42203731228144558685"/>
+  <xacro:property name="Trunk_Length" value="0.47605775481079287692"/>
   <xacro:macro name="make_waist_common" params="waist_root_link">
     <xacro:revolute_joint_ex jointName="${TorsoYawJointName}"

Commit message: Found bug with reflect. For some reason I was under the impression reflect=-1 for left which is incorrect. No clue how long I have had this backwards. I am going through everything trying to find errors. TRUST NOTHINGgit add -A.

File: robots/valkyrie_A/xacro/arm/arm.xacro (robot description, xacro)
@@ -11,7 +11,4 @@
   <xacro:property name="AJ1_Link_Height" value="0.202"/>
   <xacro:property name="AJ1_Link_Length" value="0.146"/>
-  <xacro:property name="AJ2_Link_Width" value="0.22179303376297454520"/>
-  <xacro:property name="AJ2_Link_Height" value="0.16373203016010165478"/>
-  <xacro:property name="AJ2_Link_Length" value="0.15560348965569942292"/>
   <xacro:property name="AJ3_Link_Width" value="0.136"/>
   <xacro:property name="AJ3_Link_Height" value="0.158"/>
@@ -37,7 +34,10 @@
                     material="Gold"
                     collision_mesh="${mesh_root}/arms/aj1_${prefix}.stl" />
-    <xacro:box_link name="${ShoulderRollLinkName}"
-                    width="${AJ2_Link_Width}" height="${AJ2_Link_Height}" depth="${AJ2_Link_Length}" mass="${ShoulderRollLinkMass}"
-                    origin_xyz="${ShoulderRollLinkComPosition}" origin_rpy="0 0 0"
+    <xacro:standard_link name="${ShoulderRollLinkName}"
+                    mass="${ShoulderRollLinkMass}"
+                    origin_xyz="${ShoulderRollLinkComPosition}"
+                    ixx="${ShoulderRollLinkInertia_IXX}" ixy="${ShoulderRollLinkInertia_IXY}" ixz="${ShoulderRollLinkInertia_IXZ}"
+                    iyy="${ShoulderRollLinkInertia_IYY}" iyz="${ShoulderRollLinkInertia_IYZ}" izz="${ShoulderRollLinkInertia_IZZ}"
+                    origin_rpy="0 0 0"
                     visual_mesh="${mesh_root}/arms/aj2_${prefix}.stl"
                     material="White"
@@ -56,5 +56,4 @@
                     material="Gold"
                     collision_mesh="${mesh_root}/arms/aj4_${prefix}.stl" />
-    <!-- AJ1 -->
     <xacro:revolute_joint_ex jointName="${ShoulderPitchJointName}"
                           parent="${upper_arm_root_link}" child="${ShoulderPitchLinkName}"
@@ -66,5 +65,4 @@
         <controller_gains Kp="20000" Kd="400"/>
     </xacro:revolute_joint_ex>
-    <!-- AJ2 -->
     <xacro:revolute_joint_ex jointName="${ShoulderRollJointName}"
                           parent="${ShoulderPitchLinkName}" child="${ShoulderRollLinkName}"
@@ -81,5 +79,4 @@
         <controller_gains Kp="20000" Kd="400"/>
     </xacro:revolute_joint_ex>
-    <!-- AJ3 -->
     <xacro:revolute_joint_ex jointName="${ShoulderYawJointName}"
                           parent="${ShoulderRollLinkName}" child="${ShoulderYawLinkName}"
@@ -91,5 +88,4 @@
         <controller_gains Kp="20000" Kd="400"/>
     </xacro:revolute_joint_ex>
-    <!-- AJ4 -->
     <xacro:revolute_joint_ex jointName="${ElbowPitchJointName}"
                           parent="${ShoulderYawLinkName}" child="${ElbowPitchLinkName}"
@@ -108,5 +104,4 @@
   </xacro:macro>
   <xacro:macro name="make_lower_arm" params="prefix reflect lower_arm_root_link">
-    <!-- LINKS -->
     <xacro:box_link name="${ForearmLinkName}"
                     width="${AJ5_Link_Width}" height="${AJ5_Link_Height}" depth="${AJ5_Link_Length}" mass="${ForearmYawLinkMass}"
@@ -130,5 +125,4 @@
                     material="Gold"
                     collision_mesh="${mesh_root}/arms/palm_${prefix}.stl"/>
-    <!-- AJ5 -->
     <xacro:revolute_joint_ex jointName="${ForearmYawJointName}"
                           parent="${lower_arm_root_link}" child="${ForearmLinkName}"
@@ -155,5 +149,4 @@
         <controller_gains Kp="20000" Kd="400"/>
     </xacro:revolute_joint_ex>
-    <!-- AJ7 -->
     <xacro:revolute_joint_ex jointName="${WristPitchJointName}"
                           parent="${WristRollLinkName}" child="${WristPitchLinkName}"
@@ -175,22 +168,4 @@
     <xacro:make_lower_arm prefix="${prefix}" reflect="${reflect}" lower_arm_root_link="${ElbowPitchLinkName}" />
   </xacro:macro>
-  <!-- Sensors -->
-  <xacro:macro name="v1_right_arm_sensor">
-    <xacro:camboard_sensor sensorName="/v1/RightCamBoard"
-                           parentLink="/v1/RightForearm"
-                           origin_xyz="0.049237 0.006877 -0.250708"
-                           origin_rpy="3.14 1.57 3.14"/>
-  </xacro:macro>
-  <xacro:macro name="v1_left_arm_sensor">
-    <xacro:camboard_sensor sensorName="/v1/LeftCamBoard"
-                           parentLink="/v1/LeftForearm"
-                           origin_xyz="0.045536 -0.0085 0.250708"
-                           origin_rpy="3.14 -1.57 0"/>
-  </xacro:macro>
-  <xacro:macro name="v1_arm_sensors">
-    <xacro:v1_right_arm_sensor />
-    <xacro:v1_left_arm_sensor />
-  </xacro:macro>
-  <!-- Actuators -->
   <xacro:macro name="v1_upper_arm_actuators" params="name1 type1 name2 type2 name3 type3 name4 type4">
     <actuator name="${name1}" type="${type1}"/>

File: robots/valkyrie_A/xacro/arm/mass_parameters.xacro (robot description, xacro)
@@ -4,9 +4,15 @@
   <xacro:property name="ShoulderPitchLinkComPosition" value="-0.012000 ${reflect*0.251000} 0.000000" />
   <xacro:property name="ShoulderRollLinkMass" value="3.970000" />
-  <xacro:property name="ShoulderRollLinkComPosition" value="-0.008513 ${reflect*-0.020680} 0.001088" />
+  <xacro:property name="ShoulderRollLinkComPosition" value="-0.008513 ${reflect*0.020680} 0.001088" />
+  <xacro:property name="ShoulderRollLinkInertia_IXX" value="0.009494119" />
+  <xacro:property name="ShoulderRollLinkInertia_IXY" value="-0.000067294" />
+  <xacro:property name="ShoulderRollLinkInertia_IXZ" value="0.000037177" />
+  <xacro:property name="ShoulderRollLinkInertia_IYY" value="0.007680534" />
+  <xacro:property name="ShoulderRollLinkInertia_IYZ" value="0.000008874" />
+  <xacro:property name="ShoulderRollLinkInertia_IZZ" value="0.011454772" />
   <xacro:property name="ShoulderYawLinkMass" value="3.085000" />
-  <xacro:property name="ShoulderYawLinkComPosition" value="-0.004304	${reflect*-0.209832}	-0.007295" />
+  <xacro:property name="ShoulderYawLinkComPosition" value="-0.004304	${reflect*0.209832}	-0.007295" />
   <xacro:property name="ElbowPitchLinkMass" value="1.830000" />
-  <xacro:property name="ElbowPitchLinkComPosition" value="-0.020344	${reflect*-0.014722} -0.022300" />
+  <xacro:property name="ElbowPitchLinkComPosition" value="-0.020344	${reflect*0.014722} -0.022300" />
   <xacro:property name="ForearmYawLinkMass" value="2.476" />
   <xacro:property name="ForearmYawLinkComPosition" value="0.015000	${reflect*0.110000} 0.019564" />

File: robots/valkyrie_A/xacro/leg/mass_parameters.xacro (robot description, xacro)
@@ -4,5 +4,5 @@
   <xacro:property name="HipYawLinkComPosition" value="0.02176 ${reflect*-0.00131} 0.03867" />
   <xacro:property name="HipRollLinkMass" value="3.665000" />
-  <xacro:property name="HipRollLinkComPosition" value="0.012959 ${reflect*-0.007550} -0.015950" />
+  <xacro:property name="HipRollLinkComPosition" value="0.012959 ${reflect*0.007550} -0.015950" />
   <xacro:property name="HipRollLinkInertia_IXX" value="0.005978962" />
   <xacro:property name="HipRollLinkInertia_IXY" value="${reflect*0.000234823}" />
@@ -12,5 +12,5 @@
   <xacro:property name="HipRollLinkInertia_IZZ" value="0.008193117" />
   <xacro:property name="HipPitchLinkMass" value="10.20" />
-  <xacro:property name="HipPitchLinkComPosition" value="0.016691 ${reflect*-0.091397} -0.207875" />
+  <xacro:property name="HipPitchLinkComPosition" value="0.016691 ${reflect*0.091397} -0.207875" />
   <xacro:property name="HipPitchLinkInertia_IXX" value="0.240834130" />
   <xacro:property name="HipPitchLinkInertia_IXY" value="${reflect*-0.000035915}" />
@@ -20,5 +20,5 @@
   <xacro:property name="HipPitchLinkInertia_IZZ" value="0.023276352" />
   <xacro:property name="KneePitchLinkMass" value="6.600000" />
-  <xacro:property name="KneePitchLinkComPosition" value="0.002425 ${reflect*-0.001543} -0.189511" />
+  <xacro:property name="KneePitchLinkComPosition" value="0.002425 -0.001543 -0.189511" />
   <xacro:property name="KneePitchLinkInertia_IXX" value="0.096117529" />
   <xacro:property name="KneePitchLinkInertia_IXY" value="0.000107885" />
@@ -28,5 +28,5 @@
   <xacro:property name="KneePitchLinkInertia_IZZ" value="0.013722874" />
   <xacro:property name="AnklePitchLinkMass" value="0.06" />
-  <xacro:property name="AnklePitchLinkComPosition" value="-0.001269 ${reflect*0.00009} -0.006013" />
+  <xacro:property name="AnklePitchLinkComPosition" value="-0.001269 0.00009} -0.006013" />
   <xacro:property name="AnklePitchLinkInertia_IXX" value="0.000011226" />
   <xacro:property name="AnklePitchLinkInertia_IXY" value="0.000000000" />
@@ -36,5 +36,5 @@
   <xacro:property name="AnklePitchLinkInertia_IZZ" value="0.000018792" />
   <xacro:property name="FootMass" value="3.2550" />
-  <xacro:property name="FootComPosition" value="0.040004 ${reflect*-0.00381} -0.049558" />
+  <xacro:property name="FootComPosition" value="0.040004 -0.00381 -0.049558" />
   <xacro:property name="FootInertia_IXX" value="0.008966273" />
   <xacro:property name="FootInertia_IXY" value="-0.000086029" />
