Commit message: Updated palm inertia.

File: robots/valkyrie_A/xacro/arm/arm.xacro (robot description, xacro)
@@ -10,13 +10,4 @@
   <xacro:property name="AJ1_Link_Height" value="0.202"/>
   <xacro:property name="AJ1_Link_Length" value="0.146"/>
-  <xacro:property name="AJ3_Link_Width" value="0.136"/>
-  <xacro:property name="AJ3_Link_Height" value="0.158"/>
-  <xacro:property name="AJ3_Link_Length" value="0.285"/>
-  <xacro:property name="AJ4_Link_Width" value="0.11323257841518076516"/>
-  <xacro:property name="AJ4_Link_Height" value="0.11855222975004402197"/>
-  <xacro:property name="AJ4_Link_Length" value="0.10487312631734664603"/>
-  <xacro:property name="AJ5_Link_Width" value="0.13557189311158912570"/>
-  <xacro:property name="AJ5_Link_Height" value="0.11439484172804967321"/>
-  <xacro:property name="AJ5_Link_Length" value="0.25365181285234167374"/>
   <xacro:property name="AJ6_Link_Width" value="0.03"/>
   <xacro:property name="AJ6_Link_Height" value="0.01"/>
@@ -41,13 +32,18 @@
                     material="White"
                     collision_mesh="${mesh_root}/arms/aj2_${prefix}.dae" />
-    <xacro:box_link name="${ShoulderYawLinkName}"
-                    width="${AJ3_Link_Width}" height="${AJ3_Link_Height}" depth="${AJ3_Link_Length}" mass="${ShoulderYawLinkMass}"
-                    origin_xyz="${ShoulderYawLinkComPosition}" origin_rpy="0 0 0"
+    <xacro:standard_link name="${ShoulderYawLinkName}"
+                    mass="${ShoulderYawLinkMass}"
+                    origin_xyz="${ShoulderYawLinkComPosition}"
+                    ixx="${ShoulderYawLinkInertia_IXX}" ixy="${ShoulderYawLinkInertia_IXY}" ixz="${ShoulderYawLinkInertia_IXZ}"
+                    iyy="${ShoulderYawLinkInertia_IYY}" iyz="${ShoulderYawLinkInertia_IYZ}" izz="${ShoulderYawLinkInertia_IZZ}"
+                    origin_rpy="0 0 0"
                     visual_mesh="${mesh_root}/arms/aj3_${prefix}.dae"
                     material="White"
                     collision_mesh="${mesh_root}/arms/aj3_${prefix}.dae" />
-    <xacro:box_link name="${ElbowPitchLinkName}"
-                    width="${AJ4_Link_Width}" height="${AJ4_Link_Height}" depth="${AJ4_Link_Length}" mass="${ElbowPitchLinkMass}"
+    <xacro:standard_link name="${ElbowPitchLinkName}"
+                    mass="${ElbowPitchLinkMass}"
                     origin_xyz="${ElbowPitchLinkComPosition}"
+                    ixx="${ElbowPitchLinkInertia_IXX}" ixy="${ElbowPitchLinkInertia_IXY}" ixz="${ElbowPitchLinkInertia_IXZ}"
+                    iyy="${ElbowPitchLinkInertia_IYY}" iyz="${ElbowPitchLinkInertia_IYZ}" izz="${ElbowPitchLinkInertia_IZZ}"
                     origin_rpy="0 0 0"
                     visual_mesh="${mesh_root}/arms/aj4_${prefix}.dae"
@@ -102,21 +98,27 @@
   </xacro:macro>
   <xacro:macro name="make_lower_arm" params="prefix reflect lower_arm_root_link">
-    <xacro:box_link name="${ForearmLinkName}"
-                    width="${AJ5_Link_Width}" height="${AJ5_Link_Height}" depth="${AJ5_Link_Length}" mass="${ForearmYawLinkMass}"
+    <xacro:standard_link name="${ForearmLinkName}"
+                    mass="${ForearmYawLinkMass}"
                     origin_xyz="${ForearmYawLinkComPosition}"
+                    ixx="${ForearmYawLinkInertia_IXX}" ixy="${ForearmYawLinkInertia_IXY}" ixz="${ForearmYawLinkInertia_IXZ}"
+                    iyy="${ForearmYawLinkInertia_IYY}" iyz="${ForearmYawLinkInertia_IYZ}" izz="${ForearmYawLinkInertia_IZZ}"
                     origin_rpy="0 0 0"
                     visual_mesh="${mesh_root}/arms/aj5_${prefix}.dae"
                     material="White"
                     collision_mesh="${mesh_root}/arms/aj5_${prefix}.dae" />
-    <xacro:box_link name="${WristRollLinkName}"
-                    width="${AJ6_Link_Width}" height="${AJ6_Link_Height}" depth="${AJ6_Link_Length}" mass="${WristRollLinkMass}"
+    <xacro:standard_link name="${WristRollLinkName}"
+                    mass="${WristRollLinkMass}"
                     origin_xyz="${WristRollLinkComPosition}"
+                    ixx="${WristRollLinkInertia_IXX}" ixy="${WristRollLinkInertia_IXY}" ixz="${WristRollLinkInertia_IXZ}"
+                    iyy="${WristRollLinkInertia_IYY}" iyz="${WristRollLinkInertia_IYZ}" izz="${WristRollLinkInertia_IZZ}"
                     origin_rpy="0 0 0"
                     visual_mesh="${mesh_root}/arms/aj6_${prefix}.dae"
                     material="White"
                     collision_mesh="${mesh_root}/arms/aj6_${prefix}.dae" />
-    <xacro:box_link name="${WristPitchLinkName}"
-                    width="${AJ7_Link_Width}" height="${AJ7_Link_Height}" depth="${AJ7_Link_Length}" mass="${PalmMass}"
+    <xacro:standard_link name="${WristPitchLinkName}"
+                    mass="${PalmMass}"
                     origin_xyz="${PalmComPosition}"
+                    ixx="${PalmInertia_IXX}" ixy="${PalmInertia_IXY}" ixz="${PalmInertia_IXZ}"
+                    iyy="${PalmInertia_IYY}" iyz="${PalmInertia_IYZ}" izz="${PalmInertia_IZZ}"
                     origin_rpy="0 0 0"
                     visual_mesh="${mesh_root}/arms/palm_${prefix}.dae"

File: robots/valkyrie_A/xacro/arm/mass_parameters.xacro (robot description, xacro)
@@ -28,8 +28,26 @@
   <xacro:property name="ElbowPitchLinkInertia_IZZ" value="0.007469454" />
   <xacro:property name="ForearmYawLinkMass" value="2.476" />
-  <xacro:property name="ForearmYawLinkComPosition" value="0.015000	${reflect*0.110000} 0.019564" />
+  <xacro:property name="ForearmYawLinkComPosition" value="0.015000	${reflect*0.13} 0.019564" />
+  <xacro:property name="ForearmYawLinkInertia_IXX" value="0.015011" />
+  <xacro:property name="ForearmYawLinkInertia_IXY" value="${reflect*0.001300853}" />
+  <xacro:property name="ForearmYawLinkInertia_IXZ" value="${reflect*0.000727141}" />
+  <xacro:property name="ForearmYawLinkInertia_IYY" value="0.005071567" />
+  <xacro:property name="ForearmYawLinkInertia_IYZ" value="-0.001695416" />
+  <xacro:property name="ForearmYawLinkInertia_IZZ" value="0.011365657" />
   <xacro:property name="WristRollLinkMass" value="0.14" />
   <xacro:property name="WristRollLinkComPosition" value="0 ${reflect*0} 0" />
+  <xacro:property name="WristRollLinkInertia_IXX" value="0.000030251" />
+  <xacro:property name="WristRollLinkInertia_IXY" value="${reflect*0.000000125}" />
+  <xacro:property name="WristRollLinkInertia_IXZ" value="${reflect*0.000000036}" />
+  <xacro:property name="WristRollLinkInertia_IYY" value="0.000037720" />
+  <xacro:property name="WristRollLinkInertia_IYZ" value="0.0" />
+  <xacro:property name="WristRollLinkInertia_IZZ" value="0.000009395" />
   <xacro:property name="PalmMass" value="0.712" />
   <xacro:property name="PalmComPosition" value="0.002954 ${reflect*0.052034} -0.000236" />
+  <xacro:property name="PalmInertia_IXX" value="0.000943493" />
+  <xacro:property name="PalmInertia_IXY" value="0.000034393" />
+  <xacro:property name="PalmInertia_IXZ" value="${reflect*0.000038828}" />
+  <xacro:property name="PalmInertia_IYY" value="0.000711024" />
+  <xacro:property name="PalmInertia_IYZ" value="${reflect*-0.000023429}" />
+  <xacro:property name="PalmInertia_IZZ" value="0.000610199" />
 </robot>

Commit message: Updated link inertias for fingers, neck, and converted J1's to standard links rather than box links.

File: robots/valkyrie_A/xacro/arm/arm.xacro (robot description, xacro)
@@ -7,17 +7,10 @@
   <xacro:include filename="$(find val_description)/robots/valkyrie_A/xacro/arm/frame_parameters.xacro"/>
   <xacro:include filename="$(find val_description)/robots/valkyrie_A/xacro/arm/mass_parameters.xacro"/>
-  <xacro:property name="AJ1_Link_Width" value="0.162"/>
-  <xacro:property name="AJ1_Link_Height" value="0.202"/>
-  <xacro:property name="AJ1_Link_Length" value="0.146"/>
-  <xacro:property name="AJ6_Link_Width" value="0.03"/>
-  <xacro:property name="AJ6_Link_Height" value="0.01"/>
-  <xacro:property name="AJ6_Link_Length" value="0.051"/>
-  <xacro:property name="AJ7_Link_Width" value="0.085"/>
-  <xacro:property name="AJ7_Link_Height" value="0.1"/>
-  <xacro:property name="AJ7_Link_Length" value="0.038"/>
   <xacro:macro name="make_upper_arm" params="prefix reflect upper_arm_root_link">
-    <xacro:box_link name="${ShoulderPitchLinkName}"
-                    width="${AJ1_Link_Width}" height="${AJ1_Link_Height}" depth="${AJ1_Link_Length}" mass="${ShoulderPitchLinkMass}"
+    <xacro:standard_link name="${ShoulderPitchLinkName}"
+                    mass="${ShoulderPitchLinkMass}"
                     origin_xyz="${ShoulderPitchLinkComPosition}" origin_rpy="0 0 0"
+                    ixx="${ShoulderPitchLinkInertia_IXX}" ixy="${ShoulderPitchLinkInertia_IXY}" ixz="${ShoulderPitchLinkInertia_IXZ}"
+                    iyy="${ShoulderPitchLinkInertia_IYY}" iyz="${ShoulderPitchLinkInertia_IYZ}" izz="${ShoulderPitchLinkInertia_IZZ}"
                     visual_mesh="${mesh_root}/arms/aj1_${prefix}.dae"
                     material="Gold"

File: robots/valkyrie_A/xacro/arm/mass_parameters.xacro (robot description, xacro)
@@ -3,4 +3,10 @@
   <xacro:property name="ShoulderPitchLinkMass" value="2.65" />
   <xacro:property name="ShoulderPitchLinkComPosition" value="-0.012000 ${reflect*0.251000} 0.000000" />
+  <xacro:property name="ShoulderPitchLinkInertia_IXX" value="0.013718167" />
+  <xacro:property name="ShoulderPitchLinkInertia_IXY" value="0.000000000" />
+  <xacro:property name="ShoulderPitchLinkInertia_IXZ" value="0.000000000" />
+  <xacro:property name="ShoulderPitchLinkInertia_IYY" value="0.010502833" />
+  <xacro:property name="ShoulderPitchLinkInertia_IYZ" value="0.000000000" />
+  <xacro:property name="ShoulderPitchLinkInertia_IZZ" value="0.014806433" />
   <xacro:property name="ShoulderRollLinkMass" value="3.970000" />
   <xacro:property name="ShoulderRollLinkComPosition" value="-0.008513 ${reflect*0.020680} 0.001088" />

File: robots/valkyrie_A/xacro/thumb/thumb.xacro (robot description, xacro)
@@ -89,50 +89,4 @@
     </xacro:revolute_joint>
   </xacro:macro>
-  <xacro:macro name="make_thumb_fixed" params="prefix reflect thumb_root_link">
-    <xacro:box_link name="${ThumbRollLinkName}"
-                    width="${TJ1_Link_Width}" height="${TJ1_Link_Height}" depth="${TJ1_Link_Length}" mass="${ThumbRollLinkMass}"
-                    origin_rpy="0 0 0"
-                    origin_xyz="${TJ1_Link_Origin_X} ${TJ1_Link_Origin_Y} ${TJ1_Link_Origin_Z}"
-                    visual_mesh="${mesh_root}/fingers/tf1_${prefix}.dae"
-                    material="Gold"
-                    collision_mesh="${mesh_root}/fingers/tf1_${prefix}.dae"/>
-    <xacro:box_link name="${ThumbPitch1LinkName}"
-                    width="${TJ2_Link_Width}" height="${TJ2_Link_Height}" depth="${TJ2_Link_Length}" mass="${ThumbPitch1LinkMass}"
-                    origin_rpy="0 0 0"
-                    origin_xyz="${TJ2_Link_Origin_X} ${TJ2_Link_Origin_Y} ${TJ2_Link_Origin_Z}"
-                    visual_mesh="${mesh_root}/fingers/tf2.dae"
-                    material="Gold"
-                    collision_mesh="${mesh_root}/fingers/tf2.dae"/>
-    <xacro:box_link name="${ThumbPitch2LinkName}"
-                    width="${TJ3_Link_Width}" height="${TJ3_Link_Height}" depth="${TJ3_Link_Length}" mass="${ThumbPitch2LinkMass}"
-                    origin_rpy="0 0 0"
-                    origin_xyz="${TJ3_Link_Origin_X} ${TJ3_Link_Origin_Y} ${TJ3_Link_Origin_Z}"
-                    visual_mesh="${mesh_root}/fingers/tf3.dae"
-                    material="Gold"
-                    collision_mesh="${mesh_root}/fingers/tf3.dae"/>
-    <xacro:box_link name="${ThumbPitch3LinkName}"
-                    width="${TJ4_Link_Width}" height="${TJ4_Link_Height}" depth="${TJ4_Link_Length}" mass="${ThumbPitch3LinkMass}"
-                    origin_rpy="0 0 0"
-                    origin_xyz="${TJ4_Link_Origin_X} ${TJ4_Link_Origin_Y} ${TJ4_Link_Origin_Z}"
-                    visual_mesh="${mesh_root}/fingers/tf4.dae"
-                    material="Gold"
-                    collision_mesh="${mesh_root}/fingers/tf4.dae"/>
-    <xacro:fixed_joint jointName="${ThumbRollJointName}"
-                          parent="${ThumbRollParentLinkName}" child="${ThumbRollLinkName}"
-                          origin_xyz="${ThumbRollFrameOrigin_X} ${ThumbRollFrameOrigin_Y} ${ThumbRollFrameOrigin_Z}"
-                          origin_rpy="${ThumbRollFrameOrientation_Roll} ${ThumbRollFrameOrientation_Pitch} ${ThumbRollFrameOrientation_Yaw}"/>
-    <xacro:fixed_joint jointName="${ThumbPitch1JointName}"
-                          parent="${ThumbRollLinkName}" child="${ThumbPitch1LinkName}"
-                          origin_xyz="${ThumbPitch1FrameOrigin_X} ${ThumbPitch1FrameOrigin_Y} ${ThumbPitch1FrameOrigin_Z}"
-                          origin_rpy="${ThumbPitch1FrameOrientation_Roll} ${ThumbPitch1FrameOrientation_Pitch} ${ThumbPitch1FrameOrientation_Yaw}"/>
-    <xacro:fixed_joint jointName="${ThumbPitch2JointName}"
-                          parent="${ThumbPitch1LinkName}" child="${ThumbPitch2LinkName}"
-                          origin_xyz="${ThumbPitch2FrameOrigin_X} ${ThumbPitch2FrameOrigin_Y} ${ThumbPitch2FrameOrigin_Z}"
-                          origin_rpy="${ThumbPitch2FrameOrientation_Roll} ${ThumbPitch2FrameOrientation_Pitch} ${ThumbPitch2FrameOrientation_Yaw}"/>
-    <xacro:fixed_joint jointName="${ThumbPitch3JointName}"
-                          parent="${ThumbPitch2LinkName}" child="${ThumbPitch3LinkName}"
-                          origin_xyz="${ThumbPitch3FrameOrigin_X} ${ThumbPitch3FrameOrigin_Y} ${ThumbPitch3FrameOrigin_Z}"
-                          origin_rpy="${ThumbPitch3FrameOrientation_Roll} ${ThumbPitch3FrameOrientation_Pitch} ${ThumbPitch3FrameOrientation_Yaw}"/>
-  </xacro:macro>
   <xacro:macro name="right_thumb_actuators" params="prefix api">
     <xacro:v1_actuator name="${RTA1_Actuator_Name}" api="${api}" />

File: robots/valkyrie_A/xacro/waist/mass_parameters.xacro (robot description, xacro)
@@ -1,8 +1,20 @@
 <?xml version="1.0" ?>
 <robot xmlns:xacro="http://www.ros.org/wiki/xacro" name="v1/waist/mass_parameters">
-	<xacro:property name="TorsoYawLinkMass" value="2.858" />
-	<xacro:property name="TorsoYawLinkComPosition" value="0.0 0.0 0.0" />
-	<xacro:property name="TorsoPitchLinkMass" value="0.001"/>
-	<xacro:property name="TorsoPitchLinkComPosition" value="0.0 0.0 0.0" />
+	<xacro:property name="TorsoYawLinkMass" value="0.5" />
+  <xacro:property name="TorsoYawLinkComPosition" value="0.000000 0.000000 -0.010000"/>
+  <xacro:property name="TorsoYawLinkInertia_IXX" value="0.000608427" />
+  <xacro:property name="TorsoYawLinkInertia_IXY" value="-0.000001172" />
+  <xacro:property name="TorsoYawLinkInertia_IXZ" value="0.000001647" />
+  <xacro:property name="TorsoYawLinkInertia_IYY" value="0.000620328" />
+  <xacro:property name="TorsoYawLinkInertia_IYZ" value="-0.000000233" />
+  <xacro:property name="TorsoYawLinkInertia_IZZ" value="0.001078108" />
+	<xacro:property name="TorsoPitchLinkMass" value="0.1"/>
+  <xacro:property name="TorsoPitchLinkComPosition" value="0.000000 0.000000  0.005000" />
+  <xacro:property name="TorsoPitchLinkInertia_IXX" value="0.000030320" />
+  <xacro:property name="TorsoPitchLinkInertia_IXY" value="0.000000000" />
+  <xacro:property name="TorsoPitchLinkInertia_IXZ" value="-0.000001145" />
+  <xacro:property name="TorsoPitchLinkInertia_IYY" value="0.000021274" />
+  <xacro:property name="TorsoPitchLinkInertia_IYZ" value="0.000000000" />
+  <xacro:property name="TorsoPitchLinkInertia_IZZ" value="0.000028285" />
   <xacro:property name="TorsoRollLinkMass" value="39.470000" />
   <xacro:property name="TorsoRollLinkComPosition" value="-0.178048 0.012293 0.238350" />
