Commit message: Removed a bunch of sensor xacros for sensors that no longer exist on the robot. Added some gazebo tags for sdf.

File: robots/common/sensors/microstrain.xacro (robot description, xacro)
@@ -1,4 +1,4 @@
 <?xml version="1.0" ?>
-<robot xmlns:xacro="http://www.ros.org/wiki/xacro" name="v1/microstrain">
+<robot xmlns:xacro="http://www.ros.org/wiki/xacro" name="microstrain">
   <xacro:property name="MicrostrainWidth" value="0.024"/>
   <xacro:property name="MicrostrainHeight" value="0.044"/>

File: robots/common/sensors/multisense_sl.xacro (robot description, xacro)
@@ -2,5 +2,4 @@
 <robot xmlns:xacro="http://www.ros.org/wiki/xacro" name="multisense_sl">
   <xacro:macro name="multisense_sl" params="parentLink joint_axis joint_origin_xyz joint_origin_rpy com_origin_xyz com_origin_rpy mass visual_mesh material collision_mesh">
-    	 	<!-- params="name mass origin_rpy origin_xyz ixx ixy ixz iyy iyz izz visual_mesh material collision_mesh" -->
     	<xacro:continuous_joint jointName="MultisenseSLSpinnyJointFrame"
                           parent="${parentLink}" child="hokuyo_link"
@@ -14,7 +13,14 @@
 		    	  collision_mesh="${collision_mesh}"
 		    	  />
-      <gazebo reference="hokuyo_link">
+		  <xacro:fixed_joint jointName="head_hokuyo_frame_joint"
+	           parent="hokuyo_link" child="head_hokuyo_frame_offset"
+	           origin_rpy="3.14 0.0 0.0"
+	           origin_xyz="0.16018 0.0 -0.015"/>
+      <xacro:massless_virtual_link name="head_hokuyo_frame_offset"
+                    origin_rpy="0 0 0"
+                    origin_xyz="0 0 0"/>
+      <gazebo reference="head_hokuyo_frame_offset">
         <sensor type="ray" name="head_hokuyo_sensor">
-          <parent>hokuyo_link</parent>
+          <parent>head_hokuyo_frame_offset</parent>
           <pose>0 0 0 0 0 0</pose>
           <visualize>false</visualize>
@@ -42,25 +48,32 @@
         </sensor>
       </gazebo>
-	    <xacro:massless_virtual_link name="head_hokuyo_frame_offset"
-                    origin_rpy="0 0 0"
-                    origin_xyz="0 0 0"/>
-		  <xacro:fixed_joint jointName="head_hokuyo_frame_joint"
-	           parent="hokuyo_link" child="head_hokuyo_frame_offset"
-	           origin_rpy="3.14 0.0 0.0"
-	           origin_xyz="0.16018 0.0 -0.015"/>
-      <xacro:massless_virtual_link name="left_camera_frame_offset"
-                    origin_rpy="0 0 0"
-                    origin_xyz="0 0 0"/>
       <xacro:fixed_joint jointName="left_camera_frame_joint"
          parent="${parentLink}" child="left_camera_frame_offset"
          origin_rpy="-3.14 0.1309 0.0"
        	 origin_xyz="0.18335 0.035 0.0774"/>
+      <xacro:massless_virtual_link name="left_camera_frame_offset"
+                    origin_rpy="0 0 0"
+                    origin_xyz="0 0 0"/>
+      <gazebo reference="left_camera_frame_offset">
+        <sensor type="camera" name="multisense_left_camera">
+          <parent>left_camera_frame_offset</parent>
+          <pose>0 0 0 0 0 0</pose>
+          <visualize>false</visualize>
+        </sensor>
+      </gazebo>
+      <xacro:fixed_joint jointName="right_camera_frame_joint"
+         parent="${parentLink}" child="right_camera_frame_offset"
+         origin_rpy="-3.14 0.1309 0.0"
+         origin_xyz="0.18335 -0.035 0.0774"/>
      	<xacro:massless_virtual_link name="right_camera_frame_offset"
                     origin_rpy="0 0 0"
                     origin_xyz="0 0 0"/>
-       	<xacro:fixed_joint jointName="right_camera_frame_joint"
-         parent="${parentLink}" child="right_camera_frame_offset"
-         origin_rpy="-3.14 0.1309 0.0"
-         origin_xyz="0.18335 -0.035 0.0774"/>
+      <gazebo reference="right_camera_frame_offset">
+        <sensor type="camera" name="multisense_right_camera">
+          <parent>right_camera_frame_offset</parent>
+          <pose>0 0 0 0 0 0</pose>
+          <visualize>false</visualize>
+        </sensor>
+      </gazebo>
   </xacro:macro>
 </robot>

File: robots/valkyrie_A/xacro/arm/arm.xacro (robot description, xacro)
@@ -7,5 +7,4 @@
   <xacro:include filename="$(find val_description)/robots/valkyrie_A/xacro/arm/frame_parameters.xacro"/>
   <xacro:include filename="$(find val_description)/robots/valkyrie_A/xacro/arm/mass_parameters.xacro"/>
-  <xacro:include filename="$(find val_description)/robots/valkyrie_A/xacro/sensors/camboard.xacro"/>
   <xacro:property name="AJ1_Link_Width" value="0.162"/>
   <xacro:property name="AJ1_Link_Height" value="0.202"/>
@@ -175,21 +174,4 @@
     <xacro:make_lower_arm prefix="${prefix}" reflect="${reflect}" lower_arm_root_link="${ElbowPitchLinkName}" />
   </xacro:macro>
-  <!-- Sensors -->
-  <xacro:macro name="v1_right_arm_sensor">
-    <xacro:camboard_sensor sensorName="/v1/RightCamBoard"
-                           parentLink="/v1/RightForearm"
-                           origin_xyz="0.049237 0.006877 -0.250708"
-                           origin_rpy="3.14 1.57 3.14"/>
-  </xacro:macro>
-  <xacro:macro name="v1_left_arm_sensor">
-    <xacro:camboard_sensor sensorName="/v1/LeftCamBoard"
-                           parentLink="/v1/LeftForearm"
-                           origin_xyz="0.045536 -0.0085 0.250708"
-                           origin_rpy="3.14 -1.57 0"/>
-  </xacro:macro>
-  <xacro:macro name="v1_arm_sensors">
-    <xacro:v1_right_arm_sensor />
-    <xacro:v1_left_arm_sensor />
-  </xacro:macro>
   <!-- Actuators -->
   <xacro:macro name="v1_upper_arm_actuators" params="name1 type1 name2 type2 name3 type3 name4 type4">

File: robots/valkyrie_A/xacro/common/common_bodies.xacro (robot description, xacro)
@@ -1,3 +1,3 @@
-<robot xmlns:xacro="http://ros.orgt/wiki/xacro" name="v1/common_bodies">
+<robot xmlns:xacro="http://ros.orgt/wiki/xacro" name="common_bodies">
     <xacro:include filename="$(find val_description)/robots/valkyrie_A/xacro/pelvis/pelvis.xacro" />
     <xacro:include filename="$(find val_description)/robots/valkyrie_A/xacro/waist/waist.xacro" />

File: robots/valkyrie_A/xacro/head/head.xacro (robot description, xacro)
@@ -6,5 +6,5 @@
   <xacro:include filename="$(find val_description)/robots/valkyrie_A/xacro/head/frame_parameters.xacro"/>
   <xacro:include filename="$(find val_description)/robots/valkyrie_A/xacro/head/mass_parameters.xacro"/>
-  <xacro:include filename="$(find val_description)/robots/valkyrie_A/xacro/sensors/multisense_sl.xacro"/>
+  <xacro:include filename="$(find val_description)/robots/common/sensors/multisense_sl.xacro"/>
   <xacro:property name="NJ3_Link_Radius" value="0.139"/>
   <xacro:macro name="include_head" params="lower_neck_pitch_root_link">

File: robots/valkyrie_A/xacro/leg/leg.xacro (robot description, xacro)
@@ -7,5 +7,5 @@
   <xacro:include filename="$(find val_description)/robots/valkyrie_A/xacro/leg/frame_parameters.xacro"/>
   <xacro:include filename="$(find val_description)/robots/valkyrie_A/xacro/leg/mass_parameters.xacro"/>
-  <xacro:include filename="$(find val_description)/robots/valkyrie_A/xacro/sensors/ati_force_torque.xacro"/>
+  <xacro:include filename="$(find val_description)/robots/common/sensors/ati_force_torque.xacro"/>
   <xacro:property name="LJ1_Link_Width" value="0.149"/>
   <xacro:property name="LJ1_Link_Height" value="0.185"/>

File: robots/valkyrie_A/xacro/waist/waist.xacro (robot description, xacro)
@@ -1,3 +1,3 @@
-<robot xmlns:xacro="http://www.ros.org/wiki/xacro" name="v1/waist">
+<robot xmlns:xacro="http://www.ros.org/wiki/xacro" name="waist">
   <!-- Properties -->
   <xacro:include filename="$(find val_description)/robots/valkyrie_A/xacro/waist/joint_names.xacro"/>
@@ -8,6 +8,6 @@
   <xacro:include filename="$(find val_description)/robots/valkyrie_A/xacro/waist/frame_parameters.xacro"/>
   <xacro:include filename="$(find val_description)/robots/valkyrie_A/xacro/waist/mass_parameters.xacro"/>
-  <xacro:include filename="$(find val_description)/robots/valkyrie_A/xacro/sensors/microstrain.xacro"/>
-  <xacro:include filename="$(find val_description)/robots/valkyrie_A/xacro/sensors/flea.xacro"/>
+  <xacro:include filename="$(find val_description)/robots/common/sensors/microstrain.xacro"/>
+  <xacro:include filename="$(find val_description)/robots/common/sensors/flea.xacro"/>
   <xacro:property name="Trunk_Width" value="0.47605775481079287692"/>
   <xacro:property name="Trunk_Height" value="0.39817895332782154982"/>
