Commit message: Removed some invalid tags.

File: robots/common/sensors/ati_force_torque.xacro (robot description, xacro)
@@ -11,5 +11,4 @@
     <gazebo reference="${sensorName}_Frame">
       <sensor name="${sensorName}" type="force_torque">
-        <parent link="${parentLink}"/>
         <pose>${origin_xyz} ${origin_rpy} </pose>
     	</sensor>

File: robots/common/sensors/microstrain.xacro (robot description, xacro)
@@ -15,5 +15,4 @@
     <gazebo reference="${sensorName}_Frame">
       <sensor name="${sensorName}" type="imu">
-        <parent link="${parentLink}"/>
         <pose>${origin_xyz} ${origin_rpy} </pose>
         <imu>

Commit message: Fixed sensor tag for force/torque sensor.

File: robots/common/sensors/ati_force_torque.xacro (robot description, xacro)
@@ -9,7 +9,7 @@
                        origin_rpy="${origin_rpy}"
                        origin_xyz="${origin_xyz}"/>
-    <gazebo reference="${sensorName}_Frame">
+    <gazebo reference="${sensorName}_Offset">
       <sensor name="${sensorName}" type="force_torque">
-        <pose>${origin_xyz} ${origin_rpy} </pose>
+        <frame>child</frame>
     	</sensor>
     </gazebo>

File: robots/common/sensors/multisense_sl.xacro (robot description, xacro)
@@ -22,5 +22,4 @@
       <gazebo reference="head_hokuyo_frame_offset">
         <sensor type="ray" name="head_hokuyo_sensor">
-          <parent>head_hokuyo_frame_offset</parent>
           <pose>0 0 0 0 0 0</pose>
           <visualize>false</visualize>
@@ -57,5 +56,4 @@
       <gazebo reference="left_camera_frame_offset">
         <sensor type="camera" name="multisense_left_camera">
-          <parent>left_camera_frame_offset</parent>
           <pose>0 0 0 0 0 0</pose>
           <visualize>false</visualize>
@@ -71,5 +69,4 @@
       <gazebo reference="right_camera_frame_offset">
         <sensor type="camera" name="multisense_right_camera">
-          <parent>right_camera_frame_offset</parent>
           <pose>0 0 0 0 0 0</pose>
           <visualize>false</visualize>
