Commit message: flipped joint limits not spotted earlier

File: robots/valkyrie_A/xacro/waist/joint_limits.xacro (robot description, xacro)
@@ -5,8 +5,8 @@
   <xacro:property name="TorsoRollTorqueLimit" value="150" />
   <xacro:property name="TorsoYawPositionLimit_Lower" value="-0.698" />
-  <xacro:property name="TorsoPitchPositionLimit_Lower" value="-0.698" />
+  <xacro:property name="TorsoPitchPositionLimit_Lower" value="-0.087" />
   <xacro:property name="TorsoRollPositionLimit_Lower" value="-0.262" />
   <xacro:property name="TorsoYawPositionLimit_Upper" value="0.698" />
-  <xacro:property name="TorsoPitchPositionLimit_Upper" value="0.087" />
+  <xacro:property name="TorsoPitchPositionLimit_Upper" value="0.698" />
   <xacro:property name="TorsoRollPositionLimit_Upper" value="0.262" />
   <xacro:property name="TorsoYawVelocityLimit" value="5.89" />

Commit message: Arm, torso, and neck-j1 range of motions updated and look good in RVIZ.

File: robots/valkyrie_A/xacro/waist/joint_limits.xacro (robot description, xacro)
@@ -4,10 +4,10 @@
   <xacro:property name="TorsoPitchTorqueLimit" value="150" />
   <xacro:property name="TorsoRollTorqueLimit" value="150" />
-  <xacro:property name="TorsoYawPositionLimit_Lower" value="-0.698" />
-  <xacro:property name="TorsoPitchPositionLimit_Lower" value="-0.087" />
-  <xacro:property name="TorsoRollPositionLimit_Lower" value="-0.262" />
-  <xacro:property name="TorsoYawPositionLimit_Upper" value="0.698" />
-  <xacro:property name="TorsoPitchPositionLimit_Upper" value="0.698" />
-  <xacro:property name="TorsoRollPositionLimit_Upper" value="0.262" />
+  <xacro:property name="TorsoYawPositionLimit_Lower" value="-1.329" />
+  <xacro:property name="TorsoPitchPositionLimit_Lower" value="-0.13" />
+  <xacro:property name="TorsoRollPositionLimit_Lower" value="-0.23" />
+  <xacro:property name="TorsoYawPositionLimit_Upper" value="1.181" />
+  <xacro:property name="TorsoPitchPositionLimit_Upper" value="0.666" />
+  <xacro:property name="TorsoRollPositionLimit_Upper" value="0.255" />
   <xacro:property name="TorsoYawVelocityLimit" value="5.89" />
   <xacro:property name="TorsoPitchVelocityLimit" value="9" />
