Commit message: Updated right thumb range of motion.

File: robots/valkyrie_A/xacro/thumb/joint_limits.xacro (robot description, xacro)
@@ -6,11 +6,11 @@
   <xacro:property name="ThumbPitch3TorqueLimit" value="10" />
   <xacro:property name="ThumbRollPositionLimit_Lower" value="-0.087" />
-  <xacro:property name="ThumbPitch1PositionLimit_Lower" value="-1.658" />
-  <xacro:property name="ThumbPitch2PositionLimit_Lower" value="-1.920" />
-  <xacro:property name="ThumbPitch3PositionLimit_Lower" value="-1.57" />
+  <xacro:property name="ThumbPitch1PositionLimit_Lower" value="0.175" />
+  <xacro:property name="ThumbPitch2PositionLimit_Lower" value="0.0" />
+  <xacro:property name="ThumbPitch3PositionLimit_Lower" value="0.175" />
   <xacro:property name="ThumbRollPositionLimit_Upper" value="2.356" />
-  <xacro:property name="ThumbPitch1PositionLimit_Upper" value="0.175" />
-  <xacro:property name="ThumbPitch2PositionLimit_Upper" value="0.0" />
-  <xacro:property name="ThumbPitch3PositionLimit_Upper" value="0.175" />
+  <xacro:property name="ThumbPitch1PositionLimit_Upper" value="1.658" />
+  <xacro:property name="ThumbPitch2PositionLimit_Upper" value="1.920" />
+  <xacro:property name="ThumbPitch3PositionLimit_Upper" value="1.57" />
   <xacro:property name="ThumbRollVelocityLimit" value="1" />
   <xacro:property name="ThumbPitch1VelocityLimit" value="1" />

Commit message: Fixed thumb joint limits.

File: robots/valkyrie_A/xacro/thumb/joint_limits.xacro (robot description, xacro)
@@ -5,8 +5,8 @@
   <xacro:property name="ThumbPitch2TorqueLimit" value="10" />
   <xacro:property name="ThumbPitch3TorqueLimit" value="10" />
-  <xacro:property name="ThumbRollPositionLimit_Lower" value="-0.087" />
-  <xacro:property name="ThumbPitch1PositionLimit_Lower" value="0.175" />
+  <xacro:property name="ThumbRollPositionLimit_Lower" value="0.0" />
+  <xacro:property name="ThumbPitch1PositionLimit_Lower" value="0.0" />
   <xacro:property name="ThumbPitch2PositionLimit_Lower" value="0.0" />
-  <xacro:property name="ThumbPitch3PositionLimit_Lower" value="0.175" />
+  <xacro:property name="ThumbPitch3PositionLimit_Lower" value="0.0" />
   <xacro:property name="ThumbRollPositionLimit_Upper" value="2.356" />
   <xacro:property name="ThumbPitch1PositionLimit_Upper" value="1.658" />

File: robots/valkyrie_A/xacro/thumb/thumb.xacro (robot description, xacro)
@@ -61,5 +61,10 @@
                           origin_rpy="${ThumbPitch1FrameOrientation_Roll} ${ThumbPitch1FrameOrientation_Pitch} ${ThumbPitch1FrameOrientation_Yaw}"
                           axis="${ThumbPitch1RotationAxis}">
-        <limit effort="${ThumbPitch1TorqueLimit}" lower="${ThumbPitch1PositionLimit_Lower}" upper="${ThumbPitch1PositionLimit_Upper}" velocity="${ThumbPitch1VelocityLimit}"/>
+        <xacro:if value="${(reflect+1)/2}">
+          <limit effort="${ThumbPitch1TorqueLimit}" lower="${-reflect * ThumbPitch1PositionLimit_Upper}" upper="${-reflect * ThumbPitch1PositionLimit_Lower}" velocity="${ThumbPitch1VelocityLimit}"/>
+        </xacro:if>
+        <xacro:if value="${(-reflect+1)/2}">
+          <limit effort="${ThumbPitch1TorqueLimit}" lower="${ThumbPitch1PositionLimit_Lower}" upper="${ThumbPitch1PositionLimit_Upper}" velocity="${ThumbPitch1VelocityLimit}"/>
+        </xacro:if>
     </xacro:revolute_joint>
     <xacro:revolute_joint jointName="${ThumbPitch2JointName}"
@@ -68,5 +73,10 @@
                           origin_rpy="${ThumbPitch2FrameOrientation_Roll} ${ThumbPitch2FrameOrientation_Pitch} ${ThumbPitch2FrameOrientation_Yaw}"
                           axis="${ThumbPitch2RotationAxis}">
-        <limit effort="${ThumbPitch2TorqueLimit}" lower="${ThumbPitch2PositionLimit_Lower}" upper="${ThumbPitch2PositionLimit_Upper}" velocity="${ThumbPitch2VelocityLimit}"/>
+        <xacro:if value="${(reflect+1)/2}">
+          <limit effort="${ThumbPitch2TorqueLimit}" lower="${-reflect * ThumbPitch2PositionLimit_Upper}" upper="${-reflect * ThumbPitch2PositionLimit_Lower}" velocity="${ThumbPitch2VelocityLimit}"/>
+        </xacro:if>
+        <xacro:if value="${(-reflect+1)/2}">
+          <limit effort="${ThumbPitch2TorqueLimit}" lower="${ThumbPitch2PositionLimit_Lower}" upper="${ThumbPitch2PositionLimit_Upper}" velocity="${ThumbPitch2VelocityLimit}"/>
+        </xacro:if>
     </xacro:revolute_joint>
     <xacro:revolute_joint jointName="${ThumbPitch3JointName}"
@@ -75,5 +85,10 @@
                           origin_rpy="${ThumbPitch3FrameOrientation_Roll} ${ThumbPitch3FrameOrientation_Pitch} ${ThumbPitch3FrameOrientation_Yaw}"
                           axis="${ThumbPitch3RotationAxis}">
-        <limit effort="${ThumbPitch3TorqueLimit}" lower="${ThumbPitch3PositionLimit_Lower}" upper="${ThumbPitch3PositionLimit_Upper}" velocity="${ThumbPitch3VelocityLimit}"/>
+        <xacro:if value="${(reflect+1)/2}">
+          <limit effort="${ThumbPitch3TorqueLimit}" lower="${-reflect * ThumbPitch3PositionLimit_Upper}" upper="${-reflect * ThumbPitch3PositionLimit_Lower}" velocity="${ThumbPitch3VelocityLimit}"/>
+        </xacro:if>
+        <xacro:if value="${(-reflect+1)/2}">
+          <limit effort="${ThumbPitch3TorqueLimit}" lower="${ThumbPitch3PositionLimit_Lower}" upper="${ThumbPitch3PositionLimit_Upper}" velocity="${ThumbPitch3VelocityLimit}"/>
+        </xacro:if>
     </xacro:revolute_joint>
   </xacro:macro>
