Commit message: Added multisens_sl.urdf and include that to add the multisense stuff rather than my own homegrown stuff which isn't as good.

File: robots/common/valkyrie_base.xacro (robot description, xacro)
@@ -9,5 +9,5 @@
     <xacro:v1_trunk_sensors/>
     <xacro:make_head head_root_link="${TorsoRollLinkName}" />
-    <xacro:v1_head_sensors />
+    <!-- <xacro:v1_head_sensors /> -->
     <xacro:make_arm prefix="Right" reflect="-1" arm_root_link="${TorsoRollLinkName}" />
     <xacro:make_thumb prefix="Right" reflect="-1" thumb_root_link="RightPalm"/>

File: robots/valkyrie_A/xacro/head/head.xacro (robot description, xacro)
@@ -6,5 +6,4 @@
   <xacro:include filename="$(find val_description)/robots/valkyrie_A/xacro/head/frame_parameters.xacro"/>
   <xacro:include filename="$(find val_description)/robots/valkyrie_A/xacro/head/mass_parameters.xacro"/>
-  <xacro:include filename="$(find val_description)/robots/common/sensors/multisense_sl.xacro"/>
   <xacro:property name="NJ3_Link_Radius" value="0.139"/>
   <xacro:macro name="include_head" params="lower_neck_pitch_root_link">
@@ -52,17 +51,6 @@
       <controller_gains Kp="20000" Kd="0"/>
     </xacro:revolute_joint_ex>
-  </xacro:macro>
-  <xacro:macro name="v1_head_sensors">
-    <xacro:multisense_sl parentLink="${UpperNeckPitchLinkName}"
-                  joint_axis="1 0 0"
-                  joint_origin_xyz="${HokuyoFrameOrigin_X} ${HokuyoFrameOrigin_Y} ${HokuyoFrameOrigin_Z}"
-                  joint_origin_rpy="${HokuyoFrameOrientation_Roll} ${HokuyoFrameOrientation_Pitch} ${HokuyoFrameOrientation_Yaw}"
-                  com_origin_xyz="${HokuyoLinkComPosition}"
-                  com_origin_rpy="0 0 0"
-                  mass="${HokuyoLinkMass}"
-                  visual_mesh="${mesh_root}/head/multisense_hokuyo.dae"
-                  material="White"
-                  collision_mesh="${mesh_root}/head/multisense_hokuyo.dae" />
-  </xacro:macro>
+    <xacro:fixed_joint jointName="multisense_head_root" parent="${UpperNeckPitchLinkName}" child="head" origin_xyz="0.183585961 0.0 0.075353826" origin_rpy="-3.14159 0.130899694 0.0" />
+    </xacro:macro>
   <xacro:macro name="neck_actuators" params="name1 type1 name2 type2 name3 type3">
     <actuator name="${name1}" type="${type1}"/>

File: robots/valkyrie_A_sim.xacro (robot description, xacro)
@@ -2,3 +2,4 @@
     <xacro:property name="mesh_root" value="package://val_description/meshes"/>
     <xacro:include filename="$(find val_description)/robots/common/valkyrie_base.xacro"/>
+    <xacro:include filename="$(find val_description)/urdf/multisense_sl.urdf" />
 </robot>
