Commit message: Created two xacros for val-A, one for hardware that doesn't have any multisens and one for sim that includes the multisense urdf.

File: robots/common/valkyrie_base_sim.xacro (robot description, xacro)
@@ -5,9 +5,9 @@
     <xacro:include filename="$(find val_description)/robots/valkyrie_A/xacro/common/common_bodies.xacro" />
     <xacro:make_pelvis />
-    <xacro:v1_pelvis_sensors/>
+    <xacro:v1_pelvis_sensors />
     <xacro:make_waist waist_root_link="${Pelvis_Link_Name}" />
     <xacro:v1_trunk_sensors/>
     <xacro:make_head head_root_link="${TorsoRollLinkName}" />
-    <!-- <xacro:v1_head_sensors /> -->
+    <xacro:include_multisense />
     <xacro:make_arm prefix="Right" reflect="-1" arm_root_link="${TorsoRollLinkName}" />
     <xacro:make_thumb prefix="Right" reflect="-1" thumb_root_link="RightPalm"/>

File: robots/valkyrie_A/xacro/head/head.xacro (robot description, xacro)
@@ -51,5 +51,7 @@
       <controller_gains Kp="20000" Kd="0"/>
     </xacro:revolute_joint_ex>
-    <xacro:fixed_joint jointName="multisense_head_root" parent="${UpperNeckPitchLinkName}" child="head" origin_xyz="0.183585961 0.0 0.075353826" origin_rpy="-3.14159 0.130899694 0.0" />
+    </xacro:macro>
+    <xacro:macro name="include_multisense">
+      <xacro:fixed_joint jointName="multisense_head_root" parent="${UpperNeckPitchLinkName}" child="head" origin_xyz="0.183585961 0.0 0.075353826" origin_rpy="-3.14159 0.130899694 0.0" />
     </xacro:macro>
   <xacro:macro name="neck_actuators" params="name1 type1 name2 type2 name3 type3">

File: robots/valkyrie_A_sim.xacro (robot description, xacro)
@@ -1,5 +1,5 @@
 <robot xmlns:xacro="http://ros.org/wiki/xacro" name="valkyrie">
     <xacro:property name="mesh_root" value="package://val_description/meshes"/>
-    <xacro:include filename="$(find val_description)/robots/common/valkyrie_base.xacro"/>
+    <xacro:include filename="$(find val_description)/robots/common/valkyrie_base_sim.xacro"/>
     <xacro:include filename="$(find val_description)/urdf/multisense_sl.urdf" />
 </robot>
