Commit message: Fixed hw xacro to have extra link so fixed transform to multisense root is identity.

File: robots/common/valkyrie_base_hw.xacro (robot description, xacro)
@@ -9,4 +9,5 @@
     <xacro:v1_trunk_sensors/>
     <xacro:make_head head_root_link="${TorsoRollLinkName}" />
+    <xacro:include_multisense_hw />
     <xacro:make_arm prefix="Right" reflect="-1" arm_root_link="${TorsoRollLinkName}" />
     <xacro:make_thumb prefix="Right" reflect="-1" thumb_root_link="RightPalm"/>

File: robots/common/valkyrie_base_sim.xacro (robot description, xacro)
@@ -9,5 +9,5 @@
     <xacro:v1_trunk_sensors/>
     <xacro:make_head head_root_link="${TorsoRollLinkName}" />
-    <xacro:include_multisense />
+    <xacro:include_multisense_sim />
     <xacro:make_arm prefix="Right" reflect="-1" arm_root_link="${TorsoRollLinkName}" />
     <xacro:make_thumb prefix="Right" reflect="-1" thumb_root_link="RightPalm"/>

File: robots/valkyrie_A/xacro/arm/arm.xacro (robot description, xacro)
@@ -29,5 +29,4 @@
   <xacro:property name="AJ7_Link_Length" value="0.038"/>
   <xacro:macro name="make_upper_arm" params="prefix reflect upper_arm_root_link">
-    <!-- LINKS -->
     <xacro:box_link name="${ShoulderPitchLinkName}"
                     width="${AJ1_Link_Width}" height="${AJ1_Link_Height}" depth="${AJ1_Link_Length}" mass="${ShoulderPitchLinkMass}"
@@ -55,5 +54,4 @@
                     material="Gold"
                     collision_mesh="${mesh_root}/arms/aj4_${prefix}.dae" />
-    <!-- AJ1 -->
     <xacro:revolute_joint_ex jointName="${ShoulderPitchJointName}"
                           parent="${upper_arm_root_link}" child="${ShoulderPitchLinkName}"
@@ -65,5 +63,4 @@
         <controller_gains Kp="20000" Kd="400"/>
     </xacro:revolute_joint_ex>
-    <!-- AJ2 -->
     <xacro:revolute_joint_ex jointName="${ShoulderRollJointName}"
                           parent="${ShoulderPitchLinkName}" child="${ShoulderRollLinkName}"
@@ -80,5 +77,4 @@
         <controller_gains Kp="20000" Kd="400"/>
     </xacro:revolute_joint_ex>
-    <!-- AJ3 -->
     <xacro:revolute_joint_ex jointName="${ShoulderYawJointName}"
                           parent="${ShoulderRollLinkName}" child="${ShoulderYawLinkName}"
@@ -90,5 +86,4 @@
         <controller_gains Kp="20000" Kd="400"/>
     </xacro:revolute_joint_ex>
-    <!-- AJ4 -->
     <xacro:revolute_joint_ex jointName="${ElbowPitchJointName}"
                           parent="${ShoulderYawLinkName}" child="${ElbowPitchLinkName}"
@@ -107,5 +102,4 @@
   </xacro:macro>
   <xacro:macro name="make_lower_arm" params="prefix reflect lower_arm_root_link">
-    <!-- LINKS -->
     <xacro:box_link name="${ForearmLinkName}"
                     width="${AJ5_Link_Width}" height="${AJ5_Link_Height}" depth="${AJ5_Link_Length}" mass="${ForearmYawLinkMass}"
@@ -129,5 +123,4 @@
                     material="Gold"
                     collision_mesh="${mesh_root}/arms/palm_${prefix}.dae"/>
-    <!-- AJ5 -->
     <xacro:revolute_joint_ex jointName="${ForearmYawJointName}"
                           parent="${lower_arm_root_link}" child="${ForearmLinkName}"
@@ -139,5 +132,4 @@
         <controller_gains Kp="20000" Kd="0"/>
     </xacro:revolute_joint_ex>
-    <!-- AJ6 -->
     <xacro:revolute_joint_ex jointName="${WristRollJointName}"
                           parent="${ForearmLinkName}" child="${WristRollLinkName}"
@@ -154,5 +146,4 @@
         <controller_gains Kp="20000" Kd="400"/>
     </xacro:revolute_joint_ex>
-    <!-- AJ7 -->
     <xacro:revolute_joint_ex jointName="${WristPitchJointName}"
                           parent="${WristRollLinkName}" child="${WristPitchLinkName}"
@@ -174,5 +165,4 @@
     <xacro:make_lower_arm prefix="${prefix}" reflect="${reflect}" lower_arm_root_link="${ElbowPitchLinkName}" />
   </xacro:macro>
-  <!-- Actuators -->
   <xacro:macro name="upper_arm_actuators" params="name1 type1 name2 type2 name3 type3 name4 type4">
     <actuator name="${name1}" type="${type1}"/>

File: robots/valkyrie_A/xacro/head/head.xacro (robot description, xacro)
@@ -52,6 +52,10 @@
     </xacro:revolute_joint_ex>
     </xacro:macro>
-    <xacro:macro name="include_multisense">
-      <xacro:fixed_joint jointName="multisense_head_root" parent="${UpperNeckPitchLinkName}" child="head" origin_xyz="0.183585961 0.0 0.075353826" origin_rpy="-3.14159 0.130899694 0.0" />
+    <xacro:macro name="include_multisense_sim">
+      <xacro:fixed_joint jointName="multisense_head_root_joint" parent="${UpperNeckPitchLinkName}" child="head" origin_xyz="0.183585961 0.0 0.075353826" origin_rpy="-3.14159 0.130899694 0.0" />
+    </xacro:macro>
+    <xacro:macro name="include_multisense_hw">
+      <xacro:massless_virtual_link name="miltisense_root_link" origin_xyz="0 0 0" origin_rpy="0 0 0"/>
+      <xacro:fixed_joint jointName="multisense_head_root_joint" parent="${UpperNeckPitchLinkName}" child="multisense_root_link" origin_xyz="0.183585961 0.0 0.075353826" origin_rpy="-3.14159 0.130899694 0.0" />
     </xacro:macro>
   <xacro:macro name="neck_actuators" params="name1 type1 name2 type2 name3 type3">
