Commit message: Moved a bunch of stuff around so I could get rid of the common_xacro package.

File: robots/common/generic_models.xacro (robot description, xacro)
@@ -1,4 +1,4 @@
 <?xml version="1.0" ?>
-<robot xmlns:xacro="http://www.ros.org/wiki/xacro" name="drc">
+<robot xmlns:xacro="http://www.ros.org/wiki/xacro" name="generic_models">
   <xacro:macro name="v1_actuator" params="name api">
     <actuator name="${name}" type="${api}"/>
@@ -439,200 +439,3 @@
                        origin_xyz="${origin_xyz}"/>
   </xacro:macro>
-  <xacro:macro name="v1_modes" params="jointName actuatorName">
-    <mode name="${jointName}Mode" type="mode_plugins/ModeInterface">
-      <translator name="${jointName}ModeData" type="${mode_data_interface}">
-        <joint    name="${jointName}" data="mode"/>
-        <actuator name="${actuatorName}" data="mode"/>
-      </translator>
-      <translator name="${jointName}ModeCommand" type="${mode_command_interface}">
-        <joint    name="${jointName}" data="modeCommand"/>
-        <actuator name="${actuatorName}" data="modeCommand"/>
-      </translator>
-    </mode>
-  </xacro:macro>
-  <xacro:macro name="simple_transmission" params="jointName actuatorName reduction offset">
-    <transmission name="${jointName}Transmission" type="loadable_transmissions/SimpleTransmission">
-    <mechanicalReduction>${reduction}</mechanicalReduction>
-      <jointOffset>${offset}</jointOffset>
-      <interface type="ActuatorToJointStateInterface">
-        <joint name="${jointName}" data="data"/>
-        <actuator name="${actuatorName}" data="data"/>
-      </interface>
-      <interface type="JointToActuatorPositionInterface">
-        <joint name="${jointName}" data="positionCommand"/>
-        <actuator name="${actuatorName}" data="positionCommand"/>
-      </interface>
-      <interface type="JointToActuatorVelocityInterface">
-        <joint name="${jointName}" data="velocityCommand"/>
-        <actuator name="${actuatorName}" data="velocityCommand"/>
-      </interface>
-      <interface type="JointToActuatorEffortInterface">
-        <joint name="${jointName}" data="effortCommand"/>
-        <actuator name="${actuatorName}" data="effortCommand"/>
-      </interface>
-      <interface type="JointToActuatorStateInterface">
-        <joint name="${jointName}" data="data"/>
-        <actuator name="${actuatorName}" data="data"/>
-      </interface>
-      <interface type="ActuatorToJointPositionInterface">
-        <joint name="${jointName}" data="positionCommand"/>
-        <actuator name="${actuatorName}" data="positionCommand"/>
-      </interface>
-      <interface type="ActuatorToJointVelocityInterface">
-        <joint name="${jointName}" data="velocityCommand"/>
-        <actuator name="${actuatorName}" data="velocityCommand"/>
-      </interface>
-      <interface type="ActuatorToJointEffortInterface">
-        <joint name="${jointName}" data="effortCommand"/>
-        <actuator name="${actuatorName}" data="effortCommand"/>
-      </interface>
-    </transmission>
-  </xacro:macro>
-  <xacro:macro name="pushrod_transmission" params="tranName namespace reflect joint1 joint2 actuator1 actuator2">
-    <transmission name="${tranName}" type="loadable_transmissions/PushrodTransmission">
-      <interface type="ActuatorToJointStateInterface">
-        <joint name="${joint1}" data="data"/>
-        <joint name="${joint2}" data="data"/>
-        <actuator name="${actuator1}" data="data"/>
-        <actuator name="${actuator2}" data="data"/>
-      </interface>
-      <interface type="JointToActuatorPositionInterface">
-        <joint name="${joint1}" data="positionCommand"/>
-        <joint name="${joint2}" data="positionCommand"/>
-        <actuator name="${actuator1}" data="positionCommand"/>
-        <actuator name="${actuator2}" data="positionCommand"/>
-      </interface>
-      <interface type="JointToActuatorVelocityInterface">
-        <joint name="${joint1}" data="velocityCommand"/>
-        <joint name="${joint2}" data="velocityCommand"/>
-        <actuator name="${actuator1}" data="velocityCommand"/>
-        <actuator name="${actuator2}" data="velocityCommand"/>
-      </interface>
-      <interface type="JointToActuatorEffortInterface">
-        <joint name="${joint1}" data="effortCommand"/>
-        <joint name="${joint2}" data="effortCommand"/>
-        <actuator name="${actuator1}" data="effortCommand"/>
-        <actuator name="${actuator2}" data="effortCommand"/>
-      </interface>
-      <interface type="JointToActuatorStateInterface">
-        <joint name="${joint1}" data="data"/>
-        <joint name="${joint2}" data="data"/>
-        <actuator name="${actuator1}" data="data"/>
-        <actuator name="${actuator2}" data="data"/>
-      </interface>
-      <interface type="ActuatorToJointPositionInterface">
-        <joint name="${joint1}" data="positionCommand"/>
-        <joint name="${joint2}" data="positionCommand"/>
-        <actuator name="${actuator1}" data="positionCommand"/>
-        <actuator name="${actuator2}" data="positionCommand"/>
-      </interface>
-      <interface type="ActuatorToJointVelocityInterface">
-        <joint name="${joint1}" data="velocityCommand"/>
-        <joint name="${joint2}" data="velocityCommand"/>
-        <actuator name="${actuator1}" data="velocityCommand"/>
-        <actuator name="${actuator2}" data="velocityCommand"/>
-      </interface>
-      <interface type="ActuatorToJointEffortInterface">
-        <joint name="${joint1}" data="effortCommand"/>
-        <joint name="${joint2}" data="effortCommand"/>
-        <actuator name="${actuator1}" data="effortCommand"/>
-        <actuator name="${actuator2}" data="effortCommand"/>
-      </interface>
-      <parameterNamespace name="${namespace}" />
-      <reflect data="${reflect}" />
-    </transmission>
-  </xacro:macro>
-  <xacro:macro name="finger2_transmission" params="tranName joint1 joint2 actuator">
-    <transmission name="${tranName}" type="loadable_transmissions/FingerTransmission">
-      <interface type="ActuatorToJointStateInterface">
-        <joint name="${joint1}" data="data"/>
-        <joint name="${joint2}" data="data"/>
-        <actuator name="${actuator}" data="data"/>
-      </interface>
-      <interface type="JointToActuatorPositionInterface">
-        <joint name="${joint1}" data="positionCommand"/>
-        <joint name="${joint2}" data="positionCommand"/>
-        <actuator name="${actuator}" data="positionCommand"/>
-      </interface>
-      <interface type="JointToActuatorStateInterface">
-        <joint name="${joint1}" data="data"/>
-        <joint name="${joint2}" data="data"/>
-        <actuator name="${actuator}" data="data"/>
-      </interface>
-      <interface type="ActuatorToJointPositionInterface">
-        <joint name="${joint1}" data="positionCommand"/>
-        <joint name="${joint2}" data="positionCommand"/>
-        <actuator name="${actuator}" data="positionCommand"/>
-      </interface>
-      <reducer reduction="${1/2}" offset="0"/>
-      <reducer reduction="${1/2}" offset="0"/>
-    </transmission>
-  </xacro:macro>
-  <xacro:macro name="finger3_transmission" params="tranName joint1 joint2 joint3 actuator">
-    <transmission name="${tranName}" type="loadable_transmissions/FingerTransmission">
-      <interface type="ActuatorToJointStateInterface">
-        <joint name="${joint1}" data="data"/>
-        <joint name="${joint2}" data="data"/>
-        <joint name="${joint3}" data="data"/>
-        <actuator name="${actuator}" data="data"/>
-      </interface>
-      <interface type="JointToActuatorPositionInterface">
-        <joint name="${joint1}" data="positionCommand"/>
-        <joint name="${joint2}" data="positionCommand"/>
-        <joint name="${joint3}" data="positionCommand"/>
-        <actuator name="${actuator}" data="positionCommand"/>
-      </interface>
-      <interface type="JointToActuatorStateInterface">
-        <joint name="${joint1}" data="data"/>
-        <joint name="${joint2}" data="data"/>
-        <joint name="${joint3}" data="data"/>
-        <actuator name="${actuator}" data="data"/>
-      </interface>
-      <interface type="ActuatorToJointPositionInterface">
-        <joint name="${joint1}" data="positionCommand"/>
-        <joint name="${joint2}" data="positionCommand"/>
-        <joint name="${joint3}" data="positionCommand"/>
-        <actuator name="${actuator}" data="positionCommand"/>
-      </interface>
-      <reducer reduction="${1/3}" offset="0"/>
-      <reducer reduction="${1/3}" offset="0"/>
-      <reducer reduction="${1/3}" offset="0"/>
-    </transmission>
-  </xacro:macro>
-  <xacro:macro name="finger4_transmission" params="tranName joint1 joint2 joint3 joint4 actuator">
-    <transmission name="${tranName}" type="loadable_transmissions/FingerTransmission">
-      <interface type="ActuatorToJointStateInterface">
-        <joint name="${joint1}" data="data"/>
-        <joint name="${joint2}" data="data"/>
-        <joint name="${joint3}" data="data"/>
-        <joint name="${joint4}" data="data"/>
-        <actuator name="${actuator}" data="data"/>
-      </interface>
-      <interface type="JointToActuatorPositionInterface">
-        <joint name="${joint1}" data="positionCommand"/>
-        <joint name="${joint2}" data="positionCommand"/>
-        <joint name="${joint3}" data="positionCommand"/>
-        <joint name="${joint4}" data="positionCommand"/>
-        <actuator name="${actuator}" data="positionCommand"/>
-      </interface>
-      <interface type="JointToActuatorStateInterface">
-        <joint name="${joint1}" data="data"/>
-        <joint name="${joint2}" data="data"/>
-        <joint name="${joint3}" data="data"/>
-        <joint name="${joint4}" data="data"/>
-        <actuator name="${actuator}" data="data"/>
-      </interface>
-      <interface type="ActuatorToJointPositionInterface">
-        <joint name="${joint1}" data="positionCommand"/>
-        <joint name="${joint2}" data="positionCommand"/>
-        <joint name="${joint3}" data="positionCommand"/>
-        <joint name="${joint4}" data="positionCommand"/>
-        <actuator name="${actuator}" data="positionCommand"/>
-      </interface>
-      <reducer reduction="${1/4}" offset="0"/>
-      <reducer reduction="${1/4}" offset="0"/>
-      <reducer reduction="${1/4}" offset="0"/>
-      <reducer reduction="${1/4}" offset="0"/>
-    </transmission>
-  </xacro:macro>
 </robot>

File: robots/valkyrie_A/xacro/arm/arm.xacro (robot description, xacro)
@@ -1,4 +1,4 @@
 <?xml version="1.0" ?>
-<robot xmlns:xacro="http://www.ros.org/wiki/xacro" name="v1/arm">
+<robot xmlns:xacro="http://www.ros.org/wiki/xacro" name="arm">
   <xacro:include filename="$(find val_description)/robots/valkyrie_A/xacro/arm/joint_names.xacro"/>
   <xacro:include filename="$(find val_description)/robots/valkyrie_A/xacro/arm/joint_axes.xacro"/>

File: robots/valkyrie_A/xacro/head/head.xacro (robot description, xacro)
@@ -1,3 +1,3 @@
-<robot xmlns:xacro="http://www.ros.org/wiki/xacro" name="v1/head">
+<robot xmlns:xacro="http://www.ros.org/wiki/xacro" name="head">
   <xacro:include filename="$(find val_description)/robots/valkyrie_A/xacro/head/joint_names.xacro"/>
   <xacro:include filename="$(find val_description)/robots/valkyrie_A/xacro/head/joint_axes.xacro"/>

File: robots/valkyrie_A/xacro/leg/leg.xacro (robot description, xacro)
@@ -1,4 +1,4 @@
 <?xml version="1.0" ?>
-<robot xmlns:xacro="http://www.ros.org/wiki/xacro" name="v1/leg">
+<robot xmlns:xacro="http://www.ros.org/wiki/xacro" name="leg">
   <xacro:include filename="$(find val_description)/robots/valkyrie_A/xacro/leg/joint_names.xacro"/>
   <xacro:include filename="$(find val_description)/robots/valkyrie_A/xacro/leg/joint_axes.xacro"/>

File: robots/valkyrie_A/xacro/middle_finger/middle_finger.xacro (robot description, xacro)
@@ -1,4 +1,4 @@
 <?xml version="1.0" ?>
-<robot xmlns:xacro="http://www.ros.org/wiki/xacro" name="v1/middle_finger">
+<robot xmlns:xacro="http://www.ros.org/wiki/xacro" name="middle_finger">
   <xacro:include filename="$(find val_description)/robots/valkyrie_A/xacro/middle_finger/joint_names.xacro"/>
   <xacro:include filename="$(find val_description)/robots/valkyrie_A/xacro/middle_finger/joint_axes.xacro"/>

File: robots/valkyrie_A/xacro/pinky_finger/pinky_finger.xacro (robot description, xacro)
@@ -1,4 +1,4 @@
 <?xml version="1.0" ?>
-<robot xmlns:xacro="http://www.ros.org/wiki/xacro" name="v1/pinky_finger">
+<robot xmlns:xacro="http://www.ros.org/wiki/xacro" name="pinky_finger">
   <xacro:include filename="$(find val_description)/robots/valkyrie_A/xacro/pinky_finger/joint_names.xacro"/>
   <xacro:include filename="$(find val_description)/robots/valkyrie_A/xacro/pinky_finger/joint_axes.xacro"/>

File: robots/valkyrie_A/xacro/thumb/thumb.xacro (robot description, xacro)
@@ -1,4 +1,4 @@
 <?xml version="1.0" ?>
-<robot xmlns:xacro="http://www.ros.org/wiki/xacro" name="v1/thumb">
+<robot xmlns:xacro="http://www.ros.org/wiki/xacro" name="thumb">
   <xacro:include filename="$(find val_description)/robots/valkyrie_A/xacro/thumb/joint_names.xacro"/>
   <xacro:include filename="$(find val_description)/robots/valkyrie_A/xacro/thumb/joint_axes.xacro"/>

Commit message: Updated pelvis mass, COM location, and inertia.

File: robots/common/generic_models.xacro (robot description, xacro)
@@ -43,8 +43,6 @@
         <geometry>
           <mesh filename="${visual_mesh}"/>
-          <!-- <cylinder radius="${radius}" length="${length}"/> -->
-        </geometry>
-        <origin rpy="0 0 0" xyz="0 0 0"/>
-        <!-- <origin rpy="${origin_rpy}" xyz="${origin_xyz}"/> -->
+        </geometry>
+        <origin rpy="0 0 0" xyz="0 0 0"/>
         <material name="${material}"/>
       </visual>
@@ -297,8 +295,4 @@
     </link>
   </xacro:macro>
-  <!-- May 2015: However zero mass/inertials links are still useful. (And removed with gz sdf)
-  This macro here was added to allow fixed links to have (almost) no effect on the output compound
-  sdf mass and inertia
-  -->
   <xacro:property name="massless_virtual_link_mass" value="0.0000001"/>
   <xacro:property name="massless_virtual_link_radius" value="0.0000001"/>

File: robots/valkyrie_A/xacro/arm/arm.xacro (robot description, xacro)
@@ -27,5 +27,4 @@
   <xacro:property name="AJ7_Link_Length" value="0.038"/>
   <xacro:macro name="make_upper_arm" params="prefix reflect upper_arm_root_link">
-    <!-- LINKS -->
     <xacro:box_link name="${ShoulderPitchLinkName}"
                     width="${AJ1_Link_Width}" height="${AJ1_Link_Height}" depth="${AJ1_Link_Length}" mass="${ShoulderPitchLinkMass}"
@@ -134,5 +133,4 @@
         <controller_gains Kp="20000" Kd="0"/>
     </xacro:revolute_joint_ex>
-    <!-- AJ6 -->
     <xacro:revolute_joint_ex jointName="${WristRollJointName}"
                           parent="${ForearmLinkName}" child="${WristRollLinkName}"

File: robots/valkyrie_A/xacro/leg/leg.xacro (robot description, xacro)
@@ -77,5 +77,4 @@
   </xacro:macro>
   <xacro:macro name="make_leg_joints" params="prefix reflect leg_root_link">
-    <!-- LJ1 -->
     <xacro:revolute_joint_ex jointName="${HipYawJointName}"
                           parent="${HipYawParentLinkName}" child="${HipYawLinkName}"
@@ -150,5 +149,4 @@
     <xacro:make_ankle_joints prefix="${prefix}" reflect="${reflect}" leg_root_link="${leg_root_link}" />
   </xacro:macro>
-  <!-- Sensors -->
   <xacro:macro name="v1_leg_sensors" params="prefix reflect">
     <xacro:virtual_fixed_frame_offset name="${prefix}COP"

File: robots/valkyrie_A/xacro/pelvis/pelvis.xacro (robot description, xacro)
@@ -2,7 +2,9 @@
     <xacro:property name="Pelvis_Link_Name" value="Pelvis" />
     <xacro:macro name="make_pelvis">
-        <xacro:box_link name="${Pelvis_Link_Name}"
-                        width="0.28251052337959348115" height="0.34445341259705453130" depth="0.36811588436650161116" mass="6.986"
-                        origin_xyz="0.000733954 -0.000895362 -0.0702552"
+        <xacro:standard_link name="${Pelvis_Link_Name}"
+                        mass="8.22"
+                        origin_xyz="-0.00532 -0.003512 -0.0036"
+                        ixx="0.11866378" ixy="-0.00143482" ixz="0.003271293"
+                        iyy="0.097963425" iyz="0.002159545" izz="0.083854638"
                         origin_rpy="0 0 0"
                         visual_mesh="${mesh_root}/pelvis/pelvis.stl" material="White"

File: robots/valkyrie_A/xacro/waist/waist.xacro (robot description, xacro)
@@ -1,4 +1,3 @@
 <robot xmlns:xacro="http://www.ros.org/wiki/xacro" name="v1/waist">
-  <!-- Properties -->
   <xacro:include filename="$(find val_description)/robots/valkyrie_A/xacro/waist/joint_names.xacro"/>
   <xacro:include filename="$(find val_description)/robots/valkyrie_A/xacro/waist/joint_axes.xacro"/>

Commit message: Use boxes for foot collision shape
Create a new macro: link_box_collision_mesh_visual
that uses a box for the collision shape and a mesh
for the visual.
Use this macro to for the feet with hard-coded
box size and pose.

File: robots/common/generic_models.xacro (robot description, xacro)
@@ -100,4 +100,29 @@
     </link>
   </xacro:macro>
+  <xacro:macro name="link_box_collision_mesh_visual"
+          params="name width height depth mass inertial_xyz inertial_rpy ixx ixy ixz iyy iyz izz visual_mesh material box_xyz box_rpy">
+    <link name="${name}">
+      <inertial>
+        <mass value="${mass}" />
+        <origin rpy="${inertial_rpy}" xyz="${inertial_xyz}"/>
+        <inertia ixx="${ixx}"  ixy="${ixy}" ixz="${ixz}"
+                 iyy="${iyy}" iyz="${iyz}"
+                 izz="${izz}" />
+      </inertial>
+      <visual>
+        <geometry>
+          <mesh filename="${visual_mesh}"/>
+        </geometry>
+        <origin rpy="0 0 0" xyz="0 0 0"/>
+        <material name="${material}"/>
+      </visual>
+      <collision>
+        <geometry>
+          <box size="${width} ${height} ${depth}"/>
+        </geometry>
+        <origin rpy="${box_rpy}" xyz="${box_xyz}"/>
+      </collision>
+    </link>
+  </xacro:macro>
   <xacro:macro name="virtual_link_sphere" params="name radius mass origin_xyz origin_rpy">
     <link name="${name}">

File: robots/valkyrie_A/xacro/leg/leg.xacro (robot description, xacro)
@@ -53,13 +53,17 @@
                     material="White"
                     collision_mesh="${mesh_root}/legs/lj5.dae"/>
-    <xacro:standard_link name="${AnkleRollLinkName}"
+    <xacro:link_box_collision_mesh_visual name="${AnkleRollLinkName}"
                     mass="${FootMass}"
-                    origin_xyz="${FootComPosition}"
+                    inertial_xyz="${FootComPosition}"
                     ixx="${FootInertia_IXX}" ixy="${FootInertia_IXY}" ixz="${FootInertia_IXZ}"
                     iyy="${FootInertia_IYY}" iyz="${FootInertia_IYZ}" izz="${FootInertia_IZZ}"
-                    origin_rpy="0 0 0"
+                    inertial_rpy="0 0 0"
                     visual_mesh="${mesh_root}/legs/foot_${prefix}.dae"
                     material="White"
-                    collision_mesh="${mesh_root}/legs/foot_${prefix}.dae" />
+                    width="0.27"
+                    height="0.15"
+                    depth="0.064"
+                    box_xyz="0.06 0 -0.06"
+                    box_rpy="0 0.1309 0.0" />
   </xacro:macro>
   <xacro:macro name="make_leg_joints" params="prefix reflect leg_root_link">
