Commit message: Added <always_on> tag to imu definition. Removed some unused xml macros.

File: robots/common/generic_models.xacro (robot description, xacro)
@@ -27,52 +27,4 @@
       </collision>
     </link>
-<!--    <gazebo reference="${name}">
-      <material>Gazebo/${material}</material>
-    </gazebo> -->
-  </xacro:macro>
-  <xacro:macro name="cylinder_link" params="name radius length mass origin_xyz origin_rpy visual_mesh material collision_mesh">
-    <link name="${name}">
-      <inertial>
-        <mass value="${mass}" />
-        <origin rpy="${origin_rpy}" xyz="${origin_xyz}"/>
-        <inertia ixx="${mass*(3*radius*radius + length*length)/12}" ixy="0.0" ixz="0.0"
-                 iyy="${mass*(3*radius*radius + length*length)/12}" iyz="0.0"
-                 izz="${0.5*mass*radius*radius}" />
-      </inertial>
-      <visual>
-        <geometry>
-          <mesh filename="${visual_mesh}"/>
-        </geometry>
-        <origin rpy="0 0 0" xyz="0 0 0"/>
-        <material name="${material}"/>
-      </visual>
-      <collision>
-        <geometry>
-          <mesh filename="${collision_mesh}"/>
-        </geometry>
-        <origin rpy="0 0 0" xyz="0 0 0"/>
-      </collision>
-    </link>
-    <gazebo reference="${name}">
-      <material>Gazebo/${material}</material>
-    </gazebo>
-  </xacro:macro>
-  <xacro:macro name="cylinder_link_no_mesh" params="name radius length mass origin_xyz origin_rpy">
-    <link name="${name}">
-      <inertial>
-        <mass value="${mass}" />
-        <origin rpy="${origin_rpy}" xyz="${origin_xyz}"/>
-        <inertia ixx="${mass*(3*radius*radius + length*length)/12}" ixy="0.0" ixz="0.0"
-                 iyy="${mass*(3*radius*radius + length*length)/12}" iyz="0.0"
-                 izz="${0.5*mass*radius*radius}" />
-      </inertial>
-      <visual>
-        <geometry>
-          <cylinder radius="${radius}" length="${length}"/>
-        </geometry>
-        <origin rpy="${origin_rpy}" xyz="${origin_xyz}"/>
-        <material name="Gray"/>
-      </visual>
-    </link>
   </xacro:macro>
   <xacro:macro name="link_no_mesh" params="name width height depth mass origin_xyz origin_rpy ixx ixy ixz iyy iyz izz">
@@ -98,22 +50,4 @@
         <origin rpy="${origin_rpy}" xyz="${origin_xyz}"/>
       </collision>
-    </link>
-  </xacro:macro>
-  <xacro:macro name="virtual_link_sphere" params="name radius mass origin_xyz origin_rpy">
-    <link name="${name}">
-      <inertial>
-        <mass value="${mass}" />
-        <origin rpy="${origin_rpy}" xyz="${origin_xyz}"/>
-        <inertia ixx="${2*mass*radius*radius/5}" ixy="0.0" ixz="0.0"
-                 iyy="${2*mass*radius*radius/5}" iyz="0.0"
-                 izz="${2*mass*radius*radius/5}" />
-      </inertial>
-      <visual>
-        <origin rpy="0 0 0" xyz="0 0 0"/>
-        <geometry>
-          <sphere radius="${radius}"/>
-        </geometry>
-        <material name="Gray"/>
-      </visual>
     </link>
   </xacro:macro>
@@ -239,31 +173,4 @@
     </gazebo>
   </xacro:macro>
-  <xacro:macro name="prismatic_joint_axis" params="jointName parent child origin_xyz origin_rpy axis *limits">
-    <joint name="${jointName}" type="prismatic">
-      <origin rpy="${origin_rpy}" xyz="${origin_xyz}"/>
-      <axis xyz="${axis}"/>
-      <parent link="${parent}"/>
-      <child link="${child}"/>
-      <dynamics damping="1.0" friction="0.0"/>
-      <xacro:insert_block name="limits" />
-    </joint>
-    <gazebo reference="${jointName}">
-      <implicitSpringDamper>1</implicitSpringDamper>
-    </gazebo>
-  </xacro:macro>
-  <xacro:macro name="revolute_joint_axis" params="jointName parent child origin_xyz origin_rpy axis *limits">
-    <joint name="${jointName}" type="revolute">
-      <origin rpy="${origin_rpy}" xyz="${origin_xyz}"/>
-      <axis xyz="${axis}"/>
-      <parent link="${parent}"/>
-      <child link="${child}"/>
-      <xacro:insert_block name="limits" />
-      <dynamics damping="1.0" friction="0.0"/>
-    </joint>
-    <gazebo reference="${jointName}">
-      <provideFeedback>1</provideFeedback>
-      <implicitSpringDamper>1</implicitSpringDamper>
-    </gazebo>
-  </xacro:macro>
   <xacro:macro name="fixed_joint" params="jointName parent child origin_xyz origin_rpy">
     <joint name="${jointName}" type="fixed">

File: robots/common/sensors/microstrain.xacro (robot description, xacro)
@@ -15,4 +15,5 @@
     <gazebo reference="${sensorName}_Frame">
       <sensor name="${sensorName}" type="imu">
+        <always_on>true</always_on>
         <pose>${origin_xyz} ${origin_rpy} </pose>
         <imu>

Commit message: Working on adding transmission stuff.

File: robots/common/generic_models.xacro (robot description, xacro)
@@ -133,18 +133,4 @@
     </gazebo>
   </xacro:macro>
-  <xacro:macro name="revolute_joint_damped" params="jointName parent child origin_xyz origin_rpy axis damping friction *limits">
-    <joint name="${jointName}" type="revolute">
-      <origin rpy="${origin_rpy}" xyz="${origin_xyz}"/>
-      <axis xyz="${axis}"/>
-      <parent link="${parent}"/>
-      <child link="${child}"/>
-      <dynamics damping="${damping}" friction="${friction}"/>
-      <xacro:insert_block name="limits" />
-    </joint>
-    <gazebo reference="${jointName}">
-      <provideFeedback>1</provideFeedback>
-      <implicitSpringDamper>1</implicitSpringDamper>
-    </gazebo>
-  </xacro:macro>
   <xacro:macro name="revolute_joint_ex" params="jointName parent child origin_xyz origin_rpy axis damping friction *limits *controller_gains">
     <joint name="${jointName}" type="revolute">
@@ -193,3 +179,23 @@
                        origin_xyz="${origin_xyz}"/>
   </xacro:macro>
+  <xacro:macro name="simple_transmission_force_controlled_joint" params="jointName actuatorName">
+    <transmission name="${jointName}Transmission">
+      <type>transmission_interface/SimpleTransmission</type>
+      <joint name="${jointName}">
+        <hardwareInterface>hardware_interface/EffortJointInterface</hardwareInterface>
+      </joint>
+      <actuator name="${actuatorName}"/>
+    </transmission>
+  </xacro:macro>
+  <xacro:macro name="pushrod_transmission" params="transmissionName joint1Name joint2Name actuator1Name actuator2Name">
+    <transmission name="${transmissionName}">
+      <type>transmission_interface/PushrodTransmission</type>
+      <joint name="${joint1Name}">
+        <hardwareInterface>hardware_interface/EffortJointInterface</hardwareInterface>
+      </joint>
+      <joint name="${joint1Name}">
+        <hardwareInterface>hardware_interface/EffortJointInterface</hardwareInterface>
+      </joint>
+    </transmission>
+  </xacro:macro>
 </robot>

Commit message: Have leg transmissions in URDF.

File: robots/common/generic_models.xacro (robot description, xacro)
@@ -185,4 +185,14 @@
         <hardwareInterface>hardware_interface/EffortJointInterface</hardwareInterface>
       </joint>
+      <actuator name="${actuatorName}">
+      </actuator>
+    </transmission>
+  </xacro:macro>
+  <xacro:macro name="simple_transmission_position_controlled_joint" params="jointName actuatorName">
+    <transmission name="${jointName}Transmission">
+      <type>transmission_interface/SimpleTransmission</type>
+      <joint name="${jointName}">
+        <hardwareInterface>hardware_interface/PositionJointInterface</hardwareInterface>
+      </joint>
       <actuator name="${actuatorName}"/>
     </transmission>
@@ -197,4 +207,8 @@
         <hardwareInterface>hardware_interface/EffortJointInterface</hardwareInterface>
       </joint>
+       <actuator name="${actuator1Name}">
+      </actuator>
+      <actuator name="${actuator2Name}">
+      </actuator>
     </transmission>
   </xacro:macro>

File: robots/common/valkyrie_base_hw.xacro (robot description, xacro)
@@ -21,4 +21,5 @@
     <xacro:make_pinky_finger prefix="Left" reflect="1" pinky_finger_root_link="LeftPalm"/>
     <xacro:make_leg prefix="Right" reflect="-1" leg_root_link="${Pelvis_Link_Name}" />
+    <xacro:leg_transmissions prefix="Right"/>
     <xacro:v1_leg_sensors prefix="Right" reflect="-1" />
     <xacro:make_leg prefix="Left" reflect="1" leg_root_link="${Pelvis_Link_Name}" />

File: robots/valkyrie_A/xacro/arm/actuator_names.xacro (robot description, xacro)
@@ -1,8 +1,10 @@
 <?xml version="1.0" ?>
 <robot xmlns:xacro="http://www.ros.org/wiki/xacro" name="v1/arm/joint_names">
-  <xacro:property name="ShoulderPitchActuatorName" value="/Trunk/${prefix}ArmActuator" />
-  <xacro:property name="ShoulderRollActuatorName" value="/${prefix}Arm/Actuator2" />
-  <xacro:property name="ShoulderYawActuatorName" value="/${prefix}Arm/Actuator3" />
-  <xacro:property name="ElbowPitchActuatorName" value="/${prefix}Arm/Actuator4" />
-  <xacro:property name="ForearmYawActuatorName" value="/${prefix}Arm/Actuator5" />
+  <xacro:property name="ShoulderPitchActuatorName" value="${prefix}ShoulderPitchActuator" />
+  <xacro:property name="ShoulderRollActuatorName" value="${prefix}ShoulderRollActuator" />
+  <xacro:property name="ShoulderYawActuatorName" value="${prefix}ShoulderYawActuator" />
+  <xacro:property name="ElbowPitchActuatorName" value="${prefix}ElbowPitchActuator" />
+  <xacro:property name="ForearmYawActuatorName" value="${prefix}ForearmYawActuator" />
+  <xacro:property name="WristTopActuatorName" value="${prefix}WristTopActuator" />
+  <xacro:property name="WristBottomActuatorName" value="$prefix}WristBottomActuator" />
 </robot>

File: robots/valkyrie_A/xacro/leg/leg.xacro (robot description, xacro)
@@ -2,4 +2,5 @@
 <robot xmlns:xacro="http://www.ros.org/wiki/xacro" name="leg">
   <xacro:include filename="$(find val_description)/robots/valkyrie_A/xacro/leg/joint_names.xacro"/>
+  <xacro:include filename="$(find val_description)/robots/valkyrie_A/xacro/leg/actuator_names.xacro"/>
   <xacro:include filename="$(find val_description)/robots/valkyrie_A/xacro/leg/joint_axes.xacro"/>
   <xacro:include filename="$(find val_description)/robots/valkyrie_A/xacro/leg/link_names.xacro"/>
@@ -146,11 +147,10 @@
                         origin_rpy="3.14 0.0 -1.047"/>
   </xacro:macro>
-  <xacro:macro name="leg_actuators" params="name1 type1 name2 type2 name3 type3 name4 type4 name5 type5 name6 type6">
-    <actuator name="${name1}" type="${type1}"/>
-    <actuator name="${name2}" type="${type2}"/>
-    <actuator name="${name3}" type="${type3}"/>
-    <actuator name="${name4}" type="${type4}"/>
-    <actuator name="${name5}" type="${type5}"/>
-    <actuator name="${name6}" type="${type6}"/>
+  <xacro:macro name="leg_transmissions" params="prefix">
+    <xacro:simple_transmission_force_controlled_joint jointName="${HipYawJointName}" actuatorName="${HipYawActuatorName}"/>
+    <xacro:simple_transmission_force_controlled_joint jointName="${HipRollJointName}" actuatorName="${HipRollActuatorName}"/>
+    <xacro:simple_transmission_force_controlled_joint jointName="${HipPitchJointName}" actuatorName="${HipPitchActuatorName}"/>
+    <xacro:simple_transmission_force_controlled_joint jointName="${KneePitchJointName}" actuatorName="${KneePitchActuatorName}"/>
+    <xacro:pushrod_transmission transmissionName="${prefix}AnkleTransmission" joint1Name="${AnklePitchJointName}" joint2Name="${AnkleRollJointName}" actuator1Name="${AnkleInsideActuatorName}" actuator2Name="${AnkleOutsideActuatorName}" />
   </xacro:macro>
 </robot>

Commit message: Finished adding transmission info into URDF.

File: robots/common/generic_models.xacro (robot description, xacro)
@@ -198,5 +198,5 @@
     </transmission>
   </xacro:macro>
-  <xacro:macro name="pushrod_transmission" params="transmissionName joint1Name joint2Name actuator1Name actuator2Name">
+  <xacro:macro name="pushrod_transmission_force_controlled_joints" params="transmissionName joint1Name joint2Name actuator1Name actuator2Name">
     <transmission name="${transmissionName}">
       <type>transmission_interface/PushrodTransmission</type>
@@ -213,3 +213,18 @@
     </transmission>
   </xacro:macro>
+  <xacro:macro name="pushrod_transmission_position_controlled_joints" params="transmissionName joint1Name joint2Name actuator1Name actuator2Name">
+    <transmission name="${transmissionName}">
+      <type>transmission_interface/PushrodTransmission</type>
+      <joint name="${joint1Name}">
+        <hardwareInterface>hardware_interface/EffortJointInterface</hardwareInterface>
+      </joint>
+      <joint name="${joint1Name}">
+        <hardwareInterface>hardware_interface/EffortJointInterface</hardwareInterface>
+      </joint>
+       <actuator name="${actuator1Name}">
+      </actuator>
+      <actuator name="${actuator2Name}">
+      </actuator>
+    </transmission>
+  </xacro:macro>
 </robot>

File: robots/common/valkyrie_base_hw.xacro (robot description, xacro)
@@ -5,9 +5,6 @@
     <xacro:include filename="$(find val_description)/robots/valkyrie_A/xacro/common/common_bodies.xacro" />
     <xacro:make_pelvis />
-    <xacro:v1_pelvis_sensors/>
     <xacro:make_waist waist_root_link="${Pelvis_Link_Name}" />
-    <xacro:v1_trunk_sensors/>
     <xacro:make_head head_root_link="${TorsoRollLinkName}" />
-    <xacro:include_multisense_hw />
     <xacro:make_arm prefix="Right" reflect="-1" arm_root_link="${TorsoRollLinkName}" />
     <xacro:make_thumb prefix="Right" reflect="-1" thumb_root_link="RightPalm"/>
@@ -21,7 +18,15 @@
     <xacro:make_pinky_finger prefix="Left" reflect="1" pinky_finger_root_link="LeftPalm"/>
     <xacro:make_leg prefix="Right" reflect="-1" leg_root_link="${Pelvis_Link_Name}" />
+    <xacro:make_leg prefix="Left" reflect="1" leg_root_link="${Pelvis_Link_Name}" />
+    <xacro:v1_trunk_sensors/>
+    <xacro:v1_leg_sensors prefix="Left" reflect="1" />
+    <xacro:v1_leg_sensors prefix="Right" reflect="-1" />
+    <xacro:include_multisense_hw />
+    <xacro:v1_pelvis_sensors/>
+    <xacro:waist_transmissions />
+    <xacro:leg_transmissions prefix="Left"/>
     <xacro:leg_transmissions prefix="Right"/>
-    <xacro:v1_leg_sensors prefix="Right" reflect="-1" />
-    <xacro:make_leg prefix="Left" reflect="1" leg_root_link="${Pelvis_Link_Name}" />
-    <xacro:v1_leg_sensors prefix="Left" reflect="1" />
+    <xacro:arm_transmissions prefix="Left"/>
+    <xacro:arm_transmissions prefix="Right"/>
+    <xacro:neck_transmissions />
 </robot>

File: robots/valkyrie_A/xacro/arm/arm.xacro (robot description, xacro)
@@ -2,4 +2,5 @@
 <robot xmlns:xacro="http://www.ros.org/wiki/xacro" name="arm">
   <xacro:include filename="$(find val_description)/robots/valkyrie_A/xacro/arm/joint_names.xacro"/>
+  <xacro:include filename="$(find val_description)/robots/valkyrie_A/xacro/arm/actuator_names.xacro"/>
   <xacro:include filename="$(find val_description)/robots/valkyrie_A/xacro/arm/joint_axes.xacro"/>
   <xacro:include filename="$(find val_description)/robots/valkyrie_A/xacro/arm/link_names.xacro"/>
@@ -160,18 +161,11 @@
     <xacro:make_lower_arm prefix="${prefix}" reflect="${reflect}" lower_arm_root_link="${ElbowPitchLinkName}" />
   </xacro:macro>
-  <xacro:macro name="upper_arm_actuators" params="name1 type1 name2 type2 name3 type3 name4 type4">
-    <actuator name="${name1}" type="${type1}"/>
-    <actuator name="${name2}" type="${type2}"/>
-    <actuator name="${name3}" type="${type3}"/>
-    <actuator name="${name4}" type="${type4}"/>
-  </xacro:macro>
-  <xacro:macro name="lower_arm_actuators" params="name1 type1 name2 type2 name3 type3">
-    <actuator name="${name1}" type="${type1}"/>
-    <actuator name="${name2}" type="${type2}"/>
-    <actuator name="${name3}" type="${type3}"/>
-  </xacro:macro>
-  <xacro:macro name="arm_actuators" params="name1 type1 name2 type2 name3 type3 name4 type4 name5 type5 name6 type6 name7 type7">
-    <xacro:upper_arm_actuators name1="${name1}" type1="${type1}" name2="${name2}" type2="${type2}" name3="${name3}" type3="${type3}" name4="${name4}" type4="${type4}"/>
-    <xacro:lower_arm_actuators name1="${name5}" type1="${type5}" name2="${name6}" type2="${type6}" name3="${name7}" type3="${type7}" />
+  <xacro:macro name="arm_transmissions" params="prefix">
+    <xacro:simple_transmission_force_controlled_joint jointName="${ShoulderPitchJointName}" actuatorName="${ShoulderPitchActuatorName}"/>
+    <xacro:simple_transmission_force_controlled_joint jointName="${ShoulderRollJointName}" actuatorName="${ShoulderRollActuatorName}"/>
+    <xacro:simple_transmission_force_controlled_joint jointName="${ShoulderYawJointName}" actuatorName="${ShoulderYawActuatorName}"/>
+    <xacro:simple_transmission_force_controlled_joint jointName="${ElbowPitchJointName}" actuatorName="${ElbowPitchActuatorName}"/>
+    <xacro:simple_transmission_position_controlled_joint jointName="${ForearmYawActuatorName}" actuatorName="${ForearmYawActuatorName}"/>
+    <xacro:pushrod_transmission_position_controlled_joints transmissionName="${prefix}WristTransmission" joint1Name="${AnklePitchJointName}" joint2Name="${AnkleRollJointName}" actuator1Name="${AnkleInsideActuatorName}" actuator2Name="${AnkleOutsideActuatorName}" />
   </xacro:macro>
 </robot>

File: robots/valkyrie_A/xacro/head/head.xacro (robot description, xacro)
@@ -1,4 +1,5 @@
 <robot xmlns:xacro="http://www.ros.org/wiki/xacro" name="head">
   <xacro:include filename="$(find val_description)/robots/valkyrie_A/xacro/head/joint_names.xacro"/>
+  <xacro:include filename="$(find val_description)/robots/valkyrie_A/xacro/head/actuator_names.xacro"/>
   <xacro:include filename="$(find val_description)/robots/valkyrie_A/xacro/head/joint_axes.xacro"/>
   <xacro:include filename="$(find val_description)/robots/valkyrie_A/xacro/head/link_names.xacro"/>
@@ -72,8 +73,8 @@
       <xacro:fixed_joint jointName="multisense_head_root_joint" parent="${UpperNeckPitchLinkName}" child="multisense_root_link" origin_xyz="0.183585961 0.0 0.075353826" origin_rpy="-3.14159 0.130899694 0.0" />
     </xacro:macro>
-  <xacro:macro name="neck_actuators" params="name1 type1 name2 type2 name3 type3">
-    <actuator name="${name1}" type="${type1}"/>
-    <actuator name="${name2}" type="${type2}"/>
-    <actuator name="${name3}" type="${type3}"/>
-  </xacro:macro>
+    <xacro:macro name="neck_transmissions">
+      <xacro:simple_transmission_force_controlled_joint jointName="${LowerNeckPitchJointName}" actuatorName="${LowerNeckPitchActuatorName}"/>
+      <xacro:simple_transmission_force_controlled_joint jointName="${NeckYawJointName}" actuatorName="${NeckYawActuatorName}"/>
+      <xacro:simple_transmission_force_controlled_joint jointName="${UpperNeckPitchJointName}" actuatorName="${UpperNeckPitchActuatorName}"/>
+    </xacro:macro>
 </robot>

File: robots/valkyrie_A/xacro/leg/leg.xacro (robot description, xacro)
@@ -152,5 +152,5 @@
     <xacro:simple_transmission_force_controlled_joint jointName="${HipPitchJointName}" actuatorName="${HipPitchActuatorName}"/>
     <xacro:simple_transmission_force_controlled_joint jointName="${KneePitchJointName}" actuatorName="${KneePitchActuatorName}"/>
-    <xacro:pushrod_transmission transmissionName="${prefix}AnkleTransmission" joint1Name="${AnklePitchJointName}" joint2Name="${AnkleRollJointName}" actuator1Name="${AnkleInsideActuatorName}" actuator2Name="${AnkleOutsideActuatorName}" />
+    <xacro:pushrod_transmission_force_controlled_joints transmissionName="${prefix}AnkleTransmission" joint1Name="${AnklePitchJointName}" joint2Name="${AnkleRollJointName}" actuator1Name="${AnkleInsideActuatorName}" actuator2Name="${AnkleOutsideActuatorName}" />
   </xacro:macro>
 </robot>

File: robots/valkyrie_A/xacro/waist/waist.xacro (robot description, xacro)
@@ -2,4 +2,5 @@
   <!-- Properties -->
   <xacro:include filename="$(find val_description)/robots/valkyrie_A/xacro/waist/joint_names.xacro"/>
+  <xacro:include filename="$(find val_description)/robots/valkyrie_A/xacro/waist/actuator_names.xacro"/>
   <xacro:include filename="$(find val_description)/robots/valkyrie_A/xacro/waist/joint_axes.xacro"/>
   <xacro:include filename="$(find val_description)/robots/valkyrie_A/xacro/waist/joint_axes.xacro"/>
@@ -96,3 +97,7 @@
                         frameRate="60"/>
    </xacro:macro>
+   <xacro:macro name="waist_transmissions">
+    <xacro:simple_transmission_force_controlled_joint jointName="${TorsoYawJointName}" actuatorName="${TorsoYawActuatorName}"/>
+    <xacro:pushrod_transmission_position_controlled_joints transmissionName="WaistTransmission" joint1Name="${TorsoPitchJointName}" joint2Name="${TorsoRollJointName}" actuator1Name="${WaistLeftActuatorName}" actuator2Name="${WaistRightActuatorName}" />
+   </xacro:macro>
 </robot>
