Commit message: Some typo fixes.

File: robots/common/generic_models.xacro (robot description, xacro)
@@ -204,5 +204,5 @@
         <hardwareInterface>hardware_interface/EffortJointInterface</hardwareInterface>
       </joint>
-      <joint name="${joint1Name}">
+      <joint name="${joint2Name}">
         <hardwareInterface>hardware_interface/EffortJointInterface</hardwareInterface>
       </joint>
@@ -217,8 +217,8 @@
       <type>transmission_interface/PushrodTransmission</type>
       <joint name="${joint1Name}">
-        <hardwareInterface>hardware_interface/EffortJointInterface</hardwareInterface>
-      </joint>
-      <joint name="${joint1Name}">
-        <hardwareInterface>hardware_interface/EffortJointInterface</hardwareInterface>
+        <hardwareInterface>hardware_interface/PositionJointInterface</hardwareInterface>
+      </joint>
+      <joint name="${joint2Name}">
+        <hardwareInterface>hardware_interface/PositionJointInterface</hardwareInterface>
       </joint>
        <actuator name="${actuator1Name}">

File: robots/valkyrie_A/xacro/arm/arm.xacro (robot description, xacro)
@@ -166,6 +166,6 @@
     <xacro:simple_transmission_force_controlled_joint jointName="${ShoulderYawJointName}" actuatorName="${ShoulderYawActuatorName}"/>
     <xacro:simple_transmission_force_controlled_joint jointName="${ElbowPitchJointName}" actuatorName="${ElbowPitchActuatorName}"/>
-    <xacro:simple_transmission_position_controlled_joint jointName="${ForearmYawActuatorName}" actuatorName="${ForearmYawActuatorName}"/>
-    <xacro:pushrod_transmission_position_controlled_joints transmissionName="${prefix}WristTransmission" joint1Name="${AnklePitchJointName}" joint2Name="${AnkleRollJointName}" actuator1Name="${AnkleInsideActuatorName}" actuator2Name="${AnkleOutsideActuatorName}" />
+    <xacro:simple_transmission_force_controlled_joint jointName="${ForearmYawActuatorName}" actuatorName="${ForearmYawActuatorName}"/>
+    <xacro:pushrod_transmission_position_controlled_joints transmissionName="${prefix}WristTransmission" joint1Name="${WristPitchJointName}" joint2Name="${WristRollJointName}" actuator1Name="${WristTopActuatorName}" actuator2Name="${WristBottomActuatorName}" />
   </xacro:macro>
 </robot>

File: robots/valkyrie_A/xacro/head/head.xacro (robot description, xacro)
@@ -74,7 +74,7 @@
     </xacro:macro>
     <xacro:macro name="neck_transmissions">
-      <xacro:simple_transmission_force_controlled_joint jointName="${LowerNeckPitchJointName}" actuatorName="${LowerNeckPitchActuatorName}"/>
-      <xacro:simple_transmission_force_controlled_joint jointName="${NeckYawJointName}" actuatorName="${NeckYawActuatorName}"/>
-      <xacro:simple_transmission_force_controlled_joint jointName="${UpperNeckPitchJointName}" actuatorName="${UpperNeckPitchActuatorName}"/>
+      <xacro:simple_transmission_position_controlled_joint jointName="${LowerNeckPitchJointName}" actuatorName="${LowerNeckPitchActuatorName}"/>
+      <xacro:simple_transmission_position_controlled_joint jointName="${NeckYawJointName}" actuatorName="${NeckYawActuatorName}"/>
+      <xacro:simple_transmission_position_controlled_joint jointName="${UpperNeckPitchJointName}" actuatorName="${UpperNeckPitchActuatorName}"/>
     </xacro:macro>
 </robot>
