Commit message: Added role and transmission interface type to urdf.

File: model/robots/common/xacro/common_bodies.xacro (robot description, xacro)
@@ -5,4 +5,5 @@
     <xacro:include filename="$(find val_description)/model/robots/common/xacro/arm/arm.xacro" />
     <xacro:include filename="$(find val_description)/model/robots/common/xacro/thumb/thumb.xacro" />
+    <xacro:include filename="$(find val_description)/model/robots/common/xacro/leg/leg.xacro" />
     <xacro:include filename="$(find val_description)/model/robots/common/xacro/index_finger/index_finger.xacro" />
     <xacro:include filename="$(find val_description)/model/robots/common/xacro/middle_finger/middle_finger.xacro" />

File: model/robots/common/xacro/generic_models.xacro (robot description, xacro)
@@ -184,7 +184,9 @@
       <joint name="${jointName}">
         <hardwareInterface>hardware_interface/EffortJointInterface</hardwareInterface>
+        <interface name="JointToActuatorPositionInterface"/>
       </joint>
       <actuator name="${actuatorName}">
         <node name="${nodeName}"/>
+        <interface name="ActuatorToJointPositionInterface"/>
       </actuator>
     </transmission>
@@ -195,24 +197,34 @@
       <joint name="${jointName}">
         <hardwareInterface>hardware_interface/PositionJointInterface</hardwareInterface>
+        <interface name="JointToActuatorPositionInterface"/>
       </joint>
       <actuator name="${actuatorName}">
         <node name="${nodeName}"/>
+        <interface name="ActuatorToJointPositionInterface"/>
     </actuator>
     </transmission>
   </xacro:macro>
-  <xacro:macro name="pushrod_transmission_force_controlled_joints" params="transmissionName joint1Name joint2Name actuator1Name actuator2Name actuator1Node actuator2Node">
+  <xacro:macro name="pushrod_transmission_force_controlled_joints" params="transmissionName joint1Name joint2Name actuator1Name actuator2Name actuator1Node actuator2Node joint1Role joint2Role actuator1Role actuator2Role">
     <transmission name="${transmissionName}">
       <type>transmission_interface/PushrodTransmission</type>
       <joint name="${joint1Name}">
         <hardwareInterface>hardware_interface/EffortJointInterface</hardwareInterface>
+        <interface name="JointToActuatorEffortInterface"/>
+        <role>${joint1Role}</role>
       </joint>
       <joint name="${joint2Name}">
         <hardwareInterface>hardware_interface/EffortJointInterface</hardwareInterface>
+        <interface name="JointToActuatorEffortInterface"/>
+        <role>${joint2Role}</role>
       </joint>
        <actuator name="${actuator1Name}">
         <node name="${actuator1Node}"/>
+        <interface name="ActuatorToJointEffortInterface"/>
+        <role>${actuator1Role}</role>
       </actuator>
       <actuator name="${actuator2Name}">
         <node name="${actuator2Node}"/>
+        <interface name="ActuatorToJointEffortInterface"/>
+        <role>${actuator2Role}</role>
       </actuator>
     </transmission>
@@ -223,13 +235,17 @@
       <joint name="${joint1Name}">
         <hardwareInterface>hardware_interface/PositionJointInterface</hardwareInterface>
+        <interface name="JointToActuatorPositionInterface"/>
       </joint>
       <joint name="${joint2Name}">
         <hardwareInterface>hardware_interface/PositionJointInterface</hardwareInterface>
+        <interface name="JointToActuatorPositionInterface"/>
       </joint>
        <actuator name="${actuator1Name}">
         <node name="${actuator1Node}"/>
+        <interface name="ActuatorToJointPositionInterface"/>
       </actuator>
       <actuator name="${actuator2Name}">
         <node name="${actuator2Node}"/>
+        <interface name="ActuatorToJointPositionInterface"/>
       </actuator>
     </transmission>

File: model/robots/common/xacro/leg/frame_parameters.xacro (robot description, xacro)
@@ -1,4 +1,4 @@
 <?xml version="1.0" ?>
-<robot xmlns:xacro="http://www.ros.org/wiki/xacro" name="leg_frame_parameters">
+<robot xmlns:xacro="http://www.ros.org/wiki/xacro" name="v1/leg/dh_parameters">
   <xacro:property name="HipYawFrameOrigin_X" value="0.0"/>
   <xacro:property name="HipYawFrameOrigin_Y" value="${reflect * 0.1016}"/>
@@ -19,21 +19,21 @@
   <xacro:property name="HipPitchFrameOrientation_Pitch" value="0.0"/>
   <xacro:property name="HipPitchFrameOrientation_Yaw" value="0.0"/>
-  <xacro:property name="KneePitchFrameOrigin_X" value="0.0001"/>
-  <xacro:property name="KneePitchFrameOrigin_Y" value="${reflect * 0.0361}"/>
-  <xacro:property name="KneePitchFrameOrigin_Z" value="-0.4306"/>
+  <xacro:property name="KneePitchFrameOrigin_X" value="0.000112225"/>
+  <xacro:property name="KneePitchFrameOrigin_Y" value="${reflect * 0.0361046}"/>
+  <xacro:property name="KneePitchFrameOrigin_Z" value="-0.430959"/>
   <xacro:property name="KneePitchFrameOrientation_Roll" value="0.0"/>
   <xacro:property name="KneePitchFrameOrientation_Pitch" value="0.0"/>
   <xacro:property name="KneePitchFrameOrientation_Yaw" value="0.0"/>
-  <xacro:property name="AnklePitchFrameOrigin_X" value="-0.0103"/>
+  <xacro:property name="AnklePitchFrameOrigin_X" value="-0.0102381"/>
   <xacro:property name="AnklePitchFrameOrigin_Y" value="0.0"/>
-  <xacro:property name="AnklePitchFrameOrigin_Z" value="-0.4064"/>
+  <xacro:property name="AnklePitchFrameOrigin_Z" value="-0.40627"/>
   <xacro:property name="AnklePitchFrameOrientation_Roll" value="0.0"/>
   <xacro:property name="AnklePitchFrameOrientation_Pitch" value="0.0"/>
   <xacro:property name="AnklePitchFrameOrientation_Yaw" value="0.0"/>
-  <xacro:property name="AnkleRollFrameOrigin_X" value="0.0017"/>
+  <xacro:property name="AnkleRollFrameOrigin_X" value="0.0"/>
   <xacro:property name="AnkleRollFrameOrigin_Y" value="0.0"/>
-  <xacro:property name="AnkleRollFrameOrigin_Z" value="-0.0126"/>
+  <xacro:property name="AnkleRollFrameOrigin_Z" value="0.0"/>
   <xacro:property name="AnkleRollFrameOrientation_Roll" value="0.0"/>
-  <xacro:property name="AnkleRollFrameOrientation_Pitch" value="-0.1309"/>
+  <xacro:property name="AnkleRollFrameOrientation_Pitch" value="0.0"/>
   <xacro:property name="AnkleRollFrameOrientation_Yaw" value="0.0"/>
 </robot>

File: model/robots/common/xacro/leg/leg.xacro (robot description, xacro)
@@ -4,9 +4,9 @@
   <xacro:include filename="$(find val_description)/common/xacro/actuator_names/valkyrie_actuator_names.xacro"/>
   <xacro:include filename="$(find val_description)/common/xacro/nodes/valkyrie_nodes.xacro"/>
-  <xacro:include filename="$(find val_description)/model/robots/valkyrie_A/xacro/leg/joint_axes.xacro"/>
-  <xacro:include filename="$(find val_description)/model/robots/valkyrie_A/xacro/leg/link_names.xacro"/>
-  <xacro:include filename="$(find val_description)/model/robots/valkyrie_A/xacro/leg/joint_limits.xacro"/>
-  <xacro:include filename="$(find val_description)/model/robots/valkyrie_A/xacro/leg/frame_parameters.xacro"/>
-  <xacro:include filename="$(find val_description)/model/robots/valkyrie_A/xacro/leg/mass_parameters.xacro"/>
+  <xacro:include filename="$(find val_description)/model/robots/common/xacro/leg/joint_axes.xacro"/>
+  <xacro:include filename="$(find val_description)/model/robots/common/xacro/leg/link_names.xacro"/>
+  <xacro:include filename="$(find val_description)/model/robots/common/xacro/leg/joint_limits.xacro"/>
+  <xacro:include filename="$(find val_description)/model/robots/common/xacro/leg/frame_parameters.xacro"/>
+  <xacro:include filename="$(find val_description)/model/robots/common/xacro/leg/mass_parameters.xacro"/>
   <xacro:include filename="$(find val_description)/model/robots/common/xacro/sensors/ati_force_torque.xacro"/>
   <xacro:macro name="make_leg_links" params="prefix reflect leg_root_link">
@@ -153,5 +153,5 @@
     <xacro:simple_transmission_force_controlled_joint jointName="${HipPitchJointName}" actuatorName="${HipPitchActuatorName}" nodeName="${HipPitchNode}"/>
     <xacro:simple_transmission_force_controlled_joint jointName="${KneePitchJointName}" actuatorName="${KneePitchActuatorName}" nodeName="${KneePitchNode}"/>
-    <xacro:pushrod_transmission_force_controlled_joints transmissionName="${prefix}AnkleTransmission" joint1Name="${AnklePitchJointName}" joint2Name="${AnkleRollJointName}" actuator1Name="${AnkleInsideActuatorName}" actuator2Name="${AnkleOutsideActuatorName}" actuator1Node="${AnkleInsideActuatorNode}" actuator2Node="${AnkleOutsideActuatorNode}"/>
+    <xacro:pushrod_transmission_force_controlled_joints transmissionName="${prefix}AnkleTransmission" joint1Name="${AnklePitchJointName}" joint2Name="${AnkleRollJointName}" actuator1Name="${AnkleInsideActuatorName}" actuator2Name="${AnkleOutsideActuatorName}" actuator1Node="${AnkleInsideActuatorNode}" actuator2Node="${AnkleOutsideActuatorNode}" joint1Role="pitch" joint2Role="roll" actuator1Role="insideActuator" actuator2Role="outsideActuator"/>
   </xacro:macro>
 </robot>

File: model/robots/common/xacro/waist/waist.xacro (robot description, xacro)
@@ -99,5 +99,5 @@
    <xacro:macro name="waist_transmissions">
     <xacro:simple_transmission_force_controlled_joint jointName="${TorsoYawJointName}" actuatorName="${TorsoYawActuatorName}" nodeName="${TrunkYawNode}"/>
-    <xacro:pushrod_transmission_position_controlled_joints transmissionName="WaistTransmission" joint1Name="${TorsoPitchJointName}" joint2Name="${TorsoRollJointName}" actuator1Name="${WaistLeftActuatorName}" actuator2Name="${WaistRightActuatorName}" actuator1Node="${WaistLeftActuatorNode}" actuator2Node="${WaistRightActuatorNode}"/>
+    <!-- <xacro:pushrod_transmission_force_controlled_joints transmissionName="WaistTransmission" joint1Name="${TorsoPitchJointName}" joint2Name="${TorsoRollJointName}" actuator1Name="${WaistLeftActuatorName}" actuator2Name="${WaistRightActuatorName}" actuator1Node="${WaistLeftActuatorNode}" actuator2Node="${WaistRightActuatorNode}" joint1Role="pitch" joint2Roll="roll" actuator1Roll="leftActuator" actuator2Roll="rightActuator"/> -->
    </xacro:macro>
 </robot>

File: model/robots/valkyrie_A_hw.xacro (robot description, xacro)
@@ -4,5 +4,4 @@
     <xacro:include filename="$(find val_description)/model/materials/materials.xacro" />
     <xacro:include filename="$(find val_description)/model/robots/common/xacro/common_bodies.xacro" />
-    <xacro:include filename="$(find val_description)/model/robots/valkyrie_A/xacro/leg/leg.xacro" />
     <xacro:include filename="$(find val_description)/model/robots/common/xacro/valkyrie_base_hw.xacro"/>
 </robot>

File: model/robots/valkyrie_A_sim.xacro (robot description, xacro)
@@ -4,5 +4,4 @@
     <xacro:include filename="$(find val_description)/model/materials/materials.xacro" />
     <xacro:include filename="$(find val_description)/model/robots/common/xacro/common_bodies.xacro" />
-    <xacro:include filename="$(find val_description)/model/robots/valkyrie_A/xacro/leg/leg.xacro" />
     <xacro:include filename="$(find val_description)/model/robots/common/xacro/valkyrie_base_sim.xacro"/>
     <xacro:include filename="$(find val_description)/model/urdf/multisense_sl.urdf" />

File: model/robots/valkyrie_B_hw.xacro (robot description, xacro)
@@ -4,5 +4,4 @@
     <xacro:include filename="$(find val_description)/model/materials/materials.xacro" />
     <xacro:include filename="$(find val_description)/model/robots/common/xacro/common_bodies.xacro" />
-    <xacro:include filename="$(find val_description)/model/robots/valkyrie_B/xacro/leg/leg.xacro" />
     <xacro:include filename="$(find val_description)/model/robots/common/xacro/valkyrie_base_hw.xacro"/>
 </robot>

File: model/robots/valkyrie_B_sim.xacro (robot description, xacro)
@@ -4,5 +4,4 @@
     <xacro:include filename="$(find val_description)/model/materials/materials.xacro" />
     <xacro:include filename="$(find val_description)/model/robots/common/xacro/common_bodies.xacro" />
-    <xacro:include filename="$(find val_description)/model/robots/valkyrie_B/xacro/leg/leg.xacro" />
     <xacro:include filename="$(find val_description)/model/robots/common/xacro/valkyrie_base_sim.xacro"/>
     <xacro:include filename="$(find val_description)/model/urdf/multisense_sl.urdf" />
