Commit message: Fixed install path of urdf and instance files.

File: model/robots/common/xacro/generic_models.xacro (robot description, xacro)
@@ -49,4 +49,29 @@
         </geometry>
         <origin rpy="${origin_rpy}" xyz="${origin_xyz}"/>
+      </collision>
+    </link>
+  </xacro:macro>
+  <xacro:macro name="link_box_collision_mesh_visual"
+          params="name width height depth mass inertial_xyz inertial_rpy ixx ixy ixz iyy iyz izz visual_mesh material box_xyz box_rpy">
+    <link name="${name}">
+      <inertial>
+        <mass value="${mass}" />
+        <origin rpy="${inertial_rpy}" xyz="${inertial_xyz}"/>
+        <inertia ixx="${ixx}"  ixy="${ixy}" ixz="${ixz}"
+                 iyy="${iyy}" iyz="${iyz}"
+                 izz="${izz}" />
+      </inertial>
+      <visual>
+        <geometry>
+          <mesh filename="${visual_mesh}"/>
+        </geometry>
+        <origin rpy="0 0 0" xyz="0 0 0"/>
+        <material name="${material}"/>
+      </visual>
+      <collision>
+        <geometry>
+          <box size="${width} ${height} ${depth}"/>
+        </geometry>
+        <origin rpy="${box_rpy}" xyz="${box_xyz}"/>
       </collision>
     </link>

File: model/robots/common/xacro/leg/leg.xacro (robot description, xacro)
@@ -56,5 +56,5 @@
                     material="White"
                     collision_mesh="${mesh_root}/legs/lj5.dae"/>
-    <xacro:standard_link name="${AnkleRollLinkName}"
+    <!-- <xacro:standard_link name="${AnkleRollLinkName}"
                     mass="${FootMass}"
                     origin_xyz="${FootComPosition}"
@@ -64,5 +64,18 @@
                     visual_mesh="${mesh_root}/legs/foot.dae"
                     material="White"
-                    collision_mesh="${mesh_root}/legs/foot.dae" />
+                    collision_mesh="${mesh_root}/legs/foot.dae" /> -->
+    <xacro:link_box_collision_mesh_visual name="${AnkleRollLinkName}"
+                    mass="${FootMass}"
+                    inertial_xyz="${FootComPosition}"
+                    ixx="${FootInertia_IXX}" ixy="${FootInertia_IXY}" ixz="${FootInertia_IXZ}"
+                    iyy="${FootInertia_IYY}" iyz="${FootInertia_IYZ}" izz="${FootInertia_IZZ}"
+                    inertial_rpy="0 0 0"
+                    visual_mesh="${mesh_root}/legs/foot_${prefix}.dae"
+                    material="White"
+                    width="0.27"
+                    height="0.16"
+                    depth="0.064"
+                    box_xyz="0.06 0.0 -0.06"
+                    box_rpy="0.0 0.0 0.0" />
   </xacro:macro>
   <xacro:macro name="make_leg_joints" params="prefix reflect leg_root_link">

Commit message: added macro for position interface and update neck to use position interface

File: model/robots/common/xacro/generic_models.xacro (robot description, xacro)
@@ -215,4 +215,17 @@
     </transmission>
   </xacro:macro>
+  <xacro:macro name="simple_position_transmission" params="jointName actuatorName nodeName actuatorApi">
+    <transmission name="${jointName}Transmission">
+      <type>transmission_interface/SimpleTransmission</type>
+      <joint name="${jointName}">
+        <hardwareInterface>PositionJointInterface</hardwareInterface>
+      </joint>
+      <actuator name="${actuatorName}">
+        <node name="${nodeName}"/>
+        <mechanicalReduction>1</mechanicalReduction>
+        <api name="${actuatorApi}" />
+      </actuator>
+    </transmission>
+  </xacro:macro>
   <xacro:macro name="pushrod_transmission" params="transmissionName transmissionType joint1Name joint2Name joint1Role joint2Role actuator1Name actuator2Name actuator1Node actuator2Node actuator1Api actuator2Api actuator1Role actuator2Role">
     <transmission name="${transmissionName}">

File: model/robots/common/xacro/head/head.xacro (robot description, xacro)
@@ -73,7 +73,7 @@
     </xacro:macro>
     <xacro:macro name="neck_transmissions_hw">
-      <xacro:simple_transmission jointName="${LowerNeckPitchJointName}" actuatorName="${LowerNeckPitchActuatorName}" nodeName="${LowerNeckPitchNode}" actuatorApi="${LowerNeckPitchApi}"/>
-      <xacro:simple_transmission jointName="${NeckYawJointName}" actuatorName="${NeckYawActuatorName}" nodeName="${NeckYawNode}" actuatorApi="${NeckYawApi}"/>
-      <xacro:simple_transmission jointName="${UpperNeckPitchJointName}" actuatorName="${UpperNeckPitchActuatorName}" nodeName="${UpperNeckPitchNode}" actuatorApi="${UpperNeckPitchApi}"/>
+      <xacro:simple_position_transmission jointName="${LowerNeckPitchJointName}" actuatorName="${LowerNeckPitchActuatorName}" nodeName="${LowerNeckPitchNode}" actuatorApi="${LowerNeckPitchApi}"/>
+      <xacro:simple_position_transmission jointName="${NeckYawJointName}" actuatorName="${NeckYawActuatorName}" nodeName="${NeckYawNode}" actuatorApi="${NeckYawApi}"/>
+      <xacro:simple_position_transmission jointName="${UpperNeckPitchJointName}" actuatorName="${UpperNeckPitchActuatorName}" nodeName="${UpperNeckPitchNode}" actuatorApi="${UpperNeckPitchApi}"/>
     </xacro:macro>
     <xacro:macro name="neck_transmissions_sim">
