Commit message: Fixed Franks imu xacro since I removed the old _api file.

File: model/robots/common/xacro/valkyrie_imu_base.xacro (robot description, xacro)
@@ -1,3 +1,4 @@
 <robot xmlns:xacro="http://ros.org/wiki/xacro" name="valkyrie">
+    <xacro:property name="KVHHardwareApi" value="val_imu_kvh_1750_interface/ImuKVHInterface" />
     <xacro:make_pelvis />
     <xacro:include_multisense_hw />
