Commit message: Searching through neck transforms for an error but didn't find anything.

File: model/robots/common/xacro/head/frame_parameters.xacro (robot description, xacro)
@@ -1,11 +1,11 @@
 <?xml version="1.0" ?>
 <robot xmlns:xacro="http://www.ros.org/wiki/xacro" name="v1/head/dh_parameters">
-  <xacro:property name="LowerNeckPitchFrameOrigin_X" value="0.0204"/>
+  <xacro:property name="LowerNeckPitchFrameOrigin_X" value="0.0203518"/>
   <xacro:property name="LowerNeckPitchFrameOrigin_Y" value="0.0"/>
-  <xacro:property name="LowerNeckPitchFrameOrigin_Z" value="0.3385"/>
+  <xacro:property name="LowerNeckPitchFrameOrigin_Z" value="0.33845"/>
   <xacro:property name="LowerNeckPitchFrameOrientation_Roll" value="0.0"/>
   <xacro:property name="LowerNeckPitchFrameOrientation_Pitch" value="0.0"/>
   <xacro:property name="LowerNeckPitchFrameOrientation_Yaw" value="0.0"/>
-  <xacro:property name="NeckYawFrameOrigin_X" value="-0.0519"/>
+  <xacro:property name="NeckYawFrameOrigin_X" value="-0.051924"/>
   <xacro:property name="NeckYawFrameOrigin_Y" value="0.0"/>
   <xacro:property name="NeckYawFrameOrigin_Z" value="0.0"/>
@@ -15,5 +15,5 @@
   <xacro:property name="UpperNeckPitchFrameOrigin_X" value="-0.06"/>
   <xacro:property name="UpperNeckPitchFrameOrigin_Y" value="0"/>
-  <xacro:property name="UpperNeckPitchFrameOrigin_Z" value="0.196"/>
+  <xacro:property name="UpperNeckPitchFrameOrigin_Z" value="0.195997"/>
   <xacro:property name="UpperNeckPitchFrameOrientation_Roll" value="0.0"/>
   <xacro:property name="UpperNeckPitchFrameOrientation_Pitch" value="0.0"/>
