Commit message: Added instance files for units B and C.

File: instance/instances/robots/valkyrie_A.xacro (robot description, xacro)
@@ -1,4 +1,5 @@
-<robot xmlns:xacro="http://ros.org/wiki/xacro" name="valkyrie">
+<robot xmlns:xacro="http://ros.org/wiki/xacro" name="valkyrie_A">
 	<xacro:property name="instance" value="valkyrie_A" />
+	<xacro:include filename="$(find val_description)/instance/instances/robots/xacro/serial_numbers/valkyrie_A_serials.xacro" />
     <xacro:include filename="$(find val_description)/instance/instances/robots/xacro/common/valkyrie_full_template.xacro"/>
 </robot>

File: instance/instances/robots/xacro/common/valkyrie_full_template.xacro (robot description, xacro)
@@ -1,4 +1,3 @@
 <robot xmlns:xacro="http://ros.org/wiki/xacro" name="valkyrie_template">
-	<xacro:include filename="$(find val_description)/instance/instances/robots/xacro/serial_numbers/valkyrie_A_serials.xacro" />
 	<xacro:include filename="$(find val_description)/common/xacro/nodes/valkyrie_nodes.xacro" />
 	<xacro:include filename="$(find val_description)/instance/instances/robots/xacro/limbs/leg.xacro" />
@@ -11,10 +10,10 @@
 	<xacro:all_channels/>
 	<Mechanisms>
-		<xacro:leg prefix="left" j1_serial_number="${leftLegJ1SerialNumber}" j2_serial_number="${leftLegJ2SerialNumber}" j3_serial_number="${leftLegJ3SerialNumber}" j4_serial_number="${leftLegJ4SerialNumber}" ankle_actuator0_serial="${leftAnkleActuator0SerialNumber}" ankle_actuator1_serial="${leftAnkleActuator1SerialNumber}"/>
-		<xacro:leg prefix="right" j1_serial_number="${rightLegJ1SerialNumber}" j2_serial_number="${rightLegJ2SerialNumber}" j3_serial_number="${rightLegJ3SerialNumber}" j4_serial_number="${rightLegJ4SerialNumber}" ankle_actuator0_serial="${rightAnkleActuator0SerialNumber}" ankle_actuator1_serial="${rightAnkleActuator1SerialNumber}" />
+		<xacro:leg prefix="left" j1_serial_number="${leftLegJ1SerialNumber}" j2_serial_number="${leftLegJ2SerialNumber}" j3_serial_number="${leftLegJ3SerialNumber}" j4_serial_number="${leftLegJ4SerialNumber}" ankle_left_actuator_serial="${leftAnkleActuator0SerialNumber}" ankle_right_actuator_serial="${leftAnkleActuator1SerialNumber}"/>
+		<xacro:leg prefix="right" j1_serial_number="${rightLegJ1SerialNumber}" j2_serial_number="${rightLegJ2SerialNumber}" j3_serial_number="${rightLegJ3SerialNumber}" j4_serial_number="${rightLegJ4SerialNumber}" ankle_left_actuator_serial="${rightAnkleActuator0SerialNumber}" ankle_right_actuator_serial="${rightAnkleActuator1SerialNumber}" />
 		<xacro:arm prefix="left" j1_serial_number="${leftArmJ1SerialNumber}" j2_serial_number="${leftArmJ2SerialNumber}" j3_serial_number="${leftArmJ3SerialNumber}" j4_serial_number="${leftArmJ4SerialNumber}" j5_serial_number="${leftArmJ5SerialNumber}" wrist_actuator0_serial="${leftAnkleActuator0SerialNumber}" wrist_actuator1_serial="${leftAnkleActuator1SerialNumber}" />
 		<xacro:arm prefix="right" j1_serial_number="${rightArmJ1SerialNumber}" j2_serial_number="${rightArmJ2SerialNumber}" j3_serial_number="${rightArmJ3SerialNumber}" j4_serial_number="${rightArmJ4SerialNumber}" j5_serial_number="${rightArmJ5SerialNumber}" wrist_actuator0_serial="${rightAnkleActuator0SerialNumber}" wrist_actuator1_serial="${rightAnkleActuator1SerialNumber}" />
 		<xacro:neck j1_serial_number="${neckJ1SerialNumber}" j2_serial_number="${neckJ1SerialNumber}" j3_serial_number="${neckJ1SerialNumber}" />
-		<xacro:waist j1_serial_number="${trunkSerialNumber}" waist_actuator0_serial="${waistActuator0SerialNumber}" waist_actuator1_serial="${waistActuator1SerialNumber}"/>
+		<xacro:waist j1_serial_number="${trunkSerialNumber}" waist_left_actuator_serial="${waistLeftActuatorSerialNumber}" waist_right_actuator_serial="${waistRightActuatorSerialNumber}"/>
 	</Mechanisms>
 	<Devices>

File: instance/instances/robots/xacro/limbs/arm.xacro (robot description, xacro)
@@ -8,5 +8,5 @@
     	<xacro:simple_mechanism name="${ElbowPitchJointName}" serial_number="${j4_serial_number}" node="${ElbowPitchNode}"/>
     	<xacro:simple_mechanism name="${ForearmYawJointName}" serial_number="${j5_serial_number}" node="${ForearmYawNode}"/>
-    	<xacro:two_active_joint_mechanism mechanism_name="${prefix}Wrist" joint0_name="${WristPitchJointName}" joint1_name="${WristRollJointName}" actuator0_serial="${wrist_actuator0_serial}" actuator1_serial="${wrist_actuator1_serial}" actuator0_node="${WristTopActuatorNode}" actuator1_node="${WristBottomActuatorNode}" />
+    	<xacro:two_active_joint_mechanism mechanism_name="wrist" actuator0_name="${prefix}WristTopActuator" actuator1_name="${prefix}WristBottomActuator" joint0_name="${WristPitchJointName}" joint1_name="${WristRollJointName}" actuator0_serial="${wrist_actuator0_serial}" actuator1_serial="${wrist_actuator1_serial}" actuator0_node="${WristTopActuatorNode}" actuator1_node="${WristBottomActuatorNode}" />
     </xacro:macro>
 </robot>

File: instance/instances/robots/xacro/limbs/leg.xacro (robot description, xacro)
@@ -2,10 +2,10 @@
     <xacro:include filename="$(find val_description)/instance/instances/robots/xacro/mechanisms/mechanisms.xacro"/>
     <xacro:include filename="$(find val_description)/common/xacro/joint_names/valkyrie_joint_names.xacro"/>
-    <xacro:macro name="leg" params="prefix j1_serial_number j2_serial_number j3_serial_number j4_serial_number ankle_actuator0_serial ankle_actuator1_serial" >
+    <xacro:macro name="leg" params="prefix j1_serial_number j2_serial_number j3_serial_number j4_serial_number ankle_left_actuator_serial ankle_right_actuator_serial" >
     	<xacro:simple_mechanism name="${HipYawJointName}" serial_number="${j1_serial_number}" node="${HipYawNode}"/>
     	<xacro:simple_mechanism name="${HipRollJointName}" serial_number="${j2_serial_number}" node="${HipRollNode}"/>
     	<xacro:simple_mechanism name="${HipPitchJointName}" serial_number="${j3_serial_number}" node="${HipPitchNode}"/>
     	<xacro:simple_mechanism name="${KneePitchJointName}" serial_number="${j4_serial_number}" node="${KneePitchNode}"/>
-    	<xacro:two_active_joint_mechanism mechanism_name="${prefix}Ankle" joint0_name="${AnklePitchJointName}" joint1_name="${AnkleRollJointName}" actuator0_serial="${ankle_actuator0_serial}" actuator1_serial="${ankle_actuator1_serial}" actuator0_node="${AnkleInsideActuatorNode}" actuator1_node="${AnkleOutsideActuatorNode}" />
+    	<xacro:two_active_joint_mechanism mechanism_name="ankle" actuator0_name="${prefix}AnkleLeftActuator" actuator1_name="${prefix}AnkleRightActuator" joint0_name="${AnklePitchJointName}" joint1_name="${AnkleRollJointName}" actuator0_serial="${ankle_left_actuator_serial}" actuator1_serial="${ankle_right_actuator_serial}" actuator0_node="${AnkleInsideActuatorNode}" actuator1_node="${AnkleOutsideActuatorNode}" />
     </xacro:macro>
 </robot>

File: instance/instances/robots/xacro/limbs/waist.xacro (robot description, xacro)
@@ -1,7 +1,7 @@
 <robot xmlns:xacro="http://ros.org/wiki/xacro" name="waist">
     <xacro:include filename="$(find val_description)/instance/instances/robots/xacro/mechanisms/mechanisms.xacro"/>
-    <xacro:macro name="waist" params="j1_serial_number waist_actuator0_serial waist_actuator1_serial" >
+    <xacro:macro name="waist" params="j1_serial_number waist_left_actuator_serial waist_right_actuator_serial" >
     	<xacro:simple_mechanism name="torso_yaw" serial_number="${j1_serial_number}" node="${TrunkYawNode}"/>
-    	<xacro:two_active_joint_mechanism mechanism_name="waist" joint0_name="pitch" joint1_name="roll" actuator0_serial="${waist_actuator0_serial}" actuator1_serial="${waist_actuator1_serial}" actuator0_node="${WaistLeftActuatorNode}" actuator1_node="${WaistRightActuatorNode}" />
+    	<xacro:two_active_joint_mechanism mechanism_name="waist" actuator0_name="waistLeftActuator" actuator1_name="waistRightActuator" joint0_name="pitch" joint1_name="roll" actuator0_serial="${waist_left_actuator_serial}" actuator1_serial="${waist_right_actuator_serial}" actuator0_node="${WaistLeftActuatorNode}" actuator1_node="${WaistRightActuatorNode}" />
     </xacro:macro>
 </robot>

File: instance/instances/robots/xacro/mechanisms/mechanisms.xacro (robot description, xacro)
@@ -16,10 +16,10 @@
 	</Actuator>
 </xacro:macro>
-<xacro:macro name="two_active_joint_mechanism" params="mechanism_name joint0_name joint1_name actuator0_serial actuator0_node actuator1_serial actuator1_node " >
+<xacro:macro name="two_active_joint_mechanism" params="mechanism_name actuator0_name actuator1_name joint0_name joint1_name actuator0_serial actuator0_node actuator1_serial actuator1_node " >
 	<Mechanism id="${mechanism_name}" type="complex">
 		<xacro:joint name="${joint0_name}" type="active" calibration_file="${instance}_${mechanism_name}_${joint0_name}_cal.xml"/>
 		<xacro:joint name="${joint1_name}" type="active" calibration_file="${instance}_${mechanism_name}_${joint1_name}_cal.xml"/>
-		<xacro:actuator name="${mechanism_name}_actuator0" serial_number="${actuator0_serial}" node="${actuator0_node}" />
-		<xacro:actuator name="${mechanism_name}_actuator1" serial_number="${actuator1_serial}" node="${actuator1_node}" />
+		<xacro:actuator name="${actuator0_name}" serial_number="${actuator0_serial}" node="${actuator0_node}" />
+		<xacro:actuator name="${actuator1_name}" serial_number="${actuator1_serial}" node="${actuator1_node}" />
 	</Mechanism>
 </xacro:macro>

File: instance/instances/robots/xacro/serial_numbers/valkyrie_A_serials.xacro (robot description, xacro)
@@ -17,6 +17,6 @@
 	<xacro:property name="leftArmJ4SerialNumber" value="v_f_002" />
 	<xacro:property name="leftArmJ5SerialNumber" value="v_g_005" />
-	<xacro:property name="leftWristActuator0SerialNumber" value="v_h_001" />
-	<xacro:property name="leftWristActuator1SerialNumber" value="v_h_002" />
+	<xacro:property name="leftWristActuator0SerialNumber" value="UNKNOWN" />
+	<xacro:property name="leftWristActuator1SerialNumber" value="UNKNOWN" />
 	<xacro:property name="rightArmJ1SerialNumber" value="v_a_001" />
 	<xacro:property name="rightArmJ2SerialNumber" value="v_b_003" />
@@ -24,17 +24,17 @@
 	<xacro:property name="rightArmJ4SerialNumber" value="v_f_003" />
 	<xacro:property name="rightArmJ5SerialNumber" value="v_g_003" />
-	<xacro:property name="rightWristActuator0SerialNumber" value="v_h_003" />
-	<xacro:property name="rightWristActuator1SerialNumber" value="v_h_004" />
+	<xacro:property name="rightWristActuator0SerialNumber" value="UNKNOWN" />
+	<xacro:property name="rightWristActuator1SerialNumber" value="UNKNOWN" />
 	<xacro:property name="neckJ1SerialNumber" value="v_g_006" />
 	<xacro:property name="neckJ2SerialNumber" value="v_g_007" />
 	<xacro:property name="neckJ3SerialNumber" value="v_g_008" />
 	<xacro:property name="trunkSerialNumber" value="v_a_004" />
-	<xacro:property name="waistActuator0SerialNumber" value="v_e_005" />
-	<xacro:property name="waistActuator1SerialNumber" value="v_e_006" />
-	<xacro:property name="pelvis_imu1_serial" value="134bs144" />
-	<xacro:property name="pelvis_imu2_serial" value="234bs144" />
-	<xacro:property name="torso_imu1_serial" value="134bs135" />
-	<xacro:property name="torso_imu2_serial" value="134b13144" />
-	<xacro:property name="left_foot_ATI_serial" value="FT11223" />
-	<xacro:property name="right_foot_ATI_serial" value="FT11353" />
+	<xacro:property name="waistRightActuatorSerialNumber" value="v_e_005" />
+	<xacro:property name="waistLeftActuatorSerialNumber" value="v_e_006" />
+	<xacro:property name="pelvis_imu1_serial" value="UNKNOWN" />
+	<xacro:property name="pelvis_imu2_serial" value="UNKNOWN" />
+	<xacro:property name="torso_imu1_serial" value="UNKNOWN" />
+	<xacro:property name="torso_imu2_serial" value="UNKNOWN" />
+	<xacro:property name="left_foot_ATI_serial" value="FT14020" />
+	<xacro:property name="right_foot_ATI_serial" value="FT16592" />
 </robot>
