Commit message: Fixed some actuator naming.

File: instance/instances/robots/xacro/common/valkyrie_full_template.xacro (robot description, xacro)
@@ -10,8 +10,8 @@
 	<xacro:all_channels/>
 	<Mechanisms>
-		<xacro:leg prefix="left" j1_serial_number="${leftLegJ1SerialNumber}" j2_serial_number="${leftLegJ2SerialNumber}" j3_serial_number="${leftLegJ3SerialNumber}" j4_serial_number="${leftLegJ4SerialNumber}" ankle_left_actuator_serial="${leftAnkleActuator0SerialNumber}" ankle_right_actuator_serial="${leftAnkleActuator1SerialNumber}"/>
-		<xacro:leg prefix="right" j1_serial_number="${rightLegJ1SerialNumber}" j2_serial_number="${rightLegJ2SerialNumber}" j3_serial_number="${rightLegJ3SerialNumber}" j4_serial_number="${rightLegJ4SerialNumber}" ankle_left_actuator_serial="${rightAnkleActuator0SerialNumber}" ankle_right_actuator_serial="${rightAnkleActuator1SerialNumber}" />
-		<xacro:arm prefix="left" j1_serial_number="${leftArmJ1SerialNumber}" j2_serial_number="${leftArmJ2SerialNumber}" j3_serial_number="${leftArmJ3SerialNumber}" j4_serial_number="${leftArmJ4SerialNumber}" j5_serial_number="${leftArmJ5SerialNumber}" wrist_actuator0_serial="${leftAnkleActuator0SerialNumber}" wrist_actuator1_serial="${leftAnkleActuator1SerialNumber}" />
-		<xacro:arm prefix="right" j1_serial_number="${rightArmJ1SerialNumber}" j2_serial_number="${rightArmJ2SerialNumber}" j3_serial_number="${rightArmJ3SerialNumber}" j4_serial_number="${rightArmJ4SerialNumber}" j5_serial_number="${rightArmJ5SerialNumber}" wrist_actuator0_serial="${rightAnkleActuator0SerialNumber}" wrist_actuator1_serial="${rightAnkleActuator1SerialNumber}" />
+		<xacro:leg prefix="left" j1_serial_number="${leftLegJ1SerialNumber}" j2_serial_number="${leftLegJ2SerialNumber}" j3_serial_number="${leftLegJ3SerialNumber}" j4_serial_number="${leftLegJ4SerialNumber}" ankle_left_actuator_serial="${leftAnkleLeftActuatorSerialNumber}" ankle_right_actuator_serial="${leftAnkleRightActuatorSerialNumber}"/>
+		<xacro:leg prefix="right" j1_serial_number="${rightLegJ1SerialNumber}" j2_serial_number="${rightLegJ2SerialNumber}" j3_serial_number="${rightLegJ3SerialNumber}" j4_serial_number="${rightLegJ4SerialNumber}" ankle_left_actuator_serial="${rightAnkleLeftActuatorSerialNumber}" ankle_right_actuator_serial="${rightAnkleRightActuatorSerialNumber}" />
+		<xacro:arm prefix="left" j1_serial_number="${leftArmJ1SerialNumber}" j2_serial_number="${leftArmJ2SerialNumber}" j3_serial_number="${leftArmJ3SerialNumber}" j4_serial_number="${leftArmJ4SerialNumber}" j5_serial_number="${leftArmJ5SerialNumber}" wrist_actuator0_serial="${leftWristTopActuatorSerialNumber}" wrist_actuator1_serial="${leftWristBottomActuatorSerialNumber}" />
+		<xacro:arm prefix="right" j1_serial_number="${rightArmJ1SerialNumber}" j2_serial_number="${rightArmJ2SerialNumber}" j3_serial_number="${rightArmJ3SerialNumber}" j4_serial_number="${rightArmJ4SerialNumber}" j5_serial_number="${rightArmJ5SerialNumber}" wrist_actuator0_serial="${rightWristTopActuatorSerialNumber}" wrist_actuator1_serial="${rightWristBottomActuatorSerialNumber}" />
 		<xacro:neck j1_serial_number="${neckJ1SerialNumber}" j2_serial_number="${neckJ1SerialNumber}" j3_serial_number="${neckJ1SerialNumber}" />
 		<xacro:waist j1_serial_number="${trunkSerialNumber}" waist_left_actuator_serial="${waistLeftActuatorSerialNumber}" waist_right_actuator_serial="${waistRightActuatorSerialNumber}"/>

File: instance/instances/robots/xacro/serial_numbers/valkyrie_A_serials.xacro (robot description, xacro)
@@ -4,12 +4,12 @@
 	<xacro:property name="leftLegJ3SerialNumber" value="v_c_002" />
 	<xacro:property name="leftLegJ4SerialNumber" value="v_d_001" />
-	<xacro:property name="leftAnkleActuator0SerialNumber" value="v_e_001" />
-	<xacro:property name="leftAnkleActuator1SerialNumber" value="v_e_002" />
+	<xacro:property name="leftAnkleLeftActuatorSerialNumber" value="v_e_001" />
+	<xacro:property name="leftAnkleRightActuatorSerialNumber" value="v_e_002" />
 	<xacro:property name="rightLegJ1SerialNumber" value="v_a_003" />
 	<xacro:property name="rightLegJ2SerialNumber" value="v_b_001" />
 	<xacro:property name="rightLegJ3SerialNumber" value="v_c_001" />
 	<xacro:property name="rightLegJ4SerialNumber" value="v_d_004" />
-	<xacro:property name="rightAnkleActuator0SerialNumber" value="v_e_003" />
-	<xacro:property name="rightAnkleActuator1SerialNumber" value="v_e_004" />
+	<xacro:property name="rightAnkleLeftActuatorSerialNumber" value="v_e_003" />
+	<xacro:property name="rightAnkleRightActuatorSerialNumber" value="v_e_004" />
 	<xacro:property name="leftArmJ1SerialNumber" value="v_a_005" />
 	<xacro:property name="leftArmJ2SerialNumber" value="v_b_004" />
@@ -17,6 +17,6 @@
 	<xacro:property name="leftArmJ4SerialNumber" value="v_f_002" />
 	<xacro:property name="leftArmJ5SerialNumber" value="v_g_005" />
-	<xacro:property name="leftWristActuator0SerialNumber" value="UNKNOWN" />
-	<xacro:property name="leftWristActuator1SerialNumber" value="UNKNOWN" />
+	<xacro:property name="leftWristTopActuatorSerialNumber" value="UNKNOWN" />
+	<xacro:property name="leftWristBottomActuatorSerialNumber" value="UNKNOWN" />
 	<xacro:property name="rightArmJ1SerialNumber" value="v_a_001" />
 	<xacro:property name="rightArmJ2SerialNumber" value="v_b_003" />
@@ -24,6 +24,6 @@
 	<xacro:property name="rightArmJ4SerialNumber" value="v_f_003" />
 	<xacro:property name="rightArmJ5SerialNumber" value="v_g_003" />
-	<xacro:property name="rightWristActuator0SerialNumber" value="UNKNOWN" />
-	<xacro:property name="rightWristActuator1SerialNumber" value="UNKNOWN" />
+	<xacro:property name="rightWristTopActuatorSerialNumber" value="UNKNOWN" />
+	<xacro:property name="rightWristBottomActuatorSerialNumber" value="UNKNOWN" />
 	<xacro:property name="neckJ1SerialNumber" value="v_g_006" />
 	<xacro:property name="neckJ2SerialNumber" value="v_g_007" />

File: instance/instances/robots/xacro/serial_numbers/valkyrie_B_serials.xacro (robot description, xacro)
@@ -4,12 +4,12 @@
 	<xacro:property name="leftLegJ3SerialNumber" value="v_c_004" />
 	<xacro:property name="leftLegJ4SerialNumber" value="v_d_003" />
-	<xacro:property name="leftAnkleActuator0SerialNumber" value="v_e_007" />
-	<xacro:property name="leftAnkleActuator1SerialNumber" value="v_e_008" />
+	<xacro:property name="leftAnkleLeftActuatorSerialNumber" value="v_e_007" />
+	<xacro:property name="leftAnkleRightActuatorSerialNumber" value="v_e_008" />
 	<xacro:property name="rightLegJ1SerialNumber" value="v_a_007" />
 	<xacro:property name="rightLegJ2SerialNumber" value="v_b_007" />
 	<xacro:property name="rightLegJ3SerialNumber" value="v_c_003" />
 	<xacro:property name="rightLegJ4SerialNumber" value="v_d_002" />
-	<xacro:property name="rightAnkleActuator0SerialNumber" value="v_e_009" />
-	<xacro:property name="rightAnkleActuator1SerialNumber" value="v_e_010" />
+	<xacro:property name="rightAnkleLeftActuatorSerialNumber" value="v_e_009" />
+	<xacro:property name="rightAnkleRightActuatorSerialNumber" value="v_e_010" />
 	<xacro:property name="leftArmJ1SerialNumber" value="v_a_002" />
 	<xacro:property name="leftArmJ2SerialNumber" value="v_b_008" />
@@ -17,6 +17,6 @@
 	<xacro:property name="leftArmJ4SerialNumber" value="v_f_010" />
 	<xacro:property name="leftArmJ5SerialNumber" value="UNKNOWN" />
-	<xacro:property name="leftWristActuator0SerialNumber" value="UNKNOWN" />
-	<xacro:property name="leftWristActuator1SerialNumber" value="UNKNOWN" />
+	<xacro:property name="leftWristTopActuatorSerialNumber" value="UNKNOWN" />
+	<xacro:property name="leftWristBottomActuatorSerialNumber" value="UNKNOWN" />
 	<xacro:property name="rightArmJ1SerialNumber" value="v_a_010" />
 	<xacro:property name="rightArmJ2SerialNumber" value="v_b_005" />
@@ -24,6 +24,6 @@
 	<xacro:property name="rightArmJ4SerialNumber" value="v_f_008" />
 	<xacro:property name="rightArmJ5SerialNumber" value="UNKNOWN" />
-	<xacro:property name="rightWristActuator0SerialNumber" value="UNKNOWN" />
-	<xacro:property name="rightWristActuator1SerialNumber" value="UNKNOWN" />
+	<xacro:property name="rightWristTopActuatorSerialNumber" value="UNKNOWN" />
+	<xacro:property name="rightWristBottomActuatorSerialNumber" value="UNKNOWN" />
 	<xacro:property name="neckJ1SerialNumber" value="UNKNOWN" />
 	<xacro:property name="neckJ2SerialNumber" value="UNKNOWN" />

File: instance/instances/robots/xacro/serial_numbers/valkyrie_C_serials.xacro (robot description, xacro)
@@ -4,12 +4,12 @@
 	<xacro:property name="leftLegJ3SerialNumber" value="UNKNOWN" />
 	<xacro:property name="leftLegJ4SerialNumber" value="UNKNOWN" />
-	<xacro:property name="leftAnkleActuator0SerialNumber" value="UNKNOWN" />
-	<xacro:property name="leftAnkleActuator1SerialNumber" value="UNKNOWN" />
+	<xacro:property name="leftAnkleLeftActuatorSerialNumber" value="UNKNOWN" />
+	<xacro:property name="leftAnkleRightActuatorSerialNumber" value="UNKNOWN" />
 	<xacro:property name="rightLegJ1SerialNumber" value="v_a_014" />
 	<xacro:property name="rightLegJ2SerialNumber" value="UNKNOWN" />
 	<xacro:property name="rightLegJ3SerialNumber" value="UNKNOWN" />
 	<xacro:property name="rightLegJ4SerialNumber" value="UNKNOWN" />
-	<xacro:property name="rightAnkleActuator0SerialNumber" value="UNKNOWN" />
-	<xacro:property name="rightAnkleActuator1SerialNumber" value="UNKNOWN" />
+	<xacro:property name="rightAnkleLeftActuatorSerialNumber" value="UNKNOWN" />
+	<xacro:property name="rightAnkleRightActuatorSerialNumber" value="UNKNOWN" />
 	<xacro:property name="leftArmJ1SerialNumber" value="v_a_013" />
 	<xacro:property name="leftArmJ2SerialNumber" value="v_b_009" />
@@ -17,6 +17,6 @@
 	<xacro:property name="leftArmJ4SerialNumber" value="v_f_011" />
 	<xacro:property name="leftArmJ5SerialNumber" value="UNKNOWN" />
-	<xacro:property name="leftWristActuator0SerialNumber" value="UNKNOWN" />
-	<xacro:property name="leftWristActuator1SerialNumber" value="UNKNOWN" />
+	<xacro:property name="leftWristTopActuatorSerialNumber" value="UNKNOWN" />
+	<xacro:property name="leftWristBottomActuatorSerialNumber" value="UNKNOWN" />
 	<xacro:property name="rightArmJ1SerialNumber" value="v_a_012" />
 	<xacro:property name="rightArmJ2SerialNumber" value="v_b_012" />
@@ -24,6 +24,6 @@
 	<xacro:property name="rightArmJ4SerialNumber" value="v_f_014" />
 	<xacro:property name="rightArmJ5SerialNumber" value="UNKNOWN" />
-	<xacro:property name="rightWristActuator0SerialNumber" value="UNKNOWN" />
-	<xacro:property name="rightWristActuator1SerialNumber" value="UNKNOWN" />
+	<xacro:property name="rightWristTopActuatorSerialNumber" value="UNKNOWN" />
+	<xacro:property name="rightWristBottomActuatorSerialNumber" value="UNKNOWN" />
 	<xacro:property name="neckJ1SerialNumber" value="UNKNOWN" />
 	<xacro:property name="neckJ2SerialNumber" value="UNKNOWN" />
