Commit message: Updated COM of foot and j5 link. Will soon update the mass and inertia of those links as well as shin.

File: model/robots/common/xacro/leg/mass_parameters.xacro (robot description, xacro)
@@ -34,5 +34,5 @@
   <xacro:property name="KneePitchLinkInertia_IZZ" value="0.013722874" />
   <xacro:property name="AnklePitchLinkMass" value="0.06" />
-  <xacro:property name="AnklePitchLinkComPosition" value="-0.001269 0.00009 -0.006013" />
+  <xacro:property name="AnklePitchLinkComPosition" value="0.0 0.0 0.0" />
   <xacro:property name="AnklePitchLinkInertia_IXX" value="0.000011226" />
   <xacro:property name="AnklePitchLinkInertia_IXY" value="0.000000000" />
@@ -42,5 +42,5 @@
   <xacro:property name="AnklePitchLinkInertia_IZZ" value="0.000018792" />
   <xacro:property name="FootMass" value="3.2550" />
-  <xacro:property name="FootComPosition" value="0.040004 -0.00381 -0.049558" />
+  <xacro:property name="FootComPosition" value="0.037702 0.005161 -0.047634" />
   <xacro:property name="FootInertia_IXX" value="0.008966273" />
   <xacro:property name="FootInertia_IXY" value="-0.000086029" />

Commit message: Updated foot/shin mass parameters.

File: model/robots/common/xacro/leg/mass_parameters.xacro (robot description, xacro)
@@ -25,27 +25,27 @@
   <xacro:property name="HipPitchLinkInertia_IYZ" value="${reflect*-0.001333005}" />
   <xacro:property name="HipPitchLinkInertia_IZZ" value="0.023276352" />
-  <xacro:property name="KneePitchLinkMass" value="6.600000" />
-  <xacro:property name="KneePitchLinkComPosition" value="0.002425 -0.001543 -0.189511" />
-  <xacro:property name="KneePitchLinkInertia_IXX" value="0.096117529" />
-  <xacro:property name="KneePitchLinkInertia_IXY" value="0.000107885" />
-  <xacro:property name="KneePitchLinkInertia_IXZ" value="0.006319047" />
-  <xacro:property name="KneePitchLinkInertia_IYY" value="0.097118447" />
-  <xacro:property name="KneePitchLinkInertia_IYZ" value="-0.000494739" />
-  <xacro:property name="KneePitchLinkInertia_IZZ" value="0.013722874" />
-  <xacro:property name="AnklePitchLinkMass" value="0.06" />
+  <xacro:property name="KneePitchLinkMass" value="6.200000" />
+  <xacro:property name="KneePitchLinkComPosition" value="-0.022183  0.001703  -0.189418" />
+  <xacro:property name="KneePitchLinkInertia_IXX" value="0.086935683" />
+  <xacro:property name="KneePitchLinkInertia_IXY" value="0.000099290" />
+  <xacro:property name="KneePitchLinkInertia_IXZ" value="0.000573207" />
+  <xacro:property name="KneePitchLinkInertia_IYY" value="0.091584066" />
+  <xacro:property name="KneePitchLinkInertia_IYZ" value="0.000313745" />
+  <xacro:property name="KneePitchLinkInertia_IZZ" value="0.014017272" />
+  <xacro:property name="AnklePitchLinkMass" value="0.030000" />
   <xacro:property name="AnklePitchLinkComPosition" value="0.0 0.0 0.0" />
-  <xacro:property name="AnklePitchLinkInertia_IXX" value="0.000011226" />
+  <xacro:property name="AnklePitchLinkInertia_IXX" value="0.000004377" />
   <xacro:property name="AnklePitchLinkInertia_IXY" value="0.000000000" />
-  <xacro:property name="AnklePitchLinkInertia_IXZ" value="0.000002735" />
-  <xacro:property name="AnklePitchLinkInertia_IYY" value="0.000026700" />
+  <xacro:property name="AnklePitchLinkInertia_IXZ" value="0.0" />
+  <xacro:property name="AnklePitchLinkInertia_IYY" value="0.000004322" />
   <xacro:property name="AnklePitchLinkInertia_IYZ" value="0.0" />
-  <xacro:property name="AnklePitchLinkInertia_IZZ" value="0.000018792" />
-  <xacro:property name="FootMass" value="3.2550" />
-  <xacro:property name="FootComPosition" value="0.037702 0.005161 -0.047634" />
-  <xacro:property name="FootInertia_IXX" value="0.008966273" />
-  <xacro:property name="FootInertia_IXY" value="-0.000086029" />
-  <xacro:property name="FootInertia_IXZ" value="0.003944774" />
-  <xacro:property name="FootInertia_IYY" value="0.023943858" />
-  <xacro:property name="FootInertia_IYZ" value="0.000105218" />
-  <xacro:property name="FootInertia_IZZ" value="0.028128777" />
+  <xacro:property name="AnklePitchLinkInertia_IZZ" value="0.000007015" />
+  <xacro:property name="FootMass" value="2.270000" />
+  <xacro:property name="FootComPosition" value="0.037702  0.005161  -0.047634" />
+  <xacro:property name="FootInertia_IXX" value="0.006239360" />
+  <xacro:property name="FootInertia_IXY" value="0.000217174" />
+  <xacro:property name="FootInertia_IXZ" value="0.001340587" />
+  <xacro:property name="FootInertia_IYY" value="0.017786991" />
+  <xacro:property name="FootInertia_IYZ" value="-0.000187749" />
+  <xacro:property name="FootInertia_IZZ" value="0.020774433" />
 </robot>
