Commit message: New leg meshes are done. They look pretty awful :(

File: model/robots/common/xacro/leg/leg.xacro (robot description, xacro)
@@ -61,7 +61,7 @@
                     iyy="${FootInertia_IYY}" iyz="${FootInertia_IYZ}" izz="${FootInertia_IZZ}"
                     origin_rpy="0 0 0"
-                    visual_mesh="${mesh_root}/legs/foot_${prefix}.dae"
+                    visual_mesh="${mesh_root}/legs/foot.dae"
                     material="White"
-                    collision_mesh="${mesh_root}/legs/foot_${prefix}.dae" />
+                    collision_mesh="${mesh_root}/legs/foot.dae" />
   </xacro:macro>
   <xacro:macro name="make_leg_joints" params="prefix reflect leg_root_link">

File: model/robots/common/xacro/thumb/thumb.xacro (robot description, xacro)
@@ -89,13 +89,3 @@
     </xacro:revolute_joint>
   </xacro:macro>
-  <xacro:macro name="right_thumb_actuators" params="prefix api">
-    <xacro:v1_actuator name="${RTA1_Actuator_Name}" api="${api}" />
-    <xacro:v1_actuator name="${RTA2_Actuator_Name}" api="${api}" />
-    <xacro:v1_actuator name="${RTA3_Actuator_Name}" api="${api}" />
-  </xacro:macro>
-  <xacro:macro name="left_thumb_actuators" params="prefix api">
-    <xacro:v1_actuator name="${LTA1_Actuator_Name}" api="${api}" />
-    <xacro:v1_actuator name="${LTA2_Actuator_Name}" api="${api}" />
-    <xacro:v1_actuator name="${LTA3_Actuator_Name}" api="${api}" />
-  </xacro:macro>
 </robot>

Commit message: Think I had IMU transforms messed up in the gazeob tag. Gazebo tag stuff is a bit confusing.

File: model/robots/common/xacro/leg/leg.xacro (robot description, xacro)
@@ -147,5 +147,5 @@
                        parentLink="${AnkleRollLinkName}"
                        origin_xyz="0.0189 0.0 -0.0783"
-                       origin_rpy="0.0 0.13 0.0"/>
+                       origin_rpy="0.0 0.0 0.0"/>
     <xacro:ati_force_torque_sensor sensorName="${prefix}FootSixAxis"
                         parentLink="${AnkleRollLinkName}"

File: model/robots/common/xacro/sensors/microstrain.xacro (robot description, xacro)
@@ -1,8 +1,4 @@
 <?xml version="1.0" ?>
 <robot xmlns:xacro="http://www.ros.org/wiki/xacro" name="microstrain">
-  <xacro:property name="MicrostrainWidth" value="0.024"/>
-  <xacro:property name="MicrostrainHeight" value="0.044"/>
-  <xacro:property name="MicrostrainDepth" value="0.011"/>
-  <xacro:property name="MicrostrainMass" value="0.0000001"/>
   <xacro:macro name="microstrain_sensor" params="sensorName parentLink origin_xyz origin_rpy">
     <xacro:massless_virtual_link name="${sensorName}_Frame"
@@ -13,8 +9,18 @@
                        origin_rpy="${origin_rpy}"
                        origin_xyz="${origin_xyz}"/>
+    <gazebo>
+      <plugin filename="libgazebo_ros_imu.so" name="imu_plugin_ros">
+        <alwaysOn>true</alwaysOn>
+        <bodyName>${sensorName}_Frame</bodyName>
+        <topicName>${sensorName}/imu</topicName>
+        <serviceName>${sensorName}/imu_service</serviceName>
+        <gaussianNoise>0.0</gaussianNoise>
+        <updateRate>1000.0</updateRate>
+      </plugin>
+    </gazebo>
     <gazebo reference="${sensorName}_Frame">
       <sensor name="${sensorName}" type="imu">
         <always_on>true</always_on>
-        <pose>${origin_xyz} ${origin_rpy} </pose>
+        <pose>0 0 0 0 0 0 </pose>
         <imu>
            <noise>

Commit message: Added shared memory nodes for F/T sensors in the feet.

File: model/robots/common/xacro/leg/leg.xacro (robot description, xacro)
@@ -137,5 +137,5 @@
     <xacro:make_ankle_joints prefix="${prefix}" reflect="${reflect}" leg_root_link="${leg_root_link}" />
   </xacro:macro>
-  <xacro:macro name="v1_leg_sensors" params="prefix reflect ATI_serial_number">
+  <xacro:macro name="v1_leg_sensors" params="prefix reflect ATI_serial_number ATI_node">
     <xacro:virtual_fixed_frame_offset name="${prefix}COP"
                        parentLink="${AnkleRollLinkName}"
@@ -146,5 +146,6 @@
                         origin_xyz="0.0215646 0.0 -0.051054"
                         origin_rpy="3.14 0.0 -1.047"
-                        sensor_number="${ATI_serial_number}"/>
+                        sensor_number="${ATI_serial_number}"
+                        sensor_node="${ATI_node}"/>
   </xacro:macro>
   <xacro:macro name="leg_transmissions_hw" params="prefix">

File: model/robots/common/xacro/sensors/ati_force_torque.xacro (robot description, xacro)
@@ -1,5 +1,5 @@
 <?xml version="1.0" ?>
 <robot xmlns:xacro="http://www.ros.org/wiki/xacro" name="ati_force_torque_sensor">
-  <xacro:macro name="ati_force_torque_sensor" params="sensorName parentLink origin_xyz origin_rpy sensor_number">
+  <xacro:macro name="ati_force_torque_sensor" params="sensorName parentLink origin_xyz origin_rpy sensor_number sensor_node">
 	<xacro:massless_virtual_link name="${sensorName}_Frame"
                     origin_rpy="0 0 0"
@@ -13,4 +13,5 @@
         <frame>child</frame>
         <sensor_number id="${sensor_number}" />
+        <!-- <sensor_node ide="${sensor_node}" /> -->
     	</sensor>
     </gazebo>

File: model/robots/common/xacro/valkyrie_base_hw.xacro (robot description, xacro)
@@ -16,6 +16,6 @@
     <xacro:make_leg prefix="left" reflect="1" leg_root_link="${Pelvis_Link_Name}"/>
     <xacro:v1_trunk_sensors/>
-    <xacro:v1_leg_sensors prefix="left" reflect="1" ATI_serial_number="${left_foot_ATI_serial}"/>
-    <xacro:v1_leg_sensors prefix="right" reflect="-1" ATI_serial_number="${right_foot_ATI_serial}"/>
+    <xacro:v1_leg_sensors prefix="left" reflect="1" ATI_serial_number="${left_foot_ATI_serial}" ATI_node="${left_foot_ATI_node}"/>
+    <xacro:v1_leg_sensors prefix="right" reflect="-1" ATI_serial_number="${right_foot_ATI_serial}" ATI_node="${right_foot_ATI_node}"/>
     <xacro:include_multisense_hw />
     <xacro:v1_pelvis_sensors/>

File: model/robots/common/xacro/valkyrie_base_sim.xacro (robot description, xacro)
@@ -16,6 +16,6 @@
     <xacro:make_leg prefix="left" reflect="1" leg_root_link="${Pelvis_Link_Name}"/>
     <xacro:v1_pelvis_sensors />
-    <xacro:v1_leg_sensors prefix="left" reflect="1" ATI_serial_number="${left_foot_ATI_serial}"/>
-    <xacro:v1_leg_sensors prefix="right" reflect="-1" ATI_serial_number="${right_foot_ATI_serial}"/>
+    <xacro:v1_leg_sensors prefix="left" reflect="1" ATI_serial_number="${left_foot_ATI_serial}" ATI_node="${left_foot_ATI_node}"/>
+    <xacro:v1_leg_sensors prefix="right" reflect="-1" ATI_serial_number="${right_foot_ATI_serial}" ATI_node="${right_foot_ATI_node}"/>
     <xacro:include_multisense_sim />
     <xacro:v1_trunk_sensors/>

Commit message: Fixed force_torque sensor tags. Since gazebo force_torque sensors can't attach to fixed joints I removed the extra joint/link we were using to express the frame of the sensor and added the pose tag to the sensor block.

File: model/robots/common/xacro/leg/leg.xacro (robot description, xacro)
@@ -144,4 +144,5 @@
     <xacro:ati_force_torque_sensor sensorName="${prefix}FootSixAxis"
                         parentLink="${AnkleRollLinkName}"
+                        joint_to_attach_sensor_to="${AnkleRollJointName}"
                         origin_xyz="0.0215646 0.0 -0.051054"
                         origin_rpy="3.14 0.0 -1.047"

File: model/robots/common/xacro/sensors/ati_force_torque.xacro (robot description, xacro)
@@ -1,17 +1,15 @@
 <?xml version="1.0" ?>
 <robot xmlns:xacro="http://www.ros.org/wiki/xacro" name="ati_force_torque_sensor">
-  <xacro:macro name="ati_force_torque_sensor" params="sensorName parentLink origin_xyz origin_rpy sensor_number sensor_node">
-	<xacro:massless_virtual_link name="${sensorName}_Frame"
-                    origin_rpy="0 0 0"
-                    origin_xyz="0 0 0"/>
-    <xacro:fixed_joint jointName="${sensorName}_Offset"
-                       parent="${parentLink}" child="${sensorName}_Frame"
-                       origin_rpy="${origin_rpy}"
-                       origin_xyz="${origin_xyz}"/>
-    <gazebo reference="${sensorName}_Offset">
+  <xacro:macro name="ati_force_torque_sensor" params="sensorName parentLink joint_to_attach_sensor_to origin_xyz origin_rpy sensor_number sensor_node">
+    <gazebo reference="${joint_to_attach_sensor_to}">
       <sensor name="${sensorName}" type="force_torque">
-        <frame>child</frame>
+        <pose>${origin_xyz} ${origin_rpy}</pose>
         <sensor_number id="${sensor_number}" />
-        <!-- <sensor_node ide="${sensor_node}" /> -->
+        <node ide="${sensor_node}" />
+        <always_on>true</always_on>
+        <update_rate>1000</update_rate>
+        <force_torque>
+          <frame>sensor</frame>
+        </force_torque>
     	</sensor>
     </gazebo>

Commit message: removed duplicate macro

File: model/robots/common/xacro/leg/leg.xacro (robot description, xacro)
@@ -151,18 +151,4 @@
                         sensor_api="${AtiSensorApi}" />
   </xacro:macro>
-    <xacro:macro name="v1_leg_sensors" params="prefix reflect ATI_serial_number ATI_node">
-    <xacro:virtual_fixed_frame_offset name="${prefix}COP"
-                       parentLink="${AnkleRollLinkName}"
-                       origin_xyz="0.0189 0.0 -0.0783"
-                       origin_rpy="0.0 0.0 0.0"/>
-    <xacro:ati_force_torque_sensor sensorName="${prefix}FootSixAxis"
-                        parentLink="${AnkleRollLinkName}"
-                        joint_to_attach_sensor_to="${AnkleRollJointName}"
-                        origin_xyz="0.0215646 0.0 -0.051054"
-                        origin_rpy="3.14 0.0 -1.047"
-                        sensor_number="${ATI_serial_number}"
-                        sensor_node="${ATI_node}"
-                        sensor_api="${AtiSensorApi}" />
-  </xacro:macro>
   <xacro:macro name="leg_transmissions_hw" params="prefix">
     <xacro:simple_transmission jointName="${HipYawJointName}" actuatorName="${HipYawActuatorName}" nodeName="${HipYawNode}" actuatorApi="${HipYawApi}"/>
