Commit message: Jordan & Frank: Fixed transmissions to work with Franks' transmission loader stuff. Had to do some name changes.

File: common/xacro/actuator_names/valkyrie_actuator_names.xacro (robot description, xacro)
@@ -8,6 +8,6 @@
 	<xacro:property name="HipPitchActuatorName" value="${prefix}HipPitch"/>
 	<xacro:property name="KneePitchActuatorName" value="${prefix}KneePitch"/>
-	<xacro:property name="AnkleOutsideActuatorName" value="${prefix}AnkleOutsideActuator"/>
-	<xacro:property name="AnkleInsideActuatorName" value="${prefix}AnkleInsideActuator"/>
+	<xacro:property name="AnkleRightActuatorName" value="${prefix}AnkleRightActuator"/>
+	<xacro:property name="AnkleLeftActuatorName" value="${prefix}AnkleLeftActuator"/>
 	<xacro:property name="LowerNeckPitchActuatorName" value="lowerNeckPitch"/>
 	<xacro:property name="NeckYawActuatorName" value="neckYaw"/>

File: common/xacro/api/valkyrie_api.xacro (robot description, xacro)
@@ -4,6 +4,6 @@
 	<xacro:property name="HipPitchApi" value="robot_hardware_interface/TurbodriverAPI_DRCv4" />
 	<xacro:property name="KneePitchApi" value="robot_hardware_interface/TurbodriverAPI_DRCv4" />
-	<xacro:property name="AnkleInsideActuatorApi" value="robot_hardware_interface/TurbodriverAPI_DRCv4_linear" />
-	<xacro:property name="AnkleOutsideActuatorApi" value="robot_hardware_interface/TurbodriverAPI_DRCv4_linear" />
+	<xacro:property name="AnkleRightActuatorApi" value="robot_hardware_interface/TurbodriverAPI_DRCv4_linear" />
+	<xacro:property name="AnkleLeftActuatorApi" value="robot_hardware_interface/TurbodriverAPI_DRCv4_linear" />
 	<xacro:property name="ShoulderPitchApi" value="robot_hardware_interface/TurbodriverAPI_DRCv4" />
 	<xacro:property name="ShoulderRollApi" value="robot_hardware_interface/TurbodriverAPI_DRCv4" />

File: common/xacro/nodes/valkyrie_nodes.xacro (robot description, xacro)
@@ -4,6 +4,6 @@
 	<xacro:property name="HipPitchNode" value="/${prefix}_leg/j3" />
 	<xacro:property name="KneePitchNode" value="/${prefix}_leg/j4" />
-	<xacro:property name="AnkleInsideActuatorNode" value="/${prefix}_leg/left_actuator" />
-	<xacro:property name="AnkleOutsideActuatorNode" value="/${prefix}_leg/right_actuator" />
+	<xacro:property name="AnkleLeftActuatorNode" value="/${prefix}_leg/left_actuator" />
+	<xacro:property name="AnkleRightActuatorNode" value="/${prefix}_leg/right_actuator" />
 	<xacro:property name="ShoulderPitchNode" value="/trunk/${prefix}_arm_j1" />
 	<xacro:property name="ShoulderRollNode" value="/${prefix}_arm/j2" />

File: instance/instances/robots/xacro/limbs/leg.xacro (robot description, xacro)
@@ -7,5 +7,5 @@
     	<xacro:simple_mechanism name="${HipPitchJointName}" serial_number="${j3_serial_number}" node="${HipPitchNode}"/>
     	<xacro:simple_mechanism name="${KneePitchJointName}" serial_number="${j4_serial_number}" node="${KneePitchNode}"/>
-    	<xacro:two_active_joint_mechanism mechanism_name="${prefix}Ankle" actuator0_name="${prefix}AnkleLeftActuator" actuator1_name="${prefix}AnkleRightActuator" joint0_name="${AnklePitchJointName}" joint1_name="${AnkleRollJointName}" actuator0_serial="${ankle_left_actuator_serial}" actuator1_serial="${ankle_right_actuator_serial}" actuator0_node="${AnkleInsideActuatorNode}" actuator1_node="${AnkleOutsideActuatorNode}" />
+    	<xacro:two_active_joint_mechanism mechanism_name="${prefix}Ankle" actuator0_name="${prefix}AnkleLeftActuator" actuator1_name="${prefix}AnkleRightActuator" joint0_name="${AnklePitchJointName}" joint1_name="${AnkleRollJointName}" actuator0_serial="${ankle_left_actuator_serial}" actuator1_serial="${ankle_right_actuator_serial}" actuator0_node="${AnkleLeftActuatorNode}" actuator1_node="${AnkleRightActuatorNode}" />
     </xacro:macro>
 </robot>

File: model/robots/common/xacro/arm/arm.xacro (robot description, xacro)
@@ -162,5 +162,5 @@
     <xacro:simple_transmission jointName="${ElbowPitchJointName}" actuatorName="${ElbowPitchActuatorName}" nodeName="${ElbowPitchNode}" actuatorApi="${ElbowPitchApi}"/>
     <xacro:simple_transmission jointName="${ForearmYawActuatorName}" actuatorName="${ForearmYawActuatorName}" nodeName="${ForearmYawNode}" actuatorApi="${ForearmYawApi}"/>
-    <xacro:pushrod_transmission transmissionName="${prefix}WristTransmission" joint1Name="${WristPitchJointName}" joint2Name="${WristRollJointName}" actuator1Name="${WristTopActuatorName}" actuator2Name="${WristBottomActuatorName}" actuator1Node="${WristTopActuatorNode}" actuator2Node="${WristBottomActuatorNode}" joint1Role="roll" joint2Role="pitch" actuator1Role="actuator1" actuator2Role="actuator2" actuator1Api="WristTopActuatorApi" actuator2Api="${WristBottomActuatorApi}"/>
+    <xacro:pushrod_transmission transmissionName="${prefix}WristTransmission" transmissionType="WristPushrodTransmission" joint1Name="${WristPitchJointName}" joint2Name="${WristRollJointName}" actuator1Name="${WristTopActuatorName}" actuator2Name="${WristBottomActuatorName}" actuator1Node="${WristTopActuatorNode}" actuator2Node="${WristBottomActuatorNode}" actuator1Api="WristTopActuatorApi" actuator2Api="${WristBottomActuatorApi}"/>
   </xacro:macro>
   <xacro:macro name="arm_transmissions_sim" params="prefix">

File: model/robots/common/xacro/generic_models.xacro (robot description, xacro)
@@ -215,18 +215,18 @@
     </transmission>
   </xacro:macro>
-  <xacro:macro name="pushrod_transmission" params="transmissionName joint1Name joint2Name actuator1Name actuator2Name actuator1Node actuator2Node joint1Role joint2Role actuator1Role actuator2Role actuator1Api actuator2Api">
+  <xacro:macro name="pushrod_transmission" params="transmissionName transmissionType joint1Name joint2Name actuator1Name actuator2Name actuator1Node actuator2Node actuator1Api actuator2Api">
     <transmission name="${transmissionName}">
-      <type>transmission_interface/PushrodTransmission</type>
+      <type>robot_transmission_interface/${transmissionType}</type>
       <joint name="${joint1Name}">
-        <role>${joint1Role}</role>
+        <role>joint1</role>
         <hardwareInterface>EffortJointInterface</hardwareInterface>
       </joint>
       <joint name="${joint2Name}">
-        <role>${joint2Role}</role>
+        <role>joint2</role>
         <hardwareInterface>EffortJointInterface</hardwareInterface>
       </joint>
        <actuator name="${actuator1Name}">
         <node name="${actuator1Node}"/>
-        <role>${actuator1Role}</role>
+        <role>actuator1</role>
         <mechanicalReduction>1</mechanicalReduction>
         <api name="${actuator1Api}"/>
@@ -234,5 +234,5 @@
       <actuator name="${actuator2Name}">
         <node name="${actuator2Node}"/>
-        <role>${actuator2Role}</role>
+        <role>actuator2</role>
         <mechanicalReduction>1</mechanicalReduction>
         <api name="${actuator2Api}"/>

File: model/robots/common/xacro/leg/leg.xacro (robot description, xacro)
@@ -153,5 +153,5 @@
     <xacro:simple_transmission jointName="${HipPitchJointName}" actuatorName="${HipPitchActuatorName}" nodeName="${HipPitchNode}" actuatorApi="${HipPitchApi}"/>
     <xacro:simple_transmission jointName="${KneePitchJointName}" actuatorName="${KneePitchActuatorName}" nodeName="${KneePitchNode}" actuatorApi="${KneePitchApi}"/>
-    <xacro:pushrod_transmission transmissionName="${prefix}AnkleTransmission" joint1Name="${AnklePitchJointName}" joint2Name="${AnkleRollJointName}" actuator1Name="${AnkleInsideActuatorName}" actuator2Name="${AnkleOutsideActuatorName}" actuator1Node="${AnkleInsideActuatorNode}" actuator2Node="${AnkleOutsideActuatorNode}" joint1Role="pitch" joint2Role="roll" actuator1Role="insideActuator" actuator2Role="outsideActuator" actuator1Api="${AnkleInsideActuatorApi}" actuator2Api="${AnkleOutsideActuatorApi}"/>
+    <xacro:pushrod_transmission transmissionName="${prefix}AnkleTransmission" transmissionType="AnklePushrodTransmission" joint1Name="${AnklePitchJointName}" joint2Name="${AnkleRollJointName}" actuator1Name="${AnkleLeftActuatorName}" actuator2Name="${AnkleRightActuatorName}" actuator1Node="${AnkleLeftActuatorNode}" actuator2Node="${AnkleRightActuatorNode}" actuator1Api="${AnkleLeftActuatorApi}" actuator2Api="${AnkleRightActuatorApi}"/>
   </xacro:macro>
   <xacro:macro name="leg_transmissions_sim" params="prefix">
@@ -160,6 +160,6 @@
     <xacro:simple_transmission jointName="${HipPitchJointName}" actuatorName="${HipPitchActuatorName}" nodeName="${HipPitchNode}" actuatorApi="${SimApi}"/>
     <xacro:simple_transmission jointName="${KneePitchJointName}" actuatorName="${KneePitchActuatorName}" nodeName="${KneePitchNode}" actuatorApi="${SimApi}"/>
-    <xacro:simple_transmission jointName="${AnklePitchJointName}" actuatorName="${AnkleInsideActuatorName}" nodeName="${AnkleInsideActuatorNode}" actuatorApi="${SimApi}"/>
-    <xacro:simple_transmission jointName="${AnkleRollJointName}" actuatorName="${AnkleOutsideActuatorName}" nodeName="${AnkleOutsideActuatorNode}" actuatorApi="${SimApi}"/>
+    <xacro:simple_transmission jointName="${AnklePitchJointName}" actuatorName="${AnkleLeftActuatorName}" nodeName="${AnkleLeftActuatorNode}" actuatorApi="${SimApi}"/>
+    <xacro:simple_transmission jointName="${AnkleRollJointName}" actuatorName="${AnkleRightActuatorName}" nodeName="${AnkleRightActuatorNode}" actuatorApi="${SimApi}"/>
   </xacro:macro>
 </robot>

File: model/robots/common/xacro/waist/waist.xacro (robot description, xacro)
@@ -97,5 +97,5 @@
    <xacro:macro name="waist_transmissions_hw">
     <xacro:simple_transmission jointName="${TorsoYawJointName}" actuatorName="${TorsoYawActuatorName}" nodeName="${TrunkYawNode}" actuatorApi="${TrunkYawApi}"/>
-    <xacro:pushrod_transmission transmissionName="WaistTransmission" joint1Name="${TorsoPitchJointName}" joint2Name="${TorsoRollJointName}" actuator1Name="${WaistLeftActuatorName}" actuator2Name="${WaistRightActuatorName}" actuator1Node="${WaistLeftActuatorNode}" actuator2Node="${WaistRightActuatorNode}" joint1Role="pitch" joint2Role="roll" actuator1Role="leftActuator" actuator2Role="rightActuator" actuator1Api="${WaistLeftActuatorApi}" actuator2Api="${WaistRightActuatorApi}"/>
+    <xacro:pushrod_transmission transmissionName="WaistTransmission" transmissionType="TorsoPushrodTransmission" joint1Name="${TorsoPitchJointName}" joint2Name="${TorsoRollJointName}" actuator1Name="${WaistLeftActuatorName}" actuator2Name="${WaistRightActuatorName}" actuator1Node="${WaistLeftActuatorNode}" actuator2Node="${WaistRightActuatorNode}" actuator1Api="${WaistLeftActuatorApi}" actuator2Api="${WaistRightActuatorApi}"/>
    </xacro:macro>
    <xacro:macro name="waist_transmissions_sim">

Commit message: updated nodes and names to match requirements in simulation

File: common/xacro/actuator_names/valkyrie_actuator_names.xacro (robot description, xacro)
@@ -4,4 +4,6 @@
 	<xacro:property name="WaistLeftActuatorName" value="waistLeftActuator"/>
 	<xacro:property name="WaistRightActuatorName" value="waistRightActuator"/>
+	<xacro:property name="WaistPitchActuatorSimName" value="waistPitchActuator"/>
+	<xacro:property name="WaistRollActuatorSimName" value="waistRollActuator"/>
 	<xacro:property name="HipYawActuatorName" value="${prefix}HipYaw"/>
 	<xacro:property name="HipRollActuatorName" value="${prefix}HipRoll"/>
@@ -10,4 +12,6 @@
 	<xacro:property name="AnkleRightActuatorName" value="${prefix}AnkleRightActuator"/>
 	<xacro:property name="AnkleLeftActuatorName" value="${prefix}AnkleLeftActuator"/>
+	<xacro:property name="AnkleRollActuatorSimName" value="${prefix}AnkleRollActuator"/>
+	<xacro:property name="AnklePitchActuatorSimName" value="${prefix}AnklePitchActuator"/>
 	<xacro:property name="LowerNeckPitchActuatorName" value="lowerNeckPitch"/>
 	<xacro:property name="NeckYawActuatorName" value="neckYaw"/>
@@ -20,4 +24,6 @@
 	<xacro:property name="WristBottomActuatorName" value="${prefix}WristBottomActuator"/>
 	<xacro:property name="WristTopActuatorName" value="${prefix}WristTopActuator"/>
+	<xacro:property name="WristPitchActuatorSimName" value="${prefix}WristPitchActuator"/>
+	<xacro:property name="WristRollActuatorSimName" value="${prefix}WristRollActuator"/>
 	<xacro:property name="IndexFingerPitch1ActuatorName" value="${prefix}IndexFingerPitch1"/>
 	<xacro:property name="IndexFingerPitch2ActuatorName" value="${prefix}IndexFingerPitch2"/>

File: common/xacro/api/valkyrie_api.xacro (robot description, xacro)
@@ -20,4 +20,4 @@
 	<xacro:property name="WaistRightActuatorApi" value="robot_hardware_interface/TurbodriverAPI_DRCv4_linear" />
 	<xacro:property name="AtiSensorApi" value="TurbodriverForceTorqueSensor_v1" />
-	<xacro:property name="SimApi" value="robot_hardware_interface/TurboDriverSimApiDRC_v4" />
+	<xacro:property name="SimApi" value="robot_hardware_interface/TurbodriverSimAPI_DRCv4" />
 </robot>

File: common/xacro/nodes/valkyrie_nodes.xacro (robot description, xacro)
@@ -6,4 +6,6 @@
 	<xacro:property name="AnkleLeftActuatorNode" value="/${prefix}_leg/ankle/left_actuator" />
 	<xacro:property name="AnkleRightActuatorNode" value="/${prefix}_leg/ankle/right_actuator" />
+	<xacro:property name="AnklePitchActuatorSimNode" value="/${prefix}_leg/ankle/pitch_actuator" />
+	<xacro:property name="AnkleRollActuatorSimNode" value="/${prefix}_leg/ankle/roll_actuator" />
 	<xacro:property name="ShoulderPitchNode" value="/trunk/${prefix}_arm_j1" />
 	<xacro:property name="ShoulderRollNode" value="/${prefix}_arm/j2" />
@@ -13,10 +15,14 @@
 	<xacro:property name="WristTopActuatorNode" value="/${prefix}_arm/wrist/top_actautor" />
 	<xacro:property name="WristBottomActuatorNode" value="/${prefix}_arm/wrist/bottom_actuator" />
+	<xacro:property name="WristRollActuatorSimNode" value="/${prefix}_arm/wrist/roll_actautor" />
+	<xacro:property name="WristPitchActuatorSimNode" value="/${prefix}_arm/wrist/pitch_actuator" />
 	<xacro:property name="LowerNeckPitchNode" value="/neck/j1" />
 	<xacro:property name="NeckYawNode" value="/neck/j2" />
 	<xacro:property name="UpperNeckPitchNode" value="/neck/j3" />
-	<xacro:property name="TrunkYawNode" value="/pelvis/waist" />
-	<xacro:property name="WaistLeftActuatorNode" value="/trunk/left_actuator" />
-	<xacro:property name="WaistRightActuatorNode" value="/trunk/right_actuator" />
+	<xacro:property name="TrunkYawNode" value="/pelvis/waist" /> <!--Yaw-->
+	<xacro:property name="WaistLeftActuatorNode" value="/trunk/left_actuator" /> <!--pitch-->
+	<xacro:property name="WaistRightActuatorNode" value="/trunk/right_actuator" /> <!--roll-->
+	<xacro:property name="WaistPitchActuatorSimNode" value="/trunk/pitch_actuator" /> <!--pitch-->
+	<xacro:property name="WaistRollActuatorSimNode" value="/trunk/roll_actuator" /> <!--roll-->
 	<xacro:property name="pelvis_imu1_node" value="/pelvis/sensors/imu1" />
 	<xacro:property name="pelvis_imu2_node" value="/pelvis/sensors/imu2" />
@@ -24,5 +30,7 @@
 	<xacro:property name="torso_imu2_node" value="/torso/sensors/imu2" />
 	<xacro:property name="left_foot_ATI_node" value="/left_leg/ankle/left_actuator" />
+	<xacro:property name="left_foot_Sim_ATI_node" value="/left_leg/ankle/pitch_actuator" />
 	<xacro:property name="right_foot_ATI_node" value="/right_leg/ankle/left_actuator" />
+	<xacro:property name="right_foot_Sim_ATI_node" value="/right_leg/ankle/pitch_actuator" />
 	<xacro:macro name="all_channels" >
 		<Channels>

File: model/robots/common/xacro/arm/arm.xacro (robot description, xacro)
@@ -179,6 +179,6 @@
     <xacro:simple_transmission jointName="${ElbowPitchJointName}" actuatorName="${ElbowPitchActuatorName}" nodeName="${ElbowPitchNode}" actuatorApi="${SimApi}"/>
     <xacro:simple_transmission jointName="${ForearmYawActuatorName}" actuatorName="${ForearmYawActuatorName}" nodeName="${ForearmYawNode}" actuatorApi="${SimApi}"/>
-    <xacro:simple_transmission jointName="${WristRollJointName}" actuatorName="${WristTopActuatorName}" nodeName="${WristTopActuatorNode}" actuatorApi="${SimApi}"/>
-    <xacro:simple_transmission jointName="${WristPitchJointName}" actuatorName="${WristBottomActuatorName}" nodeName="${WristBottomActuatorNode}" actuatorApi="${SimApi}"/>
+    <xacro:simple_transmission jointName="${WristRollJointName}" actuatorName="${WristRollActuatorSimName}" nodeName="${WristRollActuatorSimNode}" actuatorApi="${SimApi}"/>
+    <xacro:simple_transmission jointName="${WristPitchJointName}" actuatorName="${WristPitchActuatorSimName}" nodeName="${WristPitchActuatorSimNode}" actuatorApi="${SimApi}"/>
   </xacro:macro>
 </robot>

File: model/robots/common/xacro/leg/leg.xacro (robot description, xacro)
@@ -151,4 +151,18 @@
                         sensor_api="${AtiSensorApi}" />
   </xacro:macro>
+    <xacro:macro name="v1_leg_sensors" params="prefix reflect ATI_serial_number ATI_node">
+    <xacro:virtual_fixed_frame_offset name="${prefix}COP"
+                       parentLink="${AnkleRollLinkName}"
+                       origin_xyz="0.0189 0.0 -0.0783"
+                       origin_rpy="0.0 0.0 0.0"/>
+    <xacro:ati_force_torque_sensor sensorName="${prefix}FootSixAxis"
+                        parentLink="${AnkleRollLinkName}"
+                        joint_to_attach_sensor_to="${AnkleRollJointName}"
+                        origin_xyz="0.0215646 0.0 -0.051054"
+                        origin_rpy="3.14 0.0 -1.047"
+                        sensor_number="${ATI_serial_number}"
+                        sensor_node="${ATI_node}"
+                        sensor_api="${AtiSensorApi}" />
+  </xacro:macro>
   <xacro:macro name="leg_transmissions_hw" params="prefix">
     <xacro:simple_transmission jointName="${HipYawJointName}" actuatorName="${HipYawActuatorName}" nodeName="${HipYawNode}" actuatorApi="${HipYawApi}"/>
@@ -163,6 +177,6 @@
     <xacro:simple_transmission jointName="${HipPitchJointName}" actuatorName="${HipPitchActuatorName}" nodeName="${HipPitchNode}" actuatorApi="${SimApi}"/>
     <xacro:simple_transmission jointName="${KneePitchJointName}" actuatorName="${KneePitchActuatorName}" nodeName="${KneePitchNode}" actuatorApi="${SimApi}"/>
-    <xacro:simple_transmission jointName="${AnklePitchJointName}" actuatorName="${AnkleLeftActuatorName}" nodeName="${AnkleLeftActuatorNode}" actuatorApi="${SimApi}"/>
-    <xacro:simple_transmission jointName="${AnkleRollJointName}" actuatorName="${AnkleRightActuatorName}" nodeName="${AnkleRightActuatorNode}" actuatorApi="${SimApi}"/>
+    <xacro:simple_transmission jointName="${AnklePitchJointName}" actuatorName="${AnklePitchActuatorSimName}" nodeName="${AnklePitchActuatorSimNode}" actuatorApi="${SimApi}"/>
+    <xacro:simple_transmission jointName="${AnkleRollJointName}" actuatorName="${AnkleRollActuatorSimName}" nodeName="${AnkleRollActuatorSimNode}" actuatorApi="${SimApi}"/>
   </xacro:macro>
 </robot>

File: model/robots/common/xacro/valkyrie_base_sim.xacro (robot description, xacro)
@@ -2,5 +2,5 @@
     <gazebo>
       <plugin filename="libval_gazebo.so" name="SharedMemorySimInterfacePlugin">
-        <robotNamespace>/rrbot</robotNamespace>
+      <robotNamespace>/val</robotNamespace>
       </plugin>
     </gazebo>
@@ -21,6 +21,6 @@
     <xacro:make_leg prefix="left" reflect="1" leg_root_link="${Pelvis_Link_Name}"/>
     <xacro:v1_pelvis_sensors />
-    <xacro:v1_leg_sensors prefix="left" reflect="1" ATI_serial_number="${sim_ATI_serial}" ATI_node="${left_foot_ATI_node}"/>
-    <xacro:v1_leg_sensors prefix="right" reflect="-1" ATI_serial_number="${sim_ATI_serial}" ATI_node="${right_foot_ATI_node}"/>
+    <xacro:v1_leg_sensors prefix="left" reflect="1" ATI_serial_number="${sim_ATI_serial}" ATI_node="${left_foot_Sim_ATI_node}"/>
+    <xacro:v1_leg_sensors prefix="right" reflect="-1" ATI_serial_number="${sim_ATI_serial}" ATI_node="${right_foot_Sim_ATI_node}"/>
     <xacro:include_multisense_sim />
     <xacro:v1_trunk_sensors/>

File: model/robots/common/xacro/waist/waist.xacro (robot description, xacro)
@@ -97,6 +97,6 @@
    <xacro:macro name="waist_transmissions_sim">
     <xacro:simple_transmission jointName="${TorsoYawJointName}" actuatorName="${TorsoYawActuatorName}" nodeName="${TrunkYawNode}" actuatorApi="${SimApi}"/>
-    <xacro:simple_transmission jointName="${TorsoPitchJointName}" actuatorName="${WaistLeftActuatorName}" nodeName="${WaistLeftActuatorNode}" actuatorApi="${SimApi}"/>
-    <xacro:simple_transmission jointName="${TorsoRollJointName}" actuatorName="${WaistRightActuatorName}" nodeName="${WaistRightActuatorNode}" actuatorApi="${SimApi}"/>
+    <xacro:simple_transmission jointName="${TorsoPitchJointName}" actuatorName="${WaistPitchActuatorSimName}" nodeName="${WaistPitchActuatorSimNode}" actuatorApi="${SimApi}"/>
+    <xacro:simple_transmission jointName="${TorsoRollJointName}" actuatorName="${WaistRollActuatorSimName}" nodeName="${WaistRollActuatorSimNode}" actuatorApi="${SimApi}"/>
    </xacro:macro>
 </robot>
