Commit message: corrected nameing in macro for urdf

File: model/robots/common/xacro/sensors/microstrain.xacro (robot description, xacro)
@@ -43,5 +43,5 @@
     </gazebo>
   </xacro:macro>
-  <xacro:macro name="plugged_in_microstrain_sensor" params="sensorName parentLink origin_xyz origin_rpy sensor_node sensor_api sensor_port">
+  <xacro:macro name="usb_microstrain_sensor" params="sensorName parentLink origin_xyz origin_rpy sensor_node sensor_api sensor_port">
     <xacro:massless_virtual_link name="${sensorName}_Frame"
                     origin_rpy="0 0 0"
