Commit message: Added ports for imus. changed filter frequency on linear actuator velocity filter.

File: common/xacro/dev_ports/valkyrie_A_ports.xacro (robot description, xacro)
@@ -1,3 +1,4 @@
 <robot xmlns:xacro="http://ros.org/wiki/xacro" name="valkyrie_A_ports">
 	<xacro:property name="pelvis_middle_imu_port" value="/dev/ttyACM0" />
+	<xacro:property name="pelvis_rear_imu_port" value="/dev/ttyACM0" />
 </robot>

File: common/xacro/dev_ports/valkyrie_B_ports.xacro (robot description, xacro)
@@ -1,3 +1,4 @@
 <robot xmlns:xacro="http://ros.org/wiki/xacro" name="valkyrie_B_ports">
 	<xacro:property name="pelvis_middle_imu_port" value="/dev/serial/by-id/usb-Lord_Microstrain_Lord_Inertial_Sensor_0000__6233.47092-if00" />
+	<xacro:property name="pelvis_rear_imu_port" value="/dev/serial/by-id/usb-Lord_Microstrain_Lord_Inertial_Sensor_0000__6233.47094-if00" />
 </robot>

File: common/xacro/dev_ports/valkyrie_C_ports.xacro (robot description, xacro)
@@ -1,3 +1,4 @@
 <robot xmlns:xacro="http://ros.org/wiki/xacro" name="valkyrie_C_ports">
 	<xacro:property name="pelvis_middle_imu_port" value="/dev/serial/by-id/usb-Lord_Microstrain_Lord_Inertial_Sensor_0000__6233.47093-if00" />
+	<xacro:property name="pelvis_rear_imu_port" value="/dev/serial/by-id/usb-Lord_Microstrain_Lord_Inertial_Sensor_0000__6233.47095-if00" />
 </robot>

Commit message: updated imu data for unit B and unit C

File: common/xacro/dev_ports/valkyrie_A_ports.xacro (robot description, xacro)
@@ -1,3 +1,5 @@
 <robot xmlns:xacro="http://ros.org/wiki/xacro" name="valkyrie_A_ports">
 	<xacro:property name="pelvis_middle_imu_port" value="/dev/ttyACM0" />
+	<xacro:property name="pelvis_rear_imu_port" value="/dev/ttyACM0" />
+	<xacro:property name="torso_left_imu_port" value="/dev/ttyACM0" />
 </robot>

File: common/xacro/dev_ports/valkyrie_B_ports.xacro (robot description, xacro)
@@ -1,3 +1,5 @@
 <robot xmlns:xacro="http://ros.org/wiki/xacro" name="valkyrie_B_ports">
 	<xacro:property name="pelvis_middle_imu_port" value="/dev/serial/by-id/usb-Lord_Microstrain_Lord_Inertial_Sensor_0000__6233.47092-if00" />
+	<xacro:property name="pelvis_rear_imu_port" value="/dev/serial/by-id/usb-Lord_Microstrain_Lord_Inertial_Sensor_0000__6233.47094-if00" />
+	<xacro:property name="torso_left_imu_port" value="/dev/serial/by-id/usb-Lord_Microstrain_Lord_Inertial_Sensor_0000__6233.47100-if00" />
 </robot>

File: common/xacro/dev_ports/valkyrie_C_ports.xacro (robot description, xacro)
@@ -1,3 +1,5 @@
 <robot xmlns:xacro="http://ros.org/wiki/xacro" name="valkyrie_C_ports">
 	<xacro:property name="pelvis_middle_imu_port" value="/dev/serial/by-id/usb-Lord_Microstrain_Lord_Inertial_Sensor_0000__6233.47093-if00" />
+	<xacro:property name="pelvis_rear_imu_port" value="/dev/serial/by-id/usb-Lord_Microstrain_Lord_Inertial_Sensor_0000__6233.47095-if00" />
+	<xacro:property name="torso_left_imu_port" value="/dev/serial/by-id/usb-Lord_Microstrain_Lord_Inertial_Sensor_0000__6233.47099-if00" />
 </robot>

File: common/xacro/dev_ports/valkyrie_gazebo_ports.xacro (robot description, xacro)
@@ -1,3 +1,5 @@
 <robot xmlns:xacro="http://ros.org/wiki/xacro" name="valkyrie_gazebo_ports">
 	<xacro:property name="pelvis_middle_imu_port" value="none" />
+	<xacro:property name="pelvis_rear_imu_port" value="none" />
+	<xacro:property name="torso_left_imu_port" value="none" />
 </robot>

File: common/xacro/nodes/valkyrie_nodes.xacro (robot description, xacro)
@@ -28,5 +28,4 @@
 	<xacro:property name="pelvis_rear_imu_node" value="/sensors/rearPelvisIMU" />
 	<xacro:property name="torso_left_imu_node" value="/sensors/leftTorsoIMU" />
-	<xacro:property name="torso_right_imu_node" value="/sensors/rightTorsoIMU" />
 	<xacro:property name="left_foot_ATI_node" value="/left_leg/ankle/left_actuator" />
 	<xacro:property name="left_foot_Sim_ATI_node" value="/sensors/leftFootSixAxis" />

File: instance/instances/robots/xacro/common/valkyrie_full_template.xacro (robot description, xacro)
@@ -21,5 +21,4 @@
 		<xacro:microstrain_imu name="pelvis_rear_imu" serial_number="${pelvis_rear_imu_serial}" node="${pelvis_rear_imu_node}" />
 		<xacro:microstrain_imu name="torso_left_imu" serial_number="${torso_left_imu_serial}" node="${torso_left_imu_node}" />
-		<xacro:microstrain_imu name="torso_right_imu" serial_number="${torso_right_imu_serial}" node="${torso_right_imu_node}" />
 		<xacro:ati_force_torque name="left_foot_force_torque" serial_number="${left_foot_ATI_serial}" node="${left_foot_ATI_node}"/>
 		<xacro:ati_force_torque name="right_foot_force_torque" serial_number="${right_foot_ATI_serial}" node="${right_foot_ATI_node}"/>

File: model/robots/common/xacro/valkyrie_base_hw.xacro (robot description, xacro)
@@ -15,5 +15,5 @@
     <xacro:make_leg prefix="right" reflect="-1" leg_root_link="${Pelvis_Link_Name}"/>
     <xacro:make_leg prefix="left" reflect="1" leg_root_link="${Pelvis_Link_Name}"/>
-    <xacro:v1_trunk_sensors/>
+     <xacro:v1_trunk_sensors_usb sensor_node_tag="${torso_left_imu_node}" sensor_api_tag="${ImuSensorHardwareApi}" sensor_port_tag="${torso_left_imu_port}"/>
     <xacro:v1_leg_sensors prefix="left" reflect="1" ATI_serial_number="${left_foot_ATI_serial}" ATI_node="${left_foot_ATI_node}"/>
     <xacro:v1_leg_sensors prefix="right" reflect="-1" ATI_serial_number="${right_foot_ATI_serial}" ATI_node="${right_foot_ATI_node}"/>

File: model/robots/common/xacro/valkyrie_base_sim.xacro (robot description, xacro)
@@ -24,5 +24,5 @@
     <xacro:v1_leg_sensors prefix="right" reflect="-1" ATI_serial_number="${sim_ATI_serial}" ATI_node="${right_foot_Sim_ATI_node}"/>
     <xacro:include_multisense_sim />
-    <xacro:v1_trunk_sensors/>
+    <xacro:v1_trunk_sensors_usb sensor_node_tag="${torso_left_imu_node}" sensor_api_tag="${ImuSensorSimApi}" sensor_port_tag="${torso_left_imu_port}"/>
     <xacro:waist_transmissions_sim />
     <xacro:leg_transmissions_sim prefix="left"/>

File: model/robots/common/xacro/valkyrie_no_hands_base_hw.xacro (robot description, xacro)
@@ -7,5 +7,5 @@
     <xacro:make_leg prefix="right" reflect="-1" leg_root_link="${Pelvis_Link_Name}"/>
     <xacro:make_leg prefix="left" reflect="1" leg_root_link="${Pelvis_Link_Name}"/>
-    <xacro:v1_trunk_sensors/>
+    <xacro:v1_trunk_sensors_usb sensor_node_tag="${torso_left_imu_node}" sensor_api_tag="${ImuSensorHardwareApi}" sensor_port_tag="${torso_left_imu_port}"/>
     <xacro:v1_leg_sensors prefix="left" reflect="1" ATI_serial_number="${left_foot_ATI_serial}" ATI_node="${left_foot_ATI_node}"/>
     <xacro:v1_leg_sensors prefix="right" reflect="-1" ATI_serial_number="${right_foot_ATI_serial}" ATI_node="${right_foot_ATI_node}"/>

File: model/robots/common/xacro/waist/waist.xacro (robot description, xacro)
@@ -91,4 +91,25 @@
                         frameRate="60"/>
    </xacro:macro>
+  <xacro:macro name="v1_trunk_sensors_usb" params="sensor_node_tag sensor_api_tag sensor_port_tag">
+    <xacro:usb_microstrain_sensor sensorName="leftTorsoIMU"
+                              parentLink="${TorsoRollLinkName}"
+                              origin_xyz="-0.046863 0.134239 0.3630676"
+                              origin_rpy="1.57 0 3.14"
+                              sensor_node="${sensor_node_tag}"
+                              sensor_api="${sensor_api_tag}"
+                              sensor_port="${sensor_port_tag}" />
+    <xacro:flea3_camera sensorName="rightHazardCamera"
+                        parentLink="${TorsoRollLinkName}"
+                        origin_xyz="0.0345 -0.0406 0.1135"
+                        origin_rpy="1.57 0.0 1.57"
+                        imageFormat="R8G8B8"
+                        frameRate="60"/>
+    <xacro:flea3_camera sensorName="leftHazardCamera"
+                        parentLink="${TorsoRollLinkName}"
+                        origin_xyz="0.0345 0.0406 0.1135"
+                        origin_rpy="1.57 0.0 1.57"
+                        imageFormat="R8G8B8"
+                        frameRate="60"/>
+   </xacro:macro>
    <xacro:macro name="waist_transmissions_hw">
     <xacro:simple_transmission jointName="${TorsoYawJointName}" actuatorName="${TorsoYawActuatorName}" nodeName="${TrunkYawNode}" actuatorApi="${TrunkYawApi}"/>
