Commit message: Trying to sort out unit D's imus.

File: common/xacro/dev_ports/valkyrie_D_ports.xacro (robot description, xacro)
@@ -1,5 +1,5 @@
 <robot xmlns:xacro="http://ros.org/wiki/xacro" name="valkyrie_D_ports">
     <xacro:property name="pelvis_middle_imu_port" value="UNKNOWN" />
-    <xacro:property name="pelvis_rear_imu_port" value="/dev/serial/by-id/usb-Lord_Microstrain_Lord_Inertial_Sensor_0000__4220.47098-if00" />
-    <xacro:property name="torso_left_imu_port" value="UNKNOWN" />
+    <xacro:property name="pelvis_rear_imu_port" value="/dev/serial/by-id/usb-FTDI_USB-RS232_Cable_FTY5H9NH-if00-port0" />
+    <xacro:property name="torso_left_imu_port" value="/dev/serial/by-id/usb-Lord_Microstrain_Lord_Inertial_Sensor_0000__6233.47097-if00" />
 </robot>

Commit message: Settling on an IMU config for unit D.

File: common/xacro/dev_ports/valkyrie_D_ports.xacro (robot description, xacro)
@@ -1,5 +1,5 @@
 <robot xmlns:xacro="http://ros.org/wiki/xacro" name="valkyrie_D_ports">
     <xacro:property name="pelvis_middle_imu_port" value="UNKNOWN" />
-    <xacro:property name="pelvis_rear_imu_port" value="/dev/serial/by-id/usb-FTDI_USB-RS232_Cable_FTY5H9NH-if00-port0" />
+    <xacro:property name="pelvis_rear_imu_port" value="/dev/serial/by-id/usb-Lord_Microstrain_Lord_Inertial_Sensor_0000__6234.50971-if00" />
     <xacro:property name="torso_left_imu_port" value="/dev/serial/by-id/usb-Lord_Microstrain_Lord_Inertial_Sensor_0000__6233.47097-if00" />
 </robot>

File: model/robots/common/xacro/valkyrie_no_hands_base_hw.xacro (robot description, xacro)
@@ -11,5 +11,5 @@
     <xacro:v1_leg_sensors prefix="right" reflect="-1" ATI_serial_number="${right_foot_ATI_serial}" ATI_node="${right_foot_ATI_node}"/>
     <xacro:include_multisense_hw />
-    <xacro:v1_pelvis_rear_sensors_usb sensor_node_tag="${pelvis_rear_imu_node}" sensor_api_tag="${ImuVectorNavHardwareApi}"  sensor_port_tag="${pelvis_rear_imu_port}"/>
+    <xacro:v1_pelvis_rear_sensors_usb sensor_node_tag="${pelvis_rear_imu_node}" sensor_api_tag="${ImuMicrostrainHardwareApi}"  sensor_port_tag="${pelvis_rear_imu_port}"/>
     <xacro:waist_transmissions_hw />
     <xacro:leg_transmissions_hw prefix="left"/>

Commit message: change imu to uoe purchased sensor

File: common/xacro/dev_ports/valkyrie_D_ports.xacro (robot description, xacro)
@@ -1,5 +1,5 @@
 <robot xmlns:xacro="http://ros.org/wiki/xacro" name="valkyrie_D_ports">
     <xacro:property name="pelvis_middle_imu_port" value="UNKNOWN" />
-    <xacro:property name="pelvis_rear_imu_port" value="/dev/serial/by-id/usb-Lord_Microstrain_Lord_Inertial_Sensor_0000__6234.50971-if00" />
+    <xacro:property name="pelvis_rear_imu_port" value="/dev/serial/by-id/usb-Lord_Microstrain_Lord_Inertial_Sensor_0000__6233.51067-if00" />
     <xacro:property name="torso_left_imu_port" value="/dev/serial/by-id/usb-Lord_Microstrain_Lord_Inertial_Sensor_0000__6233.47093-if00" />
 </robot>
