Commit message: updated to allow hardware to use usb ports

File: common/xacro/dev_ports/valkyrie_C_ports.xacro (robot description, xacro)
@@ -1,3 +1,3 @@
 <robot xmlns:xacro="http://ros.org/wiki/xacro" name="valkyrie_C_ports">
-	<xacro:property name="pelvis_middle_imu_port" value="/dev/ttyACM0" />
+	<xacro:property name="pelvis_middle_imu_port" value="/dev/serial/by-id/usb-Lord_Microstrain_Lord_Inertial_Sensor_0000__6233.47093-if00" />
 </robot>

File: model/robots/common/xacro/valkyrie_base_hw.xacro (robot description, xacro)
@@ -19,5 +19,5 @@
     <xacro:v1_leg_sensors prefix="right" reflect="-1" ATI_serial_number="${right_foot_ATI_serial}" ATI_node="${right_foot_ATI_node}"/>
     <xacro:include_multisense_hw />
-    <xacro:v1_pelvis_sensors/>
+    <xacro:v1_pelvis_sensors_usb sensor_node_tag="${pelvis_middle_imu_node}" sensor_api_tag="${ImuSensorSimApi}" sensor_port_tag="${pelvis_middle_imu_port}"/>
     <xacro:waist_transmissions_hw />
     <xacro:leg_transmissions_hw prefix="left"/>

File: model/robots/common/xacro/valkyrie_no_hands_base_hw.xacro (robot description, xacro)
@@ -11,5 +11,5 @@
     <xacro:v1_leg_sensors prefix="right" reflect="-1" ATI_serial_number="${right_foot_ATI_serial}" ATI_node="${right_foot_ATI_node}"/>
     <xacro:include_multisense_hw />
-    <xacro:v1_pelvis_sensors/>
+    <xacro:v1_pelvis_sensors_usb sensor_node_tag="${pelvis_middle_imu_node}" sensor_api_tag="${ImuSensorSimApi}" sensor_port_tag="${pelvis_middle_imu_port}"/>
     <xacro:waist_transmissions_hw />
     <xacro:leg_transmissions_hw prefix="left"/>

File: model/robots/valkyrie_A_hw.xacro (robot description, xacro)
@@ -5,3 +5,4 @@
     <xacro:include filename="$(find val_description)/model/robots/common/xacro/valkyrie_base_hw.xacro"/>
     <xacro:include filename="$(find val_description)/common/xacro/serial_numbers/valkyrie_A_serials.xacro"/>
+    <xacro:include filename="$(find val_description)/common/xacro/dev_ports/valkyrie_A_ports.xacro"/>
 </robot>

File: model/robots/valkyrie_A_no_hands_hw.xacro (robot description, xacro)
@@ -5,3 +5,4 @@
     <xacro:include filename="$(find val_description)/model/robots/common/xacro/valkyrie_no_hands_base_hw.xacro"/>
     <xacro:include filename="$(find val_description)/common/xacro/serial_numbers/valkyrie_A_serials.xacro"/>
+    <xacro:include filename="$(find val_description)/common/xacro/dev_ports/valkyrie_A_ports.xacro"/>
 </robot>

Commit message: updated ports to use vectornav imu

File: common/xacro/dev_ports/valkyrie_C_ports.xacro (robot description, xacro)
@@ -1,5 +1,5 @@
 <robot xmlns:xacro="http://ros.org/wiki/xacro" name="valkyrie_C_ports">
 	<xacro:property name="pelvis_middle_imu_port" value="/dev/serial/by-id/usb-Lord_Microstrain_Lord_Inertial_Sensor_0000__6233.47093-if00" />
-	<xacro:property name="pelvis_rear_imu_port" value="/dev/serial/by-id/usb-Lord_Microstrain_Lord_Inertial_Sensor_0000__6233.47095-if00" />
+	<xacro:property name="pelvis_rear_imu_port" value="/dev/serial/by-id/usb-FTDI_USB-RS232_Cable_FTY5H9NH-if00-port0" />
 	<xacro:property name="torso_left_imu_port" value="/dev/serial/by-id/usb-Lord_Microstrain_Lord_Inertial_Sensor_0000__6233.47099-if00" />
 </robot>

File: model/robots/common/xacro/valkyrie_no_hands_base_hw.xacro (robot description, xacro)
@@ -11,5 +11,5 @@
     <xacro:v1_leg_sensors prefix="right" reflect="-1" ATI_serial_number="${right_foot_ATI_serial}" ATI_node="${right_foot_ATI_node}"/>
     <xacro:include_multisense_hw />
-    <xacro:v1_pelvis_sensors_usb sensor_node_tag="${pelvis_middle_imu_node}" sensor_api_tag="${ImuSensorHardwareApi}"  sensor_port_tag="${pelvis_middle_imu_port}"/>
+    <xacro:v1_pelvis_rear_sensors_usb sensor_node_tag="${pelvis_rear_imu_node}" sensor_api_tag="${ImuSensorHardwareApi}"  sensor_port_tag="${pelvis_rear_imu_port}"/>
     <xacro:waist_transmissions_hw />
     <xacro:leg_transmissions_hw prefix="left"/>

Commit message: Updated IMU serial for unit C.

File: common/xacro/dev_ports/valkyrie_C_ports.xacro (robot description, xacro)
@@ -1,5 +1,5 @@
 <robot xmlns:xacro="http://ros.org/wiki/xacro" name="valkyrie_C_ports">
 	<xacro:property name="pelvis_middle_imu_port" value="/dev/serial/by-id/usb-Lord_Microstrain_Lord_Inertial_Sensor_0000__6233.47093-if00" />
-	<xacro:property name="pelvis_rear_imu_port" value="/dev/serial/by-id/usb-Lord_Microstrain_Lord_Inertial_Sensor_0000__6233.47095-if00" />
+	<xacro:property name="pelvis_rear_imu_port" value="/dev/serial/by-id/usb-Lord_Microstrain_Lord_Inertial_Sensor_0000__6233.47098-if00" />
 	<xacro:property name="torso_left_imu_port" value="/dev/serial/by-id/usb-Lord_Microstrain_Lord_Inertial_Sensor_0000__6233.47099-if00" />
 </robot>

Commit message: Swapped some IMU ports on unit D.

File: common/xacro/dev_ports/valkyrie_C_ports.xacro (robot description, xacro)
@@ -1,5 +1,4 @@
 <robot xmlns:xacro="http://ros.org/wiki/xacro" name="valkyrie_C_ports">
-	<xacro:property name="pelvis_middle_imu_port" value="/dev/serial/by-id/usb-Lord_Microstrain_Lord_Inertial_Sensor_0000__6233.47093-if00" />
-	<xacro:property name="pelvis_rear_imu_port" value="/dev/serial/by-id/usb-FTDI_USB-RS232_Cable_FTY5H9NH-if00-port0" />
+	<xacro:property name="pelvis_rear_imu_port" value="/dev/serial/by-id/usb-Lord_Microstrain_Lord_Inertial_Sensor_0000__6234.50971-if00" />
 	<xacro:property name="torso_left_imu_port" value="/dev/serial/by-id/usb-Lord_Microstrain_Lord_Inertial_Sensor_0000__6233.47099-if00" />
 </robot>

File: common/xacro/dev_ports/valkyrie_D_ports.xacro (robot description, xacro)
@@ -1,5 +1,5 @@
 <robot xmlns:xacro="http://ros.org/wiki/xacro" name="valkyrie_D_ports">
     <xacro:property name="pelvis_middle_imu_port" value="UNKNOWN" />
-    <xacro:property name="pelvis_rear_imu_port" value="/dev/serial/by-id/usb-Lord_Microstrain_Lord_Inertial_Sensor_0000__6234.50971-if00" />
+    <xacro:property name="pelvis_middle_imu_port" value="/dev/serial/by-id/usb-Lord_Microstrain_Lord_Inertial_Sensor_0000__6233.47093-if00" />
     <xacro:property name="torso_left_imu_port" value="/dev/serial/by-id/usb-Lord_Microstrain_Lord_Inertial_Sensor_0000__6233.47097-if00" />
 </robot>

Commit message: New torque offsets for actuators. These come from adapting torque offsets through IHMC's controller.

File: common/xacro/dev_ports/valkyrie_C_ports.xacro (robot description, xacro)
@@ -1,3 +1,4 @@
 <robot xmlns:xacro="http://ros.org/wiki/xacro" name="valkyrie_C_ports">
+	<xacro:property name="pelvis_middle_imu_port" value="UNKNOWN" />
 	<xacro:property name="pelvis_rear_imu_port" value="/dev/serial/by-id/usb-Lord_Microstrain_Lord_Inertial_Sensor_0000__6234.50971-if00" />
 	<xacro:property name="torso_left_imu_port" value="/dev/serial/by-id/usb-Lord_Microstrain_Lord_Inertial_Sensor_0000__6233.47099-if00" />

File: common/xacro/dev_ports/valkyrie_D_ports.xacro (robot description, xacro)
@@ -1,5 +1,5 @@
 <robot xmlns:xacro="http://ros.org/wiki/xacro" name="valkyrie_D_ports">
     <xacro:property name="pelvis_middle_imu_port" value="UNKNOWN" />
-    <xacro:property name="pelvis_middle_imu_port" value="/dev/serial/by-id/usb-Lord_Microstrain_Lord_Inertial_Sensor_0000__6233.47093-if00" />
-    <xacro:property name="torso_left_imu_port" value="/dev/serial/by-id/usb-Lord_Microstrain_Lord_Inertial_Sensor_0000__6233.47097-if00" />
+    <xacro:property name="pelvis_rear_imu_port" value="/dev/serial/by-id/usb-Lord_Microstrain_Lord_Inertial_Sensor_0000__6234.50971-if00" />
+    <xacro:property name="torso_left_imu_port" value="/dev/serial/by-id/usb-Lord_Microstrain_Lord_Inertial_Sensor_0000__6233.47093-if00" />
 </robot>

Commit message: updated imu ports

File: common/xacro/dev_ports/valkyrie_C_ports.xacro (robot description, xacro)
@@ -1,5 +1,5 @@
 <robot xmlns:xacro="http://ros.org/wiki/xacro" name="valkyrie_C_ports">
 	<xacro:property name="pelvis_middle_imu_port" value="UNKNOWN" />
-	<xacro:property name="pelvis_rear_imu_port" value="/dev/serial/by-id/usb-Lord_Microstrain_Lord_Inertial_Sensor_0000__6234.50971-if00" />
+	<xacro:property name="pelvis_rear_imu_port" value="/dev/serial/by-id/usb-Lord_Microstrain_Lord_Inertial_Sensor_0000__6234.50969-if00" />
 	<xacro:property name="torso_left_imu_port" value="/dev/serial/by-id/usb-Lord_Microstrain_Lord_Inertial_Sensor_0000__6233.47099-if00" />
 </robot>

Commit message: Updated port stuff to use microstrain-15

File: common/xacro/dev_ports/valkyrie_C_ports.xacro (robot description, xacro)
@@ -1,5 +1,6 @@
 <robot xmlns:xacro="http://ros.org/wiki/xacro" name="valkyrie_C_ports">
 	<xacro:property name="pelvis_middle_imu_port" value="UNKNOWN" />
-	<xacro:property name="pelvis_rear_imu_port" value="/dev/serial/by-id/usb-Lord_Microstrain_Lord_Inertial_Sensor_0000__6234.50969-if00" />
+	<xacro:property name="pelvis_rear_imu_port" value="/dev/serial/by-id/usb-Lord_Microstrain_Lord_Inertial_Sensor_0000__6233.47251-if00" />
+	<!-- <xacro:property name="pelvis_rear_imu_port" value="/dev/serial/by-id/usb-FTDI_USB-RS422_Cable_FTXRO1OW-if00-port0" /> -->
 	<xacro:property name="torso_left_imu_port" value="/dev/serial/by-id/usb-Lord_Microstrain_Lord_Inertial_Sensor_0000__6233.47099-if00" />
 </robot>

File: model/robots/common/xacro/valkyrie_no_hands_base_hw.xacro (robot description, xacro)
@@ -11,5 +11,5 @@
     <xacro:v1_leg_sensors prefix="right" reflect="-1" ATI_serial_number="${right_foot_ATI_serial}" ATI_node="${right_foot_ATI_node}"/>
     <xacro:include_multisense_hw />
-    <xacro:v1_pelvis_rear_sensors_usb sensor_node_tag="${pelvis_rear_imu_node}" sensor_api_tag="${KVHHardwareApi}"  sensor_port_tag="${pelvis_rear_imu_port}"/>
+    <xacro:v1_pelvis_rear_sensors_usb sensor_node_tag="${pelvis_rear_imu_node}" sensor_api_tag="${ImuMicrostrainHardwareApi}"  sensor_port_tag="${pelvis_rear_imu_port}"/>
     <xacro:waist_transmissions_hw />
     <xacro:leg_transmissions_hw prefix="left"/>

Commit message: Jordan: Pulled develop and fixed IMU port for unit C.

File: common/xacro/dev_ports/valkyrie_C_ports.xacro (robot description, xacro)
@@ -3,4 +3,4 @@
 	<xacro:property name="pelvis_rear_imu_port" value="/dev/serial/by-id/usb-Lord_Microstrain_Lord_Inertial_Sensor_0000__6233.47251-if00" />
 	<!-- <xacro:property name="pelvis_rear_imu_port" value="/dev/serial/by-id/usb-FTDI_USB-RS422_Cable_FTXRO1OW-if00-port0" /> -->
-	<xacro:property name="torso_left_imu_port" value="/dev/serial/by-id/usb-Lord_Microstrain_Lord_Inertial_Sensor_0000__6233.47099-if00" />
+	<xacro:property name="torso_left_imu_port" value="/dev/serial/by-id/usb-Lord_Microstrain_Lord_Inertial_Sensor_0000__6233.47096-if00" />
 </robot>
