Commit message: update tag names to be more descriptive

File: common/xacro/dev_ports/valkyrie_B_ports.xacro (robot description, xacro)
@@ -1,3 +1,3 @@
 <robot xmlns:xacro="http://ros.org/wiki/xacro" name="valkyrie_B_ports">
-	<xacro:property name="pelvis_imu1_port" value="/dev/ttyACM0" />
+	<xacro:property name="pelvis_middle_imu_port" value="/dev/ttyACM0" />
 </robot>

File: common/xacro/dev_ports/valkyrie_C_ports.xacro (robot description, xacro)
@@ -1,3 +1,3 @@
 <robot xmlns:xacro="http://ros.org/wiki/xacro" name="valkyrie_C_ports">
-	<xacro:property name="pelvis_imu1_port" value="/dev/ttyACM0" />
+	<xacro:property name="pelvis_middle_imu_port" value="/dev/ttyACM0" />
 </robot>

File: common/xacro/dev_ports/valkyrie_gazebo_ports.xacro (robot description, xacro)
@@ -1,3 +1,3 @@
 <robot xmlns:xacro="http://ros.org/wiki/xacro" name="valkyrie_gazebo_ports">
-	<xacro:property name="pelvis_imu1_port" value="none" />
+	<xacro:property name="pelvis_middle_imu_port" value="none" />
 </robot>

File: common/xacro/nodes/valkyrie_nodes.xacro (robot description, xacro)
@@ -25,8 +25,8 @@
 	<xacro:property name="WaistPitchActuatorSimNode" value="/trunk/pitch_actuator" /> <!--pitch-->
 	<xacro:property name="WaistRollActuatorSimNode" value="/trunk/roll_actuator" /> <!--roll-->
-	<xacro:property name="pelvis_imu1_node" value="/sensors/leftPelvisIMU" />
-	<xacro:property name="pelvis_imu2_node" value="/pelvis/sensors/imu2" />
-	<xacro:property name="torso_imu1_node" value="/torso/sensors/imu1" />
-	<xacro:property name="torso_imu2_node" value="/torso/sensors/imu2" />
+	<xacro:property name="pelvis_middle_imu_node" value="/sensors/leftPelvisIMU" />
+	<xacro:property name="pelvis_rear_imu_node" value="/sensors/rightPelvisIMU" />
+	<xacro:property name="torso_left_imu_node" value="/sensors/leftTorsoIMU" />
+	<xacro:property name="torso_right_imu_node" value="/sensors/rightTorsoIMU" />
 	<xacro:property name="left_foot_ATI_node" value="/left_leg/ankle/left_actuator" />
 	<xacro:property name="left_foot_Sim_ATI_node" value="/sensors/leftFootSixAxis" />

File: common/xacro/serial_numbers/valkyrie_A_serials.xacro (robot description, xacro)
@@ -32,8 +32,8 @@
 	<xacro:property name="waistRightActuatorSerialNumber" value="v_e_005" />
 	<xacro:property name="waistLeftActuatorSerialNumber" value="v_e_006" />
-	<xacro:property name="pelvis_imu1_serial" value="UNKNOWN" />
-	<xacro:property name="pelvis_imu2_serial" value="UNKNOWN" />
-	<xacro:property name="torso_imu1_serial" value="UNKNOWN" />
-	<xacro:property name="torso_imu2_serial" value="UNKNOWN" />
+	<xacro:property name="pelvis_middle_imu_serial" value="UNKNOWN" />
+	<xacro:property name="pelvis_rear_imu_serial" value="UNKNOWN" />
+	<xacro:property name="torso_left_imu_serial" value="UNKNOWN" />
+	<xacro:property name="torso_right_imu_serial" value="UNKNOWN" />
 	<xacro:property name="left_foot_ATI_serial" value="FT14020" />
 	<xacro:property name="right_foot_ATI_serial" value="FT16592" />

File: common/xacro/serial_numbers/valkyrie_B_serials.xacro (robot description, xacro)
@@ -32,8 +32,8 @@
 	<xacro:property name="waistRightActuatorSerialNumber" value="v_e_011" />
 	<xacro:property name="waistLeftActuatorSerialNumber" value="v_e_012" />
-	<xacro:property name="pelvis_imu1_serial" value="UNKNOWN" />
-	<xacro:property name="pelvis_imu2_serial" value="UNKNOWN" />
-	<xacro:property name="torso_imu1_serial" value="UNKNOWN" />
-	<xacro:property name="torso_imu2_serial" value="UNKNOWN" />
+	<xacro:property name="pelvis_middle_imu_serial" value="UNKNOWN" />
+	<xacro:property name="pelvis_rear_imu_serial" value="UNKNOWN" />
+	<xacro:property name="torso_left_imu_serial" value="UNKNOWN" />
+	<xacro:property name="torso_right_imu_serial" value="UNKNOWN" />
 	<xacro:property name="left_foot_ATI_serial" value="FT17219" />
 	<xacro:property name="right_foot_ATI_serial" value="FT17215" />

File: common/xacro/serial_numbers/valkyrie_C_serials.xacro (robot description, xacro)
@@ -32,8 +32,8 @@
 	<xacro:property name="waistRightActuatorSerialNumber" value="v_e_014" />
 	<xacro:property name="waistLeftActuatorSerialNumber" value="v_e_013" />
-	<xacro:property name="pelvis_imu1_serial" value="UNKNOWN" />
-	<xacro:property name="pelvis_imu2_serial" value="UNKNOWN" />
-	<xacro:property name="torso_imu1_serial" value="UNKNOWN" />
-	<xacro:property name="torso_imu2_serial" value="UNKNOWN" />
+	<xacro:property name="pelvis_middle_imu_serial" value="UNKNOWN" />
+	<xacro:property name="pelvis_rear_imu_serial" value="UNKNOWN" />
+	<xacro:property name="torso_left_imu_serial" value="UNKNOWN" />
+	<xacro:property name="torso_right_imu_serial" value="UNKNOWN" />
 	<xacro:property name="left_foot_ATI_serial" value="FT17213" />
 	<xacro:property name="right_foot_ATI_serial" value="FT17217" />

File: instance/instances/robots/xacro/common/valkyrie_full_template.xacro (robot description, xacro)
@@ -18,8 +18,8 @@
 	</Mechanisms>
 	<Devices>
-		<xacro:microstrain_imu name="pelvis_imu1" serial_number="${pelvis_imu1_serial}" node="${pelvis_imu1_node}" />
-		<xacro:microstrain_imu name="pelvis_imu2" serial_number="${pelvis_imu2_serial}" node="${pelvis_imu2_node}" />
-		<xacro:microstrain_imu name="torso_imu1" serial_number="${torso_imu1_serial}" node="${torso_imu1_node}" />
-		<xacro:microstrain_imu name="torso_imu2" serial_number="${torso_imu2_serial}" node="${torso_imu2_node}" />
+		<xacro:microstrain_imu name="pelvis_middle_imu" serial_number="${pelvis_middle_imu_serial}" node="${pelvis_middle_imu_node}" />
+		<xacro:microstrain_imu name="pelvis_rear_imu" serial_number="${pelvis_rear_imu_serial}" node="${pelvis_rear_imu_node}" />
+		<xacro:microstrain_imu name="torso_left_imu" serial_number="${torso_left_imu_serial}" node="${torso_left_imu_node}" />
+		<xacro:microstrain_imu name="torso_right_imu" serial_number="${torso_right_imu_serial}" node="${torso_right_imu_node}" />
 		<xacro:ati_force_torque name="left_foot_force_torque" serial_number="${left_foot_ATI_serial}" node="${left_foot_ATI_node}"/>
 		<xacro:ati_force_torque name="right_foot_force_torque" serial_number="${right_foot_ATI_serial}" node="${right_foot_ATI_node}"/>

File: model/robots/common/xacro/pelvis/pelvis.xacro (robot description, xacro)
@@ -21,10 +21,10 @@
                                   origin_rpy="3.14159 0.0 -3.14159" />
     </xacro:macro>
-    <xacro:macro name="v1_pelvis_sensors_plugin" params="sensor_node_tag sensor_api_tag sensor_port_tag">
+    <xacro:macro name="v1_pelvis_sensors_usb" params="sensor_node_tag sensor_api_tag sensor_port_tag">
         <xacro:microstrain_sensor sensorName="pelvisRearImu"
                                   parentLink="${Pelvis_Link_Name}"
                                   origin_xyz="-0.075844901 0.0 -0.111056426"
                                   origin_rpy="-3.14159 0.476467 -3.14159" />
-        <xacro:plugged_in_microstrain_sensor sensorName="pelvisMiddleImu"
+        <xacro:usb_microstrain_sensor sensorName="pelvisMiddleImu"
                                   parentLink="${Pelvis_Link_Name}"
                                   origin_xyz="0.012 0.0 -0.108184035"

File: model/robots/common/xacro/valkyrie_base_sim.xacro (robot description, xacro)
@@ -20,5 +20,5 @@
     <xacro:make_leg prefix="right" reflect="-1" leg_root_link="${Pelvis_Link_Name}"/>
     <xacro:make_leg prefix="left" reflect="1" leg_root_link="${Pelvis_Link_Name}"/>
-    <xacro:v1_pelvis_sensors_plugin sensor_node_tag="${pelvis_imu1_node}" sensor_api_tag="${ImuSensorSimApi}" sensor_port_tag="${pelvis_imu1_port}"/>
+    <xacro:v1_pelvis_sensors_usb sensor_node_tag="${pelvis_middle_imu_node}" sensor_api_tag="${ImuSensorSimApi}" sensor_port_tag="${pelvis_middle_imu_port}"/>
     <xacro:v1_leg_sensors prefix="left" reflect="1" ATI_serial_number="${sim_ATI_serial}" ATI_node="${left_foot_Sim_ATI_node}"/>
     <xacro:v1_leg_sensors prefix="right" reflect="-1" ATI_serial_number="${sim_ATI_serial}" ATI_node="${right_foot_Sim_ATI_node}"/>

Commit message: updated ports for valkyrie B

File: common/xacro/dev_ports/valkyrie_B_ports.xacro (robot description, xacro)
@@ -1,3 +1,3 @@
 <robot xmlns:xacro="http://ros.org/wiki/xacro" name="valkyrie_B_ports">
-	<xacro:property name="pelvis_middle_imu_port" value="/dev/ttyACM0" />
+	<xacro:property name="pelvis_middle_imu_port" value="/dev/serial/by-id/usb-Lord_Microstrain_Lord_Inertial_Sensor_0000__6233.47092-if00" />
 </robot>

Commit message: Unit B walking around nicely. Just some coeff changes for not hitting force limits.

File: common/xacro/dev_ports/valkyrie_B_ports.xacro (robot description, xacro)
@@ -1,4 +1,4 @@
 <robot xmlns:xacro="http://ros.org/wiki/xacro" name="valkyrie_B_ports">
-	<xacro:property name="pelvis_middle_imu_port" value="/dev/serial/by-id/usb-Lord_Microstrain_Lord_Inertial_Sensor_0000__6233.47092-if00" />
+	<xacro:property name="pelvis_middle_imu_port" value="/dev/serial/by-id/usb-Lord_Microstrain_Lord_Inertial_Sensor_0000__6233.47087-if00" />
 	<xacro:property name="pelvis_rear_imu_port" value="/dev/serial/by-id/usb-Lord_Microstrain_Lord_Inertial_Sensor_0000__6233.47094-if00" />
 	<xacro:property name="torso_left_imu_port" value="/dev/serial/by-id/usb-Lord_Microstrain_Lord_Inertial_Sensor_0000__6233.47100-if00" />

File: model/robots/common/xacro/valkyrie_no_hands_base_hw.xacro (robot description, xacro)
@@ -11,5 +11,5 @@
     <xacro:v1_leg_sensors prefix="right" reflect="-1" ATI_serial_number="${right_foot_ATI_serial}" ATI_node="${right_foot_ATI_node}"/>
     <xacro:include_multisense_hw />
-    <xacro:v1_pelvis_sensors_usb sensor_node_tag="${pelvis_middle_imu_node}" sensor_api_tag="${ImuSensorHardwareApi}"  sensor_port_tag="${pelvis_middle_imu_port}"/>
+    <xacro:v1_pelvis_sensors_usb sensor_node_tag="${pelvis_middle_imu_node}" sensor_api_tag="${ImuSensorHardwareApi}" sensor_port_tag="${pelvis_middle_imu_port}"/>
     <xacro:waist_transmissions_hw />
     <xacro:leg_transmissions_hw prefix="left"/>

Commit message: Updated IMU port numbers on unit B.

File: common/xacro/dev_ports/valkyrie_B_ports.xacro (robot description, xacro)
@@ -1,4 +1,4 @@
 <robot xmlns:xacro="http://ros.org/wiki/xacro" name="valkyrie_B_ports">
-	<xacro:property name="pelvis_middle_imu_port" value="/dev/serial/by-id/usb-Lord_Microstrain_Lord_Inertial_Sensor_0000__6233.47087-if00" />
+	<xacro:property name="pelvis_middle_imu_port" value="/dev/serial/by-id/usb-Lord_Microstrain_Lord_Inertial_Sensor_0000__6233.47094-if00" />
 	<xacro:property name="pelvis_rear_imu_port" value="/dev/serial/by-id/usb-Lord_Microstrain_Lord_Inertial_Sensor_0000__6233.47094-if00" />
 	<xacro:property name="torso_left_imu_port" value="/dev/serial/by-id/usb-Lord_Microstrain_Lord_Inertial_Sensor_0000__6233.47100-if00" />

Commit message: modified placement, port, and orientation of vector nav imu in urdf

File: common/xacro/dev_ports/valkyrie_B_ports.xacro (robot description, xacro)
@@ -1,5 +1,5 @@
 <robot xmlns:xacro="http://ros.org/wiki/xacro" name="valkyrie_B_ports">
 	<xacro:property name="pelvis_middle_imu_port" value="/dev/serial/by-id/usb-Lord_Microstrain_Lord_Inertial_Sensor_0000__6233.47094-if00" />
-	<xacro:property name="pelvis_rear_imu_port" value="/dev/serial/by-id/usb-Lord_Microstrain_Lord_Inertial_Sensor_0000__6233.47094-if00" />
+	<xacro:property name="pelvis_rear_imu_port" value="/dev/serial/by-id/usb-FTDI_USB-RS232_Cable_FTY5H9NH-if00-port0" />
 	<xacro:property name="torso_left_imu_port" value="/dev/serial/by-id/usb-Lord_Microstrain_Lord_Inertial_Sensor_0000__6233.47100-if00" />
 </robot>

File: model/robots/common/xacro/pelvis/pelvis.xacro (robot description, xacro)
@@ -38,5 +38,5 @@
                                   parentLink="${Pelvis_Link_Name}"
                                   origin_xyz="-0.075844901 0.0 -0.111056426"
-                                  origin_rpy="-3.14159 0.476467 -3.14159"
+                                  origin_rpy="-3.14159 0.476467 0"
 				  sensor_node="${sensor_node_tag}"
 				  sensor_api="${sensor_api_tag}"

File: model/robots/common/xacro/valkyrie_no_hands_base_hw.xacro (robot description, xacro)
@@ -7,9 +7,9 @@
     <xacro:make_leg prefix="right" reflect="-1" leg_root_link="${Pelvis_Link_Name}"/>
     <xacro:make_leg prefix="left" reflect="1" leg_root_link="${Pelvis_Link_Name}"/>
-    <xacro:v1_trunk_sensors_usb sensor_node_tag="${torso_left_imu_node}" sensor_api_tag="${ImuSensorHardwareApi}" sensor_port_tag="${torso_left_imu_port}"/>
+    <xacro:v1_trunk_sensors />
     <xacro:v1_leg_sensors prefix="left" reflect="1" ATI_serial_number="${left_foot_ATI_serial}" ATI_node="${left_foot_ATI_node}"/>
     <xacro:v1_leg_sensors prefix="right" reflect="-1" ATI_serial_number="${right_foot_ATI_serial}" ATI_node="${right_foot_ATI_node}"/>
     <xacro:include_multisense_hw />
-    <xacro:v1_pelvis_sensors_usb sensor_node_tag="${pelvis_middle_imu_node}" sensor_api_tag="${ImuSensorHardwareApi}" sensor_port_tag="${pelvis_middle_imu_port}"/>
+    <xacro:v1_pelvis_rear_sensors_usb sensor_node_tag="${pelvis_rear_imu_node}" sensor_api_tag="${ImuSensorHardwareApi}" sensor_port_tag="${pelvis_rear_imu_port}"/>
     <xacro:waist_transmissions_hw />
     <xacro:leg_transmissions_hw prefix="left"/>

Commit message: pushing to pull

File: common/xacro/dev_ports/valkyrie_B_ports.xacro (robot description, xacro)
@@ -1,5 +1,6 @@
 <robot xmlns:xacro="http://ros.org/wiki/xacro" name="valkyrie_B_ports">
 	<xacro:property name="pelvis_middle_imu_port" value="/dev/serial/by-id/usb-Lord_Microstrain_Lord_Inertial_Sensor_0000__6233.47094-if00" />
-	<xacro:property name="pelvis_rear_imu_port" value="/dev/serial/by-id/usb-FTDI_USB-RS232_Cable_FTY5H9NH-if00-port0" />
-	<xacro:property name="torso_left_imu_port" value="/dev/serial/by-id/usb-Lord_Microstrain_Lord_Inertial_Sensor_0000__6233.47100-if00" />
+	<!-- <xacro:property name="pelvis_rear_imu_port" value="/dev/serial/by-id/usb-FTDI_USB-RS232_Cable_FTY5H9NH-if00-port0" /> -->
+        <xacro:property name="pelvis_rear_imu_port" value="/dev/serial/by-id/usb-Lord_Microstrain_Lord_Inertial_Sensor_0000__6233.47250-if00" />
+	<xacro:property name="torso_left_imu_port" value="/dev/serial/by-id/usb-Lord_Microstrain_Lord_Inertial_Sensor_0000__6233.47097-if00" />
 </robot>

Commit message: updated coeffes for wrobot.

File: common/xacro/dev_ports/valkyrie_B_ports.xacro (robot description, xacro)
@@ -2,5 +2,5 @@
 	<xacro:property name="pelvis_middle_imu_port" value="/dev/serial/by-id/usb-Lord_Microstrain_Lord_Inertial_Sensor_0000__6233.47094-if00" />
 	<!-- <xacro:property name="pelvis_rear_imu_port" value="/dev/serial/by-id/usb-FTDI_USB-RS232_Cable_FTY5H9NH-if00-port0" /> -->
-        <xacro:property name="pelvis_rear_imu_port" value="/dev/serial/by-id/usb-Lord_Microstrain_Lord_Inertial_Sensor_0000__6233.47250-if00" />
+        <xacro:property name="pelvis_rear_imu_port" value="/dev/serial/by-id/usb-Lord_Microstrain_Lord_Inertial_Sensor_0000__6233.47092-if00" />
 	<xacro:property name="torso_left_imu_port" value="/dev/serial/by-id/usb-Lord_Microstrain_Lord_Inertial_Sensor_0000__6233.47097-if00" />
 </robot>

Commit message: Upped force limit in linears. Wrote torque offsets to file for unit B.

File: common/xacro/dev_ports/valkyrie_B_ports.xacro (robot description, xacro)
@@ -2,5 +2,5 @@
 	<xacro:property name="pelvis_middle_imu_port" value="/dev/serial/by-id/usb-Lord_Microstrain_Lord_Inertial_Sensor_0000__6233.47094-if00" />
 	<!-- <xacro:property name="pelvis_rear_imu_port" value="/dev/serial/by-id/usb-FTDI_USB-RS232_Cable_FTY5H9NH-if00-port0" /> -->
-        <xacro:property name="pelvis_rear_imu_port" value="/dev/serial/by-id/usb-Lord_Microstrain_Lord_Inertial_Sensor_0000__6233.47092-if00" />
+        <xacro:property name="pelvis_rear_imu_port" value="/dev/serial/by-id/usb-Lord_Microstrain_Lord_Inertial_Sensor_0000__6233.47250-if00" />
 	<xacro:property name="torso_left_imu_port" value="/dev/serial/by-id/usb-Lord_Microstrain_Lord_Inertial_Sensor_0000__6233.47097-if00" />
 </robot>

Commit message: Updated imu port for unit B. Wrote torque offsets to file. Restored knee actuator damping value to previous value of 0.017.

File: common/xacro/dev_ports/valkyrie_B_ports.xacro (robot description, xacro)
@@ -2,5 +2,5 @@
 	<xacro:property name="pelvis_middle_imu_port" value="/dev/serial/by-id/usb-Lord_Microstrain_Lord_Inertial_Sensor_0000__6233.47094-if00" />
 	<!-- <xacro:property name="pelvis_rear_imu_port" value="/dev/serial/by-id/usb-FTDI_USB-RS232_Cable_FTY5H9NH-if00-port0" /> -->
-        <xacro:property name="pelvis_rear_imu_port" value="/dev/serial/by-id/usb-Lord_Microstrain_Lord_Inertial_Sensor_0000__6233.47250-if00" />
+        <xacro:property name="pelvis_rear_imu_port" value="/dev/serial/by-id/usb-Lord_Microstrain_Lord_Inertial_Sensor_0000__6233.47099-if00" />
 	<xacro:property name="torso_left_imu_port" value="/dev/serial/by-id/usb-Lord_Microstrain_Lord_Inertial_Sensor_0000__6233.47097-if00" />
 </robot>
