Commit message: Forced to change links/joints to have lowercase first letter so the node names will jive with shared memory.

File: common/xacro/nodes/valkyrie_nodes.xacro (robot description, xacro)
@@ -1,27 +1,16 @@
 <robot xmlns:xacro="http://ros.org/wiki/xacro" name="valkyrie_nodes">
-	<xacro:property name="leftLegJ1Node" value="/left_leg/j1" />
-	<xacro:property name="leftLegJ2Node" value="/left_leg/j2" />
-	<xacro:property name="leftLegJ3Node" value="/left_leg/j3" />
-	<xacro:property name="leftLegJ4Node" value="/left_leg/j4" />
-	<xacro:property name="leftAnkleActuator0Node" value="/left_leg/ankle/actuator0" />
-	<xacro:property name="leftAnkleActuator1Node" value="/left_leg/ankle/actuator1" />
-	<xacro:property name="rightLegJ1Node" value="/right_leg/j1" />
-	<xacro:property name="rightLegJ2Node" value="/right_leg/j2" />
-	<xacro:property name="rightLegJ3Node" value="/right_leg/j3" />
-	<xacro:property name="rightLegJ4Node" value="/right_leg/j4" />
-	<xacro:property name="rightAnkleActuator0Node" value="/right_leg/ankle/actuator0" />
-	<xacro:property name="rightAnkleActuator1Node" value="/right_leg/ankle/actuator1" />
-	<xacro:property name="leftArmJ1Node" value="/left_arm/j1" />
-	<xacro:property name="leftArmJ2Node" value="/left_arm/j2" />
-	<xacro:property name="leftArmJ3Node" value="/left_arm/j3" />
-	<xacro:property name="leftArmJ4Node" value="/left_arm/j4" />
-	<xacro:property name="leftWristActuator0Node" value="/left_arm/wrist/actuator0" />
-	<xacro:property name="leftWristActuator1Node" value="/left_arm/wrist/actuator1" />
-	<xacro:property name="rightArmJ1Node" value="/right_arm/j1" />
-	<xacro:property name="rightArmJ2Node" value="/right_arm/j2" />
-	<xacro:property name="rightArmJ3Node" value="/right_arm/j3" />
-	<xacro:property name="rightArmJ4Node" value="/right_arm/j4" />
-	<xacro:property name="rightWristActuator0Node" value="/right_arm/wrist/actuator0" />
-	<xacro:property name="rightWristActuator1Node" value="/right_arm/wrist/actuator1" />
+	<xacro:property name="HipYawNode" value="/${prefix}_leg/j1" />
+	<xacro:property name="HipRollNode" value="/${prefix}_leg/j2" />
+	<xacro:property name="HipPitchNode" value="/${prefix}_leg/j3" />
+	<xacro:property name="KneePitchNode" value="/${prefix}_leg/j4" />
+	<xacro:property name="AnkleInsideActuatorNode" value="/${prefix}_leg/ankle/actuator0" />
+	<xacro:property name="AnkleOutsideActuatorNode" value="/${prefix}_leg/ankle/actuator1" />
+	<xacro:property name="ShoulderPitchNode" value="/${prefix}_arm/j1" />
+	<xacro:property name="ShoulderRollNode" value="/${prefix}_arm/j2" />
+	<xacro:property name="ShoulderYawNode" value="/${prefix}_arm/j3" />
+	<xacro:property name="ElbowPitchNode" value="/${prefix}_arm/j4" />
+	<xacro:property name="ForearmYawNode" value="/${prefix}_arm/j5" />
+	<xacro:property name="WristTopActuatorNode" value="/${prefix}_arm/wrist/top_actautor" />
+	<xacro:property name="WristBottomActuatorNode" value="/${prefix}_arm/wrist/bottom_actuator" />
 	<xacro:property name="neckJ1Node" value="/neck/j1" />
 	<xacro:property name="neckJ2Node" value="/neck/j2" />

File: instance/instances/robots/xacro/common/valkyrie_full_template.xacro (robot description, xacro)
@@ -11,8 +11,8 @@
 	<xacro:all_channels/>
 	<Mechanisms>
-		<xacro:leg side="left" j1_serial_number="${leftLegJ1SerialNumber}" j2_serial_number="${leftLegJ2SerialNumber}" j3_serial_number="${leftLegJ3SerialNumber}" j4_serial_number="${leftLegJ4SerialNumber}" ankle_actuator0_serial="${leftAnkleActuator0SerialNumber}" ankle_actuator1_serial="${leftAnkleActuator1SerialNumber}" j1_node="${leftLegJ1Node}" j2_node="${leftLegJ2Node}" j3_node="${leftLegJ3Node}" j4_node="${leftLegJ4Node}" ankle_actuator0_node="${leftAnkleActuator0Node}" ankle_actuator1_node="${leftAnkleActuator1Node}" />
-		<xacro:leg side="right" j1_serial_number="${rightLegJ1SerialNumber}" j2_serial_number="${rightLegJ2SerialNumber}" j3_serial_number="${rightLegJ3SerialNumber}" j4_serial_number="${rightLegJ4SerialNumber}" ankle_actuator0_serial="${rightAnkleActuator0SerialNumber}" ankle_actuator1_serial="${rightAnkleActuator1SerialNumber}" j1_node="${rightLegJ1Node}" j2_node="${rightLegJ2Node}" j3_node="${rightLegJ3Node}" j4_node="${rightLegJ4Node}" ankle_actuator0_node="${rightAnkleActuator0Node}" ankle_actuator1_node="${rightAnkleActuator1Node}" />
-		<xacro:arm side="left" j1_serial_number="${leftArmJ1SerialNumber}" j2_serial_number="${leftArmJ2SerialNumber}" j3_serial_number="${leftArmJ3SerialNumber}" j4_serial_number="${leftArmJ4SerialNumber}" j5_serial_number="${leftArmJ5SerialNumber}" wrist_actuator0_serial="${leftAnkleActuator0SerialNumber}" wrist_actuator1_serial="${leftAnkleActuator1SerialNumber}" j1_node="${leftArmJ1Node}" j2_node="${leftArmJ2Node}" j3_node="${leftArmJ3Node}" j4_node="${leftArmJ4Node}" j5_node="${leftArmJ4Node}" wrist_actuator0_node="${leftAnkleActuator0Node}" wrist_actuator1_node="${leftAnkleActuator1Node}" />
-		<xacro:arm side="right" j1_serial_number="${rightArmJ1SerialNumber}" j2_serial_number="${rightArmJ2SerialNumber}" j3_serial_number="${rightArmJ3SerialNumber}" j4_serial_number="${rightArmJ4SerialNumber}" j5_serial_number="${rightArmJ5SerialNumber}" wrist_actuator0_serial="${rightAnkleActuator0SerialNumber}" wrist_actuator1_serial="${rightAnkleActuator1SerialNumber}" j1_node="${rightArmJ1Node}" j2_node="${rightArmJ2Node}" j3_node="${rightArmJ3Node}" j4_node="${rightArmJ4Node}" j5_node="${rightArmJ4Node}" wrist_actuator0_node="${rightAnkleActuator0Node}" wrist_actuator1_node="${rightAnkleActuator1Node}" />
+		<xacro:leg prefix="left" j1_serial_number="${leftLegJ1SerialNumber}" j2_serial_number="${leftLegJ2SerialNumber}" j3_serial_number="${leftLegJ3SerialNumber}" j4_serial_number="${leftLegJ4SerialNumber}" ankle_actuator0_serial="${leftAnkleActuator0SerialNumber}" ankle_actuator1_serial="${leftAnkleActuator1SerialNumber}"/>
+		<xacro:leg prefix="right" j1_serial_number="${rightLegJ1SerialNumber}" j2_serial_number="${rightLegJ2SerialNumber}" j3_serial_number="${rightLegJ3SerialNumber}" j4_serial_number="${rightLegJ4SerialNumber}" ankle_actuator0_serial="${rightAnkleActuator0SerialNumber}" ankle_actuator1_serial="${rightAnkleActuator1SerialNumber}" />
+		<xacro:arm prefix="left" j1_serial_number="${leftArmJ1SerialNumber}" j2_serial_number="${leftArmJ2SerialNumber}" j3_serial_number="${leftArmJ3SerialNumber}" j4_serial_number="${leftArmJ4SerialNumber}" j5_serial_number="${leftArmJ5SerialNumber}" wrist_actuator0_serial="${leftAnkleActuator0SerialNumber}" wrist_actuator1_serial="${leftAnkleActuator1SerialNumber}" />
+		<xacro:arm prefix="right" j1_serial_number="${rightArmJ1SerialNumber}" j2_serial_number="${rightArmJ2SerialNumber}" j3_serial_number="${rightArmJ3SerialNumber}" j4_serial_number="${rightArmJ4SerialNumber}" j5_serial_number="${rightArmJ5SerialNumber}" wrist_actuator0_serial="${rightAnkleActuator0SerialNumber}" wrist_actuator1_serial="${rightAnkleActuator1SerialNumber}" />
 		<xacro:neck j1_serial_number="${neckJ1SerialNumber}" j2_serial_number="${neckJ1SerialNumber}" j3_serial_number="${neckJ1SerialNumber}" j1_node="${neckJ1Node}" j2_node="${neckJ2Node}" j3_node="${neckJ3Node}" />
 		<xacro:waist j1_serial_number="${trunkSerialNumber}" waist_actuator0_serial="${waistActuator0SerialNumber}" waist_actuator1_serial="${waistActuator1SerialNumber}" j1_node="${trunkNode}" waist_actuator0_node="${waistActuator0Node}" waist_actuator1_node="${waistActuator1Node}" />

File: instance/instances/robots/xacro/limbs/arm.xacro (robot description, xacro)
@@ -1,11 +1,12 @@
 <robot xmlns:xacro="http://ros.org/wiki/xacro" name="arm">
     <xacro:include filename="$(find val_description)/instance/instances/robots/xacro/mechanisms/mechanisms.xacro"/>
-    <xacro:macro name="arm" params="side j1_serial_number j2_serial_number j3_serial_number j4_serial_number j5_serial_number wrist_actuator0_serial wrist_actuator1_serial j1_node j2_node j3_node j4_node j5_node wrist_actuator0_node wrist_actuator1_node" >
-    	<xacro:simple_mechanism name="${side}_shoulder_pitch" serial_number="${j1_serial_number}" node="${j1_node}"/>
-    	<xacro:simple_mechanism name="${side}_shoulder_roll" serial_number="${j2_serial_number}" node="${j2_node}"/>
-    	<xacro:simple_mechanism name="${side}_shoulder_yaw" serial_number="${j3_serial_number}" node="${j3_node}"/>
-    	<xacro:simple_mechanism name="${side}_elbow_pitch" serial_number="${j4_serial_number}" node="${j4_node}"/>
-    	<xacro:simple_mechanism name="${side}_forearm_yaw" serial_number="${j5_serial_number}" node="${j5_node}"/>
-    	<xacro:two_active_joint_mechanism mechanism_name="${side}_wrist" joint0_name="pitch" joint1_name="roll" actuator0_serial="${wrist_actuator0_serial}" actuator1_serial="${wrist_actuator1_serial}" actuator0_node="${wrist_actuator0_node}" actuator1_node="${wrist_actuator1_node}" />
+    <xacro:include filename="$(find val_description)/common/xacro/joint_names/valkyrie_joint_names.xacro"/>
+    <xacro:macro name="arm" params="prefix j1_serial_number j2_serial_number j3_serial_number j4_serial_number j5_serial_number wrist_actuator0_serial wrist_actuator1_serial" >
+    	<xacro:simple_mechanism name="${ShoulderPitchJointName}" serial_number="${j1_serial_number}" node="${ShoulderYawNode}"/>
+    	<xacro:simple_mechanism name="${ShoulderRollJointName}" serial_number="${j2_serial_number}" node="${ShoulderRollNode}"/>
+    	<xacro:simple_mechanism name="${ShoulderYawJointName}" serial_number="${j3_serial_number}" node="${ShoulderYawNode}"/>
+    	<xacro:simple_mechanism name="${ElbowPitchJointName}" serial_number="${j4_serial_number}" node="${ElbowPitchNode}"/>
+    	<xacro:simple_mechanism name="${ForearmYawJointName}" serial_number="${j5_serial_number}" node="${ForearmYawNode}"/>
+    	<xacro:two_active_joint_mechanism mechanism_name="${prefix}Wrist" joint0_name="${WristPitchJointName}" joint1_name="${WristRollJointName}" actuator0_serial="${wrist_actuator0_serial}" actuator1_serial="${wrist_actuator1_serial}" actuator0_node="${WristTopActuatorNode}" actuator1_node="${WristBottomActuatorNode}" />
     </xacro:macro>
 </robot>

File: instance/instances/robots/xacro/limbs/leg.xacro (robot description, xacro)
@@ -1,10 +1,11 @@
 <robot xmlns:xacro="http://ros.org/wiki/xacro" name="leg">
     <xacro:include filename="$(find val_description)/instance/instances/robots/xacro/mechanisms/mechanisms.xacro"/>
-    <xacro:macro name="leg" params="side j1_serial_number j2_serial_number j3_serial_number j4_serial_number ankle_actuator0_serial ankle_actuator1_serial j1_node j2_node j3_node j4_node ankle_actuator0_node ankle_actuator1_node" >
-    	<xacro:simple_mechanism name="${side}_hip_yaw" serial_number="${j1_serial_number}" node="${j1_node}"/>
-    	<xacro:simple_mechanism name="${side}_hip_roll" serial_number="${j2_serial_number}" node="${j2_node}"/>
-    	<xacro:simple_mechanism name="${side}_hip_pitch" serial_number="${j3_serial_number}" node="${j3_node}"/>
-    	<xacro:simple_mechanism name="${side}_knee_pitch" serial_number="${j4_serial_number}" node="${j4_node}"/>
-    	<xacro:two_active_joint_mechanism mechanism_name="${side}_ankle" joint0_name="pitch" joint1_name="roll" actuator0_serial="${ankle_actuator0_serial}" actuator1_serial="${ankle_actuator1_serial}" actuator0_node="${ankle_actuator0_node}" actuator1_node="${ankle_actuator1_node}" />
+    <xacro:include filename="$(find val_description)/common/xacro/joint_names/valkyrie_joint_names.xacro"/>
+    <xacro:macro name="leg" params="prefix j1_serial_number j2_serial_number j3_serial_number j4_serial_number ankle_actuator0_serial ankle_actuator1_serial" >
+    	<xacro:simple_mechanism name="${HipYawJointName}" serial_number="${j1_serial_number}" node="${HipYawNode}"/>
+    	<xacro:simple_mechanism name="${HipRollJointName}" serial_number="${j2_serial_number}" node="${HipRollNode}"/>
+    	<xacro:simple_mechanism name="${HipPitchJointName}" serial_number="${j3_serial_number}" node="${HipPitchNode}"/>
+    	<xacro:simple_mechanism name="${KneePitchJointName}" serial_number="${j4_serial_number}" node="${KneePitchNode}"/>
+    	<xacro:two_active_joint_mechanism mechanism_name="${prefix}Ankle" joint0_name="${AnklePitchJointName}" joint1_name="${AnkleRollJointName}" actuator0_serial="${ankle_actuator0_serial}" actuator1_serial="${ankle_actuator1_serial}" actuator0_node="${AnkleInsideActuatorNode}" actuator1_node="${AnkleOutsideActuatorNode}" />
     </xacro:macro>
 </robot>

File: instance/instances/robots/xacro/limbs/neck.xacro (robot description, xacro)
@@ -1,8 +1,9 @@
 <robot xmlns:xacro="http://ros.org/wiki/xacro" name="neck">
     <xacro:include filename="$(find val_description)/instance/instances/robots/xacro/mechanisms/mechanisms.xacro"/>
+    <xacro:include filename="$(find val_description)/common/xacro/joint_names/valkyrie_joint_names.xacro"/>
     <xacro:macro name="neck" params="j1_serial_number j2_serial_number j3_serial_number j1_node j2_node j3_node" >
-    	<xacro:simple_mechanism name="lower_neck_pitch" serial_number="${j1_serial_number}" node="${j1_node}"/>
-    	<xacro:simple_mechanism name="neck_yaw" serial_number="${j2_serial_number}" node="${j2_node}"/>
-    	<xacro:simple_mechanism name="upper_neck_pitch" serial_number="${j3_serial_number}" node="${j3_node}"/>
+    	<xacro:simple_mechanism name="${LowerNeckPitchJointName}" serial_number="${j1_serial_number}" node="${j1_node}"/>
+    	<xacro:simple_mechanism name="${NeckYawJointName}" serial_number="${j2_serial_number}" node="${j2_node}"/>
+    	<xacro:simple_mechanism name="${UpperNeckPitchJointName}" serial_number="${j3_serial_number}" node="${j3_node}"/>
     </xacro:macro>
 </robot>

File: model/robots/common/xacro/arm/arm.xacro (robot description, xacro)
@@ -1,6 +1,7 @@
 <?xml version="1.0" ?>
 <robot xmlns:xacro="http://www.ros.org/wiki/xacro" name="arm">
-  <xacro:include filename="$(find val_description)/model/robots/common/xacro/arm/joint_names.xacro"/>
-  <xacro:include filename="$(find val_description)/model/robots/common/xacro/arm/actuator_names.xacro"/>
+  <xacro:include filename="$(find val_description)/common/xacro/joint_names/valkyrie_joint_names.xacro"/>
+  <xacro:include filename="$(find val_description)/common/xacro/actuator_names/valkyrie_actuator_names.xacro"/>
+  <xacro:include filename="$(find val_description)/common/xacro/nodes/valkyrie_nodes.xacro"/>
   <xacro:include filename="$(find val_description)/model/robots/common/xacro/arm/joint_axes.xacro"/>
   <xacro:include filename="$(find val_description)/model/robots/common/xacro/arm/link_names.xacro"/>
@@ -162,10 +163,10 @@
   </xacro:macro>
   <xacro:macro name="arm_transmissions" params="prefix">
-    <xacro:simple_transmission_force_controlled_joint jointName="${ShoulderPitchJointName}" actuatorName="${ShoulderPitchActuatorName}"/>
-    <xacro:simple_transmission_force_controlled_joint jointName="${ShoulderRollJointName}" actuatorName="${ShoulderRollActuatorName}"/>
-    <xacro:simple_transmission_force_controlled_joint jointName="${ShoulderYawJointName}" actuatorName="${ShoulderYawActuatorName}"/>
-    <xacro:simple_transmission_force_controlled_joint jointName="${ElbowPitchJointName}" actuatorName="${ElbowPitchActuatorName}"/>
-    <xacro:simple_transmission_force_controlled_joint jointName="${ForearmYawActuatorName}" actuatorName="${ForearmYawActuatorName}"/>
-    <xacro:pushrod_transmission_position_controlled_joints transmissionName="${prefix}WristTransmission" joint1Name="${WristPitchJointName}" joint2Name="${WristRollJointName}" actuator1Name="${WristTopActuatorName}" actuator2Name="${WristBottomActuatorName}" />
+    <xacro:simple_transmission_force_controlled_joint jointName="${ShoulderPitchJointName}" actuatorName="${ShoulderPitchActuatorName}" nodeName="nodeNode"/>
+    <xacro:simple_transmission_force_controlled_joint jointName="${ShoulderRollJointName}" actuatorName="${ShoulderRollActuatorName}" nodeName="nodeNode"/>
+    <xacro:simple_transmission_force_controlled_joint jointName="${ShoulderYawJointName}" actuatorName="${ShoulderYawActuatorName}" nodeName="nodeNode"/>
+    <xacro:simple_transmission_force_controlled_joint jointName="${ElbowPitchJointName}" actuatorName="${ElbowPitchActuatorName}" nodeName="nodeNode"/>
+    <xacro:simple_transmission_force_controlled_joint jointName="${ForearmYawActuatorName}" actuatorName="${ForearmYawActuatorName}" nodeName="nodeNode"/>
+    <xacro:pushrod_transmission_position_controlled_joints transmissionName="${prefix}WristTransmission" joint1Name="${WristPitchJointName}" joint2Name="${WristRollJointName}" actuator1Name="${WristTopActuatorName}" actuator2Name="${WristBottomActuatorName}" actuator1Node="nodeNode" actuator2Node="nodeNode"/>
   </xacro:macro>
 </robot>

File: model/robots/common/xacro/generic_models.xacro (robot description, xacro)
@@ -179,5 +179,5 @@
                        origin_xyz="${origin_xyz}"/>
   </xacro:macro>
-  <xacro:macro name="simple_transmission_force_controlled_joint" params="jointName actuatorName">
+  <xacro:macro name="simple_transmission_force_controlled_joint" params="jointName actuatorName nodeName">
     <transmission name="${jointName}Transmission">
       <type>transmission_interface/SimpleTransmission</type>
@@ -186,8 +186,9 @@
       </joint>
       <actuator name="${actuatorName}">
-      </actuator>
-    </transmission>
-  </xacro:macro>
-  <xacro:macro name="simple_transmission_position_controlled_joint" params="jointName actuatorName">
+        <node name="${nodeName}"/>
+      </actuator>
+    </transmission>
+  </xacro:macro>
+  <xacro:macro name="simple_transmission_position_controlled_joint" params="jointName actuatorName nodeName">
     <transmission name="${jointName}Transmission">
       <type>transmission_interface/SimpleTransmission</type>
@@ -195,8 +196,10 @@
         <hardwareInterface>hardware_interface/PositionJointInterface</hardwareInterface>
       </joint>
-      <actuator name="${actuatorName}"/>
-    </transmission>
-  </xacro:macro>
-  <xacro:macro name="pushrod_transmission_force_controlled_joints" params="transmissionName joint1Name joint2Name actuator1Name actuator2Name">
+      <actuator name="${actuatorName}">
+        <node name="${nodeName}"/>
+    </actuator>
+    </transmission>
+  </xacro:macro>
+  <xacro:macro name="pushrod_transmission_force_controlled_joints" params="transmissionName joint1Name joint2Name actuator1Name actuator2Name actuator1Node actuator2Node">
     <transmission name="${transmissionName}">
       <type>transmission_interface/PushrodTransmission</type>
@@ -208,10 +211,12 @@
       </joint>
        <actuator name="${actuator1Name}">
+        <node name="${actuator1Node}"/>
       </actuator>
       <actuator name="${actuator2Name}">
-      </actuator>
-    </transmission>
-  </xacro:macro>
-  <xacro:macro name="pushrod_transmission_position_controlled_joints" params="transmissionName joint1Name joint2Name actuator1Name actuator2Name">
+        <node name="${actuator2Node}"/>
+      </actuator>
+    </transmission>
+  </xacro:macro>
+  <xacro:macro name="pushrod_transmission_position_controlled_joints" params="transmissionName joint1Name joint2Name actuator1Name actuator2Name actuator1Node actuator2Node">
     <transmission name="${transmissionName}">
       <type>transmission_interface/PushrodTransmission</type>
@@ -223,6 +228,8 @@
       </joint>
        <actuator name="${actuator1Name}">
+        <node name="${actuator1Node}"/>
       </actuator>
       <actuator name="${actuator2Name}">
+        <node name="${actuator2Node}"/>
       </actuator>
     </transmission>

File: model/robots/common/xacro/head/head.xacro (robot description, xacro)
@@ -1,5 +1,6 @@
 <robot xmlns:xacro="http://www.ros.org/wiki/xacro" name="head">
-  <xacro:include filename="$(find val_description)/model/robots/common/xacro/head/joint_names.xacro"/>
-  <xacro:include filename="$(find val_description)/model/robots/common/xacro/head/actuator_names.xacro"/>
+  <xacro:include filename="$(find val_description)/common/xacro/joint_names/valkyrie_joint_names.xacro"/>
+  <xacro:include filename="$(find val_description)/common/xacro/actuator_names/valkyrie_actuator_names.xacro"/>
+  <xacro:include filename="$(find val_description)/common/xacro/nodes/valkyrie_nodes.xacro"/>
   <xacro:include filename="$(find val_description)/model/robots/common/xacro/head/joint_axes.xacro"/>
   <xacro:include filename="$(find val_description)/model/robots/common/xacro/head/link_names.xacro"/>
@@ -74,7 +75,7 @@
     </xacro:macro>
     <xacro:macro name="neck_transmissions">
-      <xacro:simple_transmission_position_controlled_joint jointName="${LowerNeckPitchJointName}" actuatorName="${LowerNeckPitchActuatorName}"/>
-      <xacro:simple_transmission_position_controlled_joint jointName="${NeckYawJointName}" actuatorName="${NeckYawActuatorName}"/>
-      <xacro:simple_transmission_position_controlled_joint jointName="${UpperNeckPitchJointName}" actuatorName="${UpperNeckPitchActuatorName}"/>
+      <xacro:simple_transmission_position_controlled_joint jointName="${LowerNeckPitchJointName}" actuatorName="${LowerNeckPitchActuatorName}" nodeName="nodeNode"/>
+      <xacro:simple_transmission_position_controlled_joint jointName="${NeckYawJointName}" actuatorName="${NeckYawActuatorName}" nodeName="nodeNode"/>
+      <xacro:simple_transmission_position_controlled_joint jointName="${UpperNeckPitchJointName}" actuatorName="${UpperNeckPitchActuatorName}" nodeName="nodeNode"/>
     </xacro:macro>
 </robot>

File: model/robots/common/xacro/head/link_names.xacro (robot description, xacro)
@@ -2,6 +2,6 @@
 <robot xmlns:xacro="http://www.ros.org/wiki/xacro" name="v1/head/link_names">
   <xacro:property name="LowerNeckPitchParentLinkName" value="${head_root_link}" />
-  <xacro:property name="LowerNeckPitchLinkName" value="LowerNeckPitchLink" />
-  <xacro:property name="NeckYawLinkName" value="NeckYawLink" />
-  <xacro:property name="UpperNeckPitchLinkName" value="UpperNeckPitchLink" />
+  <xacro:property name="LowerNeckPitchLinkName" value="lowerNeckPitchLink" />
+  <xacro:property name="NeckYawLinkName" value="neckYawLink" />
+  <xacro:property name="UpperNeckPitchLinkName" value="upperNeckPitchLink" />
 </robot>

File: model/robots/common/xacro/index_finger/index_finger.xacro (robot description, xacro)
@@ -1,5 +1,5 @@
 <?xml version="1.0" ?>
 <robot xmlns:xacro="http://www.ros.org/wiki/xacro" name="v1/index_finger">
-  <xacro:include filename="$(find val_description)/model/robots/common/xacro/index_finger/joint_names.xacro"/>
+  <xacro:include filename="$(find val_description)/common/xacro/joint_names/valkyrie_joint_names.xacro"/>
   <xacro:include filename="$(find val_description)/model/robots/common/xacro/index_finger/joint_axes.xacro"/>
   <xacro:include filename="$(find val_description)/model/robots/common/xacro/index_finger/actuator_names.xacro"/>
