Commit message: Forced to change links/joints to have lowercase first letter so the node names will jive with shared memory.

File: model/robots/common/xacro/middle_finger/middle_finger.xacro (robot description, xacro)
@@ -1,5 +1,5 @@
 <?xml version="1.0" ?>
 <robot xmlns:xacro="http://www.ros.org/wiki/xacro" name="middle_finger">
-  <xacro:include filename="$(find val_description)/model/robots/common/xacro/middle_finger/joint_names.xacro"/>
+  <xacro:include filename="$(find val_description)/common/xacro/joint_names/valkyrie_joint_names.xacro"/>
   <xacro:include filename="$(find val_description)/model/robots/common/xacro/middle_finger/joint_axes.xacro"/>
   <xacro:include filename="$(find val_description)/model/robots/common/xacro/middle_finger/actuator_names.xacro"/>

File: model/robots/common/xacro/pinky_finger/pinky_finger.xacro (robot description, xacro)
@@ -1,5 +1,5 @@
 <?xml version="1.0" ?>
 <robot xmlns:xacro="http://www.ros.org/wiki/xacro" name="pinky_finger">
-  <xacro:include filename="$(find val_description)/model/robots/common/xacro/pinky_finger/joint_names.xacro"/>
+  <xacro:include filename="$(find val_description)/common/xacro/joint_names/valkyrie_joint_names.xacro"/>
   <xacro:include filename="$(find val_description)/model/robots/common/xacro/pinky_finger/joint_axes.xacro"/>
   <xacro:include filename="$(find val_description)/model/robots/common/xacro/pinky_finger/actuator_names.xacro"/>

File: model/robots/common/xacro/thumb/thumb.xacro (robot description, xacro)
@@ -1,5 +1,5 @@
 <?xml version="1.0" ?>
 <robot xmlns:xacro="http://www.ros.org/wiki/xacro" name="thumb">
-  <xacro:include filename="$(find val_description)/model/robots/common/xacro/thumb/joint_names.xacro"/>
+  <xacro:include filename="$(find val_description)/common/xacro/joint_names/valkyrie_joint_names.xacro"/>
   <xacro:include filename="$(find val_description)/model/robots/common/xacro/thumb/joint_axes.xacro"/>
   <xacro:include filename="$(find val_description)/model/robots/common/xacro/thumb/actuator_names.xacro"/>

File: model/robots/common/xacro/valkyrie_base_hw.xacro (robot description, xacro)
@@ -3,26 +3,26 @@
     <xacro:make_waist waist_root_link="${Pelvis_Link_Name}" />
     <xacro:make_head head_root_link="${TorsoRollLinkName}" />
-    <xacro:make_arm prefix="Right" reflect="-1" arm_root_link="${TorsoRollLinkName}" />
-    <xacro:make_thumb prefix="Right" reflect="-1" thumb_root_link="RightPalm"/>
-    <xacro:make_index_finger prefix="Right" reflect="-1" index_finger_root_link="RightPalm"/>
-    <xacro:make_middle_finger prefix="Right" reflect="-1" middle_finger_root_link="RightPalm"/>
-    <xacro:make_pinky_finger prefix="Right" reflect="-1" pinky_finger_root_link="RightPalm"/>
-    <xacro:make_arm prefix="Left" reflect="1" arm_root_link="${TorsoRollLinkName}" />
-    <xacro:make_thumb prefix="Left" reflect="1" thumb_root_link="LeftPalm"/>
-    <xacro:make_index_finger prefix="Left" reflect="1" index_finger_root_link="LeftPalm"/>
-    <xacro:make_middle_finger prefix="Left" reflect="1" middle_finger_root_link="LeftPalm"/>
-    <xacro:make_pinky_finger prefix="Left" reflect="1" pinky_finger_root_link="LeftPalm"/>
-    <xacro:make_leg prefix="Right" reflect="-1" leg_root_link="${Pelvis_Link_Name}" />
-    <xacro:make_leg prefix="Left" reflect="1" leg_root_link="${Pelvis_Link_Name}" />
+    <xacro:make_arm prefix="right" reflect="-1" arm_root_link="${TorsoRollLinkName}" />
+    <xacro:make_thumb prefix="right" reflect="-1" thumb_root_link="rightPalm"/>
+    <xacro:make_index_finger prefix="right" reflect="-1" index_finger_root_link="rightPalm"/>
+    <xacro:make_middle_finger prefix="right" reflect="-1" middle_finger_root_link="rightPalm"/>
+    <xacro:make_pinky_finger prefix="right" reflect="-1" pinky_finger_root_link="rightPalm"/>
+    <xacro:make_arm prefix="left" reflect="1" arm_root_link="${TorsoRollLinkName}" />
+    <xacro:make_thumb prefix="left" reflect="1" thumb_root_link="leftPalm"/>
+    <xacro:make_index_finger prefix="left" reflect="1" index_finger_root_link="leftPalm"/>
+    <xacro:make_middle_finger prefix="left" reflect="1" middle_finger_root_link="leftPalm"/>
+    <xacro:make_pinky_finger prefix="left" reflect="1" pinky_finger_root_link="leftPalm"/>
+    <xacro:make_leg prefix="right" reflect="-1" leg_root_link="${Pelvis_Link_Name}" />
+    <xacro:make_leg prefix="left" reflect="1" leg_root_link="${Pelvis_Link_Name}" />
     <xacro:v1_trunk_sensors/>
-    <xacro:v1_leg_sensors prefix="Left" reflect="1" />
-    <xacro:v1_leg_sensors prefix="Right" reflect="-1" />
+    <xacro:v1_leg_sensors prefix="left" reflect="1" />
+    <xacro:v1_leg_sensors prefix="right" reflect="-1" />
     <xacro:include_multisense_hw />
     <xacro:v1_pelvis_sensors/>
     <xacro:waist_transmissions />
-    <xacro:leg_transmissions prefix="Left"/>
-    <xacro:leg_transmissions prefix="Right"/>
-    <xacro:arm_transmissions prefix="Left"/>
-    <xacro:arm_transmissions prefix="Right"/>
+    <xacro:leg_transmissions prefix="left"/>
+    <xacro:leg_transmissions prefix="right"/>
+    <xacro:arm_transmissions prefix="left"/>
+    <xacro:arm_transmissions prefix="right"/>
     <xacro:neck_transmissions />
 </robot>

File: model/robots/common/xacro/valkyrie_base_sim.xacro (robot description, xacro)
@@ -3,19 +3,19 @@
     <xacro:make_waist waist_root_link="${Pelvis_Link_Name}" />
     <xacro:make_head head_root_link="${TorsoRollLinkName}" />
-    <xacro:make_arm prefix="Right" reflect="-1" arm_root_link="${TorsoRollLinkName}" />
-    <xacro:make_thumb prefix="Right" reflect="-1" thumb_root_link="RightPalm"/>
-    <xacro:make_index_finger prefix="Right" reflect="-1" index_finger_root_link="RightPalm"/>
-    <xacro:make_middle_finger prefix="Right" reflect="-1" middle_finger_root_link="RightPalm"/>
-    <xacro:make_pinky_finger prefix="Right" reflect="-1" pinky_finger_root_link="RightPalm"/>
-    <xacro:make_arm prefix="Left" reflect="1" arm_root_link="${TorsoRollLinkName}" />
-    <xacro:make_thumb prefix="Left" reflect="1" thumb_root_link="LeftPalm"/>
-    <xacro:make_index_finger prefix="Left" reflect="1" index_finger_root_link="LeftPalm"/>
-    <xacro:make_middle_finger prefix="Left" reflect="1" middle_finger_root_link="LeftPalm"/>
-    <xacro:make_pinky_finger prefix="Left" reflect="1" pinky_finger_root_link="LeftPalm"/>
-    <xacro:make_leg prefix="Right" reflect="-1" leg_root_link="${Pelvis_Link_Name}" />
-    <xacro:make_leg prefix="Left" reflect="1" leg_root_link="${Pelvis_Link_Name}" />
+    <xacro:make_arm prefix="right" reflect="-1" arm_root_link="${TorsoRollLinkName}" />
+    <xacro:make_thumb prefix="right" reflect="-1" thumb_root_link="rightPalm"/>
+    <xacro:make_index_finger prefix="right" reflect="-1" index_finger_root_link="rightPalm"/>
+    <xacro:make_middle_finger prefix="right" reflect="-1" middle_finger_root_link="rightPalm"/>
+    <xacro:make_pinky_finger prefix="right" reflect="-1" pinky_finger_root_link="rightPalm"/>
+    <xacro:make_arm prefix="left" reflect="1" arm_root_link="${TorsoRollLinkName}" />
+    <xacro:make_thumb prefix="left" reflect="1" thumb_root_link="leftPalm"/>
+    <xacro:make_index_finger prefix="left" reflect="1" index_finger_root_link="leftPalm"/>
+    <xacro:make_middle_finger prefix="left" reflect="1" middle_finger_root_link="leftPalm"/>
+    <xacro:make_pinky_finger prefix="left" reflect="1" pinky_finger_root_link="leftPalm"/>
+    <xacro:make_leg prefix="right" reflect="-1" leg_root_link="${Pelvis_Link_Name}" />
+    <xacro:make_leg prefix="left" reflect="1" leg_root_link="${Pelvis_Link_Name}" />
     <xacro:v1_pelvis_sensors />
-    <xacro:v1_leg_sensors prefix="Left" reflect="1" />
-    <xacro:v1_leg_sensors prefix="Right" reflect="-1" />
+    <xacro:v1_leg_sensors prefix="left" reflect="1" />
+    <xacro:v1_leg_sensors prefix="right" reflect="-1" />
     <xacro:include_multisense_sim />
     <xacro:v1_trunk_sensors/>

File: model/robots/common/xacro/waist/waist.xacro (robot description, xacro)
@@ -1,5 +1,6 @@
 <robot xmlns:xacro="http://www.ros.org/wiki/xacro" name="waist">
-  <xacro:include filename="$(find val_description)/model/robots/common/xacro/waist/joint_names.xacro"/>
-  <xacro:include filename="$(find val_description)/model/robots/common/xacro/waist/actuator_names.xacro"/>
+  <xacro:include filename="$(find val_description)/common/xacro/joint_names/valkyrie_joint_names.xacro"/>
+  <xacro:include filename="$(find val_description)/common/xacro/actuator_names/valkyrie_actuator_names.xacro"/>
+  <xacro:include filename="$(find val_description)/common/xacro/nodes/valkyrie_nodes.xacro"/>
   <xacro:include filename="$(find val_description)/model/robots/common/xacro/waist/joint_axes.xacro"/>
   <xacro:include filename="$(find val_description)/model/robots/common/xacro/waist/joint_axes.xacro"/>
@@ -97,6 +98,6 @@
    </xacro:macro>
    <xacro:macro name="waist_transmissions">
-    <xacro:simple_transmission_force_controlled_joint jointName="${TorsoYawJointName}" actuatorName="${TorsoYawActuatorName}"/>
-    <xacro:pushrod_transmission_position_controlled_joints transmissionName="WaistTransmission" joint1Name="${TorsoPitchJointName}" joint2Name="${TorsoRollJointName}" actuator1Name="${WaistLeftActuatorName}" actuator2Name="${WaistRightActuatorName}" />
+    <xacro:simple_transmission_force_controlled_joint jointName="${TorsoYawJointName}" actuatorName="${TorsoYawActuatorName}" nodeName="nodeNode"/>
+    <xacro:pushrod_transmission_position_controlled_joints transmissionName="WaistTransmission" joint1Name="${TorsoPitchJointName}" joint2Name="${TorsoRollJointName}" actuator1Name="${WaistLeftActuatorName}" actuator2Name="${WaistRightActuatorName}" actuator1Node="nodeNode" actuator2Node="nodeNode"/>
    </xacro:macro>
 </robot>

File: model/robots/valkyrie_A/xacro/leg/leg.xacro (robot description, xacro)
@@ -1,6 +1,7 @@
 <?xml version="1.0" ?>
 <robot xmlns:xacro="http://www.ros.org/wiki/xacro" name="leg">
-  <xacro:include filename="$(find val_description)/model/robots/valkyrie_A/xacro/leg/joint_names.xacro"/>
-  <xacro:include filename="$(find val_description)/model/robots/valkyrie_A/xacro/leg/actuator_names.xacro"/>
+  <xacro:include filename="$(find val_description)/common/xacro/joint_names/valkyrie_joint_names.xacro"/>
+  <xacro:include filename="$(find val_description)/common/xacro/actuator_names/valkyrie_actuator_names.xacro"/>
+  <xacro:include filename="$(find val_description)/common/xacro/nodes/valkyrie_nodes.xacro"/>
   <xacro:include filename="$(find val_description)/model/robots/valkyrie_A/xacro/leg/joint_axes.xacro"/>
   <xacro:include filename="$(find val_description)/model/robots/valkyrie_A/xacro/leg/link_names.xacro"/>
@@ -148,9 +149,9 @@
   </xacro:macro>
   <xacro:macro name="leg_transmissions" params="prefix">
-    <xacro:simple_transmission_force_controlled_joint jointName="${HipYawJointName}" actuatorName="${HipYawActuatorName}"/>
-    <xacro:simple_transmission_force_controlled_joint jointName="${HipRollJointName}" actuatorName="${HipRollActuatorName}"/>
-    <xacro:simple_transmission_force_controlled_joint jointName="${HipPitchJointName}" actuatorName="${HipPitchActuatorName}"/>
-    <xacro:simple_transmission_force_controlled_joint jointName="${KneePitchJointName}" actuatorName="${KneePitchActuatorName}"/>
-    <xacro:pushrod_transmission_force_controlled_joints transmissionName="${prefix}AnkleTransmission" joint1Name="${AnklePitchJointName}" joint2Name="${AnkleRollJointName}" actuator1Name="${AnkleInsideActuatorName}" actuator2Name="${AnkleOutsideActuatorName}" />
+    <xacro:simple_transmission_force_controlled_joint jointName="${HipYawJointName}" actuatorName="${HipYawActuatorName}" nodeName="nodeNode"/>
+    <xacro:simple_transmission_force_controlled_joint jointName="${HipRollJointName}" actuatorName="${HipRollActuatorName}" nodeName="nodeNode"/>
+    <xacro:simple_transmission_force_controlled_joint jointName="${HipPitchJointName}" actuatorName="${HipPitchActuatorName}" nodeName="nodeNode"/>
+    <xacro:simple_transmission_force_controlled_joint jointName="${KneePitchJointName}" actuatorName="${KneePitchActuatorName}" nodeName="nodeNode"/>
+    <xacro:pushrod_transmission_force_controlled_joints transmissionName="${prefix}AnkleTransmission" joint1Name="${AnklePitchJointName}" joint2Name="${AnkleRollJointName}" actuator1Name="${AnkleInsideActuatorName}" actuator2Name="${AnkleOutsideActuatorName}" actuator1Node="nodeNode" actuator2Node="nodeNode"/>
   </xacro:macro>
 </robot>

File: model/robots/valkyrie_B/xacro/leg/leg.xacro (robot description, xacro)
@@ -1,6 +1,7 @@
 <?xml version="1.0" ?>
 <robot xmlns:xacro="http://www.ros.org/wiki/xacro" name="leg">
-  <xacro:include filename="$(find val_description)/model/robots/valkyrie_A/xacro/leg/joint_names.xacro"/>
-  <xacro:include filename="$(find val_description)/model/robots/valkyrie_A/xacro/leg/actuator_names.xacro"/>
+    <xacro:include filename="$(find val_description)/common/xacro/joint_names/valkyrie_joint_names.xacro"/>
+  <xacro:include filename="$(find val_description)/common/xacro/actuator_names/valkyrie_actuator_names.xacro"/>
+  <xacro:include filename="$(find val_description)/common/xacro/nodes/valkyrie_nodes.xacro"/>
   <xacro:include filename="$(find val_description)/model/robots/valkyrie_A/xacro/leg/joint_axes.xacro"/>
   <xacro:include filename="$(find val_description)/model/robots/valkyrie_A/xacro/leg/link_names.xacro"/>
@@ -148,9 +149,9 @@
   </xacro:macro>
   <xacro:macro name="leg_transmissions" params="prefix">
-    <xacro:simple_transmission_force_controlled_joint jointName="${HipYawJointName}" actuatorName="${HipYawActuatorName}"/>
-    <xacro:simple_transmission_force_controlled_joint jointName="${HipRollJointName}" actuatorName="${HipRollActuatorName}"/>
-    <xacro:simple_transmission_force_controlled_joint jointName="${HipPitchJointName}" actuatorName="${HipPitchActuatorName}"/>
-    <xacro:simple_transmission_force_controlled_joint jointName="${KneePitchJointName}" actuatorName="${KneePitchActuatorName}"/>
-    <xacro:pushrod_transmission_force_controlled_joints transmissionName="${prefix}AnkleTransmission" joint1Name="${AnklePitchJointName}" joint2Name="${AnkleRollJointName}" actuator1Name="${AnkleInsideActuatorName}" actuator2Name="${AnkleOutsideActuatorName}" />
+    <xacro:simple_transmission_force_controlled_joint jointName="${HipYawJointName}" actuatorName="${HipYawActuatorName}" nodeName="nodeNode"/>
+    <xacro:simple_transmission_force_controlled_joint jointName="${HipRollJointName}" actuatorName="${HipRollActuatorName}" nodeName="nodeNode"/>
+    <xacro:simple_transmission_force_controlled_joint jointName="${HipPitchJointName}" actuatorName="${HipPitchActuatorName}" nodeName="nodeNode"/>
+    <xacro:simple_transmission_force_controlled_joint jointName="${KneePitchJointName}" actuatorName="${KneePitchActuatorName}" nodeName="nodeNode"/>
+    <xacro:pushrod_transmission_force_controlled_joints transmissionName="${prefix}AnkleTransmission" joint1Name="${AnklePitchJointName}" joint2Name="${AnkleRollJointName}" actuator1Name="${AnkleInsideActuatorName}" actuator2Name="${AnkleOutsideActuatorName}" actuator1Node="nodeNode" actuator2Node="nodeNode"/>
   </xacro:macro>
 </robot>
