Commit message: Fixed name of meshes and textures to comply with new naming.

File: common/xacro/nodes/valkyrie_nodes.xacro (robot description, xacro)
@@ -4,6 +4,6 @@
 	<xacro:property name="HipPitchNode" value="/${prefix}_leg/j3" />
 	<xacro:property name="KneePitchNode" value="/${prefix}_leg/j4" />
-	<xacro:property name="AnkleInsideActuatorNode" value="/${prefix}_leg/ankle/actuator0" />
-	<xacro:property name="AnkleOutsideActuatorNode" value="/${prefix}_leg/ankle/actuator1" />
+	<xacro:property name="AnkleInsideActuatorNode" value="/${prefix}_leg/ankle/left_actuator" />
+	<xacro:property name="AnkleOutsideActuatorNode" value="/${prefix}_leg/ankle/right_actuator" />
 	<xacro:property name="ShoulderPitchNode" value="/${prefix}_arm/j1" />
 	<xacro:property name="ShoulderRollNode" value="/${prefix}_arm/j2" />
@@ -13,10 +13,10 @@
 	<xacro:property name="WristTopActuatorNode" value="/${prefix}_arm/wrist/top_actautor" />
 	<xacro:property name="WristBottomActuatorNode" value="/${prefix}_arm/wrist/bottom_actuator" />
-	<xacro:property name="neckJ1Node" value="/neck/j1" />
-	<xacro:property name="neckJ2Node" value="/neck/j2" />
-	<xacro:property name="neckJ3Node" value="/neck/j3" />
-	<xacro:property name="trunkNode" value="/trunk/j1" />
-	<xacro:property name="waistActuator0Node" value="/trunk/waist/actuator0" />
-	<xacro:property name="waistActuator1Node" value="/trunk/waist/actuator1" />
+	<xacro:property name="LowerNeckPitchNode" value="/neck/j1" />
+	<xacro:property name="NeckYawNode" value="/neck/j2" />
+	<xacro:property name="UpperNeckPitchNode" value="/neck/j3" />
+	<xacro:property name="TrunkYawNode" value="/trunk/j1" />
+	<xacro:property name="WaistLeftActuatorNode" value="/trunk/waist/left_actuator" />
+	<xacro:property name="WaistRightActuatorNode" value="/trunk/waist/right_actuator" />
 	<xacro:property name="pelvis_imu1_node" value="/pelvis/sensors/imu1" />
 	<xacro:property name="pelvis_imu2_node" value="/pelvis/sensors/imu2" />

File: instance/instances/robots/xacro/common/valkyrie_full_template.xacro (robot description, xacro)
@@ -15,6 +15,6 @@
 		<xacro:arm prefix="left" j1_serial_number="${leftArmJ1SerialNumber}" j2_serial_number="${leftArmJ2SerialNumber}" j3_serial_number="${leftArmJ3SerialNumber}" j4_serial_number="${leftArmJ4SerialNumber}" j5_serial_number="${leftArmJ5SerialNumber}" wrist_actuator0_serial="${leftAnkleActuator0SerialNumber}" wrist_actuator1_serial="${leftAnkleActuator1SerialNumber}" />
 		<xacro:arm prefix="right" j1_serial_number="${rightArmJ1SerialNumber}" j2_serial_number="${rightArmJ2SerialNumber}" j3_serial_number="${rightArmJ3SerialNumber}" j4_serial_number="${rightArmJ4SerialNumber}" j5_serial_number="${rightArmJ5SerialNumber}" wrist_actuator0_serial="${rightAnkleActuator0SerialNumber}" wrist_actuator1_serial="${rightAnkleActuator1SerialNumber}" />
-		<xacro:neck j1_serial_number="${neckJ1SerialNumber}" j2_serial_number="${neckJ1SerialNumber}" j3_serial_number="${neckJ1SerialNumber}" j1_node="${neckJ1Node}" j2_node="${neckJ2Node}" j3_node="${neckJ3Node}" />
-		<xacro:waist j1_serial_number="${trunkSerialNumber}" waist_actuator0_serial="${waistActuator0SerialNumber}" waist_actuator1_serial="${waistActuator1SerialNumber}" j1_node="${trunkNode}" waist_actuator0_node="${waistActuator0Node}" waist_actuator1_node="${waistActuator1Node}" />
+		<xacro:neck j1_serial_number="${neckJ1SerialNumber}" j2_serial_number="${neckJ1SerialNumber}" j3_serial_number="${neckJ1SerialNumber}" />
+		<xacro:waist j1_serial_number="${trunkSerialNumber}" waist_actuator0_serial="${waistActuator0SerialNumber}" waist_actuator1_serial="${waistActuator1SerialNumber}"/>
 	</Mechanisms>
 	<Devices>

File: instance/instances/robots/xacro/limbs/neck.xacro (robot description, xacro)
@@ -2,8 +2,8 @@
     <xacro:include filename="$(find val_description)/instance/instances/robots/xacro/mechanisms/mechanisms.xacro"/>
     <xacro:include filename="$(find val_description)/common/xacro/joint_names/valkyrie_joint_names.xacro"/>
-    <xacro:macro name="neck" params="j1_serial_number j2_serial_number j3_serial_number j1_node j2_node j3_node" >
-    	<xacro:simple_mechanism name="${LowerNeckPitchJointName}" serial_number="${j1_serial_number}" node="${j1_node}"/>
-    	<xacro:simple_mechanism name="${NeckYawJointName}" serial_number="${j2_serial_number}" node="${j2_node}"/>
-    	<xacro:simple_mechanism name="${UpperNeckPitchJointName}" serial_number="${j3_serial_number}" node="${j3_node}"/>
+    <xacro:macro name="neck" params="j1_serial_number j2_serial_number j3_serial_number" >
+    	<xacro:simple_mechanism name="${LowerNeckPitchJointName}" serial_number="${j1_serial_number}" node="${LowerNeckPitchNode}"/>
+    	<xacro:simple_mechanism name="${NeckYawJointName}" serial_number="${j2_serial_number}" node="${NeckYawNode}"/>
+    	<xacro:simple_mechanism name="${UpperNeckPitchJointName}" serial_number="${j3_serial_number}" node="${UpperNeckPitchNode}"/>
     </xacro:macro>
 </robot>

File: instance/instances/robots/xacro/limbs/waist.xacro (robot description, xacro)
@@ -1,7 +1,7 @@
 <robot xmlns:xacro="http://ros.org/wiki/xacro" name="waist">
     <xacro:include filename="$(find val_description)/instance/instances/robots/xacro/mechanisms/mechanisms.xacro"/>
-    <xacro:macro name="waist" params="j1_serial_number waist_actuator0_serial waist_actuator1_serial j1_node waist_actuator0_node waist_actuator1_node" >
-    	<xacro:simple_mechanism name="torso_yaw" serial_number="${j1_serial_number}" node="${j1_node}"/>
-    	<xacro:two_active_joint_mechanism mechanism_name="waist" joint0_name="pitch" joint1_name="roll" actuator0_serial="${waist_actuator0_serial}" actuator1_serial="${waist_actuator1_serial}" actuator0_node="${waist_actuator0_node}" actuator1_node="${waist_actuator1_node}" />
+    <xacro:macro name="waist" params="j1_serial_number waist_actuator0_serial waist_actuator1_serial" >
+    	<xacro:simple_mechanism name="torso_yaw" serial_number="${j1_serial_number}" node="${TrunkYawNode}"/>
+    	<xacro:two_active_joint_mechanism mechanism_name="waist" joint0_name="pitch" joint1_name="roll" actuator0_serial="${waist_actuator0_serial}" actuator1_serial="${waist_actuator1_serial}" actuator0_node="${WaistLeftActuatorNode}" actuator1_node="${WaistRightActuatorNode}" />
     </xacro:macro>
 </robot>

File: model/robots/common/xacro/arm/arm.xacro (robot description, xacro)
@@ -163,10 +163,10 @@
   </xacro:macro>
   <xacro:macro name="arm_transmissions" params="prefix">
-    <xacro:simple_transmission_force_controlled_joint jointName="${ShoulderPitchJointName}" actuatorName="${ShoulderPitchActuatorName}" nodeName="nodeNode"/>
-    <xacro:simple_transmission_force_controlled_joint jointName="${ShoulderRollJointName}" actuatorName="${ShoulderRollActuatorName}" nodeName="nodeNode"/>
-    <xacro:simple_transmission_force_controlled_joint jointName="${ShoulderYawJointName}" actuatorName="${ShoulderYawActuatorName}" nodeName="nodeNode"/>
-    <xacro:simple_transmission_force_controlled_joint jointName="${ElbowPitchJointName}" actuatorName="${ElbowPitchActuatorName}" nodeName="nodeNode"/>
-    <xacro:simple_transmission_force_controlled_joint jointName="${ForearmYawActuatorName}" actuatorName="${ForearmYawActuatorName}" nodeName="nodeNode"/>
-    <xacro:pushrod_transmission_position_controlled_joints transmissionName="${prefix}WristTransmission" joint1Name="${WristPitchJointName}" joint2Name="${WristRollJointName}" actuator1Name="${WristTopActuatorName}" actuator2Name="${WristBottomActuatorName}" actuator1Node="nodeNode" actuator2Node="nodeNode"/>
+    <xacro:simple_transmission_force_controlled_joint jointName="${ShoulderPitchJointName}" actuatorName="${ShoulderPitchActuatorName}" nodeName="${ShoulderPitchNode}"/>
+    <xacro:simple_transmission_force_controlled_joint jointName="${ShoulderRollJointName}" actuatorName="${ShoulderRollActuatorName}" nodeName="${ShoulderRollNode}"/>
+    <xacro:simple_transmission_force_controlled_joint jointName="${ShoulderYawJointName}" actuatorName="${ShoulderYawActuatorName}" nodeName="${ShoulderYawNode}"/>
+    <xacro:simple_transmission_force_controlled_joint jointName="${ElbowPitchJointName}" actuatorName="${ElbowPitchActuatorName}" nodeName="${ElbowPitchNode}"/>
+    <xacro:simple_transmission_force_controlled_joint jointName="${ForearmYawActuatorName}" actuatorName="${ForearmYawActuatorName}" nodeName="${ForearmYawNode}"/>
+    <xacro:pushrod_transmission_position_controlled_joints transmissionName="${prefix}WristTransmission" joint1Name="${WristPitchJointName}" joint2Name="${WristRollJointName}" actuator1Name="${WristTopActuatorName}" actuator2Name="${WristBottomActuatorName}" actuator1Node="${WristTopActuatorNode}" actuator2Node="${WristBottomActuatorNode}"/>
   </xacro:macro>
 </robot>

File: model/robots/common/xacro/head/head.xacro (robot description, xacro)
@@ -75,7 +75,7 @@
     </xacro:macro>
     <xacro:macro name="neck_transmissions">
-      <xacro:simple_transmission_position_controlled_joint jointName="${LowerNeckPitchJointName}" actuatorName="${LowerNeckPitchActuatorName}" nodeName="nodeNode"/>
-      <xacro:simple_transmission_position_controlled_joint jointName="${NeckYawJointName}" actuatorName="${NeckYawActuatorName}" nodeName="nodeNode"/>
-      <xacro:simple_transmission_position_controlled_joint jointName="${UpperNeckPitchJointName}" actuatorName="${UpperNeckPitchActuatorName}" nodeName="nodeNode"/>
+      <xacro:simple_transmission_position_controlled_joint jointName="${LowerNeckPitchJointName}" actuatorName="${LowerNeckPitchActuatorName}" nodeName="${LowerNeckPitchNode}"/>
+      <xacro:simple_transmission_position_controlled_joint jointName="${NeckYawJointName}" actuatorName="${NeckYawActuatorName}" nodeName="${NeckYawNode}"/>
+      <xacro:simple_transmission_position_controlled_joint jointName="${UpperNeckPitchJointName}" actuatorName="${UpperNeckPitchActuatorName}" nodeName="${UpperNeckPitchNode}"/>
     </xacro:macro>
 </robot>

File: model/robots/common/xacro/waist/waist.xacro (robot description, xacro)
@@ -98,6 +98,6 @@
    </xacro:macro>
    <xacro:macro name="waist_transmissions">
-    <xacro:simple_transmission_force_controlled_joint jointName="${TorsoYawJointName}" actuatorName="${TorsoYawActuatorName}" nodeName="nodeNode"/>
-    <xacro:pushrod_transmission_position_controlled_joints transmissionName="WaistTransmission" joint1Name="${TorsoPitchJointName}" joint2Name="${TorsoRollJointName}" actuator1Name="${WaistLeftActuatorName}" actuator2Name="${WaistRightActuatorName}" actuator1Node="nodeNode" actuator2Node="nodeNode"/>
+    <xacro:simple_transmission_force_controlled_joint jointName="${TorsoYawJointName}" actuatorName="${TorsoYawActuatorName}" nodeName="${TrunkYawNode}"/>
+    <xacro:pushrod_transmission_position_controlled_joints transmissionName="WaistTransmission" joint1Name="${TorsoPitchJointName}" joint2Name="${TorsoRollJointName}" actuator1Name="${WaistLeftActuatorName}" actuator2Name="${WaistRightActuatorName}" actuator1Node="${WaistLeftActuatorNode}" actuator2Node="${WaistRightActuatorNode}"/>
    </xacro:macro>
 </robot>

File: model/robots/valkyrie_A/xacro/leg/leg.xacro (robot description, xacro)
@@ -149,9 +149,9 @@
   </xacro:macro>
   <xacro:macro name="leg_transmissions" params="prefix">
-    <xacro:simple_transmission_force_controlled_joint jointName="${HipYawJointName}" actuatorName="${HipYawActuatorName}" nodeName="nodeNode"/>
-    <xacro:simple_transmission_force_controlled_joint jointName="${HipRollJointName}" actuatorName="${HipRollActuatorName}" nodeName="nodeNode"/>
-    <xacro:simple_transmission_force_controlled_joint jointName="${HipPitchJointName}" actuatorName="${HipPitchActuatorName}" nodeName="nodeNode"/>
-    <xacro:simple_transmission_force_controlled_joint jointName="${KneePitchJointName}" actuatorName="${KneePitchActuatorName}" nodeName="nodeNode"/>
-    <xacro:pushrod_transmission_force_controlled_joints transmissionName="${prefix}AnkleTransmission" joint1Name="${AnklePitchJointName}" joint2Name="${AnkleRollJointName}" actuator1Name="${AnkleInsideActuatorName}" actuator2Name="${AnkleOutsideActuatorName}" actuator1Node="nodeNode" actuator2Node="nodeNode"/>
+    <xacro:simple_transmission_force_controlled_joint jointName="${HipYawJointName}" actuatorName="${HipYawActuatorName}" nodeName="${HipYawNode}"/>
+    <xacro:simple_transmission_force_controlled_joint jointName="${HipRollJointName}" actuatorName="${HipRollActuatorName}" nodeName="${HipRollNode}"/>
+    <xacro:simple_transmission_force_controlled_joint jointName="${HipPitchJointName}" actuatorName="${HipPitchActuatorName}" nodeName="${HipPitchNode}"/>
+    <xacro:simple_transmission_force_controlled_joint jointName="${KneePitchJointName}" actuatorName="${KneePitchActuatorName}" nodeName="${KneePitchNode}"/>
+    <xacro:pushrod_transmission_force_controlled_joints transmissionName="${prefix}AnkleTransmission" joint1Name="${AnklePitchJointName}" joint2Name="${AnkleRollJointName}" actuator1Name="${AnkleInsideActuatorName}" actuator2Name="${AnkleOutsideActuatorName}" actuator1Node="${AnkleInsideActuatorNode}" actuator2Node="${AnkleOutsideActuatorNode}"/>
   </xacro:macro>
 </robot>

File: model/robots/valkyrie_B/xacro/leg/leg.xacro (robot description, xacro)
@@ -149,9 +149,9 @@
   </xacro:macro>
   <xacro:macro name="leg_transmissions" params="prefix">
-    <xacro:simple_transmission_force_controlled_joint jointName="${HipYawJointName}" actuatorName="${HipYawActuatorName}" nodeName="nodeNode"/>
-    <xacro:simple_transmission_force_controlled_joint jointName="${HipRollJointName}" actuatorName="${HipRollActuatorName}" nodeName="nodeNode"/>
-    <xacro:simple_transmission_force_controlled_joint jointName="${HipPitchJointName}" actuatorName="${HipPitchActuatorName}" nodeName="nodeNode"/>
-    <xacro:simple_transmission_force_controlled_joint jointName="${KneePitchJointName}" actuatorName="${KneePitchActuatorName}" nodeName="nodeNode"/>
-    <xacro:pushrod_transmission_force_controlled_joints transmissionName="${prefix}AnkleTransmission" joint1Name="${AnklePitchJointName}" joint2Name="${AnkleRollJointName}" actuator1Name="${AnkleInsideActuatorName}" actuator2Name="${AnkleOutsideActuatorName}" actuator1Node="nodeNode" actuator2Node="nodeNode"/>
+    <xacro:simple_transmission_force_controlled_joint jointName="${HipYawJointName}" actuatorName="${HipYawActuatorName}" nodeName="${HipYawNode}"/>
+    <xacro:simple_transmission_force_controlled_joint jointName="${HipRollJointName}" actuatorName="${HipRollActuatorName}" nodeName="${HipRollNode}"/>
+    <xacro:simple_transmission_force_controlled_joint jointName="${HipPitchJointName}" actuatorName="${HipPitchActuatorName}" nodeName="${HipPitchNode}"/>
+    <xacro:simple_transmission_force_controlled_joint jointName="${KneePitchJointName}" actuatorName="${KneePitchActuatorName}" nodeName="${KneePitchNode}"/>
+    <xacro:pushrod_transmission_force_controlled_joints transmissionName="${prefix}AnkleTransmission" joint1Name="${AnklePitchJointName}" joint2Name="${AnkleRollJointName}" actuator1Name="${AnkleInsideActuatorName}" actuator2Name="${AnkleOutsideActuatorName}" actuator1Node="${AnkleInsideActuatorNode}" actuator2Node="${AnkleOutsideActuatorNode}"/>
   </xacro:macro>
 </robot>

Commit message: unit C actuator updates

File: common/xacro/nodes/valkyrie_nodes.xacro (robot description, xacro)
@@ -4,6 +4,6 @@
 	<xacro:property name="HipPitchNode" value="/${prefix}_leg/j3" />
 	<xacro:property name="KneePitchNode" value="/${prefix}_leg/j4" />
-	<xacro:property name="AnkleInsideActuatorNode" value="/${prefix}_leg/ankle/left_actuator" />
-	<xacro:property name="AnkleOutsideActuatorNode" value="/${prefix}_leg/ankle/right_actuator" />
+	<xacro:property name="AnkleInsideActuatorNode" value="/${prefix}_leg/left_actuator" />
+	<xacro:property name="AnkleOutsideActuatorNode" value="/${prefix}_leg/right_actuator" />
 	<xacro:property name="ShoulderPitchNode" value="/${prefix}_arm/j1" />
 	<xacro:property name="ShoulderRollNode" value="/${prefix}_arm/j2" />

File: instance/instances/robots/xacro/serial_numbers/valkyrie_C_serials.xacro (robot description, xacro)
@@ -1,4 +1,4 @@
 <robot xmlns:xacro="http://ros.org/wiki/xacro" name="valkyrie_C_serials">
-	<xacro:property name="leftLegJ1SerialNumber" value="v_a_015" />
+	<xacro:property name="leftLegJ1SerialNumber" value="UNKNOWN" />
 	<xacro:property name="leftLegJ2SerialNumber" value="UNKNOWN" />
 	<xacro:property name="leftLegJ3SerialNumber" value="UNKNOWN" />
@@ -6,21 +6,21 @@
 	<xacro:property name="leftAnkleLeftActuatorSerialNumber" value="UNKNOWN" />
 	<xacro:property name="leftAnkleRightActuatorSerialNumber" value="UNKNOWN" />
-	<xacro:property name="rightLegJ1SerialNumber" value="v_a_014" />
+	<xacro:property name="rightLegJ1SerialNumber" value="v_b_011" />
 	<xacro:property name="rightLegJ2SerialNumber" value="UNKNOWN" />
 	<xacro:property name="rightLegJ3SerialNumber" value="UNKNOWN" />
 	<xacro:property name="rightLegJ4SerialNumber" value="UNKNOWN" />
+	<xacro:property name="rightAnkleRightActuatorSerialNumber" value="UNKNOWN" />
 	<xacro:property name="rightAnkleLeftActuatorSerialNumber" value="UNKNOWN" />
-	<xacro:property name="rightAnkleRightActuatorSerialNumber" value="UNKNOWN" />
-	<xacro:property name="leftArmJ1SerialNumber" value="v_a_013" />
-	<xacro:property name="leftArmJ2SerialNumber" value="v_b_009" />
-	<xacro:property name="leftArmJ3SerialNumber" value="v_f_012" />
-	<xacro:property name="leftArmJ4SerialNumber" value="v_f_011" />
+	<xacro:property name="leftArmJ1SerialNumber" value="UNKNOWN" />
+	<xacro:property name="leftArmJ2SerialNumber" value="UNKNOWN" />
+	<xacro:property name="leftArmJ3SerialNumber" value="UNKNOWN" />
+	<xacro:property name="leftArmJ4SerialNumber" value="UNKNOWN" />
 	<xacro:property name="leftArmJ5SerialNumber" value="UNKNOWN" />
 	<xacro:property name="leftWristTopActuatorSerialNumber" value="UNKNOWN" />
 	<xacro:property name="leftWristBottomActuatorSerialNumber" value="UNKNOWN" />
-	<xacro:property name="rightArmJ1SerialNumber" value="v_a_012" />
-	<xacro:property name="rightArmJ2SerialNumber" value="v_b_012" />
-	<xacro:property name="rightArmJ3SerialNumber" value="v_f_013" />
-	<xacro:property name="rightArmJ4SerialNumber" value="v_f_014" />
+	<xacro:property name="rightArmJ1SerialNumber" value="UNKNOWN" />
+	<xacro:property name="rightArmJ2SerialNumber" value="UNKNOWN" />
+	<xacro:property name="rightArmJ3SerialNumber" value="UNKNOWN" />
+	<xacro:property name="rightArmJ4SerialNumber" value="UNKNOWN" />
 	<xacro:property name="rightArmJ5SerialNumber" value="UNKNOWN" />
 	<xacro:property name="rightWristTopActuatorSerialNumber" value="UNKNOWN" />
@@ -29,7 +29,7 @@
 	<xacro:property name="neckJ2SerialNumber" value="UNKNOWN" />
 	<xacro:property name="neckJ3SerialNumber" value="UNKNOWN" />
-	<xacro:property name="trunkSerialNumber" value="v_a_011" />
-	<xacro:property name="waistRightActuatorSerialNumber" value="v_e_014" />
-	<xacro:property name="waistLeftActuatorSerialNumber" value="v_e_013" />
+	<xacro:property name="trunkSerialNumber" value="UNKNOWN" />
+	<xacro:property name="waistRightActuatorSerialNumber" value="UNKNOWN" />
+	<xacro:property name="waistLeftActuatorSerialNumber" value="UNKNOWN" />
 	<xacro:property name="pelvis_imu1_serial" value="UNKNOWN" />
 	<xacro:property name="pelvis_imu2_serial" value="UNKNOWN" />
