Commit message: Valkyrie B every joint servo'd in torque control mode

File: common/xacro/nodes/valkyrie_nodes.xacro (robot description, xacro)
@@ -1,4 +1,4 @@
 <robot xmlns:xacro="http://ros.org/wiki/xacro" name="valkyrie_nodes">
-	<xacro:property name="HipYawNode" value="/${prefix}_leg/j1" />
+	<xacro:property name="HipYawNode" value="/pelvis/${prefix}_leg_j1" />
 	<xacro:property name="HipRollNode" value="/${prefix}_leg/j2" />
 	<xacro:property name="HipPitchNode" value="/${prefix}_leg/j3" />
@@ -6,5 +6,5 @@
 	<xacro:property name="AnkleInsideActuatorNode" value="/${prefix}_leg/left_actuator" />
 	<xacro:property name="AnkleOutsideActuatorNode" value="/${prefix}_leg/right_actuator" />
-	<xacro:property name="ShoulderPitchNode" value="/${prefix}_arm/j1" />
+	<xacro:property name="ShoulderPitchNode" value="/trunk/${prefix}_arm_j1" />
 	<xacro:property name="ShoulderRollNode" value="/${prefix}_arm/j2" />
 	<xacro:property name="ShoulderYawNode" value="/${prefix}_arm/j3" />
@@ -16,7 +16,7 @@
 	<xacro:property name="NeckYawNode" value="/neck/j2" />
 	<xacro:property name="UpperNeckPitchNode" value="/neck/j3" />
-	<xacro:property name="TrunkYawNode" value="/trunk/j1" />
-	<xacro:property name="WaistLeftActuatorNode" value="/trunk/waist/left_actuator" />
-	<xacro:property name="WaistRightActuatorNode" value="/trunk/waist/right_actuator" />
+	<xacro:property name="TrunkYawNode" value="/pelvis/waist" />
+	<xacro:property name="WaistLeftActuatorNode" value="/trunk/left_actuator" />
+	<xacro:property name="WaistRightActuatorNode" value="/trunk/right_actuator" />
 	<xacro:property name="pelvis_imu1_node" value="/pelvis/sensors/imu1" />
 	<xacro:property name="pelvis_imu2_node" value="/pelvis/sensors/imu2" />

File: instance/instances/robots/xacro/limbs/arm.xacro (robot description, xacro)
@@ -3,5 +3,5 @@
     <xacro:include filename="$(find val_description)/common/xacro/joint_names/valkyrie_joint_names.xacro"/>
     <xacro:macro name="arm" params="prefix j1_serial_number j2_serial_number j3_serial_number j4_serial_number j5_serial_number wrist_actuator0_serial wrist_actuator1_serial" >
-    	<xacro:simple_mechanism name="${ShoulderPitchJointName}" serial_number="${j1_serial_number}" node="${ShoulderYawNode}"/>
+    	<xacro:simple_mechanism name="${ShoulderPitchJointName}" serial_number="${j1_serial_number}" node="${ShoulderPitchNode}"/>
     	<xacro:simple_mechanism name="${ShoulderRollJointName}" serial_number="${j2_serial_number}" node="${ShoulderRollNode}"/>
     	<xacro:simple_mechanism name="${ShoulderYawJointName}" serial_number="${j3_serial_number}" node="${ShoulderYawNode}"/>

File: instance/instances/robots/xacro/serial_numbers/valkyrie_B_serials.xacro (robot description, xacro)
@@ -4,24 +4,24 @@
 	<xacro:property name="leftLegJ3SerialNumber" value="v_c_004" />
 	<xacro:property name="leftLegJ4SerialNumber" value="v_d_003" />
-	<xacro:property name="leftAnkleLeftActuatorSerialNumber" value="v_e_007" />
-	<xacro:property name="leftAnkleRightActuatorSerialNumber" value="v_e_008" />
+	<xacro:property name="leftAnkleLeftActuatorSerialNumber" value="v_e_016" />
+	<xacro:property name="leftAnkleRightActuatorSerialNumber" value="v_e_015" />
 	<xacro:property name="rightLegJ1SerialNumber" value="v_a_007" />
 	<xacro:property name="rightLegJ2SerialNumber" value="v_b_007" />
 	<xacro:property name="rightLegJ3SerialNumber" value="v_c_003" />
 	<xacro:property name="rightLegJ4SerialNumber" value="v_d_002" />
-	<xacro:property name="rightAnkleLeftActuatorSerialNumber" value="v_e_009" />
-	<xacro:property name="rightAnkleRightActuatorSerialNumber" value="v_e_010" />
+	<xacro:property name="rightAnkleLeftActuatorSerialNumber" value="v_e_018" />
+	<xacro:property name="rightAnkleRightActuatorSerialNumber" value="v_e_017" />
 	<xacro:property name="leftArmJ1SerialNumber" value="v_a_002" />
-	<xacro:property name="leftArmJ2SerialNumber" value="v_b_008" />
-	<xacro:property name="leftArmJ3SerialNumber" value="v_f_009" />
-	<xacro:property name="leftArmJ4SerialNumber" value="v_f_010" />
-	<xacro:property name="leftArmJ5SerialNumber" value="UNKNOWN" />
+	<xacro:property name="leftArmJ2SerialNumber" value="v_b_005" />
+	<xacro:property name="leftArmJ3SerialNumber" value="v_f_007" />
+	<xacro:property name="leftArmJ4SerialNumber" value="v_f_008" />
+	<xacro:property name="leftArmJ5SerialNumber" value="v_g_007" />
 	<xacro:property name="leftWristTopActuatorSerialNumber" value="UNKNOWN" />
 	<xacro:property name="leftWristBottomActuatorSerialNumber" value="UNKNOWN" />
 	<xacro:property name="rightArmJ1SerialNumber" value="v_a_010" />
-	<xacro:property name="rightArmJ2SerialNumber" value="v_b_005" />
-	<xacro:property name="rightArmJ3SerialNumber" value="v_f_007" />
-	<xacro:property name="rightArmJ4SerialNumber" value="v_f_008" />
-	<xacro:property name="rightArmJ5SerialNumber" value="UNKNOWN" />
+	<xacro:property name="rightArmJ2SerialNumber" value="v_b_008" />
+	<xacro:property name="rightArmJ3SerialNumber" value="v_f_009" />
+	<xacro:property name="rightArmJ4SerialNumber" value="v_f_010" />
+	<xacro:property name="rightArmJ5SerialNumber" value="v_g_006" />
 	<xacro:property name="rightWristTopActuatorSerialNumber" value="UNKNOWN" />
 	<xacro:property name="rightWristBottomActuatorSerialNumber" value="UNKNOWN" />

Commit message: Updated the sensor node for the force_torque sensors.

File: common/xacro/nodes/valkyrie_nodes.xacro (robot description, xacro)
@@ -23,6 +23,6 @@
 	<xacro:property name="torso_imu1_node" value="/torso/sensors/imu1" />
 	<xacro:property name="torso_imu2_node" value="/torso/sensors/imu2" />
-	<xacro:property name="left_foot_ATI_node" value="/sensors/left_leg/force_torque" />
-	<xacro:property name="right_foot_ATI_node" value="/sensors/right_leg/force_torque" />
+	<xacro:property name="left_foot_ATI_node" value="/left_leg/j6" />
+	<xacro:property name="right_foot_ATI_node" value="/right_leg/j6" />
 	<xacro:macro name="all_channels" >
 		<Channels>

Commit message: Fixed topic names of ATI sensors and ankle actuator nodes.

File: common/xacro/nodes/valkyrie_nodes.xacro (robot description, xacro)
@@ -4,6 +4,6 @@
 	<xacro:property name="HipPitchNode" value="/${prefix}_leg/j3" />
 	<xacro:property name="KneePitchNode" value="/${prefix}_leg/j4" />
-	<xacro:property name="AnkleLeftActuatorNode" value="/${prefix}_leg/left_actuator" />
-	<xacro:property name="AnkleRightActuatorNode" value="/${prefix}_leg/right_actuator" />
+	<xacro:property name="AnkleLeftActuatorNode" value="/${prefix}_leg/ankle/left_actuator" />
+	<xacro:property name="AnkleRightActuatorNode" value="/${prefix}_leg/ankle/right_actuator" />
 	<xacro:property name="ShoulderPitchNode" value="/trunk/${prefix}_arm_j1" />
 	<xacro:property name="ShoulderRollNode" value="/${prefix}_arm/j2" />
@@ -23,6 +23,6 @@
 	<xacro:property name="torso_imu1_node" value="/torso/sensors/imu1" />
 	<xacro:property name="torso_imu2_node" value="/torso/sensors/imu2" />
-	<xacro:property name="left_foot_ATI_node" value="/left_leg/j6" />
-	<xacro:property name="right_foot_ATI_node" value="/right_leg/j6" />
+	<xacro:property name="left_foot_ATI_node" value="/left_leg/ankle/left_actuator" />
+	<xacro:property name="right_foot_ATI_node" value="/right_leg/ankle/left_actuator" />
 	<xacro:macro name="all_channels" >
 		<Channels>

Commit message: update nodes for force torque sensors in sim

File: common/xacro/nodes/valkyrie_nodes.xacro (robot description, xacro)
@@ -30,7 +30,7 @@
 	<xacro:property name="torso_imu2_node" value="/torso/sensors/imu2" />
 	<xacro:property name="left_foot_ATI_node" value="/left_leg/ankle/left_actuator" />
-	<xacro:property name="left_foot_Sim_ATI_node" value="/left_leg/ankle/pitch_actuator" />
+	<xacro:property name="left_foot_Sim_ATI_node" value="/sensors/leftFootSixAxis" />
 	<xacro:property name="right_foot_ATI_node" value="/right_leg/ankle/left_actuator" />
-	<xacro:property name="right_foot_Sim_ATI_node" value="/right_leg/ankle/pitch_actuator" />
+	<xacro:property name="right_foot_Sim_ATI_node" value="/sensors/rightFootSixAxis" />
 	<xacro:macro name="all_channels" >
 		<Channels>

Commit message: update node to match new imu locations

File: common/xacro/nodes/valkyrie_nodes.xacro (robot description, xacro)
@@ -25,6 +25,6 @@
 	<xacro:property name="WaistPitchActuatorSimNode" value="/trunk/pitch_actuator" /> <!--pitch-->
 	<xacro:property name="WaistRollActuatorSimNode" value="/trunk/roll_actuator" /> <!--roll-->
-	<xacro:property name="pelvis_middle_imu_node" value="/sensors/leftPelvisIMU" />
-	<xacro:property name="pelvis_rear_imu_node" value="/sensors/rightPelvisIMU" />
+	<xacro:property name="pelvis_middle_imu_node" value="/sensors/middlePelvisIMU" />
+	<xacro:property name="pelvis_rear_imu_node" value="/sensors/rearPelvisIMU" />
 	<xacro:property name="torso_left_imu_node" value="/sensors/leftTorsoIMU" />
 	<xacro:property name="torso_right_imu_node" value="/sensors/rightTorsoIMU" />
