Commit message: Still working on urdf part of athena stuff.

File: common/xacro/nodes/valkyrie_nodes.xacro (robot description, xacro)
@@ -25,10 +25,6 @@
 	<xacro:property name="WaistPitchActuatorSimNode" value="/trunk/pitch_actuator" /> <!--pitch-->
 	<xacro:property name="WaistRollActuatorSimNode" value="/trunk/roll_actuator" /> <!--roll-->
-	<xacro:property name="ThumbRollNode" value="/forearmDriver1"/>
-	<xacro:property name="ThumbPitch1Node" value="/forearmDriver1"/>
-	<xacro:property name="ThumbPitch2Node" value="/forearmDriver1"/>
-	<xacro:property name="IndexFingerNode" value="/forearmDriver2"/>
-	<xacro:property name="MiddleFingerNode" value="/forearmDriver2"/>
-	<xacro:property name="PinkyNode" value="/forearmDriver2"/>
+	<xacro:property name="Athena1Node" value="/${prefix}_arm/athena1"/>
+	<xacro:property name="Athena2Node" value="/${prefix}_arm/athena2"/>
 	<xacro:property name="pelvis_middle_imu_node" value="/sensors/middlePelvisIMU" />
 	<xacro:property name="pelvis_rear_imu_node" value="/sensors/rearPelvisIMU" />

File: common/xacro/serial_numbers/valkyrie_A_serials.xacro (robot description, xacro)
@@ -17,6 +17,4 @@
 	<xacro:property name="leftArmJ4SerialNumber" value="v_f_002" />
 	<xacro:property name="leftArmJ5SerialNumber" value="v_g_005" />
-	<xacro:property name="leftWristTopActuatorSerialNumber" value="UNKNOWN" />
-	<xacro:property name="leftWristBottomActuatorSerialNumber" value="UNKNOWN" />
 	<xacro:property name="rightArmJ1SerialNumber" value="v_a_001" />
 	<xacro:property name="rightArmJ2SerialNumber" value="v_b_003" />
@@ -24,6 +22,4 @@
 	<xacro:property name="rightArmJ4SerialNumber" value="v_f_003" />
 	<xacro:property name="rightArmJ5SerialNumber" value="v_g_003" />
-	<xacro:property name="rightWristTopActuatorSerialNumber" value="UNKNOWN" />
-	<xacro:property name="rightWristBottomActuatorSerialNumber" value="UNKNOWN" />
 	<xacro:property name="neckJ1SerialNumber" value="v_g_006" />
 	<xacro:property name="neckJ2SerialNumber" value="v_g_007" />
@@ -32,4 +28,6 @@
 	<xacro:property name="waistRightActuatorSerialNumber" value="v_e_005" />
 	<xacro:property name="waistLeftActuatorSerialNumber" value="v_e_006" />
+	<xacro:property name="leftForearmSerialNumber" value="v_h_001"/>
+    <xacro:property name="rightForearmSerialNumber" value="v_h_002"/>
 	<xacro:property name="left_foot_ATI_serial" value="FT14020" />
 	<xacro:property name="right_foot_ATI_serial" value="FT16592" />

File: common/xacro/serial_numbers/valkyrie_B_serials.xacro (robot description, xacro)
@@ -17,6 +17,4 @@
 	<xacro:property name="leftArmJ4SerialNumber" value="v_f_008" />
 	<xacro:property name="leftArmJ5SerialNumber" value="v_g_007" />
-	<xacro:property name="leftWristTopActuatorSerialNumber" value="UNKNOWN" />
-	<xacro:property name="leftWristBottomActuatorSerialNumber" value="UNKNOWN" />
 	<xacro:property name="rightArmJ1SerialNumber" value="v_a_010" />
 	<xacro:property name="rightArmJ2SerialNumber" value="v_b_008" />
@@ -24,16 +22,12 @@
 	<xacro:property name="rightArmJ4SerialNumber" value="v_f_010" />
 	<xacro:property name="rightArmJ5SerialNumber" value="v_g_006" />
-	<xacro:property name="rightWristTopActuatorSerialNumber" value="UNKNOWN" />
-	<xacro:property name="rightWristBottomActuatorSerialNumber" value="UNKNOWN" />
-	<xacro:property name="neckJ1SerialNumber" value="BLAH1" />
-	<xacro:property name="neckJ2SerialNumber" value="BLAH2" />
-	<xacro:property name="neckJ3SerialNumber" value="BLAH3" />
+	<xacro:property name="neckJ1SerialNumber" value="v_g_009" />
+	<xacro:property name="neckJ2SerialNumber" value="v_g_010" />
+	<xacro:property name="neckJ3SerialNumber" value="v_g_011" />
 	<xacro:property name="trunkSerialNumber" value="v_a_008" />
 	<xacro:property name="waistRightActuatorSerialNumber" value="v_e_011" />
 	<xacro:property name="waistLeftActuatorSerialNumber" value="v_e_012" />
-	<xacro:property name="pelvis_middle_imu_serial" value="UNKNOWN" />
-	<xacro:property name="pelvis_rear_imu_serial" value="UNKNOWN" />
-	<xacro:property name="torso_left_imu_serial" value="UNKNOWN" />
-	<xacro:property name="torso_right_imu_serial" value="UNKNOWN" />
+	<xacro:property name="leftForearmSerialNumber" value="v_h_003"/>
+    <xacro:property name="rightForearmSerialNumber" value="v_h_004"/>
 	<xacro:property name="left_foot_ATI_serial" value="FT17219" />
 	<xacro:property name="right_foot_ATI_serial" value="FT14019" />

File: common/xacro/serial_numbers/valkyrie_C_serials.xacro (robot description, xacro)
@@ -17,6 +17,4 @@
 	<xacro:property name="leftArmJ4SerialNumber" value="v_f_011" />
 	<xacro:property name="leftArmJ5SerialNumber" value="UNKNOWN" />
-	<xacro:property name="leftWristTopActuatorSerialNumber" value="UNKNOWN" />
-	<xacro:property name="leftWristBottomActuatorSerialNumber" value="UNKNOWN" />
 	<xacro:property name="rightArmJ1SerialNumber" value="v_a_012" />
 	<xacro:property name="rightArmJ2SerialNumber" value="v_b_012" />
@@ -24,6 +22,4 @@
 	<xacro:property name="rightArmJ4SerialNumber" value="v_f_014" />
 	<xacro:property name="rightArmJ5SerialNumber" value="UNKNOWN" />
-	<xacro:property name="rightWristTopActuatorSerialNumber" value="UNKNOWN" />
-	<xacro:property name="rightWristBottomActuatorSerialNumber" value="UNKNOWN" />
 	<xacro:property name="neckJ1SerialNumber" value="v_g_001" />
 	<xacro:property name="neckJ2SerialNumber" value="v_g_002" />
@@ -32,4 +28,6 @@
 	<xacro:property name="waistRightActuatorSerialNumber" value="v_e_014" />
 	<xacro:property name="waistLeftActuatorSerialNumber" value="v_e_013" />
+	<xacro:property name="leftForearmSerialNumber" value="v_h_006"/>
+    <xacro:property name="rightForearmSerialNumber" value="v_h_005"/>
 	<xacro:property name="left_foot_ATI_serial" value="FT17212" />
 	<xacro:property name="right_foot_ATI_serial" value="FT17214" />

File: common/xacro/serial_numbers/valkyrie_D_serials.xacro (robot description, xacro)
@@ -17,6 +17,4 @@
     <xacro:property name="leftArmJ4SerialNumber" value="v_f_016" />
     <xacro:property name="leftArmJ5SerialNumber" value="UNKNOWN" />
-    <xacro:property name="leftWristTopActuatorSerialNumber" value="UNKNOWN" />
-    <xacro:property name="leftWristBottomActuatorSerialNumber" value="UNKNOWN" />
     <xacro:property name="rightArmJ1SerialNumber" value="v_a_016" />
     <xacro:property name="rightArmJ2SerialNumber" value="v_b_013" />
@@ -24,6 +22,4 @@
     <xacro:property name="rightArmJ4SerialNumber" value="v_f_015" />
     <xacro:property name="rightArmJ5SerialNumber" value="UNKNOWN" />
-    <xacro:property name="rightWristTopActuatorSerialNumber" value="UNKNOWN" />
-    <xacro:property name="rightWristBottomActuatorSerialNumber" value="UNKNOWN" />
     <xacro:property name="neckJ1SerialNumber" value="v_g_012" />
     <xacro:property name="neckJ2SerialNumber" value="v_g_013" />
@@ -32,4 +28,6 @@
     <xacro:property name="waistRightActuatorSerialNumber" value="v_e_023" />
     <xacro:property name="waistLeftActuatorSerialNumber" value="v_e_024" />
+    <xacro:property name="leftForearmSerialNumber" value="v_h_007"/>
+    <xacro:property name="rightForearmSerialNumber" value="v_h_008"/>
     <xacro:property name="left_foot_ATI_serial" value="FT14182" />
     <xacro:property name="right_foot_ATI_serial" value="FT16591" />

File: instance/instances/robots/xacro/common/valkyrie_full_template.xacro (robot description, xacro)
@@ -12,6 +12,6 @@
 		<xacro:leg prefix="left" j1_serial_number="${leftLegJ1SerialNumber}" j2_serial_number="${leftLegJ2SerialNumber}" j3_serial_number="${leftLegJ3SerialNumber}" j4_serial_number="${leftLegJ4SerialNumber}" ankle_left_actuator_serial="${leftAnkleLeftActuatorSerialNumber}" ankle_right_actuator_serial="${leftAnkleRightActuatorSerialNumber}"/>
 		<xacro:leg prefix="right" j1_serial_number="${rightLegJ1SerialNumber}" j2_serial_number="${rightLegJ2SerialNumber}" j3_serial_number="${rightLegJ3SerialNumber}" j4_serial_number="${rightLegJ4SerialNumber}" ankle_left_actuator_serial="${rightAnkleLeftActuatorSerialNumber}" ankle_right_actuator_serial="${rightAnkleRightActuatorSerialNumber}" />
-		<xacro:arm prefix="left" j1_serial_number="${leftArmJ1SerialNumber}" j2_serial_number="${leftArmJ2SerialNumber}" j3_serial_number="${leftArmJ3SerialNumber}" j4_serial_number="${leftArmJ4SerialNumber}" j5_serial_number="${leftArmJ5SerialNumber}" wrist_actuator0_serial="${leftWristTopActuatorSerialNumber}" wrist_actuator1_serial="${leftWristBottomActuatorSerialNumber}" />
-		<xacro:arm prefix="right" j1_serial_number="${rightArmJ1SerialNumber}" j2_serial_number="${rightArmJ2SerialNumber}" j3_serial_number="${rightArmJ3SerialNumber}" j4_serial_number="${rightArmJ4SerialNumber}" j5_serial_number="${rightArmJ5SerialNumber}" wrist_actuator0_serial="${rightWristTopActuatorSerialNumber}" wrist_actuator1_serial="${rightWristBottomActuatorSerialNumber}" />
+		<xacro:arm prefix="left" j1_serial_number="${leftArmJ1SerialNumber}" j2_serial_number="${leftArmJ2SerialNumber}" j3_serial_number="${leftArmJ3SerialNumber}" j4_serial_number="${leftArmJ4SerialNumber}" j5_serial_number="${leftArmJ5SerialNumber}" forearm_serial_number="${leftForearmSerialNumber}" />
+		<xacro:arm prefix="right" j1_serial_number="${rightArmJ1SerialNumber}" j2_serial_number="${rightArmJ2SerialNumber}" j3_serial_number="${rightArmJ3SerialNumber}" j4_serial_number="${rightArmJ4SerialNumber}" j5_serial_number="${rightArmJ5SerialNumber}" forearm_serial_number="${rightForearmSerialNumber}" />
 		<xacro:neck j1_serial_number="${neckJ1SerialNumber}" j2_serial_number="${neckJ2SerialNumber}" j3_serial_number="${neckJ3SerialNumber}" />
 		<xacro:waist j1_serial_number="${trunkSerialNumber}" waist_left_actuator_serial="${waistLeftActuatorSerialNumber}" waist_right_actuator_serial="${waistRightActuatorSerialNumber}"/>

File: instance/instances/robots/xacro/mechanisms/mechanisms.xacro (robot description, xacro)
@@ -6,5 +6,5 @@
 	</Mechanism>
 </xacro:macro>
-<xacro:macro name="joint" params="name type calibration_file">
+<xacro:macro name="joint" params="name type">
 	<Joint id="${name}" type="${type}">
 	</Joint>
@@ -18,9 +18,20 @@
 <xacro:macro name="two_active_joint_mechanism" params="mechanism_name actuator0_name actuator1_name joint0_name joint1_name actuator0_serial actuator0_node actuator1_serial actuator1_node " >
 	<Mechanism id="${mechanism_name}" type="complex">
-		<xacro:joint name="${joint0_name}" type="active" calibration_file="${instance}_${mechanism_name}_${joint0_name}_cal.xml"/>
-		<xacro:joint name="${joint1_name}" type="active" calibration_file="${instance}_${mechanism_name}_${joint1_name}_cal.xml"/>
+		<xacro:joint name="${joint0_name}" type="active"/>
+		<xacro:joint name="${joint1_name}" type="active"/>
 		<xacro:actuator name="${actuator0_name}" serial_number="${actuator0_serial}" node="${actuator0_node}" />
 		<xacro:actuator name="${actuator1_name}" serial_number="${actuator1_serial}" node="${actuator1_node}" />
 	</Mechanism>
 </xacro:macro>
+<xacro:macro name="forearm" params="mechanism_name serial_number athena1_node athena2_node">
+    <Mechanism id="${mechanism_name}" type="forearm">
+        <Nodes>
+            <SerialNumber id="${serial_number}"/>
+            <Nodes>
+                <Athena1 id="${athena1_node}"/>
+                <Athena2 id="${athena2_node}"/>
+            </Nodes>
+        </Nodes>
+    </Mechanism>
+</xacro:macro>
 </robot>

File: model/robots/common/xacro/arm/arm.xacro (robot description, xacro)
@@ -166,6 +166,6 @@
     <xacro:simple_transmission jointName="${ElbowPitchJointName}" actuatorName="${ElbowPitchActuatorName}" nodeName="${ElbowPitchNode}" actuatorApi="${ElbowPitchApi}"/>
     <xacro:simple_transmission jointName="${ForearmYawActuatorName}" actuatorName="${ForearmYawActuatorName}" nodeName="${ForearmYawNode}" actuatorApi="${ForearmYawApi}"/>
-    <xacro:athena1_transmission prefix="${prefix}"/>
-    <xacro:athena2_transmission prefix="${prefix}"/>
+    <xacro:athena1_transmission prefix="${prefix}" transmissionName="${prefix}ArmAthena1Transmission"/>
+    <xacro:athena2_transmission prefix="${prefix}" transmissionName="${prefix}ArmAthena2Transmission"/>
   </xacro:macro>
   <xacro:macro name="arm_transmissions_no_hands" params="prefix">

File: model/robots/common/xacro/generic_models.xacro (robot description, xacro)
@@ -275,43 +275,47 @@
     </transmission>
   </xacro:macro>
-  <xacro:macro name="athena1_transmission" params="prefix">
-    <type>robot_transmission_interface/athena1_transmission</type>
-    <joint name="${prefix}WristPitch">
-      <role>wristPitch</role>
-    </joint>
-    <joint name="${prefix}WristRoll">
-      <role>wristRoll</role>
-    </joint>
-    <joint name="${prefix}ThumbRoll">
-      <role>thumbRoll</role>
-    </joint>
-    <joint name="${prefix}ThumbPitch1">
-      <role>thumbPitch1</role>
-    </joint>
-    <actuator name="${prefix}Athena1Actuator">
-      <role>athena1Actuator</role>
-      <mechanicalReduction>1</mechanicalReduction>
-      <hardwareInterface>PositionJointInterface</hardwareInterface>
-    </actuator>
-  </xacro:macro>
-  <xacro:macro name="athena2_transmission" params="prefix">
-    <type>robot_transmission_interface/athena2_transmission</type>
-    <joint name="${prefix}ThumbPitch2">
-      <role>thumbPitch2</role>
-    </joint>
-    <joint name="${prefix}IndexFingerPitch1">
-      <role>indexFingerPitch1</role>
-    </joint>
-    <joint name="${prefix}MiddleFingerPitch1">
-      <role>middleFingerPitch1</role>
-    </joint>
-    <joint name="${prefix}PinkyPitch1">
-      <role>pinkyPitch1</role>
-    </joint>
-    <actuator name="${prefix}Athena2Actuator">
-      <role>athena2Actuator</role>
-      <mechanicalReduction>1</mechanicalReduction>
-      <hardwareInterface>PositionJointInterface</hardwareInterface>
-    </actuator>
+  <xacro:macro name="athena1_transmission" params="prefix transmissionName">
+    <transmission name="${transmissionName}">
+      <type>robot_transmission_interface/athena1_transmission</type>
+      <joint name="${prefix}WristPitch">
+        <role>wristPitch</role>
+      </joint>
+      <joint name="${prefix}WristRoll">
+        <role>wristRoll</role>
+      </joint>
+      <joint name="${prefix}ThumbRoll">
+        <role>thumbRoll</role>
+      </joint>
+      <joint name="${prefix}ThumbPitch1">
+        <role>thumbPitch1</role>
+      </joint>
+      <actuator name="${prefix}Athena1Actuator">
+        <role>athena1Actuator</role>
+        <mechanicalReduction>1</mechanicalReduction>
+        <hardwareInterface>PositionJointInterface</hardwareInterface>
+      </actuator>
+    </transmission>
+  </xacro:macro>
+  <xacro:macro name="athena2_transmission" params="prefix transmissionName">
+    <transmission name="${transmissionName}">
+      <type>robot_transmission_interface/athena2_transmission</type>
+      <joint name="${prefix}ThumbPitch2">
+        <role>thumbPitch2</role>
+      </joint>
+      <joint name="${prefix}IndexFingerPitch1">
+        <role>indexFingerPitch1</role>
+      </joint>
+      <joint name="${prefix}MiddleFingerPitch1">
+        <role>middleFingerPitch1</role>
+      </joint>
+      <joint name="${prefix}PinkyPitch1">
+        <role>pinkyPitch1</role>
+      </joint>
+      <actuator name="${prefix}Athena2Actuator">
+        <role>athena2Actuator</role>
+        <mechanicalReduction>1</mechanicalReduction>
+        <hardwareInterface>PositionJointInterface</hardwareInterface>
+      </actuator>
+    </transmission>
   </xacro:macro>
 </robot>
