Commit message: Location coeffs changed to less constricting joint range limits more suited for test bench actuator checkouts

File: common/xacro/nodes/test_bench_nodes.xacro (robot description, xacro)
@@ -1,3 +1,3 @@
 <robot xmlns:xacro="http://ros.org/wiki/xacro" name="valkyrie_nodes">
-	<xacro:property name="testbench_node" value="/left_arm/j0" />
+	<xacro:property name="testbench_node" value="/right_leg/j1" />
 </robot>

File: common/xacro/serial_numbers/test_bench_serials.xacro (robot description, xacro)
@@ -1,3 +1,3 @@
 <robot xmlns:xacro="http://ros.org/wiki/xacro" name="test_bench_serials">
-	<xacro:property name="testbench_serial_number" value="v_a_013" />
+	<xacro:property name="testbench_serial_number" value="v_c_008" />
 </robot>

Commit message: prepping tesbench instance for neck development

File: common/xacro/nodes/test_bench_nodes.xacro (robot description, xacro)
@@ -1,3 +1,5 @@
 <robot xmlns:xacro="http://ros.org/wiki/xacro" name="valkyrie_nodes">
-	<xacro:property name="testbench_node" value="/right_leg/j1" />
+	<xacro:property name="testbench_node1" value="/left_arm/j1" />
+	<xacro:property name="testbench_node2" value="/left_arm/j2" />
+	<xacro:property name="testbench_node3" value="/left_arm/j3" />
 </robot>

File: common/xacro/serial_numbers/test_bench_serials.xacro (robot description, xacro)
@@ -1,3 +1,5 @@
 <robot xmlns:xacro="http://ros.org/wiki/xacro" name="test_bench_serials">
-	<xacro:property name="testbench_serial_number" value="v_c_008" />
+	<xacro:property name="testbench_serial_number1" value="v_g_001" />
+	<xacro:property name="testbench_serial_number2" value="v_g_002" />
+	<xacro:property name="testbench_serial_number3" value="v_g_003" />
 </robot>

Commit message: calebrated wrists and added initial checkout of j5

File: common/xacro/nodes/test_bench_nodes.xacro (robot description, xacro)
@@ -1,3 +1,3 @@
 <robot xmlns:xacro="http://ros.org/wiki/xacro" name="valkyrie_nodes">
-	<xacro:property name="testbench_node" value="/right_leg/j1" />
+	<xacro:property name="testbench_node" value="/left_arm/j5" />
 </robot>

File: common/xacro/serial_numbers/test_bench_serials.xacro (robot description, xacro)
@@ -1,3 +1,3 @@
 <robot xmlns:xacro="http://ros.org/wiki/xacro" name="test_bench_serials">
-	<xacro:property name="testbench_serial_number" value="v_c_008" />
+	<xacro:property name="testbench_serial_number" value="v_g_012" />
 </robot>

File: common/xacro/serial_numbers/valkyrie_C_serials.xacro (robot description, xacro)
@@ -28,4 +28,6 @@
 	<xacro:property name="waistRightActuatorSerialNumber" value="v_e_014" />
 	<xacro:property name="waistLeftActuatorSerialNumber" value="v_e_013" />
+	<xacro:property name="leftForearmSerialNumber" value="UNKNOWN"/>
+        <xacro:property name="rightForearmSerialNumber" value="UNKNOWN"/>
 	<xacro:property name="left_foot_ATI_serial" value="FT14182" />
 	<xacro:property name="right_foot_ATI_serial" value="FT17214" />
