Commit message: UoE hand workbench configs

File: common/xacro/nodes/forearm_testbench_nodes.xacro (robot description, xacro)
@@ -1,3 +1,4 @@
 <robot xmlns:xacro="http://ros.org/wiki/xacro" name="test_bench_nodes">
+	<xacro:property name="ForearmYawNode" value="/left_arm/j5" />
 	<xacro:property name="Athena1Node" value="/left_arm/athena1" />
 	<xacro:property name="Athena2Node" value="/left_arm/athena2" />

File: common/xacro/serial_numbers/forearm_testbench_serials.xacro (robot description, xacro)
@@ -1,3 +1,4 @@
 <robot xmlns:xacro="http://ros.org/wiki/xacro" name="forearm_testbench">
 	<xacro:property name="forearm_serial_number" value="v_h_005" />
+	<xacro:property name="j5_serial_number" value="v_g_016" />
 </robot>

File: instance/instances/robots/forearm_testbench.xacro (robot description, xacro)
@@ -4,10 +4,11 @@
 	<xacro:include filename="$(find val_description)/common/xacro/nodes/forearm_testbench_nodes.xacro" />
 	<xacro:include filename="$(find val_description)/common/xacro/serial_numbers/forearm_testbench_serials.xacro" />
-    <xacro:include filename="$(find val_description)/instance/instances/robots/xacro/mechanisms/mechanisms.xacro"/>
-    <xacro:include filename="$(find val_description)/common/xacro/joint_names/valkyrie_joint_names.xacro"/>
+	<xacro:include filename="$(find val_description)/instance/instances/robots/xacro/mechanisms/mechanisms.xacro"/>
+	<xacro:include filename="$(find val_description)/common/xacro/joint_names/valkyrie_joint_names.xacro"/>
     <Channels>
     </Channels>
-    <Mechanisms>
-    <xacro:forearm mechanism_name="${prefix}Forearm" serial_number="${forearm_serial_number}" athena1_node="${Athena1Node}" athena2_node="${Athena2Node}" />
+    	<Mechanisms>
+	    	<xacro:simple_mechanism name="${ForearmYawJointName}" serial_number="${j5_serial_number}" node="${ForearmYawNode}"/>
+    		<xacro:forearm mechanism_name="${prefix}Forearm" serial_number="${forearm_serial_number}" athena1_node="${Athena1Node}" athena2_node="${Athena2Node}" />
 	</Mechanisms>
 	<Devices>

Commit message: Switch to right arm

File: common/xacro/nodes/forearm_testbench_nodes.xacro (robot description, xacro)
@@ -1,5 +1,5 @@
 <robot xmlns:xacro="http://ros.org/wiki/xacro" name="test_bench_nodes">
-	<xacro:property name="ForearmYawNode" value="/left_arm/j5" />
-	<xacro:property name="Athena1Node" value="/left_arm/athena1" />
-	<xacro:property name="Athena2Node" value="/left_arm/athena2" />
+	<xacro:property name="ForearmYawNode" value="/right_arm/j5" />
+	<xacro:property name="Athena1Node" value="/right_arm/athena1" />
+	<xacro:property name="Athena2Node" value="/right_arm/athena2" />
 </robot>

File: common/xacro/serial_numbers/forearm_testbench_serials.xacro (robot description, xacro)
@@ -1,4 +1,4 @@
 <robot xmlns:xacro="http://ros.org/wiki/xacro" name="forearm_testbench">
-	<xacro:property name="forearm_serial_number" value="v_h_005" />
-	<xacro:property name="j5_serial_number" value="v_g_016" />
+	<xacro:property name="forearm_serial_number" value="v_h_006" />
+	<xacro:property name="j5_serial_number" value="v_g_012" />
 </robot>

Commit message: Split left and right forearm testbench xacros

File: common/xacro/nodes/forearm_testbench_nodes.xacro (robot description, xacro)
@@ -1,5 +1,5 @@
 <robot xmlns:xacro="http://ros.org/wiki/xacro" name="test_bench_nodes">
-	<xacro:property name="ForearmYawNode" value="/right_arm/j5" />
-	<xacro:property name="Athena1Node" value="/right_arm/athena1" />
-	<xacro:property name="Athena2Node" value="/right_arm/athena2" />
+	<xacro:property name="ForearmYawNode" value="/${prefix}_arm/j5" />
+	<xacro:property name="Athena1Node" value="/${prefix}_arm/athena1" />
+	<xacro:property name="Athena2Node" value="/${prefix}_arm/athena2" />
 </robot>

File: instance/instances/robots/forearm_testbench_left.xacro (robot description, xacro)
@@ -3,5 +3,5 @@
 	<xacro:property name="prefix" value="left" />
 	<xacro:include filename="$(find val_description)/common/xacro/nodes/forearm_testbench_nodes.xacro" />
-	<xacro:include filename="$(find val_description)/common/xacro/serial_numbers/forearm_testbench_serials.xacro" />
+	<xacro:include filename="$(find val_description)/common/xacro/serial_numbers/forearm_left_testbench_serials.xacro" />
 	<xacro:include filename="$(find val_description)/instance/instances/robots/xacro/mechanisms/mechanisms.xacro"/>
 	<xacro:include filename="$(find val_description)/common/xacro/joint_names/valkyrie_joint_names.xacro"/>
