Commit message: Fixed orientation of torso IMU and removed some unused xacro code.

File: model/robots/common/xacro/waist/waist.xacro (robot description, xacro)
@@ -68,14 +68,9 @@
     <xacro:make_waist_common waist_root_link="${waist_root_link}"/>
   </xacro:macro>
-  <xacro:macro name="waist_actuators"  params="name1 type1 name2 type2 name3 type3">
-    <actuator name="${name1}" type="${type1}"/>
-    <actuator name="${name2}" type="${type2}"/>
-    <actuator name="${name3}" type="${type3}"/>
-  </xacro:macro>
   <xacro:macro name="v1_trunk_sensors">
     <xacro:microstrain_sensor sensorName="leftTorsoImu"
                               parentLink="${TorsoRollLinkName}"
-                              origin_xyz="-0.046863 0.134239 0.3630676"
-                              origin_rpy="1.57 0 3.14" />
+                              origin_xyz="-0.0627634 0.134239 0.3630676"
+                              origin_rpy="-1.5707 0.0 0.0" />
     <xacro:flea3_camera sensorName="rightHazardCamera"
                         parentLink="${TorsoRollLinkName}"
