Commit message: Made all sensor, link, and joint names that weren't already lowercase to be lowercase.

File: model/robots/common/xacro/pelvis/pelvis.xacro (robot description, xacro)
@@ -1,4 +1,4 @@
 <robot xmlns:xacro="http://ros.org/wiki/xacro" name="Pelvis">
-    <xacro:property name="Pelvis_Link_Name" value="Pelvis" />
+    <xacro:property name="Pelvis_Link_Name" value="pelvis" />
     <xacro:macro name="make_pelvis">
         <xacro:standard_link name="${Pelvis_Link_Name}"
@@ -12,9 +12,9 @@
     </xacro:macro>
     <xacro:macro name="v1_pelvis_sensors">
-        <xacro:microstrain_sensor sensorName="RightPelvisIMU"
+        <xacro:microstrain_sensor sensorName="rightPelvisIMU"
                                   parentLink="${Pelvis_Link_Name}"
                                   origin_xyz="0.0515 -0.115 -0.042"
                                   origin_rpy="-1.57 0.0 1.274" />
-        <xacro:microstrain_sensor sensorName="LeftPelvisIMU"
+        <xacro:microstrain_sensor sensorName="leftPelvisIMU"
                                   parentLink="${Pelvis_Link_Name}"
                                   origin_xyz="0.0515 0.115 -0.042"

File: model/robots/common/xacro/waist/link_names.xacro (robot description, xacro)
@@ -2,6 +2,6 @@
 <robot xmlns:xacro="http://www.ros.org/wiki/xacro" name="v1/waist/dh_parameters">
   <xacro:property name="TorsoYawParentLinkName" value="${waist_root_link}" />
-  <xacro:property name="TorsoYawLinkName" value="TorsoYawLink" />
-  <xacro:property name="TorsoPitchLinkName" value="TorsoPitchLink" />
-  <xacro:property name="TorsoRollLinkName" value="Torso" />
+  <xacro:property name="TorsoYawLinkName" value="torsoYawLink" />
+  <xacro:property name="TorsoPitchLinkName" value="torsoPitchLink" />
+  <xacro:property name="TorsoRollLinkName" value="torso" />
 </robot>

File: model/robots/common/xacro/waist/waist.xacro (robot description, xacro)
@@ -77,13 +77,13 @@
   </xacro:macro>
   <xacro:macro name="v1_trunk_sensors">
-    <xacro:microstrain_sensor sensorName="RightTorsoIMU"
+    <xacro:microstrain_sensor sensorName="rightTorsoIMU"
                               parentLink="${TorsoRollLinkName}"
                               origin_xyz="-0.047 -0.134 0.363"
                               origin_rpy="-1.57 0.0 3.14" />
-    <xacro:microstrain_sensor sensorName="LeftTorsoIMU"
+    <xacro:microstrain_sensor sensorName="leftTorsoIMU"
                               parentLink="${TorsoRollLinkName}"
                               origin_xyz="-0.047 0.134 0.363"
                               origin_rpy="1.57 0.0 3.14" />
-    <xacro:flea3_camera sensorName="RightHazardCamera"
+    <xacro:flea3_camera sensorName="rightHazardCamera"
                         parentLink="${TorsoRollLinkName}"
                         origin_xyz="0.0345 -0.0406 0.1135"
@@ -91,5 +91,5 @@
                         imageFormat="R8G8B8"
                         frameRate="60"/>
-    <xacro:flea3_camera sensorName="LeftHazardCamera"
+    <xacro:flea3_camera sensorName="leftHazardCamera"
                         parentLink="${TorsoRollLinkName}"
                         origin_xyz="0.0345 0.0406 0.1135"

Commit message: updated controllers for use on unit C

File: model/robots/common/xacro/pelvis/pelvis.xacro (robot description, xacro)
@@ -34,3 +34,16 @@
                                   sensor_port="${sensor_port_tag}" />
     </xacro:macro>
+    <xacro:macro name="v1_pelvis_rear_sensors_usb" params="sensor_node_tag sensor_api_tag sensor_port_tag">
+        <xacro:usb_microstrain_sensor sensorName="pelvisRearImu"
+                                  parentLink="${Pelvis_Link_Name}"
+                                  origin_xyz="-0.075844901 0.0 -0.111056426"
+                                  origin_rpy="-3.14159 0.476467 -3.14159"
+                                  sensor_node="${sensor_node_tag}"
+                                  sensor_api="${sensor_api_tag}"
+                                  sensor_port="${sensor_port_tag}" />
+        <xacro:microstrain_sensor sensorName="pelvisMiddleImu"
+                                  parentLink="${Pelvis_Link_Name}"
+                                  origin_xyz="0.0 0.0 -0.108184035"
+                                  origin_rpy="3.14159 0.0 -3.14159" />
+    </xacro:macro>
 </robot>

Commit message: Double checked IMU stuff and switched around some macros in pelvis.xacro. About to make sure it's all good on robot before merging.

File: model/robots/common/xacro/pelvis/pelvis.xacro (robot description, xacro)
@@ -18,8 +18,8 @@
         <xacro:microstrain_sensor sensorName="pelvisMiddleImu"
                                   parentLink="${Pelvis_Link_Name}"
-                                  origin_xyz="0.012 0.0 -0.108184035"
-                                  origin_rpy="3.14159 0.0 -3.14159" />
+                                  origin_xyz="0.0 0.0 -0.10819638"
+                                  origin_rpy="3.14159 0.0 0.0" />
     </xacro:macro>
-    <xacro:macro name="v1_pelvis_sensors_usb" params="sensor_node_tag sensor_api_tag sensor_port_tag">
+    <xacro:macro name="v1_pelvis_middle_sensors_usb" params="sensor_node_tag sensor_api_tag sensor_port_tag">
         <xacro:microstrain_sensor sensorName="pelvisRearImu"
                                   parentLink="${Pelvis_Link_Name}"
@@ -28,6 +28,6 @@
         <xacro:usb_microstrain_sensor sensorName="pelvisMiddleImu"
                                   parentLink="${Pelvis_Link_Name}"
-                                  origin_xyz="0.0 0.0 -0.108184035"
-                                  origin_rpy="3.14159 0.0 -3.14159"
+                                  origin_xyz="0.0 0.0 -0.10819638"
+                                  origin_rpy="3.14159 0.0 0.0"
                                   sensor_node="${sensor_node_tag}"
                                   sensor_api="${sensor_api_tag}"
@@ -38,12 +38,28 @@
                                   parentLink="${Pelvis_Link_Name}"
                                   origin_xyz="-0.075844901 0.0 -0.111056426"
-                                  origin_rpy="-3.14159 0.476467 0"
-				  sensor_node="${sensor_node_tag}"
-				  sensor_api="${sensor_api_tag}"
-				  sensor_port="${sensor_port_tag}" />
+                                  origin_rpy="-3.14159 0.476467 -3.14159"
+                        				  sensor_node="${sensor_node_tag}"
+                        				  sensor_api="${sensor_api_tag}"
+                        				  sensor_port="${sensor_port_tag}" />
         <xacro:microstrain_sensor sensorName="pelvisMiddleImu"
                                   parentLink="${Pelvis_Link_Name}"
-                                  origin_xyz="0.0 0.0 -0.108184035"
-                                  origin_rpy="3.14159 0.0 -3.14159" />
+                                  origin_xyz="0.0 0.0 -0.10819638"
+                                  origin_rpy="3.14159 0.0 0.0" />
+    </xacro:macro>
+    <xacro:macro name="v1_pelvis_sensors_usb" params="middle_sensor_node_tag middle_sensor_api_tag middle_sensor_port_tag rear_sensor_node_tag rear_sensor_api_tag rear_sensor_port_tag">
+        <xacro:usb_microstrain_sensor sensorName="pelvisRearImu"
+                                  parentLink="${Pelvis_Link_Name}"
+                                  origin_xyz="-0.075844901 0.0 -0.111056426"
+                                  origin_rpy="-3.14159 0.476467 -3.14159"
+                                  sensor_node="${rear_sensor_node_tag}"
+                                  sensor_api="${rear_sensor_api_tag}"
+                                  sensor_port="${rear_sensor_port_tag}" />
+        <xacro:usb_microstrain_sensor sensorName="pelvisMiddleImu"
+                                  parentLink="${Pelvis_Link_Name}"
+                                  origin_xyz="0.0 0.0 -0.10819638"
+                                  origin_rpy="3.14159 0.0 0.0"
+                                  sensor_node="${middle_sensor_node_tag}"
+                                  sensor_api="${middle_sensor_api_tag}"
+                                  sensor_port="${middle_sensor_port_tag}" />
     </xacro:macro>
 </robot>

File: model/robots/common/xacro/valkyrie_base_hw.xacro (robot description, xacro)
@@ -19,5 +19,5 @@
     <xacro:v1_leg_sensors prefix="right" reflect="-1" ATI_serial_number="${right_foot_ATI_serial}" ATI_node="${right_foot_ATI_node}"/>
     <xacro:include_multisense_hw />
-    <xacro:v1_pelvis_sensors_usb sensor_node_tag="${pelvis_middle_imu_node}" sensor_api_tag="${ImuMicrostrainHardwareApi}" sensor_port_tag="${pelvis_middle_imu_port}"/>
+    <xacro:v1_pelvis_middle_sensors_usb sensor_node_tag="${pelvis_middle_imu_node}" sensor_api_tag="${ImuMicrostrainHardwareApi}" sensor_port_tag="${pelvis_middle_imu_port}"/>
     <xacro:waist_transmissions_hw />
     <xacro:leg_transmissions_hw prefix="left"/>

File: model/robots/common/xacro/valkyrie_base_sim.xacro (robot description, xacro)
@@ -20,5 +20,5 @@
     <xacro:make_leg prefix="right" reflect="-1" leg_root_link="${Pelvis_Link_Name}"/>
     <xacro:make_leg prefix="left" reflect="1" leg_root_link="${Pelvis_Link_Name}"/>
-    <xacro:v1_pelvis_sensors_usb sensor_node_tag="${pelvis_middle_imu_node}" sensor_api_tag="${ImuSensorSimApi}" sensor_port_tag="${pelvis_middle_imu_port}"/>
+    <xacro:v1_pelvis_sensors_usb middle_sensor_node_tag="${pelvis_middle_imu_node}" middle_sensor_api_tag="${ImuSensorSimApi}" middle_sensor_port_tag="${pelvis_middle_imu_port}" rear_sensor_node_tag="${pelvis_rear_imu_node}" rear_sensor_api_tag="${ImuSensorSimApi}" rear_sensor_port_tag="${pelvis_rear_imu_port}"/>
     <xacro:v1_leg_sensors prefix="left" reflect="1" ATI_serial_number="${sim_ATI_serial}" ATI_node="${left_foot_Sim_ATI_node}"/>
     <xacro:v1_leg_sensors prefix="right" reflect="-1" ATI_serial_number="${sim_ATI_serial}" ATI_node="${right_foot_Sim_ATI_node}"/>
