Commit message: change pin location to TorsoRollLinkName

File: model/robots/valkyrie_sim_pinned.xacro (robot description, xacro)
@@ -11,5 +11,5 @@
     <joint name="fixed" type="fixed">
     	<parent link="world"/>
-    	<child link="${Pelvis_Link_Name}"/>
+    	<child link="${TorsoRollLinkName}"/>
   	</joint>
 </robot>

Commit message: update pin to torso

File: model/robots/valkyrie_sim_pinned.xacro (robot description, xacro)
@@ -8,8 +8,17 @@
     <xacro:include filename="$(find val_description)/common/xacro/serial_numbers/valkyrie_A_serials.xacro"/>
     <xacro:include filename="$(find val_description)/common/xacro/dev_ports/valkyrie_gazebo_ports.xacro"/>
-    <link name="world"/>
-    <joint name="fixed" type="fixed">
-    	<parent link="world"/>
-    	<child link="${TorsoRollLinkName}"/>
-  	</joint>
+    <gazebo>
+      <joint name="fixed" type="revolute">
+        <parent>world</parent>
+        <child>torso</child>
+        <axis>
+          <xyz>0 0 1</xyz>
+          <use_parent_model_frame>true</use_parent_model_frame>
+          <limit>
+            <upper>0</upper>
+            <lower>0</lower>
+          </limit>
+        </axis>
+      </joint>
+    </gazebo>
 </robot>

Commit message: change torso to  per recommendation.

File: model/robots/valkyrie_sim_pinned.xacro (robot description, xacro)
@@ -11,5 +11,5 @@
       <joint name="fixed" type="revolute">
         <parent>world</parent>
-        <child>torso</child>
+        <child>${TorsoRollLinkName}</child>
         <axis>
           <xyz>0 0 1</xyz>
