Commit message: split forearm urdf into two so don't have to recompile when switching arms

File: model/robots/forearm_right.xacro (robot description, xacro)
@@ -3,5 +3,5 @@
     <xacro:include filename="$(find val_description)/model/robots/common/xacro/generic_models.xacro" />
     <xacro:include filename="$(find val_description)/model/robots/common/xacro/common_bodies.xacro" />
-    <xacro:property name="prefix" value="left"/>
+    <xacro:property name="prefix" value="right"/>
     <xacro:property name="reflect" value="1"/>
     <link name="world"/>
