Commit message: added yaw joint to forearm urdfs

File: model/robots/forearm_left.xacro (robot description, xacro)
@@ -6,9 +6,10 @@
     <xacro:property name="reflect" value="1"/>
     <link name="world"/>
-    <joint name="fixed" type="fixed">
-        <parent link="world"/>
-        <child link="${prefix}ForearmLink"/>
-    </joint>
     <xacro:make_lower_arm prefix="${prefix}" reflect="${reflect}" lower_arm_root_link="world"/>
+    <xacro:make_thumb prefix="${prefix}" reflect="-1" thumb_root_link="${prefix}Palm"/>
+    <xacro:make_index_finger prefix="${prefix}" reflect="-1" index_finger_root_link="${prefix}Palm"/>
+    <xacro:make_middle_finger prefix="${prefix}" reflect="-1" middle_finger_root_link="${prefix}Palm"/>
+    <xacro:make_pinky_finger prefix="${prefix}" reflect="-1" pinky_finger_root_link="${prefix}Palm"/>
+    <xacro:simple_position_transmission jointName="${ForearmYawActuatorName}" actuatorName="${ForearmYawActuatorName}" nodeName="${ForearmYawNode}" actuatorApi="${ForearmYawApi}"/>
     <xacro:index_finger_transmissions_hw prefix="${prefix}" />
     <xacro:middle_finger_transmissions_hw prefix="${prefix}" />

File: model/robots/forearm_right.xacro (robot description, xacro)
@@ -6,9 +6,10 @@
     <xacro:property name="reflect" value="1"/>
     <link name="world"/>
-    <joint name="fixed" type="fixed">
-        <parent link="world"/>
-        <child link="${prefix}ForearmLink"/>
-    </joint>
     <xacro:make_lower_arm prefix="${prefix}" reflect="${reflect}" lower_arm_root_link="world"/>
+    <xacro:make_thumb prefix="${prefix}" reflect="-1" thumb_root_link="${prefix}Palm"/>
+    <xacro:make_index_finger prefix="${prefix}" reflect="-1" index_finger_root_link="${prefix}Palm"/>
+    <xacro:make_middle_finger prefix="${prefix}" reflect="-1" middle_finger_root_link="${prefix}Palm"/>
+    <xacro:make_pinky_finger prefix="${prefix}" reflect="-1" pinky_finger_root_link="${prefix}Palm"/>
+    <xacro:simple_position_transmission jointName="${ForearmYawActuatorName}" actuatorName="${ForearmYawActuatorName}" nodeName="${ForearmYawNode}" actuatorApi="${ForearmYawApi}"/>
     <xacro:index_finger_transmissions_hw prefix="${prefix}" />
     <xacro:middle_finger_transmissions_hw prefix="${prefix}" />

Commit message: updated forearm urdf for proper visualization

File: model/robots/forearm_left.xacro (robot description, xacro)
@@ -7,8 +7,8 @@
     <link name="world"/>
     <xacro:make_lower_arm prefix="${prefix}" reflect="${reflect}" lower_arm_root_link="world"/>
-    <xacro:make_thumb prefix="${prefix}" reflect="-1" thumb_root_link="${prefix}Palm"/>
-    <xacro:make_index_finger prefix="${prefix}" reflect="-1" index_finger_root_link="${prefix}Palm"/>
-    <xacro:make_middle_finger prefix="${prefix}" reflect="-1" middle_finger_root_link="${prefix}Palm"/>
-    <xacro:make_pinky_finger prefix="${prefix}" reflect="-1" pinky_finger_root_link="${prefix}Palm"/>
+    <xacro:make_thumb prefix="${prefix}" reflect="${reflect}" thumb_root_link="${prefix}Palm"/>
+    <xacro:make_index_finger prefix="${prefix}" reflect="${reflect}" index_finger_root_link="${prefix}Palm"/>
+    <xacro:make_middle_finger prefix="${prefix}" reflect="${reflect}" middle_finger_root_link="${prefix}Palm"/>
+    <xacro:make_pinky_finger prefix="${prefix}" reflect="${reflect}" pinky_finger_root_link="${prefix}Palm"/>
     <xacro:simple_position_transmission jointName="${ForearmYawActuatorName}" actuatorName="${ForearmYawActuatorName}" nodeName="${ForearmYawNode}" actuatorApi="${ForearmYawApi}"/>
     <xacro:index_finger_transmissions_hw prefix="${prefix}" />

File: model/robots/forearm_right.xacro (robot description, xacro)
@@ -4,11 +4,11 @@
     <xacro:include filename="$(find val_description)/model/robots/common/xacro/common_bodies.xacro" />
     <xacro:property name="prefix" value="right"/>
-    <xacro:property name="reflect" value="1"/>
+    <xacro:property name="reflect" value="-1"/>
     <link name="world"/>
     <xacro:make_lower_arm prefix="${prefix}" reflect="${reflect}" lower_arm_root_link="world"/>
-    <xacro:make_thumb prefix="${prefix}" reflect="-1" thumb_root_link="${prefix}Palm"/>
-    <xacro:make_index_finger prefix="${prefix}" reflect="-1" index_finger_root_link="${prefix}Palm"/>
-    <xacro:make_middle_finger prefix="${prefix}" reflect="-1" middle_finger_root_link="${prefix}Palm"/>
-    <xacro:make_pinky_finger prefix="${prefix}" reflect="-1" pinky_finger_root_link="${prefix}Palm"/>
+    <xacro:make_thumb prefix="${prefix}" reflect="${reflect}" thumb_root_link="${prefix}Palm"/>
+    <xacro:make_index_finger prefix="${prefix}" reflect="${reflect}" index_finger_root_link="${prefix}Palm"/>
+    <xacro:make_middle_finger prefix="${prefix}" reflect="${reflect}" middle_finger_root_link="${prefix}Palm"/>
+    <xacro:make_pinky_finger prefix="${prefix}" reflect="${reflect}" pinky_finger_root_link="${prefix}Palm"/>
     <xacro:simple_position_transmission jointName="${ForearmYawActuatorName}" actuatorName="${ForearmYawActuatorName}" nodeName="${ForearmYawNode}" actuatorApi="${ForearmYawApi}"/>
     <xacro:index_finger_transmissions_hw prefix="${prefix}" />
