Commit message: Have instance file for unit D. Only have serials for F/T sensors.

File: common/xacro/serial_numbers/valkyrie_D_serials.xacro (robot description, xacro)
@@ -4,12 +4,12 @@
     <xacro:property name="leftLegJ3SerialNumber" value="UNKNOWN" />
     <xacro:property name="leftLegJ4SerialNumber" value="UNKNOWN" />
-    <xacro:property name="leftAnkleLeftActuatorSerialNumber" value="v_e_009" />
-    <xacro:property name="leftAnkleRightActuatorSerialNumber" value="v_e_010" />
+    <xacro:property name="leftAnkleLeftActuatorSerialNumber" value="UNKNOWN" />
+    <xacro:property name="leftAnkleRightActuatorSerialNumber" value="UNKNOWN" />
     <xacro:property name="rightLegJ1SerialNumber" value="UNKNOWN" />
     <xacro:property name="rightLegJ2SerialNumber" value="UNKNOWN" />
     <xacro:property name="rightLegJ3SerialNumber" value="UNKNOWN" />
     <xacro:property name="rightLegJ4SerialNumber" value="UNKNOWN" />
-    <xacro:property name="rightAnkleLeftActuatorSerialNumber" value="v_e_018" />
-    <xacro:property name="rightAnkleRightActuatorSerialNumber" value="v_e_017" />
+    <xacro:property name="rightAnkleLeftActuatorSerialNumber" value="UNKNOWN" />
+    <xacro:property name="rightAnkleRightActuatorSerialNumber" value="UNKNOWN" />
     <xacro:property name="leftArmJ1SerialNumber" value="UNKNOWN" />
     <xacro:property name="leftArmJ2SerialNumber" value="UNKNOWN" />
@@ -26,16 +26,16 @@
     <xacro:property name="rightWristTopActuatorSerialNumber" value="UNKNOWN" />
     <xacro:property name="rightWristBottomActuatorSerialNumber" value="UNKNOWN" />
-    <xacro:property name="neckJ1SerialNumber" value="v_g_001" />
-    <xacro:property name="neckJ2SerialNumber" value="v_g_002" />
-    <xacro:property name="neckJ3SerialNumber" value="v_g_004" />
-    <xacro:property name="trunkSerialNumber" value="v_a_011" />
-    <xacro:property name="waistRightActuatorSerialNumber" value="v_e_014" />
-    <xacro:property name="waistLeftActuatorSerialNumber" value="v_e_013" />
+    <xacro:property name="neckJ1SerialNumber" value="UNKNOWN" />
+    <xacro:property name="neckJ2SerialNumber" value="UNKNOWN" />
+    <xacro:property name="neckJ3SerialNumber" value="UNKNOWN" />
+    <xacro:property name="trunkSerialNumber" value="UNKNOWN" />
+    <xacro:property name="waistRightActuatorSerialNumber" value="UNKNOWN" />
+    <xacro:property name="waistLeftActuatorSerialNumber" value="UNKNOWN" />
     <xacro:property name="pelvis_middle_imu_serial" value="UNKNOWN" />
     <xacro:property name="pelvis_rear_imu_serial" value="UNKNOWN" />
     <xacro:property name="torso_left_imu_serial" value="UNKNOWN" />
     <xacro:property name="torso_right_imu_serial" value="UNKNOWN" />
-    <xacro:property name="left_foot_ATI_serial" value="FT17212" />
-    <xacro:property name="right_foot_ATI_serial" value="FT17214" />
+    <xacro:property name="left_foot_ATI_serial" value="FT14182" />
+    <xacro:property name="right_foot_ATI_serial" value="FT14019" />
     <xacro:property name="sim_ATI_serial" value="FT001SIM" />
 </robot>

File: instance/instances/robots/xacro/common/valkyrie_full_template.xacro (robot description, xacro)
@@ -7,5 +7,5 @@
 	<xacro:include filename="$(find val_description)/instance/instances/robots/xacro/sensors/imu.xacro" />
 	<xacro:include filename="$(find val_description)/instance/instances/robots/xacro/sensors/ati_force_torque.xacro" />
-	<RobotInstance id="valkyrie_A" />
+	<RobotInstance id="${instance}" />
 	<xacro:all_channels/>
 	<Mechanisms>

Commit message: updaded valkyire d serials

File: common/xacro/serial_numbers/valkyrie_D_serials.xacro (robot description, xacro)
@@ -1,41 +1,41 @@
 <robot xmlns:xacro="http://ros.org/wiki/xacro" name="valkyrie_C_serials">
-    <xacro:property name="leftLegJ1SerialNumber" value="UNKNOWN" />
-    <xacro:property name="leftLegJ2SerialNumber" value="UNKNOWN" />
-    <xacro:property name="leftLegJ3SerialNumber" value="UNKNOWN" />
-    <xacro:property name="leftLegJ4SerialNumber" value="UNKNOWN" />
-    <xacro:property name="leftAnkleLeftActuatorSerialNumber" value="UNKNOWN" />
-    <xacro:property name="leftAnkleRightActuatorSerialNumber" value="UNKNOWN" />
-    <xacro:property name="rightLegJ1SerialNumber" value="UNKNOWN" />
-    <xacro:property name="rightLegJ2SerialNumber" value="UNKNOWN" />
-    <xacro:property name="rightLegJ3SerialNumber" value="UNKNOWN" />
-    <xacro:property name="rightLegJ4SerialNumber" value="UNKNOWN" />
-    <xacro:property name="rightAnkleLeftActuatorSerialNumber" value="UNKNOWN" />
-    <xacro:property name="rightAnkleRightActuatorSerialNumber" value="UNKNOWN" />
-    <xacro:property name="leftArmJ1SerialNumber" value="UNKNOWN" />
-    <xacro:property name="leftArmJ2SerialNumber" value="UNKNOWN" />
-    <xacro:property name="leftArmJ3SerialNumber" value="UNKNOWN" />
-    <xacro:property name="leftArmJ4SerialNumber" value="UNKNOWN" />
-    <xacro:property name="leftArmJ5SerialNumber" value="UNKNOWN" />
-    <xacro:property name="leftWristTopActuatorSerialNumber" value="UNKNOWN" />
-    <xacro:property name="leftWristBottomActuatorSerialNumber" value="UNKNOWN" />
-    <xacro:property name="rightArmJ1SerialNumber" value="UNKNOWN" />
-    <xacro:property name="rightArmJ2SerialNumber" value="UNKNOWN" />
-    <xacro:property name="rightArmJ3SerialNumber" value="UNKNOWN" />
-    <xacro:property name="rightArmJ4SerialNumber" value="UNKNOWN" />
-    <xacro:property name="rightArmJ5SerialNumber" value="UNKNOWN" />
-    <xacro:property name="rightWristTopActuatorSerialNumber" value="UNKNOWN" />
-    <xacro:property name="rightWristBottomActuatorSerialNumber" value="UNKNOWN" />
-    <xacro:property name="neckJ1SerialNumber" value="UNKNOWN" />
-    <xacro:property name="neckJ2SerialNumber" value="UNKNOWN" />
-    <xacro:property name="neckJ3SerialNumber" value="UNKNOWN" />
-    <xacro:property name="trunkSerialNumber" value="UNKNOWN" />
-    <xacro:property name="waistRightActuatorSerialNumber" value="UNKNOWN" />
-    <xacro:property name="waistLeftActuatorSerialNumber" value="UNKNOWN" />
-    <xacro:property name="pelvis_middle_imu_serial" value="UNKNOWN" />
-    <xacro:property name="pelvis_rear_imu_serial" value="UNKNOWN" />
-    <xacro:property name="torso_left_imu_serial" value="UNKNOWN" />
-    <xacro:property name="torso_right_imu_serial" value="UNKNOWN" />
-    <xacro:property name="left_foot_ATI_serial" value="FT14182" />
-    <xacro:property name="right_foot_ATI_serial" value="FT14019" />
-    <xacro:property name="sim_ATI_serial" value="FT001SIM" />
+	<xacro:property name="leftLegJ1SerialNumber" value="v_a_017" />
+	<xacro:property name="leftLegJ2SerialNumber" value="v_b_016" />
+	<xacro:property name="leftLegJ3SerialNumber" value="v_c_008" />
+	<xacro:property name="leftLegJ4SerialNumber" value="v_d_008" />
+	<xacro:property name="leftAnkleLeftActuatorSerialNumber" value="v_e_019" />
+	<xacro:property name="leftAnkleRightActuatorSerialNumber" value="v_e_020" />
+	<xacro:property name="rightLegJ1SerialNumber" value="v_a_018" />
+	<xacro:property name="rightLegJ2SerialNumber" value="v_b_015" />
+	<xacro:property name="rightLegJ3SerialNumber" value="v_c_009" />
+	<xacro:property name="rightLegJ4SerialNumber" value="v_d_009" />
+	<xacro:property name="rightAnkleLeftActuatorSerialNumber" value="v_e_022" />
+	<xacro:property name="rightAnkleRightActuatorSerialNumber" value="v_e_021" />
+	<xacro:property name="leftArmJ1SerialNumber" value="v_a_019" />
+	<xacro:property name="leftArmJ2SerialNumber" value="v_b_014" />
+	<xacro:property name="leftArmJ3SerialNumber" value="v_f_017" />
+	<xacro:property name="leftArmJ4SerialNumber" value="v_f_016" />
+	<xacro:property name="leftArmJ5SerialNumber" value="UNKNOWN" />
+	<xacro:property name="leftWristTopActuatorSerialNumber" value="UNKNOWN" />
+	<xacro:property name="leftWristBottomActuatorSerialNumber" value="UNKNOWN" />
+	<xacro:property name="rightArmJ1SerialNumber" value="v_a_016" />
+	<xacro:property name="rightArmJ2SerialNumber" value="v_b_013" />
+	<xacro:property name="rightArmJ3SerialNumber" value="v_f_018" />
+	<xacro:property name="rightArmJ4SerialNumber" value="v_f_015" />
+	<xacro:property name="rightArmJ5SerialNumber" value="UNKNOWN" />
+	<xacro:property name="rightWristTopActuatorSerialNumber" value="UNKNOWN" />
+	<xacro:property name="rightWristBottomActuatorSerialNumber" value="UNKNOWN" />
+	<xacro:property name="neckJ1SerialNumber" value="UNKNOWN" />
+	<xacro:property name="neckJ2SerialNumber" value="UNKNOWN" />
+	<xacro:property name="neckJ3SerialNumber" value="UNKNOWN" />
+	<xacro:property name="trunkSerialNumber" value="v_a_020" />
+	<xacro:property name="waistRightActuatorSerialNumber" value="v_e_023" />
+	<xacro:property name="waistLeftActuatorSerialNumber" value="v_e_024" />
+	<xacro:property name="pelvis_middle_imu_serial" value="UNKNOWN" />
+	<xacro:property name="pelvis_rear_imu_serial" value="UNKNOWN" />
+	<xacro:property name="torso_left_imu_serial" value="UNKNOWN" />
+	<xacro:property name="torso_right_imu_serial" value="UNKNOWN" />
+	<xacro:property name="left_foot_ATI_serial" value="FT17212" />
+	<xacro:property name="right_foot_ATI_serial" value="FT17214" />
+	<xacro:property name="sim_ATI_serial" value="FT001SIM" />
 </robot>

Commit message: Fixed a ton of actuator coeffs. Mostly fixing the velocity signal source.

File: common/xacro/serial_numbers/valkyrie_D_serials.xacro (robot description, xacro)
@@ -26,7 +26,7 @@
     <xacro:property name="rightWristTopActuatorSerialNumber" value="UNKNOWN" />
     <xacro:property name="rightWristBottomActuatorSerialNumber" value="UNKNOWN" />
-    <xacro:property name="neckJ1SerialNumber" value="v_g_012" />
+    <xacro:property name="neckJ1SerialNumber" value="v_g_014" />
     <xacro:property name="neckJ2SerialNumber" value="v_g_013" />
-    <xacro:property name="neckJ3SerialNumber" value="v_g_014" />
+    <xacro:property name="neckJ3SerialNumber" value="v_g_015" />
     <xacro:property name="trunkSerialNumber" value="v_a_020" />
     <xacro:property name="waistRightActuatorSerialNumber" value="v_e_023" />

Commit message: added instance for just forearems

File: common/xacro/serial_numbers/valkyrie_D_serials.xacro (robot description, xacro)
@@ -16,10 +16,10 @@
     <xacro:property name="leftArmJ3SerialNumber" value="v_f_017" />
     <xacro:property name="leftArmJ4SerialNumber" value="v_f_016" />
-    <xacro:property name="leftArmJ5SerialNumber" value="UNKNOWN" />
+    <xacro:property name="leftArmJ5SerialNumber" value="v_g_016" />
     <xacro:property name="rightArmJ1SerialNumber" value="v_a_016" />
     <xacro:property name="rightArmJ2SerialNumber" value="v_b_013" />
     <xacro:property name="rightArmJ3SerialNumber" value="v_f_018" />
     <xacro:property name="rightArmJ4SerialNumber" value="v_f_015" />
-    <xacro:property name="rightArmJ5SerialNumber" value="UNKNOWN" />
+    <xacro:property name="rightArmJ5SerialNumber" value="v_g_012" />
     <xacro:property name="neckJ1SerialNumber" value="v_g_014" />
     <xacro:property name="neckJ2SerialNumber" value="v_g_013" />
