Commit message: updated xacros to reference the correct force torque calibration files in simulation

File: common/xacro/serial_numbers/valkyrie_A_serials.xacro (robot description, xacro)
@@ -38,3 +38,4 @@
 	<xacro:property name="left_foot_ATI_serial" value="FT14020" />
 	<xacro:property name="right_foot_ATI_serial" value="FT16592" />
+	<xacro:property name="sim_ATI_serial" value="FT001SIM" />
 </robot>

File: common/xacro/serial_numbers/valkyrie_B_serials.xacro (robot description, xacro)
@@ -38,3 +38,4 @@
 	<xacro:property name="left_foot_ATI_serial" value="FT17219" />
 	<xacro:property name="right_foot_ATI_serial" value="FT17215" />
+    <xacro:property name="sim_ATI_serial" value="FT001SIM" />
 </robot>

File: common/xacro/serial_numbers/valkyrie_C_serials.xacro (robot description, xacro)
@@ -38,3 +38,4 @@
 	<xacro:property name="left_foot_ATI_serial" value="UNKNOWN" />
 	<xacro:property name="right_foot_ATI_serial" value="UNKNOWN" />
+	<xacro:property name="sim_ATI_serial" value="FT001SIM" />
 </robot>

File: model/robots/common/xacro/valkyrie_base_sim.xacro (robot description, xacro)
@@ -16,6 +16,6 @@
     <xacro:make_leg prefix="left" reflect="1" leg_root_link="${Pelvis_Link_Name}"/>
     <xacro:v1_pelvis_sensors />
-    <xacro:v1_leg_sensors prefix="left" reflect="1" ATI_serial_number="${left_foot_ATI_serial}" ATI_node="${left_foot_ATI_node}"/>
-    <xacro:v1_leg_sensors prefix="right" reflect="-1" ATI_serial_number="${right_foot_ATI_serial}" ATI_node="${right_foot_ATI_node}"/>
+    <xacro:v1_leg_sensors prefix="left" reflect="1" ATI_serial_number="${sim_ATI_serial}" ATI_node="${left_foot_ATI_node}"/>
+    <xacro:v1_leg_sensors prefix="right" reflect="-1" ATI_serial_number="${sim_ATI_serial}" ATI_node="${right_foot_ATI_node}"/>
     <xacro:include_multisense_sim />
     <xacro:v1_trunk_sensors/>

Commit message: Updated serials for instance file for unit D. Also removed the imu serials from xacro's since they were not being used.

File: common/xacro/serial_numbers/valkyrie_A_serials.xacro (robot description, xacro)
@@ -32,8 +32,4 @@
 	<xacro:property name="waistRightActuatorSerialNumber" value="v_e_005" />
 	<xacro:property name="waistLeftActuatorSerialNumber" value="v_e_006" />
-	<xacro:property name="pelvis_middle_imu_serial" value="UNKNOWN" />
-	<xacro:property name="pelvis_rear_imu_serial" value="UNKNOWN" />
-	<xacro:property name="torso_left_imu_serial" value="UNKNOWN" />
-	<xacro:property name="torso_right_imu_serial" value="UNKNOWN" />
 	<xacro:property name="left_foot_ATI_serial" value="FT14020" />
 	<xacro:property name="right_foot_ATI_serial" value="FT16592" />

File: common/xacro/serial_numbers/valkyrie_B_serials.xacro (robot description, xacro)
@@ -32,8 +32,4 @@
 	<xacro:property name="waistRightActuatorSerialNumber" value="v_e_011" />
 	<xacro:property name="waistLeftActuatorSerialNumber" value="v_e_012" />
-	<xacro:property name="pelvis_middle_imu_serial" value="UNKNOWN" />
-	<xacro:property name="pelvis_rear_imu_serial" value="UNKNOWN" />
-	<xacro:property name="torso_left_imu_serial" value="UNKNOWN" />
-	<xacro:property name="torso_right_imu_serial" value="UNKNOWN" />
 	<xacro:property name="left_foot_ATI_serial" value="FT17219" />
 	<xacro:property name="right_foot_ATI_serial" value="FT17217" />

File: common/xacro/serial_numbers/valkyrie_C_serials.xacro (robot description, xacro)
@@ -32,8 +32,4 @@
 	<xacro:property name="waistRightActuatorSerialNumber" value="v_e_014" />
 	<xacro:property name="waistLeftActuatorSerialNumber" value="v_e_013" />
-	<xacro:property name="pelvis_middle_imu_serial" value="UNKNOWN" />
-	<xacro:property name="pelvis_rear_imu_serial" value="UNKNOWN" />
-	<xacro:property name="torso_left_imu_serial" value="UNKNOWN" />
-	<xacro:property name="torso_right_imu_serial" value="UNKNOWN" />
 	<xacro:property name="left_foot_ATI_serial" value="FT17212" />
 	<xacro:property name="right_foot_ATI_serial" value="FT17214" />

File: common/xacro/serial_numbers/valkyrie_D_serials.xacro (robot description, xacro)
@@ -1,39 +1,35 @@
 <robot xmlns:xacro="http://ros.org/wiki/xacro" name="valkyrie_C_serials">
-    <xacro:property name="leftLegJ1SerialNumber" value="UNKNOWN" />
-    <xacro:property name="leftLegJ2SerialNumber" value="UNKNOWN" />
-    <xacro:property name="leftLegJ3SerialNumber" value="UNKNOWN" />
-    <xacro:property name="leftLegJ4SerialNumber" value="UNKNOWN" />
-    <xacro:property name="leftAnkleLeftActuatorSerialNumber" value="UNKNOWN" />
-    <xacro:property name="leftAnkleRightActuatorSerialNumber" value="UNKNOWN" />
-    <xacro:property name="rightLegJ1SerialNumber" value="UNKNOWN" />
-    <xacro:property name="rightLegJ2SerialNumber" value="UNKNOWN" />
-    <xacro:property name="rightLegJ3SerialNumber" value="UNKNOWN" />
-    <xacro:property name="rightLegJ4SerialNumber" value="UNKNOWN" />
-    <xacro:property name="rightAnkleLeftActuatorSerialNumber" value="UNKNOWN" />
-    <xacro:property name="rightAnkleRightActuatorSerialNumber" value="UNKNOWN" />
-    <xacro:property name="leftArmJ1SerialNumber" value="UNKNOWN" />
-    <xacro:property name="leftArmJ2SerialNumber" value="UNKNOWN" />
-    <xacro:property name="leftArmJ3SerialNumber" value="UNKNOWN" />
-    <xacro:property name="leftArmJ4SerialNumber" value="UNKNOWN" />
+    <xacro:property name="leftLegJ1SerialNumber" value="v_a_017" />
+    <xacro:property name="leftLegJ2SerialNumber" value="v_b_016" />
+    <xacro:property name="leftLegJ3SerialNumber" value="v_c_008" />
+    <xacro:property name="leftLegJ4SerialNumber" value="v_d_008" />
+    <xacro:property name="leftAnkleLeftActuatorSerialNumber" value="v_e_019" />
+    <xacro:property name="leftAnkleRightActuatorSerialNumber" value="v_e_020" />
+    <xacro:property name="rightLegJ1SerialNumber" value="v_a_018" />
+    <xacro:property name="rightLegJ2SerialNumber" value="v_b_015" />
+    <xacro:property name="rightLegJ3SerialNumber" value="v_c_009" />
+    <xacro:property name="rightLegJ4SerialNumber" value="v_d_005" />
+    <xacro:property name="rightAnkleLeftActuatorSerialNumber" value="v_e_022" />
+    <xacro:property name="rightAnkleRightActuatorSerialNumber" value="v_e_021" />
+    <xacro:property name="leftArmJ1SerialNumber" value="v_a_019" />
+    <xacro:property name="leftArmJ2SerialNumber" value="v_b_014" />
+    <xacro:property name="leftArmJ3SerialNumber" value="v_f_017" />
+    <xacro:property name="leftArmJ4SerialNumber" value="v_f_016" />
     <xacro:property name="leftArmJ5SerialNumber" value="UNKNOWN" />
     <xacro:property name="leftWristTopActuatorSerialNumber" value="UNKNOWN" />
     <xacro:property name="leftWristBottomActuatorSerialNumber" value="UNKNOWN" />
-    <xacro:property name="rightArmJ1SerialNumber" value="UNKNOWN" />
-    <xacro:property name="rightArmJ2SerialNumber" value="UNKNOWN" />
-    <xacro:property name="rightArmJ3SerialNumber" value="UNKNOWN" />
-    <xacro:property name="rightArmJ4SerialNumber" value="UNKNOWN" />
+    <xacro:property name="rightArmJ1SerialNumber" value="v_a_016" />
+    <xacro:property name="rightArmJ2SerialNumber" value="v_b_013" />
+    <xacro:property name="rightArmJ3SerialNumber" value="v_f_018" />
+    <xacro:property name="rightArmJ4SerialNumber" value="v_f_015" />
     <xacro:property name="rightArmJ5SerialNumber" value="UNKNOWN" />
     <xacro:property name="rightWristTopActuatorSerialNumber" value="UNKNOWN" />
     <xacro:property name="rightWristBottomActuatorSerialNumber" value="UNKNOWN" />
-    <xacro:property name="neckJ1SerialNumber" value="UNKNOWN" />
-    <xacro:property name="neckJ2SerialNumber" value="UNKNOWN" />
-    <xacro:property name="neckJ3SerialNumber" value="UNKNOWN" />
-    <xacro:property name="trunkSerialNumber" value="UNKNOWN" />
-    <xacro:property name="waistRightActuatorSerialNumber" value="UNKNOWN" />
-    <xacro:property name="waistLeftActuatorSerialNumber" value="UNKNOWN" />
-    <xacro:property name="pelvis_middle_imu_serial" value="UNKNOWN" />
-    <xacro:property name="pelvis_rear_imu_serial" value="UNKNOWN" />
-    <xacro:property name="torso_left_imu_serial" value="UNKNOWN" />
-    <xacro:property name="torso_right_imu_serial" value="UNKNOWN" />
+    <xacro:property name="neckJ1SerialNumber" value="v_g_012" />
+    <xacro:property name="neckJ2SerialNumber" value="v_g_013" />
+    <xacro:property name="neckJ3SerialNumber" value="v_g_014" />
+    <xacro:property name="trunkSerialNumber" value="v_a_020" />
+    <xacro:property name="waistRightActuatorSerialNumber" value="v_e_023" />
+    <xacro:property name="waistLeftActuatorSerialNumber" value="v_e_024" />
     <xacro:property name="left_foot_ATI_serial" value="FT14182" />
     <xacro:property name="right_foot_ATI_serial" value="FT14019" />

File: instance/instances/robots/xacro/common/valkyrie_full_template.xacro (robot description, xacro)
@@ -18,7 +18,4 @@
 	</Mechanisms>
 	<Devices>
-		<xacro:microstrain_imu name="pelvis_middle_imu" serial_number="${pelvis_middle_imu_serial}" node="${pelvis_middle_imu_node}" />
-		<xacro:microstrain_imu name="pelvis_rear_imu" serial_number="${pelvis_rear_imu_serial}" node="${pelvis_rear_imu_node}" />
-		<xacro:microstrain_imu name="torso_left_imu" serial_number="${torso_left_imu_serial}" node="${torso_left_imu_node}" />
 		<xacro:ati_force_torque name="left_foot_force_torque" serial_number="${left_foot_ATI_serial}" node="${left_foot_ATI_node}"/>
 		<xacro:ati_force_torque name="right_foot_force_torque" serial_number="${right_foot_ATI_serial}" node="${right_foot_ATI_node}"/>

Commit message: updated imu xacro to contain serial

File: common/xacro/serial_numbers/valkyrie_A_serials.xacro (robot description, xacro)
@@ -32,4 +32,6 @@
 	<xacro:property name="left_foot_ATI_serial" value="FT14020" />
 	<xacro:property name="right_foot_ATI_serial" value="FT16592" />
+	<xacro:property name="rear_pelvis_IMU_serial" value="UNKNOWN" />
+	<xacro:property name="left_torso_IMU_serial" value="UNKNOWN" />
 	<xacro:property name="sim_ATI_serial" value="FT001SIM" />
 </robot>

File: common/xacro/serial_numbers/valkyrie_B_serials.xacro (robot description, xacro)
@@ -32,4 +32,6 @@
 	<xacro:property name="left_foot_ATI_serial" value="FT17218" />
 	<xacro:property name="right_foot_ATI_serial" value="FT14018" />
+	<xacro:property name="rear_pelvis_IMU_serial" value="UNKNOWN" />
+	<xacro:property name="left_torso_IMU_serial" value="UNKNOWN" />
     <xacro:property name="sim_ATI_serial" value="FT001SIM" />
 </robot>

File: common/xacro/serial_numbers/valkyrie_C_serials.xacro (robot description, xacro)
@@ -32,4 +32,6 @@
 	<xacro:property name="left_foot_ATI_serial" value="FT16594" />
 	<xacro:property name="right_foot_ATI_serial" value="FT17214" />
+	<xacro:property name="rear_pelvis_IMU_serial" value="47251" />
+	<xacro:property name="left_torso_IMU_serial" value="47251" />
 	<xacro:property name="sim_ATI_serial" value="FT001SIM" />
 </robot>

File: common/xacro/serial_numbers/valkyrie_D_serials.xacro (robot description, xacro)
@@ -32,4 +32,6 @@
     <xacro:property name="left_foot_ATI_serial" value="FT17212" />
     <xacro:property name="right_foot_ATI_serial" value="FT16590" />
+    <xacro:property name="rear_pelvis_IMU_serial" value="UNKNOWN" />
+    <xacro:property name="left_torso_IMU_serial" value="UNKNOWN" />
     <xacro:property name="sim_ATI_serial" value="FT001SIM" />
 </robot>

File: model/robots/common/xacro/pelvis/pelvis.xacro (robot description, xacro)
@@ -21,5 +21,5 @@
                                   origin_rpy="0.0 0.0 0.7854" />
     </xacro:macro>
-    <xacro:macro name="v1_pelvis_middle_sensors_usb" params="sensor_node_tag sensor_api_tag sensor_port_tag">
+    <xacro:macro name="v1_pelvis_middle_sensors_usb" params="sensor_node_tag sensor_api_tag sensor_port_tag sensor_number_tag">
         <xacro:microstrain_sensor sensorName="pelvisRearImu"
                                   parentLink="${Pelvis_Link_Name}"
@@ -32,7 +32,8 @@
                                   sensor_node="${sensor_node_tag}"
                                   sensor_api="${sensor_api_tag}"
-                                  sensor_port="${sensor_port_tag}" />
+                                  sensor_port="${sensor_port_tag}"
+                                  sensor_number="${sensor_number_tag}"/>
     </xacro:macro>
-    <xacro:macro name="v1_pelvis_rear_sensors_usb" params="sensor_node_tag sensor_api_tag sensor_port_tag">
+    <xacro:macro name="v1_pelvis_rear_sensors_usb" params="sensor_node_tag sensor_api_tag sensor_port_tag sensor_number_tag">
         <xacro:usb_microstrain_sensor sensorName="pelvisRearImu"
                                   parentLink="${Pelvis_Link_Name}"
@@ -41,5 +42,6 @@
                         				  sensor_node="${sensor_node_tag}"
                         				  sensor_api="${sensor_api_tag}"
-                        				  sensor_port="${sensor_port_tag}" />
+                        				  sensor_port="${sensor_port_tag}"
+                                  sensor_number="${sensor_number_tag}" />
         <xacro:microstrain_sensor sensorName="pelvisMiddleImu"
                                   parentLink="${Pelvis_Link_Name}"
@@ -47,5 +49,5 @@
                                   origin_rpy="3.14159 0.0 0.0" />
     </xacro:macro>
-    <xacro:macro name="v1_pelvis_sensors_usb" params="middle_sensor_node_tag middle_sensor_api_tag middle_sensor_port_tag rear_sensor_node_tag rear_sensor_api_tag rear_sensor_port_tag">
+    <xacro:macro name="v1_pelvis_sensors_usb" params="middle_sensor_node_tag middle_sensor_api_tag middle_sensor_port_tag rear_sensor_node_tag rear_sensor_api_tag rear_sensor_port_tag sensor_number_tag" >
         <xacro:usb_microstrain_sensor sensorName="pelvisRearImu"
                                   parentLink="${Pelvis_Link_Name}"
@@ -54,5 +56,6 @@
                                   sensor_node="${rear_sensor_node_tag}"
                                   sensor_api="${rear_sensor_api_tag}"
-                                  sensor_port="${rear_sensor_port_tag}" />
+                                  sensor_port="${rear_sensor_port_tag}"
+                                  sensor_number="${sensor_number_tag}" />
         <xacro:usb_microstrain_sensor sensorName="pelvisMiddleImu"
                                   parentLink="${Pelvis_Link_Name}"
@@ -61,5 +64,6 @@
                                   sensor_node="${middle_sensor_node_tag}"
                                   sensor_api="${middle_sensor_api_tag}"
-                                  sensor_port="${middle_sensor_port_tag}" />
+                                  sensor_port="${middle_sensor_port_tag}"
+                                  sensor_number="${sensor_number_tag}" />
     </xacro:macro>
 </robot>

File: model/robots/common/xacro/sensors/microstrain.xacro (robot description, xacro)
@@ -43,5 +43,5 @@
     </gazebo>
   </xacro:macro>
-  <xacro:macro name="usb_microstrain_sensor" params="sensorName parentLink origin_xyz origin_rpy sensor_node sensor_api sensor_port">
+  <xacro:macro name="usb_microstrain_sensor" params="sensorName parentLink origin_xyz origin_rpy sensor_node sensor_api sensor_port sensor_number">
     <xacro:massless_virtual_link name="${sensorName}_Frame"
                     origin_rpy="0 0 0"
@@ -68,4 +68,5 @@
         <api name="${sensor_api}" />
         <port name="${sensor_port}" />
+        <sensor_number id="${sensor_number}"/>
         <imu>
            <noise>

File: model/robots/common/xacro/valkyrie_base_hw.xacro (robot description, xacro)
@@ -15,9 +15,9 @@
     <xacro:make_leg prefix="right" reflect="-1" leg_root_link="${Pelvis_Link_Name}"/>
     <xacro:make_leg prefix="left" reflect="1" leg_root_link="${Pelvis_Link_Name}"/>
-    <xacro:v1_trunk_sensors_usb sensor_node_tag="${torso_left_imu_node}" sensor_api_tag="${ImuMicrostrainHardwareApi}" sensor_port_tag="${torso_left_imu_port}"/>
+    <xacro:v1_trunk_sensors_usb sensor_node_tag="${torso_left_imu_node}" sensor_api_tag="${ImuMicrostrainHardwareApi}" sensor_port_tag="${torso_left_imu_port}" sensor_number_tag="${left_torso_IMU_serial}"/>
     <xacro:v1_leg_sensors prefix="left" reflect="1" ATI_serial_number="${left_foot_ATI_serial}" ATI_node="${left_foot_ATI_node}"/>
     <xacro:v1_leg_sensors prefix="right" reflect="-1" ATI_serial_number="${right_foot_ATI_serial}" ATI_node="${right_foot_ATI_node}"/>
     <xacro:include_multisense_hw />
-    <xacro:v1_pelvis_rear_sensors_usb sensor_node_tag="${pelvis_rear_imu_node}" sensor_api_tag="${ImuMicrostrainHardwareApi}"  sensor_port_tag="${pelvis_rear_imu_port}"/>
+    <xacro:v1_pelvis_rear_sensors_usb sensor_node_tag="${pelvis_rear_imu_node}" sensor_api_tag="${ImuMicrostrainHardwareApi}"  sensor_port_tag="${pelvis_rear_imu_port}" sensor_number_tag="${rear_pelvis_IMU_serial}"/>
     <xacro:waist_transmissions_hw />
     <xacro:leg_transmissions_hw prefix="left"/>

File: model/robots/common/xacro/valkyrie_base_sim.xacro (robot description, xacro)
@@ -20,9 +20,9 @@
     <xacro:make_leg prefix="right" reflect="-1" leg_root_link="${Pelvis_Link_Name}"/>
     <xacro:make_leg prefix="left" reflect="1" leg_root_link="${Pelvis_Link_Name}"/>
-    <xacro:v1_pelvis_sensors_usb middle_sensor_node_tag="${pelvis_middle_imu_node}" middle_sensor_api_tag="${ImuSensorSimApi}" middle_sensor_port_tag="${pelvis_middle_imu_port}" rear_sensor_node_tag="${pelvis_rear_imu_node}" rear_sensor_api_tag="${ImuSensorSimApi}" rear_sensor_port_tag="${pelvis_rear_imu_port}"/>
+    <xacro:v1_pelvis_sensors_usb middle_sensor_node_tag="${pelvis_middle_imu_node}" middle_sensor_api_tag="${ImuSensorSimApi}" middle_sensor_port_tag="${pelvis_middle_imu_port}" rear_sensor_node_tag="${pelvis_rear_imu_node}" rear_sensor_api_tag="${ImuSensorSimApi}" rear_sensor_port_tag="${pelvis_rear_imu_port}" sensor_number_tag="NONE"/>
     <xacro:v1_leg_sensors prefix="left" reflect="1" ATI_serial_number="${sim_ATI_serial}" ATI_node="${left_foot_Sim_ATI_node}"/>
     <xacro:v1_leg_sensors prefix="right" reflect="-1" ATI_serial_number="${sim_ATI_serial}" ATI_node="${right_foot_Sim_ATI_node}"/>
     <xacro:include_multisense_sim />
-    <xacro:v1_trunk_sensors_usb sensor_node_tag="${torso_left_imu_node}" sensor_api_tag="${ImuSensorSimApi}" sensor_port_tag="${torso_left_imu_port}"/>
+    <xacro:v1_trunk_sensors_usb sensor_node_tag="${torso_left_imu_node}" sensor_api_tag="${ImuSensorSimApi}" sensor_port_tag="${torso_left_imu_port}" sensor_number_tag="${rear_pelvis_IMU_serial}"/>
     <xacro:waist_transmissions_sim />
     <xacro:leg_transmissions_sim prefix="left"/>

File: model/robots/common/xacro/valkyrie_imu_base.xacro (robot description, xacro)
@@ -2,4 +2,4 @@
     <xacro:make_pelvis />
     <xacro:include_multisense_hw />
-    <xacro:v1_pelvis_middle_sensors_usb sensor_node_tag="${pelvis_middle_imu_node}" sensor_api_tag="${KVHHardwareApi}"  sensor_port_tag="${pelvis_middle_imu_port}"/>
+    <xacro:v1_pelvis_middle_sensors_usb sensor_node_tag="${pelvis_middle_imu_node}" sensor_api_tag="${KVHHardwareApi}"  sensor_port_tag="${pelvis_middle_imu_port}" sensor_number_tag="3dmConfigTest"/>
 </robot>

File: model/robots/common/xacro/valkyrie_no_hands_base_hw.xacro (robot description, xacro)
@@ -7,9 +7,9 @@
     <xacro:make_leg prefix="right" reflect="-1" leg_root_link="${Pelvis_Link_Name}"/>
     <xacro:make_leg prefix="left" reflect="1" leg_root_link="${Pelvis_Link_Name}"/>
-    <xacro:v1_trunk_sensors_usb sensor_node_tag="${torso_left_imu_node}" sensor_api_tag="${ImuMicrostrainHardwareApi}" sensor_port_tag="${torso_left_imu_port}"/>
+    <xacro:v1_trunk_sensors_usb sensor_node_tag="${torso_left_imu_node}" sensor_api_tag="${ImuMicrostrainHardwareApi}" sensor_port_tag="${torso_left_imu_port}" sensor_number_tag="${left_torso_IMU_serial}"/>
     <xacro:v1_leg_sensors prefix="left" reflect="1" ATI_serial_number="${left_foot_ATI_serial}" ATI_node="${left_foot_ATI_node}"/>
     <xacro:v1_leg_sensors prefix="right" reflect="-1" ATI_serial_number="${right_foot_ATI_serial}" ATI_node="${right_foot_ATI_node}"/>
     <xacro:include_multisense_hw />
-    <xacro:v1_pelvis_rear_sensors_usb sensor_node_tag="${pelvis_rear_imu_node}" sensor_api_tag="${ImuMicrostrainHardwareApi}"  sensor_port_tag="${pelvis_rear_imu_port}"/>
+    <xacro:v1_pelvis_rear_sensors_usb sensor_node_tag="${pelvis_rear_imu_node}" sensor_api_tag="${ImuMicrostrainHardwareApi}"  sensor_port_tag="${pelvis_rear_imu_port}" sensor_number_tag="${rear_pelvis_IMU_serial}"/>
     <xacro:waist_transmissions_hw />
     <xacro:leg_transmissions_hw prefix="left"/>

File: model/robots/common/xacro/waist/waist.xacro (robot description, xacro)
@@ -86,5 +86,5 @@
                         frameRate="60"/>
    </xacro:macro>
-  <xacro:macro name="v1_trunk_sensors_usb" params="sensor_node_tag sensor_api_tag sensor_port_tag">
+  <xacro:macro name="v1_trunk_sensors_usb" params="sensor_node_tag sensor_api_tag sensor_port_tag sensor_number_tag">
     <xacro:usb_microstrain_sensor sensorName="leftTorsoImu"
                               parentLink="${TorsoRollLinkName}"
@@ -93,5 +93,6 @@
                               sensor_node="${sensor_node_tag}"
                               sensor_api="${sensor_api_tag}"
-                              sensor_port="${sensor_port_tag}" />
+                              sensor_port="${sensor_port_tag}"
+                              sensor_number="${sensor_number_tag}" />
     <xacro:flea3_camera sensorName="rightHazardCamera"
                         parentLink="${TorsoRollLinkName}"
