Commit message: Removed a bunch of sim urdfs and condensed them into a single one. Also updated unit C's serials and created an urdf for it.

File: common/xacro/serial_numbers/valkyrie_C_serials.xacro (robot description, xacro)
@@ -1,41 +1,41 @@
 <robot xmlns:xacro="http://ros.org/wiki/xacro" name="valkyrie_C_serials">
-	<xacro:property name="leftLegJ1SerialNumber" value="UNKNOWN" />
-	<xacro:property name="leftLegJ2SerialNumber" value="UNKNOWN" />
-	<xacro:property name="leftLegJ3SerialNumber" value="UNKNOWN" />
-	<xacro:property name="leftLegJ4SerialNumber" value="UNKNOWN" />
-	<xacro:property name="leftAnkleLeftActuatorSerialNumber" value="UNKNOWN" />
-	<xacro:property name="leftAnkleRightActuatorSerialNumber" value="UNKNOWN" />
-	<xacro:property name="rightLegJ1SerialNumber" value="v_b_011" />
-	<xacro:property name="rightLegJ2SerialNumber" value="UNKNOWN" />
-	<xacro:property name="rightLegJ3SerialNumber" value="UNKNOWN" />
-	<xacro:property name="rightLegJ4SerialNumber" value="UNKNOWN" />
-	<xacro:property name="rightAnkleRightActuatorSerialNumber" value="UNKNOWN" />
-	<xacro:property name="rightAnkleLeftActuatorSerialNumber" value="UNKNOWN" />
-	<xacro:property name="leftArmJ1SerialNumber" value="UNKNOWN" />
-	<xacro:property name="leftArmJ2SerialNumber" value="UNKNOWN" />
-	<xacro:property name="leftArmJ3SerialNumber" value="UNKNOWN" />
-	<xacro:property name="leftArmJ4SerialNumber" value="UNKNOWN" />
+	<xacro:property name="leftLegJ1SerialNumber" value="v_a_015" />
+	<xacro:property name="leftLegJ2SerialNumber" value="v_b_011" />
+	<xacro:property name="leftLegJ3SerialNumber" value="v_c_007" />
+	<xacro:property name="leftLegJ4SerialNumber" value="v_d_007" />
+	<xacro:property name="leftAnkleLeftActuatorSerialNumber" value="v_e_009" />
+	<xacro:property name="leftAnkleRightActuatorSerialNumber" value="v_e_010" />
+	<xacro:property name="rightLegJ1SerialNumber" value="v_a_014" />
+	<xacro:property name="rightLegJ2SerialNumber" value="v_b_010" />
+	<xacro:property name="rightLegJ3SerialNumber" value="v_c_006" />
+	<xacro:property name="rightLegJ4SerialNumber" value="v_d_006" />
+	<xacro:property name="rightAnkleRightActuatorSerialNumber" value="v_e_008" />
+	<xacro:property name="rightAnkleLeftActuatorSerialNumber" value="v_e_007" />
+	<xacro:property name="leftArmJ1SerialNumber" value="v_a_013" />
+	<xacro:property name="leftArmJ2SerialNumber" value="v_b_009" />
+	<xacro:property name="leftArmJ3SerialNumber" value="v_f_012" />
+	<xacro:property name="leftArmJ4SerialNumber" value="v_f_011" />
 	<xacro:property name="leftArmJ5SerialNumber" value="UNKNOWN" />
 	<xacro:property name="leftWristTopActuatorSerialNumber" value="UNKNOWN" />
 	<xacro:property name="leftWristBottomActuatorSerialNumber" value="UNKNOWN" />
-	<xacro:property name="rightArmJ1SerialNumber" value="UNKNOWN" />
-	<xacro:property name="rightArmJ2SerialNumber" value="UNKNOWN" />
-	<xacro:property name="rightArmJ3SerialNumber" value="UNKNOWN" />
-	<xacro:property name="rightArmJ4SerialNumber" value="UNKNOWN" />
+	<xacro:property name="rightArmJ1SerialNumber" value="v_a_012" />
+	<xacro:property name="rightArmJ2SerialNumber" value="v_b_012" />
+	<xacro:property name="rightArmJ3SerialNumber" value="v_f_013" />
+	<xacro:property name="rightArmJ4SerialNumber" value="v_f_014" />
 	<xacro:property name="rightArmJ5SerialNumber" value="UNKNOWN" />
 	<xacro:property name="rightWristTopActuatorSerialNumber" value="UNKNOWN" />
 	<xacro:property name="rightWristBottomActuatorSerialNumber" value="UNKNOWN" />
-	<xacro:property name="neckJ1SerialNumber" value="UNKNOWN" />
-	<xacro:property name="neckJ2SerialNumber" value="UNKNOWN" />
-	<xacro:property name="neckJ3SerialNumber" value="UNKNOWN" />
-	<xacro:property name="trunkSerialNumber" value="UNKNOWN" />
-	<xacro:property name="waistRightActuatorSerialNumber" value="UNKNOWN" />
-	<xacro:property name="waistLeftActuatorSerialNumber" value="UNKNOWN" />
+	<xacro:property name="neckJ1SerialNumber" value="v_g_001" />
+	<xacro:property name="neckJ2SerialNumber" value="v_g_002" />
+	<xacro:property name="neckJ3SerialNumber" value="v_g_004" />
+	<xacro:property name="trunkSerialNumber" value="v_a_011" />
+	<xacro:property name="waistRightActuatorSerialNumber" value="v_e_014" />
+	<xacro:property name="waistLeftActuatorSerialNumber" value="v_e_013" />
 	<xacro:property name="pelvis_imu1_serial" value="UNKNOWN" />
 	<xacro:property name="pelvis_imu2_serial" value="UNKNOWN" />
 	<xacro:property name="torso_imu1_serial" value="UNKNOWN" />
 	<xacro:property name="torso_imu2_serial" value="UNKNOWN" />
-	<xacro:property name="left_foot_ATI_serial" value="UNKNOWN" />
-	<xacro:property name="right_foot_ATI_serial" value="UNKNOWN" />
+	<xacro:property name="left_foot_ATI_serial" value="FT17213" />
+	<xacro:property name="right_foot_ATI_serial" value="FT17217" />
 	<xacro:property name="sim_ATI_serial" value="FT001SIM" />
 </robot>

File: model/robots/valkyrie_A_sim.xacro (robot description, xacro)
@@ -1,3 +1,3 @@
-<robot xmlns:xacro="http://ros.org/wiki/xacro" name="valkyrie_A_sim">
+<robot xmlns:xacro="http://ros.org/wiki/xacro" name="valkyrie_sim">
     <xacro:property name="mesh_root" value="package://val_description/model/meshes"/>
     <xacro:include filename="$(find val_description)/model/robots/common/xacro/generic_models.xacro" />

Commit message: switch calibration file used in urdf for unit C

File: common/xacro/serial_numbers/valkyrie_C_serials.xacro (robot description, xacro)
@@ -36,6 +36,6 @@
 	<xacro:property name="torso_left_imu_serial" value="UNKNOWN" />
 	<xacro:property name="torso_right_imu_serial" value="UNKNOWN" />
-	<xacro:property name="left_foot_ATI_serial" value="FT17213" />
-	<xacro:property name="right_foot_ATI_serial" value="FT17215" />
+	<xacro:property name="left_foot_ATI_serial" value="FT17212" />
+	<xacro:property name="right_foot_ATI_serial" value="FT17214" />
 	<xacro:property name="sim_ATI_serial" value="FT001SIM" />
 </robot>

Commit message: updated coefs for unit B

File: common/xacro/serial_numbers/valkyrie_C_serials.xacro (robot description, xacro)
@@ -7,9 +7,9 @@
 	<xacro:property name="leftAnkleRightActuatorSerialNumber" value="v_e_010" />
 	<xacro:property name="rightLegJ1SerialNumber" value="v_a_014" />
-	<xacro:property name="rightLegJ2SerialNumber" value="v_b_007" />
-	<xacro:property name="rightLegJ3SerialNumber" value="v_c_003" />
-	<xacro:property name="rightLegJ4SerialNumber" value="v_d_002" />
-	<xacro:property name="rightAnkleLeftActuatorSerialNumber" value="v_e_018" />
-	<xacro:property name="rightAnkleRightActuatorSerialNumber" value="v_e_017" />
+	<xacro:property name="rightLegJ2SerialNumber" value="v_b_015" />
+	<xacro:property name="rightLegJ3SerialNumber" value="v_c_009" />
+	<xacro:property name="rightLegJ4SerialNumber" value="v_d_005" />
+	<xacro:property name="rightAnkleLeftActuatorSerialNumber" value="v_e_021" />
+	<xacro:property name="rightAnkleRightActuatorSerialNumber" value="v_e_022" />
 	<xacro:property name="leftArmJ1SerialNumber" value="v_a_013" />
 	<xacro:property name="leftArmJ2SerialNumber" value="v_b_009" />

File: model/robots/common/xacro/valkyrie_no_hands_base_hw.xacro (robot description, xacro)
@@ -11,5 +11,5 @@
     <xacro:v1_leg_sensors prefix="right" reflect="-1" ATI_serial_number="${right_foot_ATI_serial}" ATI_node="${right_foot_ATI_node}"/>
     <xacro:include_multisense_hw />
-    <xacro:v1_pelvis_rear_sensors_usb sensor_node_tag="${pelvis_rear_imu_node}" sensor_api_tag="${ImuSensorHardwareApi}"  sensor_port_tag="${pelvis_rear_imu_port}"/>
+    <xacro:v1_pelvis_sensors_usb sensor_node_tag="${pelvis_middle_imu_node}" sensor_api_tag="${ImuSensorHardwareApi}"  sensor_port_tag="${pelvis_middle_imu_port}"/>
     <xacro:waist_transmissions_hw />
     <xacro:leg_transmissions_hw prefix="left"/>

Commit message: updated coeffs and serials

File: common/xacro/serial_numbers/valkyrie_C_serials.xacro (robot description, xacro)
@@ -7,9 +7,9 @@
 	<xacro:property name="leftAnkleRightActuatorSerialNumber" value="v_e_010" />
 	<xacro:property name="rightLegJ1SerialNumber" value="v_a_014" />
-	<xacro:property name="rightLegJ2SerialNumber" value="v_b_015" />
-	<xacro:property name="rightLegJ3SerialNumber" value="v_c_009" />
-	<xacro:property name="rightLegJ4SerialNumber" value="v_d_005" />
-	<xacro:property name="rightAnkleLeftActuatorSerialNumber" value="v_e_021" />
-	<xacro:property name="rightAnkleRightActuatorSerialNumber" value="v_e_022" />
+	<xacro:property name="rightLegJ2SerialNumber" value="v_b_007" />
+	<xacro:property name="rightLegJ3SerialNumber" value="v_c_003" />
+	<xacro:property name="rightLegJ4SerialNumber" value="v_d_002" />
+	<xacro:property name="rightAnkleLeftActuatorSerialNumber" value="v_e_018" />
+	<xacro:property name="rightAnkleRightActuatorSerialNumber" value="v_e_017" />
 	<xacro:property name="leftArmJ1SerialNumber" value="v_a_013" />
 	<xacro:property name="leftArmJ2SerialNumber" value="v_b_009" />

Commit message: Serial swap for moving unit C's left leg to unit D.

File: common/xacro/serial_numbers/valkyrie_C_serials.xacro (robot description, xacro)
@@ -1,9 +1,9 @@
 <robot xmlns:xacro="http://ros.org/wiki/xacro" name="valkyrie_C_serials">
 	<xacro:property name="leftLegJ1SerialNumber" value="v_a_015" />
-	<xacro:property name="leftLegJ2SerialNumber" value="v_b_011" />
-	<xacro:property name="leftLegJ3SerialNumber" value="v_c_007" />
-	<xacro:property name="leftLegJ4SerialNumber" value="v_d_007" />
-	<xacro:property name="leftAnkleLeftActuatorSerialNumber" value="v_e_009" />
-	<xacro:property name="leftAnkleRightActuatorSerialNumber" value="v_e_010" />
+	<xacro:property name="leftLegJ2SerialNumber" value="v_b_016" />
+    <xacro:property name="leftLegJ3SerialNumber" value="v_c_008" />
+    <xacro:property name="leftLegJ4SerialNumber" value="v_d_008" />
+    <xacro:property name="leftAnkleLeftActuatorSerialNumber" value="v_e_019" />
+    <xacro:property name="leftAnkleRightActuatorSerialNumber" value="v_e_020" />
 	<xacro:property name="rightLegJ1SerialNumber" value="v_a_014" />
 	<xacro:property name="rightLegJ2SerialNumber" value="v_b_007" />

File: common/xacro/serial_numbers/valkyrie_D_serials.xacro (robot description, xacro)
@@ -1,9 +1,9 @@
 <robot xmlns:xacro="http://ros.org/wiki/xacro" name="valkyrie_C_serials">
     <xacro:property name="leftLegJ1SerialNumber" value="v_a_017" />
-    <xacro:property name="leftLegJ2SerialNumber" value="v_b_016" />
-    <xacro:property name="leftLegJ3SerialNumber" value="v_c_008" />
-    <xacro:property name="leftLegJ4SerialNumber" value="v_d_008" />
-    <xacro:property name="leftAnkleLeftActuatorSerialNumber" value="v_e_019" />
-    <xacro:property name="leftAnkleRightActuatorSerialNumber" value="v_e_020" />
+    <xacro:property name="leftLegJ2SerialNumber" value="v_b_011" />
+    <xacro:property name="leftLegJ3SerialNumber" value="v_c_007" />
+    <xacro:property name="leftLegJ4SerialNumber" value="v_d_007" />
+    <xacro:property name="leftAnkleLeftActuatorSerialNumber" value="v_e_009" />
+    <xacro:property name="leftAnkleRightActuatorSerialNumber" value="v_e_010" />
     <xacro:property name="rightLegJ1SerialNumber" value="v_a_018" />
     <xacro:property name="rightLegJ2SerialNumber" value="v_b_010" />

Commit message: Forgot to swap left foot ATI sensor serials. Swapping them here.

File: common/xacro/serial_numbers/valkyrie_C_serials.xacro (robot description, xacro)
@@ -32,5 +32,5 @@
 	<xacro:property name="waistRightActuatorSerialNumber" value="v_e_014" />
 	<xacro:property name="waistLeftActuatorSerialNumber" value="v_e_013" />
-	<xacro:property name="left_foot_ATI_serial" value="FT17212" />
+	<xacro:property name="left_foot_ATI_serial" value="FT14182" />
 	<xacro:property name="right_foot_ATI_serial" value="FT17214" />
 	<xacro:property name="sim_ATI_serial" value="FT001SIM" />

File: common/xacro/serial_numbers/valkyrie_D_serials.xacro (robot description, xacro)
@@ -32,5 +32,5 @@
     <xacro:property name="waistRightActuatorSerialNumber" value="v_e_023" />
     <xacro:property name="waistLeftActuatorSerialNumber" value="v_e_024" />
-    <xacro:property name="left_foot_ATI_serial" value="FT14182" />
+    <xacro:property name="left_foot_ATI_serial" value="FT17212" />
     <xacro:property name="right_foot_ATI_serial" value="FT16590" />
     <xacro:property name="sim_ATI_serial" value="FT001SIM" />

Commit message: Fixed ATI serials for unit C. calibrated a few of unit C's joints.

File: common/xacro/serial_numbers/valkyrie_C_serials.xacro (robot description, xacro)
@@ -29,6 +29,6 @@
 	<xacro:property name="waistLeftActuatorSerialNumber" value="v_e_013" />
 	<xacro:property name="leftForearmSerialNumber" value="UNKNOWN"/>
-        <xacro:property name="rightForearmSerialNumber" value="UNKNOWN"/>
-	<xacro:property name="left_foot_ATI_serial" value="FT14182" />
+    <xacro:property name="rightForearmSerialNumber" value="UNKNOWN"/>
+	<xacro:property name="left_foot_ATI_serial" value="FT16594" />
 	<xacro:property name="right_foot_ATI_serial" value="FT17214" />
 	<xacro:property name="sim_ATI_serial" value="FT001SIM" />

Commit message: Fixed serial of ATI load cell on foot.

File: common/xacro/serial_numbers/valkyrie_C_serials.xacro (robot description, xacro)
@@ -31,5 +31,5 @@
     <xacro:property name="rightForearmSerialNumber" value="UNKNOWN"/>
 	<xacro:property name="left_foot_ATI_serial" value="FT16594" />
-	<xacro:property name="right_foot_ATI_serial" value="FT14019" />
+	<xacro:property name="right_foot_ATI_serial" value="FT14018" />
 	<xacro:property name="sim_ATI_serial" value="FT001SIM" />
 </robot>

Commit message: updated imu serial numbers for unit C

File: common/xacro/serial_numbers/valkyrie_C_serials.xacro (robot description, xacro)
@@ -33,5 +33,5 @@
 	<xacro:property name="right_foot_ATI_serial" value="FT17214" />
 	<xacro:property name="rear_pelvis_IMU_serial" value="47251" />
-	<xacro:property name="left_torso_IMU_serial" value="47251" />
+	<xacro:property name="left_torso_IMU_serial" value="47099" />
 	<xacro:property name="sim_ATI_serial" value="FT001SIM" />
 </robot>

Commit message: Added forearm J5 serials to Unit C xacro

File: common/xacro/serial_numbers/valkyrie_C_serials.xacro (robot description, xacro)
@@ -16,10 +16,10 @@
 	<xacro:property name="leftArmJ3SerialNumber" value="v_f_012" />
 	<xacro:property name="leftArmJ4SerialNumber" value="v_f_011" />
-	<xacro:property name="leftArmJ5SerialNumber" value="UNKNOWN" />
+	<xacro:property name="leftArmJ5SerialNumber" value="v_g_018" />
 	<xacro:property name="rightArmJ1SerialNumber" value="v_a_012" />
 	<xacro:property name="rightArmJ2SerialNumber" value="v_b_012" />
 	<xacro:property name="rightArmJ3SerialNumber" value="v_f_013" />
 	<xacro:property name="rightArmJ4SerialNumber" value="v_f_014" />
-	<xacro:property name="rightArmJ5SerialNumber" value="UNKNOWN" />
+	<xacro:property name="rightArmJ5SerialNumber" value="v_g_017" />
 	<xacro:property name="neckJ1SerialNumber" value="v_g_001" />
 	<xacro:property name="neckJ2SerialNumber" value="v_g_002" />

Commit message: added forearms to val C serial numbers

File: common/xacro/serial_numbers/valkyrie_C_serials.xacro (robot description, xacro)
@@ -28,6 +28,6 @@
 	<xacro:property name="waistRightActuatorSerialNumber" value="v_e_014" />
 	<xacro:property name="waistLeftActuatorSerialNumber" value="v_e_013" />
-	<xacro:property name="leftForearmSerialNumber" value="UNKNOWN"/>
-    <xacro:property name="rightForearmSerialNumber" value="UNKNOWN"/>
+	<xacro:property name="leftForearmSerialNumber" value="v_h_007"/>
+    <xacro:property name="rightForearmSerialNumber" value="v_h_008"/>
 	<xacro:property name="left_foot_ATI_serial" value="FT16594" />
 	<xacro:property name="right_foot_ATI_serial" value="FT17214" />
