Commit message: updated coeffs for fingers

File: common/xacro/serial_numbers/forearm_testbench_serials.xacro (robot description, xacro)
@@ -1,3 +1,3 @@
 <robot xmlns:xacro="http://ros.org/wiki/xacro" name="forearm_testbench">
-	<xacro:property name="forearm_serial_number" value="v_h_003" />
+	<xacro:property name="forearm_serial_number" value="v_h_006" />
 </robot>

File: common/xacro/serial_numbers/valkyrie_D_serials.xacro (robot description, xacro)
@@ -28,6 +28,6 @@
     <xacro:property name="waistRightActuatorSerialNumber" value="v_e_023" />
     <xacro:property name="waistLeftActuatorSerialNumber" value="v_e_024" />
-    <xacro:property name="leftForearmSerialNumber" value="v_h_007"/>
-    <xacro:property name="rightForearmSerialNumber" value="v_h_008"/>
+    <xacro:property name="leftForearmSerialNumber" value="v_h_005"/>
+    <xacro:property name="rightForearmSerialNumber" value="v_h_006"/>
     <xacro:property name="left_foot_ATI_serial" value="FT14182" />
     <xacro:property name="right_foot_ATI_serial" value="FT14019" />

Commit message: pulled devel

File: common/xacro/serial_numbers/forearm_testbench_serials.xacro (robot description, xacro)
@@ -1,3 +1,3 @@
 <robot xmlns:xacro="http://ros.org/wiki/xacro" name="forearm_testbench">
-	<xacro:property name="forearm_serial_number" value="v_h_006" />
+	<xacro:property name="forearm_serial_number" value="v_h_005" />
 </robot>

File: common/xacro/serial_numbers/test_bench_serials.xacro (robot description, xacro)
@@ -1,3 +1,3 @@
 <robot xmlns:xacro="http://ros.org/wiki/xacro" name="test_bench_serials">
-	<xacro:property name="testbench_serial_number" value="v_g_012" />
+	<xacro:property name="testbench_serial_number" value="v_g_016" />
 </robot>

Commit message: updated to have two instance files for forearm testbench

File: common/xacro/serial_numbers/forearm_testbench_serials.xacro (robot description, xacro)
@@ -1,3 +1,4 @@
 <robot xmlns:xacro="http://ros.org/wiki/xacro" name="forearm_testbench">
+	<xacro:property name="testbench_serial_number" value="v_g_016" />
 	<xacro:property name="forearm_serial_number" value="v_h_005" />
 </robot>

File: instance/instances/robots/forearm_testbench_right.xacro (robot description, xacro)
@@ -1,6 +1,6 @@
-<robot xmlns:xacro="http://ros.org/wiki/xacro" name="forearm_testbench">
-	<xacro:property name="instance" value="forearm_testbench" />
-	<xacro:property name="prefix" value="left" />
-	<xacro:include filename="$(find val_description)/common/xacro/nodes/forearm_testbench_nodes.xacro" />
+<robot xmlns:xacro="http://ros.org/wiki/xacro" name="forearm_testbench_right">
+	<xacro:property name="instance" value="forearm_testbench_right" />
+	<xacro:property name="prefix" value="right" />
+	<xacro:include filename="$(find val_description)/common/xacro/nodes/forearm_testbench_nodes_right.xacro" />
 	<xacro:include filename="$(find val_description)/common/xacro/serial_numbers/forearm_testbench_serials.xacro" />
     <xacro:include filename="$(find val_description)/instance/instances/robots/xacro/mechanisms/mechanisms.xacro"/>
@@ -9,4 +9,5 @@
     </Channels>
     <Mechanisms>
+    <xacro:simple_mechanism name="testbench_actuator" serial_number="${testbench_serial_number}" node="${testbench_node}"/>
     <xacro:forearm mechanism_name="${prefix}Forearm" serial_number="${forearm_serial_number}" athena1_node="${Athena1Node}" athena2_node="${Athena2Node}" />
 	</Mechanisms>

Commit message: updated serials for forearm actuators

File: common/xacro/serial_numbers/forearm_testbench_serials.xacro (robot description, xacro)
@@ -1,5 +1,4 @@
 <robot xmlns:xacro="http://ros.org/wiki/xacro" name="forearm_testbench">
 	<xacro:property name="testbench_serial_number" value="v_g_016" />
-	<xacro:property name="forearm_serial_number" value="v_h_007" />
-	<xacro:property name="j5_serial_number" value="v_g_016" />
+	<xacro:property name="forearm_serial_number" value="v_h_003" />
 </robot>

Commit message: updated forearm testbench serials

File: common/xacro/serial_numbers/forearm_testbench_serials.xacro (robot description, xacro)
@@ -1,4 +1,4 @@
 <robot xmlns:xacro="http://ros.org/wiki/xacro" name="forearm_testbench">
-	<xacro:property name="testbench_serial_number" value="v_g_016" />
-	<xacro:property name="forearm_serial_number" value="v_h_003" />
+	<xacro:property name="testbench_serial_number" value="v_g_006" />
+	<xacro:property name="forearm_serial_number" value="v_h_004" />
 </robot>

Commit message: corrected compile error

File: common/xacro/serial_numbers/forearm_testbench_serials.xacro (robot description, xacro)
@@ -1,4 +1,4 @@
 <robot xmlns:xacro="http://ros.org/wiki/xacro" name="forearm_testbench">
-	<xacro:property name="testbench_serial_number" value="v_g_016" />
+	<xacro:property name="forearm_yaw_serial_number" value="v_g_016" />
 	<xacro:property name="forearm_serial_number" value="v_h_003" />
 </robot>
