Commit message: Added F/T sensor serial number to urdf.

File: common/xacro/serial_numbers/valkyrie_B_serials.xacro (robot description, xacro)
@@ -36,5 +36,5 @@
 	<xacro:property name="torso_imu1_serial" value="UNKNOWN" />
 	<xacro:property name="torso_imu2_serial" value="UNKNOWN" />
-	<xacro:property name="left_foot_ATI_serial" value="UNKNOWN" />
-	<xacro:property name="right_foot_ATI_serial" value="UNKNOWN" />
+	<xacro:property name="left_foot_ATI_serial" value="FT17219" />
+	<xacro:property name="right_foot_ATI_serial" value="FT17215" />
 </robot>

File: model/robots/common/xacro/leg/leg.xacro (robot description, xacro)
@@ -143,5 +143,5 @@
     <xacro:make_ankle_joints prefix="${prefix}" reflect="${reflect}" leg_root_link="${leg_root_link}" />
   </xacro:macro>
-  <xacro:macro name="v1_leg_sensors" params="prefix reflect">
+  <xacro:macro name="v1_leg_sensors" params="prefix reflect ATI_serial_number">
     <xacro:virtual_fixed_frame_offset name="${prefix}COP"
                        parentLink="${AnkleRollLinkName}"
@@ -151,5 +151,6 @@
                         parentLink="${AnkleRollLinkName}"
                         origin_xyz="0.0215646 0.0 -0.051054"
-                        origin_rpy="3.14 0.0 -1.047"/>
+                        origin_rpy="3.14 0.0 -1.047"
+                        sensor_number="${ATI_serial_number}"/>
   </xacro:macro>
   <xacro:macro name="leg_transmissions_hw" params="prefix">

File: model/robots/common/xacro/sensors/ati_force_torque.xacro (robot description, xacro)
@@ -1,5 +1,5 @@
 <?xml version="1.0" ?>
 <robot xmlns:xacro="http://www.ros.org/wiki/xacro" name="ati_force_torque_sensor">
-  <xacro:macro name="ati_force_torque_sensor" params="sensorName parentLink origin_xyz origin_rpy">
+  <xacro:macro name="ati_force_torque_sensor" params="sensorName parentLink origin_xyz origin_rpy sensor_number">
 	<xacro:massless_virtual_link name="${sensorName}_Frame"
                     origin_rpy="0 0 0"
@@ -12,4 +12,5 @@
       <sensor name="${sensorName}" type="force_torque">
         <frame>child</frame>
+        <sensor_number id="${sensor_number}" />
     	</sensor>
     </gazebo>

File: model/robots/common/xacro/valkyrie_base_hw.xacro (robot description, xacro)
@@ -13,9 +13,9 @@
     <xacro:make_middle_finger prefix="left" reflect="1" middle_finger_root_link="leftPalm"/>
     <xacro:make_pinky_finger prefix="left" reflect="1" pinky_finger_root_link="leftPalm"/>
-    <xacro:make_leg prefix="right" reflect="-1" leg_root_link="${Pelvis_Link_Name}" />
-    <xacro:make_leg prefix="left" reflect="1" leg_root_link="${Pelvis_Link_Name}" />
+    <xacro:make_leg prefix="right" reflect="-1" leg_root_link="${Pelvis_Link_Name}"/>
+    <xacro:make_leg prefix="left" reflect="1" leg_root_link="${Pelvis_Link_Name}"/>
     <xacro:v1_trunk_sensors/>
-    <xacro:v1_leg_sensors prefix="left" reflect="1" />
-    <xacro:v1_leg_sensors prefix="right" reflect="-1" />
+    <xacro:v1_leg_sensors prefix="left" reflect="1" ATI_serial_number="${left_foot_ATI_serial}"/>
+    <xacro:v1_leg_sensors prefix="right" reflect="-1" ATI_serial_number="${right_foot_ATI_serial}"/>
     <xacro:include_multisense_hw />
     <xacro:v1_pelvis_sensors/>

File: model/robots/common/xacro/valkyrie_base_sim.xacro (robot description, xacro)
@@ -13,9 +13,9 @@
     <xacro:make_middle_finger prefix="left" reflect="1" middle_finger_root_link="leftPalm"/>
     <xacro:make_pinky_finger prefix="left" reflect="1" pinky_finger_root_link="leftPalm"/>
-    <xacro:make_leg prefix="right" reflect="-1" leg_root_link="${Pelvis_Link_Name}" />
-    <xacro:make_leg prefix="left" reflect="1" leg_root_link="${Pelvis_Link_Name}" />
+    <xacro:make_leg prefix="right" reflect="-1" leg_root_link="${Pelvis_Link_Name}"/>
+    <xacro:make_leg prefix="left" reflect="1" leg_root_link="${Pelvis_Link_Name}"/>
     <xacro:v1_pelvis_sensors />
-    <xacro:v1_leg_sensors prefix="left" reflect="1" />
-    <xacro:v1_leg_sensors prefix="right" reflect="-1" />
+    <xacro:v1_leg_sensors prefix="left" reflect="1" ATI_serial_number="${left_foot_ATI_serial}"/>
+    <xacro:v1_leg_sensors prefix="right" reflect="-1" ATI_serial_number="${right_foot_ATI_serial}"/>
     <xacro:include_multisense_sim />
     <xacro:v1_trunk_sensors/>

File: model/robots/valkyrie_A_sim.xacro (robot description, xacro)
@@ -5,3 +5,4 @@
     <xacro:include filename="common/xacro/valkyrie_base_sim.xacro"/>
     <xacro:include filename="../urdf/multisense_sl.urdf" />
+    <xacro:include filename="../../common/xacro/serial_numbers/valkyrie_A_serials.xacro"/>
 </robot>

File: model/robots/valkyrie_B_sim.xacro (robot description, xacro)
@@ -5,3 +5,4 @@
     <xacro:include filename="common/xacro/valkyrie_base_sim.xacro"/>
     <xacro:include filename="../urdf/multisense_sl.urdf" />
+    <xacro:include filename="../../common/xacro/serial_numbers/valkyrie_B_serials.xacro"/>
 </robot>

Commit message: Fixed copy paste error in val instance file template.

File: common/xacro/serial_numbers/valkyrie_B_serials.xacro (robot description, xacro)
@@ -26,7 +26,7 @@
 	<xacro:property name="rightWristTopActuatorSerialNumber" value="UNKNOWN" />
 	<xacro:property name="rightWristBottomActuatorSerialNumber" value="UNKNOWN" />
-	<xacro:property name="neckJ1SerialNumber" value="UNKNOWN" />
-	<xacro:property name="neckJ2SerialNumber" value="UNKNOWN" />
-	<xacro:property name="neckJ3SerialNumber" value="UNKNOWN" />
+	<xacro:property name="neckJ1SerialNumber" value="BLAH1" />
+	<xacro:property name="neckJ2SerialNumber" value="BLAH2" />
+	<xacro:property name="neckJ3SerialNumber" value="BLAH3" />
 	<xacro:property name="trunkSerialNumber" value="v_a_008" />
 	<xacro:property name="waistRightActuatorSerialNumber" value="v_e_011" />

File: instance/instances/robots/xacro/common/valkyrie_full_template.xacro (robot description, xacro)
@@ -14,5 +14,5 @@
 		<xacro:arm prefix="left" j1_serial_number="${leftArmJ1SerialNumber}" j2_serial_number="${leftArmJ2SerialNumber}" j3_serial_number="${leftArmJ3SerialNumber}" j4_serial_number="${leftArmJ4SerialNumber}" j5_serial_number="${leftArmJ5SerialNumber}" wrist_actuator0_serial="${leftWristTopActuatorSerialNumber}" wrist_actuator1_serial="${leftWristBottomActuatorSerialNumber}" />
 		<xacro:arm prefix="right" j1_serial_number="${rightArmJ1SerialNumber}" j2_serial_number="${rightArmJ2SerialNumber}" j3_serial_number="${rightArmJ3SerialNumber}" j4_serial_number="${rightArmJ4SerialNumber}" j5_serial_number="${rightArmJ5SerialNumber}" wrist_actuator0_serial="${rightWristTopActuatorSerialNumber}" wrist_actuator1_serial="${rightWristBottomActuatorSerialNumber}" />
-		<xacro:neck j1_serial_number="${neckJ1SerialNumber}" j2_serial_number="${neckJ1SerialNumber}" j3_serial_number="${neckJ1SerialNumber}" />
+		<xacro:neck j1_serial_number="${neckJ1SerialNumber}" j2_serial_number="${neckJ2SerialNumber}" j3_serial_number="${neckJ3SerialNumber}" />
 		<xacro:waist j1_serial_number="${trunkSerialNumber}" waist_left_actuator_serial="${waistLeftActuatorSerialNumber}" waist_right_actuator_serial="${waistRightActuatorSerialNumber}"/>
 	</Mechanisms>

Commit message: Swapped serial numbers of right legs between units be and C.

File: common/xacro/serial_numbers/valkyrie_B_serials.xacro (robot description, xacro)
@@ -7,9 +7,9 @@
 	<xacro:property name="leftAnkleRightActuatorSerialNumber" value="v_e_015" />
 	<xacro:property name="rightLegJ1SerialNumber" value="v_a_007" />
-	<xacro:property name="rightLegJ2SerialNumber" value="v_b_007" />
-	<xacro:property name="rightLegJ3SerialNumber" value="v_c_003" />
-	<xacro:property name="rightLegJ4SerialNumber" value="v_d_002" />
-	<xacro:property name="rightAnkleLeftActuatorSerialNumber" value="v_e_018" />
-	<xacro:property name="rightAnkleRightActuatorSerialNumber" value="v_e_017" />
+	<xacro:property name="rightLegJ2SerialNumber" value="v_b_010" />
+	<xacro:property name="rightLegJ3SerialNumber" value="v_c_006" />
+	<xacro:property name="rightLegJ4SerialNumber" value="v_d_006" />
+	<xacro:property name="rightAnkleRightActuatorSerialNumber" value="v_e_008" />
+	<xacro:property name="rightAnkleLeftActuatorSerialNumber" value="v_e_007" />
 	<xacro:property name="leftArmJ1SerialNumber" value="v_a_002" />
 	<xacro:property name="leftArmJ2SerialNumber" value="v_b_005" />
@@ -37,5 +37,5 @@
 	<xacro:property name="torso_imu2_serial" value="UNKNOWN" />
 	<xacro:property name="left_foot_ATI_serial" value="FT17219" />
-	<xacro:property name="right_foot_ATI_serial" value="FT17215" />
+	<xacro:property name="right_foot_ATI_serial" value="FT17217" />
     <xacro:property name="sim_ATI_serial" value="FT001SIM" />
 </robot>

File: common/xacro/serial_numbers/valkyrie_C_serials.xacro (robot description, xacro)
@@ -7,9 +7,9 @@
 	<xacro:property name="leftAnkleRightActuatorSerialNumber" value="v_e_010" />
 	<xacro:property name="rightLegJ1SerialNumber" value="v_a_014" />
-	<xacro:property name="rightLegJ2SerialNumber" value="v_b_010" />
-	<xacro:property name="rightLegJ3SerialNumber" value="v_c_006" />
-	<xacro:property name="rightLegJ4SerialNumber" value="v_d_006" />
-	<xacro:property name="rightAnkleRightActuatorSerialNumber" value="v_e_008" />
-	<xacro:property name="rightAnkleLeftActuatorSerialNumber" value="v_e_007" />
+	<xacro:property name="rightLegJ2SerialNumber" value="v_b_007" />
+	<xacro:property name="rightLegJ3SerialNumber" value="v_c_003" />
+	<xacro:property name="rightLegJ4SerialNumber" value="v_d_002" />
+	<xacro:property name="rightAnkleLeftActuatorSerialNumber" value="v_e_018" />
+	<xacro:property name="rightAnkleRightActuatorSerialNumber" value="v_e_017" />
 	<xacro:property name="leftArmJ1SerialNumber" value="v_a_013" />
 	<xacro:property name="leftArmJ2SerialNumber" value="v_b_009" />
@@ -37,5 +37,5 @@
 	<xacro:property name="torso_imu2_serial" value="UNKNOWN" />
 	<xacro:property name="left_foot_ATI_serial" value="FT17213" />
-	<xacro:property name="right_foot_ATI_serial" value="FT17217" />
+	<xacro:property name="right_foot_ATI_serial" value="FT17215" />
 	<xacro:property name="sim_ATI_serial" value="FT001SIM" />
 </robot>

Commit message: Fixed serial number of ATI's in feet to have correct calibration file.

File: common/xacro/serial_numbers/valkyrie_B_serials.xacro (robot description, xacro)
@@ -36,6 +36,6 @@
 	<xacro:property name="torso_left_imu_serial" value="UNKNOWN" />
 	<xacro:property name="torso_right_imu_serial" value="UNKNOWN" />
-	<xacro:property name="left_foot_ATI_serial" value="FT17219" />
-	<xacro:property name="right_foot_ATI_serial" value="FT17217" />
+	<xacro:property name="left_foot_ATI_serial" value="FT17218" />
+	<xacro:property name="right_foot_ATI_serial" value="FT17216" />
     <xacro:property name="sim_ATI_serial" value="FT001SIM" />
 </robot>

Commit message: updated actuator and force torque serials

File: common/xacro/serial_numbers/valkyrie_B_serials.xacro (robot description, xacro)
@@ -7,9 +7,9 @@
 	<xacro:property name="leftAnkleRightActuatorSerialNumber" value="v_e_015" />
 	<xacro:property name="rightLegJ1SerialNumber" value="v_a_007" />
-	<xacro:property name="rightLegJ2SerialNumber" value="v_b_010" />
-	<xacro:property name="rightLegJ3SerialNumber" value="v_c_006" />
-	<xacro:property name="rightLegJ4SerialNumber" value="v_d_006" />
-	<xacro:property name="rightAnkleRightActuatorSerialNumber" value="v_e_008" />
-	<xacro:property name="rightAnkleLeftActuatorSerialNumber" value="v_e_007" />
+	<xacro:property name="rightLegJ2SerialNumber" value="v_b_015" />
+	<xacro:property name="rightLegJ3SerialNumber" value="v_c_009" />
+	<xacro:property name="rightLegJ4SerialNumber" value="v_d_005" />
+	<xacro:property name="rightAnkleRightActuatorSerialNumber" value="v_e_021" />
+	<xacro:property name="rightAnkleLeftActuatorSerialNumber" value="v_e_022" />
 	<xacro:property name="leftArmJ1SerialNumber" value="v_a_002" />
 	<xacro:property name="leftArmJ2SerialNumber" value="v_b_005" />
@@ -37,5 +37,5 @@
 	<xacro:property name="torso_right_imu_serial" value="UNKNOWN" />
 	<xacro:property name="left_foot_ATI_serial" value="FT17219" />
-	<xacro:property name="right_foot_ATI_serial" value="FT17217" />
+	<xacro:property name="right_foot_ATI_serial" value="FT14019" />
     <xacro:property name="sim_ATI_serial" value="FT001SIM" />
 </robot>

File: common/xacro/serial_numbers/valkyrie_D_serials.xacro (robot description, xacro)
@@ -7,9 +7,9 @@
     <xacro:property name="leftAnkleRightActuatorSerialNumber" value="v_e_020" />
     <xacro:property name="rightLegJ1SerialNumber" value="v_a_018" />
-    <xacro:property name="rightLegJ2SerialNumber" value="v_b_015" />
-    <xacro:property name="rightLegJ3SerialNumber" value="v_c_009" />
-    <xacro:property name="rightLegJ4SerialNumber" value="v_d_005" />
-    <xacro:property name="rightAnkleLeftActuatorSerialNumber" value="v_e_022" />
-    <xacro:property name="rightAnkleRightActuatorSerialNumber" value="v_e_021" />
+    <xacro:property name="rightLegJ2SerialNumber" value="v_b_010" />
+    <xacro:property name="rightLegJ3SerialNumber" value="v_c_006" />
+    <xacro:property name="rightLegJ4SerialNumber" value="v_d_006" />
+    <xacro:property name="rightAnkleLeftActuatorSerialNumber" value="v_e_008" />
+    <xacro:property name="rightAnkleRightActuatorSerialNumber" value="v_e_007" />
     <xacro:property name="leftArmJ1SerialNumber" value="v_a_019" />
     <xacro:property name="leftArmJ2SerialNumber" value="v_b_014" />
@@ -33,5 +33,5 @@
     <xacro:property name="waistLeftActuatorSerialNumber" value="v_e_024" />
     <xacro:property name="left_foot_ATI_serial" value="FT14182" />
-    <xacro:property name="right_foot_ATI_serial" value="FT14019" />
+    <xacro:property name="right_foot_ATI_serial" value="FT16591" />
     <xacro:property name="sim_ATI_serial" value="FT001SIM" />
 </robot>

Commit message: current working version of unit B coeffs

File: common/xacro/serial_numbers/valkyrie_B_serials.xacro (robot description, xacro)
@@ -7,9 +7,9 @@
 	<xacro:property name="leftAnkleRightActuatorSerialNumber" value="v_e_015" />
 	<xacro:property name="rightLegJ1SerialNumber" value="v_a_007" />
-	<xacro:property name="rightLegJ2SerialNumber" value="v_b_015" />
-	<xacro:property name="rightLegJ3SerialNumber" value="v_c_009" />
-	<xacro:property name="rightLegJ4SerialNumber" value="v_d_005" />
-	<xacro:property name="rightAnkleRightActuatorSerialNumber" value="v_e_021" />
-	<xacro:property name="rightAnkleLeftActuatorSerialNumber" value="v_e_022" />
+	<xacro:property name="rightLegJ2SerialNumber" value="v_b_010" />
+	<xacro:property name="rightLegJ3SerialNumber" value="v_c_006" />
+	<xacro:property name="rightLegJ4SerialNumber" value="v_d_006" />
+	<xacro:property name="rightAnkleRightActuatorSerialNumber" value="v_e_008" />
+	<xacro:property name="rightAnkleLeftActuatorSerialNumber" value="v_e_007" />
 	<xacro:property name="leftArmJ1SerialNumber" value="v_a_002" />
 	<xacro:property name="leftArmJ2SerialNumber" value="v_b_005" />

File: common/xacro/serial_numbers/valkyrie_D_serials.xacro (robot description, xacro)
@@ -7,9 +7,9 @@
     <xacro:property name="leftAnkleRightActuatorSerialNumber" value="v_e_020" />
     <xacro:property name="rightLegJ1SerialNumber" value="v_a_018" />
-    <xacro:property name="rightLegJ2SerialNumber" value="v_b_010" />
-    <xacro:property name="rightLegJ3SerialNumber" value="v_c_006" />
-    <xacro:property name="rightLegJ4SerialNumber" value="v_d_006" />
-    <xacro:property name="rightAnkleLeftActuatorSerialNumber" value="v_e_008" />
-    <xacro:property name="rightAnkleRightActuatorSerialNumber" value="v_e_007" />
+    <xacro:property name="rightLegJ2SerialNumber" value="v_b_015" />
+    <xacro:property name="rightLegJ3SerialNumber" value="v_c_009" />
+    <xacro:property name="rightLegJ4SerialNumber" value="v_d_005" />
+    <xacro:property name="rightAnkleLeftActuatorSerialNumber" value="v_e_021" />
+    <xacro:property name="rightAnkleRightActuatorSerialNumber" value="v_e_022" />
     <xacro:property name="leftArmJ1SerialNumber" value="v_a_019" />
     <xacro:property name="leftArmJ2SerialNumber" value="v_b_014" />

Commit message: Swapped serials to match robots.

File: common/xacro/serial_numbers/valkyrie_B_serials.xacro (robot description, xacro)
@@ -37,5 +37,5 @@
 	<xacro:property name="torso_right_imu_serial" value="UNKNOWN" />
 	<xacro:property name="left_foot_ATI_serial" value="FT17219" />
-	<xacro:property name="right_foot_ATI_serial" value="FT14019" />
+	<xacro:property name="right_foot_ATI_serial" value="FT16590" />
     <xacro:property name="sim_ATI_serial" value="FT001SIM" />
 </robot>

File: common/xacro/serial_numbers/valkyrie_D_serials.xacro (robot description, xacro)
@@ -33,5 +33,5 @@
     <xacro:property name="waistLeftActuatorSerialNumber" value="v_e_024" />
     <xacro:property name="left_foot_ATI_serial" value="FT14182" />
-    <xacro:property name="right_foot_ATI_serial" value="FT16591" />
+    <xacro:property name="right_foot_ATI_serial" value="FT14019" />
     <xacro:property name="sim_ATI_serial" value="FT001SIM" />
 </robot>

Commit message: Recal'd left ankle and fixed FT sensor serial for left foot.

File: common/xacro/serial_numbers/valkyrie_B_serials.xacro (robot description, xacro)
@@ -36,5 +36,5 @@
 	<xacro:property name="torso_left_imu_serial" value="UNKNOWN" />
 	<xacro:property name="torso_right_imu_serial" value="UNKNOWN" />
-	<xacro:property name="left_foot_ATI_serial" value="FT17219" />
+	<xacro:property name="left_foot_ATI_serial" value="FT17218" />
 	<xacro:property name="right_foot_ATI_serial" value="FT16590" />
     <xacro:property name="sim_ATI_serial" value="FT001SIM" />

Commit message: Emergency leg swap. Swapped serials.

File: common/xacro/serial_numbers/valkyrie_B_serials.xacro (robot description, xacro)
@@ -7,9 +7,9 @@
 	<xacro:property name="leftAnkleRightActuatorSerialNumber" value="v_e_015" />
 	<xacro:property name="rightLegJ1SerialNumber" value="v_a_007" />
-	<xacro:property name="rightLegJ2SerialNumber" value="v_b_010" />
-	<xacro:property name="rightLegJ3SerialNumber" value="v_c_006" />
-	<xacro:property name="rightLegJ4SerialNumber" value="v_d_006" />
-	<xacro:property name="rightAnkleRightActuatorSerialNumber" value="v_e_008" />
-	<xacro:property name="rightAnkleLeftActuatorSerialNumber" value="v_e_007" />
+	<xacro:property name="rightLegJ2SerialNumber" value="v_b_015" />
+    <xacro:property name="rightLegJ3SerialNumber" value="v_c_009" />
+    <xacro:property name="rightLegJ4SerialNumber" value="v_d_005" />
+    <xacro:property name="rightAnkleLeftActuatorSerialNumber" value="v_e_021" />
+    <xacro:property name="rightAnkleRightActuatorSerialNumber" value="v_e_022" />
 	<xacro:property name="leftArmJ1SerialNumber" value="v_a_002" />
 	<xacro:property name="leftArmJ2SerialNumber" value="v_b_005" />
@@ -37,5 +37,5 @@
 	<xacro:property name="torso_right_imu_serial" value="UNKNOWN" />
 	<xacro:property name="left_foot_ATI_serial" value="FT17218" />
-	<xacro:property name="right_foot_ATI_serial" value="FT16590" />
+	<xacro:property name="right_foot_ATI_serial" value="FT14019" />
     <xacro:property name="sim_ATI_serial" value="FT001SIM" />
 </robot>

File: common/xacro/serial_numbers/valkyrie_D_serials.xacro (robot description, xacro)
@@ -7,9 +7,9 @@
     <xacro:property name="leftAnkleRightActuatorSerialNumber" value="v_e_020" />
     <xacro:property name="rightLegJ1SerialNumber" value="v_a_018" />
-    <xacro:property name="rightLegJ2SerialNumber" value="v_b_015" />
-    <xacro:property name="rightLegJ3SerialNumber" value="v_c_009" />
-    <xacro:property name="rightLegJ4SerialNumber" value="v_d_005" />
-    <xacro:property name="rightAnkleLeftActuatorSerialNumber" value="v_e_021" />
-    <xacro:property name="rightAnkleRightActuatorSerialNumber" value="v_e_022" />
+    <xacro:property name="rightLegJ2SerialNumber" value="v_b_010" />
+    <xacro:property name="rightLegJ3SerialNumber" value="v_c_006" />
+    <xacro:property name="rightLegJ4SerialNumber" value="v_d_006" />
+    <xacro:property name="rightAnkleRightActuatorSerialNumber" value="v_e_008" />
+    <xacro:property name="rightAnkleLeftActuatorSerialNumber" value="v_e_007" />
     <xacro:property name="leftArmJ1SerialNumber" value="v_a_019" />
     <xacro:property name="leftArmJ2SerialNumber" value="v_b_014" />
@@ -33,5 +33,5 @@
     <xacro:property name="waistLeftActuatorSerialNumber" value="v_e_024" />
     <xacro:property name="left_foot_ATI_serial" value="FT14182" />
-    <xacro:property name="right_foot_ATI_serial" value="FT14019" />
+    <xacro:property name="right_foot_ATI_serial" value="FT16590" />
     <xacro:property name="sim_ATI_serial" value="FT001SIM" />
 </robot>
