Commit message: updated robot serials

File: common/xacro/serial_numbers/valkyrie_B_serials.xacro (robot description, xacro)
@@ -1,15 +1,15 @@
 <robot xmlns:xacro="http://ros.org/wiki/xacro" name="valkyrie_B_serials">
 	<xacro:property name="leftLegJ1SerialNumber" value="v_a_009" />
-	<xacro:property name="leftLegJ2SerialNumber" value="v_b_006" />
-	<xacro:property name="leftLegJ3SerialNumber" value="v_c_004" />
-	<xacro:property name="leftLegJ4SerialNumber" value="v_d_003" />
+	<xacro:property name="leftLegJ2SerialNumber" value="v_b_016" />
+	<xacro:property name="leftLegJ3SerialNumber" value="v_c_008" />
+	<xacro:property name="leftLegJ4SerialNumber" value="v_d_008" />
 	<xacro:property name="leftAnkleLeftActuatorSerialNumber" value="v_e_016" />
 	<xacro:property name="leftAnkleRightActuatorSerialNumber" value="v_e_015" />
 	<xacro:property name="rightLegJ1SerialNumber" value="v_a_007" />
 	<xacro:property name="rightLegJ2SerialNumber" value="v_b_015" />
-    <xacro:property name="rightLegJ3SerialNumber" value="v_c_009" />
-    <xacro:property name="rightLegJ4SerialNumber" value="v_d_005" />
-    <xacro:property name="rightAnkleLeftActuatorSerialNumber" value="v_e_021" />
-    <xacro:property name="rightAnkleRightActuatorSerialNumber" value="v_e_022" />
+        <xacro:property name="rightLegJ3SerialNumber" value="v_c_009" />
+        <xacro:property name="rightLegJ4SerialNumber" value="v_d_005" />
+        <xacro:property name="rightAnkleLeftActuatorSerialNumber" value="v_e_021" />
+        <xacro:property name="rightAnkleRightActuatorSerialNumber" value="v_e_022" />
 	<xacro:property name="leftArmJ1SerialNumber" value="v_a_002" />
 	<xacro:property name="leftArmJ2SerialNumber" value="v_b_005" />

File: common/xacro/serial_numbers/valkyrie_C_serials.xacro (robot description, xacro)
@@ -1,9 +1,9 @@
 <robot xmlns:xacro="http://ros.org/wiki/xacro" name="valkyrie_C_serials">
 	<xacro:property name="leftLegJ1SerialNumber" value="v_a_015" />
-	<xacro:property name="leftLegJ2SerialNumber" value="v_b_016" />
-    <xacro:property name="leftLegJ3SerialNumber" value="v_c_008" />
-    <xacro:property name="leftLegJ4SerialNumber" value="v_d_008" />
-    <xacro:property name="leftAnkleLeftActuatorSerialNumber" value="v_e_019" />
-    <xacro:property name="leftAnkleRightActuatorSerialNumber" value="v_e_020" />
+	<xacro:property name="leftLegJ2SerialNumber" value="v_b_006" />
+        <xacro:property name="leftLegJ3SerialNumber" value="v_c_004" />
+        <xacro:property name="leftLegJ4SerialNumber" value="v_d_003" />
+        <xacro:property name="leftAnkleLeftActuatorSerialNumber" value="v_e_019" />
+        <xacro:property name="leftAnkleRightActuatorSerialNumber" value="v_e_020" />
 	<xacro:property name="rightLegJ1SerialNumber" value="v_a_014" />
 	<xacro:property name="rightLegJ2SerialNumber" value="v_b_007" />

Commit message: Another leg swap. Updated serials accordingly.

File: common/xacro/serial_numbers/valkyrie_B_serials.xacro (robot description, xacro)
@@ -7,9 +7,9 @@
 	<xacro:property name="leftAnkleRightActuatorSerialNumber" value="v_e_015" />
 	<xacro:property name="rightLegJ1SerialNumber" value="v_a_007" />
-	<xacro:property name="rightLegJ2SerialNumber" value="v_b_015" />
-        <xacro:property name="rightLegJ3SerialNumber" value="v_c_009" />
-        <xacro:property name="rightLegJ4SerialNumber" value="v_d_005" />
-        <xacro:property name="rightAnkleLeftActuatorSerialNumber" value="v_e_021" />
-        <xacro:property name="rightAnkleRightActuatorSerialNumber" value="v_e_022" />
+	<xacro:property name="rightLegJ2SerialNumber" value="v_b_007" />
+	<xacro:property name="rightLegJ3SerialNumber" value="v_c_003" />
+	<xacro:property name="rightLegJ4SerialNumber" value="v_d_002" />
+	<xacro:property name="rightAnkleLeftActuatorSerialNumber" value="v_e_018" />
+	<xacro:property name="rightAnkleRightActuatorSerialNumber" value="v_e_017" />
 	<xacro:property name="leftArmJ1SerialNumber" value="v_a_002" />
 	<xacro:property name="leftArmJ2SerialNumber" value="v_b_005" />
@@ -31,5 +31,5 @@
     <xacro:property name="rightForearmSerialNumber" value="v_h_004"/>
 	<xacro:property name="left_foot_ATI_serial" value="FT17218" />
-	<xacro:property name="right_foot_ATI_serial" value="FT14019" />
+	<xacro:property name="right_foot_ATI_serial" value="FT17214" />
     <xacro:property name="sim_ATI_serial" value="FT001SIM" />
 </robot>

File: common/xacro/serial_numbers/valkyrie_C_serials.xacro (robot description, xacro)
@@ -2,14 +2,14 @@
 	<xacro:property name="leftLegJ1SerialNumber" value="v_a_015" />
 	<xacro:property name="leftLegJ2SerialNumber" value="v_b_006" />
-        <xacro:property name="leftLegJ3SerialNumber" value="v_c_004" />
-        <xacro:property name="leftLegJ4SerialNumber" value="v_d_003" />
-        <xacro:property name="leftAnkleLeftActuatorSerialNumber" value="v_e_019" />
-        <xacro:property name="leftAnkleRightActuatorSerialNumber" value="v_e_020" />
+    <xacro:property name="leftLegJ3SerialNumber" value="v_c_004" />
+    <xacro:property name="leftLegJ4SerialNumber" value="v_d_003" />
+    <xacro:property name="leftAnkleLeftActuatorSerialNumber" value="v_e_019" />
+    <xacro:property name="leftAnkleRightActuatorSerialNumber" value="v_e_020" />
 	<xacro:property name="rightLegJ1SerialNumber" value="v_a_014" />
-	<xacro:property name="rightLegJ2SerialNumber" value="v_b_007" />
-	<xacro:property name="rightLegJ3SerialNumber" value="v_c_003" />
-	<xacro:property name="rightLegJ4SerialNumber" value="v_d_002" />
-	<xacro:property name="rightAnkleLeftActuatorSerialNumber" value="v_e_018" />
-	<xacro:property name="rightAnkleRightActuatorSerialNumber" value="v_e_017" />
+	<xacro:property name="rightLegJ2SerialNumber" value="v_b_015" />
+    <xacro:property name="rightLegJ3SerialNumber" value="v_c_009" />
+    <xacro:property name="rightLegJ4SerialNumber" value="v_d_005" />
+    <xacro:property name="rightAnkleLeftActuatorSerialNumber" value="v_e_021" />
+    <xacro:property name="rightAnkleRightActuatorSerialNumber" value="v_e_022" />
 	<xacro:property name="leftArmJ1SerialNumber" value="v_a_013" />
 	<xacro:property name="leftArmJ2SerialNumber" value="v_b_009" />
@@ -31,5 +31,5 @@
     <xacro:property name="rightForearmSerialNumber" value="UNKNOWN"/>
 	<xacro:property name="left_foot_ATI_serial" value="FT16594" />
-	<xacro:property name="right_foot_ATI_serial" value="FT17214" />
+	<xacro:property name="right_foot_ATI_serial" value="FT14019" />
 	<xacro:property name="sim_ATI_serial" value="FT001SIM" />
 </robot>

Commit message: Coeff fixes and a serial swap due to a swapping of legs.

File: common/xacro/serial_numbers/valkyrie_B_serials.xacro (robot description, xacro)
@@ -7,9 +7,9 @@
 	<xacro:property name="leftAnkleRightActuatorSerialNumber" value="v_e_015" />
 	<xacro:property name="rightLegJ1SerialNumber" value="v_a_007" />
-	<xacro:property name="rightLegJ2SerialNumber" value="v_b_007" />
-	<xacro:property name="rightLegJ3SerialNumber" value="v_c_003" />
-	<xacro:property name="rightLegJ4SerialNumber" value="v_d_002" />
-	<xacro:property name="rightAnkleLeftActuatorSerialNumber" value="v_e_018" />
-	<xacro:property name="rightAnkleRightActuatorSerialNumber" value="v_e_017" />
+	<xacro:property name="rightLegJ2SerialNumber" value="v_b_015" />
+    <xacro:property name="rightLegJ3SerialNumber" value="v_c_009" />
+    <xacro:property name="rightLegJ4SerialNumber" value="v_d_009" />
+    <xacro:property name="rightAnkleLeftActuatorSerialNumber" value="v_e_021" />
+    <xacro:property name="rightAnkleRightActuatorSerialNumber" value="v_e_022" />
 	<xacro:property name="leftArmJ1SerialNumber" value="v_a_002" />
 	<xacro:property name="leftArmJ2SerialNumber" value="v_b_005" />
@@ -31,5 +31,5 @@
     <xacro:property name="rightForearmSerialNumber" value="v_h_004"/>
 	<xacro:property name="left_foot_ATI_serial" value="FT17218" />
-	<xacro:property name="right_foot_ATI_serial" value="FT17214" />
+	<xacro:property name="right_foot_ATI_serial" value="FT14018" />
     <xacro:property name="sim_ATI_serial" value="FT001SIM" />
 </robot>

File: common/xacro/serial_numbers/valkyrie_C_serials.xacro (robot description, xacro)
@@ -7,9 +7,9 @@
     <xacro:property name="leftAnkleRightActuatorSerialNumber" value="v_e_020" />
 	<xacro:property name="rightLegJ1SerialNumber" value="v_a_014" />
-	<xacro:property name="rightLegJ2SerialNumber" value="v_b_015" />
-    <xacro:property name="rightLegJ3SerialNumber" value="v_c_009" />
-    <xacro:property name="rightLegJ4SerialNumber" value="v_d_005" />
-    <xacro:property name="rightAnkleLeftActuatorSerialNumber" value="v_e_021" />
-    <xacro:property name="rightAnkleRightActuatorSerialNumber" value="v_e_022" />
+	<xacro:property name="rightLegJ2SerialNumber" value="v_b_007" />
+	<xacro:property name="rightLegJ3SerialNumber" value="v_c_003" />
+	<xacro:property name="rightLegJ4SerialNumber" value="v_d_002" />
+	<xacro:property name="rightAnkleLeftActuatorSerialNumber" value="v_e_018" />
+	<xacro:property name="rightAnkleRightActuatorSerialNumber" value="v_e_017" />
 	<xacro:property name="leftArmJ1SerialNumber" value="v_a_013" />
 	<xacro:property name="leftArmJ2SerialNumber" value="v_b_009" />
@@ -31,5 +31,5 @@
     <xacro:property name="rightForearmSerialNumber" value="UNKNOWN"/>
 	<xacro:property name="left_foot_ATI_serial" value="FT16594" />
-	<xacro:property name="right_foot_ATI_serial" value="FT14018" />
+	<xacro:property name="right_foot_ATI_serial" value="FT17214" />
 	<xacro:property name="sim_ATI_serial" value="FT001SIM" />
 </robot>

Commit message: First madness commit

File: common/xacro/serial_numbers/valkyrie_B_serials.xacro (robot description, xacro)
@@ -7,5 +7,5 @@
 	<xacro:property name="leftAnkleRightActuatorSerialNumber" value="v_e_015" />
 	<xacro:property name="rightLegJ1SerialNumber" value="v_a_007" />
-	<xacro:property name="rightLegJ2SerialNumber" value="v_b_015" />
+	<xacro:property name="rightLegJ2SerialNumber" value="v_b_001" />
     <xacro:property name="rightLegJ3SerialNumber" value="v_c_009" />
     <xacro:property name="rightLegJ4SerialNumber" value="v_d_009" />

Commit message: updated valkyrie_B_serials for actuator swap

File: common/xacro/serial_numbers/valkyrie_B_serials.xacro (robot description, xacro)
@@ -7,5 +7,5 @@
 	<xacro:property name="leftAnkleRightActuatorSerialNumber" value="v_e_015" />
 	<xacro:property name="rightLegJ1SerialNumber" value="v_a_007" />
-	<xacro:property name="rightLegJ2SerialNumber" value="v_b_001" />
+	<xacro:property name="rightLegJ2SerialNumber" value="v_b_015" />
     <xacro:property name="rightLegJ3SerialNumber" value="v_c_009" />
     <xacro:property name="rightLegJ4SerialNumber" value="v_d_009" />

Commit message: neck j1 swap for unit B

File: common/xacro/serial_numbers/valkyrie_B_serials.xacro (robot description, xacro)
@@ -22,5 +22,5 @@
 	<xacro:property name="rightArmJ4SerialNumber" value="v_f_010" />
 	<xacro:property name="rightArmJ5SerialNumber" value="v_g_006" />
-	<xacro:property name="neckJ1SerialNumber" value="v_g_009" />
+	<xacro:property name="neckJ1SerialNumber" value="v_g_019" />
 	<xacro:property name="neckJ2SerialNumber" value="v_g_010" />
 	<xacro:property name="neckJ3SerialNumber" value="v_g_011" />
