Commit message: Fixing inertias and COM's of elbow pitch links. I was not properly reflecting the COM's and was just doing stupid with the inertias.

File: model/robots/common/xacro/arm/mass_parameters.xacro (robot description, xacro)
@@ -26,11 +26,11 @@
   <xacro:property name="ShoulderYawLinkInertia_IZZ" value="0.041879481" />
   <xacro:property name="ElbowPitchLinkMass" value="1.830000" />
-  <xacro:property name="ElbowPitchLinkComPosition" value="-0.020344	${reflect*0.014722} -0.022300" />
-  <xacro:property name="ElbowPitchLinkInertia_IXX" value="0.004285137" />
-  <xacro:property name="ElbowPitchLinkInertia_IXY" value="${reflect*-0.000408334}" />
-  <xacro:property name="ElbowPitchLinkInertia_IXZ" value="${reflect*0.003326627}" />
-  <xacro:property name="ElbowPitchLinkInertia_IYY" value="0.008440601" />
-  <xacro:property name="ElbowPitchLinkInertia_IYZ" value="0.000140731" />
-  <xacro:property name="ElbowPitchLinkInertia_IZZ" value="0.007469454" />
+  <xacro:property name="ElbowPitchLinkComPosition" value="-0.020344	${reflect*0.014722} ${reflect*0.022300}" />
+  <xacro:property name="ElbowPitchLinkInertia_IXX" value="0.003314516" />
+  <xacro:property name="ElbowPitchLinkInertia_IXY" value="${reflect*0.000535099}" />
+  <xacro:property name="ElbowPitchLinkInertia_IXZ" value="${reflect*0.000728077}" />
+  <xacro:property name="ElbowPitchLinkInertia_IYY" value="0.003505669" />
+  <xacro:property name="ElbowPitchLinkInertia_IYZ" value="-0.000423865" />
+  <xacro:property name="ElbowPitchLinkInertia_IZZ" value="0.003011283" />
   <xacro:property name="ForearmYawLinkMass" value="2.476" />
   <xacro:property name="ForearmYawLinkComPosition" value="0.015000	${reflect*0.13} 0.019564" />

Commit message: Fixed reflect on shoulder yaw COM.

File: model/robots/common/xacro/arm/mass_parameters.xacro (robot description, xacro)
@@ -18,5 +18,5 @@
   <xacro:property name="ShoulderRollLinkInertia_IZZ" value="0.011454772" />
   <xacro:property name="ShoulderYawLinkMass" value="3.085000" />
-  <xacro:property name="ShoulderYawLinkComPosition" value="-0.004304	${reflect*0.209832}	-0.007295" />
+  <xacro:property name="ShoulderYawLinkComPosition" value="-0.004304	${reflect*0.209832}	${reflect*0.007295}" />
   <xacro:property name="ShoulderYawLinkInertia_IXX" value="0.039355177" />
   <xacro:property name="ShoulderYawLinkInertia_IXY" value="0.007827077" />

Commit message: Fixed reflection of shoulder yaw COM and inertia.

File: model/robots/common/xacro/arm/mass_parameters.xacro (robot description, xacro)
@@ -20,8 +20,8 @@
   <xacro:property name="ShoulderYawLinkComPosition" value="-0.004304	${reflect*0.209832}	${reflect*0.007295}" />
   <xacro:property name="ShoulderYawLinkInertia_IXX" value="0.039355177" />
-  <xacro:property name="ShoulderYawLinkInertia_IXY" value="0.007827077" />
+  <xacro:property name="ShoulderYawLinkInertia_IXY" value="${reflect*-0.007827077}" />
   <xacro:property name="ShoulderYawLinkInertia_IXZ" value="${reflect*-0.000753947}" />
   <xacro:property name="ShoulderYawLinkInertia_IYY" value="0.004905765" />
-  <xacro:property name="ShoulderYawLinkInertia_IYZ" value="${reflect*-0.002723873}" />
+  <xacro:property name="ShoulderYawLinkInertia_IYZ" value="${reflect*0.002723873}" />
   <xacro:property name="ShoulderYawLinkInertia_IZZ" value="0.041879481" />
   <xacro:property name="ElbowPitchLinkMass" value="1.830000" />

Commit message: Fixed a few more inertia params for arms.

File: model/robots/common/xacro/arm/mass_parameters.xacro (robot description, xacro)
@@ -35,9 +35,9 @@
   <xacro:property name="ForearmYawLinkMass" value="2.476" />
   <xacro:property name="ForearmYawLinkComPosition" value="0.015000	${reflect*0.13} 0.019564" />
-  <xacro:property name="ForearmYawLinkInertia_IXX" value="0.015011" />
+  <xacro:property name="ForearmYawLinkInertia_IXX" value="0.011755430" />
   <xacro:property name="ForearmYawLinkInertia_IXY" value="${reflect*0.001300853}" />
-  <xacro:property name="ForearmYawLinkInertia_IXZ" value="${reflect*0.000727141}" />
+  <xacro:property name="ForearmYawLinkInertia_IXZ" value="-0.000727141" />
   <xacro:property name="ForearmYawLinkInertia_IYY" value="0.005071567" />
-  <xacro:property name="ForearmYawLinkInertia_IYZ" value="-0.001695416" />
+  <xacro:property name="ForearmYawLinkInertia_IYZ" value="${reflect*0.001695416}" />
   <xacro:property name="ForearmYawLinkInertia_IZZ" value="0.011365657" />
   <xacro:property name="WristRollLinkMass" value="0.14" />

Commit message: Fixed some inertia parameters of shoulder roll link.

File: model/robots/common/xacro/arm/mass_parameters.xacro (robot description, xacro)
@@ -10,5 +10,5 @@
   <xacro:property name="ShoulderPitchLinkInertia_IZZ" value="0.014806433" />
   <xacro:property name="ShoulderRollLinkMass" value="3.970000" />
-  <xacro:property name="ShoulderRollLinkComPosition" value="-0.008513 ${reflect*0.020680} 0.001088" />
+  <xacro:property name="ShoulderRollLinkComPosition" value="-0.008513 ${reflect*0.020680} ${reflect*-0.001088}" />
   <xacro:property name="ShoulderRollLinkInertia_IXX" value="0.009494119" />
   <xacro:property name="ShoulderRollLinkInertia_IXY" value="${reflect*0.000067294}" />
@@ -16,5 +16,5 @@
   <xacro:property name="ShoulderRollLinkInertia_IYY" value="0.007680534" />
   <xacro:property name="ShoulderRollLinkInertia_IYZ" value="0.000008874" />
-  <xacro:property name="ShoulderRollLinkInertia_IZZ" value="0.011454772" />
+  <xacro:property name="ShoulderRollLinkInertia_IZZ" value="0.012454772" />
   <xacro:property name="ShoulderYawLinkMass" value="3.085000" />
   <xacro:property name="ShoulderYawLinkComPosition" value="-0.004304	${reflect*0.209832}	${reflect*0.007295}" />

Commit message: Updated COM and inertia since we are flipping the right arm now.

File: model/robots/common/xacro/arm/mass_parameters.xacro (robot description, xacro)
@@ -2,5 +2,5 @@
 <robot xmlns:xacro="http://www.ros.org/wiki/xacro" name="v1/arm/mass_parameters">
   <xacro:property name="ShoulderPitchLinkMass" value="2.65" />
-  <xacro:property name="ShoulderPitchLinkComPosition" value="-0.012000 ${reflect*0.251000} 0.000000" />
+  <xacro:property name="ShoulderPitchLinkComPosition" value="${reflect*-0.012000} ${reflect*0.251000} 0.000000" />
   <xacro:property name="ShoulderPitchLinkInertia_IXX" value="0.013718167" />
   <xacro:property name="ShoulderPitchLinkInertia_IXY" value="0.000000000" />
@@ -10,11 +10,11 @@
   <xacro:property name="ShoulderPitchLinkInertia_IZZ" value="0.014806433" />
   <xacro:property name="ShoulderRollLinkMass" value="3.970000" />
-  <xacro:property name="ShoulderRollLinkComPosition" value="-0.008513 ${reflect*0.020680} ${reflect*-0.001088}" />
-  <xacro:property name="ShoulderRollLinkInertia_IXX" value="0.009494119" />
-  <xacro:property name="ShoulderRollLinkInertia_IXY" value="${reflect*0.000067294}" />
-  <xacro:property name="ShoulderRollLinkInertia_IXZ" value="${reflect*-0.000037177}" />
-  <xacro:property name="ShoulderRollLinkInertia_IYY" value="0.007680534" />
-  <xacro:property name="ShoulderRollLinkInertia_IYZ" value="0.000008874" />
-  <xacro:property name="ShoulderRollLinkInertia_IZZ" value="0.012454772" />
+  <xacro:property name="ShoulderRollLinkComPosition" value="${reflect*-0.008513) ${reflect*0.020680} -0.001088" />
+  <xacro:property name="ShoulderRollLinkInertia_IXX" value="0.014598842" />
+  <xacro:property name="ShoulderRollLinkInertia_IXY" value="-0.00066764" />
+  <xacro:property name="ShoulderRollLinkInertia_IXZ" value="${reflect*-0.00003629}" />
+  <xacro:property name="ShoulderRollLinkInertia_IYY" value="0.006452136" />
+  <xacro:property name="ShoulderRollLinkInertia_IYZ" value="${reflect*-0.00008283}" />
+  <xacro:property name="ShoulderRollLinkInertia_IZZ" value="0.016848319" />
   <xacro:property name="ShoulderYawLinkMass" value="3.085000" />
   <xacro:property name="ShoulderYawLinkComPosition" value="-0.004304	${reflect*0.209832}	${reflect*0.007295}" />

Commit message: Fixed typo in xacro file that I introduced. Giggity.

File: model/robots/common/xacro/arm/mass_parameters.xacro (robot description, xacro)
@@ -10,5 +10,5 @@
   <xacro:property name="ShoulderPitchLinkInertia_IZZ" value="0.014806433" />
   <xacro:property name="ShoulderRollLinkMass" value="3.970000" />
-  <xacro:property name="ShoulderRollLinkComPosition" value="${reflect*-0.008513) ${reflect*0.020680} -0.001088" />
+  <xacro:property name="ShoulderRollLinkComPosition" value="${reflect*-0.008513} ${reflect*0.020680} -0.001088" />
   <xacro:property name="ShoulderRollLinkInertia_IXX" value="0.014598842" />
   <xacro:property name="ShoulderRollLinkInertia_IXY" value="-0.00066764" />
