Commit message: Have urdf's generating again.

File: model/robots/common/xacro/arm/arm.xacro (robot description, xacro)
@@ -1,11 +1,11 @@
 <?xml version="1.0" ?>
 <robot xmlns:xacro="http://www.ros.org/wiki/xacro" name="arm">
-  <xacro:include filename="$(find val_description)/robots/common/xacro/arm/joint_names.xacro"/>
-  <xacro:include filename="$(find val_description)/robots/common/xacro/arm/actuator_names.xacro"/>
-  <xacro:include filename="$(find val_description)/robots/common/xacro/arm/joint_axes.xacro"/>
-  <xacro:include filename="$(find val_description)/robots/common/xacro/arm/link_names.xacro"/>
-  <xacro:include filename="$(find val_description)/robots/common/xacro/arm/joint_limits.xacro"/>
-  <xacro:include filename="$(find val_description)/robots/common/xacro/arm/frame_parameters.xacro"/>
-  <xacro:include filename="$(find val_description)/robots/common/xacro/arm/mass_parameters.xacro"/>
+  <xacro:include filename="$(find val_description)/model/robots/common/xacro/arm/joint_names.xacro"/>
+  <xacro:include filename="$(find val_description)/model/robots/common/xacro/arm/actuator_names.xacro"/>
+  <xacro:include filename="$(find val_description)/model/robots/common/xacro/arm/joint_axes.xacro"/>
+  <xacro:include filename="$(find val_description)/model/robots/common/xacro/arm/link_names.xacro"/>
+  <xacro:include filename="$(find val_description)/model/robots/common/xacro/arm/joint_limits.xacro"/>
+  <xacro:include filename="$(find val_description)/model/robots/common/xacro/arm/frame_parameters.xacro"/>
+  <xacro:include filename="$(find val_description)/model/robots/common/xacro/arm/mass_parameters.xacro"/>
   <xacro:macro name="make_upper_arm" params="prefix reflect upper_arm_root_link">
     <xacro:standard_link name="${ShoulderPitchLinkName}"

File: model/robots/common/xacro/common_bodies.xacro (robot description, xacro)
@@ -1,10 +1,10 @@
 <robot xmlns:xacro="http://ros.orgt/wiki/xacro" name="common_bodies">
-    <xacro:include filename="$(find val_description)/robots/common/xacro/pelvis/pelvis.xacro" />
-    <xacro:include filename="$(find val_description)/robots/common/xacro/waist/waist.xacro" />
-    <xacro:include filename="$(find val_description)/robots/common/xacro/head/head.xacro" />
-    <xacro:include filename="$(find val_description)/robots/common/xacro/arm/arm.xacro" />
-    <xacro:include filename="$(find val_description)/robots/common/xacro/thumb/thumb.xacro" />
-    <xacro:include filename="$(find val_description)/robots/common/xacro/index_finger/index_finger.xacro" />
-    <xacro:include filename="$(find val_description)/robots/common/xacro/middle_finger/middle_finger.xacro" />
-    <xacro:include filename="$(find val_description)/robots/common/xacro/pinky_finger/pinky_finger.xacro" />
+    <xacro:include filename="$(find val_description)/model/robots/common/xacro/pelvis/pelvis.xacro" />
+    <xacro:include filename="$(find val_description)/model/robots/common/xacro/waist/waist.xacro" />
+    <xacro:include filename="$(find val_description)/model/robots/common/xacro/head/head.xacro" />
+    <xacro:include filename="$(find val_description)/model/robots/common/xacro/arm/arm.xacro" />
+    <xacro:include filename="$(find val_description)/model/robots/common/xacro/thumb/thumb.xacro" />
+    <xacro:include filename="$(find val_description)/model/robots/common/xacro/index_finger/index_finger.xacro" />
+    <xacro:include filename="$(find val_description)/model/robots/common/xacro/middle_finger/middle_finger.xacro" />
+    <xacro:include filename="$(find val_description)/model/robots/common/xacro/pinky_finger/pinky_finger.xacro" />
 </robot>

File: model/robots/common/xacro/head/head.xacro (robot description, xacro)
@@ -1,10 +1,10 @@
 <robot xmlns:xacro="http://www.ros.org/wiki/xacro" name="head">
-  <xacro:include filename="$(find val_description)/robots/common/xacro/head/joint_names.xacro"/>
-  <xacro:include filename="$(find val_description)/robots/common/xacro/head/actuator_names.xacro"/>
-  <xacro:include filename="$(find val_description)/robots/common/xacro/head/joint_axes.xacro"/>
-  <xacro:include filename="$(find val_description)/robots/common/xacro/head/link_names.xacro"/>
-  <xacro:include filename="$(find val_description)/robots/common/xacro/head/joint_limits.xacro"/>
-  <xacro:include filename="$(find val_description)/robots/common/xacro/head/frame_parameters.xacro"/>
-  <xacro:include filename="$(find val_description)/robots/common/xacro/head/mass_parameters.xacro"/>
+  <xacro:include filename="$(find val_description)/model/robots/common/xacro/head/joint_names.xacro"/>
+  <xacro:include filename="$(find val_description)/model/robots/common/xacro/head/actuator_names.xacro"/>
+  <xacro:include filename="$(find val_description)/model/robots/common/xacro/head/joint_axes.xacro"/>
+  <xacro:include filename="$(find val_description)/model/robots/common/xacro/head/link_names.xacro"/>
+  <xacro:include filename="$(find val_description)/model/robots/common/xacro/head/joint_limits.xacro"/>
+  <xacro:include filename="$(find val_description)/model/robots/common/xacro/head/frame_parameters.xacro"/>
+  <xacro:include filename="$(find val_description)/model/robots/common/xacro/head/mass_parameters.xacro"/>
   <xacro:property name="NJ3_Link_Radius" value="0.139"/>
   <xacro:macro name="include_head" params="lower_neck_pitch_root_link">

File: model/robots/common/xacro/index_finger/index_finger.xacro (robot description, xacro)
@@ -1,11 +1,11 @@
 <?xml version="1.0" ?>
 <robot xmlns:xacro="http://www.ros.org/wiki/xacro" name="v1/index_finger">
-  <xacro:include filename="$(find val_description)/robots/common/xacro/index_finger/joint_names.xacro"/>
-  <xacro:include filename="$(find val_description)/robots/common/xacro/index_finger/joint_axes.xacro"/>
-  <xacro:include filename="$(find val_description)/robots/common/xacro/index_finger/actuator_names.xacro"/>
-  <xacro:include filename="$(find val_description)/robots/common/xacro/index_finger/link_names.xacro"/>
-  <xacro:include filename="$(find val_description)/robots/common/xacro/index_finger/joint_limits.xacro"/>
-  <xacro:include filename="$(find val_description)/robots/common/xacro/index_finger/frame_parameters.xacro"/>
-  <xacro:include filename="$(find val_description)/robots/common/xacro/index_finger/mass_parameters.xacro"/>
+  <xacro:include filename="$(find val_description)/model/robots/common/xacro/index_finger/joint_names.xacro"/>
+  <xacro:include filename="$(find val_description)/model/robots/common/xacro/index_finger/joint_axes.xacro"/>
+  <xacro:include filename="$(find val_description)/model/robots/common/xacro/index_finger/actuator_names.xacro"/>
+  <xacro:include filename="$(find val_description)/model/robots/common/xacro/index_finger/link_names.xacro"/>
+  <xacro:include filename="$(find val_description)/model/robots/common/xacro/index_finger/joint_limits.xacro"/>
+  <xacro:include filename="$(find val_description)/model/robots/common/xacro/index_finger/frame_parameters.xacro"/>
+  <xacro:include filename="$(find val_description)/model/robots/common/xacro/index_finger/mass_parameters.xacro"/>
   <xacro:macro name="make_index_finger" params="prefix reflect index_finger_root_link">
     <xacro:standard_link name="${IndexFingerPitch1LinkName}"

File: model/robots/common/xacro/middle_finger/middle_finger.xacro (robot description, xacro)
@@ -1,11 +1,11 @@
 <?xml version="1.0" ?>
 <robot xmlns:xacro="http://www.ros.org/wiki/xacro" name="middle_finger">
-  <xacro:include filename="$(find val_description)/robots/common/xacro/middle_finger/joint_names.xacro"/>
-  <xacro:include filename="$(find val_description)/robots/common/xacro/middle_finger/joint_axes.xacro"/>
-  <xacro:include filename="$(find val_description)/robots/common/xacro/middle_finger/actuator_names.xacro"/>
-  <xacro:include filename="$(find val_description)/robots/common/xacro/middle_finger/link_names.xacro"/>
-  <xacro:include filename="$(find val_description)/robots/common/xacro/middle_finger/joint_limits.xacro"/>
-  <xacro:include filename="$(find val_description)/robots/common/xacro/middle_finger/frame_parameters.xacro"/>
-  <xacro:include filename="$(find val_description)/robots/common/xacro/middle_finger/mass_parameters.xacro"/>
+  <xacro:include filename="$(find val_description)/model/robots/common/xacro/middle_finger/joint_names.xacro"/>
+  <xacro:include filename="$(find val_description)/model/robots/common/xacro/middle_finger/joint_axes.xacro"/>
+  <xacro:include filename="$(find val_description)/model/robots/common/xacro/middle_finger/actuator_names.xacro"/>
+  <xacro:include filename="$(find val_description)/model/robots/common/xacro/middle_finger/link_names.xacro"/>
+  <xacro:include filename="$(find val_description)/model/robots/common/xacro/middle_finger/joint_limits.xacro"/>
+  <xacro:include filename="$(find val_description)/model/robots/common/xacro/middle_finger/frame_parameters.xacro"/>
+  <xacro:include filename="$(find val_description)/model/robots/common/xacro/middle_finger/mass_parameters.xacro"/>
   <xacro:macro name="make_middle_finger" params="prefix reflect middle_finger_root_link">
     <xacro:standard_link name="${MiddleFingerPitch1LinkName}"

File: model/robots/common/xacro/pinky_finger/pinky_finger.xacro (robot description, xacro)
@@ -1,11 +1,11 @@
 <?xml version="1.0" ?>
 <robot xmlns:xacro="http://www.ros.org/wiki/xacro" name="pinky_finger">
-  <xacro:include filename="$(find val_description)/robots/common/xacro/pinky_finger/joint_names.xacro"/>
-  <xacro:include filename="$(find val_description)/robots/common/xacro/pinky_finger/joint_axes.xacro"/>
-  <xacro:include filename="$(find val_description)/robots/common/xacro/pinky_finger/actuator_names.xacro"/>
-  <xacro:include filename="$(find val_description)/robots/common/xacro/pinky_finger/link_names.xacro"/>
-  <xacro:include filename="$(find val_description)/robots/common/xacro/pinky_finger/joint_limits.xacro"/>
-  <xacro:include filename="$(find val_description)/robots/common/xacro/pinky_finger/frame_parameters.xacro"/>
-  <xacro:include filename="$(find val_description)/robots/common/xacro/pinky_finger/mass_parameters.xacro"/>
+  <xacro:include filename="$(find val_description)/model/robots/common/xacro/pinky_finger/joint_names.xacro"/>
+  <xacro:include filename="$(find val_description)/model/robots/common/xacro/pinky_finger/joint_axes.xacro"/>
+  <xacro:include filename="$(find val_description)/model/robots/common/xacro/pinky_finger/actuator_names.xacro"/>
+  <xacro:include filename="$(find val_description)/model/robots/common/xacro/pinky_finger/link_names.xacro"/>
+  <xacro:include filename="$(find val_description)/model/robots/common/xacro/pinky_finger/joint_limits.xacro"/>
+  <xacro:include filename="$(find val_description)/model/robots/common/xacro/pinky_finger/frame_parameters.xacro"/>
+  <xacro:include filename="$(find val_description)/model/robots/common/xacro/pinky_finger/mass_parameters.xacro"/>
   <xacro:macro name="make_pinky_finger" params="prefix reflect pinky_finger_root_link">
     <xacro:standard_link name="${PinkyPitch1LinkName}"

File: model/robots/common/xacro/thumb/thumb.xacro (robot description, xacro)
@@ -1,11 +1,11 @@
 <?xml version="1.0" ?>
 <robot xmlns:xacro="http://www.ros.org/wiki/xacro" name="thumb">
-  <xacro:include filename="$(find val_description)/robots/common/xacro/thumb/joint_names.xacro"/>
-  <xacro:include filename="$(find val_description)/robots/common/xacro/thumb/joint_axes.xacro"/>
-  <xacro:include filename="$(find val_description)/robots/common/xacro/thumb/actuator_names.xacro"/>
-  <xacro:include filename="$(find val_description)/robots/common/xacro/thumb/link_names.xacro"/>
-  <xacro:include filename="$(find val_description)/robots/common/xacro/thumb/joint_limits.xacro"/>
-  <xacro:include filename="$(find val_description)/robots/common/xacro/thumb/frame_parameters.xacro"/>
-  <xacro:include filename="$(find val_description)/robots/common/xacro/thumb/mass_parameters.xacro"/>
+  <xacro:include filename="$(find val_description)/model/robots/common/xacro/thumb/joint_names.xacro"/>
+  <xacro:include filename="$(find val_description)/model/robots/common/xacro/thumb/joint_axes.xacro"/>
+  <xacro:include filename="$(find val_description)/model/robots/common/xacro/thumb/actuator_names.xacro"/>
+  <xacro:include filename="$(find val_description)/model/robots/common/xacro/thumb/link_names.xacro"/>
+  <xacro:include filename="$(find val_description)/model/robots/common/xacro/thumb/joint_limits.xacro"/>
+  <xacro:include filename="$(find val_description)/model/robots/common/xacro/thumb/frame_parameters.xacro"/>
+  <xacro:include filename="$(find val_description)/model/robots/common/xacro/thumb/mass_parameters.xacro"/>
   <xacro:macro name="make_thumb" params="prefix reflect thumb_root_link">
     <xacro:standard_link name="${ThumbRollLinkName}"

File: model/robots/common/xacro/waist/waist.xacro (robot description, xacro)
@@ -1,13 +1,13 @@
 <robot xmlns:xacro="http://www.ros.org/wiki/xacro" name="waist">
-  <xacro:include filename="$(find val_description)/robots/common/xacro/waist/joint_names.xacro"/>
-  <xacro:include filename="$(find val_description)/robots/common/xacro/waist/actuator_names.xacro"/>
-  <xacro:include filename="$(find val_description)/robots/common/xacro/waist/joint_axes.xacro"/>
-  <xacro:include filename="$(find val_description)/robots/common/xacro/waist/joint_axes.xacro"/>
-  <xacro:include filename="$(find val_description)/robots/common/xacro/waist/link_names.xacro"/>
-  <xacro:include filename="$(find val_description)/robots/common/xacro/waist/joint_limits.xacro"/>
-  <xacro:include filename="$(find val_description)/robots/common/xacro/waist/frame_parameters.xacro"/>
-  <xacro:include filename="$(find val_description)/robots/common/xacro/waist/mass_parameters.xacro"/>
-  <xacro:include filename="$(find val_description)/robots/common/xacro/sensors/microstrain.xacro"/>
-  <xacro:include filename="$(find val_description)/robots/common/xacro/sensors/flea.xacro"/>
+  <xacro:include filename="$(find val_description)/model/robots/common/xacro/waist/joint_names.xacro"/>
+  <xacro:include filename="$(find val_description)/model/robots/common/xacro/waist/actuator_names.xacro"/>
+  <xacro:include filename="$(find val_description)/model/robots/common/xacro/waist/joint_axes.xacro"/>
+  <xacro:include filename="$(find val_description)/model/robots/common/xacro/waist/joint_axes.xacro"/>
+  <xacro:include filename="$(find val_description)/model/robots/common/xacro/waist/link_names.xacro"/>
+  <xacro:include filename="$(find val_description)/model/robots/common/xacro/waist/joint_limits.xacro"/>
+  <xacro:include filename="$(find val_description)/model/robots/common/xacro/waist/frame_parameters.xacro"/>
+  <xacro:include filename="$(find val_description)/model/robots/common/xacro/waist/mass_parameters.xacro"/>
+  <xacro:include filename="$(find val_description)/model/robots/common/xacro/sensors/microstrain.xacro"/>
+  <xacro:include filename="$(find val_description)/model/robots/common/xacro/sensors/flea.xacro"/>
   <xacro:macro name="make_waist_common" params="waist_root_link">
     <xacro:revolute_joint_ex jointName="${TorsoYawJointName}"

File: model/robots/valkyrie_A/xacro/leg/frame_parameters.xacro (robot description, xacro)
@@ -1,4 +1,4 @@
 <?xml version="1.0" ?>
-<robot xmlns:xacro="http://www.ros.org/wiki/xacro" name="v1/leg/dh_parameters">
+<robot xmlns:xacro="http://www.ros.org/wiki/xacro" name="leg_frame_parameters">
   <xacro:property name="HipYawFrameOrigin_X" value="0.0"/>
   <xacro:property name="HipYawFrameOrigin_Y" value="${reflect * 0.1016}"/>

File: model/robots/valkyrie_A/xacro/leg/joint_names.xacro (robot description, xacro)
@@ -1,4 +1,4 @@
 <?xml version="1.0" ?>
-<robot xmlns:xacro="http://www.ros.org/wiki/xacro" name="v1/leg/joint_names">
+<robot xmlns:xacro="http://www.ros.org/wiki/xacro" name="leg_joint_names">
   <xacro:property name="HipYawJointName" value="${prefix}HipYaw" />
   <xacro:property name="HipRollJointName" value="${prefix}HipRoll" />

File: model/robots/valkyrie_A/xacro/leg/leg.xacro (robot description, xacro)
@@ -1,12 +1,12 @@
 <?xml version="1.0" ?>
 <robot xmlns:xacro="http://www.ros.org/wiki/xacro" name="leg">
-  <xacro:include filename="$(find val_description)/robots/valkyrie_A/xacro/leg/joint_names.xacro"/>
-  <xacro:include filename="$(find val_description)/robots/valkyrie_A/xacro/leg/actuator_names.xacro"/>
-  <xacro:include filename="$(find val_description)/robots/valkyrie_A/xacro/leg/joint_axes.xacro"/>
-  <xacro:include filename="$(find val_description)/robots/valkyrie_A/xacro/leg/link_names.xacro"/>
-  <xacro:include filename="$(find val_description)/robots/valkyrie_A/xacro/leg/joint_limits.xacro"/>
-  <xacro:include filename="$(find val_description)/robots/valkyrie_A/xacro/leg/frame_parameters.xacro"/>
-  <xacro:include filename="$(find val_description)/robots/valkyrie_A/xacro/leg/mass_parameters.xacro"/>
-  <xacro:include filename="$(find val_description)/robots/common/xacro/sensors/ati_force_torque.xacro"/>
+  <xacro:include filename="$(find val_description)/model/robots/valkyrie_A/xacro/leg/joint_names.xacro"/>
+  <xacro:include filename="$(find val_description)/model/robots/valkyrie_A/xacro/leg/actuator_names.xacro"/>
+  <xacro:include filename="$(find val_description)/model/robots/valkyrie_A/xacro/leg/joint_axes.xacro"/>
+  <xacro:include filename="$(find val_description)/model/robots/valkyrie_A/xacro/leg/link_names.xacro"/>
+  <xacro:include filename="$(find val_description)/model/robots/valkyrie_A/xacro/leg/joint_limits.xacro"/>
+  <xacro:include filename="$(find val_description)/model/robots/valkyrie_A/xacro/leg/frame_parameters.xacro"/>
+  <xacro:include filename="$(find val_description)/model/robots/valkyrie_A/xacro/leg/mass_parameters.xacro"/>
+  <xacro:include filename="$(find val_description)/model/robots/common/xacro/sensors/ati_force_torque.xacro"/>
   <xacro:macro name="make_leg_links" params="prefix reflect leg_root_link">
     <xacro:standard_link name="${HipYawLinkName}"

File: model/robots/valkyrie_A_hw.xacro (robot description, xacro)
@@ -1,8 +1,8 @@
 <robot xmlns:xacro="http://ros.org/wiki/xacro" name="valkyrie">
-    <xacro:property name="mesh_root" value="package://val_description/meshes"/>
-    <xacro:include filename="$(find val_description)/robots/common/xacro/generic_models.xacro" />
-    <xacro:include filename="$(find val_description)/materials/materials.xacro" />
-    <xacro:include filename="$(find val_description)/robots/common/xacro/common_bodies.xacro" />
-    <xacro:include filename="$(find val_description)/robots/valkyrie_A/xacro/leg/leg.xacro" />
-    <xacro:include filename="$(find val_description)/robots/common/xacro/valkyrie_base_hw.xacro"/>
+    <xacro:property name="mesh_root" value="package://val_description/model/meshes"/>
+    <xacro:include filename="$(find val_description)/model/robots/common/xacro/generic_models.xacro" />
+    <xacro:include filename="$(find val_description)/model/materials/materials.xacro" />
+    <xacro:include filename="$(find val_description)/model/robots/common/xacro/common_bodies.xacro" />
+    <xacro:include filename="$(find val_description)/model/robots/valkyrie_A/xacro/leg/leg.xacro" />
+    <xacro:include filename="$(find val_description)/model/robots/common/xacro/valkyrie_base_hw.xacro"/>
 </robot>

File: model/robots/valkyrie_A_sim.xacro (robot description, xacro)
@@ -1,9 +1,9 @@
 <robot xmlns:xacro="http://ros.org/wiki/xacro" name="valkyrie">
-    <xacro:property name="mesh_root" value="package://val_description/meshes"/>
-    <xacro:include filename="$(find val_description)/robots/common/xacro/generic_models.xacro" />
-    <xacro:include filename="$(find val_description)/materials/materials.xacro" />
-    <xacro:include filename="$(find val_description)/robots/common/xacro/common_bodies.xacro" />
-    <xacro:include filename="$(find val_description)/robots/valkyrie_A/xacro/leg/leg.xacro" />
-    <xacro:include filename="$(find val_description)/robots/common/xacro/valkyrie_base_sim.xacro"/>
-    <xacro:include filename="$(find val_description)/urdf/multisense_sl.urdf" />
+    <xacro:property name="mesh_root" value="package://val_description/model/meshes"/>
+    <xacro:include filename="$(find val_description)/model/robots/common/xacro/generic_models.xacro" />
+    <xacro:include filename="$(find val_description)/model/materials/materials.xacro" />
+    <xacro:include filename="$(find val_description)/model/robots/common/xacro/common_bodies.xacro" />
+    <xacro:include filename="$(find val_description)/model/robots/valkyrie_A/xacro/leg/leg.xacro" />
+    <xacro:include filename="$(find val_description)/model/robots/common/xacro/valkyrie_base_sim.xacro"/>
+    <xacro:include filename="$(find val_description)/model/urdf/multisense_sl.urdf" />
 </robot>

File: model/robots/valkyrie_B/xacro/leg/link_names.xacro (robot description, xacro)
@@ -1,4 +1,4 @@
 <?xml version="1.0" ?>
-<robot xmlns:xacro="http://www.ros.org/wiki/xacro" name="v1/leg/link_names">
+<robot xmlns:xacro="http://www.ros.org/wiki/xacro" name="leg_link_names">
   <xacro:property name="HipYawParentLinkName" value="${leg_root_link}" />
   <xacro:property name="HipYawLinkName" value="${prefix}HipYawLink" />

File: model/robots/valkyrie_B_hw.xacro (robot description, xacro)
@@ -1,8 +1,8 @@
 <robot xmlns:xacro="http://ros.org/wiki/xacro" name="valkyrie">
-    <xacro:property name="mesh_root" value="package://val_description/meshes"/>
-    <xacro:include filename="$(find val_description)/robots/common/xacro/generic_models.xacro" />
-    <xacro:include filename="$(find val_description)/materials/materials.xacro" />
-    <xacro:include filename="$(find val_description)/robots/common/xacro/common_bodies.xacro" />
-    <xacro:include filename="$(find val_description)/robots/valkyrie_B/xacro/leg/leg.xacro" />
-    <xacro:include filename="$(find val_description)/robots/common/xacro/valkyrie_base_hw.xacro"/>
+    <xacro:property name="mesh_root" value="package://val_description/model/meshes"/>
+    <xacro:include filename="$(find val_description)/model/robots/common/xacro/generic_models.xacro" />
+    <xacro:include filename="$(find val_description)/model/materials/materials.xacro" />
+    <xacro:include filename="$(find val_description)/model/robots/common/xacro/common_bodies.xacro" />
+    <xacro:include filename="$(find val_description)/model/robots/valkyrie_B/xacro/leg/leg.xacro" />
+    <xacro:include filename="$(find val_description)/model/robots/common/xacro/valkyrie_base_hw.xacro"/>
 </robot>
