Commit message: Have urdf's generating again.

File: model/robots/valkyrie_B_sim.xacro (robot description, xacro)
@@ -1,9 +1,9 @@
 <robot xmlns:xacro="http://ros.org/wiki/xacro" name="valkyrie">
-    <xacro:property name="mesh_root" value="package://val_description/meshes"/>
-    <xacro:include filename="$(find val_description)/robots/common/xacro/generic_models.xacro" />
-    <xacro:include filename="$(find val_description)/materials/materials.xacro" />
-    <xacro:include filename="$(find val_description)/robots/common/xacro/common_bodies.xacro" />
-    <xacro:include filename="$(find val_description)/robots/valkyrie_B/xacro/leg/leg.xacro" />
-    <xacro:include filename="$(find val_description)/robots/common/xacro/valkyrie_base_sim.xacro"/>
-    <xacro:include filename="$(find val_description)/urdf/multisense_sl.urdf" />
+    <xacro:property name="mesh_root" value="package://val_description/model/meshes"/>
+    <xacro:include filename="$(find val_description)/model/robots/common/xacro/generic_models.xacro" />
+    <xacro:include filename="$(find val_description)/model/materials/materials.xacro" />
+    <xacro:include filename="$(find val_description)/model/robots/common/xacro/common_bodies.xacro" />
+    <xacro:include filename="$(find val_description)/model/robots/valkyrie_B/xacro/leg/leg.xacro" />
+    <xacro:include filename="$(find val_description)/model/robots/common/xacro/valkyrie_base_sim.xacro"/>
+    <xacro:include filename="$(find val_description)/model/urdf/multisense_sl.urdf" />
 </robot>

File: model/urdf/multisense_sl.urdf (robot description, URDF)
Before this commit: robot multisense_sl, 12 links, 11 joints
Links:
- link hokuyo_link: geometry collision box size=0.08 0.06 0.04238; collision cylinder length=0.047 radius=0.024425

Commit message: Removed some old files and changing the transmission tags a bit.

File: model/robots/common/xacro/arm/arm.xacro (robot description, xacro)
@@ -163,10 +163,10 @@
   </xacro:macro>
   <xacro:macro name="arm_transmissions" params="prefix">
-    <xacro:simple_transmission_force_controlled_joint jointName="${ShoulderPitchJointName}" actuatorName="${ShoulderPitchActuatorName}" nodeName="${ShoulderPitchNode}"/>
-    <xacro:simple_transmission_force_controlled_joint jointName="${ShoulderRollJointName}" actuatorName="${ShoulderRollActuatorName}" nodeName="${ShoulderRollNode}"/>
-    <xacro:simple_transmission_force_controlled_joint jointName="${ShoulderYawJointName}" actuatorName="${ShoulderYawActuatorName}" nodeName="${ShoulderYawNode}"/>
-    <xacro:simple_transmission_force_controlled_joint jointName="${ElbowPitchJointName}" actuatorName="${ElbowPitchActuatorName}" nodeName="${ElbowPitchNode}"/>
-    <xacro:simple_transmission_force_controlled_joint jointName="${ForearmYawActuatorName}" actuatorName="${ForearmYawActuatorName}" nodeName="${ForearmYawNode}"/>
-    <xacro:pushrod_transmission_position_controlled_joints transmissionName="${prefix}WristTransmission" joint1Name="${WristPitchJointName}" joint2Name="${WristRollJointName}" actuator1Name="${WristTopActuatorName}" actuator2Name="${WristBottomActuatorName}" actuator1Node="${WristTopActuatorNode}" actuator2Node="${WristBottomActuatorNode}"/>
+    <xacro:simple_transmission jointName="${ShoulderPitchJointName}" actuatorName="${ShoulderPitchActuatorName}" nodeName="${ShoulderPitchNode}"/>
+    <xacro:simple_transmission jointName="${ShoulderRollJointName}" actuatorName="${ShoulderRollActuatorName}" nodeName="${ShoulderRollNode}"/>
+    <xacro:simple_transmission jointName="${ShoulderYawJointName}" actuatorName="${ShoulderYawActuatorName}" nodeName="${ShoulderYawNode}"/>
+    <xacro:simple_transmission jointName="${ElbowPitchJointName}" actuatorName="${ElbowPitchActuatorName}" nodeName="${ElbowPitchNode}"/>
+    <xacro:simple_transmission jointName="${ForearmYawActuatorName}" actuatorName="${ForearmYawActuatorName}" nodeName="${ForearmYawNode}"/>
+    <xacro:pushrod_transmission transmissionName="${prefix}WristTransmission" joint1Name="${WristPitchJointName}" joint2Name="${WristRollJointName}" actuator1Name="${WristTopActuatorName}" actuator2Name="${WristBottomActuatorName}" actuator1Node="${WristTopActuatorNode}" actuator2Node="${WristBottomActuatorNode}"/>
   </xacro:macro>
 </robot>

File: model/robots/common/xacro/generic_models.xacro (robot description, xacro)
@@ -179,81 +179,38 @@
                        origin_xyz="${origin_xyz}"/>
   </xacro:macro>
-  <xacro:macro name="simple_transmission_force_controlled_joint" params="jointName actuatorName nodeName">
+  <xacro:macro name="simple_transmission" params="jointName actuatorName nodeName apiType">
     <transmission name="${jointName}Transmission">
       <type>transmission_interface/SimpleTransmission</type>
       <joint name="${jointName}">
-        <hardwareInterface>hardware_interface/EffortJointInterface</hardwareInterface>
-        <interface name="JointToActuatorPositionInterface"/>
       </joint>
       <actuator name="${actuatorName}">
         <node name="${nodeName}"/>
-        <interface name="ActuatorToJointPositionInterface"/>
         <mechanicalReduction>1</mechanicalReduction>
+        <api name="${apiType}" />
       </actuator>
     </transmission>
   </xacro:macro>
-  <xacro:macro name="simple_transmission_position_controlled_joint" params="jointName actuatorName nodeName">
-    <transmission name="${jointName}Transmission">
-      <type>transmission_interface/SimpleTransmission</type>
-      <joint name="${jointName}">
-        <hardwareInterface>hardware_interface/PositionJointInterface</hardwareInterface>
-        <interface name="JointToActuatorPositionInterface"/>
-      </joint>
-      <actuator name="${actuatorName}">
-        <node name="${nodeName}"/>
-        <interface name="ActuatorToJointPositionInterface"/>
-        <mechanicalReduction>1</mechanicalReduction>
-    </actuator>
-    </transmission>
-  </xacro:macro>
-  <xacro:macro name="pushrod_transmission_force_controlled_joints" params="transmissionName joint1Name joint2Name actuator1Name actuator2Name actuator1Node actuator2Node joint1Role joint2Role actuator1Role actuator2Role">
+  <xacro:macro name="pushrod_transmission" params="transmissionName joint1Name joint2Name actuator1Name actuator2Name actuator1Node actuator2Node joint1Role joint2Role actuator1Role actuator2Role api1Type api2Type">
     <transmission name="${transmissionName}">
       <type>transmission_interface/PushrodTransmission</type>
       <joint name="${joint1Name}">
-        <hardwareInterface>hardware_interface/EffortJointInterface</hardwareInterface>
-        <interface name="JointToActuatorEffortInterface"/>
         <role>${joint1Role}</role>
       </joint>
       <joint name="${joint2Name}">
-        <hardwareInterface>hardware_interface/EffortJointInterface</hardwareInterface>
-        <interface name="JointToActuatorEffortInterface"/>
         <role>${joint2Role}</role>
       </joint>
        <actuator name="${actuator1Name}">
         <node name="${actuator1Node}"/>
-        <interface name="ActuatorToJointEffortInterface"/>
         <role>${actuator1Role}</role>
         <mechanicalReduction>1</mechanicalReduction>
+        <api name="${api1Type}"/>
       </actuator>
       <actuator name="${actuator2Name}">
         <node name="${actuator2Node}"/>
-        <interface name="ActuatorToJointEffortInterface"/>
         <role>${actuator2Role}</role>
         <mechanicalReduction>1</mechanicalReduction>
+        <api name="${api2Type}"/>
       </actuator>
     </transmission>
   </xacro:macro>
-  <xacro:macro name="pushrod_transmission_position_controlled_joints" params="transmissionName joint1Name joint2Name actuator1Name actuator2Name actuator1Node actuator2Node">
-    <transmission name="${transmissionName}">
-      <type>transmission_interface/PushrodTransmission</type>
-      <joint name="${joint1Name}">
-        <hardwareInterface>hardware_interface/PositionJointInterface</hardwareInterface>
-        <interface name="JointToActuatorPositionInterface"/>
-      </joint>
-      <joint name="${joint2Name}">
-        <hardwareInterface>hardware_interface/PositionJointInterface</hardwareInterface>
-        <interface name="JointToActuatorPositionInterface"/>
-      </joint>
-       <actuator name="${actuator1Name}">
-        <node name="${actuator1Node}"/>
-        <interface name="ActuatorToJointPositionInterface"/>
-        <mechanicalReduction>1</mechanicalReduction>
-      </actuator>
-      <actuator name="${actuator2Name}">
-        <node name="${actuator2Node}"/>
-        <interface name="ActuatorToJointPositionInterface"/>
-        <mechanicalReduction>1</mechanicalReduction>
-      </actuator>
-    </transmission>
-  </xacro:macro>
 </robot>

File: model/robots/common/xacro/head/head.xacro (robot description, xacro)
@@ -75,7 +75,7 @@
     </xacro:macro>
     <xacro:macro name="neck_transmissions">
-      <xacro:simple_transmission_position_controlled_joint jointName="${LowerNeckPitchJointName}" actuatorName="${LowerNeckPitchActuatorName}" nodeName="${LowerNeckPitchNode}"/>
-      <xacro:simple_transmission_position_controlled_joint jointName="${NeckYawJointName}" actuatorName="${NeckYawActuatorName}" nodeName="${NeckYawNode}"/>
-      <xacro:simple_transmission_position_controlled_joint jointName="${UpperNeckPitchJointName}" actuatorName="${UpperNeckPitchActuatorName}" nodeName="${UpperNeckPitchNode}"/>
+      <xacro:simple_transmission jointName="${LowerNeckPitchJointName}" actuatorName="${LowerNeckPitchActuatorName}" nodeName="${LowerNeckPitchNode}"/>
+      <xacro:simple_transmission jointName="${NeckYawJointName}" actuatorName="${NeckYawActuatorName}" nodeName="${NeckYawNode}"/>
+      <xacro:simple_transmission jointName="${UpperNeckPitchJointName}" actuatorName="${UpperNeckPitchActuatorName}" nodeName="${UpperNeckPitchNode}"/>
     </xacro:macro>
 </robot>

File: model/robots/common/xacro/index_finger/index_finger.xacro (robot description, xacro)
@@ -3,5 +3,4 @@
   <xacro:include filename="$(find val_description)/common/xacro/joint_names/valkyrie_joint_names.xacro"/>
   <xacro:include filename="$(find val_description)/model/robots/common/xacro/index_finger/joint_axes.xacro"/>
-  <xacro:include filename="$(find val_description)/model/robots/common/xacro/index_finger/actuator_names.xacro"/>
   <xacro:include filename="$(find val_description)/model/robots/common/xacro/index_finger/link_names.xacro"/>
   <xacro:include filename="$(find val_description)/model/robots/common/xacro/index_finger/joint_limits.xacro"/>

File: model/robots/common/xacro/leg/leg.xacro (robot description, xacro)
@@ -149,9 +149,9 @@
   </xacro:macro>
   <xacro:macro name="leg_transmissions" params="prefix">
-    <xacro:simple_transmission_force_controlled_joint jointName="${HipYawJointName}" actuatorName="${HipYawActuatorName}" nodeName="${HipYawNode}"/>
-    <xacro:simple_transmission_force_controlled_joint jointName="${HipRollJointName}" actuatorName="${HipRollActuatorName}" nodeName="${HipRollNode}"/>
-    <xacro:simple_transmission_force_controlled_joint jointName="${HipPitchJointName}" actuatorName="${HipPitchActuatorName}" nodeName="${HipPitchNode}"/>
-    <xacro:simple_transmission_force_controlled_joint jointName="${KneePitchJointName}" actuatorName="${KneePitchActuatorName}" nodeName="${KneePitchNode}"/>
-    <xacro:pushrod_transmission_force_controlled_joints transmissionName="${prefix}AnkleTransmission" joint1Name="${AnklePitchJointName}" joint2Name="${AnkleRollJointName}" actuator1Name="${AnkleInsideActuatorName}" actuator2Name="${AnkleOutsideActuatorName}" actuator1Node="${AnkleInsideActuatorNode}" actuator2Node="${AnkleOutsideActuatorNode}" joint1Role="pitch" joint2Role="roll" actuator1Role="insideActuator" actuator2Role="outsideActuator"/>
+    <xacro:simple_transmission jointName="${HipYawJointName}" actuatorName="${HipYawActuatorName}" nodeName="${HipYawNode}"/>
+    <xacro:simple_transmission jointName="${HipRollJointName}" actuatorName="${HipRollActuatorName}" nodeName="${HipRollNode}"/>
+    <xacro:simple_transmission jointName="${HipPitchJointName}" actuatorName="${HipPitchActuatorName}" nodeName="${HipPitchNode}"/>
+    <xacro:simple_transmission jointName="${KneePitchJointName}" actuatorName="${KneePitchActuatorName}" nodeName="${KneePitchNode}"/>
+    <xacro:pushrod_transmission transmissionName="${prefix}AnkleTransmission" joint1Name="${AnklePitchJointName}" joint2Name="${AnkleRollJointName}" actuator1Name="${AnkleInsideActuatorName}" actuator2Name="${AnkleOutsideActuatorName}" actuator1Node="${AnkleInsideActuatorNode}" actuator2Node="${AnkleOutsideActuatorNode}" joint1Role="pitch" joint2Role="roll" actuator1Role="insideActuator" actuator2Role="outsideActuator"/>
   </xacro:macro>
 </robot>

File: model/robots/common/xacro/middle_finger/middle_finger.xacro (robot description, xacro)
@@ -3,5 +3,4 @@
   <xacro:include filename="$(find val_description)/common/xacro/joint_names/valkyrie_joint_names.xacro"/>
   <xacro:include filename="$(find val_description)/model/robots/common/xacro/middle_finger/joint_axes.xacro"/>
-  <xacro:include filename="$(find val_description)/model/robots/common/xacro/middle_finger/actuator_names.xacro"/>
   <xacro:include filename="$(find val_description)/model/robots/common/xacro/middle_finger/link_names.xacro"/>
   <xacro:include filename="$(find val_description)/model/robots/common/xacro/middle_finger/joint_limits.xacro"/>

File: model/robots/common/xacro/pinky_finger/pinky_finger.xacro (robot description, xacro)
@@ -3,5 +3,4 @@
   <xacro:include filename="$(find val_description)/common/xacro/joint_names/valkyrie_joint_names.xacro"/>
   <xacro:include filename="$(find val_description)/model/robots/common/xacro/pinky_finger/joint_axes.xacro"/>
-  <xacro:include filename="$(find val_description)/model/robots/common/xacro/pinky_finger/actuator_names.xacro"/>
   <xacro:include filename="$(find val_description)/model/robots/common/xacro/pinky_finger/link_names.xacro"/>
   <xacro:include filename="$(find val_description)/model/robots/common/xacro/pinky_finger/joint_limits.xacro"/>

File: model/robots/common/xacro/thumb/thumb.xacro (robot description, xacro)
@@ -3,5 +3,4 @@
   <xacro:include filename="$(find val_description)/common/xacro/joint_names/valkyrie_joint_names.xacro"/>
   <xacro:include filename="$(find val_description)/model/robots/common/xacro/thumb/joint_axes.xacro"/>
-  <xacro:include filename="$(find val_description)/model/robots/common/xacro/thumb/actuator_names.xacro"/>
   <xacro:include filename="$(find val_description)/model/robots/common/xacro/thumb/link_names.xacro"/>
   <xacro:include filename="$(find val_description)/model/robots/common/xacro/thumb/joint_limits.xacro"/>

File: model/robots/common/xacro/waist/waist.xacro (robot description, xacro)
@@ -98,6 +98,6 @@
    </xacro:macro>
    <xacro:macro name="waist_transmissions">
-    <xacro:simple_transmission_force_controlled_joint jointName="${TorsoYawJointName}" actuatorName="${TorsoYawActuatorName}" nodeName="${TrunkYawNode}"/>
-    <xacro:pushrod_transmission_force_controlled_joints transmissionName="WaistTransmission" joint1Name="${TorsoPitchJointName}" joint2Name="${TorsoRollJointName}" actuator1Name="${WaistLeftActuatorName}" actuator2Name="${WaistRightActuatorName}" actuator1Node="${WaistLeftActuatorNode}" actuator2Node="${WaistRightActuatorNode}" joint1Role="pitch" joint2Role="roll" actuator1Role="leftActuator" actuator2Role="rightActuator"/>
+    <xacro:simple_transmission jointName="${TorsoYawJointName}" actuatorName="${TorsoYawActuatorName}" nodeName="${TrunkYawNode}"/>
+    <xacro:pushrod_transmission transmissionName="WaistTransmission" joint1Name="${TorsoPitchJointName}" joint2Name="${TorsoRollJointName}" actuator1Name="${WaistLeftActuatorName}" actuator2Name="${WaistRightActuatorName}" actuator1Node="${WaistLeftActuatorNode}" actuator2Node="${WaistRightActuatorNode}" joint1Role="pitch" joint2Role="roll" actuator1Role="leftActuator" actuator2Role="rightActuator"/>
    </xacro:macro>
 </robot>
