Commit message: Added a simple transmissions to sim urdf. Finished moving things around in hw transmissions.

File: model/robots/common/xacro/arm/arm.xacro (robot description, xacro)
@@ -4,4 +4,5 @@
   <xacro:include filename="$(find val_description)/common/xacro/actuator_names/valkyrie_actuator_names.xacro"/>
   <xacro:include filename="$(find val_description)/common/xacro/nodes/valkyrie_nodes.xacro"/>
+  <xacro:include filename="$(find val_description)/common/xacro/api/valkyrie_api.xacro"/>
   <xacro:include filename="$(find val_description)/model/robots/common/xacro/arm/joint_axes.xacro"/>
   <xacro:include filename="$(find val_description)/model/robots/common/xacro/arm/link_names.xacro"/>
@@ -162,11 +163,20 @@
     <xacro:make_lower_arm prefix="${prefix}" reflect="${reflect}" lower_arm_root_link="${ElbowPitchLinkName}" />
   </xacro:macro>
-  <xacro:macro name="arm_transmissions" params="prefix">
-    <xacro:simple_transmission jointName="${ShoulderPitchJointName}" actuatorName="${ShoulderPitchActuatorName}" nodeName="${ShoulderPitchNode}"/>
-    <xacro:simple_transmission jointName="${ShoulderRollJointName}" actuatorName="${ShoulderRollActuatorName}" nodeName="${ShoulderRollNode}"/>
-    <xacro:simple_transmission jointName="${ShoulderYawJointName}" actuatorName="${ShoulderYawActuatorName}" nodeName="${ShoulderYawNode}"/>
-    <xacro:simple_transmission jointName="${ElbowPitchJointName}" actuatorName="${ElbowPitchActuatorName}" nodeName="${ElbowPitchNode}"/>
-    <xacro:simple_transmission jointName="${ForearmYawActuatorName}" actuatorName="${ForearmYawActuatorName}" nodeName="${ForearmYawNode}"/>
-    <xacro:pushrod_transmission transmissionName="${prefix}WristTransmission" joint1Name="${WristPitchJointName}" joint2Name="${WristRollJointName}" actuator1Name="${WristTopActuatorName}" actuator2Name="${WristBottomActuatorName}" actuator1Node="${WristTopActuatorNode}" actuator2Node="${WristBottomActuatorNode}"/>
+  <xacro:macro name="arm_transmissions_hw" params="prefix">
+    <xacro:simple_transmission jointName="${ShoulderPitchJointName}" actuatorName="${ShoulderPitchActuatorName}" nodeName="${ShoulderPitchNode}" actuatorApi="${ShoulderPitchApi}"/>
+    <xacro:simple_transmission jointName="${ShoulderRollJointName}" actuatorName="${ShoulderRollActuatorName}" nodeName="${ShoulderRollNode}" actuatorApi="${ShoulderRollApi}"/>
+    <xacro:simple_transmission jointName="${ShoulderYawJointName}" actuatorName="${ShoulderYawActuatorName}" nodeName="${ShoulderYawNode}" actuatorApi="${ShoulderYawApi}"/>
+    <xacro:simple_transmission jointName="${ElbowPitchJointName}" actuatorName="${ElbowPitchActuatorName}" nodeName="${ElbowPitchNode}" actuatorApi="${ElbowPitchApi}"/>
+    <xacro:simple_transmission jointName="${ForearmYawActuatorName}" actuatorName="${ForearmYawActuatorName}" nodeName="${ForearmYawNode}" actuatorApi="${ForearmYawApi}"/>
+    <xacro:pushrod_transmission transmissionName="${prefix}WristTransmission" joint1Name="${WristPitchJointName}" joint2Name="${WristRollJointName}" actuator1Name="${WristTopActuatorName}" actuator2Name="${WristBottomActuatorName}" actuator1Node="${WristTopActuatorNode}" actuator2Node="${WristBottomActuatorNode}" joint1Role="roll" joint2Role="pitch" actuator1Role="actuator1" actuator2Role="actuator2" actuator1Api="WristTopActuatorApi" actuator2Api="${WristBottomActuatorApi}"/>
+  </xacro:macro>
+  <xacro:macro name="arm_transmissions_sim" params="prefix">
+    <xacro:simple_transmission jointName="${ShoulderPitchJointName}" actuatorName="${ShoulderPitchActuatorName}" nodeName="${ShoulderPitchNode}" actuatorApi="${SimApi}"/>
+    <xacro:simple_transmission jointName="${ShoulderRollJointName}" actuatorName="${ShoulderRollActuatorName}" nodeName="${ShoulderRollNode}" actuatorApi="${SimApi}"/>
+    <xacro:simple_transmission jointName="${ShoulderYawJointName}" actuatorName="${ShoulderYawActuatorName}" nodeName="${ShoulderYawNode}" actuatorApi="${SimApi}"/>
+    <xacro:simple_transmission jointName="${ElbowPitchJointName}" actuatorName="${ElbowPitchActuatorName}" nodeName="${ElbowPitchNode}" actuatorApi="${SimApi}"/>
+    <xacro:simple_transmission jointName="${ForearmYawActuatorName}" actuatorName="${ForearmYawActuatorName}" nodeName="${ForearmYawNode}" actuatorApi="${SimApi}"/>
+    <xacro:simple_transmission jointName="${WristRollJointName}" actuatorName="${WristTopActuatorName}" nodeName="${WristTopActuatorNode}" actuatorApi="${SimApi}"/>
+    <xacro:simple_transmission jointName="${WristPitchJointName}" actuatorName="${WristBottomActuatorName}" nodeName="${WristBottomActuatorNode}" actuatorApi="${SimApi}"/>
   </xacro:macro>
 </robot>

File: model/robots/common/xacro/generic_models.xacro (robot description, xacro)
@@ -179,5 +179,5 @@
                        origin_xyz="${origin_xyz}"/>
   </xacro:macro>
-  <xacro:macro name="simple_transmission" params="jointName actuatorName nodeName apiType">
+  <xacro:macro name="simple_transmission" params="jointName actuatorName nodeName actuatorApi">
     <transmission name="${jointName}Transmission">
       <type>transmission_interface/SimpleTransmission</type>
@@ -187,9 +187,9 @@
         <node name="${nodeName}"/>
         <mechanicalReduction>1</mechanicalReduction>
-        <api name="${apiType}" />
+        <api name="${actuatorApi}" />
       </actuator>
     </transmission>
   </xacro:macro>
-  <xacro:macro name="pushrod_transmission" params="transmissionName joint1Name joint2Name actuator1Name actuator2Name actuator1Node actuator2Node joint1Role joint2Role actuator1Role actuator2Role api1Type api2Type">
+  <xacro:macro name="pushrod_transmission" params="transmissionName joint1Name joint2Name actuator1Name actuator2Name actuator1Node actuator2Node joint1Role joint2Role actuator1Role actuator2Role actuator1Api actuator2Api">
     <transmission name="${transmissionName}">
       <type>transmission_interface/PushrodTransmission</type>
@@ -204,5 +204,5 @@
         <role>${actuator1Role}</role>
         <mechanicalReduction>1</mechanicalReduction>
-        <api name="${api1Type}"/>
+        <api name="${actuator1Api}"/>
       </actuator>
       <actuator name="${actuator2Name}">
@@ -210,5 +210,5 @@
         <role>${actuator2Role}</role>
         <mechanicalReduction>1</mechanicalReduction>
-        <api name="${api2Type}"/>
+        <api name="${actuator2Api}"/>
       </actuator>
     </transmission>

File: model/robots/common/xacro/head/head.xacro (robot description, xacro)
@@ -3,4 +3,5 @@
   <xacro:include filename="$(find val_description)/common/xacro/actuator_names/valkyrie_actuator_names.xacro"/>
   <xacro:include filename="$(find val_description)/common/xacro/nodes/valkyrie_nodes.xacro"/>
+  <xacro:include filename="$(find val_description)/common/xacro/api/valkyrie_api.xacro"/>
   <xacro:include filename="$(find val_description)/model/robots/common/xacro/head/joint_axes.xacro"/>
   <xacro:include filename="$(find val_description)/model/robots/common/xacro/head/link_names.xacro"/>
@@ -74,8 +75,13 @@
       <xacro:fixed_joint jointName="multisense_head_root_joint" parent="${UpperNeckPitchLinkName}" child="multisense_root_link" origin_xyz="0.183585961 0.0 0.075353826" origin_rpy="-3.14159 0.130899694 0.0" />
     </xacro:macro>
-    <xacro:macro name="neck_transmissions">
-      <xacro:simple_transmission jointName="${LowerNeckPitchJointName}" actuatorName="${LowerNeckPitchActuatorName}" nodeName="${LowerNeckPitchNode}"/>
-      <xacro:simple_transmission jointName="${NeckYawJointName}" actuatorName="${NeckYawActuatorName}" nodeName="${NeckYawNode}"/>
-      <xacro:simple_transmission jointName="${UpperNeckPitchJointName}" actuatorName="${UpperNeckPitchActuatorName}" nodeName="${UpperNeckPitchNode}"/>
+    <xacro:macro name="neck_transmissions_hw">
+      <xacro:simple_transmission jointName="${LowerNeckPitchJointName}" actuatorName="${LowerNeckPitchActuatorName}" nodeName="${LowerNeckPitchNode}" actuatorApi="${LowerNeckPitchApi}"/>
+      <xacro:simple_transmission jointName="${NeckYawJointName}" actuatorName="${NeckYawActuatorName}" nodeName="${NeckYawNode}" actuatorApi="${NeckYawApi}"/>
+      <xacro:simple_transmission jointName="${UpperNeckPitchJointName}" actuatorName="${UpperNeckPitchActuatorName}" nodeName="${UpperNeckPitchNode}" actuatorApi="${UpperNeckPitchApi}"/>
+    </xacro:macro>
+    <xacro:macro name="neck_transmissions_sim">
+      <xacro:simple_transmission jointName="${LowerNeckPitchJointName}" actuatorName="${LowerNeckPitchActuatorName}" nodeName="${LowerNeckPitchNode}" actuatorApi="${SimApi}"/>
+      <xacro:simple_transmission jointName="${NeckYawJointName}" actuatorName="${NeckYawActuatorName}" nodeName="${NeckYawNode}" actuatorApi="${SimApi}"/>
+      <xacro:simple_transmission jointName="${UpperNeckPitchJointName}" actuatorName="${UpperNeckPitchActuatorName}" nodeName="${UpperNeckPitchNode}" actuatorApi="${SimApi}"/>
     </xacro:macro>
 </robot>

File: model/robots/common/xacro/leg/leg.xacro (robot description, xacro)
@@ -1,7 +1,8 @@
 <?xml version="1.0" ?>
 <robot xmlns:xacro="http://www.ros.org/wiki/xacro" name="leg">
-    <xacro:include filename="$(find val_description)/common/xacro/joint_names/valkyrie_joint_names.xacro"/>
+  <xacro:include filename="$(find val_description)/common/xacro/joint_names/valkyrie_joint_names.xacro"/>
   <xacro:include filename="$(find val_description)/common/xacro/actuator_names/valkyrie_actuator_names.xacro"/>
   <xacro:include filename="$(find val_description)/common/xacro/nodes/valkyrie_nodes.xacro"/>
+  <xacro:include filename="$(find val_description)/common/xacro/api/valkyrie_api.xacro"/>
   <xacro:include filename="$(find val_description)/model/robots/common/xacro/leg/joint_axes.xacro"/>
   <xacro:include filename="$(find val_description)/model/robots/common/xacro/leg/link_names.xacro"/>
@@ -148,10 +149,18 @@
                         origin_rpy="3.14 0.0 -1.047"/>
   </xacro:macro>
-  <xacro:macro name="leg_transmissions" params="prefix">
-    <xacro:simple_transmission jointName="${HipYawJointName}" actuatorName="${HipYawActuatorName}" nodeName="${HipYawNode}"/>
-    <xacro:simple_transmission jointName="${HipRollJointName}" actuatorName="${HipRollActuatorName}" nodeName="${HipRollNode}"/>
-    <xacro:simple_transmission jointName="${HipPitchJointName}" actuatorName="${HipPitchActuatorName}" nodeName="${HipPitchNode}"/>
-    <xacro:simple_transmission jointName="${KneePitchJointName}" actuatorName="${KneePitchActuatorName}" nodeName="${KneePitchNode}"/>
-    <xacro:pushrod_transmission transmissionName="${prefix}AnkleTransmission" joint1Name="${AnklePitchJointName}" joint2Name="${AnkleRollJointName}" actuator1Name="${AnkleInsideActuatorName}" actuator2Name="${AnkleOutsideActuatorName}" actuator1Node="${AnkleInsideActuatorNode}" actuator2Node="${AnkleOutsideActuatorNode}" joint1Role="pitch" joint2Role="roll" actuator1Role="insideActuator" actuator2Role="outsideActuator"/>
+  <xacro:macro name="leg_transmissions_hw" params="prefix">
+    <xacro:simple_transmission jointName="${HipYawJointName}" actuatorName="${HipYawActuatorName}" nodeName="${HipYawNode}" actuatorApi="${HipYawApi}"/>
+    <xacro:simple_transmission jointName="${HipRollJointName}" actuatorName="${HipRollActuatorName}" nodeName="${HipRollNode}" actuatorApi="${HipRollApi}"/>
+    <xacro:simple_transmission jointName="${HipPitchJointName}" actuatorName="${HipPitchActuatorName}" nodeName="${HipPitchNode}" actuatorApi="${HipPitchApi}"/>
+    <xacro:simple_transmission jointName="${KneePitchJointName}" actuatorName="${KneePitchActuatorName}" nodeName="${KneePitchNode}" actuatorApi="${KneePitchApi}"/>
+    <xacro:pushrod_transmission transmissionName="${prefix}AnkleTransmission" joint1Name="${AnklePitchJointName}" joint2Name="${AnkleRollJointName}" actuator1Name="${AnkleInsideActuatorName}" actuator2Name="${AnkleOutsideActuatorName}" actuator1Node="${AnkleInsideActuatorNode}" actuator2Node="${AnkleOutsideActuatorNode}" joint1Role="pitch" joint2Role="roll" actuator1Role="insideActuator" actuator2Role="outsideActuator" actuator1Api="${AnkleInsideActuatorApi}" actuator2Api="${AnkleOutsideActuatorApi}"/>
+  </xacro:macro>
+  <xacro:macro name="leg_transmissions_sim" params="prefix">
+    <xacro:simple_transmission jointName="${HipYawJointName}" actuatorName="${HipYawActuatorName}" nodeName="${HipYawNode}" actuatorApi="${SimApi}"/>
+    <xacro:simple_transmission jointName="${HipRollJointName}" actuatorName="${HipRollActuatorName}" nodeName="${HipRollNode}" actuatorApi="${SimApi}"/>
+    <xacro:simple_transmission jointName="${HipPitchJointName}" actuatorName="${HipPitchActuatorName}" nodeName="${HipPitchNode}" actuatorApi="${SimApi}"/>
+    <xacro:simple_transmission jointName="${KneePitchJointName}" actuatorName="${KneePitchActuatorName}" nodeName="${KneePitchNode}" actuatorApi="${SimApi}"/>
+    <xacro:simple_transmission jointName="${AnklePitchJointName}" actuatorName="${AnkleInsideActuatorName}" nodeName="${AnkleInsideActuatorNode}" actuatorApi="${SimApi}"/>
+    <xacro:simple_transmission jointName="${AnkleRollJointName}" actuatorName="${AnkleOutsideActuatorName}" nodeName="${AnkleOutsideActuatorNode}" actuatorApi="${SimApi}"/>
   </xacro:macro>
 </robot>

File: model/robots/common/xacro/valkyrie_base_hw.xacro (robot description, xacro)
@@ -20,9 +20,9 @@
     <xacro:include_multisense_hw />
     <xacro:v1_pelvis_sensors/>
-    <xacro:waist_transmissions />
-    <xacro:leg_transmissions prefix="left"/>
-    <xacro:leg_transmissions prefix="right"/>
-    <xacro:arm_transmissions prefix="left"/>
-    <xacro:arm_transmissions prefix="right"/>
-    <xacro:neck_transmissions />
+    <xacro:waist_transmissions_hw />
+    <xacro:leg_transmissions_hw prefix="left"/>
+    <xacro:leg_transmissions_hw prefix="right"/>
+    <xacro:arm_transmissions_hw prefix="left"/>
+    <xacro:arm_transmissions_hw prefix="right"/>
+    <xacro:neck_transmissions_hw />
 </robot>

File: model/robots/common/xacro/valkyrie_base_sim.xacro (robot description, xacro)
@@ -20,3 +20,9 @@
     <xacro:include_multisense_sim />
     <xacro:v1_trunk_sensors/>
+    <xacro:waist_transmissions_sim />
+    <xacro:leg_transmissions_sim prefix="left"/>
+    <xacro:leg_transmissions_sim prefix="right"/>
+    <xacro:arm_transmissions_sim prefix="left"/>
+    <xacro:arm_transmissions_sim prefix="right"/>
+    <xacro:neck_transmissions_sim />
 </robot>

File: model/robots/common/xacro/waist/waist.xacro (robot description, xacro)
@@ -3,4 +3,5 @@
   <xacro:include filename="$(find val_description)/common/xacro/actuator_names/valkyrie_actuator_names.xacro"/>
   <xacro:include filename="$(find val_description)/common/xacro/nodes/valkyrie_nodes.xacro"/>
+  <xacro:include filename="$(find val_description)/common/xacro/api/valkyrie_api.xacro"/>
   <xacro:include filename="$(find val_description)/model/robots/common/xacro/waist/joint_axes.xacro"/>
   <xacro:include filename="$(find val_description)/model/robots/common/xacro/waist/joint_axes.xacro"/>
@@ -97,7 +98,12 @@
                         frameRate="60"/>
    </xacro:macro>
-   <xacro:macro name="waist_transmissions">
-    <xacro:simple_transmission jointName="${TorsoYawJointName}" actuatorName="${TorsoYawActuatorName}" nodeName="${TrunkYawNode}"/>
-    <xacro:pushrod_transmission transmissionName="WaistTransmission" joint1Name="${TorsoPitchJointName}" joint2Name="${TorsoRollJointName}" actuator1Name="${WaistLeftActuatorName}" actuator2Name="${WaistRightActuatorName}" actuator1Node="${WaistLeftActuatorNode}" actuator2Node="${WaistRightActuatorNode}" joint1Role="pitch" joint2Role="roll" actuator1Role="leftActuator" actuator2Role="rightActuator"/>
+   <xacro:macro name="waist_transmissions_hw">
+    <xacro:simple_transmission jointName="${TorsoYawJointName}" actuatorName="${TorsoYawActuatorName}" nodeName="${TrunkYawNode}" actuatorApi="${TrunkYawApi}"/>
+    <xacro:pushrod_transmission transmissionName="WaistTransmission" joint1Name="${TorsoPitchJointName}" joint2Name="${TorsoRollJointName}" actuator1Name="${WaistLeftActuatorName}" actuator2Name="${WaistRightActuatorName}" actuator1Node="${WaistLeftActuatorNode}" actuator2Node="${WaistRightActuatorNode}" joint1Role="pitch" joint2Role="roll" actuator1Role="leftActuator" actuator2Role="rightActuator" actuator1Api="${WaistLeftActuatorApi}" actuator2Api="${WaistRightActuatorApi}"/>
+   </xacro:macro>
+   <xacro:macro name="waist_transmissions_sim">
+    <xacro:simple_transmission jointName="${TorsoYawJointName}" actuatorName="${TorsoYawActuatorName}" nodeName="${TrunkYawNode}" actuatorApi="${SimApi}"/>
+    <xacro:simple_transmission jointName="${TorsoPitchJointName}" actuatorName="${WaistLeftActuatorName}" nodeName="${WaistLeftActuatorNode}" actuatorApi="${SimApi}"/>
+    <xacro:simple_transmission jointName="${TorsoRollJointName}" actuatorName="${WaistRightActuatorName}" nodeName="${WaistRightActuatorNode}" actuatorApi="${SimApi}"/>
    </xacro:macro>
 </robot>
