Commit message: remove references to gazebo colors which aren't referenced in urdf
the colors were removed by 485b59e4036b574286c72c7e8cbea9c5129e7b52
this commit removed materials.xacro from valkyrie_A_sim.xacro

File: model/robots/common/xacro/arm/arm.xacro (robot description, xacro)
@@ -17,5 +17,4 @@
                     iyy="${ShoulderPitchLinkInertia_IYY}" iyz="${ShoulderPitchLinkInertia_IYZ}" izz="${ShoulderPitchLinkInertia_IZZ}"
                     visual_mesh="${mesh_root}/arms/aj1_${prefix}.dae"
-                    material="Gold"
                     collision_mesh="${mesh_root}/arms/aj1_${prefix}.dae" />
     <xacro:standard_link name="${ShoulderRollLinkName}"
@@ -26,5 +25,4 @@
                     origin_rpy="0 0 0"
                     visual_mesh="${mesh_root}/arms/aj2_${prefix}.dae"
-                    material="White"
                     collision_mesh="${mesh_root}/arms/aj2_${prefix}.dae" />
     <xacro:standard_link name="${ShoulderYawLinkName}"
@@ -35,5 +33,4 @@
                     origin_rpy="0 0 0"
                     visual_mesh="${mesh_root}/arms/aj3_${prefix}.dae"
-                    material="White"
                     collision_mesh="${mesh_root}/arms/aj3_${prefix}.dae" />
     <xacro:standard_link name="${ElbowPitchLinkName}"
@@ -44,5 +41,4 @@
                     origin_rpy="0 0 0"
                     visual_mesh="${mesh_root}/arms/aj4_${prefix}.dae"
-                    material="Gold"
                     collision_mesh="${mesh_root}/arms/aj4_${prefix}.dae" />
     <xacro:revolute_joint_ex jointName="${ShoulderPitchJointName}"
@@ -101,5 +97,4 @@
                     origin_rpy="0 0 0"
                     visual_mesh="${mesh_root}/arms/aj5_${prefix}.dae"
-                    material="White"
                     collision_mesh="${mesh_root}/arms/aj5_${prefix}.dae" />
     <xacro:standard_link name="${WristRollLinkName}"
@@ -110,5 +105,4 @@
                     origin_rpy="0 0 0"
                     visual_mesh="${mesh_root}/arms/aj6_${prefix}.dae"
-                    material="White"
                     collision_mesh="${mesh_root}/arms/aj6_${prefix}.dae" />
     <xacro:standard_link name="${WristPitchLinkName}"
@@ -119,5 +113,4 @@
                     origin_rpy="0 0 0"
                     visual_mesh="${mesh_root}/arms/palm_${prefix}.dae"
-                    material="Gold"
                     collision_mesh="${mesh_root}/arms/palm_${prefix}.dae"/>
     <xacro:revolute_joint_ex jointName="${ForearmYawJointName}"

File: model/robots/common/xacro/generic_models.xacro (robot description, xacro)
@@ -4,5 +4,5 @@
     <actuator name="${name}" type="${api}"/>
   </xacro:macro>
-  <xacro:macro name="standard_link" params="name mass origin_rpy origin_xyz ixx ixy ixz iyy iyz izz visual_mesh material collision_mesh">
+  <xacro:macro name="standard_link" params="name mass origin_rpy origin_xyz ixx ixy ixz iyy iyz izz visual_mesh collision_mesh">
     <link name="${name}">
       <inertial>
@@ -18,5 +18,4 @@
           </geometry>
           <origin rpy="0.0 0.0 0.0" xyz="0.0 0.0 0.0"/>
-          <material name="${material}"/>
         </visual>
         <collision>
@@ -53,5 +52,5 @@
   </xacro:macro>
   <xacro:macro name="link_box_collision_mesh_visual"
-          params="name width height depth mass inertial_xyz inertial_rpy ixx ixy ixz iyy iyz izz visual_mesh material box_xyz box_rpy">
+          params="name width height depth mass inertial_xyz inertial_rpy ixx ixy ixz iyy iyz izz visual_mesh box_xyz box_rpy">
     <link name="${name}">
       <inertial>
@@ -67,5 +66,4 @@
         </geometry>
         <origin rpy="0 0 0" xyz="0 0 0"/>
-        <material name="${material}"/>
       </visual>
       <collision>

File: model/robots/common/xacro/head/head.xacro (robot description, xacro)
@@ -20,5 +20,4 @@
                         iyy="${LowerNeckPitchLinkInertia_IYY}" iyz="${LowerNeckPitchLinkInertia_IYZ}" izz="${LowerNeckPitchLinkInertia_IZZ}"
                         visual_mesh="${mesh_root}/head/neckj1.dae"
-                        material="White"
                         collision_mesh="${mesh_root}/head/neckj1.dae"/>
     <xacro:standard_link name="${NeckYawLinkName}"
@@ -29,5 +28,4 @@
                         iyy="${NeckYawLinkInertia_IYY}" iyz="${NeckYawLinkInertia_IYZ}" izz="${NeckYawLinkInertia_IZZ}"
                         visual_mesh="${mesh_root}/head/neckj2.dae"
-                        material="White"
                         collision_mesh="${mesh_root}/head/neckj2.dae" />
     <xacro:standard_link name="${UpperNeckPitchLinkName}"
@@ -38,5 +36,4 @@
                        origin_rpy="0 0 0"
                        visual_mesh="${mesh_root}/head/head_multisense_no_visor.dae"
-                       material="White"
                        collision_mesh="${mesh_root}/head/head_multisense_no_visor.dae"/>
     <xacro:revolute_joint_ex jointName="${LowerNeckPitchJointName}"

File: model/robots/common/xacro/index_finger/index_finger.xacro (robot description, xacro)
@@ -15,5 +15,4 @@
                     origin_rpy="0 0 0"
                     visual_mesh="${mesh_root}/fingers/indexj1_${prefix}.dae"
-                    material="Gold"
                     collision_mesh="${mesh_root}/fingers/indexj1_${prefix}.dae"/>
     <xacro:standard_link name="${IndexFingerPitch2LinkName}"
@@ -24,5 +23,4 @@
                     origin_rpy="0 0 0"
                     visual_mesh="${mesh_root}/fingers/indexj2_${prefix}.dae"
-                    material="Gold"
                     collision_mesh="${mesh_root}/fingers/indexj2_${prefix}.dae"/>
     <xacro:standard_link name="${IndexFingerPitch3LinkName}"
@@ -33,5 +31,4 @@
                     origin_rpy="0 0 0"
                     visual_mesh="${mesh_root}/fingers/indexj3_${prefix}.dae"
-                    material="Gold"
                     collision_mesh="${mesh_root}/fingers/indexj3_${prefix}.dae"/>
     <xacro:revolute_joint jointName="${IndexFingerPitch1JointName}"

File: model/robots/common/xacro/leg/leg.xacro (robot description, xacro)
@@ -18,5 +18,4 @@
                     iyy="${HipYawLinkInertia_IYY}" iyz="${HipYawLinkInertia_IYZ}" izz="${HipYawLinkInertia_IZZ}"
                     visual_mesh="${mesh_root}/legs/lj1_${prefix}.dae"
-                    material="Gold"
                     collision_mesh="${mesh_root}/legs/lj1_${prefix}.dae"/>
     <xacro:standard_link name="${HipRollLinkName}"
@@ -27,5 +26,4 @@
                     origin_rpy="0 0 0"
                     visual_mesh="${mesh_root}/legs/lj2_${prefix}.dae"
-                    material="White"
                     collision_mesh="${mesh_root}/legs/lj2_${prefix}.dae"/>
     <xacro:standard_link name="${HipPitchLinkName}"
@@ -36,5 +34,4 @@
                     origin_rpy="0 0 0"
                     visual_mesh="${mesh_root}/legs/lj3_${prefix}.dae"
-                    material="White"
                     collision_mesh="${mesh_root}/legs/lj3_${prefix}.dae"/>
     <xacro:standard_link name="${KneePitchLinkName}"
@@ -45,5 +42,4 @@
                     origin_rpy="0 0 0"
                     visual_mesh="${mesh_root}/legs/lj4_${prefix}.dae"
-                    material="White"
                     collision_mesh="${mesh_root}/legs/lj4_${prefix}.dae"/>
     <xacro:standard_link name="${AnklePitchLinkName}"
@@ -54,5 +50,4 @@
                     origin_rpy="0 0 0"
                     visual_mesh="${mesh_root}/legs/lj5.dae"
-                    material="White"
                     collision_mesh="${mesh_root}/legs/lj5.dae"/>
     <xacro:link_box_collision_mesh_visual name="${AnkleRollLinkName}"
@@ -63,5 +58,4 @@
                     inertial_rpy="0 0 0"
                     visual_mesh="${mesh_root}/legs/foot.dae"
-                    material="White"
                     width="0.27"
                     height="0.16"

File: model/robots/common/xacro/middle_finger/middle_finger.xacro (robot description, xacro)
@@ -15,5 +15,4 @@
                     origin_rpy="0 0 0"
                     visual_mesh="${mesh_root}/fingers/middlej1_${prefix}.dae"
-                    material="Gold"
                     collision_mesh="${mesh_root}/fingers/middlej1_${prefix}.dae"/>
     <xacro:standard_link name="${MiddleFingerPitch2LinkName}"
@@ -24,5 +23,4 @@
                     origin_rpy="0 0 0"
                     visual_mesh="${mesh_root}/fingers/middlej2_${prefix}.dae"
-                    material="Gold"
                     collision_mesh="${mesh_root}/fingers/middlej2_${prefix}.dae"/>
     <xacro:standard_link name="${MiddleFingerPitch3LinkName}"
@@ -33,5 +31,4 @@
                     origin_rpy="0 0 0"
                     visual_mesh="${mesh_root}/fingers/middlej3_${prefix}.dae"
-                    material="Gold"
                     collision_mesh="${mesh_root}/fingers/middlej3_${prefix}.dae"/>
     <xacro:revolute_joint jointName="${MiddleFingerPitch1JointName}"

File: model/robots/common/xacro/pelvis/pelvis.xacro (robot description, xacro)
@@ -8,5 +8,5 @@
                         iyy="0.097963425" iyz="0.002159545" izz="0.083854638"
                         origin_rpy="0 0 0"
-                        visual_mesh="${mesh_root}/pelvis/pelvis.dae" material="White"
+                        visual_mesh="${mesh_root}/pelvis/pelvis.dae"
                         collision_mesh="${mesh_root}/pelvis/pelvis.dae"/>
     </xacro:macro>

File: model/robots/common/xacro/pinky_finger/pinky_finger.xacro (robot description, xacro)
@@ -15,5 +15,4 @@
                     origin_rpy="0 0 0"
                     visual_mesh="${mesh_root}/fingers/pinkyj1_${prefix}.dae"
-                    material="Gold"
                     collision_mesh="${mesh_root}/fingers/pinkyj1_${prefix}.dae"/>
     <xacro:standard_link name="${PinkyPitch2LinkName}"
@@ -24,5 +23,4 @@
                     origin_rpy="0 0 0"
                     visual_mesh="${mesh_root}/fingers/pinkyj2_${prefix}.dae"
-                    material="Gold"
                     collision_mesh="${mesh_root}/fingers/pinkyj2_${prefix}.dae"/>
     <xacro:standard_link name="${PinkyPitch3LinkName}"
@@ -33,5 +31,4 @@
                     origin_rpy="0 0 0"
                     visual_mesh="${mesh_root}/fingers/pinkyj3_${prefix}.dae"
-                    material="Gold"
                     collision_mesh="${mesh_root}/fingers/pinkyj3_${prefix}.dae"/>
     <xacro:revolute_joint jointName="${PinkyPitch1JointName}"

File: model/robots/common/xacro/thumb/thumb.xacro (robot description, xacro)
@@ -15,5 +15,4 @@
                     origin_rpy="0 0 0"
                     visual_mesh="${mesh_root}/fingers/thumbj1_${prefix}.dae"
-                    material="Gold"
                     collision_mesh="${mesh_root}/fingers/thumbj1_${prefix}.dae"/>
     <xacro:standard_link name="${ThumbPitch1LinkName}"
@@ -24,5 +23,4 @@
                     origin_rpy="0 0 0"
                     visual_mesh="${mesh_root}/fingers/thumbj2_${prefix}.dae"
-                    material="Gold"
                     collision_mesh="${mesh_root}/fingers/thumbj2_${prefix}.dae"/>
     <xacro:standard_link name="${ThumbPitch2LinkName}"
@@ -33,5 +31,4 @@
                     origin_rpy="0 0 0"
                     visual_mesh="${mesh_root}/fingers/thumbj3_${prefix}.dae"
-                    material="Gold"
                     collision_mesh="${mesh_root}/fingers/thumbj3_${prefix}.dae"/>
     <xacro:standard_link name="${ThumbPitch3LinkName}"
@@ -42,5 +39,4 @@
                     origin_rpy="0 0 0"
                     visual_mesh="${mesh_root}/fingers/thumbj4_${prefix}.dae"
-                    material="Gold"
                     collision_mesh="${mesh_root}/fingers/thumbj4_${prefix}.dae"/>
     <xacro:revolute_joint jointName="${ThumbRollJointName}"

File: model/robots/common/xacro/waist/waist.xacro (robot description, xacro)
@@ -49,5 +49,4 @@
                     iyy="${TorsoYawLinkInertia_IYY}" iyz="${TorsoYawLinkInertia_IYZ}" izz="${TorsoYawLinkInertia_IZZ}"
                     visual_mesh="${mesh_root}/torso/torsoyaw.dae"
-                    material="White"
                     collision_mesh="${mesh_root}/torso/torsoyaw.dae" />
     <xacro:standard_link name="${TorsoPitchLinkName}"
@@ -58,5 +57,4 @@
                     iyy="${TorsoPitchLinkInertia_IYY}" iyz="${TorsoPitchLinkInertia_IYZ}" izz="${TorsoPitchLinkInertia_IZZ}"
                     visual_mesh="${mesh_root}/torso/torsopitch.dae"
-                    material="White"
                     collision_mesh="${mesh_root}/torso/torsopitch.dae" />
     <xacro:standard_link name="${TorsoRollLinkName}"
@@ -67,5 +65,4 @@
                     origin_xyz="${TorsoRollLinkComPosition}"
                     visual_mesh="${mesh_root}/torso/torso.dae"
-                    material="White"
                     collision_mesh="${mesh_root}/torso/torso.dae" />
     <xacro:make_waist_common waist_root_link="${waist_root_link}"/>

Commit message: Added macros for urdfs with no hands.

File: model/robots/common/xacro/arm/arm.xacro (robot description, xacro)
@@ -156,4 +156,7 @@
     <xacro:make_lower_arm prefix="${prefix}" reflect="${reflect}" lower_arm_root_link="${ElbowPitchLinkName}" />
   </xacro:macro>
+  <xacro:macro name="make_arm_no_hands" params="prefix reflect arm_root_link">
+    <xacro:make_upper_arm prefix="${prefix}" reflect="${reflect}" upper_arm_root_link="${arm_root_link}" />
+  </xacro:macro>
   <xacro:macro name="arm_transmissions_hw" params="prefix">
     <xacro:simple_transmission jointName="${ShoulderPitchJointName}" actuatorName="${ShoulderPitchActuatorName}" nodeName="${ShoulderPitchNode}" actuatorApi="${ShoulderPitchApi}"/>
@@ -163,4 +166,10 @@
     <xacro:simple_transmission jointName="${ForearmYawActuatorName}" actuatorName="${ForearmYawActuatorName}" nodeName="${ForearmYawNode}" actuatorApi="${ForearmYawApi}"/>
     <xacro:pushrod_transmission transmissionName="${prefix}WristTransmission" transmissionType="WristPushrodTransmission" joint1Name="${WristPitchJointName}" joint2Name="${WristRollJointName}" actuator1Name="${WristTopActuatorName}" actuator2Name="${WristBottomActuatorName}" actuator1Node="${WristTopActuatorNode}" actuator2Node="${WristBottomActuatorNode}" actuator1Api="${WristTopActuatorApi}" actuator2Api="${WristBottomActuatorApi}"/>
+  </xacro:macro>
+  <xacro:macro name="arm_transmissions_no_hands" params="prefix">
+    <xacro:simple_transmission jointName="${ShoulderPitchJointName}" actuatorName="${ShoulderPitchActuatorName}" nodeName="${ShoulderPitchNode}" actuatorApi="${ShoulderPitchApi}"/>
+    <xacro:simple_transmission jointName="${ShoulderRollJointName}" actuatorName="${ShoulderRollActuatorName}" nodeName="${ShoulderRollNode}" actuatorApi="${ShoulderRollApi}"/>
+    <xacro:simple_transmission jointName="${ShoulderYawJointName}" actuatorName="${ShoulderYawActuatorName}" nodeName="${ShoulderYawNode}" actuatorApi="${ShoulderYawApi}"/>
+    <xacro:simple_transmission jointName="${ElbowPitchJointName}" actuatorName="${ElbowPitchActuatorName}" nodeName="${ElbowPitchNode}" actuatorApi="${ElbowPitchApi}"/>
   </xacro:macro>
   <xacro:macro name="arm_transmissions_sim" params="prefix">

Commit message: Added new transmission role stuff according to Franks changes to val_control.

File: model/robots/common/xacro/arm/arm.xacro (robot description, xacro)
@@ -165,5 +165,5 @@
     <xacro:simple_transmission jointName="${ElbowPitchJointName}" actuatorName="${ElbowPitchActuatorName}" nodeName="${ElbowPitchNode}" actuatorApi="${ElbowPitchApi}"/>
     <xacro:simple_transmission jointName="${ForearmYawActuatorName}" actuatorName="${ForearmYawActuatorName}" nodeName="${ForearmYawNode}" actuatorApi="${ForearmYawApi}"/>
-    <xacro:pushrod_transmission transmissionName="${prefix}WristTransmission" transmissionType="WristPushrodTransmission" joint1Name="${WristPitchJointName}" joint2Name="${WristRollJointName}" actuator1Name="${WristTopActuatorName}" actuator2Name="${WristBottomActuatorName}" actuator1Node="${WristTopActuatorNode}" actuator2Node="${WristBottomActuatorNode}" actuator1Api="${WristTopActuatorApi}" actuator2Api="${WristBottomActuatorApi}"/>
+    <xacro:pushrod_transmission transmissionName="${prefix}WristTransmission" transmissionType="WristPushrodTransmission" joint1Name="${WristPitchJointName}" joint2Name="${WristRollJointName}" joint1Role="roll" joint2Role="pitch" actuator1Name="${WristTopActuatorName}" actuator2Name="${WristBottomActuatorName}" actuator1Node="${WristTopActuatorNode}" actuator2Node="${WristBottomActuatorNode}" actuator1Api="${WristTopActuatorApi}" actuator2Api="${WristBottomActuatorApi}" actuator1Role="top" actuator2Role="bottom"/>
   </xacro:macro>
   <xacro:macro name="arm_transmissions_no_hands" params="prefix">

File: model/robots/common/xacro/generic_models.xacro (robot description, xacro)
@@ -215,18 +215,18 @@
     </transmission>
   </xacro:macro>
-  <xacro:macro name="pushrod_transmission" params="transmissionName transmissionType joint1Name joint2Name actuator1Name actuator2Name actuator1Node actuator2Node actuator1Api actuator2Api">
+  <xacro:macro name="pushrod_transmission" params="transmissionName transmissionType joint1Name joint2Name joint1Role joint2Role actuator1Name actuator2Name actuator1Node actuator2Node actuator1Api actuator2Api actuator1Role actuator2Role">
     <transmission name="${transmissionName}">
       <type>robot_transmission_interface/${transmissionType}</type>
       <joint name="${joint1Name}">
-        <role>joint1</role>
+        <role>${joint1Role}</role>
         <hardwareInterface>EffortJointInterface</hardwareInterface>
       </joint>
       <joint name="${joint2Name}">
-        <role>joint2</role>
+        <role>${joint2Role}</role>
         <hardwareInterface>EffortJointInterface</hardwareInterface>
       </joint>
        <actuator name="${actuator1Name}">
         <node name="${actuator1Node}"/>
-        <role>actuator1</role>
+        <role>${actuator1Role}</role>
         <mechanicalReduction>1</mechanicalReduction>
         <api name="${actuator1Api}"/>
@@ -234,5 +234,5 @@
       <actuator name="${actuator2Name}">
         <node name="${actuator2Node}"/>
-        <role>actuator2</role>
+        <role>${actuator2Role}</role>
         <mechanicalReduction>1</mechanicalReduction>
         <api name="${actuator2Api}"/>

File: model/robots/common/xacro/leg/leg.xacro (robot description, xacro)
@@ -156,5 +156,5 @@
     <xacro:simple_transmission jointName="${HipPitchJointName}" actuatorName="${HipPitchActuatorName}" nodeName="${HipPitchNode}" actuatorApi="${HipPitchApi}"/>
     <xacro:simple_transmission jointName="${KneePitchJointName}" actuatorName="${KneePitchActuatorName}" nodeName="${KneePitchNode}" actuatorApi="${KneePitchApi}"/>
-    <xacro:pushrod_transmission transmissionName="${prefix}AnkleTransmission" transmissionType="AnklePushrodTransmission" joint1Name="${AnklePitchJointName}" joint2Name="${AnkleRollJointName}" actuator1Name="${AnkleRightActuatorName}" actuator2Name="${AnkleLeftActuatorName}" actuator1Node="${AnkleRightActuatorNode}" actuator2Node="${AnkleLeftActuatorNode}" actuator1Api="${AnkleRightActuatorApi}" actuator2Api="${AnkleLeftActuatorApi}"/>
+    <xacro:pushrod_transmission transmissionName="${prefix}AnkleTransmission" transmissionType="AnklePushrodTransmission" joint1Name="${AnklePitchJointName}" joint2Name="${AnkleRollJointName}" joint1Role="pitch" joint2Role="roll" actuator1Name="${AnkleRightActuatorName}" actuator2Name="${AnkleLeftActuatorName}" actuator1Node="${AnkleRightActuatorNode}" actuator2Node="${AnkleLeftActuatorNode}" actuator1Api="${AnkleRightActuatorApi}" actuator2Api="${AnkleLeftActuatorApi}" actuator1Role="right" actuator2Role="left"/>
   </xacro:macro>
   <xacro:macro name="leg_transmissions_sim" params="prefix">

File: model/robots/common/xacro/waist/waist.xacro (robot description, xacro)
@@ -97,5 +97,5 @@
    <xacro:macro name="waist_transmissions_hw">
     <xacro:simple_transmission jointName="${TorsoYawJointName}" actuatorName="${TorsoYawActuatorName}" nodeName="${TrunkYawNode}" actuatorApi="${TrunkYawApi}"/>
-    <xacro:pushrod_transmission transmissionName="WaistTransmission" transmissionType="TorsoPushrodTransmission" joint1Name="${TorsoPitchJointName}" joint2Name="${TorsoRollJointName}" actuator1Name="${WaistRightActuatorName}" actuator2Name="${WaistLeftActuatorName}" actuator1Node="${WaistRightActuatorNode}" actuator2Node="${WaistLeftActuatorNode}" actuator1Api="${WaistRightActuatorApi}" actuator2Api="${WaistLeftActuatorApi}"/>
+    <xacro:pushrod_transmission transmissionName="waistTransmission" transmissionType="TorsoPushrodTransmission" joint1Name="${TorsoPitchJointName}" joint2Name="${TorsoRollJointName}" joint1Role="roll" joint2Role="pitch" actuator1Name="${WaistRightActuatorName}" actuator2Name="${WaistLeftActuatorName}" actuator1Node="${WaistRightActuatorNode}" actuator2Node="${WaistLeftActuatorNode}" actuator1Api="${WaistRightActuatorApi}" actuator2Api="${WaistLeftActuatorApi}" actuator1Role="left" actuator2Role="right"/>
    </xacro:macro>
    <xacro:macro name="waist_transmissions_sim">
