Commit message: Added new pushrod transmissions for the wrists since they are pushrod joints with position controlled actuators.

File: model/robots/common/xacro/arm/arm.xacro (robot description, xacro)
@@ -166,5 +166,5 @@
     <xacro:simple_transmission jointName="${ElbowPitchJointName}" actuatorName="${ElbowPitchActuatorName}" nodeName="${ElbowPitchNode}" actuatorApi="${ElbowPitchApi}"/>
     <xacro:simple_transmission jointName="${ForearmYawActuatorName}" actuatorName="${ForearmYawActuatorName}" nodeName="${ForearmYawNode}" actuatorApi="${ForearmYawApi}"/>
-    <xacro:pushrod_transmission transmissionName="${prefix}WristTransmission" transmissionType="WristPushrodTransmission" joint1Name="${WristPitchJointName}" joint2Name="${WristRollJointName}" joint1Role="roll" joint2Role="pitch" actuator1Name="${WristTopActuatorName}" actuator2Name="${WristBottomActuatorName}" actuator1Node="${WristTopActuatorNode}" actuator2Node="${WristBottomActuatorNode}" actuator1Api="${WristTopActuatorApi}" actuator2Api="${WristBottomActuatorApi}" actuator1Role="top" actuator2Role="bottom"/>
+    <xacro:pushrod_transmission_position_control transmissionName="${prefix}WristTransmission" transmissionType="WristPushrodTransmission" joint1Name="${WristPitchJointName}" joint2Name="${WristRollJointName}" joint1Role="roll" joint2Role="pitch" actuator1Name="${WristTopActuatorName}" actuator2Name="${WristBottomActuatorName}" actuator1Node="${WristTopActuatorNode}" actuator2Node="${WristBottomActuatorNode}" actuator1Api="${WristTopActuatorApi}" actuator2Api="${WristBottomActuatorApi}" actuator1Role="top" actuator2Role="bottom"/>
   </xacro:macro>
   <xacro:macro name="arm_transmissions_no_hands" params="prefix">
@@ -180,6 +180,6 @@
     <xacro:simple_transmission jointName="${ElbowPitchJointName}" actuatorName="${ElbowPitchActuatorName}" nodeName="${ElbowPitchNode}" actuatorApi="${SimApi}"/>
     <xacro:simple_transmission jointName="${ForearmYawActuatorName}" actuatorName="${ForearmYawActuatorName}" nodeName="${ForearmYawNode}" actuatorApi="${SimApi}"/>
-    <xacro:simple_transmission jointName="${WristRollJointName}" actuatorName="${WristRollActuatorSimName}" nodeName="${WristRollActuatorSimNode}" actuatorApi="${SimApi}"/>
-    <xacro:simple_transmission jointName="${WristPitchJointName}" actuatorName="${WristPitchActuatorSimName}" nodeName="${WristPitchActuatorSimNode}" actuatorApi="${SimApi}"/>
+    <xacro:simple_position_transmission jointName="${WristRollJointName}" actuatorName="${WristRollActuatorSimName}" nodeName="${WristRollActuatorSimNode}" actuatorApi="${SimApi}"/>
+    <xacro:simple_position_transmission jointName="${WristPitchJointName}" actuatorName="${WristPitchActuatorSimName}" nodeName="${WristPitchActuatorSimNode}" actuatorApi="${SimApi}"/>
   </xacro:macro>
 </robot>

File: model/robots/common/xacro/generic_models.xacro (robot description, xacro)
@@ -253,3 +253,30 @@
     </transmission>
   </xacro:macro>
+  <xacro:macro name="pushrod_transmission_position_control" params="transmissionName transmissionType joint1Name joint2Name joint1Role joint2Role actuator1Name actuator2Name actuator1Node actuator2Node actuator1Api actuator2Api actuator1Role actuator2Role">
+    <transmission name="${transmissionName}">
+      <type>robot_transmission_interface/${transmissionType}</type>
+      <joint name="${joint1Name}">
+        <role>${joint1Role}</role>
+        <hardwareInterface>PositionJointInterface</hardwareInterface>
+      </joint>
+      <joint name="${joint2Name}">
+        <role>${joint2Role}</role>
+        <hardwareInterface>PositionJointInterface</hardwareInterface>
+      </joint>
+       <actuator name="${actuator1Name}">
+        <node name="${actuator1Node}"/>
+        <role>${actuator1Role}</role>
+        <mechanicalReduction>1</mechanicalReduction>
+        <api name="${actuator1Api}"/>
+      </actuator>
+      <actuator name="${actuator2Name}">
+        <node name="${actuator2Node}"/>
+        <role>${actuator2Role}</role>
+        <mechanicalReduction>1</mechanicalReduction>
+        <api name="${actuator2Api}"/>
+      </actuator>
+    </transmission>
+  </xacro:macro>
+  <xacro:macro name="finger_transmission" params="transmissionName transmissionType joint1Name joint2Name joint3Name joint1Role joint2Role joint3Role actuator1Name actuator2Name actuator3Name actuator1Api actuator1Role actuator2Role actuator3Role">
+  </xacro:macro>
 </robot>

File: model/robots/common/xacro/thumb/thumb.xacro (robot description, xacro)
@@ -84,3 +84,6 @@
     </xacro:revolute_joint>
   </xacro:macro>
+  <xacro:macro name="thumb_transmissions" params="prefix">
+    <xacro:simple_transmission jointName="${ThumbRollJointName}" actuatorName="${ThumbRollActuatorName}" nodeName="${ThumbRollNodeName}" actuatorApi="${SimApi}"/>
+  </xacro:macro>
 </robot>

Commit message: Another attempt at getting the athena urdf entry's correct.

File: model/robots/common/xacro/arm/arm.xacro (robot description, xacro)
@@ -166,5 +166,6 @@
     <xacro:simple_transmission jointName="${ElbowPitchJointName}" actuatorName="${ElbowPitchActuatorName}" nodeName="${ElbowPitchNode}" actuatorApi="${ElbowPitchApi}"/>
     <xacro:simple_transmission jointName="${ForearmYawActuatorName}" actuatorName="${ForearmYawActuatorName}" nodeName="${ForearmYawNode}" actuatorApi="${ForearmYawApi}"/>
-    <xacro:pushrod_transmission_position_control transmissionName="${prefix}WristTransmission" transmissionType="WristPushrodTransmission" joint1Name="${WristPitchJointName}" joint2Name="${WristRollJointName}" joint1Role="roll" joint2Role="pitch" actuator1Name="${WristTopActuatorName}" actuator2Name="${WristBottomActuatorName}" actuator1Node="${WristTopActuatorNode}" actuator2Node="${WristBottomActuatorNode}" actuator1Api="${WristTopActuatorApi}" actuator2Api="${WristBottomActuatorApi}" actuator1Role="top" actuator2Role="bottom"/>
+    <xacro:athena1_transmission prefix="${prefix}"/>
+    <xacro:athena2_transmission prefix="${prefix}"/>
   </xacro:macro>
   <xacro:macro name="arm_transmissions_no_hands" params="prefix">

File: model/robots/common/xacro/generic_models.xacro (robot description, xacro)
@@ -277,17 +277,38 @@
   <xacro:macro name="athena1_transmission" params="prefix">
     <type>robot_transmission_interface/athena1_transmission</type>
-    <joint name="wristPitch">
+    <joint name="${prefix}WristPitch">
       <role>wristPitch</role>
     </joint>
-    <joint name="wristRoll">
+    <joint name="${prefix}WristRoll">
       <role>wristRoll</role>
     </joint>
-    <actuator name="wristTopActuator">
-      <role>="wristTopActuator"</role>
+    <joint name="${prefix}ThumbRoll">
+      <role>thumbRoll</role>
+    </joint>
+    <joint name="${prefix}ThumbPitch1">
+      <role>thumbPitch1</role>
+    </joint>
+    <actuator name="${prefix}Athena1Actuator">
+      <role>athena1Actuator</role>
       <mechanicalReduction>1</mechanicalReduction>
       <hardwareInterface>PositionJointInterface</hardwareInterface>
     </actuator>
-    <actuator name="wristBottomActuator">
-      <role>="wristBottomActuator"</role>
+  </xacro:macro>
+  <xacro:macro name="athena2_transmission" params="prefix">
+    <type>robot_transmission_interface/athena2_transmission</type>
+    <joint name="${prefix}ThumbPitch2">
+      <role>thumbPitch2</role>
+    </joint>
+    <joint name="${prefix}IndexFingerPitch1">
+      <role>indexFingerPitch1</role>
+    </joint>
+    <joint name="${prefix}MiddleFingerPitch1">
+      <role>middleFingerPitch1</role>
+    </joint>
+    <joint name="${prefix}PinkyPitch1">
+      <role>pinkyPitch1</role>
+    </joint>
+    <actuator name="${prefix}Athena2Actuator">
+      <role>athena2Actuator</role>
       <mechanicalReduction>1</mechanicalReduction>
       <hardwareInterface>PositionJointInterface</hardwareInterface>

File: model/robots/common/xacro/valkyrie_base_hw.xacro (robot description, xacro)
@@ -26,11 +26,3 @@
     <xacro:arm_transmissions_hw prefix="right"/>
     <xacro:neck_transmissions_hw />
-    <xacro:thumb_transmissions prefix="left"/>
-    <xacro:thumb_transmissions prefix="right"/>
-    <xacro:index_finger_transmissions prefix="left"/>
-    <xacro:index_finger_transmissions prefix="right"/>
-    <xacro:middle_finger_transmissions prefix="left"/>
-    <xacro:middle_finger_transmissions prefix="right"/>
-    <xacro:pinky_finger_transmissions prefix="left"/>
-    <xacro:pinky_finger_transmissions prefix="right"/>
 </robot>

Commit message: added reflect arg to forearm transmissions

File: model/robots/common/xacro/arm/arm.xacro (robot description, xacro)
@@ -159,10 +159,10 @@
     <xacro:make_upper_arm prefix="${prefix}" reflect="${reflect}" upper_arm_root_link="${arm_root_link}" />
   </xacro:macro>
-  <xacro:macro name="arm_transmissions_hw" params="prefix">
+  <xacro:macro name="arm_transmissions_hw" params="prefix reflect">
     <xacro:simple_transmission jointName="${ShoulderPitchJointName}" actuatorName="${ShoulderPitchActuatorName}" nodeName="${ShoulderPitchNode}" actuatorApi="${ShoulderPitchApi}"/>
     <xacro:simple_transmission jointName="${ShoulderRollJointName}" actuatorName="${ShoulderRollActuatorName}" nodeName="${ShoulderRollNode}" actuatorApi="${ShoulderRollApi}"/>
     <xacro:simple_transmission jointName="${ShoulderYawJointName}" actuatorName="${ShoulderYawActuatorName}" nodeName="${ShoulderYawNode}" actuatorApi="${ShoulderYawApi}"/>
     <xacro:simple_transmission jointName="${ElbowPitchJointName}" actuatorName="${ElbowPitchActuatorName}" nodeName="${ElbowPitchNode}" actuatorApi="${ElbowPitchApi}"/>
-    <xacro:simple_position_transmission jointName="${ForearmYawActuatorName}" actuatorName="${ForearmYawActuatorName}" nodeName="${ForearmYawNode}" actuatorApi="${ForearmYawApi}"/>
+    <xacro:simple_forearm_position_transmission jointName="${ForearmYawActuatorName}" actuatorName="${ForearmYawActuatorName}" nodeName="${ForearmYawNode}" actuatorApi="${ForearmYawApi}" reflect="${reflect}"/>
     <xacro:athena1_transmission prefix="${prefix}" transmissionName="${prefix}ArmAthena1Transmission" actuatorApi="${Athena1Api}" nodeName="${Athena1Node}"/>
     <xacro:athena2_transmission prefix="${prefix}" transmissionName="${prefix}ArmAthena2Transmission" actuatorApi="${Athena2Api}" nodeName="${Athena2Node}"/>

File: model/robots/common/xacro/generic_models.xacro (robot description, xacro)
@@ -225,4 +225,17 @@
     </transmission>
   </xacro:macro>
+  <xacro:macro name="simple_forearm_position_transmission" params="jointName actuatorName nodeName actuatorApi reflect">
+    <transmission name="${jointName}Transmission">
+      <type>transmission_interface/SimpleTransmission</type>
+      <joint name="${jointName}">
+        <hardwareInterface>PositionJointInterface</hardwareInterface>
+      </joint>
+      <actuator name="${actuatorName}">
+        <node name="${nodeName}"/>
+        <mechanicalReduction>${reflect}</mechanicalReduction>
+        <api name="${actuatorApi}" />
+      </actuator>
+    </transmission>
+  </xacro:macro>
   <xacro:macro name="pushrod_transmission" params="transmissionName transmissionType joint1Name joint2Name joint1Role joint2Role actuator1Name actuator2Name actuator1Node actuator2Node actuator1Api actuator2Api actuator1Role actuator2Role">
     <transmission name="${transmissionName}">

File: model/robots/common/xacro/index_finger/index_finger.xacro (robot description, xacro)
@@ -69,8 +69,8 @@
     </xacro:revolute_joint>
   </xacro:macro>
-  <xacro:macro name="index_finger_transmissions_hw" params="prefix">
-    <xacro:simple_position_transmission jointName="${IndexFingerPitch1JointName}" actuatorName="${prefix}IndexPitch1Actuator" nodeName="${IndexFingerPitch1Node}" actuatorApi="${IndexFingerApi}"/>
-    <xacro:simple_position_transmission jointName="${IndexFingerPitch2JointName}" actuatorName="${prefix}IndexPitch2Actuator" nodeName="${IndexFingerPitch2Node}" actuatorApi="${IndexFingerApi}"/>
-    <xacro:simple_position_transmission jointName="${IndexFingerPitch3JointName}" actuatorName="${prefix}IndexPitch3Actuator" nodeName="${IndexFingerPitch3Node}" actuatorApi="${IndexFingerApi}"/>
+  <xacro:macro name="index_finger_transmissions_hw" params="prefix reflect">
+    <xacro:simple_forearm_position_transmission jointName="${IndexFingerPitch1JointName}" actuatorName="${prefix}IndexPitch1Actuator" nodeName="${IndexFingerPitch1Node}" actuatorApi="${IndexFingerApi}" reflect="${reflect}"/>
+    <xacro:simple_forearm_position_transmission jointName="${IndexFingerPitch2JointName}" actuatorName="${prefix}IndexPitch2Actuator" nodeName="${IndexFingerPitch2Node}" actuatorApi="${IndexFingerApi}" reflect="${reflect}"/>
+    <xacro:simple_forearm_position_transmission jointName="${IndexFingerPitch3JointName}" actuatorName="${prefix}IndexPitch3Actuator" nodeName="${IndexFingerPitch3Node}" actuatorApi="${IndexFingerApi}" reflect="${reflect}"/>
   </xacro:macro>
 </robot>

File: model/robots/common/xacro/middle_finger/middle_finger.xacro (robot description, xacro)
@@ -69,8 +69,8 @@
     </xacro:revolute_joint>
   </xacro:macro>
-  <xacro:macro name="middle_finger_transmissions_hw" params="prefix">
-    <xacro:simple_position_transmission jointName="${MiddleFingerPitch1JointName}" actuatorName="${prefix}MiddlePitch1Actuator" nodeName="${MiddleFingerPitch1Node}" actuatorApi="${MiddleFingerApi}"/>
-    <xacro:simple_position_transmission jointName="${MiddleFingerPitch2JointName}" actuatorName="${prefix}MiddlePitch2Actuator" nodeName="${MiddleFingerPitch2Node}" actuatorApi="${MiddleFingerApi}"/>
-    <xacro:simple_position_transmission jointName="${MiddleFingerPitch3JointName}" actuatorName="${prefix}MiddlePitch3Actuator" nodeName="${MiddleFingerPitch3Node}" actuatorApi="${MiddleFingerApi}"/>
+  <xacro:macro name="middle_finger_transmissions_hw" params="prefix reflect">
+    <xacro:simple_forearm_position_transmission jointName="${MiddleFingerPitch1JointName}" actuatorName="${prefix}MiddlePitch1Actuator" nodeName="${MiddleFingerPitch1Node}" actuatorApi="${MiddleFingerApi}" reflect="${reflect}"/>
+    <xacro:simple_forearm_position_transmission jointName="${MiddleFingerPitch2JointName}" actuatorName="${prefix}MiddlePitch2Actuator" nodeName="${MiddleFingerPitch2Node}" actuatorApi="${MiddleFingerApi}" reflect="${reflect}"/>
+    <xacro:simple_forearm_position_transmission jointName="${MiddleFingerPitch3JointName}" actuatorName="${prefix}MiddlePitch3Actuator" nodeName="${MiddleFingerPitch3Node}" actuatorApi="${MiddleFingerApi}" reflect="${reflect}"/>
   </xacro:macro>
 </robot>

File: model/robots/common/xacro/pinky_finger/pinky_finger.xacro (robot description, xacro)
@@ -69,8 +69,8 @@
     </xacro:revolute_joint>
   </xacro:macro>
-  <xacro:macro name="pinky_finger_transmissions_hw" params="prefix">
-    <xacro:simple_position_transmission jointName="${PinkyPitch1JointName}" actuatorName="${prefix}PinkyPitch1Actuator" nodeName="${PinkyPitch1Node}" actuatorApi="${PinkyApi}"/>
-    <xacro:simple_position_transmission jointName="${PinkyPitch2JointName}" actuatorName="${prefix}PinkyPitch2Actuator" nodeName="${PinkyPitch2Node}" actuatorApi="${PinkyApi}"/>
-    <xacro:simple_position_transmission jointName="${PinkyPitch3JointName}" actuatorName="${prefix}PinkyPitch3Actuator" nodeName="${PinkyPitch3Node}" actuatorApi="${PinkyApi}"/>
+  <xacro:macro name="pinky_finger_transmissions_hw" params="prefix reflect">
+    <xacro:simple_forearm_position_transmission jointName="${PinkyPitch1JointName}" actuatorName="${prefix}PinkyPitch1Actuator" nodeName="${PinkyPitch1Node}" actuatorApi="${PinkyApi}" reflect="${reflect}"/>
+    <xacro:simple_forearm_position_transmission jointName="${PinkyPitch2JointName}" actuatorName="${prefix}PinkyPitch2Actuator" nodeName="${PinkyPitch2Node}" actuatorApi="${PinkyApi}" reflect="${reflect}"/>
+    <xacro:simple_forearm_position_transmission jointName="${PinkyPitch3JointName}" actuatorName="${prefix}PinkyPitch3Actuator" nodeName="${PinkyPitch3Node}" actuatorApi="${PinkyApi}" reflect="${reflect}"/>
   </xacro:macro>
 </robot>

File: model/robots/common/xacro/thumb/thumb.xacro (robot description, xacro)
@@ -84,9 +84,9 @@
     </xacro:revolute_joint>
   </xacro:macro>
-  <xacro:macro name="thumb_transmissions_hw" params="prefix">
+  <xacro:macro name="thumb_transmissions_hw" params="prefix reflect">
     <xacro:simple_position_transmission jointName="${ThumbRollJointName}" actuatorName="${prefix}ThumbRollActuator" nodeName="${ThumbRollNode}" actuatorApi="${ThumbFingerApi}"/>
-    <xacro:simple_position_transmission jointName="${ThumbPitch1JointName}" actuatorName="${prefix}ThumbPitch1Actuator" nodeName="${ThumbPitch1Node}" actuatorApi="${ThumbFingerApi}"/>
-    <xacro:simple_position_transmission jointName="${ThumbPitch2JointName}" actuatorName="${prefix}ThumbPitch2Actuator" nodeName="${ThumbPitch2Node}" actuatorApi="${ThumbFingerApi}"/>
-    <xacro:simple_position_transmission jointName="${ThumbPitch3JointName}" actuatorName="${prefix}ThumbPitch3Actuator" nodeName="${ThumbPitch3Node}" actuatorApi="${ThumbFingerApi}"/>
+    <xacro:simple_forearm_position_transmission jointName="${ThumbPitch1JointName}" actuatorName="${prefix}ThumbPitch1Actuator" nodeName="${ThumbPitch1Node}" actuatorApi="${ThumbFingerApi}" reflect="${reflect}"/>
+    <xacro:simple_forearm_position_transmission jointName="${ThumbPitch2JointName}" actuatorName="${prefix}ThumbPitch2Actuator" nodeName="${ThumbPitch2Node}" actuatorApi="${ThumbFingerApi}" reflect="${reflect}"/>
+    <xacro:simple_forearm_position_transmission jointName="${ThumbPitch3JointName}" actuatorName="${prefix}ThumbPitch3Actuator" nodeName="${ThumbPitch3Node}" actuatorApi="${ThumbFingerApi}" reflect="${reflect}"/>
   </xacro:macro>
 </robot>

File: model/robots/common/xacro/valkyrie_base_hw.xacro (robot description, xacro)
@@ -23,14 +23,14 @@
     <xacro:leg_transmissions_hw prefix="left"/>
     <xacro:leg_transmissions_hw prefix="right"/>
-    <xacro:arm_transmissions_hw prefix="left"/>
-    <xacro:arm_transmissions_hw prefix="right"/>
+    <xacro:arm_transmissions_hw prefix="left" reflect="1"/>
+    <xacro:arm_transmissions_hw prefix="right" reflect="-1"/>
     <xacro:neck_transmissions_hw />
-    <xacro:index_finger_transmissions_hw prefix="left" />
-    <xacro:middle_finger_transmissions_hw prefix="left" />
-    <xacro:pinky_finger_transmissions_hw prefix="left" />
-    <xacro:thumb_transmissions_hw prefix="left" />
-    <xacro:index_finger_transmissions_hw prefix="right" />
-    <xacro:middle_finger_transmissions_hw prefix="right" />
-    <xacro:pinky_finger_transmissions_hw prefix="right" />
-    <xacro:thumb_transmissions_hw prefix="right" />
+    <xacro:index_finger_transmissions_hw prefix="left" reflect="1" />
+    <xacro:middle_finger_transmissions_hw prefix="left" reflect="1"/>
+    <xacro:pinky_finger_transmissions_hw prefix="left" reflect="1"/>
+    <xacro:thumb_transmissions_hw prefix="left" reflect="1"/>
+    <xacro:index_finger_transmissions_hw prefix="right" reflect="-1"/>
+    <xacro:middle_finger_transmissions_hw prefix="right" reflect="-1"/>
+    <xacro:pinky_finger_transmissions_hw prefix="right" reflect="-1"/>
+    <xacro:thumb_transmissions_hw prefix="right" reflect="-1"/>
 </robot>

File: model/robots/forearm_left.xacro (robot description, xacro)
@@ -12,8 +12,8 @@
     </joint>
     <xacro:make_lower_arm prefix="${prefix}" reflect="${reflect}" lower_arm_root_link="world"/>
-    <xacro:index_finger_transmissions_hw prefix="${prefix}" />
-    <xacro:middle_finger_transmissions_hw prefix="${prefix}" />
-    <xacro:pinky_finger_transmissions_hw prefix="${prefix}" />
-    <xacro:thumb_transmissions_hw prefix="${prefix}" />
+    <xacro:index_finger_transmissions_hw prefix="${prefix}" reflect="${reflect}"/>
+    <xacro:middle_finger_transmissions_hw prefix="${prefix}" reflect="${reflect}"/>
+    <xacro:pinky_finger_transmissions_hw prefix="${prefix}" reflect="${reflect}"/>
+    <xacro:thumb_transmissions_hw prefix="${prefix}" reflect="${reflect}"/>
     <xacro:athena1_transmission prefix="${prefix}" transmissionName="${prefix}ArmAthena1Transmission" actuatorApi="${Athena1Api}" nodeName="${Athena1Node}"/>
     <xacro:athena2_transmission prefix="${prefix}" transmissionName="${prefix}ArmAthena2Transmission" actuatorApi="${Athena2Api}" nodeName="${Athena2Node}"/>

File: model/robots/forearm_right.xacro (robot description, xacro)
@@ -12,8 +12,8 @@
     </joint>
     <xacro:make_lower_arm prefix="${prefix}" reflect="${reflect}" lower_arm_root_link="world"/>
-    <xacro:index_finger_transmissions_hw prefix="${prefix}" />
-    <xacro:middle_finger_transmissions_hw prefix="${prefix}" />
-    <xacro:pinky_finger_transmissions_hw prefix="${prefix}" />
-    <xacro:thumb_transmissions_hw prefix="${prefix}" />
+    <xacro:index_finger_transmissions_hw prefix="${prefix}" reflect="-1"/>
+    <xacro:middle_finger_transmissions_hw prefix="${prefix}" reflect="-1"/>
+    <xacro:pinky_finger_transmissions_hw prefix="${prefix}" reflect="-1"/>
+    <xacro:thumb_transmissions_hw prefix="${prefix}" reflect="-1"/>
     <xacro:athena1_transmission prefix="${prefix}" transmissionName="${prefix}ArmAthena1Transmission" actuatorApi="${Athena1Api}" nodeName="${Athena1Node}"/>
     <xacro:athena2_transmission prefix="${prefix}" transmissionName="${prefix}ArmAthena2Transmission" actuatorApi="${Athena2Api}" nodeName="${Athena2Node}"/>
