Commit message: Updated API's since changing TurbodriverAPI_linear to TurbodriverAPI_linear_futek.

File: common/xacro/api/valkyrie_A_api.xacro (robot description, xacro)
@@ -4,6 +4,6 @@
     <xacro:property name="HipPitchApi" value="robot_hardware_interface/TurbodriverAPI" />
     <xacro:property name="KneePitchApi" value="robot_hardware_interface/TurbodriverAPI" />
-    <xacro:property name="AnkleRightActuatorApi" value="robot_hardware_interface/TurbodriverAPI_linear" />
-    <xacro:property name="AnkleLeftActuatorApi" value="robot_hardware_interface/TurbodriverAPI_linear" />
+    <xacro:property name="AnkleRightActuatorApi" value="robot_hardware_interface/TurbodriverAPI_linear_futek" />
+    <xacro:property name="AnkleLeftActuatorApi" value="robot_hardware_interface/TurbodriverAPI_linear_futek" />
     <xacro:property name="ShoulderPitchApi" value="robot_hardware_interface/TurbodriverAPI" />
     <xacro:property name="ShoulderRollApi" value="robot_hardware_interface/TurbodriverAPI" />
@@ -11,12 +11,12 @@
     <xacro:property name="ElbowPitchApi" value="robot_hardware_interface/TurbodriverAPI" />
     <xacro:property name="ForearmYawApi" value="robot_hardware_interface/TurbodriverAPI" />
-    <xacro:property name="WristTopActuatorApi" value="robot_hardware_interface/TurbodriverAPI_linear" />
-    <xacro:property name="WristBottomActuatorApi" value="robot_hardware_interface/TurbodriverAPI_linear" />
+    <xacro:property name="WristTopActuatorApi" value="robot_hardware_interface/TurbodriverAPI_linear_futek" />
+    <xacro:property name="WristBottomActuatorApi" value="robot_hardware_interface/TurbodriverAPI_linear_futek" />
     <xacro:property name="LowerNeckPitchApi" value="robot_hardware_interface/TurbodriverAPI" />
     <xacro:property name="NeckYawApi" value="robot_hardware_interface/TurbodriverAPI" />
     <xacro:property name="UpperNeckPitchApi" value="robot_hardware_interface/TurbodriverAPI" />
     <xacro:property name="TrunkYawApi" value="robot_hardware_interface/TurbodriverAPI" />
-    <xacro:property name="WaistLeftActuatorApi" value="robot_hardware_interface/TurbodriverAPI_linear" />
-    <xacro:property name="WaistRightActuatorApi" value="robot_hardware_interface/TurbodriverAPI_linear" />
+    <xacro:property name="WaistLeftActuatorApi" value="robot_hardware_interface/TurbodriverAPI_linear_futek" />
+    <xacro:property name="WaistRightActuatorApi" value="robot_hardware_interface/TurbodriverAPI_linear_futek" />
     <xacro:property name="AtiSensorApi" value="TurbodriverForceTorqueSensor" />
     <xacro:property name="ImuMicrostrainHardwareApi" value="val_imu_3dm_gx4_15_interface/Imu3dmGx415Interface" />

File: common/xacro/api/valkyrie_C_api.xacro (robot description, xacro)
@@ -4,6 +4,6 @@
     <xacro:property name="HipPitchApi" value="robot_hardware_interface/TurbodriverAPI" />
     <xacro:property name="KneePitchApi" value="robot_hardware_interface/TurbodriverAPI" />
-    <xacro:property name="AnkleRightActuatorApi" value="robot_hardware_interface/TurbodriverAPI_linear" />
-    <xacro:property name="AnkleLeftActuatorApi" value="robot_hardware_interface/TurbodriverAPI_linear" />
+    <xacro:property name="AnkleRightActuatorApi" value="robot_hardware_interface/TurbodriverAPI_linear_futek" />
+    <xacro:property name="AnkleLeftActuatorApi" value="robot_hardware_interface/TurbodriverAPI_linear_futek" />
     <xacro:property name="ShoulderPitchApi" value="robot_hardware_interface/TurbodriverAPI" />
     <xacro:property name="ShoulderRollApi" value="robot_hardware_interface/TurbodriverAPI" />
@@ -11,12 +11,12 @@
     <xacro:property name="ElbowPitchApi" value="robot_hardware_interface/TurbodriverAPI" />
     <xacro:property name="ForearmYawApi" value="robot_hardware_interface/TurbodriverAPI" />
-    <xacro:property name="WristTopActuatorApi" value="robot_hardware_interface/TurbodriverAPI_linear" />
-    <xacro:property name="WristBottomActuatorApi" value="robot_hardware_interface/TurbodriverAPI_linear" />
+    <xacro:property name="WristTopActuatorApi" value="robot_hardware_interface/TurbodriverAPI_linear_futek" />
+    <xacro:property name="WristBottomActuatorApi" value="robot_hardware_interface/TurbodriverAPI_linear_futek" />
     <xacro:property name="LowerNeckPitchApi" value="robot_hardware_interface/TurbodriverAPI" />
     <xacro:property name="NeckYawApi" value="robot_hardware_interface/TurbodriverAPI" />
     <xacro:property name="UpperNeckPitchApi" value="robot_hardware_interface/TurbodriverAPI" />
     <xacro:property name="TrunkYawApi" value="robot_hardware_interface/TurbodriverAPI" />
-    <xacro:property name="WaistLeftActuatorApi" value="robot_hardware_interface/TurbodriverAPI_linear_renishaw" />
-    <xacro:property name="WaistRightActuatorApi" value="robot_hardware_interface/TurbodriverAPI_linear_renishaw" />
+    <xacro:property name="WaistLeftActuatorApi" value="robot_hardware_interface/TurbodriverAPI_linear_Renishaw" />
+    <xacro:property name="WaistRightActuatorApi" value="robot_hardware_interface/TurbodriverAPI_linear_Renishaw" />
     <xacro:property name="AtiSensorApi" value="TurbodriverForceTorqueSensor" />
     <xacro:property name="ImuMicrostrainHardwareApi" value="val_imu_3dm_gx4_15_interface/Imu3dmGx415Interface" />
