Commit message: Fixed api names in valkyrie_api.xacro.

File: common/xacro/api/valkyrie_api.xacro (robot description, xacro)
@@ -1,22 +1,22 @@
 <robot xmlns:xacro="http://ros.org/wiki/xacro" name="valkyrie_api">
-	<xacro:property name="HipYawApi" value="TurboDriverDRC_v4" />
-	<xacro:property name="HipRollApi" value="TurboDriverDRC_v4" />
-	<xacro:property name="HipPitchApi" value="TurboDriverDRC_v4" />
-	<xacro:property name="KneePitchApi" value="TurboDriverDRC_v4" />
-	<xacro:property name="AnkleInsideActuatorApi" value="TurboDriverDRC_v4_linear" />
-	<xacro:property name="AnkleOutsideActuatorApi" value="TurboDriverDRC_v4_linear" />
-	<xacro:property name="ShoulderPitchApi" value="TurboDriverDRC_v4" />
-	<xacro:property name="ShoulderRollApi" value="TurboDriverDRC_v4" />
-	<xacro:property name="ShoulderYawApi" value="TurboDriverDRC_v4" />
-	<xacro:property name="ElbowPitchApi" value="TurboDriverDRC_v4" />
-	<xacro:property name="ForearmYawApi" value="TurboDriverDRC_v4" />
-	<xacro:property name="WristTopActuatorApi" value="TurboDriverDRC_v4_linear" />
-	<xacro:property name="WristBottomActuatorApi" value="TurboDriverDRC_v4_linear" />
-	<xacro:property name="LowerNeckPitchApi" value="TurboDriverDRC_v4" />
-	<xacro:property name="NeckYawApi" value="TurboDriverDRC_v4" />
-	<xacro:property name="UpperNeckPitchApi" value="TurboDriverDRC_v4" />
-	<xacro:property name="TrunkYawApi" value="TurboDriverDRC_v4" />
-	<xacro:property name="WaistLeftActuatorApi" value="TurboDriverDRC_v4_linear" />
-	<xacro:property name="WaistRightActuatorApi" value="TurboDriverDRC_v4_linear" />
-	<xacro:property name="SimApi" value="TurboDriverDRC_v4" />
+	<xacro:property name="HipYawApi" value="robot_hardware_interface/TurbodriverAPI_DRCv4" />
+	<xacro:property name="HipRollApi" value="robot_hardware_interface/TurbodriverAPI_DRCv4" />
+	<xacro:property name="HipPitchApi" value="robot_hardware_interface/TurbodriverAPI_DRCv4" />
+	<xacro:property name="KneePitchApi" value="robot_hardware_interface/TurbodriverAPI_DRCv4" />
+	<xacro:property name="AnkleInsideActuatorApi" value="robot_hardware_interface/TurbodriverAPI_DRCv4_linear" />
+	<xacro:property name="AnkleOutsideActuatorApi" value="robot_hardware_interface/TurbodriverAPI_DRCv4_linear" />
+	<xacro:property name="ShoulderPitchApi" value="robot_hardware_interface/TurbodriverAPI_DRCv4" />
+	<xacro:property name="ShoulderRollApi" value="robot_hardware_interface/TurbodriverAPI_DRCv4" />
+	<xacro:property name="ShoulderYawApi" value="robot_hardware_interface/TurbodriverAPI_DRCv4" />
+	<xacro:property name="ElbowPitchApi" value="robot_hardware_interface/TurbodriverAPI_DRCv4" />
+	<xacro:property name="ForearmYawApi" value="robot_hardware_interface/TurbodriverAPI_DRCv4" />
+	<xacro:property name="WristTopActuatorApi" value="robot_hardware_interface/TurbodriverAPI_DRCv4_linear" />
+	<xacro:property name="WristBottomActuatorApi" value="robot_hardware_interface/TurbodriverAPI_DRCv4_linear" />
+	<xacro:property name="LowerNeckPitchApi" value="robot_hardware_interface/TurbodriverAPI_DRCv4" />
+	<xacro:property name="NeckYawApi" value="robot_hardware_interface/TurbodriverAPI_DRCv4" />
+	<xacro:property name="UpperNeckPitchApi" value="robot_hardware_interface/TurbodriverAPI_DRCv4" />
+	<xacro:property name="TrunkYawApi" value="robot_hardware_interface/TurbodriverAPI_DRCv4" />
+	<xacro:property name="WaistLeftActuatorApi" value="robot_hardware_interface/TurbodriverAPI_DRCv4_linear" />
+	<xacro:property name="WaistRightActuatorApi" value="robot_hardware_interface/TurbodriverAPI_DRCv4_linear" />
+	<xacro:property name="SimApi" value="robot_hardware_interface/TurboDriverSimApiDRC_v4" />
 </robot>

Commit message: added api tag to force-torque sensor

File: common/xacro/api/valkyrie_api.xacro (robot description, xacro)
@@ -19,4 +19,5 @@
 	<xacro:property name="WaistLeftActuatorApi" value="robot_hardware_interface/TurbodriverAPI_DRCv4_linear" />
 	<xacro:property name="WaistRightActuatorApi" value="robot_hardware_interface/TurbodriverAPI_DRCv4_linear" />
+	<xacro:property name="AtiSensorApi" value="TurbodriverForceTorqueSensor_v1.xml" />
 	<xacro:property name="SimApi" value="robot_hardware_interface/TurboDriverSimApiDRC_v4" />
 </robot>

File: model/robots/common/xacro/leg/leg.xacro (robot description, xacro)
@@ -148,5 +148,6 @@
                         origin_rpy="3.14 0.0 -1.047"
                         sensor_number="${ATI_serial_number}"
-                        sensor_node="${ATI_node}"/>
+                        sensor_node="${ATI_node}"
+                        sensor_api="${AtiSensorApi}" />
   </xacro:macro>
   <xacro:macro name="leg_transmissions_hw" params="prefix">

File: model/robots/common/xacro/sensors/ati_force_torque.xacro (robot description, xacro)
@@ -1,5 +1,5 @@
 <?xml version="1.0" ?>
 <robot xmlns:xacro="http://www.ros.org/wiki/xacro" name="ati_force_torque_sensor">
-  <xacro:macro name="ati_force_torque_sensor" params="sensorName parentLink joint_to_attach_sensor_to origin_xyz origin_rpy sensor_number sensor_node">
+  <xacro:macro name="ati_force_torque_sensor" params="sensorName parentLink joint_to_attach_sensor_to origin_xyz origin_rpy sensor_number sensor_node sensor_api">
     <gazebo reference="${joint_to_attach_sensor_to}">
       <sensor name="${sensorName}" type="force_torque">
@@ -7,4 +7,5 @@
         <sensor_number id="${sensor_number}" />
         <node ide="${sensor_node}" />
+        <api name="${sensor_api}" />
         <always_on>true</always_on>
         <update_rate>1000</update_rate>

Commit message: Removed .xml from api tag for F/T sensor.

File: common/xacro/api/valkyrie_api.xacro (robot description, xacro)
@@ -19,5 +19,5 @@
 	<xacro:property name="WaistLeftActuatorApi" value="robot_hardware_interface/TurbodriverAPI_DRCv4_linear" />
 	<xacro:property name="WaistRightActuatorApi" value="robot_hardware_interface/TurbodriverAPI_DRCv4_linear" />
-	<xacro:property name="AtiSensorApi" value="TurbodriverForceTorqueSensor_v1.xml" />
+	<xacro:property name="AtiSensorApi" value="TurbodriverForceTorqueSensor_v1" />
 	<xacro:property name="SimApi" value="robot_hardware_interface/TurboDriverSimApiDRC_v4" />
 </robot>

Commit message: added xacro files for adding imus

File: common/xacro/api/valkyrie_api.xacro (robot description, xacro)
@@ -20,4 +20,6 @@
 	<xacro:property name="WaistRightActuatorApi" value="robot_hardware_interface/TurbodriverAPI_DRCv4_linear" />
 	<xacro:property name="AtiSensorApi" value="TurbodriverForceTorqueSensor_v1" />
+	<xacro:property name="ImuSensorHardwareApi" value="imu_3dm_gx4_interface/Imu3dmGx4Interface" />
+	<xacro:property name="ImuSensorSimApi" value="imu_gazebo_interface/ImuGazeboInterface" />
 	<xacro:property name="SimApi" value="robot_hardware_interface/TurbodriverSimAPI_DRCv4" />
 </robot>

File: common/xacro/nodes/valkyrie_nodes.xacro (robot description, xacro)
@@ -25,5 +25,5 @@
 	<xacro:property name="WaistPitchActuatorSimNode" value="/trunk/pitch_actuator" /> <!--pitch-->
 	<xacro:property name="WaistRollActuatorSimNode" value="/trunk/roll_actuator" /> <!--roll-->
-	<xacro:property name="pelvis_imu1_node" value="/pelvis/sensors/imu1" />
+	<xacro:property name="pelvis_imu1_node" value="/sensors/leftPelvisIMU" />
 	<xacro:property name="pelvis_imu2_node" value="/pelvis/sensors/imu2" />
 	<xacro:property name="torso_imu1_node" value="/torso/sensors/imu1" />

File: model/robots/common/xacro/pelvis/pelvis.xacro (robot description, xacro)
@@ -21,3 +21,16 @@
                                   origin_rpy="3.14159 0.0 -3.14159" />
     </xacro:macro>
+    <xacro:macro name="v1_pelvis_sensors_plugin" params="sensor_node_tag sensor_api_tag sensor_port_tag">
+        <xacro:microstrain_sensor sensorName="pelvisRearImu"
+                                  parentLink="${Pelvis_Link_Name}"
+                                  origin_xyz="-0.075844901 0.0 -0.111056426"
+                                  origin_rpy="-3.14159 0.476467 -3.14159" />
+        <xacro:plugged_in_microstrain_sensor sensorName="pelvisMiddleImu"
+                                  parentLink="${Pelvis_Link_Name}"
+                                  origin_xyz="0.012 0.0 -0.108184035"
+                                  origin_rpy="3.14159 0.0 -3.14159"
+                                  sensor_node="${sensor_node_tag}"
+                                  sensor_api="${sensor_api_tag}"
+                                  sensor_port="${sensor_port_tag}" />
+    </xacro:macro>
 </robot>

File: model/robots/common/xacro/sensors/microstrain.xacro (robot description, xacro)
@@ -43,3 +43,48 @@
     </gazebo>
   </xacro:macro>
+  <xacro:macro name="plugged_in_microstrain_sensor" params="sensorName parentLink origin_xyz origin_rpy sensor_node sensor_api sensor_port">
+    <xacro:massless_virtual_link name="${sensorName}_Frame"
+                    origin_rpy="0 0 0"
+                    origin_xyz="0 0 0"/>
+    <xacro:fixed_joint jointName="${sensorName}_Offset"
+                       parent="${parentLink}" child="${sensorName}_Frame"
+                       origin_rpy="${origin_rpy}"
+                       origin_xyz="${origin_xyz}"/>
+    <gazebo>
+      <plugin filename="libgazebo_ros_imu.so" name="imu_plugin_ros">
+        <alwaysOn>true</alwaysOn>
+        <bodyName>${sensorName}_Frame</bodyName>
+        <topicName>${sensorName}/imu</topicName>
+        <serviceName>${sensorName}/imu_service</serviceName>
+        <gaussianNoise>0.0</gaussianNoise>
+        <updateRate>1000.0</updateRate>
+      </plugin>
+    </gazebo>
+    <gazebo reference="${sensorName}_Frame">
+      <sensor name="${sensorName}" type="imu">
+        <always_on>true</always_on>
+        <pose>0 0 0 0 0 0 </pose>
+        <node name="${sensor_node}" />
+        <api name="${sensor_api}" />
+        <port name="${sensor_port}" />
+        <imu>
+           <noise>
+               <type>gaussian</type>
+               <rate>
+                   <mean>0</mean>
+                   <stddev>0.0002</stddev>
+                   <bias_mean>7.5e-06</bias_mean>
+                   <bias_stddev>8e-07</bias_stddev>
+               </rate>
+               <accel>
+                   <mean>0</mean>
+                   <stddev>0.017</stddev>
+                   <bias_mean>0.1</bias_mean>
+                   <bias_stddev>0.001</bias_stddev>
+               </accel>
+           </noise>
+        </imu>
+        </sensor>
+    </gazebo>
+  </xacro:macro>
 </robot>

File: model/robots/common/xacro/valkyrie_base_sim.xacro (robot description, xacro)
@@ -20,5 +20,5 @@
     <xacro:make_leg prefix="right" reflect="-1" leg_root_link="${Pelvis_Link_Name}"/>
     <xacro:make_leg prefix="left" reflect="1" leg_root_link="${Pelvis_Link_Name}"/>
-    <xacro:v1_pelvis_sensors />
+    <xacro:v1_pelvis_sensors_plugin sensor_node_tag="${pelvis_imu1_node}" sensor_api_tag="${ImuSensorSimApi}" sensor_port_tag="${pelvis_imu1_port}"/>
     <xacro:v1_leg_sensors prefix="left" reflect="1" ATI_serial_number="${sim_ATI_serial}" ATI_node="${left_foot_Sim_ATI_node}"/>
     <xacro:v1_leg_sensors prefix="right" reflect="-1" ATI_serial_number="${sim_ATI_serial}" ATI_node="${right_foot_Sim_ATI_node}"/>

File: model/robots/valkyrie_B_hw.xacro (robot description, xacro)
@@ -5,3 +5,4 @@
     <xacro:include filename="$(find val_description)/model/robots/common/xacro/valkyrie_base_hw.xacro"/>
     <xacro:include filename="$(find val_description)/common/xacro/serial_numbers/valkyrie_B_serials.xacro"/>
+    <xacro:include filename="$(find val_description)/common/xacro/dev_ports/valkyrie_B_ports.xacro"/>
 </robot>

File: model/robots/valkyrie_B_no_hands_hw.xacro (robot description, xacro)
@@ -5,3 +5,4 @@
     <xacro:include filename="$(find val_description)/model/robots/common/xacro/valkyrie_no_hands_base_hw.xacro"/>
     <xacro:include filename="$(find val_description)/common/xacro/serial_numbers/valkyrie_B_serials.xacro"/>
+    <xacro:include filename="$(find val_description)/common/xacro/dev_ports/valkyrie_B_ports.xacro"/>
 </robot>

File: model/robots/valkyrie_C_hw.xacro (robot description, xacro)
@@ -5,3 +5,4 @@
     <xacro:include filename="$(find val_description)/model/robots/common/xacro/valkyrie_base_hw.xacro"/>
     <xacro:include filename="$(find val_description)/common/xacro/serial_numbers/valkyrie_C_serials.xacro"/>
+    <xacro:include filename="$(find val_description)/common/xacro/dev_ports/valkyrie_C_ports.xacro"/>
 </robot>

File: model/robots/valkyrie_C_no_hands_hw.xacro (robot description, xacro)
@@ -5,3 +5,4 @@
     <xacro:include filename="$(find val_description)/model/robots/common/xacro/valkyrie_no_hands_base_hw.xacro"/>
     <xacro:include filename="$(find val_description)/common/xacro/serial_numbers/valkyrie_C_serials.xacro"/>
+    <xacro:include filename="$(find val_description)/common/xacro/dev_ports/valkyrie_C_ports.xacro"/>
 </robot>

File: model/robots/valkyrie_remote_sim.xacro (robot description, xacro)
@@ -6,3 +6,4 @@
     <xacro:include filename="$(find val_description)/model/urdf/multisense_sl_remote.urdf" />
     <xacro:include filename="$(find val_description)/common/xacro/serial_numbers/valkyrie_A_serials.xacro"/>
+    <xacro:include filename="$(find val_description)/common/xacro/dev_ports/valkyrie_gazebo_ports.xacro"/>
 </robot>

File: model/robots/valkyrie_remote_sim_pinned.xacro (robot description, xacro)
@@ -7,4 +7,5 @@
     <xacro:include filename="$(find val_description)/model/urdf/multisense_sl_remote.urdf" />
     <xacro:include filename="$(find val_description)/common/xacro/serial_numbers/valkyrie_A_serials.xacro"/>
+    <xacro:include filename="$(find val_description)/common/xacro/dev_ports/valkyrie_gazebo_ports.xacro"/>
     <link name="world"/>
     <joint name="fixed" type="fixed">

File: model/robots/valkyrie_sim.xacro (robot description, xacro)
@@ -6,3 +6,4 @@
     <xacro:include filename="$(find val_description)/model/urdf/multisense_sl.urdf" />
     <xacro:include filename="$(find val_description)/common/xacro/serial_numbers/valkyrie_A_serials.xacro"/>
+    <xacro:include filename="$(find val_description)/common/xacro/dev_ports/valkyrie_gazebo_ports.xacro"/>
 </robot>

File: model/robots/valkyrie_sim_pinned.xacro (robot description, xacro)
@@ -7,4 +7,5 @@
     <xacro:include filename="$(find val_description)/model/urdf/multisense_sl.urdf" />
     <xacro:include filename="$(find val_description)/common/xacro/serial_numbers/valkyrie_A_serials.xacro"/>
+    <xacro:include filename="$(find val_description)/common/xacro/dev_ports/valkyrie_gazebo_ports.xacro"/>
     <link name="world"/>
     <joint name="fixed" type="fixed">

Commit message: updated plugin names for imus

File: common/xacro/api/valkyrie_api.xacro (robot description, xacro)
@@ -20,6 +20,6 @@
 	<xacro:property name="WaistRightActuatorApi" value="robot_hardware_interface/TurbodriverAPI_DRCv4_linear" />
 	<xacro:property name="AtiSensorApi" value="TurbodriverForceTorqueSensor_v1" />
-	<xacro:property name="ImuSensorHardwareApi" value="imu_3dm_gx4_interface/Imu3dmGx4Interface" />
-	<xacro:property name="ImuSensorSimApi" value="imu_gazebo_interface/ImuGazeboInterface" />
+	<xacro:property name="ImuSensorHardwareApi" value="val_imu_3dm_gx4_15_interface/Imu3dmGx415Interface" />
+	<xacro:property name="ImuSensorSimApi" value="val_imu_gazebo_interface/ImuGazeboInterface" />
 	<xacro:property name="SimApi" value="robot_hardware_interface/TurbodriverSimAPI_DRCv4" />
 </robot>

Commit message: Gotta break to fix something for Wolfgang.

File: common/xacro/api/valkyrie_api.xacro (robot description, xacro)
@@ -19,4 +19,10 @@
 	<xacro:property name="WaistLeftActuatorApi" value="robot_hardware_interface/TurbodriverAPI_DRCv4_linear" />
 	<xacro:property name="WaistRightActuatorApi" value="robot_hardware_interface/TurbodriverAPI_DRCv4_linear" />
+	<xacro:property name="ThumbRollApi" value="robot_hardware_interface/ThumbRollApi"/>
+	<xacro:property name="ThumbPitch1Api" value="robot_hardware_interface/ThumbPitch1Api"/>
+	<xacro:property name="ThumbPitch2Api" value="robot_hardware_interface/ThumbPitch2Api"/>
+	<xacro:property name="IndexFingerApi" value="robot_hardware_interface/IndexFingerApi"/>
+	<xacro:property name="MiddleFingerApi" value="robot_hardware_interface/MiddleFingerApi"/>
+	<xacro:property name="PinkyApi" value="robot_hardware_interface/PinkyFingerApi"/>
 	<xacro:property name="AtiSensorApi" value="TurbodriverForceTorqueSensor_v1" />
 	<xacro:property name="ImuSensorHardwareApi" value="val_imu_3dm_gx4_15_interface/Imu3dmGx415Interface" />

File: common/xacro/nodes/valkyrie_nodes.xacro (robot description, xacro)
@@ -25,4 +25,10 @@
 	<xacro:property name="WaistPitchActuatorSimNode" value="/trunk/pitch_actuator" /> <!--pitch-->
 	<xacro:property name="WaistRollActuatorSimNode" value="/trunk/roll_actuator" /> <!--roll-->
+	<xacro:property name="ThumbRollNode" value="/forearmDriver1"/>
+	<xacro:property name="ThumbPitch1Node" value="/forearmDriver1"/>
+	<xacro:property name="ThumbPitch2Node" value="/forearmDriver1"/>
+	<xacro:property name="IndexFingerNode" value="/forearmDriver2"/>
+	<xacro:property name="MiddleFingerNode" value="/forearmDriver2"/>
+	<xacro:property name="PinkyNode" value="/forearmDriver2"/>
 	<xacro:property name="pelvis_middle_imu_node" value="/sensors/middlePelvisIMU" />
 	<xacro:property name="pelvis_rear_imu_node" value="/sensors/rearPelvisIMU" />

File: model/robots/common/xacro/generic_models.xacro (robot description, xacro)
@@ -1,7 +1,4 @@
 <?xml version="1.0" ?>
 <robot xmlns:xacro="http://www.ros.org/wiki/xacro" name="generic_models">
-  <xacro:macro name="v1_actuator" params="name api">
-    <actuator name="${name}" type="${api}"/>
-  </xacro:macro>
   <xacro:macro name="standard_link" params="name mass origin_rpy origin_xyz ixx ixy ixz iyy iyz izz visual_mesh collision_mesh">
     <link name="${name}">
@@ -278,5 +275,22 @@
     </transmission>
   </xacro:macro>
-  <xacro:macro name="finger_transmission" params="transmissionName transmissionType joint1Name joint2Name joint3Name joint1Role joint2Role joint3Role actuator1Name actuator2Name actuator3Name actuator1Api actuator1Role actuator2Role actuator3Role">
+  <xacro:macro name="athena1_transmission" params="prefix">
+    <type>robot_transmission_interface/athena1_transmission</type>
+    <joint name="wristPitch">
+      <role>wristPitch</role>
+    </joint>
+    <joint name="wristRoll">
+      <role>wristRoll</role>
+    </joint>
+    <actuator name="wristTopActuator">
+      <role>="wristTopActuator"</role>
+      <mechanicalReduction>1</mechanicalReduction>
+      <hardwareInterface>PositionJointInterface</hardwareInterface>
+    </actuator>
+    <actuator name="wristBottomActuator">
+      <role>="wristBottomActuator"</role>
+      <mechanicalReduction>1</mechanicalReduction>
+      <hardwareInterface>PositionJointInterface</hardwareInterface>
+    </actuator>
   </xacro:macro>
 </robot>

File: model/robots/common/xacro/index_finger/index_finger.xacro (robot description, xacro)
@@ -69,9 +69,3 @@
     </xacro:revolute_joint>
   </xacro:macro>
-  <xacro:macro name="v1_right_index_finger_actuators" params="prefix api">
-    <xacro:v1_actuator name="${RPFA_Actuator_Name}" api="${api}" />
-  </xacro:macro>
-  <xacro:macro name="v1_left_index_finger_actuators" params="prefix api">
-    <xacro:v1_actuator name="${LPFA_Actuator_Name}" api="${api}" />
-  </xacro:macro>
 </robot>

File: model/robots/common/xacro/middle_finger/middle_finger.xacro (robot description, xacro)
@@ -69,9 +69,3 @@
     </xacro:revolute_joint>
   </xacro:macro>
-  <xacro:macro name="v1_right_middle_finger_actuators" params="prefix api">
-    <xacro:v1_actuator name="${RMFA_Actuator_Name}" api="${api}" />
-  </xacro:macro>
-  <xacro:macro name="v1_left_middle_finger_actuators" params="prefix api">
-    <xacro:v1_actuator name="${LMFA_Actuator_Name}" api="${api}" />
-  </xacro:macro>
 </robot>

File: model/robots/common/xacro/pinky_finger/pinky_finger.xacro (robot description, xacro)
@@ -69,9 +69,3 @@
     </xacro:revolute_joint>
   </xacro:macro>
-  <xacro:macro name="v1_right_pinky_finger_actuators" params="prefix api">
-    <xacro:v1_actuator name="${RLFA_Actuator_Name}" api="${api}" />
-  </xacro:macro>
-  <xacro:macro name="v1_left_pinky_finger_actuators" params="prefix api">
-    <xacro:v1_actuator name="${LLFA_Actuator_Name}" api="${api}" />
-  </xacro:macro>
 </robot>

File: model/robots/common/xacro/thumb/thumb.xacro (robot description, xacro)
@@ -84,6 +84,3 @@
     </xacro:revolute_joint>
   </xacro:macro>
-  <xacro:macro name="thumb_transmissions" params="prefix">
-    <xacro:simple_transmission jointName="${ThumbRollJointName}" actuatorName="${ThumbRollActuatorName}" nodeName="${ThumbRollNodeName}" actuatorApi="${SimApi}"/>
-  </xacro:macro>
 </robot>

File: model/robots/common/xacro/valkyrie_base_hw.xacro (robot description, xacro)
@@ -26,3 +26,11 @@
     <xacro:arm_transmissions_hw prefix="right"/>
     <xacro:neck_transmissions_hw />
+    <xacro:thumb_transmissions prefix="left"/>
+    <xacro:thumb_transmissions prefix="right"/>
+    <xacro:index_finger_transmissions prefix="left"/>
+    <xacro:index_finger_transmissions prefix="right"/>
+    <xacro:middle_finger_transmissions prefix="left"/>
+    <xacro:middle_finger_transmissions prefix="right"/>
+    <xacro:pinky_finger_transmissions prefix="left"/>
+    <xacro:pinky_finger_transmissions prefix="right"/>
 </robot>
