Commit message: Updated API's for new names.

File: common/xacro/api/valkyrie_api.xacro (robot description, xacro)
@@ -1,25 +1,25 @@
 <robot xmlns:xacro="http://ros.org/wiki/xacro" name="valkyrie_api">
-	<xacro:property name="HipYawApi" value="robot_hardware_interface/TurbodriverAPI_DRCv4" />
-	<xacro:property name="HipRollApi" value="robot_hardware_interface/TurbodriverAPI_DRCv4" />
-	<xacro:property name="HipPitchApi" value="robot_hardware_interface/TurbodriverAPI_DRCv4" />
-	<xacro:property name="KneePitchApi" value="robot_hardware_interface/TurbodriverAPI_DRCv4" />
-	<xacro:property name="AnkleRightActuatorApi" value="robot_hardware_interface/TurbodriverAPI_DRCv4_linear" />
-	<xacro:property name="AnkleLeftActuatorApi" value="robot_hardware_interface/TurbodriverAPI_DRCv4_linear" />
-	<xacro:property name="ShoulderPitchApi" value="robot_hardware_interface/TurbodriverAPI_DRCv4" />
-	<xacro:property name="ShoulderRollApi" value="robot_hardware_interface/TurbodriverAPI_DRCv4" />
-	<xacro:property name="ShoulderYawApi" value="robot_hardware_interface/TurbodriverAPI_DRCv4" />
-	<xacro:property name="ElbowPitchApi" value="robot_hardware_interface/TurbodriverAPI_DRCv4" />
-	<xacro:property name="ForearmYawApi" value="robot_hardware_interface/TurbodriverAPI_DRCv4" />
-	<xacro:property name="WristTopActuatorApi" value="robot_hardware_interface/TurbodriverAPI_DRCv4_linear" />
-	<xacro:property name="WristBottomActuatorApi" value="robot_hardware_interface/TurbodriverAPI_DRCv4_linear" />
-	<xacro:property name="LowerNeckPitchApi" value="robot_hardware_interface/TurbodriverAPI_DRCv4" />
-	<xacro:property name="NeckYawApi" value="robot_hardware_interface/TurbodriverAPI_DRCv4" />
-	<xacro:property name="UpperNeckPitchApi" value="robot_hardware_interface/TurbodriverAPI_DRCv4" />
-	<xacro:property name="TrunkYawApi" value="robot_hardware_interface/TurbodriverAPI_DRCv4" />
-	<xacro:property name="WaistLeftActuatorApi" value="robot_hardware_interface/TurbodriverAPI_DRCv4_linear" />
-	<xacro:property name="WaistRightActuatorApi" value="robot_hardware_interface/TurbodriverAPI_DRCv4_linear" />
+	<xacro:property name="HipYawApi" value="robot_hardware_interface/TurbodriverAPI" />
+	<xacro:property name="HipRollApi" value="robot_hardware_interface/TurbodriverAPI" />
+	<xacro:property name="HipPitchApi" value="robot_hardware_interface/TurbodriverAPI" />
+	<xacro:property name="KneePitchApi" value="robot_hardware_interface/TurbodriverAPI" />
+	<xacro:property name="AnkleRightActuatorApi" value="robot_hardware_interface/TurbodriverAPI_linear" />
+	<xacro:property name="AnkleLeftActuatorApi" value="robot_hardware_interface/TurbodriverAPI_linear" />
+	<xacro:property name="ShoulderPitchApi" value="robot_hardware_interface/TurbodriverAPI" />
+	<xacro:property name="ShoulderRollApi" value="robot_hardware_interface/TurbodriverAPI" />
+	<xacro:property name="ShoulderYawApi" value="robot_hardware_interface/TurbodriverAPI" />
+	<xacro:property name="ElbowPitchApi" value="robot_hardware_interface/TurbodriverAPI" />
+	<xacro:property name="ForearmYawApi" value="robot_hardware_interface/TurbodriverAPI" />
+	<xacro:property name="WristTopActuatorApi" value="robot_hardware_interface/TurbodriverAPI_linear" />
+	<xacro:property name="WristBottomActuatorApi" value="robot_hardware_interface/TurbodriverAPI_linear" />
+	<xacro:property name="LowerNeckPitchApi" value="robot_hardware_interface/TurbodriverAPI" />
+	<xacro:property name="NeckYawApi" value="robot_hardware_interface/TurbodriverAPI" />
+	<xacro:property name="UpperNeckPitchApi" value="robot_hardware_interface/TurbodriverAPI" />
+	<xacro:property name="TrunkYawApi" value="robot_hardware_interface/TurbodriverAPI" />
+	<xacro:property name="WaistLeftActuatorApi" value="robot_hardware_interface/TurbodriverAPI_linear" />
+	<xacro:property name="WaistRightActuatorApi" value="robot_hardware_interface/TurbodriverAPI_linear" />
 	<xacro:property name="AtiSensorApi" value="TurbodriverForceTorqueSensor_v1" />
 	<xacro:property name="ImuSensorHardwareApi" value="val_imu_3dm_gx4_15_interface/Imu3dmGx415Interface" />
 	<xacro:property name="ImuSensorSimApi" value="val_imu_gazebo_interface/ImuGazeboInterface" />
-	<xacro:property name="SimApi" value="robot_hardware_interface/TurbodriverSimAPI_DRCv4" />
+	<xacro:property name="SimApi" value="robot_hardware_interface/TurbodriverSimAPI" />
 </robot>

Commit message: Updates since removing _v1 and _v2 from all API names.

File: common/xacro/api/valkyrie_api.xacro (robot description, xacro)
@@ -19,5 +19,5 @@
 	<xacro:property name="WaistLeftActuatorApi" value="robot_hardware_interface/TurbodriverAPI_linear" />
 	<xacro:property name="WaistRightActuatorApi" value="robot_hardware_interface/TurbodriverAPI_linear" />
-	<xacro:property name="AtiSensorApi" value="TurbodriverForceTorqueSensor_v1" />
+	<xacro:property name="AtiSensorApi" value="TurbodriverForceTorqueSensor" />
 	<xacro:property name="ImuSensorHardwareApi" value="val_imu_3dm_gx4_15_interface/Imu3dmGx415Interface" />
 	<xacro:property name="ImuSensorSimApi" value="val_imu_gazebo_interface/ImuGazeboInterface" />

Commit message: First cut of forearm testbench urdf.

File: common/xacro/api/valkyrie_api.xacro (robot description, xacro)
@@ -19,4 +19,10 @@
 	<xacro:property name="WaistLeftActuatorApi" value="robot_hardware_interface/TurbodriverAPI_DRCv4_linear" />
 	<xacro:property name="WaistRightActuatorApi" value="robot_hardware_interface/TurbodriverAPI_DRCv4_linear" />
+	<xacro:property name="ThumbRollApi" value="robot_hardware_interface/TurbodriverAPI_DRCv4" />
+	<xacro:property name="ThumbPitch1Api" value="robot_hardware_interface/TurbodriverAPI_DRCv4" />
+	<xacro:property name="ThumbPitch2Api" value="robot_hardware_interface/TurbodriverAPI_DRCv4" />
+	<xacro:property name="IndexFingerPitch1Api" value="robot_hardware_interface/TurbodriverAPI_DRCv4" />
+	<xacro:property name="MiddleFingerPitch1Api" value="robot_hardware_interface/TurbodriverAPI_DRCv4" />
+	<xacro:property name="PinkyPitch1Api" value="robot_hardware_interface/TurbodriverAPI_DRCv4" />
 	<xacro:property name="AtiSensorApi" value="TurbodriverForceTorqueSensor_v1" />
 	<xacro:property name="ImuSensorHardwareApi" value="val_imu_3dm_gx4_15_interface/Imu3dmGx415Interface" />

File: common/xacro/nodes/valkyrie_nodes.xacro (robot description, xacro)
@@ -13,6 +13,6 @@
 	<xacro:property name="ElbowPitchNode" value="/${prefix}_arm/j4" />
 	<xacro:property name="ForearmYawNode" value="/${prefix}_arm/j5" />
-	<xacro:property name="WristTopActuatorNode" value="/${prefix}_arm/wrist/top_actautor" />
-	<xacro:property name="WristBottomActuatorNode" value="/${prefix}_arm/wrist/bottom_actuator" />
+	<xacro:property name="WristTopActuatorNode" value="/${prefix}_arm/forearm/n7" />
+	<xacro:property name="WristBottomActuatorNode" value="/${prefix}_arm/forearm/n8" />
 	<xacro:property name="WristRollActuatorSimNode" value="/${prefix}_arm/wrist/roll_actautor" />
 	<xacro:property name="WristPitchActuatorSimNode" value="/${prefix}_arm/wrist/pitch_actuator" />
@@ -25,4 +25,10 @@
 	<xacro:property name="WaistPitchActuatorSimNode" value="/trunk/pitch_actuator" /> <!--pitch-->
 	<xacro:property name="WaistRollActuatorSimNode" value="/trunk/roll_actuator" /> <!--roll-->
+	<xacro:property name="ThumbRollNode" value="/${prefix}_arm/forearm/n1" />
+	<xacro:property name="ThumbPitch1Node" value="/${prefix}_arm/forearm/n2" />
+	<xacro:property name="ThumbPitch2Node" value="/${prefix}_arm/forearm/n3" />
+	<xacro:property name="IndexFingerPitch1Node" value="/${prefix}_arm/forearm/n4"/>
+	<xacro:property name="MiddleFingerPitch1Node" value="/${prefix}_arm/forearm/n5"/>
+	<xacro:property name="PinkyPitch1Node" value="/${prefix}_arm/forearm/n6"/>
 	<xacro:property name="pelvis_middle_imu_node" value="/sensors/middlePelvisIMU" />
 	<xacro:property name="pelvis_rear_imu_node" value="/sensors/rearPelvisIMU" />

File: model/robots/common/xacro/arm/arm.xacro (robot description, xacro)
@@ -166,5 +166,5 @@
     <xacro:simple_transmission jointName="${ElbowPitchJointName}" actuatorName="${ElbowPitchActuatorName}" nodeName="${ElbowPitchNode}" actuatorApi="${ElbowPitchApi}"/>
     <xacro:simple_transmission jointName="${ForearmYawActuatorName}" actuatorName="${ForearmYawActuatorName}" nodeName="${ForearmYawNode}" actuatorApi="${ForearmYawApi}"/>
-    <xacro:pushrod_transmission transmissionName="${prefix}WristTransmission" transmissionType="WristPushrodTransmission" joint1Name="${WristPitchJointName}" joint2Name="${WristRollJointName}" joint1Role="roll" joint2Role="pitch" actuator1Name="${WristTopActuatorName}" actuator2Name="${WristBottomActuatorName}" actuator1Node="${WristTopActuatorNode}" actuator2Node="${WristBottomActuatorNode}" actuator1Api="${WristTopActuatorApi}" actuator2Api="${WristBottomActuatorApi}" actuator1Role="top" actuator2Role="bottom"/>
+    <xacro:pushrod_transmission_position transmissionName="${prefix}WristTransmission" transmissionType="WristPushrodTransmission" joint1Name="${WristPitchJointName}" joint2Name="${WristRollJointName}" joint1Role="roll" joint2Role="pitch" actuator1Name="${WristTopActuatorName}" actuator2Name="${WristBottomActuatorName}" actuator1Node="${WristTopActuatorNode}" actuator2Node="${WristBottomActuatorNode}" actuator1Api="${WristTopActuatorApi}" actuator2Api="${WristBottomActuatorApi}" actuator1Role="top" actuator2Role="bottom"/>
   </xacro:macro>
   <xacro:macro name="arm_transmissions_no_hands" params="prefix">

File: model/robots/common/xacro/arm/link_names.xacro (robot description, xacro)
@@ -1,4 +1,4 @@
 <?xml version="1.0" ?>
-<robot xmlns:xacro="http://www.ros.org/wiki/xacro" name="v1/arm/link_names">
+<robot xmlns:xacro="http://www.ros.org/wiki/xacro" name="arm_link_names">
   <xacro:property name="ShoulderPitchParentLinkName" value="${arm_root_link}" />
   <xacro:property name="ShoulderPitchLinkName" value="${prefix}ShoulderPitchLink" />

File: model/robots/common/xacro/generic_models.xacro (robot description, xacro)
@@ -253,3 +253,28 @@
     </transmission>
   </xacro:macro>
+  <xacro:macro name="pushrod_transmission_position" params="transmissionName transmissionType joint1Name joint2Name joint1Role joint2Role actuator1Name actuator2Name actuator1Node actuator2Node actuator1Api actuator2Api actuator1Role actuator2Role">
+    <transmission name="${transmissionName}">
+      <type>robot_transmission_interface/${transmissionType}</type>
+      <joint name="${joint1Name}">
+        <role>${joint1Role}</role>
+        <hardwareInterface>PositionJointInterface</hardwareInterface>
+      </joint>
+      <joint name="${joint2Name}">
+        <role>${joint2Role}</role>
+        <hardwareInterface>PositionJointInterface</hardwareInterface>
+      </joint>
+       <actuator name="${actuator1Name}">
+        <node name="${actuator1Node}"/>
+        <role>${actuator1Role}</role>
+        <mechanicalReduction>1</mechanicalReduction>
+        <api name="${actuator1Api}"/>
+      </actuator>
+      <actuator name="${actuator2Name}">
+        <node name="${actuator2Node}"/>
+        <role>${actuator2Role}</role>
+        <mechanicalReduction>1</mechanicalReduction>
+        <api name="${actuator2Api}"/>
+      </actuator>
+    </transmission>
+  </xacro:macro>
 </robot>

File: model/robots/common/xacro/index_finger/index_finger.xacro (robot description, xacro)
@@ -69,9 +69,6 @@
     </xacro:revolute_joint>
   </xacro:macro>
-  <xacro:macro name="v1_right_index_finger_actuators" params="prefix api">
-    <xacro:v1_actuator name="${RPFA_Actuator_Name}" api="${api}" />
-  </xacro:macro>
-  <xacro:macro name="v1_left_index_finger_actuators" params="prefix api">
-    <xacro:v1_actuator name="${LPFA_Actuator_Name}" api="${api}" />
+  <xacro:macro name="index_finger_transmissions" params="prefix">
+    <xacro:simple_position_transmission jointName="${IndexFingerPitch1JointName}" actuatorName="${IndexFingerPitch1ActuatorName}" nodeName="${IndexFingerPitch1Node}" actuatorApi="${IndexFingerPitch1Api}"/>
   </xacro:macro>
 </robot>

File: model/robots/common/xacro/middle_finger/middle_finger.xacro (robot description, xacro)
@@ -69,9 +69,6 @@
     </xacro:revolute_joint>
   </xacro:macro>
-  <xacro:macro name="v1_right_middle_finger_actuators" params="prefix api">
-    <xacro:v1_actuator name="${RMFA_Actuator_Name}" api="${api}" />
-  </xacro:macro>
-  <xacro:macro name="v1_left_middle_finger_actuators" params="prefix api">
-    <xacro:v1_actuator name="${LMFA_Actuator_Name}" api="${api}" />
+  <xacro:macro name="middle_finger_transmissions" params="prefix">
+    <xacro:simple_position_transmission jointName="${MiddleFingerPitch1JointName}" actuatorName="${MiddleFingerPitch1ActuatorName}" nodeName="${MiddleFingerPitch1Node}" actuatorApi="${MiddleFingerPitch1Api}"/>
   </xacro:macro>
 </robot>

File: model/robots/common/xacro/pinky_finger/pinky_finger.xacro (robot description, xacro)
@@ -7,5 +7,5 @@
   <xacro:include filename="$(find val_description)/model/robots/common/xacro/pinky_finger/frame_parameters.xacro"/>
   <xacro:include filename="$(find val_description)/model/robots/common/xacro/pinky_finger/mass_parameters.xacro"/>
-  <xacro:macro name="make_pinky_finger" params="prefix reflect pinky_finger_root_link">
+  <xacro:macro name="make_pinky" params="prefix reflect pinky_finger_root_link">
     <xacro:standard_link name="${PinkyPitch1LinkName}"
                     mass="${PinkyPitch1LinkMass}"
@@ -69,9 +69,6 @@
     </xacro:revolute_joint>
   </xacro:macro>
-  <xacro:macro name="v1_right_pinky_finger_actuators" params="prefix api">
-    <xacro:v1_actuator name="${RLFA_Actuator_Name}" api="${api}" />
-  </xacro:macro>
-  <xacro:macro name="v1_left_pinky_finger_actuators" params="prefix api">
-    <xacro:v1_actuator name="${LLFA_Actuator_Name}" api="${api}" />
+  <xacro:macro name="pinky_transmissions" params="prefix">
+    <xacro:simple_position_transmission jointName="${PinkyPitch1JointName}" actuatorName="${PinkyPitch1ActuatorName}" nodeName="${PinkyPitch1Node}" actuatorApi="${PinkyPitch1Api}"/>
   </xacro:macro>
 </robot>

File: model/robots/common/xacro/thumb/thumb.xacro (robot description, xacro)
@@ -84,3 +84,8 @@
     </xacro:revolute_joint>
   </xacro:macro>
+  <xacro:macro name="thumb_transmissions" params="prefix">
+    <xacro:simple_position_transmission jointName="${ThumbRollJointName}" actuatorName="${ThumbRollActuatorName}" nodeName="${ThumbRollNode}" actuatorApi="${ThumbRollApi}"/>
+    <xacro:simple_position_transmission jointName="${ThumbPitch1JointName}" actuatorName="${ThumbPitch1ActuatorName}" nodeName="${ThumbPitch1Node}" actuatorApi="${ThumbPitch1Api}"/>
+    <xacro:simple_position_transmission jointName="${ThumbPitch2JointName}" actuatorName="${ThumbPitch2ActuatorName}" nodeName="${ThumbPitch2Node}" actuatorApi="${ThumbPitch2Api}"/>
+  </xacro:macro>
 </robot>

Commit message: added api tag for vectornav imu

File: common/xacro/api/valkyrie_api.xacro (robot description, xacro)
@@ -20,5 +20,6 @@
 	<xacro:property name="WaistRightActuatorApi" value="robot_hardware_interface/TurbodriverAPI_linear" />
 	<xacro:property name="AtiSensorApi" value="TurbodriverForceTorqueSensor" />
-	<xacro:property name="ImuSensorHardwareApi" value="val_imu_3dm_gx4_15_interface/Imu3dmGx415Interface" />
+	<xacro:property name="ImuMicrostrainHardwareApi" value="val_imu_3dm_gx4_15_interface/Imu3dmGx415Interface" />
+	<xacro:property name="ImuVectorNavHardwareApi" value="val_imu_vectornav_vn100_interface/ImuVecotNavInterface" />
 	<xacro:property name="ImuSensorSimApi" value="val_imu_gazebo_interface/ImuGazeboInterface" />
 	<xacro:property name="SimApi" value="robot_hardware_interface/TurbodriverSimAPI" />

File: model/robots/common/xacro/valkyrie_base_hw.xacro (robot description, xacro)
@@ -15,9 +15,9 @@
     <xacro:make_leg prefix="right" reflect="-1" leg_root_link="${Pelvis_Link_Name}"/>
     <xacro:make_leg prefix="left" reflect="1" leg_root_link="${Pelvis_Link_Name}"/>
-     <xacro:v1_trunk_sensors_usb sensor_node_tag="${torso_left_imu_node}" sensor_api_tag="${ImuSensorHardwareApi}" sensor_port_tag="${torso_left_imu_port}"/>
+    <xacro:v1_trunk_sensors_usb sensor_node_tag="${torso_left_imu_node}" sensor_api_tag="${ImuMicrostrainHardwareApi}" sensor_port_tag="${torso_left_imu_port}"/>
     <xacro:v1_leg_sensors prefix="left" reflect="1" ATI_serial_number="${left_foot_ATI_serial}" ATI_node="${left_foot_ATI_node}"/>
     <xacro:v1_leg_sensors prefix="right" reflect="-1" ATI_serial_number="${right_foot_ATI_serial}" ATI_node="${right_foot_ATI_node}"/>
     <xacro:include_multisense_hw />
-    <xacro:v1_pelvis_sensors_usb sensor_node_tag="${pelvis_middle_imu_node}" sensor_api_tag="${ImuSensorHardwareApi}" sensor_port_tag="${pelvis_middle_imu_port}"/>
+    <xacro:v1_pelvis_sensors_usb sensor_node_tag="${pelvis_middle_imu_node}" sensor_api_tag="${ImuMicrostrainHardwareApi}" sensor_port_tag="${pelvis_middle_imu_port}"/>
     <xacro:waist_transmissions_hw />
     <xacro:leg_transmissions_hw prefix="left"/>

File: model/robots/common/xacro/valkyrie_no_hands_base_hw.xacro (robot description, xacro)
@@ -7,9 +7,9 @@
     <xacro:make_leg prefix="right" reflect="-1" leg_root_link="${Pelvis_Link_Name}"/>
     <xacro:make_leg prefix="left" reflect="1" leg_root_link="${Pelvis_Link_Name}"/>
-    <xacro:v1_trunk_sensors />
+    <xacro:v1_trunk_sensors_usb sensor_node_tag="${torso_left_imu_node}" sensor_api_tag="${ImuMicrostrainHardwareApi}" sensor_port_tag="${torso_left_imu_port}"/>
     <xacro:v1_leg_sensors prefix="left" reflect="1" ATI_serial_number="${left_foot_ATI_serial}" ATI_node="${left_foot_ATI_node}"/>
     <xacro:v1_leg_sensors prefix="right" reflect="-1" ATI_serial_number="${right_foot_ATI_serial}" ATI_node="${right_foot_ATI_node}"/>
     <xacro:include_multisense_hw />
-    <xacro:v1_pelvis_rear_sensors_usb sensor_node_tag="${pelvis_rear_imu_node}" sensor_api_tag="${ImuSensorHardwareApi}" sensor_port_tag="${pelvis_rear_imu_port}"/>
+    <xacro:v1_pelvis_rear_sensors_usb sensor_node_tag="${pelvis_rear_imu_node}" sensor_api_tag="${ImuVectorNavHardwareApi}" sensor_port_tag="${pelvis_rear_imu_port}"/>
     <xacro:waist_transmissions_hw />
     <xacro:leg_transmissions_hw prefix="left"/>

Commit message: updated athena macros to include api and node tags

File: common/xacro/api/valkyrie_api.xacro (robot description, xacro)
@@ -29,3 +29,5 @@
 	<xacro:property name="PinkyApi" value="robot_hardware_interface/PinkyFingerApi"/>
 	<xacro:property name="SimApi" value="robot_hardware_interface/TurbodriverSimAPI" />
+	<xacro:property name="Athena1Api" value="robot_hardware_interface/AthenaForearmAPI" />
+	<xacro:property name="Athena2Api" value="robot_hardware_interface/AthenaFingerAPI" />
 </robot>

File: model/robots/common/xacro/arm/arm.xacro (robot description, xacro)
@@ -166,6 +166,6 @@
     <xacro:simple_transmission jointName="${ElbowPitchJointName}" actuatorName="${ElbowPitchActuatorName}" nodeName="${ElbowPitchNode}" actuatorApi="${ElbowPitchApi}"/>
     <xacro:simple_transmission jointName="${ForearmYawActuatorName}" actuatorName="${ForearmYawActuatorName}" nodeName="${ForearmYawNode}" actuatorApi="${ForearmYawApi}"/>
-    <xacro:athena1_transmission prefix="${prefix}" transmissionName="${prefix}ArmAthena1Transmission"/>
-    <xacro:athena2_transmission prefix="${prefix}" transmissionName="${prefix}ArmAthena2Transmission"/>
+    <xacro:athena1_transmission prefix="${prefix}" transmissionName="${prefix}ArmAthena1Transmission" actuatorApi="${Athena1Api}" nodeName="${Athena1Node}"/>
+    <xacro:athena2_transmission prefix="${prefix}" transmissionName="${prefix}ArmAthena2Transmission" actuatorApi="${Athena2Api}" nodeName="${Athena2Node}"/>
   </xacro:macro>
   <xacro:macro name="arm_transmissions_no_hands" params="prefix">

File: model/robots/common/xacro/generic_models.xacro (robot description, xacro)
@@ -275,5 +275,5 @@
     </transmission>
   </xacro:macro>
-  <xacro:macro name="athena1_transmission" params="prefix transmissionName">
+  <xacro:macro name="athena1_transmission" params="prefix transmissionName actuatorApi nodeName">
     <transmission name="${transmissionName}">
       <type>robot_transmission_interface/AthenaForearmTransmission</type>
@@ -292,10 +292,12 @@
       <actuator name="${prefix}Athena1Actuator">
         <role>athena1Actuator</role>
-        <mechanicalReduction>1</mechanicalReduction>
-        <hardwareInterface>PositionJointInterface</hardwareInterface>
-      </actuator>
-    </transmission>
-  </xacro:macro>
-  <xacro:macro name="athena2_transmission" params="prefix transmissionName">
+        <node name="${nodeName}"/>
+        <mechanicalReduction>1</mechanicalReduction>
+        <hardwareInterface>PositionJointInterface</hardwareInterface>
+        <api name="${actuatorApi}"/>
+      </actuator>
+    </transmission>
+  </xacro:macro>
+  <xacro:macro name="athena2_transmission" params="prefix transmissionName actuatorApi nodeName">
     <transmission name="${transmissionName}">
       <type>robot_transmission_interface/AthenaFingerTransmission</type>
@@ -314,6 +316,8 @@
       <actuator name="${prefix}Athena2Actuator">
         <role>athena2Actuator</role>
-        <mechanicalReduction>1</mechanicalReduction>
-        <hardwareInterface>PositionJointInterface</hardwareInterface>
+        <node name="${nodeName}"/>
+        <mechanicalReduction>1</mechanicalReduction>
+        <hardwareInterface>PositionJointInterface</hardwareInterface>
+        <api name="${actuatorApi}"/>
       </actuator>
     </transmission>

File: model/robots/forearm.xacro (robot description, xacro)
@@ -11,5 +11,5 @@
     </joint>
     <xacro:make_lower_arm prefix="${prefix}" reflect="${reflect}" lower_arm_root_link="world"/>
-    <xacro:athena1_transmission prefix="${prefix}" transmissionName="${prefix}ArmAthena1Transmission"/>
-    <xacro:athena2_transmission prefix="${prefix}" transmissionName="${prefix}ArmAthena2Transmission"/>
+    <xacro:athena1_transmission prefix="${prefix}" transmissionName="${prefix}ArmAthena1Transmission" actuatorApi="${Athena1Api}" nodeName="${Athena1Node}"/>
+    <xacro:athena2_transmission prefix="${prefix}" transmissionName="${prefix}ArmAthena2Transmission" actuatorApi="${Athena2Api}" nodeName="${Athena2Node}"/>
 </robot>
