Commit message: updated instance and description to match new athena code'

File: common/xacro/api/valkyrie_api.xacro (robot description, xacro)
@@ -29,5 +29,5 @@
 	<xacro:property name="PinkyApi" value="robot_hardware_interface/PinkyFingerApi"/>
 	<xacro:property name="SimApi" value="robot_hardware_interface/TurbodriverSimAPI" />
-	<xacro:property name="Athena1Api" value="robot_hardware_interface/AthenaForearmAPI" />
-	<xacro:property name="Athena2Api" value="robot_hardware_interface/AthenaFingerAPI" />
+	<xacro:property name="Athena1Api" value="athena_forearm_interface/AthenaForearmAPI" />
+	<xacro:property name="Athena2Api" value="athena_finger_interface/AthenaFingerAPI" />
 </robot>

File: common/xacro/nodes/forearm_testbench_nodes.xacro (robot description, xacro)
@@ -1,4 +1,4 @@
 <robot xmlns:xacro="http://ros.org/wiki/xacro" name="test_bench_nodes">
-	<xacro:property name="Athena1Node" value="/forearm/forearm_driver1" />
-	<xacro:property name="Athena2Node" value="/forearm/forearm_driver2" />
+	<xacro:property name="Athena1Node" value="/left_arm/athena1" />
+	<xacro:property name="Athena2Node" value="/left_arm/athena2" />
 </robot>

Commit message: added finger transmissions for midas output

File: common/xacro/api/valkyrie_api.xacro (robot description, xacro)
@@ -22,10 +22,8 @@
 	<xacro:property name="ImuSensorHardwareApi" value="val_imu_3dm_gx4_15_interface/Imu3dmGx415Interface" />
 	<xacro:property name="ImuSensorSimApi" value="val_imu_gazebo_interface/ImuGazeboInterface" />
-	<xacro:property name="ThumbRollApi" value="robot_hardware_interface/ThumbRollApi"/>
-	<xacro:property name="ThumbPitch1Api" value="robot_hardware_interface/ThumbPitch1Api"/>
-	<xacro:property name="ThumbPitch2Api" value="robot_hardware_interface/ThumbPitch2Api"/>
-	<xacro:property name="IndexFingerApi" value="robot_hardware_interface/IndexFingerApi"/>
-	<xacro:property name="MiddleFingerApi" value="robot_hardware_interface/MiddleFingerApi"/>
-	<xacro:property name="PinkyApi" value="robot_hardware_interface/PinkyFingerApi"/>
+	<xacro:property name="ThumbFingerApi" value="midas_finger_interface/MidasFingerAPI" />
+	<xacro:property name="IndexFingerApi" value="midas_finger_interface/MidasFingerAPI"/>
+	<xacro:property name="MiddleFingerApi" value="midas_finger_interface/MidasFingerAPI"/>
+	<xacro:property name="PinkyApi" value="midas_finger_interface/MidasFingerAPI"/>
 	<xacro:property name="SimApi" value="robot_hardware_interface/TurbodriverSimAPI" />
 	<xacro:property name="Athena1Api" value="athena_forearm_interface/AthenaForearmAPI" />

File: common/xacro/nodes/valkyrie_nodes.xacro (robot description, xacro)
@@ -34,4 +34,17 @@
 	<xacro:property name="right_foot_ATI_node" value="/right_leg/ankle/left_actuator" />
 	<xacro:property name="right_foot_Sim_ATI_node" value="/sensors/rightFootSixAxis" />
+	<xacro:property name="IndexFingerPitch1Node" value="/${prefix}_arm/forearm_sensors/index/pitch_1"/>
+	<xacro:property name="IndexFingerPitch2Node" value="/${prefix}_arm/forearm_sensors/index/pitch_2"/>
+	<xacro:property name="IndexFingerPitch3Node" value="/${prefix}_arm/forearm_sensors/index/pitch_3"/>
+	<xacro:property name="MiddleFingerPitch1Node" value="/${prefix}_arm/forearm_sensors/middle/pitch_1"/>
+	<xacro:property name="MiddleFingerPitch2Node" value="/${prefix}_arm/forearm_sensors/middle/pitch_2"/>
+	<xacro:property name="MiddleFingerPitch3Node" value="/${prefix}_arm/forearm_sensors/middle/pitch_3"/>
+	<xacro:property name="PinkyPitch1Node" value="/${prefix}_arm/forearm_sensors/pinky/pitch_1"/>
+	<xacro:property name="PinkyPitch2Node" value="/${prefix}_arm/forearm_sensors/pinky/pitch_2"/>
+	<xacro:property name="PinkyPitch3Node" value="/${prefix}_arm/forearm_sensors/pinky/pitch_3"/>
+	<xacro:property name="ThumbRollNode" value="/${prefix}_arm/forearm_sensors/thumb/roll"/>
+	<xacro:property name="ThumbPitch1Node" value="/${prefix}_arm/forearm_sensors/thumb/pitch_1"/>
+	<xacro:property name="ThumbPitch2Node" value="/${prefix}_arm/forearm_sensors/thumb/pitch_2"/>
+	<xacro:property name="ThumbPitch3Node" value="/${prefix}_arm/forearm_sensors/thumb/pitch_3"/>
 	<xacro:macro name="all_channels" >
 		<Channels>

File: model/robots/common/xacro/generic_models.xacro (robot description, xacro)
@@ -286,9 +286,9 @@
         <hardwareInterface>PositionJointInterface</hardwareInterface>
       </joint>
-      <joint name="${prefix}ThumbRoll">
+      <joint name="${prefix}ThumbMotorRoll">
         <role>thumbRoll</role>
         <hardwareInterface>PositionJointInterface</hardwareInterface>
       </joint>
-      <joint name="${prefix}ThumbPitch1">
+      <joint name="${prefix}ThumbMotorPitch1">
         <role>thumbPitch1</role>
         <hardwareInterface>PositionJointInterface</hardwareInterface>
@@ -306,17 +306,17 @@
     <transmission name="${transmissionName}">
       <type>robot_transmission_interface/AthenaFingerTransmission</type>
-      <joint name="${prefix}ThumbPitch2">
+      <joint name="${prefix}ThumbMotorPitch2">
         <role>thumbPitch2</role>
         <hardwareInterface>PositionJointInterface</hardwareInterface>
       </joint>
-      <joint name="${prefix}IndexFingerPitch1">
+      <joint name="${prefix}IndexFingerMotorPitch1">
         <role>indexFingerPitch1</role>
         <hardwareInterface>PositionJointInterface</hardwareInterface>
       </joint>
-      <joint name="${prefix}MiddleFingerPitch1">
+      <joint name="${prefix}MiddleFingerMotorPitch1">
         <role>middleFingerPitch1</role>
         <hardwareInterface>PositionJointInterface</hardwareInterface>
       </joint>
-      <joint name="${prefix}PinkyPitch1">
+      <joint name="${prefix}PinkyMotorPitch1">
         <role>pinkyPitch1</role>
         <hardwareInterface>PositionJointInterface</hardwareInterface>

File: model/robots/common/xacro/index_finger/index_finger.xacro (robot description, xacro)
@@ -69,3 +69,8 @@
     </xacro:revolute_joint>
   </xacro:macro>
+  <xacro:macro name="index_finger_transmissions_hw" params="prefix">
+    <xacro:simple_position_transmission jointName="${IndexFingerPitch1JointName}" actuatorName="${prefix}IndexPitch1Actuator" nodeName="${IndexFingerPitch1Node}" actuatorApi="${IndexFingerApi}"/>
+    <xacro:simple_position_transmission jointName="${IndexFingerPitch2JointName}" actuatorName="${prefix}IndexPitch2Actuator" nodeName="${IndexFingerPitch2Node}" actuatorApi="${IndexFingerApi}"/>
+    <xacro:simple_position_transmission jointName="${IndexFingerPitch3JointName}" actuatorName="${prefix}IndexPitch3Actuator" nodeName="${IndexFingerPitch3Node}" actuatorApi="${IndexFingerApi}"/>
+  </xacro:macro>
 </robot>

File: model/robots/common/xacro/middle_finger/middle_finger.xacro (robot description, xacro)
@@ -69,3 +69,8 @@
     </xacro:revolute_joint>
   </xacro:macro>
+  <xacro:macro name="middle_finger_transmissions_hw" params="prefix">
+    <xacro:simple_position_transmission jointName="${MiddleFingerPitch1JointName}" actuatorName="${prefix}MiddlePitch1Actuator" nodeName="${MiddleFingerPitch1Node}" actuatorApi="${MiddleFingerApi}"/>
+    <xacro:simple_position_transmission jointName="${MiddleFingerPitch2JointName}" actuatorName="${prefix}MiddlePitch2Actuator" nodeName="${MiddleFingerPitch2Node}" actuatorApi="${MiddleFingerApi}"/>
+    <xacro:simple_position_transmission jointName="${MiddleFingerPitch3JointName}" actuatorName="${prefix}MiddlePitch3Actuator" nodeName="${MiddleFingerPitch3Node}" actuatorApi="${MiddleFingerApi}"/>
+  </xacro:macro>
 </robot>

File: model/robots/common/xacro/pinky_finger/pinky_finger.xacro (robot description, xacro)
@@ -69,3 +69,8 @@
     </xacro:revolute_joint>
   </xacro:macro>
+  <xacro:macro name="pinky_finger_transmissions_hw" params="prefix">
+    <xacro:simple_position_transmission jointName="${PinkyPitch1JointName}" actuatorName="${prefix}PinkyPitch1Actuator" nodeName="${PinkyPitch1Node}" actuatorApi="${PinkyApi}"/>
+    <xacro:simple_position_transmission jointName="${PinkyPitch2JointName}" actuatorName="${prefix}PinkyPitch2Actuator" nodeName="${PinkyPitch2Node}" actuatorApi="${PinkyApi}"/>
+    <xacro:simple_position_transmission jointName="${PinkyPitch3JointName}" actuatorName="${prefix}PinkyPitch3Actuator" nodeName="${PinkyPitch3Node}" actuatorApi="${PinkyApi}"/>
+  </xacro:macro>
 </robot>

File: model/robots/common/xacro/thumb/thumb.xacro (robot description, xacro)
@@ -84,3 +84,9 @@
     </xacro:revolute_joint>
   </xacro:macro>
+  <xacro:macro name="thumb_transmissions_hw" params="prefix">
+    <xacro:simple_position_transmission jointName="${ThumbRollJointName}" actuatorName="${prefix}ThumbRollActuator" nodeName="${ThumbRollNode}" actuatorApi="${ThumbFingerApi}"/>
+    <xacro:simple_position_transmission jointName="${ThumbPitch1JointName}" actuatorName="${prefix}ThumbPitch1Actuator" nodeName="${ThumbPitch1Node}" actuatorApi="${ThumbFingerApi}"/>
+    <xacro:simple_position_transmission jointName="${ThumbPitch2JointName}" actuatorName="${prefix}ThumbPitch2Actuator" nodeName="${ThumbPitch2Node}" actuatorApi="${ThumbFingerApi}"/>
+    <xacro:simple_position_transmission jointName="${ThumbPitch3JointName}" actuatorName="${prefix}ThumbPitch3Actuator" nodeName="${ThumbPitch3Node}" actuatorApi="${ThumbFingerApi}"/>
+  </xacro:macro>
 </robot>

File: model/robots/forearm.xacro (robot description, xacro)
@@ -11,4 +11,8 @@
     </joint>
     <xacro:make_lower_arm prefix="${prefix}" reflect="${reflect}" lower_arm_root_link="world"/>
+    <xacro:index_finger_transmissions_hw prefix="${prefix}" />
+    <xacro:middle_finger_transmissions_hw prefix="${prefix}" />
+    <xacro:pinky_finger_transmissions_hw prefix="${prefix}" />
+    <xacro:thumb_transmissions_hw prefix="${prefix}" />
     <xacro:athena1_transmission prefix="${prefix}" transmissionName="${prefix}ArmAthena1Transmission" actuatorApi="${Athena1Api}" nodeName="${Athena1Node}"/>
     <xacro:athena2_transmission prefix="${prefix}" transmissionName="${prefix}ArmAthena2Transmission" actuatorApi="${Athena2Api}" nodeName="${Athena2Node}"/>

Commit message: added urdf for testing kvh imu

File: common/xacro/api/valkyrie_api.xacro (robot description, xacro)
@@ -22,4 +22,5 @@
 	<xacro:property name="ImuMicrostrainHardwareApi" value="val_imu_3dm_gx4_15_interface/Imu3dmGx415Interface" />
 	<xacro:property name="ImuVectorNavHardwareApi" value="val_imu_vectornav_vn100_interface/ImuVecotNavInterface" />
+	<xacro:property name="KVHHardwareApi" value="val_imu_kvh_1750_interface/ImuKVHInterface" />
 	<xacro:property name="ImuSensorSimApi" value="val_imu_gazebo_interface/ImuGazeboInterface" />
 	<xacro:property name="ThumbFingerApi" value="midas_finger_interface/MidasFingerAPI" />

File: model/robots/common/xacro/valkyrie_no_hands_base_hw.xacro (robot description, xacro)
@@ -11,5 +11,5 @@
     <xacro:v1_leg_sensors prefix="right" reflect="-1" ATI_serial_number="${right_foot_ATI_serial}" ATI_node="${right_foot_ATI_node}"/>
     <xacro:include_multisense_hw />
-    <xacro:v1_pelvis_rear_sensors_usb sensor_node_tag="${pelvis_rear_imu_node}" sensor_api_tag="${ImuMicrostrainHardwareApi}"  sensor_port_tag="${pelvis_rear_imu_port}"/>
+    <xacro:v1_pelvis_rear_sensors_usb sensor_node_tag="${pelvis_rear_imu_node}" sensor_api_tag="${KVHHardwareApi}"  sensor_port_tag="${pelvis_rear_imu_port}"/>
     <xacro:waist_transmissions_hw />
     <xacro:leg_transmissions_hw prefix="left"/>

Commit message: added renishaw api to api files

File: common/xacro/api/valkyrie_api.xacro (robot description, xacro)
@@ -17,6 +17,6 @@
 	<xacro:property name="UpperNeckPitchApi" value="robot_hardware_interface/TurbodriverAPI" />
 	<xacro:property name="TrunkYawApi" value="robot_hardware_interface/TurbodriverAPI" />
-	<xacro:property name="WaistLeftActuatorApi" value="robot_hardware_interface/TurbodriverAPI_linear" />
-	<xacro:property name="WaistRightActuatorApi" value="robot_hardware_interface/TurbodriverAPI_linear" />
+	<xacro:property name="WaistLeftActuatorApi" value="robot_hardware_interface/TurbodriverAPI_linear_Renishaw" />
+	<xacro:property name="WaistRightActuatorApi" value="robot_hardware_interface/TurbodriverAPI_linear_Renishaw" />
 	<xacro:property name="AtiSensorApi" value="TurbodriverForceTorqueSensor" />
 	<xacro:property name="ImuMicrostrainHardwareApi" value="val_imu_3dm_gx4_15_interface/Imu3dmGx415Interface" />

Commit message: updated api for futeks

File: common/xacro/api/valkyrie_api.xacro (robot description, xacro)
@@ -4,6 +4,6 @@
 	<xacro:property name="HipPitchApi" value="robot_hardware_interface/TurbodriverAPI" />
 	<xacro:property name="KneePitchApi" value="robot_hardware_interface/TurbodriverAPI" />
-	<xacro:property name="AnkleRightActuatorApi" value="robot_hardware_interface/TurbodriverAPI_linear" />
-	<xacro:property name="AnkleLeftActuatorApi" value="robot_hardware_interface/TurbodriverAPI_linear" />
+	<xacro:property name="AnkleRightActuatorApi" value="robot_hardware_interface/TurbodriverAPI_linear_futek" />
+	<xacro:property name="AnkleLeftActuatorApi" value="robot_hardware_interface/TurbodriverAPI_linear_futek" />
 	<xacro:property name="ShoulderPitchApi" value="robot_hardware_interface/TurbodriverAPI" />
 	<xacro:property name="ShoulderRollApi" value="robot_hardware_interface/TurbodriverAPI" />
@@ -11,6 +11,6 @@
 	<xacro:property name="ElbowPitchApi" value="robot_hardware_interface/TurbodriverAPI" />
 	<xacro:property name="ForearmYawApi" value="robot_hardware_interface/TurbodriverAPI" />
-	<xacro:property name="WristTopActuatorApi" value="robot_hardware_interface/TurbodriverAPI_linear" />
-	<xacro:property name="WristBottomActuatorApi" value="robot_hardware_interface/TurbodriverAPI_linear" />
+	<xacro:property name="WristTopActuatorApi" value="robot_hardware_interface/TurbodriverAPI_linear_futek" />
+	<xacro:property name="WristBottomActuatorApi" value="robot_hardware_interface/TurbodriverAPI_linear_futek" />
 	<xacro:property name="LowerNeckPitchApi" value="robot_hardware_interface/TurbodriverAPI" />
 	<xacro:property name="NeckYawApi" value="robot_hardware_interface/TurbodriverAPI" />
