Commit message: Switched unit C to use renishaw sensors on all linears.

File: common/xacro/api/valkyrie_C_api.xacro (robot description, xacro)
@@ -4,6 +4,6 @@
     <xacro:property name="HipPitchApi" value="robot_hardware_interface/TurbodriverAPI" />
     <xacro:property name="KneePitchApi" value="robot_hardware_interface/TurbodriverAPI" />
-    <xacro:property name="AnkleRightActuatorApi" value="robot_hardware_interface/TurbodriverAPI_linear_futek" />
-    <xacro:property name="AnkleLeftActuatorApi" value="robot_hardware_interface/TurbodriverAPI_linear_futek" />
+    <xacro:property name="AnkleRightActuatorApi" value="robot_hardware_interface/TurbodriverAPI_linear_Renishaw" />
+    <xacro:property name="AnkleLeftActuatorApi" value="robot_hardware_interface/TurbodriverAPI_linear_Renishaw" />
     <xacro:property name="ShoulderPitchApi" value="robot_hardware_interface/TurbodriverAPI" />
     <xacro:property name="ShoulderRollApi" value="robot_hardware_interface/TurbodriverAPI" />
@@ -11,6 +11,6 @@
     <xacro:property name="ElbowPitchApi" value="robot_hardware_interface/TurbodriverAPI" />
     <xacro:property name="ForearmYawApi" value="robot_hardware_interface/TurbodriverAPI" />
-    <xacro:property name="WristTopActuatorApi" value="robot_hardware_interface/TurbodriverAPI_linear_futek" />
-    <xacro:property name="WristBottomActuatorApi" value="robot_hardware_interface/TurbodriverAPI_linear_futek" />
+    <xacro:property name="WristTopActuatorApi" value="robot_hardware_interface/TurbodriverAPI_linear_Renishaw" />
+    <xacro:property name="WristBottomActuatorApi" value="robot_hardware_interface/TurbodriverAPI_linear_Renishaw" />
     <xacro:property name="LowerNeckPitchApi" value="robot_hardware_interface/TurbodriverAPI" />
     <xacro:property name="NeckYawApi" value="robot_hardware_interface/TurbodriverAPI" />
